Commit message: correct most of the files to complete the hovering, aerial transform, vel control from joy

File: aerial_robot_model/robots/dragon2.urdf.xacro (robot description, xacro)
@@ -5,5 +5,5 @@
   <xacro:include filename="$(find aerial_robot_model)/urdf/dragon2/dragon2_link.urdf.xacro" />
   <xacro:include filename="$(find aerial_robot_model)/urdf/dragon2/dragon2_head.urdf.xacro" />
-  <xacro:dragon_head self="link0"/>
+  <xacro:dragon_head self="link0"  gripper="1" />
   <xacro:dragon_link parent="link0" self="link1"/>
   <xacro:dragon_link parent="link1" self="link2"/>
@@ -14,4 +14,4 @@
 <!-- two gripper mode -->
   <xacro:dragon_link parent="link5" self="link6"/>
-  <xacro:dragon_head2 parent="link6" self="link7"/>
+  <xacro:dragon_head2 parent="link6" self="link7" gripper="1"/>
 </robot>

File: aerial_robot_model/urdf/dragon2/dragon2_head.urdf.xacro (robot description, xacro)
@@ -62,6 +62,8 @@
     </link>
   </xacro:macro>
-  <xacro:macro name="dragon_head" params="self">
-    <xacro:pr2_gripper self="${self}"/>
+  <xacro:macro name="dragon_head" params="self gripper">
+    <xacro:if value="${gripper}">
+      <xacro:pr2_gripper self="${self}"/>
+    </xacro:if>
     <link name="${self}_rear_junction">
       <visual>
@@ -73,6 +75,8 @@
     </link>
   </xacro:macro>
-  <xacro:macro name="dragon_head2" params="parent self">
-    <xacro:pr2_gripper self="${self}"/>
+  <xacro:macro name="dragon_head2" params="parent self gripper">
+    <xacro:if value="${gripper}">
+      <xacro:pr2_gripper self="${self}"/>
+    </xacro:if>
     <joint name="${parent}_${self}_joint" type="fixed">
       <parent link="${parent}_rear_junction"/>
