Commit message: some of the changes to be update

File: aerial_robot_model/robots/dragon.urdf.xacro (robot description, xacro)
@@ -5,10 +5,9 @@
   <xacro:include filename="$(find aerial_robot_model)/urdf/dragon/dragon_link.urdf.xacro" />
   <xacro:include filename="$(find aerial_robot_model)/urdf/dragon/dragon_head.urdf.xacro" />
-  <xacro:dragon_head />
+  <xacro:dragon_head self="link0"  gripper="0" />
   <xacro:dragon_link parent="link0" self="link1"/>
   <xacro:dragon_link parent="link1" self="link2"/>
   <xacro:dragon_link parent="link2" self="link3"/>
   <xacro:dragon_link parent="link3" self="link4"/>
-  <xacro:dragon_link parent="link4" self="link5"/>
-  <xacro:dragon_end_link parent="link5" self="link6"/>
+  <xacro:dragon_head2 parent="link4" self="link5" gripper="0"/>
 </robot>

File: aerial_robot_model/robots/dragon2.urdf.xacro (robot description, xacro)
@@ -11,7 +11,9 @@
   <xacro:dragon_link parent="link3" self="link4"/>
   <xacro:dragon_link parent="link4" self="link5"/>
+  <xacro:dragon_link parent="link5" self="link6"/>
+  <xacro:dragon_link parent="link6" self="link7"/>
+  <xacro:dragon_link parent="link7" self="link8"/>
 <!--    <xacro:dragon_end_link parent="link5" self="link6"/>  -->
 <!-- two gripper mode -->
-  <xacro:dragon_link parent="link5" self="link6"/>
-  <xacro:dragon_head2 parent="link6" self="link7" gripper="1"/>
+  <xacro:dragon_head2 parent="link8" self="link9" gripper="1"/>
 </robot>

File: aerial_robot_model/robots/other_objects/street_lamp.urdf.xacro (robot description, xacro)
@@ -1,9 +1,9 @@
 <?xml version="1.0"?>
 <robot name="streetlamp">
-    <link name="street_lamp">
+    <link name="base_link">
       <visual>
         <origin rpy="0 0 0" xyz="0 0 0"/>
         <geometry>
-          <mesh filename="package://aerial_robot_model/urdf/other_objects/StreetLamp.dae" scale="1 1 1"/>
+          <mesh filename="package://aerial_robot_model/urdf/other_objects/street_lamp.dae" scale="0.2 0.2 0.2"/>
         </geometry>
       </visual>

File: aerial_robot_model/urdf/dragon/dragon_head.urdf.xacro (robot description, xacro)
@@ -2,133 +2,78 @@
 <robot
     xmlns:xacro="http://www.ros.org/wiki/xacro" name="dragon_head" >
-<!--
-  <xacro:macro name="dragon_head">
-    <link name="left_eye">
+  <xacro:macro name="pr2_gripper" params="self">
+    <joint name="${self}_left_gripper_joint" type="revolute">
+      <axis xyz="0 0 1"/>
+      <limit effort="1000.0" lower="0.0" upper="0.548" velocity="0.5"/>
+      <origin rpy="0 0 0" xyz="0.015 0.01 0"/>
+      <parent link="${self}_head_base"/>
+      <child link="${self}_left_gripper"/>
+    </joint>
+    <link name="${self}_left_gripper">
       <visual>
+        <origin rpy="0.0 0 0" xyz="0 0 0"/>
         <geometry>
-          <sphere radius="${tail_width*.2}"/>
-        </geometry>
-        <material name="Red">
-          <color rgba=".7 .0 .0 1"/>
-        </material>
-      </visual>
-    </link>
-    <joint name="left_eye_head_cylinder_joint" type="fixed">
-      <parent link="head_cylinder"/>
-      <child link="left_eye"/>
-      <origin rpy="0 0 0" xyz="${tail_len*.2} ${tail_width*.5*.707} ${tail_width*.5*.707}"/>
-    </joint>
-    <link name="right_eye">
-      <visual>
-        <geometry>
-          <sphere radius="${tail_width*.2}"/>
-        </geometry>
-        <material name="Red">
-          <color rgba=".7 .0 .0 1"/>
-        </material>
-      </visual>
-    </link>
-    <joint name="right_eye_head_cylinder_joint" type="fixed">
-      <parent link="head_cylinder"/>
-      <child link="right_eye"/>
-      <origin rpy="0 0 0" xyz="${tail_len*.2} ${-tail_width*.5*.707} ${tail_width*.5*.707}"/>
-    </joint>
-    <link name="head_sphere">
-      <visual>
-        <geometry>
-          <sphere radius="${tail_width*.5}"/>
+          <mesh filename="package://aerial_robot_model/urdf/mesh_model/l_finger.dae"/>
         </geometry>
         <xacro:link_color />
       </visual>
     </link>
-    <joint name="head_sphere_head_cylinder_joint" type="fixed">
-      <parent link="head_cylinder"/>
-      <child link="head_sphere"/>
-      <origin rpy="0 0 0" xyz="${tail_len*.25} 0 0"/>
+    <joint name="${self}_left_tip_joint" type="fixed">
+      <parent link="${self}_left_gripper"/>
+      <child link="${self}_left_tip"/>
     </joint>
-    <link name="head_cylinder">
+    <link name="${self}_left_tip">
       <visual>
+        <origin rpy="0.0 0 0" xyz="0.09137 0.00495 0"/>
         <geometry>
-          <cylinder length="${tail_len*.5}" radius="${tail_width*.5}"/>
-        </geometry>
-        <origin rpy="0 1.57075 0 " xyz="0 0 0"/>
-        <xacro:link_color />
-      </visual>
-    </link>
-    <link name="link0_rear_junction">
-      <visual>
-        <geometry>
-          <box size="0.01 ${tail_width} ${abdomen_height}"/>
+          <mesh filename="package://pr2_description/meshes/gripper_v0/l_finger_tip.dae"/>
         </geometry>
         <xacro:link_color />
       </visual>
     </link>
-    <joint name="link0_rear_junction_abdomen_joint" type="fixed">
-      <parent link="head_cylinder"/>
-      <child link="link0_rear_junction"/>
-      <origin rpy="0 0 0" xyz="${-tail_len*.25-.005} 0 0"/>
+    <joint name="${self}_right_gripper_joint" type="revolute">
+      <axis xyz="0 0 -1"/>
+      <limit effort="1000.0" lower="0.0" upper="0.548" velocity="0.5"/>
+      <origin rpy="0 0 0" xyz="0.015 -0.01 0"/>
+      <parent link="${self}_head_base"/>
+      <child link="${self}_right_gripper"/>
     </joint>
-  </xacro:macro>
--->
-  <xacro:macro name="dragon_head">
-  <joint name="left_gripper_joint" type="revolute">
-    <axis xyz="0 0 1"/>
-    <limit effort="1000.0" lower="0.0" upper="0.548" velocity="0.5"/>
-    <origin rpy="0 0 0" xyz="0.015 0.01 0"/>
-    <parent link="link0_rear_junction"/>
-    <child link="left_gripper"/>
-  </joint>
- <link name="left_gripper">
-    <visual>
-      <origin rpy="0.0 0 0" xyz="0 0 0"/>
-      <geometry>
-        <mesh filename="package://aerial_robot_model/urdf/mesh_model/l_finger.dae"/>
-      </geometry>
-      <xacro:link_color />
-    </visual>
- </link>
-  <joint name="left_tip_joint" type="fixed">
-    <parent link="left_gripper"/>
-    <child link="left_tip"/>
-  </joint>
-  <link name="left_tip">
-    <visual>
-      <origin rpy="0.0 0 0" xyz="0.09137 0.00495 0"/>
-      <geometry>
-        <mesh filename="package://pr2_description/meshes/gripper_v0/l_finger_tip.dae"/>
-      </geometry>
-      <xacro:link_color />
-    </visual>
-  </link>
-  <joint name="right_gripper_joint" type="revolute">
-    <axis xyz="0 0 -1"/>
-    <limit effort="1000.0" lower="0.0" upper="0.548" velocity="0.5"/>
-    <origin rpy="0 0 0" xyz="0.015 -0.01 0"/>
-    <parent link="link0_rear_junction"/>
-    <child link="right_gripper"/>
-  </joint>
-  <link name="right_gripper">
-    <visual>
-      <origin rpy="-3.1415 0 0" xyz="0 0 0"/>
-      <geometry>
-        <mesh filename="package://aerial_robot_model/urdf/mesh_model/l_finger.dae"/>
-      </geometry>
-      <xacro:link_color />
-    </visual>
-  </link>
-  <joint name="right_tip_joint" type="fixed">
-    <parent link="right_gripper"/>
-    <child link="right_tip"/>
-  </joint>
-  <link name="right_tip">
-    <visual>
-      <origin rpy="-3.1415 0 0" xyz="0.09137 0.00495 0"/>
-      <geometry>
-        <mesh filename="package://pr2_description/meshes/gripper_v0/l_finger_tip.dae"/>
-      </geometry>
-      <xacro:link_color />
-    </visual>
-  </link>
-    <link name="link0_rear_junction">
+    <link name="${self}_right_gripper">
+      <visual>
+        <origin rpy="-3.1415 0 0" xyz="0 0 0"/>
+        <geometry>
+          <mesh filename="package://aerial_robot_model/urdf/mesh_model/l_finger.dae"/>
+        </geometry>
+        <xacro:link_color />
+      </visual>
+    </link>
+    <joint name="${self}_right_tip_joint" type="fixed">
+      <parent link="${self}_right_gripper"/>
+      <child link="${self}_right_tip"/>
+    </joint>
+    <link name="${self}_right_tip">
+      <visual>
+        <origin rpy="-3.1415 0 0" xyz="0.09137 0.00495 0"/>
+        <geometry>
+          <mesh filename="package://pr2_description/meshes/gripper_v0/l_finger_tip.dae"/>
+        </geometry>
+        <xacro:link_color />
+      </visual>
+    </link>
+    <link name="${self}_head_base">
+      <visual>
+        <geometry>
+          <box size="0.01 ${tail_width*.5} ${abdomen_height*.5}"/>
+        </geometry>
+        <xacro:link_color />
+      </visual>
+    </link>
+    <joint name="${self}_roll_joint" type="continuous">
+      <parent link="${self}_rear_junction"/>
+      <child link="${self}_head_base"/>
+      <origin rpy="0 0 0" xyz="0 0 0"/>
+      <axis xyz="1 0 0"/>
+    </joint>
+    <link name="${self}_rear_junction">
       <visual>
         <geometry>
@@ -139,3 +84,18 @@
     </link>
   </xacro:macro>
+  <xacro:macro name="dragon_head" params="self gripper">
+    <xacro:if value="${gripper}">
+      <xacro:pr2_gripper self="${self}"/>
+    </xacro:if>
+  </xacro:macro>
+  <xacro:macro name="dragon_head2" params="parent self gripper">
+    <xacro:if value="${gripper}">
+      <xacro:pr2_gripper self="${self}"/>
+    </xacro:if>
+    <joint name="${parent}_${self}_joint" type="fixed">
+      <parent link="${parent}_rear_junction"/>
+      <child link="${self}_rear_junction"/>
+      <origin rpy="-1.5708  3.1415 0" xyz="-0.01 0 0"/>
+    </joint>
+  </xacro:macro>
 </robot>

File: aerial_robot_model/urdf/dragon2/dragon2_head.urdf.xacro (robot description, xacro)
@@ -7,5 +7,5 @@
       <limit effort="1000.0" lower="0.0" upper="0.548" velocity="0.5"/>
       <origin rpy="0 0 0" xyz="0.015 0.01 0"/>
-      <parent link="${self}_rear_junction"/>
+      <parent link="${self}_head_base"/>
       <child link="${self}_left_gripper"/>
     </joint>
@@ -36,5 +36,5 @@
       <limit effort="1000.0" lower="0.0" upper="0.548" velocity="0.5"/>
       <origin rpy="0 0 0" xyz="0.015 -0.01 0"/>
-      <parent link="${self}_rear_junction"/>
+      <parent link="${self}_head_base"/>
       <child link="${self}_right_gripper"/>
     </joint>
@@ -61,4 +61,18 @@
       </visual>
     </link>
+    <link name="${self}_head_base">
+      <visual>
+        <geometry>
+          <box size="0.01 ${tail_width*.5} ${abdomen_height*.5}"/>
+        </geometry>
+        <xacro:link_color />
+      </visual>
+    </link>
+    <joint name="${self}_roll_joint" type="continuous">
+      <parent link="${self}_rear_junction"/>
+      <child link="${self}_head_base"/>
+      <origin rpy="0 0 0" xyz="0 0 0"/>
+      <axis xyz="1 0 0"/>
+    </joint>
   </xacro:macro>
   <xacro:macro name="dragon_head" params="self gripper">
@@ -79,9 +93,4 @@
       <xacro:pr2_gripper self="${self}"/>
     </xacro:if>
-    <joint name="${parent}_${self}_joint" type="fixed">
-      <parent link="${parent}_rear_junction"/>
-      <child link="${self}_rear_junction"/>
-      <origin rpy="-1.5708  3.1415 0" xyz="-0.01 0 0"/>
-    </joint>
     <link name="${self}_rear_junction">
       <visual>
@@ -92,4 +101,9 @@
       </visual>
     </link>
+    <joint name="${parent}_${self}_joint" type="fixed">
+      <parent link="${parent}_rear_junction"/>
+      <child link="${self}_rear_junction"/>
+      <origin rpy="-1.5708  3.1415 0" xyz="-0.01 0 0"/>
+    </joint>
   </xacro:macro>
 </robot>
