Commit message: some commit about gazebo multirotr

File: aerial_robot_model/robots/hydra3.urdf (robot description, URDF)
Before this commit: robot hydra3, 7 links, 6 joints
Links:
- removed link joint2
- removed link joint3
- removed link link3
- removed link link4
- link link1: mass None -> 0.5; geometry collision cylinder length=0.1 radius=0.155; visual mesh filename=package://aerial_robot_model/urdf/hydra3/mesh/hydra_link1.s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 scale=.001 .001 .001
- link link2: mass None -> 0.5; geometry collision cylinder length=0.1 radius=0.155; visual mesh filename=package://aerial_robot_model/urdf/hydra3/mesh/hydra_link4.s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 scale=.001 .001 .001
Joints:
- removed joint joint2
- removed joint joint2_link3
- removed joint joint3
- removed joint joint3_link4

File: aerial_robot_model/urdf/hydra3/hydra3_common.xacro (robot description, xacro)
@@ -4,6 +4,7 @@
   <xacro:property name="pi" value="3.1415926535897931" />
   <xacro:property name="link_length" value=".44" />
+  <xacro:property name="protector_radius" value=".155" />
   <xacro:macro name="link_color">
-    <material name="gray">
+    <material name="color">
       <color rgba="0.75 .5 .2 1"/>
     </material>

File: aerial_robot_model/urdf/hydra3/hydra3_link.urdf.xacro (robot description, xacro)
@@ -6,4 +6,10 @@
     <xacro:if value="${head}">
       <link name="link${self}">
+        <collision>
+          <origin xyz="0 0 0" rpy="0 0 0"/>
+          <geometry>
+          <cylinder length="0.1" radius="${protector_radius}"/>
+          </geometry>
+        </collision>
         <visual>
           <origin rpy="0 0 ${pi}" xyz="0 0 0"/>
@@ -13,4 +19,12 @@
           <xacro:link_color />
         </visual>
+        <inertial>
+          <origin xyz="0 0 0" rpy="0 0 0"/>
+          <mass value="0.5"/>
+          <inertia
+	      ixx="0.1" ixy="0.0" ixz="0.0"
+	      iyy="0.01" iyz="0.0"
+	      izz="0.11"/>
+        </inertial>
       </link>
       <joint name="joint${self}" type="revolute">
@@ -20,6 +34,28 @@
         <origin rpy="0 0 0" xyz="-${link_length*.5} 0 0"/>
         <axis xyz="0 0 1"/>
+        <dynamics damping="0.8"/>
       </joint>
-      <link name="joint${self}">  </link>
+      <link name="joint${self}">
+        <collision>
+          <origin rpy="0 0 0" xyz="0 0 0"/>
+          <geometry>
+            <cylinder length="0.05" radius="0.02"/>
+          </geometry>
+        </collision>
+        <visual>
+          <origin rpy="0 0 0" xyz="0 0 0"/>
+          <geometry>
+            <cylinder length="0.001" radius="0.001"/>
+          </geometry>
+          <material name="color">
+            <color rgba="0.75 .5 .2 1"/>
+          </material>
+        </visual>
+        <inertial>
+          <origin rpy="0 0 0" xyz="0 0 0"/>
+          <mass value="0.1"/>
+          <inertia ixx="0.00005" ixy="0.0" ixz="0.0" iyy="0.00005" iyz="0.0" izz="0.0001"/>
+        </inertial>
+      </link>
       <joint name="joint${self}_link${child}" type="fixed">
         <parent link="joint${self}"/>
@@ -31,4 +67,10 @@
       <xacro:if value="${tail}">
         <link name="link${self}">
+          <collision>
+            <origin xyz="0 0 0" rpy="0 0 0"/>
+            <geometry>
+              <cylinder length="${protector_radius}" radius="0.1"/>
+            </geometry>
+          </collision>
           <visual>
             <origin rpy="0 0 ${pi}" xyz="0 0 0"/>
@@ -38,4 +80,12 @@
             <xacro:link_color />
           </visual>
+          <inertial>
+            <origin xyz="0 0 0" rpy="0 0 0"/>
+            <mass value="0.5"/>
+            <inertia
+	        ixx="0.1" ixy="0.0" ixz="0.0"
+	        iyy="0.01" iyz="0.0"
+	        izz="0.11"/>
+          </inertial>
         </link>
       </xacro:if>
@@ -43,4 +93,10 @@
         <xacro:if value="${imu}">
           <link name="link${self}">
+            <collision>
+              <origin xyz="0 0 0" rpy="0 0 0"/>
+              <geometry>
+                <cylinder length="${protector_radius}" radius="0.1"/>
+              </geometry>
+            </collision>
             <visual>
               <origin rpy="0 0 ${pi}" xyz="0 0 0"/>
@@ -50,8 +106,22 @@
               <xacro:link_color />
             </visual>
+            <inertial>
+              <origin xyz="0 0 0" rpy="0 0 0"/>
+              <mass value="0.5"/>
+              <inertia
+	          ixx="0.1" ixy="0.0" ixz="0.0"
+	          iyy="0.01" iyz="0.0"
+	          izz="0.11"/>
+            </inertial>
           </link>
         </xacro:if>
         <xacro:unless value="${imu}">
           <link name="link${self}">
+            <collision>
+              <origin xyz="0 0 0" rpy="0 0 0"/>
+              <geometry>
+                <cylinder length="0.1" radius="${protector_radius}"/>
+              </geometry>
+            </collision>
             <visual>
               <origin rpy="0 0 ${pi}" xyz="0 0 0"/>
@@ -61,4 +131,12 @@
               <xacro:link_color />
             </visual>
+            <inertial>
+              <origin xyz="0 0 0" rpy="0 0 0"/>
+              <mass value="0.5"/>
+              <inertia
+	          ixx="0.1" ixy="0.0" ixz="0.0"
+	          iyy="0.01" iyz="0.0"
+	          izz="0.11"/>
+            </inertial>
           </link>
         </xacro:unless>
@@ -69,6 +147,28 @@
           <origin rpy="0 0 0" xyz="-${link_length*.5} 0 0"/>
           <axis xyz="0 0 1"/>
+          <dynamics damping="0.7"/>
         </joint>
-        <link name="joint${self}">  </link>
+        <link name="joint${self}">
+          <collision>
+            <origin rpy="0 0 0" xyz="0 0 0"/>
+            <geometry>
+              <cylinder length="0.05" radius="0.02"/>
+            </geometry>
+          </collision>
+          <visual>
+            <origin rpy="0 0 0" xyz="0 0 0"/>
+            <geometry>
+              <cylinder length="0.001" radius="0.001"/>
+            </geometry>
+            <material name="color">
+              <color rgba="0.75 .5 .2 1"/>
+            </material>
+          </visual>
+          <inertial>
+            <origin rpy="0 0 0" xyz="0 0 0"/>
+            <mass value="0.1"/>
+            <inertia ixx="0.00005" ixy="0.0" ixz="0.0" iyy="0.00005" iyz="0.0" izz="0.0001"/>
+          </inertial>
+        </link>
         <joint name="joint${self}_link${child}" type="fixed">
           <parent link="joint${self}"/>
