Commit message: 1. Update the hydrus3 model which has original color: SolidEdge Collada Export 2. Refine the urdf xacro description for hydrus3 3. Add Gazebo elements to urdf xacro file
4. merge gazebo display launch file to aerial_robot_model.lunach

File: aerial_robot_model/robots/hydrus3.urdf.xacro (robot description, xacro)
@@ -8,3 +8,10 @@
   <xacro:hydrus3_link self="3" child="4" head="false" tail="false" imu="false"/>
   <xacro:hydrus3_link self="4" child="5" head="false" tail="true" imu="false"/>
+  <!-- gazebo elements: hw interface -->
+  <gazebo>
+    <plugin name="gazebo_ros_control" filename="libgazebo_ros_control.so">
+      <robotNamespace>/hydra3</robotNamespace>
+      <robotSimType>gazebo_ros_control/DefaultRobotHWSim</robotSimType>
+    </plugin>
+  </gazebo>
 </robot>

File: aerial_robot_model/urdf/hydrus3/hydrus3_common.xacro (robot description, xacro)
@@ -5,8 +5,17 @@
   <xacro:property name="link_length" value=".44" />
   <xacro:property name="protector_radius" value=".155" />
-  <xacro:macro name="link_color">
-    <material name="color">
-      <color rgba="0.75 .5 .2 1"/>
-    </material>
+  <xacro:macro name="link_model" params="self">
+    <collision>
+      <origin xyz="0 0 0" rpy="0 0 0"/>
+      <geometry>
+        <cylinder length="${protector_radius}" radius="0.1"/>
+      </geometry>
+    </collision>
+    <visual>
+      <origin rpy="${-pi/2} 0 ${pi}" xyz="0 0 0"/>
+      <geometry>
+        <mesh filename="package://aerial_robot_model/urdf/hydrus3/mesh/hydrus3_link${self}.dae"/>
+      </geometry>
+    </visual>
   </xacro:macro>
 </robot>

File: aerial_robot_model/urdf/hydrus3/hydrus3_link.urdf.xacro (robot description, xacro)
@@ -6,24 +6,13 @@
     <xacro:if value="${head}">
       <link name="link${self}">
-        <collision>
-          <origin xyz="0 0 0" rpy="0 0 0"/>
-          <geometry>
-          <cylinder length="0.1" radius="${protector_radius}"/>
-          </geometry>
-        </collision>
-        <visual>
-          <origin rpy="0 0 ${pi}" xyz="0 0 0"/>
-          <geometry>
-            <mesh filename="package://aerial_robot_model/urdf/hydrus3/mesh/hydrus3_link1.dae"/>
-          </geometry>
-          <xacro:link_color />
-        </visual>
+        <xacro:link_model self="1" />
+        <!-- TODO: check precise inertial -->
         <inertial>
           <origin xyz="0 0 0" rpy="0 0 0"/>
           <mass value="0.5"/>
           <inertia
-	      ixx="0.1" ixy="0.0" ixz="0.0"
-	      iyy="0.01" iyz="0.0"
-	      izz="0.11"/>
+              ixx="0.1" ixy="0.0" ixz="0.0"
+              iyy="0.01" iyz="0.0"
+              izz="0.11"/>
         </inertial>
       </link>
@@ -63,82 +52,46 @@
         <origin rpy="0 0 0" xyz="-${link_length*.5} 0 0"/>
       </joint>
-    </xacro:if>
+    </xacro:if> <!-- var_head -->
     <xacro:unless value="${head}">
       <xacro:if value="${tail}">
         <link name="link${self}">
-          <collision>
-            <origin xyz="0 0 0" rpy="0 0 0"/>
-            <geometry>
-              <cylinder length="${protector_radius}" radius="0.1"/>
-            </geometry>
-          </collision>
-          <visual>
-            <origin rpy="0 0 ${pi}" xyz="0 0 0"/>
-            <geometry>
-              <mesh filename="package://aerial_robot_model/urdf/hydrus3/mesh/hydrus3_link4.dae" />
-            </geometry>
-            <xacro:link_color />
-          </visual>
+          <xacro:link_model self="4" />
           <inertial>
             <origin xyz="0 0 0" rpy="0 0 0"/>
             <mass value="0.5"/>
             <inertia
-	        ixx="0.1" ixy="0.0" ixz="0.0"
-	        iyy="0.01" iyz="0.0"
-	        izz="0.11"/>
+                ixx="0.1" ixy="0.0" ixz="0.0"
+                iyy="0.01" iyz="0.0"
+                izz="0.11"/>
           </inertial>
         </link>
-      </xacro:if>
+      </xacro:if> <!-- var_tail -->
       <xacro:unless value="${tail}">
         <xacro:if value="${imu}">
           <link name="link${self}">
-            <collision>
-              <origin xyz="0 0 0" rpy="0 0 0"/>
-              <geometry>
-                <cylinder length="${protector_radius}" radius="0.1"/>
-              </geometry>
-            </collision>
-            <visual>
-              <origin rpy="0 0 ${pi}" xyz="0 0 0"/>
-              <geometry>
-                <mesh filename="package://aerial_robot_model/urdf/hydrus3/mesh/hydrus3_link2.dae"/>
-              </geometry>
-              <xacro:link_color />
-            </visual>
+            <xacro:link_model self="2" />
             <inertial>
               <origin xyz="0 0 0" rpy="0 0 0"/>
               <mass value="0.5"/>
               <inertia
-	          ixx="0.1" ixy="0.0" ixz="0.0"
-	          iyy="0.01" iyz="0.0"
-	          izz="0.11"/>
+                  ixx="0.1" ixy="0.0" ixz="0.0"
+                  iyy="0.01" iyz="0.0"
+                  izz="0.11"/>
             </inertial>
           </link>
-        </xacro:if>
-        <xacro:unless value="${imu}">
+        </xacro:if> <!-- var_imu -->
+        <xacro:unless value="${imu}"> <!-- var_imu -->
           <link name="link${self}">
-            <collision>
-              <origin xyz="0 0 0" rpy="0 0 0"/>
-              <geometry>
-                <cylinder length="0.1" radius="${protector_radius}"/>
-              </geometry>
-            </collision>
-            <visual>
-              <origin rpy="0 0 ${pi}" xyz="0 0 0"/>
-              <geometry>
-                <mesh filename="package://aerial_robot_model/urdf/hydrus3/mesh/hydrus3_link3.dae"/>
-              </geometry>
-              <xacro:link_color />
-            </visual>
+            <xacro:link_model self="3" />
             <inertial>
               <origin xyz="0 0 0" rpy="0 0 0"/>
               <mass value="0.5"/>
               <inertia
-	          ixx="0.1" ixy="0.0" ixz="0.0"
-	          iyy="0.01" iyz="0.0"
-	          izz="0.11"/>
+                  ixx="0.1" ixy="0.0" ixz="0.0"
+                  iyy="0.01" iyz="0.0"
+                  izz="0.11"/>
             </inertial>
           </link>
-        </xacro:unless>
+        </xacro:unless> <!-- var_imu -->
         <joint name="joint${self}" type="revolute">
           <limit effort="100.0" lower="-1.57" upper="1.57" velocity="0.5"/>
@@ -176,6 +129,22 @@
           <origin rpy="0 0 0" xyz="-${link_length*.5} 0 0"/>
         </joint>
-      </xacro:unless>
-    </xacro:unless>
+      </xacro:unless> <!-- var_tail -->
+    </xacro:unless> <!-- var_head -->
+    <!-- gazebo elements -->
+    <!-- transmission interface -->
+    <xacro:unless value="${tail}">
+      <transmission name="tran${self}">
+        <type>transmission_interface/SimpleTransmission</type>
+        <joint name="joint${self}">
+          <!-- TODO: effort is torque, maybe position is enough -->
+          <hardwareInterface>EffortJointInterface</hardwareInterface>
+        </joint>
+        <actuator name="servo{self}">
+          <!-- TODO: effort is torque, maybe position is enough -->
+          <hardwareInterface>EffortJointInterface</hardwareInterface>
+          <mechanicalReduction>1</mechanicalReduction>
+        </actuator>
+      </transmission>
+    </xacro:unless> <!-- var_tail -->
   </xacro:macro>
 </robot>

Commit message: Improve the discription of transformable aerial robot's urdf: 1. Change the kinematics rule: the link origin of link n is at the joint n-1, so we also create a virtual link_center link;  the x axis of link n is towrads joint n, which is opposite to the previous one. 2. Specify the dynamics of the link: inertia parameters.

File: aerial_robot_model/robots/hydrus3.urdf.xacro (robot description, xacro)
@@ -4,7 +4,7 @@
   <xacro:include filename="$(find aerial_robot_model)/urdf/hydrus3/hydrus3_common.xacro" />
   <xacro:include filename="$(find aerial_robot_model)/urdf/hydrus3/hydrus3_link.urdf.xacro" />
-  <xacro:hydrus3_link self="1" child="2" head="true" tail="false" imu="false"/>
-  <xacro:hydrus3_link self="2" child="3" head="false" tail="false" imu="true"/>
-  <xacro:hydrus3_link self="3" child="4" head="false" tail="false" imu="false"/>
-  <xacro:hydrus3_link self="4" child="5" head="false" tail="true" imu="false"/>
+  <xacro:hydrus3_link self="1" child="2" head="true" tail="false" imu="false" m_link="0.607" i_xx="${protector_inertia * .5}" i_yy="${joint_inertia + pc_inertia + rod_inertia + protector_inertia * .5}" i_zz="${joint_inertia + pc_inertia + rod_inertia + protector_inertia}" />
+  <xacro:hydrus3_link self="2" child="3" head="false" tail="false" imu="true" m_link="0.557" i_xx="${protector_inertia * .5}" i_yy="${joint_inertia + rod_inertia + protector_inertia * .5}" i_zz="${joint_inertia + rod_inertia + protector_inertia}"/>
+  <xacro:hydrus3_link self="3" child="4" head="false" tail="false" imu="false" m_link="0.487" i_xx="${protector_inertia * .5}" i_yy="${joint_inertia + rod_inertia + protector_inertia * .5}" i_zz="${joint_inertia + rod_inertia + protector_inertia}"/>
+  <xacro:hydrus3_link self="4" child="5" head="false" tail="true" imu="false" m_link="0.45" i_xx="${protector_inertia * .5}" i_yy="${rod_inertia + protector_inertia * .5}" i_zz="${rod_inertia + protector_inertia}"/>
 </robot>

File: aerial_robot_model/urdf/hydrus3/hydrus3_common.xacro (robot description, xacro)
@@ -5,13 +5,23 @@
   <xacro:property name="link_length" value=".44" />
   <xacro:property name="protector_radius" value=".155" />
+  <xacro:property name="protector_mass" value=".05" />
+  <xacro:property name="pc_mass" value=".1" />
+  <xacro:property name="rotor_mass" value=".05" /> <!-- [g] -->
+  <xacro:property name="rotor_radius" value=".015" /> <!-- [g] -->
+  <xacro:property name="rotor_height" value=".05" /> <!-- [m] -->
+  <xacro:property name="max_force" value="100" /> <!-- [m] -->
+  <xacro:property name="joint_inertia" value="${.0785 * .205 * .205}" /> <!-- mass * dist * dist -->
+  <xacro:property name="rod_inertia" value="${link_length * link_length * 0.1 /12}" /> <!-- mass * dist * dist -->
+  <xacro:property name="pc_inertia" value="${pc_mass * .189 * .189}" /> <!-- mass * dist * dist -->
+  <xacro:property name="protector_inertia" value="${protector_mass * protector_radius * protector_radius}" /> <!-- mass * dist * dist -->
   <xacro:macro name="link_model" params="self">
     <collision>
       <origin xyz="0 0 0" rpy="0 0 0"/>
       <geometry>
-        <cylinder length="${protector_radius}" radius="0.1"/>
+        <cylinder length="${protector_radius}" radius="0.09"/>
       </geometry>
     </collision>
     <visual>
-      <origin rpy="${-pi/2} 0 ${pi}" xyz="0 0 0"/>
+      <origin rpy="${-pi/2} 0 0" xyz="${link_length*.5} 0 0"/>
       <geometry>
         <mesh filename="package://aerial_robot_model/urdf/hydrus3/mesh/hydrus3_link${self}.dae"/>
@@ -19,3 +29,15 @@
     </visual>
   </xacro:macro>
+  <!-- friction -->
+  <xacro:macro name="friction" params="self">
+    <gazebo reference="link${self}">
+      <mu1>0.0001</mu1>
+      <mu2>0.0001</mu2>
+    </gazebo>
+  </xacro:macro>
+  <xacro:macro name="damping_factor" params="link">
+    <gazebo reference="${link}">
+      <dampingFactor>0.00</dampingFactor>
+    </gazebo>
+  </xacro:macro>
 </robot>

File: aerial_robot_model/urdf/hydrus3/hydrus3_link.urdf.xacro (robot description, xacro)
@@ -2,133 +2,101 @@
 <robot
     xmlns:xacro="http://www.ros.org/wiki/xacro" name="hydrus3_link" >
-  <!-- problem: the direction of the link is opposite, because the joint!! -->
-  <xacro:macro name="hydrus3_link" params="self child head tail imu">
-    <xacro:if value="${head}">
-      <link name="link${self}">
+  <!-- D-H kai description(different from prof.nakamura) -->
+  <xacro:macro name="hydrus3_link" params="self child head tail imu m_link i_xx i_yy i_zz">
+    <!-- link -->
+    <link name="link${self}">
+      <!-- visual & collisiont -->
+      <xacro:if value="${head}">
         <xacro:link_model self="1" />
-        <!-- TODO: check precise inertial -->
-        <inertial>
-          <origin xyz="0 0 0" rpy="0 0 0"/>
-          <mass value="0.5"/>
-          <inertia
-              ixx="0.1" ixy="0.0" ixz="0.0"
-              iyy="0.01" iyz="0.0"
-              izz="0.11"/>
-        </inertial>
-      </link>
+      </xacro:if>
+      <xacro:unless value="${head}">
+        <xacro:if value="${imu}">
+          <xacro:link_model self="2" />
+        </xacro:if>
+        <xacro:unless value="${imu}">
+          <xacro:if value="${tail}">
+            <xacro:link_model self="4" />
+          </xacro:if>
+          <xacro:unless value="${tail}">
+            <xacro:link_model self="3" />
+          </xacro:unless>
+        </xacro:unless>
+      </xacro:unless>
+      <inertial>
+        <origin xyz="${link_length*.5} 0 0" rpy="0 0 0"/>
+        <mass value="${m_link}"/>
+<!--
+        <inertia
+            ixx="0.0001" ixy="0.0" ixz="0.0"
+            iyy="0.005" iyz="0.0"
+            izz="0.0051"/>
+            </inertial>
+-->
+        <inertia
+            ixx="${i_xx}" ixy="0.0" ixz="0.0"
+            iyy="${i_yy}" iyz="0.0"
+            izz="${i_zz}"/>
+            </inertial>
+    </link>
+    <xacro:damping_factor link ="link${self}"/>
+    <!-- link center(virtual) -->
+    <!-- not good -->
+    <joint name="center${self}" type="fixed">
+      <parent link="link${self}"/>
+      <child link="link${self}_center"/>
+      <origin rpy="0 0 0" xyz="${link_length*.5} 0 0"/>
+      <axis xyz="0 0 1"/>
+    </joint>
+    <link name="link${self}_center">
+      <!-- visual & collisiont -->
+      <inertial>
+        <origin xyz="0 0 0" rpy="0 0 0"/>
+        <mass value="0.001"/>
+        <inertia
+            ixx="0.00000001" ixy="0.0" ixz="0.0"
+            iyy="0.00000001" iyz="0.0"
+            izz="0.00000002"/>
+      </inertial>
+    </link>
+    <xacro:damping_factor link ="link${self}_center"/>
+    <!-- rotor -->
+    <joint name="rotor${self}" type="continuous">
+      <limit effort="100.0" lower="0" upper="${max_force}" velocity="0.5"/> <!-- force range -->
+      <parent link="link${self}"/>
+      <child link="propeller${self}"/>
+      <origin rpy="0 0 0" xyz="${link_length*.5} 0 0"/>
+      <axis xyz="0 0 1"/>
+    </joint>
+    <link name="propeller${self}">
+      <!-- visual & collisiont -->
+      <inertial>
+        <origin xyz="0 0 0" rpy="0 0 0"/>
+        <mass value="${rotor_mass}"/>
+        <inertia
+            ixx="${rotor_mass * .25 * rotor_radius * rotor_radius}" ixy="0.0" ixz="0.0"
+            iyy="${rotor_mass * .25 * rotor_radius * rotor_radius}" iyz="0.0"
+            izz="${rotor_mass * .5 * rotor_radius * rotor_radius}"/>
+      </inertial>
+    </link>
+    <xacro:damping_factor link ="propeller${self}"/>
+    <!-- joint -->>
+    <xacro:unless value="${tail}">
       <joint name="joint${self}" type="revolute">
-        <limit effort="100.0" lower="-1.57" upper="1.57" velocity="0.5"/>
+        <limit effort="3.1" lower="-1.57" upper="1.57" velocity="0.5"/>
         <parent link="link${self}"/>
-        <child link="joint${self}"/>
-        <origin rpy="0 0 0" xyz="-${link_length*.5} 0 0"/>
+        <child link="link${child}"/>
+        <origin rpy="0 0 0" xyz="${link_length} 0 0"/>
         <axis xyz="0 0 1"/>
-        <dynamics damping="0.8"/>
-      </joint>
-      <link name="joint${self}">
-        <collision>
-          <origin rpy="0 0 0" xyz="0 0 0"/>
-          <geometry>
-            <cylinder length="0.05" radius="0.02"/>
-          </geometry>
-        </collision>
-        <visual>
-          <origin rpy="0 0 0" xyz="0 0 0"/>
-          <geometry>
-            <cylinder length="0.001" radius="0.001"/>
-          </geometry>
-          <material name="color">
-            <color rgba="0.75 .5 .2 1"/>
-          </material>
-        </visual>
-        <inertial>
-          <origin rpy="0 0 0" xyz="0 0 0"/>
-          <mass value="0.1"/>
-          <inertia ixx="0.00005" ixy="0.0" ixz="0.0" iyy="0.00005" iyz="0.0" izz="0.0001"/>
-        </inertial>
-      </link>
-      <joint name="joint${self}_link${child}" type="fixed">
-        <parent link="joint${self}"/>
+        <dynamics damping="0.8" friction="0.05"/>
+        </joint>
+<!--
+      <joint name="joint${self}" type="fixed">
+        <parent link="link${self}"/>
         <child link="link${child}"/>
-        <origin rpy="0 0 0" xyz="-${link_length*.5} 0 0"/>
-      </joint>
-    </xacro:if> <!-- var_head -->
-    <xacro:unless value="${head}">
-      <xacro:if value="${tail}">
-        <link name="link${self}">
-          <xacro:link_model self="4" />
-          <inertial>
-            <origin xyz="0 0 0" rpy="0 0 0"/>
-            <mass value="0.5"/>
-            <inertia
-                ixx="0.1" ixy="0.0" ixz="0.0"
-                iyy="0.01" iyz="0.0"
-                izz="0.11"/>
-          </inertial>
-        </link>
-      </xacro:if> <!-- var_tail -->
-      <xacro:unless value="${tail}">
-        <xacro:if value="${imu}">
-          <link name="link${self}">
-            <xacro:link_model self="2" />
-            <inertial>
-              <origin xyz="0 0 0" rpy="0 0 0"/>
-              <mass value="0.5"/>
-              <inertia
-                  ixx="0.1" ixy="0.0" ixz="0.0"
-                  iyy="0.01" iyz="0.0"
-                  izz="0.11"/>
-            </inertial>
-          </link>
-        </xacro:if> <!-- var_imu -->
-        <xacro:unless value="${imu}"> <!-- var_imu -->
-          <link name="link${self}">
-            <xacro:link_model self="3" />
-            <inertial>
-              <origin xyz="0 0 0" rpy="0 0 0"/>
-              <mass value="0.5"/>
-              <inertia
-                  ixx="0.1" ixy="0.0" ixz="0.0"
-                  iyy="0.01" iyz="0.0"
-                  izz="0.11"/>
-            </inertial>
-          </link>
-        </xacro:unless> <!-- var_imu -->
-        <joint name="joint${self}" type="revolute">
-          <limit effort="100.0" lower="-1.57" upper="1.57" velocity="0.5"/>
-          <parent link="link${self}"/>
-          <child link="joint${self}"/>
-          <origin rpy="0 0 0" xyz="-${link_length*.5} 0 0"/>
-          <axis xyz="0 0 1"/>
-          <dynamics damping="0.7"/>
+        <origin rpy="0 0 ${pi/2}" xyz="${link_length} 0 0"/>
+        <axis xyz="0 0 1"/>
         </joint>
-        <link name="joint${self}">
-          <collision>
-            <origin rpy="0 0 0" xyz="0 0 0"/>
-            <geometry>
-              <cylinder length="0.05" radius="0.02"/>
-            </geometry>
-          </collision>
-          <visual>
-            <origin rpy="0 0 0" xyz="0 0 0"/>
-            <geometry>
-              <cylinder length="0.001" radius="0.001"/>
-            </geometry>
-            <material name="color">
-              <color rgba="0.75 .5 .2 1"/>
-            </material>
-          </visual>
-          <inertial>
-            <origin rpy="0 0 0" xyz="0 0 0"/>
-            <mass value="0.1"/>
-            <inertia ixx="0.00005" ixy="0.0" ixz="0.0" iyy="0.00005" iyz="0.0" izz="0.0001"/>
-          </inertial>
-        </link>
-        <joint name="joint${self}_link${child}" type="fixed">
-          <parent link="joint${self}"/>
-          <child link="link${child}"/>
-          <origin rpy="0 0 0" xyz="-${link_length*.5} 0 0"/>
-        </joint>
-      </xacro:unless> <!-- var_tail -->
-    </xacro:unless> <!-- var_head -->
+-->
+</xacro:unless> <!-- var_tail -->
     <!-- hardware interface -->
     <xacro:unless value="${tail}">
@@ -137,13 +105,26 @@
         <joint name="joint${self}">
           <!-- TODO: effort is torque, maybe position is enough -->
-          <hardwareInterface>EffortJointInterface</hardwareInterface>
+          <hardwareInterface>hardware_interface/EffortJointInterface</hardwareInterface>
         </joint>
         <actuator name="servo{self}">
           <!-- TODO: effort is torque, maybe position is enough -->
-          <hardwareInterface>EffortJointInterface</hardwareInterface>
+          <hardwareInterface>hardware_interface/EffortJointInterface</hardwareInterface>
           <mechanicalReduction>1</mechanicalReduction>
         </actuator>
       </transmission>
     </xacro:unless> <!-- var_tail -->
+    <transmission name="rotor_tran${self}">
+      <type>transmission_interface/SimpleTransmission</type>
+      <joint name="rotor${self}">
+        <!-- TODO: effort is torque, maybe position is enough -->
+        <hardwareInterface>RotorInterface</hardwareInterface>
+      </joint>
+      <actuator name="rotor${self}">
+        <!-- TODO: effort is torque, maybe position is enough -->
+        <hardwareInterface>RotorInterface</hardwareInterface>
+        <mechanicalReduction>1</mechanicalReduction>
+      </actuator>
+    </transmission>
+    <xacro:friction self ="${self}"/>
   </xacro:macro>
 </robot>
