Commit message: improve the model description of hydrus3

File: aerial_robot_model/robots/hydrus3.urdf.xacro (robot description, xacro)
@@ -4,7 +4,7 @@
   <xacro:include filename="$(find aerial_robot_model)/urdf/hydrus3/hydrus3_common.xacro" />
   <xacro:include filename="$(find aerial_robot_model)/urdf/hydrus3/hydrus3_link.urdf.xacro" />
-  <xacro:hydrus3_link self="1" child="2" head="true" tail="false" imu="false" m_link="0.607" i_xx="${protector_inertia * .5}" i_yy="${joint_inertia + pc_inertia + rod_inertia + protector_inertia * .5}" i_zz="${joint_inertia + pc_inertia + rod_inertia + protector_inertia}" />
-  <xacro:hydrus3_link self="2" child="3" head="false" tail="false" imu="true" m_link="0.557" i_xx="${protector_inertia * .5}" i_yy="${joint_inertia + rod_inertia + protector_inertia * .5}" i_zz="${joint_inertia + rod_inertia + protector_inertia}"/>
-  <xacro:hydrus3_link self="3" child="4" head="false" tail="false" imu="false" m_link="0.487" i_xx="${protector_inertia * .5}" i_yy="${joint_inertia + rod_inertia + protector_inertia * .5}" i_zz="${joint_inertia + rod_inertia + protector_inertia}"/>
-  <xacro:hydrus3_link self="4" child="5" head="false" tail="true" imu="false" m_link="0.45" i_xx="${protector_inertia * .5}" i_yy="${rod_inertia + protector_inertia * .5}" i_zz="${rod_inertia + protector_inertia}"/>
+  <xacro:hydrus3_link self="1" child="2" head="true" tail="false" imu="false" />
+  <xacro:hydrus3_link self="2" child="3" head="false" tail="false" imu="true" />
+  <xacro:hydrus3_link self="3" child="4" head="false" tail="false" imu="false" />
+  <xacro:hydrus3_link self="4" child="5" head="false" tail="true" imu="false" />
 </robot>

File: aerial_robot_model/urdf/hydrus3/hydrus3_common.xacro (robot description, xacro)
@@ -3,21 +3,34 @@
     xmlns:xacro="http://www.ros.org/wiki/xacro" name="hydrus3_common" >
   <xacro:property name="pi" value="3.1415926535897931" />
+  <!-- kinematics [m] -->
   <xacro:property name="link_length" value=".44" />
-  <xacro:property name="protector_radius" value=".155" />
-  <xacro:property name="protector_mass" value=".05" />
-  <xacro:property name="pc_mass" value=".1" />
-  <xacro:property name="rotor_mass" value=".05" /> <!-- [g] -->
-  <xacro:property name="rotor_radius" value=".015" /> <!-- [g] -->
+  <xacro:property name="link_rod_length" value=".4" />
+  <xacro:property name="protector_radius" value=".1425" />
+  <xacro:property name="link_joint_offset" value="-0.205" /> <!-- [m] -->
+  <xacro:property name="rotor_radius" value=".015" /> <!-- [m] -->
   <xacro:property name="rotor_height" value=".05" /> <!-- [m] -->
-  <xacro:property name="max_force" value="100" /> <!-- [m] -->
-  <xacro:property name="joint_inertia" value="${.0785 * .205 * .205}" /> <!-- mass * dist * dist -->
-  <xacro:property name="rod_inertia" value="${link_length * link_length * 0.1 /12}" /> <!-- mass * dist * dist -->
-  <xacro:property name="pc_inertia" value="${pc_mass * .189 * .189}" /> <!-- mass * dist * dist -->
+  <xacro:property name="pc_offset" value="-0.189" /> <!-- [m] -->
+  <xacro:property name="fc_offset" value="0.166" /> <!-- [m] -->
+  <!-- dynamics [Kg] -->
+  <xacro:property name="link_rod_mass" value="0.1" />
+  <xacro:property name="link_center_mass" value=".241" />
+  <xacro:property name="joint_mass" value=".0785" />
+  <xacro:property name="protector_mass" value=".048" />
+  <xacro:property name="protector_holder_mass" value=".047" />
+  <xacro:property name="fc_mass" value=".022" />
+  <xacro:property name="pc_mass" value=".104" />
+  <xacro:property name="rotor_mass" value=".05" /> <!-- exclude from center mass -->
+  <xacro:property name="max_force" value="10" /> <!-- [m] -->
+  <xacro:property name="joint_inertia" value="${joint_mass * link_joint_offset * link_joint_offset}" /> <!-- mass * dist * dist -->
+  <xacro:property name="link_rod_inertia" value="${link_rod_mass * link_rod_length * link_rod_length /12}" /> <!-- mass * dist * dist -->
+  <xacro:property name="pc_inertia" value="${pc_mass * pc_offset * pc_offset}" /> <!-- mass * dist * dist -->
+  <xacro:property name="fc_inertia" value="${fc_mass * fc_offset * fc_offset}" /> <!-- mass * dist * dist -->
   <xacro:property name="protector_inertia" value="${protector_mass * protector_radius * protector_radius}" /> <!-- mass * dist * dist -->
+  <xacro:property name="protector_holder_inertia" value="${protector_holder_mass * protector_radius * protector_radius}" /> <!-- mass * dist * dist -->
   <xacro:macro name="link_model" params="self">
     <collision>
       <origin xyz="0 0 0" rpy="0 0 0"/>
       <geometry>
-        <cylinder length="${protector_radius}" radius="0.09"/>
+        <cylinder length="0.13" radius="${protector_radius}"/>
       </geometry>
     </collision>
@@ -28,4 +41,29 @@
       </geometry>
     </visual>
+  </xacro:macro>
+  <xacro:macro name="link_inertial" params="head tail imu">
+    <xacro:if value="${head}">
+      <mass value="${link_rod_mass + link_center_mass + protector_mass + protector_holder_mass + pc_mass - rotor_mass}"/>
+      <inertia
+          ixx="${protector_inertia / 2 }" ixy="0.0" ixz="0.0"
+          iyy="${link_rod_inertia + protector_holder_inertia + protector_inertia /2 + pc_inertia}" iyz="0.0"
+          izz="${link_rod_inertia + protector_holder_inertia + protector_inertia + pc_inertia}"/>
+    </xacro:if>
+    <xacro:unless value="${head}">
+      <xacro:if value="${imu}">
+      <mass value="${link_rod_mass + link_center_mass + joint_mass + protector_mass + protector_holder_mass + fc_mass - rotor_mass}"/>
+      <inertia
+          ixx="${protector_inertia / 2 }" ixy="0.0" ixz="0.0"
+          iyy="${joint_inertia + link_rod_inertia + protector_holder_inertia + protector_inertia /2 + fc_inertia}" iyz="0.0"
+          izz="${joint_inertia + link_rod_inertia + protector_holder_inertia + protector_inertia + fc_inertia}"/>
+      </xacro:if>
+      <xacro:unless value="${imu}">
+        <mass value="${link_rod_mass + link_center_mass + joint_mass + protector_mass + protector_holder_mass - rotor_mass}"/>
+        <inertia
+            ixx="${protector_inertia / 2 }" ixy="0.0" ixz="0.0"
+            iyy="${joint_inertia + link_rod_inertia + protector_holder_inertia + protector_inertia /2}" iyz="0.0"
+            izz="${joint_inertia + link_rod_inertia + protector_holder_inertia + protector_inertia}"/>
+      </xacro:unless>
+    </xacro:unless>
   </xacro:macro>
   <!-- friction -->

File: aerial_robot_model/urdf/hydrus3/hydrus3_link.urdf.xacro (robot description, xacro)
@@ -3,7 +3,12 @@
     xmlns:xacro="http://www.ros.org/wiki/xacro" name="hydrus3_link" >
   <!-- D-H kai description(different from prof.nakamura) -->
-  <xacro:macro name="hydrus3_link" params="self child head tail imu m_link i_xx i_yy i_zz">
+  <xacro:macro name="hydrus3_link" params="self child head tail imu">
     <!-- link -->
     <link name="link${self}">
+      <!-- inertial -->
+      <inertial>
+        <origin xyz="${link_length*.5} 0 0" rpy="0 0 0"/>
+        <xacro:link_inertial head = "${head}" tail = "${tail}" imu = "${imu}" />
+      </inertial>
       <!-- visual & collisiont -->
       <xacro:if value="${head}">
@@ -23,19 +28,4 @@
         </xacro:unless>
       </xacro:unless>
-      <inertial>
-        <origin xyz="${link_length*.5} 0 0" rpy="0 0 0"/>
-        <mass value="${m_link}"/>
-<!--
-        <inertia
-            ixx="0.0001" ixy="0.0" ixz="0.0"
-            iyy="0.005" iyz="0.0"
-            izz="0.0051"/>
-            </inertial>
--->
-        <inertia
-            ixx="${i_xx}" ixy="0.0" ixz="0.0"
-            iyy="${i_yy}" iyz="0.0"
-            izz="${i_zz}"/>
-            </inertial>
     </link>
     <xacro:damping_factor link ="link${self}"/>
@@ -89,14 +79,6 @@
         <axis xyz="0 0 1"/>
         <dynamics damping="0.8" friction="0.05"/>
-        </joint>
-<!--
-      <joint name="joint${self}" type="fixed">
-        <parent link="link${self}"/>
-        <child link="link${child}"/>
-        <origin rpy="0 0 ${pi/2}" xyz="${link_length} 0 0"/>
-        <axis xyz="0 0 1"/>
-        </joint>
--->
-</xacro:unless> <!-- var_tail -->
+      </joint>
+    </xacro:unless> <!-- var_tail -->
     <!-- hardware interface -->
     <xacro:unless value="${tail}">
