Commit message: modified the cog/pricipal_calc for hydra3, as well as the modelling

File: aerial_robot_model/robots/test/test.urdf (robot description, URDF)
Before this commit: robot test, 3 links, 2 joints
Links:
- removed link abdomen2
- removed link abdomen3
- link abdomen: geometry visual mesh filename=package://aerial_robot_model/urdf/hydra3/mesh/hydra_link3.s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 scale=.001 .001 .001
Joints:
- removed joint tiltrotor_pitch_joint
- removed joint tiltrotor_roll_joint
