Commit message: Change the model of hydrus3 from stl style to dea style, which is more compatible for gazebo and eus.

File: aerial_robot_model/urdf/hydrus3/hydrus3_link.urdf.xacro (robot description, xacro)
@@ -15,5 +15,5 @@
           <origin rpy="0 0 ${pi}" xyz="0 0 0"/>
           <geometry>
-            <mesh filename="package://aerial_robot_model/urdf/hydrus3/mesh/hydrus3_link1.stl" scale=".001 .001 .001"/>
+            <mesh filename="package://aerial_robot_model/urdf/hydrus3/mesh/hydrus3_link1.dae"/>
           </geometry>
           <xacro:link_color />
@@ -76,5 +76,5 @@
             <origin rpy="0 0 ${pi}" xyz="0 0 0"/>
             <geometry>
-              <mesh filename="package://aerial_robot_model/urdf/hydrus3/mesh/hydrus3_link4.stl" scale=".001 .001 .001"/>
+              <mesh filename="package://aerial_robot_model/urdf/hydrus3/mesh/hydrus3_link4.dae" />
             </geometry>
             <xacro:link_color />
@@ -102,5 +102,5 @@
               <origin rpy="0 0 ${pi}" xyz="0 0 0"/>
               <geometry>
-                <mesh filename="package://aerial_robot_model/urdf/hydrus3/mesh/hydrus3_link2.stl" scale=".001 .001 .001"/>
+                <mesh filename="package://aerial_robot_model/urdf/hydrus3/mesh/hydrus3_link2.dae"/>
               </geometry>
               <xacro:link_color />
@@ -127,5 +127,5 @@
               <origin rpy="0 0 ${pi}" xyz="0 0 0"/>
               <geometry>
-                <mesh filename="package://aerial_robot_model/urdf/hydrus3/mesh/hydrus3_link3.stl" scale=".001 .001 .001"/>
+                <mesh filename="package://aerial_robot_model/urdf/hydrus3/mesh/hydrus3_link3.dae"/>
               </geometry>
               <xacro:link_color />
