Commit message: Update the description of hydrus3 common/link urdf, new elements: base_inertia

File: aerial_robot_model/urdf/hydrus3/hydrus3_common.xacro (robot description, xacro)
@@ -12,5 +12,6 @@
   <xacro:property name="pc_offset" value="-0.189" /> <!-- [m] -->
   <xacro:property name="fc_offset" value="0.166" /> <!-- [m] -->
-  <!-- dynamics [Kg] -->
+  <!-- inertial parameter -->
+  <!-- mass [Kg] -->
   <xacro:property name="link_rod_mass" value="0.1" />
   <xacro:property name="link_center_mass" value=".241" />
@@ -21,5 +22,6 @@
   <xacro:property name="pc_mass" value=".104" />
   <xacro:property name="rotor_mass" value=".05" /> <!-- exclude from center mass -->
-  <xacro:property name="max_force" value="10" /> <!-- [m] -->
+  <xacro:property name="base_mass" value="${link_rod_mass + link_center_mass + joint_mass + protector_mass + protector_holder_mass - rotor_mass}" /> <!-- exclude from center mass -->
+  <!-- inertial [N*m*m] -->
   <xacro:property name="joint_inertia" value="${joint_mass * link_joint_offset * link_joint_offset}" /> <!-- mass * dist * dist -->
   <xacro:property name="link_rod_inertia" value="${link_rod_mass * link_rod_length * link_rod_length /12}" /> <!-- mass * dist * dist -->
@@ -28,7 +30,12 @@
   <xacro:property name="protector_inertia" value="${protector_mass * protector_radius * protector_radius}" /> <!-- mass * dist * dist -->
   <xacro:property name="protector_holder_inertia" value="${protector_holder_mass * protector_radius * protector_radius}" /> <!-- mass * dist * dist -->
-  <xacro:macro name="link_model" params="self">
+  <xacro:property name="base_ixx" value="${protector_inertia / 2}" />
+  <xacro:property name="base_iyy" value="${joint_inertia + link_rod_inertia + protector_holder_inertia + protector_inertia /2}" />
+  <xacro:property name="base_izz" value="${joint_inertia + link_rod_inertia + protector_holder_inertia + protector_inertia}" />
+  <!-- dynamics [N] -->
+  <xacro:property name="max_force" value="10" /> <!-- [m] -->
+  <xacro:macro name="link_model" params="type">
     <collision>
-      <origin xyz="0 0 0" rpy="0 0 0"/>
+      <origin xyz="0 0 0" rpy="${link_length*.5} 0 0"/>
       <geometry>
         <cylinder length="0.13" radius="${protector_radius}"/>
@@ -38,32 +45,14 @@
       <origin rpy="${-pi/2} 0 0" xyz="${link_length*.5} 0 0"/>
       <geometry>
-        <mesh filename="package://aerial_robot_model/urdf/hydrus3/mesh/hydrus3_link${self}.dae"/>
+        <mesh filename="package://aerial_robot_model/urdf/hydrus3/mesh/hydrus3_link${type}.dae"/>
       </geometry>
     </visual>
   </xacro:macro>
-  <xacro:macro name="link_inertial" params="head tail imu">
-    <xacro:if value="${head}">
-      <mass value="${link_rod_mass + link_center_mass + protector_mass + protector_holder_mass + pc_mass - rotor_mass}"/>
-      <inertia
-          ixx="${protector_inertia / 2 }" ixy="0.0" ixz="0.0"
-          iyy="${link_rod_inertia + protector_holder_inertia + protector_inertia /2 + pc_inertia}" iyz="0.0"
-          izz="${link_rod_inertia + protector_holder_inertia + protector_inertia + pc_inertia}"/>
-    </xacro:if>
-    <xacro:unless value="${head}">
-      <xacro:if value="${imu}">
-      <mass value="${link_rod_mass + link_center_mass + joint_mass + protector_mass + protector_holder_mass + fc_mass - rotor_mass}"/>
-      <inertia
-          ixx="${protector_inertia / 2 }" ixy="0.0" ixz="0.0"
-          iyy="${joint_inertia + link_rod_inertia + protector_holder_inertia + protector_inertia /2 + fc_inertia}" iyz="0.0"
-          izz="${joint_inertia + link_rod_inertia + protector_holder_inertia + protector_inertia + fc_inertia}"/>
-      </xacro:if>
-      <xacro:unless value="${imu}">
-        <mass value="${link_rod_mass + link_center_mass + joint_mass + protector_mass + protector_holder_mass - rotor_mass}"/>
+  <xacro:macro name="link_inertial" params="extra_mass extra_ixx extra_iyy extra_izz">
+    <mass value="${base_mass + extra_mass}"/>
         <inertia
-            ixx="${protector_inertia / 2 }" ixy="0.0" ixz="0.0"
-            iyy="${joint_inertia + link_rod_inertia + protector_holder_inertia + protector_inertia /2}" iyz="0.0"
-            izz="${joint_inertia + link_rod_inertia + protector_holder_inertia + protector_inertia}"/>
-      </xacro:unless>
-    </xacro:unless>
+            ixx="${base_ixx + extra_ixx}" ixy="0.0" ixz="0.0"
+            iyy="${base_iyy + extra_iyy}" iyz="0.0"
+            izz="${base_izz + extra_izz}"/>
   </xacro:macro>
   <!-- friction -->

File: aerial_robot_model/urdf/hydrus3/hydrus3_link.urdf.xacro (robot description, xacro)
@@ -3,29 +3,47 @@
     xmlns:xacro="http://www.ros.org/wiki/xacro" name="hydrus3_link" >
   <!-- D-H kai description(different from prof.nakamura) -->
-  <xacro:macro name="hydrus3_link" params="self child head tail imu">
+  <xacro:macro name="hydrus3_link" params="self child general fc pc">
     <!-- link -->
     <link name="link${self}">
-      <!-- inertial -->
+      <!-- common inertial -->
       <inertial>
         <origin xyz="${link_length*.5} 0 0" rpy="0 0 0"/>
-        <xacro:link_inertial head = "${head}" tail = "${tail}" imu = "${imu}" />
+        <!-- mass and inertia -->
+        <!-- head -->
+        <xacro:if value="${self == 1}">
+          <xacro:link_inertial extra_mass = "${pc_mass}" extra_ixx = "0" extra_iyy = "${pc_inertia}" extra_izz = "${pc_inertia}" />
+        </xacro:if>
+        <!-- tail -->
+        <xacro:if value="${self == child}">
+          <xacro:link_inertial extra_mass = "0" extra_ixx = "0" extra_iyy = "0" extra_izz = "0" />
+        </xacro:if>
+        <!-- fc -->
+        <xacro:if value="${fc}">
+          <xacro:link_inertial extra_mass = "${fc_mass}" extra_ixx = "0" extra_iyy = "${fc_inertia}" extra_izz = "${fc_inertia}" />
+        </xacro:if>
+        <!-- pc: no -->
+        <!-- general -->
+        <xacro:if value="${general}">
+          <xacro:link_inertial extra_mass = "0" extra_ixx = "0" extra_iyy = "0" extra_izz = "0" />
+        </xacro:if>
       </inertial>
-      <!-- visual & collisiont -->
-      <xacro:if value="${head}">
-        <xacro:link_model self="1" />
+      <!-- sepcial inertia & visual & collision -->
+      <!-- head -->
+      <xacro:if value="${self == 1}">
+        <xacro:link_model type="1" />
       </xacro:if>
-      <xacro:unless value="${head}">
-        <xacro:if value="${imu}">
-          <xacro:link_model self="2" />
-        </xacro:if>
-        <xacro:unless value="${imu}">
-          <xacro:if value="${tail}">
-            <xacro:link_model self="4" />
-          </xacro:if>
-          <xacro:unless value="${tail}">
-            <xacro:link_model self="3" />
-          </xacro:unless>
-        </xacro:unless>
-      </xacro:unless>
+      <!-- tail -->
+      <xacro:if value="${self == child}">
+        <xacro:link_model type="4" />
+      </xacro:if>
+      <!-- fc -->
+      <xacro:if value="${fc}">
+        <xacro:link_model type="2" />
+      </xacro:if>
+      <!-- pc: no -->
+      <!-- general -->
+      <xacro:if value="${general}">
+        <xacro:link_model type="3" />
+      </xacro:if>
     </link>
     <xacro:damping_factor link ="link${self}"/>
@@ -71,5 +89,5 @@
     <xacro:damping_factor link ="propeller${self}"/>
     <!-- joint -->>
-    <xacro:unless value="${tail}">
+    <xacro:unless value="${self == child}">
       <joint name="joint${self}" type="revolute">
         <limit effort="3.1" lower="-1.57" upper="1.57" velocity="0.5"/>
@@ -80,7 +98,7 @@
         <dynamics damping="0.8" friction="0.05"/>
       </joint>
-    </xacro:unless> <!-- var_tail -->
+    </xacro:unless>
     <!-- hardware interface -->
-    <xacro:unless value="${tail}">
+    <xacro:unless value="${self == child}">
       <transmission name="joint_tran${self}">
         <type>transmission_interface/SimpleTransmission</type>
@@ -95,5 +113,5 @@
         </actuator>
       </transmission>
-    </xacro:unless> <!-- var_tail -->
+    </xacro:unless>
     <transmission name="rotor_tran${self}">
       <type>transmission_interface/SimpleTransmission</type>

Commit message: Fix the wrong origion setting for the collision model

File: aerial_robot_model/urdf/hydrus3/hydrus3_common.xacro (robot description, xacro)
@@ -37,5 +37,5 @@
   <xacro:macro name="link_model" params="type">
     <collision>
-      <origin xyz="0 0 0" rpy="${link_length*.5} 0 0"/>
+      <origin rpy="0 0 0" xyz="${link_length*.5} 0 0"/>
       <geometry>
         <cylinder length="0.13" radius="${protector_radius}"/>

Commit message: modified the urdf model and related tf publisher code to be suitable for KDL based kinematics

File: aerial_robot_model/urdf/hydrus3/hydrus3_common.xacro (robot description, xacro)
@@ -30,5 +30,5 @@
   <xacro:macro name="link_model" params="type">
     <collision>
-      <origin rpy="0 0 0" xyz="0 0 0"/>
+      <origin rpy="0 0 0" xyz="${link_length* 0.5} 0 0"/>
       <geometry>
         <cylinder length="0.13" radius="${protector_radius}"/>
@@ -36,5 +36,5 @@
     </collision>
     <visual>
-      <origin rpy="${-pi/2} 0 0" xyz="0 0 0"/>
+      <origin rpy="${-pi/2} 0 0" xyz="${link_length* 0.5} 0 0"/>
       <geometry>
         <mesh filename="package://aerial_robot_model/urdf/hydrus3/mesh/hydrus3_link${type}.dae"/>

File: aerial_robot_model/urdf/hydrus3/hydrus3_link.urdf.xacro (robot description, xacro)
@@ -6,22 +6,7 @@
     <!-- link -->
     <link name="link${self}">
+      <!-- common inertial -->
       <inertial>
-        <origin xyz="0 0 0" rpy="0 0 0"/>
-        <mass value="0.0000001"/>
-        <inertia
-            ixx="0.00000001" ixy="0.0" ixz="0.0"
-            iyy="0.00000001" iyz="0.0"
-            izz="0.00000002"/>
-      </inertial>
-    </link>
-    <joint name="link${self}2center" type="fixed">
-      <parent link="link${self}"/>
-      <child link="link${self}_center"/>
-      <origin rpy="0 0 0" xyz="${link_length* 0.5} 0 0"/>
-      <axis xyz="0 0 1"/>
-    </joint>
-    <link name="link${self}_center">
-      <inertial>
-        <origin xyz="0 0 0" rpy="0 0 0"/>
+        <origin xyz="${link_length* 0.5} 0 0" rpy="0 0 0"/>
         <mass value="${link_rod_mass + link_center_mass + protector_mass + protector_holder_mass - rotor_mass}" /> <!-- exclude from center mass -->
         <inertia
@@ -53,7 +38,7 @@
     <joint name="rotor${self}" type="continuous">
       <limit effort="100.0" lower="0" upper="${max_force}" velocity="0.5"/> <!-- force range -->
-      <parent link="link${self}_center"/>
+      <parent link="link${self}"/>
       <child link="propeller${self}"/>
-      <origin rpy="0 0 0" xyz="0 0 0"/>
+      <origin rpy="0 0 0" xyz="${link_length* 0.5} 0 0"/>
       <axis xyz="0 0 1"/>
     </joint>
@@ -71,4 +56,24 @@
     <xacro:damping_factor link ="propeller${self}"/>
     <!-- extra module -->
+    <!-- head -->
+    <xacro:if value="${self == 1}">
+      <!-- dummy root link for KDL -->
+      <link name="root">
+        <inertial>
+          <origin xyz="0 0 0" rpy="0 0 0"/>
+          <mass value="0.00001"/>
+          <inertia
+              ixx="0.000001" ixy="0.0" ixz="0.0"
+              iyy="0.000001" iyz="0.0"
+              izz="0.000002"/>
+        </inertial>
+      </link>
+      <joint name="root_joint" type="fixed">
+        <parent link="root"/>
+        <child link="link${self}"/>
+        <origin rpy="0 0 0" xyz="0 0 0"/>
+        <axis xyz="0 0 1"/>
+      </joint>
+    </xacro:if>
     <!-- pc -->
     <xacro:if value="${pc}">

File: aerial_robot_model/urdf/hydrusx/hydrusx_common.xacro (robot description, xacro)
@@ -44,5 +44,5 @@
   <xacro:macro name="link_model" params="type">
     <collision>
-      <origin rpy="0 0 0" xyz="0 0 -0.03"/>
+      <origin rpy="0 0 0" xyz="${link_length* 0.5} 0 -0.03"/>
       <geometry>
         <cylinder length="0.15" radius="${protector_radius}"/>
@@ -50,5 +50,5 @@
     </collision>
     <visual>
-      <origin rpy="${-pi/2} 0 0" xyz="0 0 0"/>
+      <origin rpy="${-pi/2} 0 0" xyz="${link_length* 0.5} 0 0"/>
       <geometry>
         <mesh filename="package://aerial_robot_model/urdf/hydrusx/mesh/hydrusx_link${type}.dae"/>

File: aerial_robot_model/urdf/hydrusx/hydrusx_link.urdf.xacro (robot description, xacro)
@@ -8,21 +8,5 @@
       <!-- common inertial -->
       <inertial>
-        <origin xyz="0 0 0" rpy="0 0 0"/>
-        <mass value="0.0000001"/>
-        <inertia
-            ixx="0.00000001" ixy="0.0" ixz="0.0"
-            iyy="0.00000001" iyz="0.0"
-            izz="0.00000002"/>
-      </inertial>
-    </link>
-    <joint name="link${self}2center" type="fixed">
-      <parent link="link${self}"/>
-      <child link="link${self}_center"/>
-      <origin rpy="0 0 0" xyz="${link_length* 0.5} 0 0"/>
-      <axis xyz="0 0 1"/>
-    </joint>
-    <link name="link${self}_center">
-      <inertial>
-        <origin xyz="0 0 0" rpy="0 0 0"/>
+        <origin xyz="${link_length* 0.5} 0 0" rpy="0 0 0"/>
         <mass value="${link_rod_mass + link_center_mass + protector_mass + protector_holder_mass - rotor_mass}" /> <!-- exclude from center mass -->
         <inertia
@@ -57,7 +41,7 @@
     <joint name="rotor${self}" type="continuous">
       <limit effort="100.0" lower="0" upper="${max_force}" velocity="0.5"/> <!-- force range -->
-      <parent link="link${self}_center"/>
+      <parent link="link${self}"/>
       <child link="propeller${self}"/>
-      <origin rpy="0 0 0" xyz="0 0 0"/>
+      <origin rpy="0 0 0" xyz="${link_length* 0.5} 0 0"/>
       <axis xyz="0 0 1"/>
     </joint>
@@ -77,4 +61,21 @@
     <!-- head -->
     <xacro:if value="${self == 1}">
+      <!-- dummy root link for KDL -->
+      <link name="root">
+        <inertial>
+          <origin xyz="0 0 0" rpy="0 0 0"/>
+          <mass value="0.00001"/>
+          <inertia
+              ixx="0.000001" ixy="0.0" ixz="0.0"
+              iyy="0.000001" iyz="0.0"
+              izz="0.000002"/>
+        </inertial>
+      </link>
+      <joint name="root_joint" type="fixed">
+        <parent link="root"/>
+        <child link="link${self}"/>
+        <origin rpy="0 0 0" xyz="0 0 0"/>
+        <axis xyz="0 0 1"/>
+      </joint>
       <xacro:extra_module name = "head" parent = "${self}" mass = "${head_leg_mass}" offset = "${link_length * 0.5 + head_leg_offset}" />
       <!-- battery -->
