Commit message: Update the model for hydrusx model

File: aerial_robot_model/urdf/hydrusx/hydrusx_common.xacro (robot description, xacro)
@@ -3,10 +3,77 @@
     xmlns:xacro="http://www.ros.org/wiki/xacro" name="hydrusx_common" >
   <xacro:property name="pi" value="3.1415926535897931" />
+  <!-- kinematics [m] -->
   <xacro:property name="link_length" value=".6" />
-  <xacro:property name="protector_radius" value=".2" />
-  <xacro:macro name="link_color">
-    <material name="color">
-      <color rgba="0.75 .5 .2 1"/>
-    </material>
+  <xacro:property name="link_rod_length" value=".528" />
+  <xacro:property name="protector_radius" value=".1925" />
+  <xacro:property name="link_joint_offset" value="0.3" /> <!-- [m] -->
+  <xacro:property name="rotor_radius" value=".02" /> <!-- [m] -->
+  <xacro:property name="rotor_height" value=".05" /> <!-- [m] -->
+  <xacro:property name="pc_offset" value="0.22" /> <!-- [m] -->
+  <xacro:property name="fc_offset" value="-0.28" /> <!-- [m] -->
+  <xacro:property name="tail_leg_offset" value="0.235" /> <!-- [m] -->
+  <xacro:property name="head_leg_offset" value="-0.247" /> <!-- [m] -->
+  <xacro:property name="sensor_offset" value="-0.215" /> <!-- [m] -->
+  <!-- inertial paramters -->
+  <!-- mass [Kg] -->
+  <xacro:property name="link_center_mass" value=".4046" />
+  <xacro:property name="joint_mass" value=".2075" />
+  <xacro:property name="link_rod_mass" value="0.099" />
+  <xacro:property name="protector_mass" value=".05" />
+  <xacro:property name="protector_holder_mass" value=".0386" />
+  <xacro:property name="fc_mass" value=".03" />
+  <xacro:property name="pc_mass" value=".24" />
+  <xacro:property name="tail_leg_mass" value="0.0623" />
+  <xacro:property name="head_leg_mass" value="0.0623" />
+  <xacro:property name="sensor_mass" value="0.06" />
+  <xacro:property name="rotor_mass" value=".05" /> <!-- exclude from center mass -->
+  <xacro:property name="base_mass" value="${link_rod_mass + link_center_mass + joint_mass + protector_mass + protector_holder_mass - rotor_mass}" /> <!-- exclude from center mass -->
+  <!-- inertial [N*m*m] -->
+  <xacro:property name="joint_inertia" value="${joint_mass * link_joint_offset * link_joint_offset}" /> <!-- mass * dist * dist -->
+  <xacro:property name="link_rod_inertia" value="${link_rod_mass * link_rod_length * link_rod_length /12}" /> <!-- mass * dist * dist -->
+  <xacro:property name="pc_inertia" value="${pc_mass * pc_offset * pc_offset}" /> <!-- mass * dist * dist -->
+  <xacro:property name="fc_inertia" value="${fc_mass * fc_offset * fc_offset}" /> <!-- mass * dist * dist -->
+  <xacro:property name="sensor_inertia" value="${sensor_mass * sensor_offset * sensor_offset}" /> <!-- mass * dist * dist -->
+  <xacro:property name="head_leg_inertia" value="${head_leg_mass * head_leg_offset * head_leg_offset}" /> <!-- mass * dist * dist -->
+  <xacro:property name="tail_leg_inertia" value="${tail_leg_mass * tail_leg_offset * tail_leg_offset}" /> <!-- mass * dist * dist -->
+  <xacro:property name="protector_inertia" value="${protector_mass * protector_radius * protector_radius}" /> <!-- mass * dist * dist -->
+  <xacro:property name="protector_holder_inertia" value="${protector_holder_mass * protector_radius * protector_radius}" /> <!-- mass * dist * dist -->
+  <xacro:property name="base_ixx" value="${protector_inertia / 2}" />
+  <xacro:property name="base_iyy" value="${joint_inertia + link_rod_inertia + protector_holder_inertia + protector_inertia /2}" />
+  <xacro:property name="base_izz" value="${joint_inertia + link_rod_inertia + protector_holder_inertia + protector_inertia}" />
+  <!-- dynamics -->
+  <xacro:property name="max_force" value="18" /> <!-- [N] -->
+  <xacro:macro name="link_model" params="type">
+    <collision>
+      <origin xyz="0 0 0" rpy="${link_length*.5} 0 0"/>
+      <geometry>
+        <cylinder length="0.10" radius="${protector_radius}"/>
+      </geometry>
+    </collision>
+    <visual>
+      <origin rpy="${-pi/2} 0 0" xyz="${link_length*.5} 0 0"/>
+      <geometry>
+        <mesh filename="package://aerial_robot_model/urdf/hydrusx/mesh/hydrusx_link${type}.dae"/>
+      </geometry>
+    </visual>
+  </xacro:macro>
+  <xacro:macro name="link_inertial" params="extra_mass extra_ixx extra_iyy extra_izz">
+    <mass value="${base_mass + extra_mass}"/>
+        <inertia
+            ixx="${base_ixx + extra_ixx}" ixy="0.0" ixz="0.0"
+            iyy="${base_iyy + extra_iyy}" iyz="0.0"
+            izz="${base_izz + extra_izz}"/>
+  </xacro:macro>
+  <!-- friction -->
+  <xacro:macro name="friction" params="self">
+    <gazebo reference="link${self}">
+      <mu1>0.0001</mu1>
+      <mu2>0.0001</mu2>
+    </gazebo>
+  </xacro:macro>
+  <xacro:macro name="damping_factor" params="link">
+    <gazebo reference="${link}">
+      <dampingFactor>0.00</dampingFactor>
+    </gazebo>
   </xacro:macro>
 </robot>

File: aerial_robot_model/urdf/hydrusx/hydrusx_link.urdf.xacro (robot description, xacro)
@@ -2,206 +2,135 @@
 <robot
     xmlns:xacro="http://www.ros.org/wiki/xacro" name="hydrusx_link" >
-  <xacro:macro name="hydrusx_link" params="self child head tail imu pc">
-    <xacro:if value="${head}">
-      <link name="link${self}">
-        <collision>
-          <origin xyz="0 0 0" rpy="0 0 0"/>
-          <geometry>
-          <cylinder length="0.1" radius="${protector_radius}"/>
-          </geometry>
-        </collision>
-        <visual>
-          <origin rpy="0 0 0" xyz="0 0 0"/>
-          <geometry>
-            <mesh filename="package://aerial_robot_model/urdf/hydrusx/mesh/hydrusx_link1.dae"/>
-          </geometry>
-          <xacro:link_color />
-        </visual>
-        <inertial>
-          <origin xyz="0 0 0" rpy="0 0 0"/>
-          <mass value="0.5"/>
-          <inertia
-	      ixx="0.1" ixy="0.0" ixz="0.0"
-	      iyy="0.01" iyz="0.0"
-	      izz="0.11"/>
-        </inertial>
-      </link>
+  <!-- D-H kai description(different from prof.nakamura) -->
+  <xacro:macro name="hydrusx_link" params="self child general fc pc">
+    <!-- link -->
+    <link name="link${self}">
+      <!-- common inertial -->
+      <inertial>
+        <origin xyz="${link_length*.5} 0 0" rpy="0 0 0"/>
+        <!-- mass and inertia -->
+        <!-- head -->
+        <xacro:if value="${self == 1}">
+          <xacro:link_inertial extra_mass = "${head_leg_mass}" extra_ixx = "0" extra_iyy = "${head_leg_inertia}" extra_izz = "${head_leg_inertia}" />
+        </xacro:if>
+        <!-- tail -->
+        <xacro:if value="${self == child}">
+          <xacro:link_inertial extra_mass = "${tail_leg_mass}" extra_ixx = "0" extra_iyy = "${tail_leg_inertia}" extra_izz = "${tail_leg_inertia}" />
+        </xacro:if>
+        <!-- fc -->
+        <xacro:if value="${fc}">
+          <xacro:link_inertial extra_mass = "${sensor_mass + fc_mass}" extra_ixx = "0" extra_iyy = "${sensor_inertia + fc_inertia}" extra_izz = "${sensor_inertia + fc_inertia}" />
+        </xacro:if>
+        <!-- pc: -->
+        <xacro:if value="${pc}">
+          <xacro:link_inertial extra_mass = "${pc_mass}" extra_ixx = "0" extra_iyy = "${pc_inertia}" extra_izz = "${pc_inertia}" />
+        </xacro:if>
+        <!-- general -->
+        <xacro:if value="${general}">
+          <xacro:link_inertial extra_mass = "0" extra_ixx = "0" extra_iyy = "0" extra_izz = "0" />
+        </xacro:if>
+      </inertial>
+      <!-- sepcial inertia & visual & collision -->
+      <!-- head -->
+      <xacro:if value="${self == 1}">
+        <xacro:link_model type="1" />
+      </xacro:if>
+      <!-- tail -->
+      <xacro:if value="${self == child}">
+        <xacro:link_model type="4" />
+      </xacro:if>
+      <!-- fc -->
+      <xacro:if value="${fc}">
+        <xacro:link_model type="3" />
+      </xacro:if>
+      <!-- pc: -->
+      <xacro:if value="${pc}">
+        <xacro:link_model type="2" />
+      </xacro:if>
+      <!-- general -->
+      <xacro:if value="${general}">
+        <xacro:link_model type="5" />
+      </xacro:if>
+    </link>
+    <xacro:damping_factor link ="link${self}"/>
+    <!-- link center(virtual) -->
+    <!-- not good -->
+    <joint name="center${self}" type="fixed">
+      <parent link="link${self}"/>
+      <child link="link${self}_center"/>
+      <origin rpy="0 0 0" xyz="${link_length*.5} 0 0"/>
+      <axis xyz="0 0 1"/>
+    </joint>
+    <link name="link${self}_center">
+      <!-- visual & collisiont -->
+      <inertial>
+        <origin xyz="0 0 0" rpy="0 0 0"/>
+        <mass value="0.001"/>
+        <inertia
+            ixx="0.00000001" ixy="0.0" ixz="0.0"
+            iyy="0.00000001" iyz="0.0"
+            izz="0.00000002"/>
+      </inertial>
+    </link>
+    <xacro:damping_factor link ="link${self}_center"/>
+    <!-- rotor -->
+    <joint name="rotor${self}" type="continuous">
+      <limit effort="100.0" lower="0" upper="${max_force}" velocity="0.5"/> <!-- force range -->
+      <parent link="link${self}"/>
+      <child link="propeller${self}"/>
+      <origin rpy="0 0 0" xyz="${link_length*.5} 0 0"/>
+      <axis xyz="0 0 1"/>
+    </joint>
+    <link name="propeller${self}">
+      <!-- visual & collisiont -->
+      <inertial>
+        <origin xyz="0 0 0" rpy="0 0 0"/>
+        <mass value="${rotor_mass}"/>
+        <inertia
+            ixx="${rotor_mass * .25 * rotor_radius * rotor_radius}" ixy="0.0" ixz="0.0"
+            iyy="${rotor_mass * .25 * rotor_radius * rotor_radius}" iyz="0.0"
+            izz="${rotor_mass * .5 * rotor_radius * rotor_radius}"/>
+      </inertial>
+    </link>
+    <xacro:damping_factor link ="propeller${self}"/>
+    <!-- joint -->>
+    <xacro:unless value="${self == child}">
       <joint name="joint${self}" type="revolute">
-        <limit effort="100.0" lower="-1.57" upper="1.57" velocity="0.5"/>
+        <limit effort="3.1" lower="-1.57" upper="1.57" velocity="0.5"/>
         <parent link="link${self}"/>
-        <child link="joint${self}"/>
-        <origin rpy="0 0 0" xyz="-${link_length*.5} 0 0"/>
+        <child link="link${child}"/>
+        <origin rpy="0 0 0" xyz="${link_length} 0 0"/>
         <axis xyz="0 0 1"/>
-        <dynamics damping="0.8"/>
+        <dynamics damping="0.8" friction="0.05"/>
       </joint>
-      <link name="joint${self}">
-        <collision>
-          <origin rpy="0 0 0" xyz="0 0 0"/>
-          <geometry>
-            <cylinder length="0.05" radius="0.02"/>
-          </geometry>
-        </collision>
-        <visual>
-          <origin rpy="0 0 0" xyz="0 0 0"/>
-          <geometry>
-            <cylinder length="0.001" radius="0.001"/>
-          </geometry>
-          <material name="color">
-            <color rgba="0.75 .5 .2 1"/>
-          </material>
-        </visual>
-        <inertial>
-          <origin rpy="0 0 0" xyz="0 0 0"/>
-          <mass value="0.1"/>
-          <inertia ixx="0.00005" ixy="0.0" ixz="0.0" iyy="0.00005" iyz="0.0" izz="0.0001"/>
-        </inertial>
-      </link>
-      <joint name="joint${self}_link${child}" type="fixed">
-        <parent link="joint${self}"/>
-        <child link="link${child}"/>
-        <origin rpy="0 0 0" xyz="-${link_length*.5} 0 0"/>
+    </xacro:unless>
+    <!-- hardware interface -->
+    <xacro:unless value="${self == child}">
+      <transmission name="joint_tran${self}">
+        <type>transmission_interface/SimpleTransmission</type>
+        <joint name="joint${self}">
+          <!-- TODO: effort is torque, maybe position is enough -->
+          <hardwareInterface>hardware_interface/EffortJointInterface</hardwareInterface>
+        </joint>
+        <actuator name="servo{self}">
+          <!-- TODO: effort is torque, maybe position is enough -->
+          <hardwareInterface>hardware_interface/EffortJointInterface</hardwareInterface>
+          <mechanicalReduction>1</mechanicalReduction>
+        </actuator>
+      </transmission>
+    </xacro:unless>
+    <transmission name="rotor_tran${self}">
+      <type>transmission_interface/SimpleTransmission</type>
+      <joint name="rotor${self}">
+        <!-- TODO: effort is torque, maybe position is enough -->
+        <hardwareInterface>RotorInterface</hardwareInterface>
       </joint>
-    </xacro:if>
-    <xacro:unless value="${head}">
-      <xacro:if value="${tail}">
-        <link name="link${self}">
-          <collision>
-            <origin xyz="0 0 0" rpy="0 0 0"/>
-            <geometry>
-              <cylinder length="${protector_radius}" radius="0.1"/>
-            </geometry>
-          </collision>
-          <visual>
-            <origin rpy="0 0 0" xyz="0 0 0"/>
-            <geometry>
-              <mesh filename="package://aerial_robot_model/urdf/hydrusx/mesh/hydrusx_link5.dae" />
-            </geometry>
-            <xacro:link_color />
-          </visual>
-          <inertial>
-            <origin xyz="0 0 0" rpy="0 0 0"/>
-            <mass value="0.5"/>
-            <inertia
-	        ixx="0.1" ixy="0.0" ixz="0.0"
-	        iyy="0.01" iyz="0.0"
-	        izz="0.11"/>
-          </inertial>
-        </link>
-      </xacro:if>
-      <xacro:unless value="${tail}">
-        <xacro:if value="${imu}">
-          <link name="link${self}">
-            <collision>
-              <origin xyz="0 0 0" rpy="0 0 0"/>
-              <geometry>
-                <cylinder length="${protector_radius}" radius="0.1"/>
-              </geometry>
-            </collision>
-            <visual>
-              <origin rpy="0 0 0" xyz="0 0 0"/>
-              <geometry>
-                <mesh filename="package://aerial_robot_model/urdf/hydrusx/mesh/hydrusx_link4.dae"/>
-              </geometry>
-              <xacro:link_color />
-            </visual>
-            <inertial>
-              <origin xyz="0 0 0" rpy="0 0 0"/>
-              <mass value="0.5"/>
-              <inertia
-	          ixx="0.1" ixy="0.0" ixz="0.0"
-	          iyy="0.01" iyz="0.0"
-	          izz="0.11"/>
-            </inertial>
-          </link>
-        </xacro:if>
-        <xacro:unless value="${imu}">
-          <xacro:if value="${pc}">
-            <link name="link${self}">
-              <collision>
-                <origin xyz="0 0 0" rpy="0 0 0"/>
-                <geometry>
-                  <cylinder length="${protector_radius}" radius="0.1"/>
-                </geometry>
-              </collision>
-              <visual>
-                <origin rpy="0 0 0" xyz="0 0 0"/>
-                <geometry>
-                  <mesh filename="package://aerial_robot_model/urdf/hydrusx/mesh/hydrusx_link3.dae"/>
-                </geometry>
-                <xacro:link_color />
-              </visual>
-              <inertial>
-                <origin xyz="0 0 0" rpy="0 0 0"/>
-                <mass value="0.5"/>
-                <inertia
-	            ixx="0.1" ixy="0.0" ixz="0.0"
-	            iyy="0.01" iyz="0.0"
-	            izz="0.11"/>
-              </inertial>
-            </link>
-          </xacro:if>
-          <xacro:unless value="${pc}">
-            <link name="link${self}">
-              <collision>
-                <origin xyz="0 0 0" rpy="0 0 0"/>
-                <geometry>
-                  <cylinder length="0.1" radius="${protector_radius}"/>
-                </geometry>
-              </collision>
-              <visual>
-                <origin rpy="0 0 0" xyz="0 0 0"/>
-                <geometry>
-                  <mesh filename="package://aerial_robot_model/urdf/hydrusx/mesh/hydrusx_link2.dae"/>
-                </geometry>
-                <xacro:link_color />
-              </visual>
-              <inertial>
-                <origin xyz="0 0 0" rpy="0 0 0"/>
-                <mass value="0.5"/>
-                <inertia
-	            ixx="0.1" ixy="0.0" ixz="0.0"
-	            iyy="0.01" iyz="0.0"
-	            izz="0.11"/>
-              </inertial>
-            </link>
-          </xacro:unless>
-        </xacro:unless>
-        <joint name="joint${self}" type="revolute">
-          <limit effort="100.0" lower="-1.57" upper="1.57" velocity="0.5"/>
-          <parent link="link${self}"/>
-          <child link="joint${self}"/>
-          <origin rpy="0 0 0" xyz="-${link_length*.5} 0 0"/>
-          <axis xyz="0 0 1"/>
-          <dynamics damping="0.7"/>
-        </joint>
-        <link name="joint${self}">
-          <collision>
-            <origin rpy="0 0 0" xyz="0 0 0"/>
-            <geometry>
-              <cylinder length="0.05" radius="0.02"/>
-            </geometry>
-          </collision>
-          <visual>
-            <origin rpy="0 0 0" xyz="0 0 0"/>
-            <geometry>
-              <cylinder length="0.001" radius="0.001"/>
-            </geometry>
-            <material name="color">
-              <color rgba="0.75 .5 .2 1"/>
-            </material>
-          </visual>
-          <inertial>
-            <origin rpy="0 0 0" xyz="0 0 0"/>
-            <mass value="0.1"/>
-            <inertia ixx="0.00005" ixy="0.0" ixz="0.0" iyy="0.00005" iyz="0.0" izz="0.0001"/>
-          </inertial>
-        </link>
-        <joint name="joint${self}_link${child}" type="fixed">
-          <parent link="joint${self}"/>
-          <child link="link${child}"/>
-          <origin rpy="0 0 0" xyz="-${link_length*.5} 0 0"/>
-        </joint>
-      </xacro:unless>
-    </xacro:unless>
+      <actuator name="rotor${self}">
+        <!-- TODO: effort is torque, maybe position is enough -->
+        <hardwareInterface>RotorInterface</hardwareInterface>
+        <mechanicalReduction>1</mechanicalReduction>
+      </actuator>
+    </transmission>
+    <xacro:friction self ="${self}"/>
   </xacro:macro>
 </robot>

Commit message: Setup for the hydrusx series(quad, hex) in the simulation system

File: aerial_robot_model/urdf/hydrusx/hydrusx_common.xacro (robot description, xacro)
@@ -46,7 +46,7 @@
   <xacro:macro name="link_model" params="type">
     <collision>
-      <origin xyz="0 0 0" rpy="${link_length*.5} 0 0"/>
+      <origin rpy="0 0 0" xyz="${link_length*.5} 0 -0.03"/>
       <geometry>
-        <cylinder length="0.10" radius="${protector_radius}"/>
+        <cylinder length="0.15" radius="${protector_radius}"/>
       </geometry>
     </collision>
