Commit message: Update the hydrusx model dscription

File: aerial_robot_model/urdf/hydrusx/hydrusx_common.xacro (robot description, xacro)
@@ -7,44 +7,42 @@
   <xacro:property name="link_rod_length" value=".528" />
   <xacro:property name="protector_radius" value=".1925" />
-  <xacro:property name="link_joint_offset" value="0.3" /> <!-- [m] -->
-  <xacro:property name="rotor_radius" value=".02" /> <!-- [m] -->
-  <xacro:property name="rotor_height" value=".05" /> <!-- [m] -->
-  <xacro:property name="pc_offset" value="0.22" /> <!-- [m] -->
-  <xacro:property name="fc_offset" value="-0.28" /> <!-- [m] -->
-  <xacro:property name="tail_leg_offset" value="0.235" /> <!-- [m] -->
-  <xacro:property name="head_leg_offset" value="-0.247" /> <!-- [m] -->
-  <xacro:property name="sensor_offset" value="-0.215" /> <!-- [m] -->
+  <xacro:property name="link_joint_offset" value="0.3" />
+  <xacro:property name="rotor_radius" value=".02" />
+  <xacro:property name="rotor_height" value=".05" />
+  <xacro:property name="bat_offset" value="0.0" />
+  <xacro:property name="pc_c_offset" value="0.22" />
+  <xacro:property name="pc_v_offset" value="-0.2" />
+  <xacro:property name="pcs_cable_offset" value="0.0" />
+  <xacro:property name="fc_offset" value="-0.26" />
+  <xacro:property name="sensor_c_offset" value="-0.215" />
+  <xacro:property name="sensor_v_offset" value="-0.01" />
+  <xacro:property name="head_leg_offset" value="-0.25" />
+  <xacro:property name="tail_leg_offset" value="0.235" />
   <!-- inertial paramters -->
   <!-- mass [Kg] -->
-  <xacro:property name="link_center_mass" value=".4046" />
+  <xacro:property name="link_rod_mass" value="0.099" />
+  <xacro:property name="link_center_mass" value=".211" />
   <xacro:property name="joint_mass" value=".2075" />
-  <xacro:property name="link_rod_mass" value="0.099" />
   <xacro:property name="protector_mass" value=".05" />
   <xacro:property name="protector_holder_mass" value=".0386" />
+  <xacro:property name="bat_mass" value="0.41" />
   <xacro:property name="fc_mass" value=".03" />
-  <xacro:property name="pc_mass" value=".24" />
-  <xacro:property name="tail_leg_mass" value="0.0623" />
+  <xacro:property name="pc_c_mass" value=".1" />
+  <xacro:property name="pc_v_mass" value=".24" />
+  <xacro:property name="pcs_cable_mass" value=".03" />
   <xacro:property name="head_leg_mass" value="0.0623" />
-  <xacro:property name="sensor_mass" value="0.06" />
+  <xacro:property name="tail_leg_mass" value="0.09" />
+  <xacro:property name="sensor_c_mass" value="0.065" />
+  <xacro:property name="sensor_v_mass" value="0.18" />
   <xacro:property name="rotor_mass" value=".05" /> <!-- exclude from center mass -->
-  <xacro:property name="base_mass" value="${link_rod_mass + link_center_mass + joint_mass + protector_mass + protector_holder_mass - rotor_mass}" /> <!-- exclude from center mass -->
   <!-- inertial [N*m*m] -->
-  <xacro:property name="joint_inertia" value="${joint_mass * link_joint_offset * link_joint_offset}" /> <!-- mass * dist * dist -->
   <xacro:property name="link_rod_inertia" value="${link_rod_mass * link_rod_length * link_rod_length /12}" /> <!-- mass * dist * dist -->
-  <xacro:property name="pc_inertia" value="${pc_mass * pc_offset * pc_offset}" /> <!-- mass * dist * dist -->
-  <xacro:property name="fc_inertia" value="${fc_mass * fc_offset * fc_offset}" /> <!-- mass * dist * dist -->
-  <xacro:property name="sensor_inertia" value="${sensor_mass * sensor_offset * sensor_offset}" /> <!-- mass * dist * dist -->
-  <xacro:property name="head_leg_inertia" value="${head_leg_mass * head_leg_offset * head_leg_offset}" /> <!-- mass * dist * dist -->
-  <xacro:property name="tail_leg_inertia" value="${tail_leg_mass * tail_leg_offset * tail_leg_offset}" /> <!-- mass * dist * dist -->
   <xacro:property name="protector_inertia" value="${protector_mass * protector_radius * protector_radius}" /> <!-- mass * dist * dist -->
   <xacro:property name="protector_holder_inertia" value="${protector_holder_mass * protector_radius * protector_radius}" /> <!-- mass * dist * dist -->
-  <xacro:property name="base_ixx" value="${protector_inertia / 2}" />
-  <xacro:property name="base_iyy" value="${joint_inertia + link_rod_inertia + protector_holder_inertia + protector_inertia /2}" />
-  <xacro:property name="base_izz" value="${joint_inertia + link_rod_inertia + protector_holder_inertia + protector_inertia}" />
   <!-- dynamics -->
   <xacro:property name="max_force" value="18" /> <!-- [N] -->
   <xacro:macro name="link_model" params="type">
     <collision>
-      <origin rpy="0 0 0" xyz="${link_length*.5} 0 -0.03"/>
+      <origin rpy="0 0 0" xyz="0 0 -0.03"/>
       <geometry>
         <cylinder length="0.15" radius="${protector_radius}"/>
@@ -52,5 +50,5 @@
     </collision>
     <visual>
-      <origin rpy="${-pi/2} 0 0" xyz="${link_length*.5} 0 0"/>
+      <origin rpy="${-pi/2} 0 0" xyz="0 0 0"/>
       <geometry>
         <mesh filename="package://aerial_robot_model/urdf/hydrusx/mesh/hydrusx_link${type}.dae"/>
@@ -58,10 +56,21 @@
     </visual>
   </xacro:macro>
-  <xacro:macro name="link_inertial" params="extra_mass extra_ixx extra_iyy extra_izz">
-    <mass value="${base_mass + extra_mass}"/>
+  <xacro:macro name="extra_module" params="name parent mass offset">
+    <joint name="link2${name}" type="fixed">
+      <parent link="link${parent}"/>
+      <child link="${name}"/>
+      <origin rpy="0 0 0" xyz="${offset} 0 0"/>
+      <axis xyz="0 0 1"/>
+    </joint>
+    <link name="${name}">
+      <inertial>
+        <origin xyz="0 0 0" rpy="0 0 0"/>
+        <mass value="${mass}"/>
         <inertia
-            ixx="${base_ixx + extra_ixx}" ixy="0.0" ixz="0.0"
-            iyy="${base_iyy + extra_iyy}" iyz="0.0"
-            izz="${base_izz + extra_izz}"/>
+            ixx="0.00001" ixy="0.0" ixz="0.0"
+            iyy="0.00001" iyz="0.0"
+            izz="0.00002"/>
+      </inertial>
+    </link>
   </xacro:macro>
   <!-- friction -->

File: aerial_robot_model/urdf/hydrusx/hydrusx_link.urdf.xacro (robot description, xacro)
@@ -8,26 +8,26 @@
       <!-- common inertial -->
       <inertial>
-        <origin xyz="${link_length*.5} 0 0" rpy="0 0 0"/>
-        <!-- mass and inertia -->
-        <!-- head -->
-        <xacro:if value="${self == 1}">
-          <xacro:link_inertial extra_mass = "${head_leg_mass}" extra_ixx = "0" extra_iyy = "${head_leg_inertia}" extra_izz = "${head_leg_inertia}" />
-        </xacro:if>
-        <!-- tail -->
-        <xacro:if value="${self == child}">
-          <xacro:link_inertial extra_mass = "${tail_leg_mass}" extra_ixx = "0" extra_iyy = "${tail_leg_inertia}" extra_izz = "${tail_leg_inertia}" />
-        </xacro:if>
-        <!-- fc -->
-        <xacro:if value="${fc}">
-          <xacro:link_inertial extra_mass = "${sensor_mass + fc_mass}" extra_ixx = "0" extra_iyy = "${sensor_inertia + fc_inertia}" extra_izz = "${sensor_inertia + fc_inertia}" />
-        </xacro:if>
-        <!-- pc: -->
-        <xacro:if value="${pc}">
-          <xacro:link_inertial extra_mass = "${pc_mass}" extra_ixx = "0" extra_iyy = "${pc_inertia}" extra_izz = "${pc_inertia}" />
-        </xacro:if>
-        <!-- general -->
-        <xacro:if value="${general}">
-          <xacro:link_inertial extra_mass = "0" extra_ixx = "0" extra_iyy = "0" extra_izz = "0" />
-        </xacro:if>
+        <origin xyz="0 0 0" rpy="0 0 0"/>
+        <mass value="0.0000001"/>
+        <inertia
+            ixx="0.00000001" ixy="0.0" ixz="0.0"
+            iyy="0.00000001" iyz="0.0"
+            izz="0.00000002"/>
+      </inertial>
+    </link>
+    <joint name="link${self}2center" type="fixed">
+      <parent link="link${self}"/>
+      <child link="link${self}_center"/>
+      <origin rpy="0 0 0" xyz="${link_length* 0.5} 0 0"/>
+      <axis xyz="0 0 1"/>
+    </joint>
+    <link name="link${self}_center">
+      <inertial>
+        <origin xyz="0 0 0" rpy="0 0 0"/>
+        <mass value="${link_rod_mass + link_center_mass + protector_mass + protector_holder_mass - rotor_mass}" /> <!-- exclude from center mass -->
+        <inertia
+            ixx="${protector_inertia / 2}" ixy="0.0" ixz="0.0"
+            iyy="${link_rod_inertia + protector_holder_inertia + protector_inertia /2}" iyz="0.0"
+            izz="${link_rod_inertia + protector_holder_inertia + protector_inertia}"/>
       </inertial>
       <!-- sepcial inertia & visual & collision -->
@@ -54,30 +54,10 @@
     </link>
     <xacro:damping_factor link ="link${self}"/>
-    <!-- link center(virtual) -->
-    <!-- not good -->
-    <joint name="center${self}" type="fixed">
-      <parent link="link${self}"/>
-      <child link="link${self}_center"/>
-      <origin rpy="0 0 0" xyz="${link_length*.5} 0 0"/>
-      <axis xyz="0 0 1"/>
-    </joint>
-    <link name="link${self}_center">
-      <!-- visual & collisiont -->
-      <inertial>
-        <origin xyz="0 0 0" rpy="0 0 0"/>
-        <mass value="0.001"/>
-        <inertia
-            ixx="0.00000001" ixy="0.0" ixz="0.0"
-            iyy="0.00000001" iyz="0.0"
-            izz="0.00000002"/>
-      </inertial>
-    </link>
-    <xacro:damping_factor link ="link${self}_center"/>
     <!-- rotor -->
     <joint name="rotor${self}" type="continuous">
       <limit effort="100.0" lower="0" upper="${max_force}" velocity="0.5"/> <!-- force range -->
-      <parent link="link${self}"/>
+      <parent link="link${self}_center"/>
       <child link="propeller${self}"/>
-      <origin rpy="0 0 0" xyz="${link_length*.5} 0 0"/>
+      <origin rpy="0 0 0" xyz="0 0 0"/>
       <axis xyz="0 0 1"/>
     </joint>
@@ -94,4 +74,39 @@
     </link>
     <xacro:damping_factor link ="propeller${self}"/>
+    <!-- extra module -->
+    <!-- head -->
+    <xacro:if value="${self == 1}">
+      <xacro:extra_module name = "head" parent = "${self}" mass = "${head_leg_mass}" offset = "${link_length * 0.5 + head_leg_offset}" />
+      <!-- battery -->
+      <xacro:extra_module name = "bat${self}" parent = "${self}" mass = "${bat_mass}" offset = "${link_length * 0.5 + bat_offset}" />
+    </xacro:if>
+    <!-- tail -->
+    <xacro:if value="${self == child}">
+      <xacro:extra_module name = "tail" parent = "${self}" mass = "${tail_leg_mass}" offset = "${link_length * 0.5 + tail_leg_offset}" />
+      <!-- battery -->
+      <xacro:extra_module name = "bat${self}" parent = "${self}" mass = "${bat_mass}" offset = "${link_length * 0.5 + bat_offset}" />
+    </xacro:if>
+    <!-- fc -->
+    <xacro:if value="${fc}">
+      <xacro:extra_module name = "fc" parent = "${self}" mass = "${fc_mass}" offset = "${link_length * 0.5 + fc_offset}" />
+      <!-- sensor for control -->
+      <xacro:extra_module name = "sensor_c" parent = "${self}" mass = "${sensor_c_mass}" offset = "${link_length * 0.5 + sensor_c_offset}" />
+      <!-- sensor for vision -->
+      <xacro:extra_module name = "sensor_v" parent = "${self}" mass = "${sensor_v_mass}" offset = "${link_length * 0.5 + sensor_v_offset}" />
+    </xacro:if>
+    <!-- pc -->
+    <xacro:if value="${pc}">
+      <!-- control side -->
+      <xacro:extra_module name = "pc_c" parent = "${self}" mass = "${pc_c_mass}" offset = "${link_length * 0.5 + pc_c_offset}" />
+      <!-- visual side -->
+      <xacro:extra_module name = "pc_v" parent = "${self}" mass = "${pc_v_mass}" offset = "${link_length * 0.5 + pc_v_offset}" />
+      <!-- pcs calble -->
+      <xacro:extra_module name = "pcs_cable" parent = "${self}" mass = "${pcs_cable_mass}" offset = "${link_length * 0.5 + pcs_cable_offset}" />
+    </xacro:if>
+    <!-- general -->
+    <xacro:if value="${general}">
+      <!-- battery -->
+      <xacro:extra_module name = "bat${self}" parent = "${self}" mass = "${bat_mass}" offset = "${link_length * 0.5 + bat_offset}" />
+    </xacro:if>
     <!-- joint -->>
     <xacro:unless value="${self == child}">
@@ -104,4 +119,5 @@
         <dynamics damping="0.8" friction="0.05"/>
       </joint>
+      <xacro:extra_module name = "joint${self}_module" parent = "${self}" mass = "${joint_mass}" offset = "${link_length* 0.5 + link_joint_offset}" />
     </xacro:unless>
     <!-- hardware interface -->
