Commit message: Update the hydrus3 model dscription

File: aerial_robot_model/robots/hydrus3/penta.urdf.xacro (robot description, xacro)
@@ -4,5 +4,5 @@
   <xacro:include filename="$(find aerial_robot_model)/urdf/hydrus3/hydrus3_common.xacro" />
   <xacro:include filename="$(find aerial_robot_model)/urdf/hydrus3/hydrus3_link.urdf.xacro" />
-  <xacro:hydrus3_link self="1" child="2" general="false" fc="false" pc="pc"  />
+  <xacro:hydrus3_link self="1" child="2" general="false" fc="false" pc="true"  />
   <xacro:hydrus3_link self="2" child="3" general="true" fc="false" pc="false" />
   <xacro:hydrus3_link self="3" child="4" general="false" fc="true" pc="false" />

File: aerial_robot_model/robots/hydrus3/quad.urdf.xacro (robot description, xacro)
@@ -4,5 +4,5 @@
   <xacro:include filename="$(find aerial_robot_model)/urdf/hydrus3/hydrus3_common.xacro" />
   <xacro:include filename="$(find aerial_robot_model)/urdf/hydrus3/hydrus3_link.urdf.xacro" />
-  <xacro:hydrus3_link self="1" child="2" general="false" fc="false" pc="pc"  />
+  <xacro:hydrus3_link self="1" child="2" general="false" fc="false" pc="true"  />
   <xacro:hydrus3_link self="2" child="3" general="false" fc="true" pc="false" />
   <xacro:hydrus3_link self="3" child="4" general="true" fc="false" pc="false" />

File: aerial_robot_model/urdf/hydrus3/hydrus3_common.xacro (robot description, xacro)
@@ -7,9 +7,9 @@
   <xacro:property name="link_rod_length" value=".4" />
   <xacro:property name="protector_radius" value=".1425" />
-  <xacro:property name="link_joint_offset" value="-0.205" /> <!-- [m] -->
-  <xacro:property name="rotor_radius" value=".015" /> <!-- [m] -->
-  <xacro:property name="rotor_height" value=".05" /> <!-- [m] -->
-  <xacro:property name="pc_offset" value="-0.189" /> <!-- [m] -->
-  <xacro:property name="fc_offset" value="0.166" /> <!-- [m] -->
+  <xacro:property name="link_joint_offset" value="-0.205" />
+  <xacro:property name="rotor_radius" value=".015" />
+  <xacro:property name="rotor_height" value=".05" />
+  <xacro:property name="pc_offset" value="-0.189" /> <!-- from link_cetner -->
+  <xacro:property name="fc_offset" value="0.166" /> <!-- from link_cetner -->
   <!-- inertial parameter -->
   <!-- mass [Kg] -->
@@ -22,20 +22,13 @@
   <xacro:property name="pc_mass" value=".104" />
   <xacro:property name="rotor_mass" value=".05" /> <!-- exclude from center mass -->
-  <xacro:property name="base_mass" value="${link_rod_mass + link_center_mass + joint_mass + protector_mass + protector_holder_mass - rotor_mass}" /> <!-- exclude from center mass -->
   <!-- inertial [N*m*m] -->
-  <xacro:property name="joint_inertia" value="${joint_mass * link_joint_offset * link_joint_offset}" /> <!-- mass * dist * dist -->
   <xacro:property name="link_rod_inertia" value="${link_rod_mass * link_rod_length * link_rod_length /12}" /> <!-- mass * dist * dist -->
-  <xacro:property name="pc_inertia" value="${pc_mass * pc_offset * pc_offset}" /> <!-- mass * dist * dist -->
-  <xacro:property name="fc_inertia" value="${fc_mass * fc_offset * fc_offset}" /> <!-- mass * dist * dist -->
   <xacro:property name="protector_inertia" value="${protector_mass * protector_radius * protector_radius}" /> <!-- mass * dist * dist -->
   <xacro:property name="protector_holder_inertia" value="${protector_holder_mass * protector_radius * protector_radius}" /> <!-- mass * dist * dist -->
-  <xacro:property name="base_ixx" value="${protector_inertia / 2}" />
-  <xacro:property name="base_iyy" value="${joint_inertia + link_rod_inertia + protector_holder_inertia + protector_inertia /2}" />
-  <xacro:property name="base_izz" value="${joint_inertia + link_rod_inertia + protector_holder_inertia + protector_inertia}" />
   <!-- dynamics [N] -->
   <xacro:property name="max_force" value="10" /> <!-- [m] -->
   <xacro:macro name="link_model" params="type">
     <collision>
-      <origin rpy="0 0 0" xyz="${link_length*.5} 0 0"/>
+      <origin rpy="0 0 0" xyz="0 0 0"/>
       <geometry>
         <cylinder length="0.13" radius="${protector_radius}"/>
@@ -43,5 +36,5 @@
     </collision>
     <visual>
-      <origin rpy="${-pi/2} 0 0" xyz="${link_length*.5} 0 0"/>
+      <origin rpy="${-pi/2} 0 0" xyz="0 0 0"/>
       <geometry>
         <mesh filename="package://aerial_robot_model/urdf/hydrus3/mesh/hydrus3_link${type}.dae"/>
@@ -49,10 +42,21 @@
     </visual>
   </xacro:macro>
-  <xacro:macro name="link_inertial" params="extra_mass extra_ixx extra_iyy extra_izz">
-    <mass value="${base_mass + extra_mass}"/>
+  <xacro:macro name="extra_module" params="name parent mass offset">
+    <joint name="link2${name}" type="fixed">
+      <parent link="link${parent}"/>
+      <child link="${name}"/>
+      <origin rpy="0 0 0" xyz="${offset} 0 0"/>
+      <axis xyz="0 0 1"/>
+    </joint>
+    <link name="${name}">
+      <inertial>
+        <origin xyz="0 0 0" rpy="0 0 0"/>
+        <mass value="${mass}"/>
         <inertia
-            ixx="${base_ixx + extra_ixx}" ixy="0.0" ixz="0.0"
-            iyy="${base_iyy + extra_iyy}" iyz="0.0"
-            izz="${base_izz + extra_izz}"/>
+            ixx="0.00001" ixy="0.0" ixz="0.0"
+            iyy="0.00001" iyz="0.0"
+            izz="0.00002"/>
+      </inertial>
+    </link>
   </xacro:macro>
   <!-- friction -->

File: aerial_robot_model/urdf/hydrus3/hydrus3_link.urdf.xacro (robot description, xacro)
@@ -6,25 +6,27 @@
     <!-- link -->
     <link name="link${self}">
-      <!-- common inertial -->
       <inertial>
-        <origin xyz="${link_length*.5} 0 0" rpy="0 0 0"/>
-        <!-- mass and inertia -->
-        <!-- head -->
-        <xacro:if value="${self == 1}">
-          <xacro:link_inertial extra_mass = "${pc_mass}" extra_ixx = "0" extra_iyy = "${pc_inertia}" extra_izz = "${pc_inertia}" />
-        </xacro:if>
-        <!-- tail -->
-        <xacro:if value="${self == child}">
-          <xacro:link_inertial extra_mass = "0" extra_ixx = "0" extra_iyy = "0" extra_izz = "0" />
-        </xacro:if>
-        <!-- fc -->
-        <xacro:if value="${fc}">
-          <xacro:link_inertial extra_mass = "${fc_mass}" extra_ixx = "0" extra_iyy = "${fc_inertia}" extra_izz = "${fc_inertia}" />
-        </xacro:if>
-        <!-- pc: no -->
-        <!-- general -->
-        <xacro:if value="${general}">
-          <xacro:link_inertial extra_mass = "0" extra_ixx = "0" extra_iyy = "0" extra_izz = "0" />
-        </xacro:if>
+        <origin xyz="0 0 0" rpy="0 0 0"/>
+        <mass value="0.0000001"/>
+        <inertia
+            ixx="0.00000001" ixy="0.0" ixz="0.0"
+            iyy="0.00000001" iyz="0.0"
+            izz="0.00000002"/>
+      </inertial>
+    </link>
+    <joint name="link${self}2center" type="fixed">
+      <parent link="link${self}"/>
+      <child link="link${self}_center"/>
+      <origin rpy="0 0 0" xyz="${link_length* 0.5} 0 0"/>
+      <axis xyz="0 0 1"/>
+    </joint>
+    <link name="link${self}_center">
+      <inertial>
+        <origin xyz="0 0 0" rpy="0 0 0"/>
+        <mass value="${link_rod_mass + link_center_mass + protector_mass + protector_holder_mass - rotor_mass}" /> <!-- exclude from center mass -->
+        <inertia
+            ixx="${protector_inertia / 2}" ixy="0.0" ixz="0.0"
+            iyy="${link_rod_inertia + protector_holder_inertia + protector_inertia /2}" iyz="0.0"
+            izz="${link_rod_inertia + protector_holder_inertia + protector_inertia}"/>
       </inertial>
       <!-- sepcial inertia & visual & collision -->
@@ -48,30 +50,10 @@
     </link>
     <xacro:damping_factor link ="link${self}"/>
-    <!-- link center(virtual) -->
-    <!-- not good -->
-    <joint name="center${self}" type="fixed">
-      <parent link="link${self}"/>
-      <child link="link${self}_center"/>
-      <origin rpy="0 0 0" xyz="${link_length*.5} 0 0"/>
-      <axis xyz="0 0 1"/>
-    </joint>
-    <link name="link${self}_center">
-      <!-- visual & collisiont -->
-      <inertial>
-        <origin xyz="0 0 0" rpy="0 0 0"/>
-        <mass value="0.001"/>
-        <inertia
-            ixx="0.00000001" ixy="0.0" ixz="0.0"
-            iyy="0.00000001" iyz="0.0"
-            izz="0.00000002"/>
-      </inertial>
-    </link>
-    <xacro:damping_factor link ="link${self}_center"/>
     <!-- rotor -->
     <joint name="rotor${self}" type="continuous">
       <limit effort="100.0" lower="0" upper="${max_force}" velocity="0.5"/> <!-- force range -->
-      <parent link="link${self}"/>
+      <parent link="link${self}_center"/>
       <child link="propeller${self}"/>
-      <origin rpy="0 0 0" xyz="${link_length*.5} 0 0"/>
+      <origin rpy="0 0 0" xyz="0 0 0"/>
       <axis xyz="0 0 1"/>
     </joint>
@@ -88,5 +70,14 @@
     </link>
     <xacro:damping_factor link ="propeller${self}"/>
-    <!-- joint -->>
+    <!-- extra module -->
+    <!-- pc -->
+    <xacro:if value="${pc}">
+      <xacro:extra_module name = "pc" parent = "${self}" mass = "${pc_mass}" offset = "${link_length* 0.5 + pc_offset}" />
+    </xacro:if>
+    <!-- fc -->
+    <xacro:if value="${fc}">
+      <xacro:extra_module name = "fc" parent = "${self}" mass = "${fc_mass}" offset = "${link_length* 0.5 + fc_offset}" />
+    </xacro:if>
+    <!-- joint -->
     <xacro:unless value="${self == child}">
       <joint name="joint${self}" type="revolute">
@@ -98,4 +89,5 @@
         <dynamics damping="0.8" friction="0.05"/>
       </joint>
+      <xacro:extra_module name = "joint${self}_module" parent = "${child}" mass = "${joint_mass}" offset = "${link_length* 0.5 + link_joint_offset}" /> <!-- special -->
     </xacro:unless>
     <!-- hardware interface -->

Commit message: Modified the robot xacro file and yaml to be suitable for the new rotor direction configuration

File: aerial_robot_model/robots/hydrus3/penta.urdf.xacro (robot description, xacro)
@@ -4,8 +4,8 @@
   <xacro:include filename="$(find aerial_robot_model)/urdf/hydrus3/hydrus3_common.xacro" />
   <xacro:include filename="$(find aerial_robot_model)/urdf/hydrus3/hydrus3_link.urdf.xacro" />
-  <xacro:hydrus3_link self="1" child="2" general="false" fc="false" pc="true"  />
-  <xacro:hydrus3_link self="2" child="3" general="true" fc="false" pc="false" />
-  <xacro:hydrus3_link self="3" child="4" general="false" fc="true" pc="false" />
-  <xacro:hydrus3_link self="4" child="5" general="true" fc="false" pc="false" />
-  <xacro:hydrus3_link self="5" child="5" general="false" fc="false" pc="false" />
+  <xacro:hydrus3_link self="1" child="2" rotor_direction="-1" general="false" fc="false" pc="true"  />
+  <xacro:hydrus3_link self="2" child="3" rotor_direction="1" general="true" fc="false" pc="false" />
+  <xacro:hydrus3_link self="3" child="4" rotor_direction="-1" general="false" fc="true" pc="false" />
+  <xacro:hydrus3_link self="4" child="5" rotor_direction="1" general="true" fc="false" pc="false" />
+  <xacro:hydrus3_link self="5" child="5" rotor_direction="-1" general="false" fc="false" pc="false" />
 </robot>

File: aerial_robot_model/robots/hydrus3/quad.urdf.xacro (robot description, xacro)
@@ -4,7 +4,7 @@
   <xacro:include filename="$(find aerial_robot_model)/urdf/hydrus3/hydrus3_common.xacro" />
   <xacro:include filename="$(find aerial_robot_model)/urdf/hydrus3/hydrus3_link.urdf.xacro" />
-  <xacro:hydrus3_link self="1" child="2" general="false" fc="false" pc="true"  />
-  <xacro:hydrus3_link self="2" child="3" general="false" fc="true" pc="false" />
-  <xacro:hydrus3_link self="3" child="4" general="true" fc="false" pc="false" />
-  <xacro:hydrus3_link self="4" child="4" general="false" fc="false" pc="false" />
+  <xacro:hydrus3_link self="1" child="2" rotor_direction="-1" general="false" fc="false" pc="true"  />
+  <xacro:hydrus3_link self="2" child="3" rotor_direction="1" general="false" fc="true" pc="false" />
+  <xacro:hydrus3_link self="3" child="4" rotor_direction="-1" general="true" fc="false" pc="false" />
+  <xacro:hydrus3_link self="4" child="4" rotor_direction="1" general="false" fc="false" pc="false" />
 </robot>

File: aerial_robot_model/robots/hydrusx/hex.urdf.xacro (robot description, xacro)
@@ -4,9 +4,9 @@
   <xacro:include filename="$(find aerial_robot_model)/urdf/hydrusx/hydrusx_common.xacro" />
   <xacro:include filename="$(find aerial_robot_model)/urdf/hydrusx/hydrusx_link.urdf.xacro" />
-  <xacro:hydrusx_link self="1" child="2" general="false" fc="false" pc="false"/>
-  <xacro:hydrusx_link self="2" child="3" general="true" fc="false" pc="false"/>
-  <xacro:hydrusx_link self="3" child="4" general="false" fc="false" pc="true"/>
-  <xacro:hydrusx_link self="4" child="5" general="false" fc="true" pc="false"/>
-  <xacro:hydrusx_link self="5" child="6" general="true" fc="false" pc="false"/>
-  <xacro:hydrusx_link self="6" child="6" general="false" fc="false" pc="false"/>
+  <xacro:hydrusx_link self="1" child="2" rotor_direction="-1" general="false" fc="false" pc="false"/>
+  <xacro:hydrusx_link self="2" child="3" rotor_direction="1"  general="true"  fc="false" pc="false"/>
+  <xacro:hydrusx_link self="3" child="4" rotor_direction="-1" general="false" fc="false" pc="true"/>
+  <xacro:hydrusx_link self="4" child="5" rotor_direction="1"  general="false" fc="true"  pc="false"/>
+  <xacro:hydrusx_link self="5" child="6" rotor_direction="-1" general="true"  fc="false" pc="false"/>
+  <xacro:hydrusx_link self="6" child="6" rotor_direction="1"  general="false" fc="false" pc="false"/>
 </robot>

File: aerial_robot_model/robots/hydrusx/quad.urdf.xacro (robot description, xacro)
@@ -4,7 +4,7 @@
   <xacro:include filename="$(find aerial_robot_model)/urdf/hydrusx/hydrusx_common.xacro" />
   <xacro:include filename="$(find aerial_robot_model)/urdf/hydrusx/hydrusx_link.urdf.xacro" />
-  <xacro:hydrusx_link self="1" child="2" general="false" fc="false" pc="false"/>
-  <xacro:hydrusx_link self="2" child="3" general="false" fc="false" pc="true"/>
-  <xacro:hydrusx_link self="3" child="4" general="false" fc="true" pc="false"/>
-  <xacro:hydrusx_link self="4" child="4" general="false" fc="false" pc="false"/>
+  <xacro:hydrusx_link self="1" child="2" rotor_direction="-1" general="false" fc="false" pc="false"/>
+  <xacro:hydrusx_link self="2" child="3" rotor_direction="1"  general="false" fc="false" pc="true"/>
+  <xacro:hydrusx_link self="3" child="4" rotor_direction="-1" general="false" fc="true"  pc="false"/>
+  <xacro:hydrusx_link self="4" child="4" rotor_direction="1"  general="false" fc="false" pc="false"/>
 </robot>

File: aerial_robot_model/urdf/hydrus3/hydrus3_link.urdf.xacro (robot description, xacro)
@@ -3,5 +3,5 @@
     xmlns:xacro="http://www.ros.org/wiki/xacro" name="hydrus3_link" >
   <!-- D-H kai description(different from prof.nakamura) -->
-  <xacro:macro name="hydrus3_link" params="self child general fc pc">
+  <xacro:macro name="hydrus3_link" params="self child rotor_direction general fc pc">
     <!-- link -->
     <link name="link${self}">
@@ -41,5 +41,5 @@
       <child link="propeller${self}"/>
       <origin rpy="0 0 0" xyz="${link_length* 0.5} 0 0"/>
-      <axis xyz="0 0 1"/>
+      <axis xyz="0 0 ${rotor_direction}"/>
     </joint>
     <link name="propeller${self}">

File: aerial_robot_model/urdf/hydrusx/hydrusx_link.urdf.xacro (robot description, xacro)
@@ -3,5 +3,5 @@
     xmlns:xacro="http://www.ros.org/wiki/xacro" name="hydrusx_link" >
   <!-- D-H kai description(different from prof.nakamura) -->
-  <xacro:macro name="hydrusx_link" params="self child general fc pc">
+  <xacro:macro name="hydrusx_link" params="self child rotor_direction general fc pc">
     <!-- link -->
     <link name="link${self}">
@@ -44,5 +44,5 @@
       <child link="propeller${self}"/>
       <origin rpy="0 0 0" xyz="${link_length* 0.5} 0 0"/>
-      <axis xyz="0 0 1"/>
+      <axis xyz="0 0 ${rotor_direction}"/>
     </joint>
     <link name="propeller${self}">
