Commit message: Update model: 1. Add stl model for dragon, which is lighter than dae file 2. Fix the wrong origin position of ducted_fan_gimbal_pitch 3. Update the collision model for each module 4. Update the max force for dragon model 5. Update the friction paramter for the each type of joint

File: aerial_robot_model/urdf/dragon/dragon_common.xacro (robot description, xacro)
@@ -13,16 +13,16 @@
   <xacro:property name="gimbal_pitch_z_offset" value="0.037" />
   <!-- dynamics -->
-  <xacro:property name="max_force" value="18" /> <!-- [N] -->
+  <xacro:property name="max_force" value="30" /> <!-- [N] -->
   <xacro:macro name="link_model" params="type">
     <collision>
-      <origin rpy="0 ${pi/2} 0" xyz="${link_length* 0.5} 0 0"/>
+      <origin rpy="0 0 0" xyz="${link_length* 0.5} 0 0"/>
       <geometry>
-        <cylinder length="${link_length}" radius="0.2"/>
+        <box size="0.05 0.05 0.1686"/>
       </geometry>
     </collision>
     <visual>
-      <origin rpy="${-pi/2} 0 0" xyz="${link_length* 0.5} 0 0"/>
+      <origin rpy="0 0 0" xyz="${link_length* 0.5} 0 0"/>
       <geometry>
-        <mesh filename="package://aerial_robot_model/urdf/dragon/mesh/ducted_fan_${type}.dae"/>
+        <mesh filename="package://aerial_robot_model/urdf/dragon/mesh/ducted_fan_${type}.stl" scale="0.001 0.001 0.001"/>
       </geometry>
     </visual>
@@ -31,6 +31,7 @@
   <xacro:macro name="friction" params="self">
     <gazebo reference="link${self}">
-      <mu1>0.0001</mu1>
-      <mu2>0.0001</mu2>
+      <mu1>0.2</mu1>
+      <mu2>0.2</mu2>
+      <material>Gazebo/Black</material>
     </gazebo>
   </xacro:macro>

File: aerial_robot_model/urdf/dragon/dragon_link.urdf.xacro (robot description, xacro)
@@ -63,8 +63,7 @@
       <origin rpy="0 0 0" xyz="${link_length/2} 0 0"/>
       <axis xyz="1 0 0"/>
-      <dynamics damping="0.8" friction="0.05"/>
+      <dynamics damping="0.1" friction="0.0"/>
     </joint>
     <link name="gimbal${self}_roll_module">
-      <!-- common inertial -->
       <inertial>
         <origin xyz="${gimbal_roll_x_offset - 17.20968 * 0.001} ${0.41439 * 0.001} ${15.61551 * 0.001}" rpy="0 0 0"/>
@@ -74,17 +73,14 @@
             ixy="0" ixz="-0.0002" iyz="0.0"/>
       </inertial>
-      <collision>
+      <visual>
         <origin xyz="${gimbal_roll_x_offset} 0 0" rpy="0 0 0"/>
         <geometry>
-          <cylinder length="150" radius="0.05"/>
-        </geometry>
-      </collision>
-      <visual>
-        <origin xyz="${gimbal_roll_x_offset} 0 0" rpy="${-pi/2} 0 0"/>
-        <geometry>
-          <mesh filename="package://aerial_robot_model/urdf/dragon/mesh/ducted_fan_gimbal_roll.dae"/>
+          <mesh filename="package://aerial_robot_model/urdf/dragon/mesh/ducted_fan_gimbal_roll.stl" scale="0.001 0.001 0.001"/>
         </geometry>
       </visual>
     </link>
+    <gazebo reference="gimbal${self}_roll_module">
+      <material>Gazebo/Red</material>
+    </gazebo>
     <!-- gimbal pitch -->
     <joint name="gimbal${self}_pitch" type="revolute">
@@ -94,10 +90,9 @@
       <origin rpy="0 0 0" xyz="0 0 ${gimbal_pitch_z_offset}"/>
       <axis xyz="0 1 0"/>
-      <dynamics damping="0.8" friction="0.05"/>
+      <dynamics damping="0.1" friction="0.0"/>
     </joint>
     <link name="gimbal${self}_pitch_module">
-      <!-- common inertial -->
       <inertial>
-        <origin xyz="0 0.47 -7.38" rpy="0 0 0"/>
+        <origin xyz="0 ${0.47 * 0.001}  ${-7.38 * 0.001}" rpy="0 0 0"/>
         <mass value=".4187" />
         <inertia
@@ -105,20 +100,17 @@
             ixy="0" ixz="0.0" iyz="0.0"/>
       </inertial>
-      <collision>
-        <origin xyz="0 0 0" rpy="${pi/2} 0 0"/>
+      <visual>
+        <origin xyz="0 0 0" rpy="0 0 0"/>
         <geometry>
-          <cylinder length="0.3" radius="0.05"/>
-        </geometry>
-      </collision>
-      <visual>
-        <origin xyz="0 0 0" rpy="${-pi/2} 0 0"/>
-        <geometry>
-          <mesh filename="package://aerial_robot_model/urdf/dragon/mesh/ducted_fan_gimbal_pitch.dae"/>
+          <mesh filename="package://aerial_robot_model/urdf/dragon/mesh/ducted_fan_gimbal_pitch.stl" scale="0.001 0.001 0.001"/>
         </geometry>
       </visual>
     </link>
+    <gazebo reference="gimbal${self}_pitch_module">
+      <material>Gazebo/Black</material>
+    </gazebo>
     <!-- rotor -->
     <joint name="rotor${self}" type="continuous">
-      <limit effort="100.0" lower="0" upper="${max_force}" velocity="0.5"/> <!-- force range -->
+      <limit effort="100.0" lower="0" upper="${max_force}" velocity="0.5"/>
       <parent link="gimbal${self}_pitch_module"/>
       <child link="propeller${self}"/>
@@ -128,14 +120,14 @@
     <link name="propeller${self}">
       <inertial>
-        <origin xyz="0 0 0" rpy="0 0 0"/>
-        <mass value="0.000001"/>
+        <origin xyz="0 0 0.1" rpy="0 0 0"/>
+        <mass value="0.0001"/>
         <inertia
-            ixx="0.000001" ixy="0.0" ixz="0.0"
-            iyy="0.000001" iyz="0.0"
-            izz="0.000002"/>
+            ixx="0.00001" ixy="0.0" ixz="0.0"
+            iyy="0.00001" iyz="0.0"
+            izz="0.00002"/>
       </inertial>
     </link>
     <xacro:damping_factor link ="propeller${self}"/>
-    <!-- joint -->>
+    <!-- joint -->
     <xacro:unless value="${self == child}">
       <joint name="joint${self}_pitch" type="revolute">
@@ -158,13 +150,13 @@
         </inertial>
         <collision>
-          <origin rpy="0 0 0" xyz="${inter_joint_x_offset} 0 0"/>
+          <origin rpy="0 0 0" xyz="${2 * inter_joint_x_offset} 0 0"/>
           <geometry>
-            <cylinder length="0.15" radius="0.15"/>
+            <cylinder length="0.1686" radius="0.011"/>
           </geometry>
         </collision>
         <visual>
-          <origin rpy="${-pi/2} 0 0" xyz="${inter_joint_x_offset} 0 0"/>
+          <origin rpy="0 0 0" xyz="${inter_joint_x_offset} 0 0"/>
           <geometry>
-            <mesh filename="package://aerial_robot_model/urdf/dragon/mesh/inter_joint_junction.dae"/>
+            <mesh filename="package://aerial_robot_model/urdf/dragon/mesh/inter_joint_junction.stl" scale="0.001 0.001 0.001"/>
           </geometry>
         </visual>
@@ -178,4 +170,9 @@
         <dynamics damping="0.8" friction="0.05"/>
       </joint>
+      <gazebo reference="inter_joint${self}">
+        <mu1>0.2</mu1>
+        <mu2>0.2</mu2>
+        <material>Gazebo/Red</material>
+      </gazebo>
     </xacro:unless>
     <xacro:if value="${self == 1}">
@@ -200,11 +197,23 @@
     <!-- hardware interface -->
     <xacro:unless value="${self == child}">
-      <transmission name="joint_tran${self}">
+      <transmission name="joint${self}_pitch_tran">
         <type>transmission_interface/SimpleTransmission</type>
-        <joint name="joint${self}">
+        <joint name="joint${self}_pitch">
           <!-- TODO: effort is torque, maybe position is enough -->
           <hardwareInterface>hardware_interface/EffortJointInterface</hardwareInterface>
         </joint>
-        <actuator name="servo{self}">
+        <actuator name="joint_servo{self}_pitch">
+          <!-- TODO: effort is torque, maybe position is enough -->
+          <hardwareInterface>hardware_interface/EffortJointInterface</hardwareInterface>
+          <mechanicalReduction>1</mechanicalReduction>
+        </actuator>
+      </transmission>
+      <transmission name="joint${self}_yaw_tran">
+        <type>transmission_interface/SimpleTransmission</type>
+        <joint name="joint${self}_yaw">
+          <!-- TODO: effort is torque, maybe position is enough -->
+          <hardwareInterface>hardware_interface/EffortJointInterface</hardwareInterface>
+        </joint>
+        <actuator name="joint_servo{self}_yaw">
           <!-- TODO: effort is torque, maybe position is enough -->
           <hardwareInterface>hardware_interface/EffortJointInterface</hardwareInterface>
@@ -213,16 +222,34 @@
       </transmission>
     </xacro:unless>
-    <transmission name="rotor_tran${self}">
+    <transmission name="gimbal${self}_roll_tran">
+      <type>transmission_interface/SimpleTransmission</type>
+      <joint name="gimbal${self}_roll">
+        <hardwareInterface>hardware_interface/EffortJointInterface</hardwareInterface>
+      </joint>
+      <actuator name="gimbal_servo{self}_roll">
+        <hardwareInterface>hardware_interface/EffortJointInterface</hardwareInterface>
+        <mechanicalReduction>1</mechanicalReduction>
+      </actuator>
+    </transmission>
+    <transmission name="gimbal${self}_pitch_tran">
+      <type>transmission_interface/SimpleTransmission</type>
+      <joint name="gimbal${self}_pitch">
+        <hardwareInterface>hardware_interface/EffortJointInterface</hardwareInterface>
+      </joint>
+      <actuator name="gimbal_servo{self}_pitch">
+        <hardwareInterface>hardware_interface/EffortJointInterface</hardwareInterface>
+        <mechanicalReduction>1</mechanicalReduction>
+      </actuator>
+    </transmission>
+    <transmission name="rotor${self}_tran">
       <type>transmission_interface/SimpleTransmission</type>
       <joint name="rotor${self}">
-        <!-- TODO: effort is torque, maybe position is enough -->
         <hardwareInterface>RotorInterface</hardwareInterface>
       </joint>
       <actuator name="rotor${self}">
-        <!-- TODO: effort is torque, maybe position is enough -->
         <hardwareInterface>RotorInterface</hardwareInterface>
         <mechanicalReduction>1</mechanicalReduction>
       </actuator>
-    </transmission>
+      </transmission>
     <xacro:friction self ="${self}"/>
   </xacro:macro>

Commit message: Add color for stl model in rviz

File: aerial_robot_model/urdf/dragon/dragon_common.xacro (robot description, xacro)
@@ -12,4 +12,11 @@
   <xacro:property name="gimbal_roll_x_offset" value="-0.01" />
   <xacro:property name="gimbal_pitch_z_offset" value="0.037" />
+  <!-- material color for rviz -->
+  <material name="black">
+    <color rgba="0 0 0 1"/>
+  </material>
+  <material name="red">
+    <color rgba="1 0 0 1"/>
+  </material>
   <!-- dynamics -->
   <xacro:property name="max_force" value="30" /> <!-- [N] -->
@@ -26,4 +33,5 @@
         <mesh filename="package://aerial_robot_model/urdf/dragon/mesh/ducted_fan_${type}.stl" scale="0.001 0.001 0.001"/>
       </geometry>
+      <material name="black"/>
     </visual>
   </xacro:macro>

File: aerial_robot_model/urdf/dragon/dragon_link.urdf.xacro (robot description, xacro)
@@ -77,4 +77,5 @@
         <geometry>
           <mesh filename="package://aerial_robot_model/urdf/dragon/mesh/ducted_fan_gimbal_roll.stl" scale="0.001 0.001 0.001"/>
+          <material name="red"/>
         </geometry>
       </visual>
@@ -105,4 +106,5 @@
           <mesh filename="package://aerial_robot_model/urdf/dragon/mesh/ducted_fan_gimbal_pitch.stl" scale="0.001 0.001 0.001"/>
         </geometry>
+        <material name="black"/>
       </visual>
     </link>
@@ -160,4 +162,5 @@
             <mesh filename="package://aerial_robot_model/urdf/dragon/mesh/inter_joint_junction.stl" scale="0.001 0.001 0.001"/>
           </geometry>
+          <material name="red"/>
         </visual>
       </link>
