Commit message: Update the package, especially for the robot model

File: robots/dragon/robots/quad.gazebo.xacro (robot description, xacro)
@@ -2,5 +2,5 @@
 <robot
     xmlns:xacro="http://www.ros.org/wiki/xacro" name="dragon" >
-  <xacro:include filename="$(find aerial_robot_model)/robots/dragon/quad.urdf.xacro" />
+  <xacro:include filename="$(find dragon)/robots/quad.urdf.xacro" />
   <!-- gazebo elements: hw interface -->
   <gazebo>

File: robots/dragon/robots/quad.urdf.xacro (robot description, xacro)
@@ -2,6 +2,6 @@
 <robot
     xmlns:xacro="http://www.ros.org/wiki/xacro" name="dragon" >
-  <xacro:include filename="$(find aerial_robot_model)/urdf/dragon/dragon_common.xacro" />
-  <xacro:include filename="$(find aerial_robot_model)/urdf/dragon/dragon_link.urdf.xacro" />
+  <xacro:include filename="$(find dragon)/urdf/dragon_common.xacro" />
+  <xacro:include filename="$(find dragon)/urdf/dragon_link.urdf.xacro" />
   <xacro:dragon_module self="1" child="2" baselink="false" />
   <xacro:dragon_module self="2" child="3" baselink="true" />

File: robots/dragon/urdf/dragon_common.xacro (robot description, xacro)
@@ -31,5 +31,5 @@
       <origin rpy="0 0 0" xyz="${link_length* 0.5} 0 0"/>
       <geometry>
-        <mesh filename="package://aerial_robot_model/urdf/dragon/mesh/ducted_fan_${type}.stl" scale="0.001 0.001 0.001"/>
+        <mesh filename="package://dragon/urdf/mesh/ducted_fan_${type}.stl" scale="0.001 0.001 0.001"/>
       </geometry>
       <material name="black"/>

File: robots/dragon/urdf/dragon_link.urdf.xacro (robot description, xacro)
@@ -76,5 +76,5 @@
         <origin xyz="${gimbal_roll_x_offset} 0 0" rpy="0 0 0"/>
         <geometry>
-          <mesh filename="package://aerial_robot_model/urdf/dragon/mesh/ducted_fan_gimbal_roll.stl" scale="0.001 0.001 0.001"/>
+          <mesh filename="package://dragon/urdf/mesh/ducted_fan_gimbal_roll.stl" scale="0.001 0.001 0.001"/>
           <material name="red"/>
         </geometry>
@@ -104,5 +104,5 @@
         <origin xyz="0 0 0" rpy="0 0 0"/>
         <geometry>
-          <mesh filename="package://aerial_robot_model/urdf/dragon/mesh/ducted_fan_gimbal_pitch.stl" scale="0.001 0.001 0.001"/>
+          <mesh filename="package://dragon/urdf/mesh/ducted_fan_gimbal_pitch.stl" scale="0.001 0.001 0.001"/>
         </geometry>
         <material name="black"/>
@@ -160,5 +160,5 @@
           <origin rpy="0 0 0" xyz="${inter_joint_x_offset} 0 0"/>
           <geometry>
-            <mesh filename="package://aerial_robot_model/urdf/dragon/mesh/inter_joint_junction.stl" scale="0.001 0.001 0.001"/>
+            <mesh filename="package://dragon/urdf/mesh/inter_joint_junction.stl" scale="0.001 0.001 0.001"/>
           </geometry>
           <material name="red"/>
