Commit message: Change the name of thrust point from "propeller"

File: robots/hydrus/urdf/hydrus3/hydrus3_link.urdf.xacro (robot description, xacro)
@@ -39,9 +39,9 @@
       <limit effort="100.0" lower="0" upper="${max_force}" velocity="0.5"/> <!-- force range -->
       <parent link="link${self}"/>
-      <child link="propeller${self}"/>
+      <child link="thrust${self}"/>
       <origin rpy="0 0 0" xyz="${link_length* 0.5} 0 0"/>
       <axis xyz="0 0 ${rotor_direction}"/>
     </joint>
-    <link name="propeller${self}">
+    <link name="thrust${self}">
       <!-- visual & collisiont -->
       <inertial>
@@ -54,5 +54,5 @@
       </inertial>
     </link>
-    <xacro:damping_factor link ="propeller${self}"/>
+    <xacro:damping_factor link ="thrust${self}"/>
     <!-- extra module -->
     <!-- head -->

File: robots/hydrus/urdf/hydrusx/hydrusx_link.urdf.xacro (robot description, xacro)
@@ -42,9 +42,9 @@
       <limit effort="100.0" lower="0" upper="${max_force}" velocity="0.5"/> <!-- force range -->
       <parent link="link${self}"/>
-      <child link="propeller${self}"/>
+      <child link="thrust${self}"/>
       <origin rpy="0 0 0" xyz="${link_length* 0.5} 0 0"/>
       <axis xyz="0 0 ${rotor_direction}"/>
     </joint>
-    <link name="propeller${self}">
+    <link name="thrust${self}">
       <!-- visual & collisiont -->
       <inertial>
@@ -63,5 +63,5 @@
         </collision>
     </link>
-    <xacro:damping_factor link ="propeller${self}"/>
+    <xacro:damping_factor link ="thrust${self}"/>
     <!-- extra module -->
     <!-- head -->
