Commit message: update the hydrusx model based on intel euclid

File: robots/hydrus/robots/hydrusx/quad.urdf.xacro (robot description, xacro)
@@ -5,5 +5,5 @@
   <xacro:include filename="$(find hydrus)/urdf/hydrusx/hydrusx_link.urdf.xacro" />
   <xacro:hydrusx_link self="1" child="2" rotor_direction="-1" general="false" fc="false" pc="false"/>
-  <xacro:hydrusx_link self="2" child="3" rotor_direction="1"  general="false" fc="false" pc="true"/>
+  <xacro:hydrusx_link self="2" child="3" rotor_direction="1"  general="true" fc="false" pc="false"/>
   <xacro:hydrusx_link self="3" child="4" rotor_direction="-1" general="false" fc="true"  pc="false"/>
   <xacro:hydrusx_link self="4" child="4" rotor_direction="1"  general="false" fc="false" pc="false"/>

File: robots/hydrus/urdf/hydrusx/hydrusx_common.xacro (robot description, xacro)
@@ -11,6 +11,6 @@
   <xacro:property name="rotor_height" value=".05" />
   <xacro:property name="bat_offset" value="0.0" />
-  <xacro:property name="pc_c_offset" value="0.22" />
-  <xacro:property name="pc_v_offset" value="-0.2" />
+  <xacro:property name="pc_c_offset" value="0.0" />  <!-- odroid u4: 0.22, euclid: 0 -->
+  <xacro:property name="pc_v_offset" value="0.2" />  <!-- odroid u4: -0.2, euclid: 0.2 -->
   <xacro:property name="pcs_cable_offset" value="0.0" />
   <xacro:property name="fc_offset" value="-0.26" />
@@ -26,7 +26,7 @@
   <xacro:property name="protector_mass" value=".05" />
   <xacro:property name="protector_holder_mass" value=".0386" />
-  <xacro:property name="bat_mass" value="0.41" />
+  <xacro:property name="bat_mass" value="0.364" /> <!-- hyperon: 0.41, white: 0.364 -->
   <xacro:property name="fc_mass" value=".03" />
-  <xacro:property name="pc_c_mass" value=".1" />
+  <xacro:property name="pc_c_mass" value=".13" /> <!-- odoroid u4: 0.1, euclid: 0.13 -->
   <xacro:property name="pc_v_mass" value=".24" />
   <xacro:property name="pcs_cable_mass" value=".03" />

File: robots/hydrus/urdf/hydrusx/hydrusx_link.urdf.xacro (robot description, xacro)
@@ -93,15 +93,6 @@
       <!-- sensor for control -->
       <xacro:extra_module name = "sensor_c" parent = "${self}" mass = "${sensor_c_mass}" offset = "${link_length * 0.5 + sensor_c_offset}" />
-      <!-- sensor for vision -->
-      <xacro:extra_module name = "sensor_v" parent = "${self}" mass = "${sensor_v_mass}" offset = "${link_length * 0.5 + sensor_v_offset}" />
-    </xacro:if>
-    <!-- pc -->
-    <xacro:if value="${pc}">
       <!-- control side -->
       <xacro:extra_module name = "pc_c" parent = "${self}" mass = "${pc_c_mass}" offset = "${link_length * 0.5 + pc_c_offset}" />
-      <!-- visual side -->
-      <xacro:extra_module name = "pc_v" parent = "${self}" mass = "${pc_v_mass}" offset = "${link_length * 0.5 + pc_v_offset}" />
-      <!-- pcs calble -->
-      <xacro:extra_module name = "pcs_cable" parent = "${self}" mass = "${pcs_cable_mass}" offset = "${link_length * 0.5 + pcs_cable_offset}" />
     </xacro:if>
     <!-- general -->

Commit message: Update the model of hydrusx quad type for IJRR2017.

File: robots/hydrus/robots/hydrusx/quad.urdf.xacro (robot description, xacro)
@@ -5,5 +5,5 @@
   <xacro:include filename="$(find hydrus)/urdf/hydrusx/hydrusx_link.urdf.xacro" />
   <xacro:hydrusx_link self="1" child="2" rotor_direction="-1" general="false" fc="false" pc="false"/>
-  <xacro:hydrusx_link self="2" child="3" rotor_direction="1"  general="true" fc="false" pc="false"/>
+  <xacro:hydrusx_link self="2" child="3" rotor_direction="1"  general="false" fc="false" pc="true"/>
   <xacro:hydrusx_link self="3" child="4" rotor_direction="-1" general="false" fc="true"  pc="false"/>
   <xacro:hydrusx_link self="4" child="4" rotor_direction="1"  general="false" fc="false" pc="false"/>

File: robots/hydrus/urdf/hydrusx/hydrusx_common.xacro (robot description, xacro)
@@ -11,5 +11,5 @@
   <xacro:property name="rotor_height" value=".05" />
   <xacro:property name="bat_offset" value="0.0" />
-  <xacro:property name="pc_c_offset" value="0.0" />  <!-- odroid u4: 0.22, euclid: 0 -->
+  <xacro:property name="pc_c_offset" value="0.22" />  <!-- odroid u4: 0.22, euclid: 0 -->
   <xacro:property name="pc_v_offset" value="0.2" />  <!-- odroid u4: -0.2, euclid: 0.2 -->
   <xacro:property name="pcs_cable_offset" value="0.0" />
@@ -26,7 +26,7 @@
   <xacro:property name="protector_mass" value=".05" />
   <xacro:property name="protector_holder_mass" value=".0386" />
-  <xacro:property name="bat_mass" value="0.364" /> <!-- hyperon: 0.41, white: 0.364 -->
+  <xacro:property name="bat_mass" value="0.193" /> <!-- hyperon: 0.41, white(2700mAh): 0.364, white(1300mAh): 0.193 -->
   <xacro:property name="fc_mass" value=".03" />
-  <xacro:property name="pc_c_mass" value=".13" /> <!-- odoroid u4: 0.1, euclid: 0.13 -->
+  <xacro:property name="pc_c_mass" value=".14" /> <!-- odoroid u4: 0.1, euclid: 0.13 -->
   <xacro:property name="pc_v_mass" value=".24" />
   <xacro:property name="pcs_cable_mass" value=".03" />

File: robots/hydrus/urdf/hydrusx/hydrusx_link.urdf.xacro (robot description, xacro)
@@ -100,5 +100,15 @@
       <xacro:extra_module name = "sensor_c" parent = "${self}" mass = "${sensor_c_mass}" offset = "${link_length * 0.5 + sensor_c_offset}" />
       <!-- control side -->
+      <!--
       <xacro:extra_module name = "pc_c" parent = "${self}" mass = "${pc_c_mass}" offset = "${link_length * 0.5 + pc_c_offset}" />
+      -->
+      <!-- battery -->
+      <xacro:extra_module name = "bat${self}" parent = "${self}" mass = "${bat_mass}" offset = "${link_length * 0.5 + bat_offset}" />
+    </xacro:if>
+    <!-- pc -->
+    <xacro:if value="${pc}">
+      <xacro:extra_module name = "pc_c" parent = "${self}" mass = "${pc_c_mass}" offset = "${link_length * 0.5 + pc_c_offset}" />
+      <!-- battery -->
+      <xacro:extra_module name = "bat${self}" parent = "${self}" mass = "${bat_mass}" offset = "${link_length * 0.5 + bat_offset}" />
     </xacro:if>
     <!-- general -->
