Commit message: Add simulated sensor plugins in hydrusx quad type for the egomotion estimation in gazebo

File: robots/hydrus/robots/hydrusx/quad.gazebo.xacro (robot description, xacro)
@@ -11,3 +11,34 @@
     </plugin>
   </gazebo>
+  <!-- sensor plugins -->
+  <!-- 1. imu -->
+  <gazebo reference="fc">
+    <gravity>true</gravity>
+    <sensor name="imu_sensor" type="imu">
+      <always_on>true</always_on>
+      <update_rate>200</update_rate>
+      <visualize>true</visualize>
+      <topic>imu_test</topic>
+      <plugin filename="libgazebo_ros_imu_sensor.so" name="imu_plugin">
+        <topicName>imu</topicName>
+        <bodyName>imu_link</bodyName>
+        <updateRateHZ>200.0</updateRateHZ>
+        <gaussianNoise>0.001</gaussianNoise>
+        <xyzOffset>0 0 0</xyzOffset>
+        <rpyOffset>0 0 0</rpyOffset>
+        <frameName>imu_link</frameName>
+      </plugin>
+      <pose>0 0 0 0 0 0</pose>
+    </sensor>
+  </gazebo>
+  <!-- 2. one point laser sensor: leddarone -->
+  <xacro:include filename="$(find hector_sensors_description)/urdf/sonar_sensor.urdf.xacro" />
+  <xacro:sonar_sensor name="leddarone" parent="link3" ros_topic="leddarone_temp" update_rate="30" min_range="0.05" max_range="20.0" field_of_view="0" ray_count="1">
+    <origin xyz="0.073 0.03 -0.02" rpy="0 ${90*pi/180} 0"/>  <!-- y is for the avoidance of ray with the parent link collision model -->
+  </xacro:sonar_sensor>
+  <!-- 3. downward camera -->
+<xacro:include filename="$(find hector_sensors_description)/urdf/generic_camera.urdf.xacro" />
+  <xacro:generic_camera name="downwards_cam" parent="link3" ros_topic="/camera/image" cam_info_topic="/camera/camera_info" update_rate="30" res_x="640" res_y="480" image_format="R8G8B8" hfov="54">
+    <origin xyz="0.1 0.0 -0.05" rpy="0 ${90*pi/180} 0"/>
+  </xacro:generic_camera>
 </robot>

File: robots/hydrus/urdf/hydrusx/hydrusx_common.xacro (robot description, xacro)
@@ -57,9 +57,9 @@
     </visual>
   </xacro:macro>
-  <xacro:macro name="extra_module" params="name parent mass offset">
+  <xacro:macro name="extra_module" params="name *origin parent mass">
     <joint name="link2${name}" type="fixed">
+      <xacro:insert_block name="origin" />
       <parent link="link${parent}"/>
       <child link="${name}"/>
-      <origin rpy="0 0 0" xyz="${offset} 0 0"/>
       <axis xyz="0 0 1"/>
     </joint>
@@ -81,4 +81,8 @@
       <mu2>0.1</mu2>
     </gazebo>
+    <gazebo reference="rotor{self}">
+      <mu1>0.1</mu1>
+      <mu2>0.1</mu2>
+    </gazebo>
   </xacro:macro>
   <xacro:macro name="damping_factor" params="link">

File: robots/hydrus/urdf/hydrusx/hydrusx_link.urdf.xacro (robot description, xacro)
@@ -84,36 +84,52 @@
         <axis xyz="0 0 1"/>
       </joint>
-      <xacro:extra_module name = "head" parent = "${self}" mass = "${head_leg_mass}" offset = "${link_length * 0.5 + head_leg_offset}" />
+      <xacro:extra_module name = "head" parent = "${self}" mass = "${head_leg_mass}" >
+        <origin xyz="${link_length * 0.5 + head_leg_offset} 0.0 0.0" rpy="0 0 0"/>
+      </xacro:extra_module>
       <!-- battery -->
-      <xacro:extra_module name = "bat${self}" parent = "${self}" mass = "${bat_mass}" offset = "${link_length * 0.5 + bat_offset}" />
+      <xacro:extra_module name = "bat${self}" parent = "${self}" mass = "${bat_mass}" >
+        <origin xyz="${link_length * 0.5 + bat_offset} 0.0 0.0" rpy="0 0 0"/>
+      </xacro:extra_module>
     </xacro:if>
     <!-- tail -->
     <xacro:if value="${self == child}">
-      <xacro:extra_module name = "tail" parent = "${self}" mass = "${tail_leg_mass}" offset = "${link_length * 0.5 + tail_leg_offset}" />
+      <xacro:extra_module name = "tail" parent = "${self}" mass = "${tail_leg_mass}" >
+        <origin xyz="${link_length * 0.5 + tail_leg_offset} 0.0 0.0" rpy="0 0 0"/>
+      </xacro:extra_module>
       <!-- battery -->
-      <xacro:extra_module name = "bat${self}" parent = "${self}" mass = "${bat_mass}" offset = "${link_length * 0.5 + bat_offset}" />
+      <xacro:extra_module name = "bat${self}" parent = "${self}" mass = "${bat_mass}" >
+        <origin xyz="${link_length * 0.5 + bat_offset} 0.0 0.0" rpy="0 0 0"/>
+      </xacro:extra_module>
     </xacro:if>
     <!-- fc -->
     <xacro:if value="${fc}">
-      <xacro:extra_module name = "fc" parent = "${self}" mass = "${fc_mass}" offset = "${link_length * 0.5 + fc_offset}" />
+      <xacro:extra_module name = "fc" parent = "${self}" mass = "${fc_mass}" >
+        <origin xyz="${link_length * 0.5 + fc_offset} 0.0 0.035" rpy="0 0 0"/>
+      </xacro:extra_module>
       <!-- sensor for control -->
-      <xacro:extra_module name = "sensor_c" parent = "${self}" mass = "${sensor_c_mass}" offset = "${link_length * 0.5 + sensor_c_offset}" />
-      <!-- control side -->
-      <!--
-      <xacro:extra_module name = "pc_c" parent = "${self}" mass = "${pc_c_mass}" offset = "${link_length * 0.5 + pc_c_offset}" />
-      -->
+      <xacro:extra_module name = "sensor_c" parent = "${self}" mass = "${sensor_c_mass}" >
+        <origin xyz="${link_length * 0.5 + sensor_c_offset} 0.0 0.0" rpy="0 0 0"/>
+      </xacro:extra_module>
       <!-- battery -->
-      <xacro:extra_module name = "bat${self}" parent = "${self}" mass = "${bat_mass}" offset = "${link_length * 0.5 + bat_offset}" />
+      <xacro:extra_module name = "bat${self}" parent = "${self}" mass = "${bat_mass}" >
+        <origin xyz="${link_length * 0.5 + bat_offset} 0.0 0.0" rpy="0 0 0"/>
+      </xacro:extra_module>
     </xacro:if>
     <!-- pc -->
     <xacro:if value="${pc}">
-      <xacro:extra_module name = "pc_c" parent = "${self}" mass = "${pc_c_mass}" offset = "${link_length * 0.5 + pc_c_offset}" />
+      <xacro:extra_module name = "pc_c" parent = "${self}" mass = "${pc_c_mass}" >
+        <origin xyz="${link_length * 0.5 + pc_c_offset} 0.0 0.0" rpy="0 0 0"/>
+      </xacro:extra_module>
       <!-- battery -->
-      <xacro:extra_module name = "bat${self}" parent = "${self}" mass = "${bat_mass}" offset = "${link_length * 0.5 + bat_offset}" />
+      <xacro:extra_module name = "bat${self}" parent = "${self}" mass = "${bat_mass}" >
+        <origin xyz="${link_length * 0.5 + bat_offset} 0.0 0.0" rpy="0 0 0"/>
+      </xacro:extra_module>
     </xacro:if>
     <!-- general -->
     <xacro:if value="${general}">
       <!-- battery -->
-      <xacro:extra_module name = "bat${self}" parent = "${self}" mass = "${bat_mass}" offset = "${link_length * 0.5 + bat_offset}" />
+      <xacro:extra_module name = "bat${self}" parent = "${self}" mass = "${bat_mass}" >
+        <origin xyz="${link_length * 0.5 + bat_offset} 0.0 0.0" rpy="0 0 0"/>
+      </xacro:extra_module>
     </xacro:if>
     <!-- joint -->>
@@ -127,5 +143,7 @@
         <dynamics damping="0.8" friction="0.05"/>
       </joint>
-      <xacro:extra_module name = "joint${self}_module" parent = "${self}" mass = "${joint_mass}" offset = "${link_length* 0.5 + link_joint_offset}" />
+      <xacro:extra_module name = "joint${self}_module" parent = "${self}" mass = "${joint_mass}" >
+        <origin xyz="${link_length* 0.5 + link_joint_offset} 0.0 0.0" rpy="0 0 0"/>
+      </xacro:extra_module>
     </xacro:unless>
     <!-- hardware interface -->

Commit message: Improve the mono optical flow estimation based on the epipolar constraint

File: robots/hydrus/robots/hydrusx/quad.gazebo.xacro (robot description, xacro)
@@ -38,7 +38,7 @@
   </xacro:sonar_sensor>
   <!-- 3. downward camera -->
-<xacro:include filename="$(find hector_sensors_description)/urdf/generic_camera.urdf.xacro" />
-  <xacro:generic_camera name="downwards_cam" parent="link3" ros_topic="/camera/image" cam_info_topic="/camera/camera_info" update_rate="30" res_x="640" res_y="480" image_format="R8G8B8" hfov="54">
-    <origin xyz="0.1 0.0 -0.05" rpy="0 ${90*pi/180} 0"/>
+  <xacro:include filename="$(find hector_sensors_description)/urdf/generic_camera.urdf.xacro" />
+  <xacro:generic_camera name="downwards_cam" parent="link3" ros_topic="/camera/image" cam_info_topic="/camera/camera_info" update_rate="20" res_x="640" res_y="480" image_format="R8G8B8" hfov="54">
+    <origin xyz="0.1 0.0 -0.05" rpy="0 ${pi/2} 0"/>
   </xacro:generic_camera>
 </robot>
