Commit message: Improve launch file for special model

File: robots/hydrus_xi/urdf/common.xacro (robot description, xacro)
@@ -44,6 +44,4 @@
       <xacro:if value="${visible == 1}">
         <visual>
-          <!-- the origin of link_frame and visual_frame should be identical -->
-          <!--origin rpy="${-pi/2} 0 0" xyz="0 0 0"/-->
           <geometry>
             <mesh filename="${model_url}"/>
@@ -51,4 +49,22 @@
         </visual>
       </xacro:if>
+    </link>
+  </xacro:macro>
+  <xacro:macro name="extra_module_collision" params="name parent *origin *inertial visible:=0 model_url:=0 *collision">
+    <joint name="${parent}2${name}" type="fixed">
+      <parent link="${parent}"/>
+      <child link="${name}"/>
+      <xacro:insert_block name="origin" />
+    </joint>
+    <link name="${name}">
+      <xacro:insert_block name="inertial" />
+      <xacro:if value="${visible == 1}">
+        <visual>
+          <geometry>
+            <mesh filename="${model_url}"/>
+          </geometry>
+        </visual>
+      </xacro:if>
+      <xacro:insert_block name="collision"/>
     </link>
   </xacro:macro>
