Commit message: add hydrus_xi branch type model

File: robots/hydrus_xi/urdf/branch_type_link.urdf.xacro (robot description, xacro)
@@ -2,5 +2,96 @@
 <robot
     xmlns:xacro="http://www.ros.org/wiki/xacro" name="hydrus_xi_link">
-  <xacro:macro name="hydrus_xi_link" params="self child rotor_direction link_type">
+  <xacro:macro name="hydrus_xi_center_link" params="child1 child2 child3">
+    #### dummy root link for KDL ####
+    <link name="root">
+      <inertial>
+        <origin xyz="0 0 0" rpy="0 0 0"/>
+        <mass value="0.00001"/>
+        <inertia
+            ixx="0.000001" ixy="0.0" ixz="0.0"
+            iyy="0.000001" iyz="0.0"
+            izz="0.000001"/>
+      </inertial>
+    </link>
+    <joint name="root_joint" type="fixed">
+      <parent link="root"/>
+      <child link="center_link"/>
+      <origin rpy="0 0 0" xyz="0 0 0"/>
+      <axis xyz="0 0 1"/>
+    </joint>
+    #### link ####
+    <link name="center_link">
+      <inertial>
+        <origin xyz="0.294295 -0.000052 0.028894" rpy="0 0 0"/>
+        <mass value="0.714766"/>
+        <inertia
+            ixx="0.008182" iyy="0.019328" izz="0.023801"
+            ixy="-0.000016" ixz="0.010020" iyz="-0.000003"/>
+      </inertial>
+      <xacro:mesh_model type="link/center_link">
+        <origin xyz="0 0 0" rpy="0 0 0"/>
+      </xacro:mesh_model>
+    </link>
+    <xacro:damping_factor link="center_link"/>
+    #### joints ####
+    #### link joint ####
+    <joint name="joint${child1}" type="revolute">
+      <limit effort="3.3" lower="-1.57" upper="1.57" velocity="0.5"/>
+      <parent link="center_link"/>
+      <child link="link${child1}"/>
+      <origin rpy="0 0 ${pi / 2.0}" xyz="0 0.1255 0.016"/>
+      <axis xyz="0 0 1"/>
+      <dynamics damping="0.8" friction="0.05"/>
+    </joint>
+    <joint name="joint${child2}" type="revolute">
+      <limit effort="3.3" lower="-1.57" upper="1.57" velocity="0.5"/>
+      <parent link="center_link"/>
+      <child link="link${child2}"/>
+      <origin rpy="0 0 ${pi * 7.0 / 6.0}" xyz="-0.10869 -0.06275 0.016"/>
+      <axis xyz="0 0 1"/>
+      <dynamics damping="0.8" friction="0.05"/>
+    </joint>
+    <joint name="joint${child3}" type="revolute">
+      <limit effort="3.3" lower="-1.57" upper="1.57" velocity="0.5"/>
+      <parent link="center_link"/>
+      <child link="link${child3}"/>
+      <origin rpy="0 0 ${pi * 11.0 / 6.0}" xyz="0.10869 -0.06275 0.016"/>
+      <axis xyz="0 0 1"/>
+      <dynamics damping="0.8" friction="0.05"/>
+    </joint>
+    #### hardware interface ####
+    <transmission name="joint_tran${child1}">
+      <type>transmission_interface/SimpleTransmission</type>
+      <joint name="joint${child1}">
+        <hardwareInterface>hardware_interface/EffortJointInterface</hardwareInterface>
+      </joint>
+      <actuator name="servo${child1}">
+        <hardwareInterface>hardware_interface/EffortJointInterface</hardwareInterface>
+        <mechanicalReduction>1</mechanicalReduction>
+      </actuator>
+    </transmission>
+    <transmission name="joint_tran${child2}">
+      <type>transmission_interface/SimpleTransmission</type>
+      <joint name="joint${child2}">
+        <hardwareInterface>hardware_interface/EffortJointInterface</hardwareInterface>
+      </joint>
+      <actuator name="servo${child2}">
+        <hardwareInterface>hardware_interface/EffortJointInterface</hardwareInterface>
+        <mechanicalReduction>1</mechanicalReduction>
+      </actuator>
+    </transmission>
+    <transmission name="joint_tran${child3}">
+      <type>transmission_interface/SimpleTransmission</type>
+      <joint name="joint${child3}">
+        <hardwareInterface>hardware_interface/EffortJointInterface</hardwareInterface>
+      </joint>
+      <actuator name="servo${child3}">
+        <hardwareInterface>hardware_interface/EffortJointInterface</hardwareInterface>
+        <mechanicalReduction>1</mechanicalReduction>
+      </actuator>
+    </transmission>
+    <xacro:friction self="center_link"/>
+  </xacro:macro>
+  <xacro:macro name="hydrus_xi_branch_type_link" params="self child rotor_direction link_type">
     #### link ####
     <link name="link${self}">
@@ -14,18 +105,5 @@
         </inertial>
         <xacro:mesh_model type="link/general_link">
-          <origin xyz="0 0 0" rpy="0 0 0"/>
-        </xacro:mesh_model>
-        <xacro:link_collision_model/>
-      </xacro:if>
-      <xacro:if value="${link_type == 'head'}">
-        <inertial>
-          <origin xyz="0.32159 -0.0000232075 0.020785" rpy="0 0 0"/>
-          <mass value="0.64047"/>
-          <inertia
-              ixx="0.008485" iyy="0.015088" izz="0.019250"
-              ixy="-0.000009" ixz="0.007973" iyz="-0.000001"/>
-        </inertial>
-        <xacro:mesh_model type="link/head_link">
-          <origin xyz="0 0 0" rpy="0 0 0"/>
+          <origin xyz="0.6 0 0" rpy="0 0 ${pi}"/>
         </xacro:mesh_model>
         <xacro:link_collision_model/>
@@ -39,6 +117,6 @@
               ixy="-0.000016" ixz="0.009513" iyz="-0.000003"/>
         </inertial>
-        <xacro:mesh_model type="link/end_link">
-          <origin xyz="0 0 0" rpy="0 0 0"/>
+        <xacro:mesh_model type="link/head_link">
+          <origin xyz="0.6 0 0" rpy="0 0 ${pi}"/>
         </xacro:mesh_model>
         <xacro:link_collision_model/>
@@ -90,27 +168,8 @@
     </link>
     <xacro:damping_factor link="thrust${self}"/>
-    #### dummy root link for KDL ####
-    <xacro:if value="${self == 1}">
-      <link name="root">
-        <inertial>
-          <origin xyz="0 0 0" rpy="0 0 0"/>
-          <mass value="0.00001"/>
-          <inertia
-              ixx="0.000001" ixy="0.0" ixz="0.0"
-              iyy="0.000001" iyz="0.0"
-              izz="0.000001"/>
-        </inertial>
-      </link>
-      <joint name="root_joint" type="fixed">
-        <parent link="root"/>
-        <child link="link${self}"/>
-        <origin rpy="0 0 0" xyz="0 0 0"/>
-        <axis xyz="0 0 1"/>
-      </joint>
-    </xacro:if>
     #### joints ####
     #### link joint ####
     <xacro:unless value="${self == child}">
-      <joint name="joint${self}" type="revolute">
+      <joint name="joint${child}" type="revolute">
         <limit effort="3.3" lower="-1.57" upper="1.57" velocity="0.5"/>
         <parent link="link${self}"/>
@@ -148,5 +207,5 @@
     <xacro:extra_module name="bat${self}" parent="link${self}" visible="1"
                         model_url="package://hydrus_xi/urdf/mesh/modules/battery/battery.dae">
-      <origin xyz="0.3133 0.0 -0.048" rpy="0 0 ${pi / 2.0}"/>
+      <origin xyz="0.2867 0.0 -0.048" rpy="0 0 ${pi / 2.0}"/>
       <inertial>
         <origin xyz="0 0 0" rpy="0 0 0"/>
@@ -160,10 +219,10 @@
     #### hardware interface ####
     <xacro:unless value="${self == child}">
-      <transmission name="joint_tran${self}">
+      <transmission name="joint_tran${child}">
         <type>transmission_interface/SimpleTransmission</type>
-        <joint name="joint${self}">
+        <joint name="joint${child}">
           <hardwareInterface>hardware_interface/EffortJointInterface</hardwareInterface>
         </joint>
-        <actuator name="servo{self}">
+        <actuator name="servo{child}">
           <hardwareInterface>hardware_interface/EffortJointInterface</hardwareInterface>
           <mechanicalReduction>1</mechanicalReduction>

Commit message: fix params of hydrus_xi branch type

File: robots/hydrus_xi/urdf/branch_type_link.urdf.xacro (robot description, xacro)
@@ -40,5 +40,5 @@
       <parent link="center_link"/>
       <child link="link${child1}"/>
-      <origin rpy="0 0 0" xyz="0.1255 0 0.016"/>
+      <origin rpy="0 0 ${pi * 4.0 / 3.0}" xyz="-0.06275 -0.10869 0.016"/>
       <axis xyz="0 0 1"/>
       <dynamics damping="0.8" friction="0.05"/>
@@ -48,5 +48,5 @@
       <parent link="center_link"/>
       <child link="link${child2}"/>
-      <origin rpy="0 0 ${pi * 2.0 / 3.0}" xyz="-0.06275 0.10869 0.016"/>
+      <origin rpy="0 0 0" xyz="0.1255 0 0.016"/>
       <axis xyz="0 0 1"/>
       <dynamics damping="0.8" friction="0.05"/>
@@ -56,5 +56,5 @@
       <parent link="center_link"/>
       <child link="link${child3}"/>
-      <origin rpy="0 0 ${pi * 4.0 / 3.0}" xyz="-0.06275 -0.10869 0.016"/>
+      <origin rpy="0 0 ${pi * 2.0 / 3.0}" xyz="-0.06275 0.10869 0.016"/>
       <axis xyz="0 0 1"/>
       <dynamics damping="0.8" friction="0.05"/>
@@ -185,5 +185,5 @@
       <parent link="link${self}"/>
       <child link="gimbal_link${self}"/>
-      <origin rpy="0 0 ${pi}" xyz="0.2984 0 0.05967"/>
+      <origin rpy="0 0 0" xyz="0.2984 0 0.05967"/>
       <axis xyz="0 0 1"/>
       <dynamics damping="0.8" friction="0.05"/>

Commit message: fix servo param

File: robots/hydrus_xi/urdf/branch_type_link.urdf.xacro (robot description, xacro)
@@ -42,5 +42,5 @@
       <origin rpy="0 0 0" xyz="0.1555 0.0 0.015"/>
       <axis xyz="0 0 1"/>
-      <dynamics damping="0.8" friction="0.05"/>
+      <dynamics damping="0.8" friction="0.0"/>
     </joint>
     <joint name="joint${child2}" type="revolute">
@@ -50,5 +50,5 @@
       <origin rpy="0 0 ${pi * 2.0 / 3.0}" xyz="-0.07775 0.13467 0.015"/>
       <axis xyz="0 0 1"/>
-      <dynamics damping="0.8" friction="0.05"/>
+      <dynamics damping="0.8" friction="0.0"/>
     </joint>
     <joint name="joint${child3}" type="revolute">
@@ -58,5 +58,5 @@
       <origin rpy="0 0 ${pi * 4.0 / 3.0}" xyz="-0.07775 -0.13467 0.015"/>
       <axis xyz="0 0 1"/>
-      <dynamics damping="0.8" friction="0.05"/>
+      <dynamics damping="0.8" friction="0.0"/>
     </joint>
     #### hardware interface ####
@@ -177,5 +177,5 @@
         <origin rpy="0 0 0" xyz="${link_length} 0 0"/>
         <axis xyz="0 0 1"/>
-        <dynamics damping="0.8" friction="0.05"/>
+        <dynamics damping="0.8" friction="0.0"/>
       </joint>
     </xacro:unless>
@@ -187,5 +187,5 @@
       <origin rpy="0 0 0" xyz="0.2984 0 0.05967"/>
       <axis xyz="0 0 1"/>
-      <dynamics damping="0.8" friction="0.05"/>
+      <dynamics damping="0.8" friction="0.0"/>
     </joint>
     #### rotor parent link joint (virtual) ####

Commit message: change servo angle speed

File: robots/hydrus_xi/urdf/branch_type_link.urdf.xacro (robot description, xacro)
@@ -37,5 +37,5 @@
     #### link joint ####
     <joint name="joint${child1}" type="revolute">
-      <limit effort="6.6" lower="-1.57" upper="1.57" velocity="0.5"/>
+      <limit effort="6.6" lower="-1.57" upper="1.57" velocity="3.0"/>
       <parent link="center_link"/>
       <child link="link${child1}"/>
@@ -45,5 +45,5 @@
     </joint>
     <joint name="joint${child2}" type="revolute">
-      <limit effort="6.6" lower="-1.57" upper="1.57" velocity="0.5"/>
+      <limit effort="6.6" lower="-1.57" upper="1.57" velocity="3.0"/>
       <parent link="center_link"/>
       <child link="link${child2}"/>
@@ -53,5 +53,5 @@
     </joint>
     <joint name="joint${child3}" type="revolute">
-      <limit effort="6.6" lower="-1.57" upper="1.57" velocity="0.5"/>
+      <limit effort="6.6" lower="-1.57" upper="1.57" velocity="3.0"/>
       <parent link="center_link"/>
       <child link="link${child3}"/>
@@ -172,5 +172,5 @@
     <xacro:unless value="${self == child}">
       <joint name="joint${child}" type="revolute">
-        <limit effort="6.6" lower="${-pi * 0.5}" upper="${pi * 0.5}" velocity="0.5"/>
+        <limit effort="6.6" lower="${-pi * 0.5}" upper="${pi * 0.5}" velocity="3.0"/>
         <parent link="link${self}"/>
         <child link="link${child}"/>
@@ -182,5 +182,5 @@
     #### gimbal joint ####
     <joint name="gimbal${self}" type="revolute">
-      <limit effort="3.1" lower="-3.1415" upper="3.1415" velocity="0.5"/>
+      <limit effort="3.1" lower="-3.1415" upper="3.1415" velocity="3.0"/>
       <parent link="link${self}"/>
       <child link="gimbal_link${self}"/>

Commit message: modify model collision

File: robots/hydrus_xi/urdf/branch_type_link.urdf.xacro (robot description, xacro)
@@ -32,4 +32,10 @@
         <origin xyz="0 0 0" rpy="0 0 0"/>
       </xacro:mesh_model>
+      <collision>
+        <origin rpy="0 0 0" xyz="0 0 0"/>
+        <geometry>
+          <cylinder length="0.20" radius="0.1"/>
+        </geometry>
+      </collision>
     </link>
     <xacro:damping_factor link="center_link"/>
@@ -137,10 +143,10 @@
         <origin xyz="0 0 0" rpy="0 0 0"/>
       </xacro:mesh_model>
-      <!-- <collision> -->
-      <!--   <origin rpy="0 0 0" xyz="0 0 ${- collision_rotor_height / 2}"/> -->
-      <!--   <geometry> -->
-      <!--     <cylinder length="${collision_rotor_height}" radius="${protector_radius + 0.01}"/> -->
-      <!--   </geometry> -->
-      <!-- </collision> -->
+      <collision>
+        <origin rpy="0 0 0" xyz="0 0 ${- collision_rotor_height / 2}"/>
+        <geometry>
+          <cylinder length="${collision_rotor_height}" radius="${protector_radius + 0.01}"/>
+        </geometry>
+      </collision>
     </link>
     <xacro:damping_factor link="gimbal_link${self}"/>

File: robots/hydrus_xi/urdf/common.xacro (robot description, xacro)
@@ -4,4 +4,5 @@
   <!-- kinematics [m] -->
   <xacro:property name="link_length" value="0.6"/>
+  <xacro:property name="link_height" value="0.28"/>
   <xacro:property name="protector_radius" value="0.1925"/>
   <xacro:property name="fc_x_offset" value="0.566"/>
@@ -29,5 +30,5 @@
       <origin rpy="0 0 0" xyz="${link_length* 0.5} 0 0"/>
       <geometry>
-        <box size="${link_length} 0.05 0.25"/>
+        <box size="${link_length} 0.05 ${link_height}"/>
       </geometry>
     </collision>

Commit message: modify to 15inch prop

File: robots/hydrus_xi/urdf/branch_type_link.urdf.xacro (robot description, xacro)
@@ -105,5 +105,5 @@
         <inertial>
           <origin xyz="0.300691 0.000051 0.027824" rpy="0 0 0"/>
-          <mass value="0.736958"/>
+          <mass value="0.606958"/>
           <inertia
               ixx="0.008461" iyy="0.022896" izz="0.027105"
@@ -117,9 +117,9 @@
       <xacro:if value="${link_type == 'end'}">
         <inertial>
-          <origin xyz="0.300691 0.000051 0.027824" rpy="0 0 0"/>
-          <mass value="0.736958"/>
+          <origin xyz="0.271325 0.000023 0.018067" rpy="0 0 0"/>
+          <mass value="0.527057"/>
           <inertia
-              ixx="0.008461" iyy="0.022896" izz="0.027105"
-              ixy="0.000029" ixz="0.013452" iyz="0.000003"/>
+              ixx="0.008981" iyy="0.018237" izz="0.021912"
+              ixy="0.000009" ixz="0.005609" iyz="0.000001"/>
         </inertial>
         <xacro:mesh_model type="link/end_link1">
@@ -135,5 +135,5 @@
       <inertial>
         <origin xyz="-0.006114 0.000001 0.032778" rpy="0 0 0"/>
-        <mass value="0.140963"/>
+        <mass value="0.23599752692"/>
         <inertia
             ixx="0.001" iyy="0.001" izz="0.001"

Commit message: modify for experiment

File: robots/hydrus_xi/urdf/branch_type_link.urdf.xacro (robot description, xacro)
@@ -191,5 +191,5 @@
       <parent link="link${self}"/>
       <child link="gimbal_link${self}"/>
-      <origin rpy="0 0 0" xyz="0.2984 0 0.05967"/>
+      <origin rpy="0 0 ${pi}" xyz="0.2984 0 0.05967"/>
       <axis xyz="0 0 1"/>
       <dynamics damping="0.8" friction="0.0"/>

Commit message: update hydrus_xi branch type mesh model

File: robots/hydrus_xi/urdf/branch_type_link.urdf.xacro (robot description, xacro)
@@ -104,9 +104,9 @@
       <xacro:if value="${link_type == 'middle'}">
         <inertial>
-          <origin xyz="0.300691 0.000051 0.027824" rpy="0 0 0"/>
-          <mass value="0.606958"/>
+          <origin xyz="0.313051 0.000071 0.011024" rpy="0 0 0"/>
+          <mass value="0.535052"/>
           <inertia
-              ixx="0.008461" iyy="0.022896" izz="0.027105"
-              ixy="0.000029" ixz="0.013452" iyz="0.000003"/>
+              ixx="0.000808" iyy="0.014148" izz="0.013428"
+              ixy="0.000030" ixz="0.005073" iyz="0.000002"/>
         </inertial>
         <xacro:mesh_model type="link/middle_link">
@@ -117,9 +117,9 @@
       <xacro:if value="${link_type == 'end'}">
         <inertial>
-          <origin xyz="0.271325 0.000023 0.018067" rpy="0 0 0"/>
-          <mass value="0.527057"/>
+          <origin xyz="0.272827 0.000033 -0.006011" rpy="0 0 0"/>
+          <mass value="0.455151"/>
           <inertia
-              ixx="0.008981" iyy="0.018237" izz="0.021912"
-              ixy="0.000009" ixz="0.005609" iyz="0.000001"/>
+              ixx="0.001020" iyy="0.009477" izz="0.008530"
+              ixy="0.000009" ixz="-0.002418" iyz="0.000000"/>
         </inertial>
         <xacro:mesh_model type="link/end_link1">
@@ -134,9 +134,9 @@
     <link name="gimbal_link${self}">
       <inertial>
-        <origin xyz="-0.006114 0.000001 0.032778" rpy="0 0 0"/>
-        <mass value="0.23599752692"/>
-        <inertia
-            ixx="0.001" iyy="0.001" izz="0.001"
-            ixy="0" ixz="0" iyz="0"/>
+        <origin xyz="-0.009927 0.000000 0.050828" rpy="0 0 0"/>
+        <mass value="0.252140"/>
+        <inertia
+            ixx="0.004032" iyy="0.003374" izz="0.006517"
+            ixy="-0.000000" ixz="-0.001309" iyz="0.000000"/>
       </inertial>
       <xacro:mesh_model type="link/propeller_link">
@@ -187,9 +187,9 @@
     </xacro:unless>
     #### gimbal joint ####
-    <joint name="gimbal${self}" type="revolute">
-      <limit effort="3.1" lower="-3.1415" upper="3.1415" velocity="3.0"/>
+    <joint name="gimbal${self}" type="continuous">
+      <limit effort="3.1" lower="${pi * -6}" upper="${pi * 6}" velocity="20.0"/>
       <parent link="link${self}"/>
       <child link="gimbal_link${self}"/>
-      <origin rpy="0 0 ${pi}" xyz="0.2984 0 0.05967"/>
+      <origin rpy="0 0 ${pi}" xyz="0.2984 0 0.04867"/>
       <axis xyz="0 0 1"/>
       <dynamics damping="0.8" friction="0.0"/>
@@ -199,5 +199,5 @@
       <parent link="gimbal_link${self}"/>
       <child link="rotor_parent${self}"/>
-      <origin rpy="0 ${thrust_tilt_angle} 0" xyz="0 0 0.05091"/>
+      <origin rpy="0 ${thrust_tilt_angle} 0" xyz="0 0 0.06041"/>
       <axis xyz="0 0 ${rotor_direction}"/>
     </joint>

Commit message: Modify propeller link inertia

File: robots/hydrus_xi/urdf/branch_type_link.urdf.xacro (robot description, xacro)
@@ -134,9 +134,9 @@
     <link name="gimbal_link${self}">
       <inertial>
-        <origin xyz="-0.009927 0.000000 0.050828" rpy="0 0 0"/>
-        <mass value="0.252140"/>
-        <inertia
-            ixx="0.004032" iyy="0.003374" izz="0.006517"
-            ixy="-0.000000" ixz="-0.001309" iyz="0.000000"/>
+        <origin xyz="-0.010664 0.000000 0.049923" rpy="0 0 0"/>
+        <mass value="0.237140"/>
+        <inertia
+            ixx="0.004029" iyy="0.003369" izz="0.006515"
+            ixy="-0.000000" ixz="-0.001310" iyz="0.000000"/>
       </inertial>
       <xacro:mesh_model type="link/propeller_link">

Commit message: Refactor the jacobian calculation for thrust force (lambda) and joint torque

File: robots/hydrus_xi/urdf/branch_type_link.urdf.xacro (robot description, xacro)
@@ -47,5 +47,5 @@
       <child link="link${child1}"/>
       <origin rpy="0 0 0" xyz="0.1555 0.0 0.015"/>
-      <axis xyz="0 0 1"/>
+      <axis xyz="0 1 0"/>
       <dynamics damping="0.8" friction="0.0"/>
     </joint>
@@ -55,5 +55,5 @@
       <child link="link${child2}"/>
       <origin rpy="0 0 ${pi * 2.0 / 3.0}" xyz="-0.07775 0.13467 0.015"/>
-      <axis xyz="0 0 1"/>
+      <axis xyz="0 1 0"/>
       <dynamics damping="0.8" friction="0.0"/>
     </joint>
@@ -63,5 +63,5 @@
       <child link="link${child3}"/>
       <origin rpy="0 0 ${pi * 4.0 / 3.0}" xyz="-0.07775 -0.13467 0.015"/>
-      <axis xyz="0 0 1"/>
+      <axis xyz="0 1 0"/>
       <dynamics damping="0.8" friction="0.0"/>
     </joint>

Commit message: - Refactor aerial_robot_model/src/transformable_aerial_robot_model: separate into several source files with different functions: general api, kinematics, statics, statiblity - Refactor the numerical jacobian solution as rostest code to compare with analytical results

File: robots/hydrus_xi/urdf/branch_type_link.urdf.xacro (robot description, xacro)
@@ -47,5 +47,5 @@
       <child link="link${child1}"/>
       <origin rpy="0 0 0" xyz="0.1555 0.0 0.015"/>
-      <axis xyz="0 1 0"/>
+      <axis xyz="1 0 0"/>
       <dynamics damping="0.8" friction="0.0"/>
     </joint>
@@ -55,5 +55,5 @@
       <child link="link${child2}"/>
       <origin rpy="0 0 ${pi * 2.0 / 3.0}" xyz="-0.07775 0.13467 0.015"/>
-      <axis xyz="0 1 0"/>
+      <axis xyz="1 0 0"/>
       <dynamics damping="0.8" friction="0.0"/>
     </joint>
@@ -63,5 +63,5 @@
       <child link="link${child3}"/>
       <origin rpy="0 0 ${pi * 4.0 / 3.0}" xyz="-0.07775 -0.13467 0.015"/>
-      <axis xyz="0 1 0"/>
+      <axis xyz="1 0 0"/>
       <dynamics damping="0.8" friction="0.0"/>
     </joint>
