Commit message: Create quad (under-actuated) type of hydrus_xi

File: robots/hydrus_xi/urdf/link.urdf.xacro (robot description, xacro)
@@ -122,6 +122,6 @@
     </xacro:unless>
     #### gimbal joint ####
-    <joint name="gimbal${self}" type="revolute">
-      <limit effort="3.1" lower="-3.1415" upper="3.1415" velocity="0.5"/>
+    <joint name="gimbal${self}" type="continuous">
+      <limit effort="3.1" lower="${pi * -6}" upper="${pi * 6}" velocity="20.0"/>
       <parent link="link${self}"/>
       <child link="gimbal_link${self}"/>

Commit message: fix gimbal link module weight (again)

File: robots/hydrus_xi/urdf/link.urdf.xacro (robot description, xacro)
@@ -51,5 +51,5 @@
       <inertial>
         <origin xyz="-0.006114 0.000001 0.032778" rpy="0 0 0"/>
-        <mass value="0.140963"/>
+        <mass value="0.260"/>
         <inertia
             ixx="0.001" iyy="0.001" izz="0.001"
