Commit message: fixed HydrusXI model files

File: robots/hydrus_xi/robots/octo.urdf.xacro (robot description, xacro)
@@ -5,6 +5,6 @@
   <xacro:include filename="$(find hydrus_xi)/urdf/hydrus_xi_link.urdf.xacro" />
   <!--  model type 1: baselink (attached with imu, pc): fixed_n-->
-  <!--  model type 2: fixed_p_link -->
-  <!--  model type 3: fixed_n_link -->
+  <!--  model type 2: fixed_n_link -->
+  <!--  model type 3: fixed_p_link -->
   <xacro:hydrus_xi_module self="1" child="2" rotor_direction="-1"  link_type="1" />
   <xacro:hydrus_xi_module self="2" child="3" rotor_direction="1"  link_type="3" />

File: robots/hydrus_xi/urdf/hydrus_xi_common.xacro (robot description, xacro)
@@ -32,13 +32,11 @@
     </collision>
     <visual>
-      <origin rpy="${- pi / 2} 0 0" xyz="${link_length* 0.5} 0 0"/>
-      <!-- <origin rpy="0 0 0" xyz="${link_length* 0.5} 0 0"/>  STL-->
+      <!--<origin rpy="${- pi / 2} 0 0" xyz="${link_length* 0.5} 0 0"/> -->
+      <origin rpy="0 0 0" xyz="${link_length* 0.5} 0 0"/>
       <geometry>
-        <mesh filename="package://hydrus_xi/urdf/mesh/${type}.dae"/>
-        <!-- STL
-            <mesh filename="package://hydrus_xi/urdf/mesh/${type}.stl" scale="0.001 0.001 0.001"/>
-        -->
+        <!--<mesh filename="package://hydrus_xi/urdf/mesh/${type}.dae"/> -->
+        <mesh filename="package://hydrus_xi/urdf/mesh/${type}.stl" scale="0.001 0.001 0.001"/>
       </geometry>
-      <!-- <material name="black"/> STL-->
+      <material name="black"/>
     </visual>
   </xacro:macro>

File: robots/hydrus_xi/urdf/hydrus_xi_link.urdf.xacro (robot description, xacro)
@@ -16,4 +16,20 @@
         </inertial>
         <xacro:link_model type="baselink" />
+        <link name="fc">
+          <inertial>
+            <origin xyz="0 0 0" rpy="0 0 0"/>
+            <mass value="0.00001"/>
+            <inertia
+                ixx="0.000001" ixy="0.0" ixz="0.0"
+                iyy="0.000001" iyz="0.0"
+                izz="0.000002"/>
+          </inertial>
+        </link>
+        <joint name="fc_joint" type="fixed">
+          <child link="fc"/>
+          <parent link="link${self}"/>
+          <origin rpy="0 0 0" xyz="${fc_x_offset} 0 ${fc_z_offset}"/>
+          <axis xyz="0 0 1"/>
+        </joint>
       </xacro:if>
       <!-- fixed_n_link -->
@@ -93,4 +109,18 @@
         <axis xyz="0 0 1"/>
       </joint>
+    </xacro:if>
+    <!-- joint -->>
+    <xacro:unless value="${self == child}">
+      <joint name="joint${self}" type="revolute">
+        <limit effort="3.1" lower="-1.57" upper="1.57" velocity="0.5"/>
+        <parent link="link${self}"/>
+        <child link="link${child}"/>
+        <origin rpy="0 0 0" xyz="${link_length} 0 0"/>
+        <axis xyz="0 0 1"/>
+        <dynamics damping="0.8" friction="0.05"/>
+      </joint>
+    </xacro:unless>
+    <!-- fc -->
+    <xacro:if value="${link_type == 1}">
       <link name="fc">
         <inertial>
@@ -110,15 +140,4 @@
       </joint>
     </xacro:if>
-    <!-- joint -->>
-    <xacro:unless value="${self == child}">
-      <joint name="joint${self}" type="revolute">
-        <limit effort="3.1" lower="-1.57" upper="1.57" velocity="0.5"/>
-        <parent link="link${self}"/>
-        <child link="link${child}"/>
-        <origin rpy="0 0 0" xyz="${link_length} 0 0"/>
-        <axis xyz="0 0 1"/>
-        <dynamics damping="0.8" friction="0.05"/>
-      </joint>
-    </xacro:unless>
     <!-- hardware interface -->
     <xacro:unless value="${self == child}">
