Commit message: add small white battery mass data

File: robots/hydrus/urdf/hydrusx/hydrusx_common.xacro (robot description, xacro)
@@ -26,5 +26,5 @@
   <xacro:property name="protector_mass" value=".05" />
   <xacro:property name="protector_holder_mass" value=".0386" />
-  <xacro:property name="bat_mass" value="0.364" /> <!-- hyperon: 0.41, white: 0.364 -->
+  <xacro:property name="bat_mass" value="0.192" /> <!-- hyperon: 0.41, white(big): 0.364, white(small): 0.192 -->
   <xacro:property name="fc_mass" value=".03" />
   <xacro:property name="pc_c_mass" value=".13" /> <!-- odoroid u4: 0.1, euclid: 0.13 -->

Commit message: Update the collsion model for hydrusx

File: robots/hydrus/urdf/hydrusx/hydrusx_common.xacro (robot description, xacro)
@@ -43,8 +43,9 @@
   <xacro:property name="max_force" value="18" /> <!-- [N] -->
   <xacro:macro name="link_model" params="type">
+    <!-- for fcl in planning -->
     <collision>
       <origin rpy="0 0 0" xyz="${link_length* 0.5} 0 -0.03"/>
       <geometry>
-        <cylinder length="0.15" radius="${protector_radius}"/>
+        <box size="${link_length} 0.05 0.15"/>
       </geometry>
     </collision>

File: robots/hydrus/urdf/hydrusx/hydrusx_link.urdf.xacro (robot description, xacro)
@@ -56,4 +56,10 @@
             izz="${rotor_mass * .5 * rotor_radius * rotor_radius}"/>
       </inertial>
+      <collision>
+        <origin rpy="0 0 0" xyz="0 0 -0.03"/>
+        <geometry>
+          <cylinder length="0.15" radius="${protector_radius + 0.01}"/>
+        </geometry>
+        </collision>
     </link>
     <xacro:damping_factor link ="propeller${self}"/>

Commit message: Update parameters about control for hydrusx quad

File: robots/hydrus/urdf/hydrusx/hydrusx_common.xacro (robot description, xacro)
@@ -33,5 +33,5 @@
   <xacro:property name="head_leg_mass" value="0.0623" />
   <xacro:property name="tail_leg_mass" value="0.09" />
-  <xacro:property name="sensor_c_mass" value="0.065" />
+  <xacro:property name="sensor_c_mass" value="0.03" /> <!-- gps: 0.43 -->
   <xacro:property name="sensor_v_mass" value="0.18" />
   <xacro:property name="rotor_mass" value=".05" /> <!-- exclude from center mass -->

Commit message: Update the model of hydrusx (for quad type), which does not have rollors

File: robots/hydrus/urdf/hydrusx/hydrusx_common.xacro (robot description, xacro)
@@ -23,5 +23,5 @@
   <xacro:property name="link_rod_mass" value="0.099" />
   <xacro:property name="link_center_mass" value=".211" />
-  <xacro:property name="joint_mass" value=".2075" />
+  <xacro:property name="joint_mass" value=".19" /> <!-- rollor: 0.15 -->
   <xacro:property name="protector_mass" value=".05" />
   <xacro:property name="protector_holder_mass" value=".0386" />
@@ -31,6 +31,6 @@
   <xacro:property name="pc_v_mass" value=".24" />
   <xacro:property name="pcs_cable_mass" value=".03" />
-  <xacro:property name="head_leg_mass" value="0.0623" />
-  <xacro:property name="tail_leg_mass" value="0.09" />
+  <xacro:property name="head_leg_mass" value="0.045" /> <!-- rollor: 0.017 -->
+  <xacro:property name="tail_leg_mass" value="0.073" /> <!-- rollor: 0.017 -->
   <xacro:property name="sensor_c_mass" value="0.03" /> <!-- gps: 0.43 -->
   <xacro:property name="sensor_v_mass" value="0.18" />
