Commit message: Implement end-effector IK program based on Jacobian Inverse (sr-inverse)

File: robots/hydrus/urdf/hydrusx/hydrusx_link.urdf.xacro (robot description, xacro)
@@ -120,5 +120,5 @@
     <xacro:unless value="${self == child}">
       <joint name="joint${self}" type="revolute">
-        <limit effort="3.1" lower="-1.57" upper="1.57" velocity="0.5"/>
+        <limit effort="3.1" lower="-1.6" upper="1.6" velocity="0.5"/>
         <parent link="link${self}"/>
         <child link="link${child}"/>
