Commit message: Modified the zed mini position cofiguration to be idnetical to the real model

File: robots/hydrus/robots/quad/tx2_zed_201810.urdf.xacro (robot description, xacro)
@@ -84,5 +84,5 @@
     </inertial>
     <visual>
-      <origin xyz="${-22.5 * 0.001} 0 ${-19 * 0.001}" rpy="0 ${pi/2} ${pi/2}"/>
+      <origin xyz="${-14.75 * 0.001} 0 ${-19 * 0.001}" rpy="0 ${pi/2} ${-pi}"/>
       <geometry>
         <mesh filename="package://hydrus/urdf/mesh/modules/sensor/zed_mini_servo_down.dae"/>
@@ -90,4 +90,16 @@
     </visual>
   </link>
+  <!-- to create the zed center frame -->
+  <xacro:extra_module name = "zed_camera_center" parent = "zed_mini_servo_down" visible = "0" >
+    <origin xyz="${-14.75 * 0.001} 0 ${-19 * 0.001}" rpy="0 ${pi/2} ${pi/2}"/>
+    <inertial>
+      <mass value = "0.0" />
+      <origin xyz="0 0 0" rpy="0 0 0"/>
+      <inertia
+          ixx="0.0" ixy="0.0" ixz="0.0"
+          iyy="0.0" iyz="0.0"
+          izz="0.0"/>
+    </inertial>
+  </xacro:extra_module>
   <transmission name="zed_mini_servo_joint_tran">
     <type>transmission_interface/SimpleTransmission</type>

Commit message: temp

File: robots/hydrus/robots/quad/tx2_zed_201810.urdf.xacro (robot description, xacro)
@@ -78,5 +78,5 @@
     <inertial>
       <origin xyz="${-22.5 * 0.001} 0 ${-14 * 0.001}" rpy="0 0 0"/>
-      <mass value="0.08" />
+      <mass value="0.093" />
       <inertia
           ixx="0.00001" iyy="0.00012" izz="0.00013"

Commit message: Imrpove the urdf description of Hydrus: 1. precise inertial paramteres from CAD softerware (solid edge) 2. add leg and battery on/off flag for link module for more model option regarding to different types of legs and battereis

File: robots/hydrus/robots/quad/tx2_zed_201810.urdf.xacro (robot description, xacro)
@@ -7,8 +7,8 @@
   <xacro:extra_module name = "fc" parent = "link2" visible = "1"
                       model_url = "package://hydrus/urdf/mesh/modules/flight_controller/fc_euclid201806.dae"> <!-- same with intel euclid -->
-    <origin xyz="${link_length/2 + 0.2281} ${-4.4*0.001} 0.03533" rpy="0 0 0"/>
+    <origin xyz="${link_length / 2 + 0.2281} ${-4.4*0.001} 0.03533" rpy="0 0 0"/>
     <inertial>
-      <mass value = "0.0457" />
-      <origin xyz="${8.7*0.001} ${4.4*0.001} -0.01" rpy="0 0 0"/>
+      <mass value = "0.05" />
+      <origin xyz="${11.48*0.001} ${4.3*0.001} ${-9.4*0.001}" rpy="0 0 0"/>
       <inertia
           ixx="0.00001" ixy="0.0" ixz="0.0"
@@ -22,10 +22,9 @@
     <origin xyz="${link_length/2 + 0.206} 0.0 0.18" rpy="0 0 0"/>
     <inertial>
-      <mass value = "0.044" />
-      <origin xyz="0.0 0.0 -0.08" rpy="0 0 0"/>
+      <origin xyz="0.000000 0.000000 -0.062510" rpy="0 0 0"/>
+      <mass value="0.053000"/>
       <inertia
-          ixx="0.00001" ixy="0.0" ixz="0.0"
-          iyy="0.00001" iyz="0.0"
-          izz="0.00002"/>
+          ixx="0.000503" iyy="0.000503" izz="0.000010"
+          ixy="0.000000" ixz="0.000000" iyz="0.000000"/>
     </inertial>
   </xacro:extra_module>
@@ -43,13 +42,14 @@
   <!-- processor: jetson tx2 -->
   <xacro:extra_module name = "pc" parent = "link3" visible = "1"
-                      model_url = "package://hydrus/urdf/mesh/modules/processor/jetson_tx2.dae">
-    <origin xyz="${link_length/2 - 0.2134} 0.0 -0.0192" rpy="${pi/2} 0 ${pi}"/>
+                      model_url = "package://hydrus/urdf/mesh/modules/processor/jetson_tx2.dae"
+                      scale="0.001" >
+    <origin xyz="0.086 0.0 ${-0.0192}" rpy="${pi/2} 0 ${pi}"/>
     <inertial>
-      <mass value = "0.1672" />
-      <origin xyz="0 0 ${-5 * 0.001}" rpy="0 0 0"/>
+      <mass value = "0.181" />
+      <origin xyz="0 ${-5 * 0.001} 0" rpy="0 0 0"/>
       <inertia
           ixx="0.00001" ixy="0.0" ixz="0.0"
           iyy="0.00001" iyz="0.0"
-          izz="0.00002"/>
+          izz="0.00001"/>
     </inertial>
   </xacro:extra_module>
@@ -57,19 +57,19 @@
   <xacro:extra_module name = "zed_mini_servo_up" parent = "link2" visible = "1"
                       model_url = "package://hydrus/urdf/mesh/modules/sensor/zed_mini_servo_up.dae">
-    <origin xyz="${link_length/2 + 0.28714} 0.0 -0.04015" rpy="0 0 0"/>
+    <origin xyz="${link_length/2 + 0.28715} 0.0 -0.04015" rpy="0 0 0"/>
     <inertial>
-      <mass value = "0.017" />
-      <origin xyz="${-20 * 0.001} 0 ${5 * 0.001}" rpy="0 0 0"/>
+      <mass value = "0.021" />
+      <origin xyz="${-21.77 * 0.001} 0 ${10.3 * 0.001}" rpy="0 0 0"/>
       <inertia
-          ixx="0.00000" ixy="0.0" ixz="0.0"
-          iyy="0.00001" iyz="0.0"
-          izz="0.00001"/>
+          ixx="0.0" ixy="0.0" ixz="0.0"
+          iyy="0.0" iyz="0.0"
+          izz="0.0"/>
     </inertial>
   </xacro:extra_module>
   <joint name="zed_mini_servo_joint" type="revolute">
     <limit effort="0.2" lower="-1.6" upper="1.6" velocity="0.1"/>
-    <parent link="link2"/>
+    <parent link="zed_mini_servo_up"/>
     <child link="zed_mini_servo_down"/>
-    <origin rpy="0 0 0" xyz="${link_length/2 + 0.28714} 0.0 -0.04015"/>
+    <origin rpy="0 0 0" xyz="0 0.0 0"/>
     <axis xyz="1 0 0"/>
     <dynamics damping="0.01" friction="0.0"/>
@@ -77,8 +77,8 @@
   <link name="zed_mini_servo_down">
     <inertial>
-      <origin xyz="${-22.5 * 0.001} 0 ${-14 * 0.001}" rpy="0 0 0"/>
-      <mass value="0.093" />
+      <origin xyz="${-21.35 * 0.001} 0 ${-16.4 * 0.001}" rpy="0 0 0"/>
+      <mass value="0.079" />
       <inertia
-          ixx="0.00001" iyy="0.00012" izz="0.00013"
+          ixx="0.00001" iyy="0.00012" izz="0.00012"
           ixy="0" ixz="0" iyz="0"/>
     </inertial>

File: robots/hydrus/urdf/common.xacro (robot description, xacro)
@@ -4,39 +4,27 @@
   <!-- kinematics [m] -->
   <xacro:property name="link_length" value=".6" />
-  <xacro:property name="link_rod_length" value=".528" />
   <xacro:property name="protector_radius" value=".1925" />
-  <xacro:property name="link_joint_offset" value="0.3" />
-  <xacro:property name="rotor_radius" value=".02" />
-  <xacro:property name="rotor_height" value=".05" />
-  <xacro:property name="bat_offset" value="0.0" />
-  <xacro:property name="head_leg_offset" value="-0.25" />
-  <xacro:property name="end_leg_offset" value="0.235" />
-  <!-- inertial paramters -->
-  <!-- mass [Kg] -->
-  <xacro:property name="link_rod_mass" value="0.099" />
-  <xacro:property name="link_center_mass" value=".211" />
-  <xacro:property name="joint_mass" value=".19" /> <!-- rollor: 0.15 -->
-  <xacro:property name="protector_mass" value=".05" />
-  <xacro:property name="protector_holder_mass" value=".0386" />
-  <xacro:property name="bat_mass" value="0.193" /> <!-- hyperon: 0.41, white(2700mAh): 0.364, white(1300mAh): 0.193 -->
-  <xacro:property name="head_leg_mass" value="0.045" /> <!-- rollor: 0.017 -->
-  <xacro:property name="end_leg_mass" value="0.073" /> <!-- rollor: 0.017 -->
-  <xacro:property name="rotor_mass" value=".05" /> <!-- exclude from center mass -->
+  <xacro:property name="head_leg_offset" value="0.0525" />
+  <xacro:property name="general_leg_offset" value="0.05" />
+  <xacro:property name="end_leg_offset" value="0.5355" />
   <!-- collision model parameter -->
-  <xacro:property name="collision_model_height" value="0.14" />
-  <xacro:property name="collision_model_z_offset" value="-0.0215" />
-  <!-- inertial [N*m*m] -->
-  <xacro:property name="link_rod_inertia" value="${link_rod_mass * link_rod_length * link_rod_length /12}" /> <!-- mass * dist * dist -->
-  <xacro:property name="protector_inertia" value="${protector_mass * protector_radius * protector_radius}" /> <!-- mass * dist * dist -->
-  <xacro:property name="protector_holder_inertia" value="${protector_holder_mass * protector_radius * protector_radius}" /> <!-- mass * dist * dist -->
+  <xacro:property name="leg_collision_model_height" value="0.1715" />
   <!-- dynamics -->
   <xacro:property name="max_force" value="18" /> <!-- [N] -->
-  <xacro:macro name="link_model" params="type">
+  <xacro:macro name="link_model" params="type with_leg:=${with_leg}">
     <!-- for fcl in planning -->
     <collision>
-      <origin rpy="0 0 0" xyz="${link_length* 0.5} 0 ${collision_model_z_offset}"/>
-      <geometry>
-        <box size="${link_length} 0.05 ${collision_model_height}"/>
-      </geometry>
+      <xacro:if value="${with_leg == 1}">
+        <origin rpy="0 0 0" xyz="${link_length* 0.5} 0 ${- leg_collision_model_height / 2}"/>
+        <geometry>
+          <box size="${link_length} 0.05 ${leg_collision_model_height}"/>
+        </geometry>
+      </xacro:if>
+      <xacro:unless value="${with_leg == 1}">
+        <origin rpy="0 0 0" xyz="${link_length* 0.5} 0 0"/>
+        <geometry>
+          <box size="${link_length} 0.05 0.1"/>
+        </geometry>
+      </xacro:unless>
     </collision>
     <visual>
@@ -47,5 +35,5 @@
     </visual>
   </xacro:macro>
-  <xacro:macro name="extra_module" params="name parent *origin *inertial visible:=0 model_url:=0">
+  <xacro:macro name="extra_module" params="name parent *origin *inertial visible:=0 model_url:=1 scale:=1">
     <joint name="${parent}2${name}" type="fixed">
       <parent link="${parent}"/>
@@ -60,9 +48,30 @@
           <origin rpy="${-pi/2} 0 0" xyz="0 0 0"/>
           <geometry>
-            <mesh filename="${model_url}"/>
+            <mesh filename="${model_url}" scale= "${scale} ${scale} ${scale}"/>
           </geometry>
         </visual>
-        </xacro:if>
+      </xacro:if>
     </link>
+  </xacro:macro>
+  <xacro:macro name="standard_leg" params="parent self:=${self} *origin">
+      <xacro:extra_module name = "leg${self}" parent = "${parent}" visible = "1"
+                          model_url = "package://hydrus/urdf/mesh/modules/mechanical/standard_legs.dae" >
+        <xacro:insert_block name="origin" />
+        <inertial>
+          <!-- short leg:
+          <origin xyz="0.0 0.0 -0.055380" rpy="0 0 0"/>
+          <mass value="0.043000"/>
+          <inertia
+              ixx="0.000088" iyy="0.000088" izz="0.000000"
+              ixy="0.000000" ixz="0.000000" iyz="0.000000"/>
+          -->
+          <!-- standard leg: -->
+          <origin xyz="0.0 0.0 -0.0852" rpy="0 0 0"/>
+          <mass value="0.047000"/>
+          <inertia
+              ixx="0.000259" iyy="-0.000281" izz="0.000010"
+              ixy="0.000000" ixz="0.000000" iyz="0.000000"/>
+        </inertial>
+      </xacro:extra_module>
   </xacro:macro>
   <!-- friction -->

File: robots/hydrus/urdf/link.urdf.xacro (robot description, xacro)
@@ -3,19 +3,16 @@
     xmlns:xacro="http://www.ros.org/wiki/xacro" name="hydrusx_link" >
   <!-- D-H kai description(different from prof.nakamura) -->
-  <xacro:macro name="hydrusx_link" params="self child rotor_direction">
+  <xacro:macro name="hydrusx_link" params="self child rotor_direction with_leg:=1 with_battery:=1">
     <!-- link -->
     <link name="link${self}">
-      <!-- common inertial -->
-      <inertial>
-        <origin xyz="${link_length* 0.5} 0 0" rpy="0 0 0"/>
-        <mass value="${link_rod_mass + link_center_mass + protector_mass + protector_holder_mass - rotor_mass}" /> <!-- exclude from center mass -->
-        <inertia
-            ixx="${protector_inertia / 2}" ixy="0.0" ixz="0.0"
-            iyy="${link_rod_inertia + protector_holder_inertia + protector_inertia /2}" iyz="0.0"
-            izz="${link_rod_inertia + protector_holder_inertia + protector_inertia}"/>
-      </inertial>
-      <!-- sepcial inertia & visual & collision -->
       <!-- head -->
       <xacro:if value="${self == 1}">
+        <inertial>
+          <origin xyz="${link_length* 0.5 + 0.055120} 0.0 0.011580" rpy="0 0 0"/>
+          <mass value="0.566650"/>
+          <inertia
+              ixx="0.001804" iyy="0.017972" izz="0.019248"
+              ixy="0.000021" ixz="0.000372" iyz="0.000000"/>
+        </inertial>
         <xacro:link_model type="head" />
       </xacro:if>
@@ -23,9 +20,23 @@
         <!-- tail -->
         <xacro:if value="${self == child}">
+          <inertial>
+            <origin xyz="${link_length * 0.5 + -0.013450} 0.0 0.012830" rpy="0 0 0"/>
+            <mass value="0.495530"/>
+            <inertia
+                ixx="0.001758" iyy="0.013619" izz="0.014910"
+                ixy="0.000020" ixz="-0.000076" iyz="0.000000"/>
+          </inertial>
           <xacro:link_model type="end" />
         </xacro:if>
         <xacro:unless value="${self == child}">
           <!-- general -->
-            <xacro:link_model type="general" />
+          <inertial>
+            <origin xyz="${link_length * 0.5 + 0.038190} 0.0 0.010950" rpy="0 0 0"/>
+            <mass value="0.597720"/>
+            <inertia
+                ixx="0.001828" iyy="0.021127" izz="0.022388"
+                ixy="0.000021" ixz="0.000260" iyz="0.000000"/>
+          </inertial>
+          <xacro:link_model type="general" />
         </xacro:unless>
       </xacro:unless>
@@ -44,32 +55,65 @@
       <inertial>
         <origin xyz="0 0 0" rpy="0 0 0"/>
-        <mass value="${rotor_mass}"/>
+        <mass value="0.0001"/>
         <inertia
-            ixx="${rotor_mass * .25 * rotor_radius * rotor_radius}" ixy="0.0" ixz="0.0"
-            iyy="${rotor_mass * .25 * rotor_radius * rotor_radius}" iyz="0.0"
-            izz="${rotor_mass * .5 * rotor_radius * rotor_radius}"/>
+            ixx="0.00001" ixy="0.0" ixz="0.0"
+            iyy="0.00001" iyz="0.0"
+            izz="0.00002"/>
       </inertial>
       <collision>
-        <origin rpy="0 0 0" xyz="0 0 ${collision_model_z_offset}"/>
+        <origin rpy="0 0 0" xyz="0 0 0"/>
         <geometry>
-          <cylinder length="${collision_model_height}" radius="${protector_radius + 0.01}"/>
+          <cylinder length="0.1" radius="${protector_radius + 0.01}"/>
         </geometry>
-        </collision>
+      </collision>
     </link>
     <xacro:damping_factor link ="thrust${self}"/>
-    <!-- battery -->
-    <xacro:extra_module name = "bat${self}" parent = "link${self}" >
-      <origin xyz="${link_length/2 + bat_offset} 0.0 -0.054" rpy="0 0 0"/>
-      <inertial>
-        <origin xyz="0 0 0" rpy="0 0 0"/>
-        <mass value="${bat_mass}"/>
-        <inertia
-          ixx="0.00001" ixy="0.0" ixz="0.0"
-          iyy="0.00001" iyz="0.0"
-          izz="0.00002"/>
-      </inertial>
-    </xacro:extra_module>
-    <!-- extra module -->
-    <!-- head -->
+    <!-- battery: -->
+    <!-- use default battery: -->
+    <xacro:if value="${with_battery == 1}">
+      <xacro:extra_module name = "bat${self}" parent = "link${self}" visible = "1"
+                          model_url = "package://hydrus/urdf/mesh/modules/battery/VOLTON-PG-1300LP2-6s.stl" scale="0.001">
+        <origin xyz="${link_length/2} 0.0 -0.048" rpy="${pi/2} 0 0"/>
+        <inertial>
+          <origin xyz="0 0 0" rpy="0 0 0"/>
+          <mass value="0.194"/>
+          <inertia
+              ixx="0.00012" ixy="0.00005" ixz="0.00011"
+              iyy="0.0" iyz="0.0"
+              izz="0.0"/>
+        </inertial>
+      </xacro:extra_module>
+    </xacro:if>
+    <!-- leg -->
+    <xacro:if value="${with_leg == 1}">
+      <!-- head -->
+      <xacro:if value="${self == 1}">
+        <xacro:standard_leg parent = "link${self}" >
+          <origin xyz="${head_leg_offset} 0.0 0" rpy="0 0 0"/>
+        </xacro:standard_leg>
+      </xacro:if>
+      <xacro:unless value="${self == 1}">
+        <xacro:standard_leg parent = "link${self}" >
+          <origin xyz="${general_leg_offset} 0.0 0" rpy="0 0 0"/>
+        </xacro:standard_leg>
+        <!-- tail -->
+        <xacro:if value="${self == child}">
+          <xacro:standard_leg parent = "link${self}" self= "${self + 1}" >
+            <origin xyz="${end_leg_offset} 0.0 0" rpy="0 0 0"/>
+          </xacro:standard_leg>
+        </xacro:if>
+      </xacro:unless>
+    </xacro:if>
+    <!-- joint -->
+    <xacro:unless value="${self == child}">
+      <joint name="joint${self}" type="revolute">
+        <limit effort="10.0" lower="-1.57" upper="1.57" velocity="0.5"/>
+        <parent link="link${self}"/>
+        <child link="link${child}"/>
+        <origin rpy="0 0 0" xyz="${link_length} 0 0"/>
+        <axis xyz="0 0 1"/>
+        <dynamics damping="0.9" friction="0.05"/>
+      </joint>
+    </xacro:unless>
     <xacro:if value="${self == 1}">
       <!-- dummy root link for KDL -->
@@ -90,52 +134,5 @@
         <axis xyz="0 0 1"/>
       </joint>
-      <xacro:extra_module name = "head_leg" parent = "link${self}" >
-        <origin xyz="${link_length * 0.5 + head_leg_offset} 0.0 -0.03" rpy="0 0 0"/>
-        <inertial>
-          <mass value="${head_leg_mass}"/>
-          <origin xyz="0.0 0.0 0.0" rpy="0 0 0"/>
-          <inertia
-              ixx="0.000001" ixy="0.0" ixz="0.0"
-              iyy="0.000001" iyz="0.0"
-              izz="0.000002"/>
-        </inertial>
-      </xacro:extra_module>
     </xacro:if>
-    <!-- tail -->
-    <xacro:if value="${self == child}">
-      <xacro:extra_module name = "end_leg" parent = "link${self}" >
-        <origin xyz="${link_length * 0.5 + end_leg_offset} 0.0 -0.03" rpy="0 0 0"/>
-        <inertial>
-          <mass value="${end_leg_mass}"/>
-          <origin xyz="0.0 0.0 0.0" rpy="0 0 0"/>
-          <inertia
-              ixx="0.000001" ixy="0.0" ixz="0.0"
-              iyy="0.000001" iyz="0.0"
-              izz="0.000002"/>
-        </inertial>
-      </xacro:extra_module>
-    </xacro:if>
-    <!-- joint -->>
-    <xacro:unless value="${self == child}">
-      <joint name="joint${self}" type="revolute">
-        <limit effort="3.1" lower="-1.6" upper="1.6" velocity="0.5"/>
-        <parent link="link${self}"/>
-        <child link="link${child}"/>
-        <origin rpy="0 0 0" xyz="${link_length} 0 0"/>
-        <axis xyz="0 0 1"/>
-        <dynamics damping="0.8" friction="0.05"/>
-      </joint>
-      <xacro:extra_module name = "joint${self}_module" parent = "link${self}" >
-        <origin xyz="${link_length * 0.5 + link_joint_offset} 0.0 0.0" rpy="0 0 0"/>
-        <inertial>
-          <mass value="${joint_mass}"/>
-          <origin xyz="0.0 0.0 0.0" rpy="0 0 0"/>
-          <inertia
-              ixx="0.000001" ixy="0.0" ixz="0.0"
-              iyy="0.000001" iyz="0.0"
-              izz="0.000002"/>
-        </inertial>
-      </xacro:extra_module>
-</xacro:unless>
     <!-- hardware interface -->
     <xacro:unless value="${self == child}">

Commit message: Add leddar one range sensor (altimeter) for hydrus (quad tx2 zed type), and set the altitude estimation (imu + range sensor) to be active as default.

File: robots/hydrus/robots/quad/tx2_zed_201810.urdf.xacro (robot description, xacro)
@@ -38,4 +38,16 @@
           iyy="0.000001" iyz="0.0"
           izz="0.000002"/>
+    </inertial>
+  </xacro:extra_module>
+  <!-- leddar one -->
+  <xacro:extra_module name = "leddarone" parent = "link3" visible = "1"
+                      model_url = "package://hydrus/urdf/mesh/modules/sensor/leddar_one_tx2_attached_mode.dae">
+    <origin xyz="0.0866 0.0 -0.06267" rpy="0 ${pi} 0"/>
+    <inertial>
+      <origin xyz="-0.007950 0.000000 -0.000140" rpy="0 0 0"/>
+      <mass value="0.029000"/>
+      <inertia
+          ixx="0.000010" iyy="0.000008" izz="0.000008"
+          ixy="0.000000" ixz="0.000000" iyz="0.000000"/>
     </inertial>
   </xacro:extra_module>

Commit message: Update the battert arrangement for hydrus quad model with tx2 + zed mini

File: robots/hydrus/robots/quad/tx2_zed_201810.urdf.xacro (robot description, xacro)
@@ -3,5 +3,33 @@
     xmlns:xacro="http://www.ros.org/wiki/xacro" name="hydrusx" >
   <!-- basic kinematics model -->
-  <xacro:include filename="$(find hydrus)/robots/quad/default.urdf.xacro" />
+  <xacro:include filename="$(find hydrus)/urdf/common.xacro" />
+  <xacro:include filename="$(find hydrus)/urdf/link.urdf.xacro" />
+  <xacro:hydrusx_link self="1" child="2" rotor_direction="-1" with_battery = "0" />
+  <xacro:hydrusx_link self="2" child="3" rotor_direction="1"  with_battery = "0" />
+  <xacro:hydrusx_link self="3" child="4" rotor_direction="-1" with_battery = "0" />
+  <xacro:hydrusx_link self="4" child="4" rotor_direction="1"  with_battery = "0"/>
+  <!-- special battery arrangement -->
+  <xacro:extra_module name = "bat1" parent = "link1" visible = "1"
+                      model_url = "package://hydrus/urdf/mesh/modules/battery/Kypom-3000-6s.stl" scale="0.001">
+    <origin xyz="${link_length/2} 0.0 -0.048" rpy="${pi/2} 0 0"/>
+    <inertial>
+      <origin xyz="0 0 0" rpy="0 0 0"/>
+      <mass value="0.4108"/>
+      <inertia
+          ixx="0.0001" iyy="0.0006" izz="0.0006"
+          ixy="0.0" ixz="0.0"  iyz="0.0"/>
+    </inertial>
+  </xacro:extra_module>
+  <xacro:extra_module name = "bat2" parent = "link4" visible = "1"
+                      model_url = "package://hydrus/urdf/mesh/modules/battery/Kypom-3000-6s.stl" scale="0.001">
+    <origin xyz="${link_length/2} 0.0 -0.048" rpy="${pi/2} 0 0"/>
+    <inertial>
+      <origin xyz="0 0 0" rpy="0 0 0"/>
+      <mass value="0.4108"/>
+      <inertia
+          ixx="0.0001" iyy="0.0006" izz="0.0006"
+          ixy="0.0" ixz="0.0"  iyz="0.0"/>
+    </inertial>
+  </xacro:extra_module>
   <!-- oboard sensors and processors -->
   <xacro:include filename="$(find hydrus)/robots/onboards/tx2_zed_201810/onboards.urdf.xacro" />
