Commit message: add hydrus_xi xavier models remove hydrus_xi euclid models

File: robots/hydrus_xi/robots/hex/xavier201811.gazebo.xacro (robot description, xacro)
@@ -2,5 +2,5 @@
 <robot
     xmlns:xacro="http://www.ros.org/wiki/xacro" name="hydrus_xi" >
-  <xacro:include filename="$(find hydrus_xi)/robots/quad/euclid201806.urdf.xacro" />
+  <xacro:include filename="$(find hydrus_xi)/robots/hex/xavier201811.urdf.xacro" />
   <!-- gazebo -->
   <xacro:include filename="$(find hydrus_xi)/robots/default.gazebo.xacro" />

File: robots/hydrus_xi/robots/hex/xavier201811.urdf.xacro (robot description, xacro)
@@ -16,16 +16,15 @@
     </inertial>
   </xacro:extra_module>
-  <!-- processor: euclid -->
-  <!-- <xacro:extra_module name = "pc" parent = "link2" visible = "1" -->
-  <!--                     model_url = "package://hydrus/urdf/mesh/modules/processor/intel_euclid_201806.dae"> -->
-  <!--   <origin xyz="${link_length/2 + 0.1565 + 0.063} 0.0 -0.0394" rpy="0 0 ${-pi/2}"/> -->
-  <!--   <inertial> -->
-  <!--     <mass value = "0.164" /> -->
-  <!--     <origin xyz="${0.03*0.001} ${0.72*0.001} ${2.9 * 0.001}" rpy="0 0 0"/> -->
-  <!--     <inertia -->
-  <!--         ixx="0.00001" ixy="0.0" ixz="0.0" -->
-  <!--         iyy="0.00001" iyz="0.0" -->
-  <!--         izz="0.00002"/> -->
-  <!--   </inertial> -->
-  <!-- </xacro:extra_module> -->
+  <xacro:extra_module name = "pc" parent = "link3" visible = "1"
+                      model_url = "package://hydrus_xi/urdf/mesh/modules/pc/xavier.dae">
+    <origin xyz="0.47375 0.0 -0.0805" rpy="0 0 0"/>
+    <inertial>
+      <mass value = "0.559" />
+      <origin xyz="-0.00086 -0.00012 0.02982" rpy="0 0 0"/>
+      <inertia
+          ixx="0.00001" ixy="0.0" ixz="0.0"
+          iyy="0.00001" iyz="0.0"
+          izz="0.00002"/>
+    </inertial>
+  </xacro:extra_module>
 </robot>

File: robots/hydrus_xi/robots/quad/xavier201811.gazebo.xacro (robot description, xacro)
@@ -2,5 +2,5 @@
 <robot
     xmlns:xacro="http://www.ros.org/wiki/xacro" name="hydrus_xi" >
-  <xacro:include filename="$(find hydrus_xi)/robots/hex/euclid201806.urdf.xacro" />
+  <xacro:include filename="$(find hydrus_xi)/robots/quad/xavier201811.urdf.xacro" />
   <!-- gazebo -->
   <xacro:include filename="$(find hydrus_xi)/robots/default.gazebo.xacro" />

File: robots/hydrus_xi/robots/quad/xavier201811.urdf.xacro (robot description, xacro)
@@ -16,16 +16,16 @@
     </inertial>
   </xacro:extra_module>
-  <!-- processor: euclid -->
-  <!-- <xacro:extra_module name = "pc" parent = "link2" visible = "1" -->
-  <!--                     model_url = "package://hydrus/urdf/mesh/modules/processor/intel_euclid_201806.dae"> -->
-  <!--   <origin xyz="${link_length/2 + 0.1565 + 0.063} 0.0 -0.0394" rpy="0 0 ${-pi/2}"/> -->
-  <!--   <inertial> -->
-  <!--     <mass value = "0.164" /> -->
-  <!--     <origin xyz="${0.03*0.001} ${0.72*0.001} ${2.9 * 0.001}" rpy="0 0 0"/> -->
-  <!--     <inertia -->
-  <!--         ixx="0.00001" ixy="0.0" ixz="0.0" -->
-  <!--         iyy="0.00001" iyz="0.0" -->
-  <!--         izz="0.00002"/> -->
-  <!--   </inertial> -->
-  <!-- </xacro:extra_module> -->
+  #### processor: xavier ####
+  <xacro:extra_module name = "pc" parent = "link2" visible = "1"
+                      model_url = "package://hydrus_xi/urdf/mesh/modules/pc/xavier.dae">
+    <origin xyz="0.47375 0.0 -0.0805" rpy="0 0 0"/>
+    <inertial>
+      <mass value = "0.559" />
+      <origin xyz="-0.00086 -0.00012 0.02982" rpy="0 0 0"/>
+      <inertia
+          ixx="0.00001" ixy="0.0" ixz="0.0"
+          iyy="0.00001" iyz="0.0"
+          izz="0.00002"/>
+    </inertial>
+  </xacro:extra_module>
 </robot>

File: robots/hydrus_xi/urdf/common.xacro (robot description, xacro)
@@ -11,4 +11,5 @@
   <!-- mass [Kg] -->
   <xacro:property name="rotor_mass" value="0.02"/> <!-- exclude from center mass -->
+  <xacro:property name="bat_mass" value="0.193"/> <!-- 1300mAh -->
   <!-- dynamics -->
   <xacro:property name="max_force" value="24"/> <!-- [N] -->

File: robots/hydrus_xi/urdf/link.urdf.xacro (robot description, xacro)
@@ -145,4 +145,16 @@
       <axis xyz="0 0 ${rotor_direction}"/>
     </joint>
+    #### battery ####
+    <xacro:extra_module name="bat${self}" parent="link${self}" >
+      <origin xyz="0.3133 0.0 -0.048" rpy="0 0 0"/>
+      <inertial>
+        <origin xyz="0 0 0" rpy="0 0 0"/>
+        <mass value="${bat_mass}"/>
+        <inertia
+          ixx="0.00001" ixy="0.0" ixz="0.0"
+          iyy="0.00001" iyz="0.0"
+          izz="0.00002"/>
+      </inertial>
+    </xacro:extra_module>
     #### hardware interface ####
     <xacro:unless value="${self == child}">
