Commit message: fix hydrus_xi link.urdf.xacro (squash into ef02)

File: robots/hydrus_xi/robots/hex/default.urdf.xacro (robot description, xacro)
@@ -4,9 +4,9 @@
   <xacro:include filename="$(find hydrus_xi)/urdf/common.xacro" />
   <xacro:include filename="$(find hydrus_xi)/urdf/link.urdf.xacro" />
-  <xacro:hydrus_xi_link self="1" child="2" rotor_direction="-1" link_type="head"/>
-  <xacro:hydrus_xi_link self="2" child="3" rotor_direction="1"  link_type="general"/>
-  <xacro:hydrus_xi_link self="3" child="4" rotor_direction="-1" link_type="general"/>
-  <xacro:hydrus_xi_link self="4" child="5" rotor_direction="1"  link_type="general"/>
-  <xacro:hydrus_xi_link self="5" child="6" rotor_direction="-1" link_type="general"/>
-  <xacro:hydrus_xi_link self="6" child="6" rotor_direction="1"  link_type="end"/>
+  <xacro:hydrus_xi_link self="1" child="2" rotor_direction="1" link_type="head"/>
+  <xacro:hydrus_xi_link self="2" child="3" rotor_direction="-1"  link_type="general"/>
+  <xacro:hydrus_xi_link self="3" child="4" rotor_direction="1" link_type="general"/>
+  <xacro:hydrus_xi_link self="4" child="5" rotor_direction="-1"  link_type="general"/>
+  <xacro:hydrus_xi_link self="5" child="6" rotor_direction="1" link_type="general"/>
+  <xacro:hydrus_xi_link self="6" child="6" rotor_direction="-1"  link_type="end"/>
 </robot>

File: robots/hydrus_xi/urdf/link.urdf.xacro (robot description, xacro)
@@ -126,5 +126,5 @@
       <parent link="link${self}"/>
       <child link="gimbal_link${self}"/>
-      <origin rpy="0 0 0" xyz="0.3016 0 0.05967"/>
+      <origin rpy="0 0 3.14159" xyz="0.3016 0 0.05967"/>
       <axis xyz="0 0 1"/>
       <dynamics damping="0.8" friction="0.05"/>
