Commit message: remove battery and PC

File: robots/hydrus_xi/robots/hex/xavier201811.urdf.xacro (robot description, xacro)
@@ -16,15 +16,15 @@
     </inertial>
   </xacro:extra_module>
-  <xacro:extra_module name = "pc" parent = "link3" visible = "1"
-                      model_url = "package://hydrus_xi/urdf/mesh/modules/pc/xavier.dae">
-    <origin xyz="0.47375 0.0 -0.0805" rpy="0 0 0"/>
-    <inertial>
-      <mass value = "0.559" />
-      <origin xyz="-0.00086 -0.00012 0.02982" rpy="0 0 0"/>
-      <inertia
-          ixx="0.00001" ixy="0.0" ixz="0.0"
-          iyy="0.00001" iyz="0.0"
-          izz="0.00002"/>
-    </inertial>
-  </xacro:extra_module>
+  <!-- <xacro:extra_module name = "pc" parent = "link3" visible = "1" -->
+  <!--                     model_url = "package://hydrus_xi/urdf/mesh/modules/pc/xavier.dae"> -->
+  <!--   <origin xyz="0.47375 0.0 -0.0805" rpy="0 0 0"/> -->
+  <!--   <inertial> -->
+  <!--     <mass value = "0.559" /> -->
+  <!--     <origin xyz="-0.00086 -0.00012 0.02982" rpy="0 0 0"/> -->
+  <!--     <inertia -->
+  <!--         ixx="0.00001" ixy="0.0" ixz="0.0" -->
+  <!--         iyy="0.00001" iyz="0.0" -->
+  <!--         izz="0.00002"/> -->
+  <!--   </inertial> -->
+  <!-- </xacro:extra_module> -->
 </robot>

File: robots/hydrus_xi/urdf/link.urdf.xacro (robot description, xacro)
@@ -146,15 +146,15 @@
     </joint>
     #### battery ####
-    <xacro:extra_module name="bat${self}" parent="link${self}" >
-      <origin xyz="0.3133 0.0 -0.048" rpy="0 0 0"/>
-      <inertial>
-        <origin xyz="0 0 0" rpy="0 0 0"/>
-        <mass value="${bat_mass}"/>
-        <inertia
-          ixx="0.00001" ixy="0.0" ixz="0.0"
-          iyy="0.00001" iyz="0.0"
-          izz="0.00002"/>
-      </inertial>
-    </xacro:extra_module>
+    <!-- <xacro:extra_module name="bat${self}" parent="link${self}" > -->
+    <!--   <origin xyz="0.3133 0.0 -0.048" rpy="0 0 0"/> -->
+    <!--   <inertial> -->
+    <!--     <origin xyz="0 0 0" rpy="0 0 0"/> -->
+    <!--     <mass value="${bat_mass}"/> -->
+    <!--     <inertia -->
+    <!--       ixx="0.00001" ixy="0.0" ixz="0.0" -->
+    <!--       iyy="0.00001" iyz="0.0" -->
+    <!--       izz="0.00002"/> -->
+    <!--   </inertial> -->
+    <!-- </xacro:extra_module> -->
     #### hardware interface ####
     <xacro:unless value="${self == child}">

Commit message: Revert "remove battery and PC"
This reverts commit e8f39c0f715d09e0f7afa78034c96c4c9d811e78.

File: robots/hydrus_xi/robots/hex/xavier201811.urdf.xacro (robot description, xacro)
@@ -16,15 +16,15 @@
     </inertial>
   </xacro:extra_module>
-  <!-- <xacro:extra_module name = "pc" parent = "link3" visible = "1" -->
-  <!--                     model_url = "package://hydrus_xi/urdf/mesh/modules/pc/xavier.dae"> -->
-  <!--   <origin xyz="0.47375 0.0 -0.0805" rpy="0 0 0"/> -->
-  <!--   <inertial> -->
-  <!--     <mass value = "0.559" /> -->
-  <!--     <origin xyz="-0.00086 -0.00012 0.02982" rpy="0 0 0"/> -->
-  <!--     <inertia -->
-  <!--         ixx="0.00001" ixy="0.0" ixz="0.0" -->
-  <!--         iyy="0.00001" iyz="0.0" -->
-  <!--         izz="0.00002"/> -->
-  <!--   </inertial> -->
-  <!-- </xacro:extra_module> -->
+  <xacro:extra_module name = "pc" parent = "link3" visible = "1"
+                      model_url = "package://hydrus_xi/urdf/mesh/modules/pc/xavier.dae">
+    <origin xyz="0.47375 0.0 -0.0805" rpy="0 0 0"/>
+    <inertial>
+      <mass value = "0.559" />
+      <origin xyz="-0.00086 -0.00012 0.02982" rpy="0 0 0"/>
+      <inertia
+          ixx="0.00001" ixy="0.0" ixz="0.0"
+          iyy="0.00001" iyz="0.0"
+          izz="0.00002"/>
+    </inertial>
+  </xacro:extra_module>
 </robot>

File: robots/hydrus_xi/urdf/link.urdf.xacro (robot description, xacro)
@@ -146,15 +146,15 @@
     </joint>
     #### battery ####
-    <!-- <xacro:extra_module name="bat${self}" parent="link${self}" > -->
-    <!--   <origin xyz="0.3133 0.0 -0.048" rpy="0 0 0"/> -->
-    <!--   <inertial> -->
-    <!--     <origin xyz="0 0 0" rpy="0 0 0"/> -->
-    <!--     <mass value="${bat_mass}"/> -->
-    <!--     <inertia -->
-    <!--       ixx="0.00001" ixy="0.0" ixz="0.0" -->
-    <!--       iyy="0.00001" iyz="0.0" -->
-    <!--       izz="0.00002"/> -->
-    <!--   </inertial> -->
-    <!-- </xacro:extra_module> -->
+    <xacro:extra_module name="bat${self}" parent="link${self}" >
+      <origin xyz="0.3133 0.0 -0.048" rpy="0 0 0"/>
+      <inertial>
+        <origin xyz="0 0 0" rpy="0 0 0"/>
+        <mass value="${bat_mass}"/>
+        <inertia
+          ixx="0.00001" ixy="0.0" ixz="0.0"
+          iyy="0.00001" iyz="0.0"
+          izz="0.00002"/>
+      </inertial>
+    </xacro:extra_module>
     #### hardware interface ####
     <xacro:unless value="${self == child}">
