Commit message: Update the configurarion regarding to egomotion estimation for following models: - quad - hex - hex_branch (default mode) - hex_branch with hokuyo

File: robots/hydrus_xi/robots/hex_branch/xavier_hokuyo.urdf.xacro (robot description, xacro)
@@ -26,8 +26,45 @@
     </inertial>
   </xacro:extra_module>
+  <!-- zed mini setero -->
+  <xacro:extra_module name = "zed_camera_center" parent = "center_link" visible = "1"
+                      model_url = "package://hydrus_xi/urdf/mesh/sensor/zed_mini.dae">
+    <origin xyz="0.05504 0.09534  0.029" rpy="0 0 ${pi/3}"/>
+    <inertial>
+      <origin xyz="0.000430 0.006110 0.000000" rpy="0 0 0"/>
+      <mass value="0.090000"/>
+      <inertia
+          ixx="0.000117" iyy="0.000010" izz="0.000117"
+          ixy="0.000000" ixz="0.000000" iyz="0.000000"/>
+    </inertial>
+  </xacro:extra_module>
+  <!-- leddar one -->
+  <xacro:extra_module name = "leddar_one" parent = "center_link" visible = "1"
+                      model_url = "package://hydrus_xi/urdf/mesh/sensor/leddar_one.dae">
+    <origin xyz="0.082 0.0 -0.027" rpy="0 ${pi} ${-pi/2}"/>
+    <inertial>
+      <origin xyz="0.000000 -0.009700 -0.004610" rpy="0 0 0"/>
+      <mass value="0.028000"/>
+      <inertia
+          ixx="0.000007" iyy="0.000009" izz="0.000007"
+          ixy="0.000000" ixz="0.000000" iyz="0.000001"/>
+    </inertial>
+  </xacro:extra_module>
   <!-- Hokuyo UST-20LX -->
+  <!-- https://www.hokuyo-aut.co.jp/search/single.php?serial=16 -->
   <xacro:include filename="$(find hydrus_xi)/robots/sensor/hokuyo_ust20lx.urdf.xacro" />
   <xacro:hokuyo_ust20lx name="laser" parent="center_link" ros_topic="scan" update_rate="40" ray_count="1081" min_angle="-135" max_angle="135">
-    <origin xyz="0.0 0.0 0.250" rpy="0 0 ${pi}"/>
+    <origin xyz="0.0 0.0 ${0.220 + 0.01 + 0.0474}" rpy="0 0 ${pi}"/>
   </xacro:hokuyo_ust20lx>
+  <!-- gps -->
+  <xacro:extra_module name = "gps" parent = "center_link" visible = "1"
+                      model_url = "package://hydrus_xi/urdf/mesh/sensor/gps_m8nblox.dae">
+    <origin xyz="0.0 0.0 0.3" rpy="0 0 0"/>
+    <inertial>
+      <origin xyz="0.0 0.0 0.0" rpy="0 0 0"/>
+      <mass value="0.03"/>
+      <inertia
+          ixx="0.0" iyy="0.0" izz="0.0"
+          ixy="0.0" ixz="0.0" iyz="0.0"/>
+    </inertial>
+  </xacro:extra_module>
 </robot>

File: robots/hydrus_xi/robots/sensor/hokuyo_ust20lx.urdf.xacro (robot description, xacro)
@@ -10,5 +10,5 @@
       <inertial>
         <origin xyz="-0.000570 0.000005 -0.064301" rpy="0 0 0"/>
-        <mass value="0.210930"/>
+        <mass value="0.2568"/> <!-- old: 0.210930 -->
         <inertia
             ixx="0.002067" iyy="0.002077" izz="0.000470"
