Commit message: update center_link model

File: robots/hydrus_xi/robots/hex_branch/xavier201811.urdf.xacro (robot description, xacro)
@@ -6,5 +6,5 @@
   <xacro:extra_module name = "fc" parent = "center_link" visible = "1"
                       model_url = "package://hydrus_xi/urdf/mesh/modules/flight_controller/fc3.dae">
-    <origin xyz="-0.0129 -0.0169 0.04133" rpy="0 0 0"/>
+    <origin xyz="-0.0129 -0.0044 0.03933" rpy="0 0 0"/>
     <inertial>
       <origin xyz="0.012999 0.004396 -0.004856" rpy="0 0 0"/>
@@ -17,5 +17,5 @@
   <xacro:extra_module name = "pc" parent = "center_link" visible = "1"
                       model_url = "package://hydrus_xi/urdf/mesh/modules/pc/xavier_2.dae">
-    <origin xyz="-0.0005 0.0125 -0.0775" rpy="0 0 ${pi / 2.0}"/>
+    <origin xyz="-0.01075 0.0005 -0.0775" rpy="0 0 0"/>
     <inertial>
       <origin xyz="-0.000890 -0.000110 0.028700" rpy="0 0 0"/>

File: robots/hydrus_xi/urdf/branch_type_link.urdf.xacro (robot description, xacro)
@@ -37,24 +37,24 @@
     #### link joint ####
     <joint name="joint${child1}" type="revolute">
-      <limit effort="3.3" lower="-1.57" upper="1.57" velocity="0.5"/>
+      <limit effort="6.6" lower="-1.57" upper="1.57" velocity="0.5"/>
       <parent link="center_link"/>
       <child link="link${child1}"/>
-      <origin rpy="0 0 ${pi * 4.0 / 3.0}" xyz="-0.06275 -0.10869 0.016"/>
+      <origin rpy="0 0 0" xyz="0.1555 0.0 0.015"/>
       <axis xyz="0 0 1"/>
       <dynamics damping="0.8" friction="0.05"/>
     </joint>
     <joint name="joint${child2}" type="revolute">
-      <limit effort="3.3" lower="-1.57" upper="1.57" velocity="0.5"/>
+      <limit effort="6.6" lower="-1.57" upper="1.57" velocity="0.5"/>
       <parent link="center_link"/>
       <child link="link${child2}"/>
-      <origin rpy="0 0 0" xyz="0.1255 0 0.016"/>
+      <origin rpy="0 0 ${pi * 2.0 / 3.0}" xyz="-0.07775 0.13467 0.015"/>
       <axis xyz="0 0 1"/>
       <dynamics damping="0.8" friction="0.05"/>
     </joint>
     <joint name="joint${child3}" type="revolute">
-      <limit effort="3.3" lower="-1.57" upper="1.57" velocity="0.5"/>
+      <limit effort="6.6" lower="-1.57" upper="1.57" velocity="0.5"/>
       <parent link="center_link"/>
       <child link="link${child3}"/>
-      <origin rpy="0 0 ${pi * 2.0 / 3.0}" xyz="-0.06275 0.10869 0.016"/>
+      <origin rpy="0 0 ${pi * 4.0 / 3.0}" xyz="-0.07775 -0.13467 0.015"/>
       <axis xyz="0 0 1"/>
       <dynamics damping="0.8" friction="0.05"/>

Commit message: Modify xavier201811 sensor config

File: robots/hydrus_xi/robots/hex_branch/xavier201811.urdf.xacro (robot description, xacro)
@@ -26,3 +26,27 @@
     </inertial>
   </xacro:extra_module>
+  <!-- zed mini setero -->
+  <xacro:extra_module name = "zed_camera_center" parent = "center_link" visible = "1"
+                      model_url = "package://hydrus_xi/urdf/mesh/sensor/zed_mini.dae">
+    <origin xyz="0.05504 0.09534  0.029" rpy="0 0 ${pi/3}"/>
+    <inertial>
+      <origin xyz="0.000430 0.006110 0.000000" rpy="0 0 0"/>
+      <mass value="0.090000"/>
+      <inertia
+          ixx="0.000117" iyy="0.000010" izz="0.000117"
+          ixy="0.000000" ixz="0.000000" iyz="0.000000"/>
+    </inertial>
+  </xacro:extra_module>
+  <!-- leddar one -->
+  <xacro:extra_module name = "leddarone" parent = "center_link" visible = "1"
+                      model_url = "package://hydrus_xi/urdf/mesh/sensor/leddar_one.dae">
+    <origin xyz="0.082 0.0 -0.027" rpy="0 ${pi} ${-pi/2}"/>
+    <inertial>
+      <origin xyz="0.000000 -0.009700 -0.004610" rpy="0 0 0"/>
+      <mass value="0.028000"/>
+      <inertia
+          ixx="0.000007" iyy="0.000009" izz="0.000007"
+          ixy="0.000000" ixz="0.000000" iyz="0.000001"/>
+    </inertial>
+  </xacro:extra_module>
 </robot>
