Commit message: Fix the wrong "arg" assignment: simulation -> real_machine for sensors.launch.includes

File: robots/hydrus/robots/hex/euclid201806.urdf.xacro (robot description, xacro)
@@ -34,5 +34,5 @@
     <inertial>
       <mass value = "0.164" />
-      <origin xyz="${0.03*0.001} ${0.72*0.001} ${2.9 * 0.0001}" rpy="0 0 0"/>
+      <origin xyz="${0.03*0.001} ${0.72*0.001} ${2.9 * 0.001}" rpy="0 0 0"/>
       <inertia
           ixx="0.00001" ixy="0.0" ixz="0.0"

File: robots/hydrus/robots/quad/euclid201806.urdf.xacro (robot description, xacro)
@@ -47,5 +47,5 @@
     <inertial>
       <mass value = "0.164" />
-      <origin xyz="${0.03*0.001} ${0.72*0.001} ${2.9 * 0.0001}" rpy="0 0 0"/>
+      <origin xyz="${0.03*0.001} ${0.72*0.001} ${2.9 * 0.001}" rpy="0 0 0"/>
       <inertia
           ixx="0.00001" ixy="0.0" ixz="0.0"

Commit message: Update the fc urdf model for hydrus minor model (hex + intel euclid, quad + intel euclid)

File: robots/hydrus/robots/hex/euclid201806.urdf.xacro (robot description, xacro)
@@ -7,8 +7,8 @@
   <xacro:extra_module name = "fc" parent = "link3" visible = "1"
                       model_url = "package://hydrus/urdf/mesh/modules/flight_controller/fc_euclid201806.dae">
-    <origin xyz="${link_length/2 + 0.241} 0.0 0.0348" rpy="0 0 0"/>
+    <origin xyz="${link_length / 2 + 0.2281} ${-4.4*0.001} 0.03533" rpy="0 0 0"/>
     <inertial>
-      <mass value = "0.033" />
-      <origin xyz="0.0 0.0 -0.01" rpy="0 0 0"/>
+      <mass value = "0.05" />
+      <origin xyz="${11.48*0.001} ${4.3*0.001} ${-9.4*0.001}" rpy="0 0 0"/>
       <inertia
           ixx="0.00001" ixy="0.0" ixz="0.0"
@@ -17,6 +17,6 @@
     </inertial>
   </xacro:extra_module>
-  <xacro:extra_module name = "magnet" parent = "link3">
-    <origin xyz="${link_length/2 + 0.241} 0.0 0.0348" rpy="0 0 0"/>
+  <xacro:extra_module name = "magnet" parent = "fc">
+    <origin xyz="0.0 0.0 0.0" rpy="0 0 0"/>
     <inertial>
       <mass value = "0.00001" />

File: robots/hydrus/robots/quad/euclid201806.urdf.xacro (robot description, xacro)
@@ -7,8 +7,8 @@
   <xacro:extra_module name = "fc" parent = "link2" visible = "1"
                       model_url = "package://hydrus/urdf/mesh/modules/flight_controller/fc_euclid201806.dae">
-    <origin xyz="${link_length/2 + 0.2281} ${-4.4*0.001} 0.03533" rpy="0 0 0"/>
+    <origin xyz="${link_length / 2 + 0.2281} ${-4.4*0.001} 0.03533" rpy="0 0 0"/>
     <inertial>
-      <mass value = "0.0457" />
-      <origin xyz="${8.7*0.001} ${4.4*0.001} -0.01" rpy="0 0 0"/>
+      <mass value = "0.05" />
+      <origin xyz="${11.48*0.001} ${4.3*0.001} ${-9.4*0.001}" rpy="0 0 0"/>
       <inertia
           ixx="0.00001" ixy="0.0" ixz="0.0"
@@ -22,10 +22,9 @@
     <origin xyz="${link_length/2 + 0.206} 0.0 0.18" rpy="0 0 0"/>
     <inertial>
-      <mass value = "0.044" />
-      <origin xyz="0.0 0.0 -0.08" rpy="0 0 0"/>
+      <origin xyz="0.000000 0.000000 -0.062510" rpy="0 0 0"/>
+      <mass value="0.053000"/>
       <inertia
-          ixx="0.00001" ixy="0.0" ixz="0.0"
-          iyy="0.00001" iyz="0.0"
-          izz="0.00002"/>
+          ixx="0.000503" iyy="0.000503" izz="0.000010"
+          ixy="0.000000" ixz="0.000000" iyz="0.000000"/>
     </inertial>
   </xacro:extra_module>
