Commit message: add offset zed left camera

File: robots/hydrus/robots/onboards/tx2_zed_201810/onboards.gazebo.xacro (robot description, xacro)
@@ -6,5 +6,5 @@
   <!-- stereo camera: depth, color based on left camera -->
   <xacro:extra_module name = "zed_left_camera_frame" parent = "zed_camera_center">
-    <origin xyz="0 0.03 0" rpy="0 0 0"/>
+    <origin xyz="0.002 0.03 0" rpy="0 0 0"/>
     <inertial>
       <mass value = "0.00001" />

Commit message: Refactor the robot model with regard to hydrus - delete unnecessary hex type - merge the onboard module description into the robot urdf

File: robots/hydrus/robots/onboards/tx2_zed_201810/onboards.gazebo.xacro (robot description, xacro)
@@ -2,73 +2,3 @@
 <robot
     xmlns:xacro="http://www.ros.org/wiki/xacro" name="hydrusx" >
-  <!-- gazebo plugin for controller and common sensors -->
-  <xacro:include filename="$(find hydrus)/robots/default.gazebo.xacro" />
-  <!-- stereo camera: depth, color based on left camera -->
-  <xacro:extra_module name = "zed_left_camera_frame" parent = "zed_camera_center">
-    <origin xyz="0.002 0.03 0" rpy="0 0 0"/>
-    <inertial>
-      <mass value = "0.00001" />
-      <origin xyz="0 0 0" rpy="0 0 0"/>
-      <inertia
-          ixx="0.000001" ixy="0.0" ixz="0.0"
-          iyy="0.000001" iyz="0.0"
-          izz="0.000002"/>
-    </inertial>
-  </xacro:extra_module>
-  <xacro:extra_module name = "zed_left_camera_optical_frame" parent = "zed_left_camera_frame">
-    <origin xyz="0 0 0" rpy="${-pi / 2} 0 ${-pi / 2}"/>
-    <inertial>
-      <mass value = "0.00001" />
-      <origin xyz="0 0 0" rpy="0 0 0"/>
-      <inertia
-          ixx="0.000001" ixy="0.0" ixz="0.0"
-          iyy="0.000001" iyz="0.0"
-          izz="0.000002"/>
-    </inertial>
-  </xacro:extra_module>
-  <gazebo reference="zed_left_camera_frame">
-    <sensor type="depth" name="zed_depth_camera">
-      <update_rate>20.0</update_rate>
-      <camera name="head">
-        <horizontal_fov>1.57</horizontal_fov>
-        <image>
-          <width>1280</width>
-          <height>720</height>
-          <format>RGB</format>
-        </image>
-        <clip>
-          <near>0.02</near>
-          <far>300</far>
-        </clip>
-        <noise>
-          <type>gaussian</type>
-          <mean>0.0</mean>
-          <stddev>0.007</stddev>
-        </noise>
-      </camera>
-      <plugin name="depth_camera" filename="libgazebo_ros_openni_kinect.so">
-        <baseline>0.06</baseline>
-        <alwaysOn>true</alwaysOn>
-        <updateRate>0.0</updateRate>
-        <cameraName>zed</cameraName>
-        <imageTopicName>rgb/image_rect_color</imageTopicName>
-        <cameraInfoTopicName>rgb/camera_info</cameraInfoTopicName>
-        <depthImageTopicName>depth/depth_registered</depthImageTopicName>
-        <depthImageInfoTopicName>depth/camera_info</depthImageInfoTopicName>
-        <pointCloudTopicName>point_cloud/cloud_registered</pointCloudTopicName>
-        <frameName>zed_left_camera_optical_frame</frameName>
-        <pointCloudCutoff>0.05</pointCloudCutoff>
-        <distortionK1>0</distortionK1>
-        <distortionK2>0</distortionK2>
-        <distortionK3>0</distortionK3>
-        <distortionT1>0</distortionT1>
-        <distortionT2>0</distortionT2>
-        <CxPrime>0</CxPrime>
-        <Cx>0</Cx>
-        <Cy>0</Cy>
-        <focalLength>0</focalLength>
-        <hackBaseline>0</hackBaseline>
-      </plugin>
-    </sensor>
-  </gazebo>
 </robot>
