Commit message: Update the hydrus model (old version: joint with MX28AR)

File: robots/hydrus/robots/quad/tx2_zed_201810/robot.urdf.xacro (robot description, xacro)
@@ -11,6 +11,6 @@
   <!-- special battery arrangement -->
   <xacro:extra_module name = "bat1" parent = "link1" visible = "1"
-                      model_url = "package://hydrus/urdf/mesh/modules/battery/Kypom-3000-6s.stl" scale="0.001">
-    <origin xyz="${link_length/2} 0.0 -0.048" rpy="${pi/2} 0 0"/>
+                      model_url = "package://hydrus/urdf/mesh/battery/Kypom-3000-6s.dae" >
+    <origin xyz="${link_length/2} 0.0 -0.048" rpy="0 0 0"/>
     <inertial>
       <origin xyz="0 0 0" rpy="0 0 0"/>
@@ -22,6 +22,6 @@
   </xacro:extra_module>
   <xacro:extra_module name = "bat2" parent = "link4" visible = "1"
-                      model_url = "package://hydrus/urdf/mesh/modules/battery/Kypom-3000-6s.stl" scale="0.001">
-    <origin xyz="${link_length/2} 0.0 -0.048" rpy="${pi/2} 0 0"/>
+                      model_url = "package://hydrus/urdf/mesh/battery/Kypom-3000-6s.dae" >
+    <origin xyz="${link_length/2} 0.0 -0.048" rpy="0 0 0"/>
     <inertial>
       <origin xyz="0 0 0" rpy="0 0 0"/>
@@ -36,5 +36,5 @@
   <!-- 1.1 flight controller -->
   <xacro:extra_module name = "fc" parent = "link2" visible = "1"
-                      model_url = "package://hydrus/urdf/mesh/modules/flight_controller/fc_euclid201806.dae"> <!-- same with intel euclid -->
+                      model_url = "package://hydrus/urdf/mesh/ver1/flight_controller/fc_euclid201806.dae"> <!-- same with intel euclid -->
     <origin xyz="${link_length / 2 + 0.2281} ${-4.4*0.001} 0.03533" rpy="0 0 0"/>
     <inertial>
@@ -50,7 +50,7 @@
   <!-- 1.2 processor: jetson tx2 -->
   <xacro:extra_module name = "pc" parent = "link3" visible = "1"
-                      model_url = "package://hydrus/urdf/mesh/modules/processor/jetson_tx2.dae"
+                      model_url = "package://hydrus/urdf/mesh/ver1/processor/jetson_tx2.dae"
                       scale="0.001" >
-    <origin xyz="0.086 0.0 ${-0.0192}" rpy="${pi/2} 0 ${pi}"/>
+    <origin xyz="0.086 0.0 ${-0.0192}" rpy="0 0 ${pi}"/>
     <inertial>
       <mass value = "0.181" />
@@ -66,5 +66,5 @@
   <!-- 2.1 leddar one -->
   <xacro:extra_module name = "leddarone" parent = "link3" visible = "1"
-                      model_url = "package://hydrus/urdf/mesh/modules/sensor/leddar_one_tx2_attached_mode.dae">
+                      model_url = "package://hydrus/urdf/mesh/sensor/leddar_one_tx2_attached_mode.dae">
     <origin xyz="0.0866 0.0 -0.06267" rpy="0 ${pi} 0"/>
     <inertial>
@@ -79,6 +79,6 @@
   <!-- 2.2 gps -->
   <xacro:extra_module name = "gps" parent = "link2" visible = "1"
-                      model_url = "package://hydrus/urdf/mesh/modules/sensor/gps_ublox_m8n.dae">
-    <origin xyz="${link_length/2 + 0.206} 0.0 0.18" rpy="0 0 0"/>
+                      model_url = "package://hydrus/urdf/mesh/sensor/gps_ublox_m8n.dae">
+    <origin xyz="${link_length/2 + 0.1925} 0.0 0.152" rpy="0 0 0"/>
     <inertial>
       <origin xyz="0.000000 0.000000 -0.062510" rpy="0 0 0"/>
@@ -103,5 +103,5 @@
   <!-- 2.3 sensor: zed mini with servo -->
   <xacro:extra_module name = "zed_mini_servo_up" parent = "link2" visible = "1"
-                      model_url = "package://hydrus/urdf/mesh/modules/sensor/zed_mini_servo_up.dae">
+                      model_url = "package://hydrus/urdf/mesh/ver1/sensor/zed_mini_servo_up.dae">
     <origin xyz="${link_length/2 + 0.28715} 0.0 -0.04015" rpy="0 0 0"/>
     <inertial>
@@ -131,7 +131,7 @@
     </inertial>
     <visual>
-      <origin xyz="${-14.75 * 0.001} 0 ${-19 * 0.001}" rpy="0 ${pi/2} ${-pi}"/>
+      <origin xyz="${-14.75 * 0.001} 0 ${-19 * 0.001}" rpy="0 ${pi/2} ${pi/2}"/>
       <geometry>
-        <mesh filename="package://hydrus/urdf/mesh/modules/sensor/zed_mini_servo_down.dae"/>
+        <mesh filename="package://hydrus/urdf/mesh/ver1/sensor/zed_mini_servo_down.dae"/>
       </geometry>
     </visual>

File: robots/hydrus/urdf/common.xacro (robot description, xacro)
@@ -29,7 +29,7 @@
     </collision>
     <visual>
-      <origin rpy="${-pi/2} 0 0" xyz="${link_length* 0.5} 0 0"/>
+      <origin rpy="0 0 0" xyz="${link_length* 0.5} 0 0"/>
       <geometry>
-        <mesh filename="package://hydrus/urdf/mesh/link/${type}_link.dae"/>
+        <mesh filename="package://hydrus/urdf/mesh/ver1/link/${type}_link.dae"/>
       </geometry>
     </visual>
@@ -45,6 +45,5 @@
       <xacro:if value="${visible == 1}">
         <visual>
-          <!-- the origin of link_frame and visual_frame should be identical -->
-          <origin rpy="${-pi/2} 0 0" xyz="0 0 0"/>
+          <origin rpy="0 0 0" xyz="0 0 0"/>
           <geometry>
             <mesh filename="${model_url}" scale= "${scale} ${scale} ${scale}"/>
@@ -56,5 +55,5 @@
   <xacro:macro name="standard_leg" params="parent self:=${self} *origin">
       <xacro:extra_module name = "leg${self}" parent = "${parent}" visible = "1"
-                          model_url = "package://hydrus/urdf/mesh/modules/mechanical/standard_legs.dae" >
+                          model_url = "package://hydrus/urdf/mesh/ver1/leg/standard_legs.dae" >
         <xacro:insert_block name="origin" />
         <inertial>

Commit message: Add the new version of hydrus model, which is the standard model for MBZIRC. This commit also remains the old version, which is compatible by specifying the correct onboard_model (e.g. tx2_zed_201810)

File: robots/hydrus/robots/quad/tx2_zed_201810/robot.urdf.xacro (robot description, xacro)
@@ -5,8 +5,8 @@
   <xacro:include filename="$(find hydrus)/urdf/common.xacro" />
   <xacro:include filename="$(find hydrus)/urdf/link.urdf.xacro" />
-  <xacro:hydrusx_link self="1" child="2" rotor_direction="-1" with_battery = "0" />
-  <xacro:hydrusx_link self="2" child="3" rotor_direction="1"  with_battery = "0" />
-  <xacro:hydrusx_link self="3" child="4" rotor_direction="-1" with_battery = "0" />
-  <xacro:hydrusx_link self="4" child="4" rotor_direction="1"  with_battery = "0"/>
+  <xacro:hydrusx_link links="4" self="1" rotor_direction="-1" with_battery = "0" old_version = "1" />
+  <xacro:hydrusx_link links="4" self="2" rotor_direction="1"  with_battery = "0" old_version = "1" />
+  <xacro:hydrusx_link links="4" self="3" rotor_direction="-1" with_battery = "0" old_version = "1" />
+  <xacro:hydrusx_link links="4" self="4" rotor_direction="1"  with_battery = "0" old_version = "1" />
   <!-- special battery arrangement -->
   <xacro:extra_module name = "bat1" parent = "link1" visible = "1"

File: robots/hydrus/urdf/common.xacro (robot description, xacro)
@@ -5,12 +5,15 @@
   <xacro:property name="link_length" value=".6" />
   <xacro:property name="protector_radius" value=".1925" />
-  <xacro:property name="head_leg_offset" value="0.0525" />
-  <xacro:property name="general_leg_offset" value="0.05" />
-  <xacro:property name="end_leg_offset" value="0.5355" />
+  <xacro:property name="head_leg_offset" value="${0.3 - 0.25884}" />
+  <xacro:property name="end_leg_offset" value="${0.3 + 0.25884}" />
+  <!-- old version -->
+  <xacro:property name="head_leg_offset_old_version" value="0.0525" />
+  <xacro:property name="general_leg_offset_old_version" value="0.05" />
+  <xacro:property name="end_leg_offset_old_version" value="0.5355" />
   <!-- collision model parameter -->
   <xacro:property name="leg_collision_model_height" value="0.1715" />
   <!-- dynamics -->
   <xacro:property name="max_force" value="18" /> <!-- [N] -->
-  <xacro:macro name="link_model" params="type with_leg:=${with_leg}">
+  <xacro:macro name="link_model" params="type with_leg:=${with_leg} old_version:=${old_version}">
     <!-- for fcl in planning -->
     <collision>
@@ -29,8 +32,16 @@
     </collision>
     <visual>
-      <origin rpy="0 0 0" xyz="${link_length* 0.5} 0 0"/>
-      <geometry>
-        <mesh filename="package://hydrus/urdf/mesh/ver1/link/${type}_link.dae"/>
-      </geometry>
+      <xacro:if value="${old_version == 1}">
+        <origin rpy="0 0 0" xyz="${link_length* 0.5} 0 0"/>
+        <geometry>
+          <mesh filename="package://hydrus/urdf/mesh/ver1/link/${type}_link.dae"/>
+        </geometry>
+      </xacro:if>
+      <xacro:unless value="${old_version == 1}">
+        <origin rpy="0 0 0" xyz="${link_length* 0.5} 0 0"/>
+        <geometry>
+          <mesh filename="package://hydrus/urdf/mesh/ver2/link//link${type}.dae"/>
+        </geometry>
+      </xacro:unless>
     </visual>
   </xacro:macro>
@@ -53,24 +64,50 @@
     </link>
   </xacro:macro>
-  <xacro:macro name="standard_leg" params="parent self:=${self} *origin">
-      <xacro:extra_module name = "leg${self}" parent = "${parent}" visible = "1"
-                          model_url = "package://hydrus/urdf/mesh/ver1/leg/standard_legs.dae" >
-        <xacro:insert_block name="origin" />
-        <inertial>
-          <!-- short leg:
-          <origin xyz="0.0 0.0 -0.055380" rpy="0 0 0"/>
-          <mass value="0.043000"/>
-          <inertia
-              ixx="0.000088" iyy="0.000088" izz="0.000000"
-              ixy="0.000000" ixz="0.000000" iyz="0.000000"/>
-          -->
-          <!-- standard leg: -->
-          <origin xyz="0.0 0.0 -0.0852" rpy="0 0 0"/>
-          <mass value="0.047000"/>
-          <inertia
-              ixx="0.000259" iyy="-0.000281" izz="0.000010"
-              ixy="0.000000" ixz="0.000000" iyz="0.000000"/>
-        </inertial>
-      </xacro:extra_module>
+  <xacro:macro name="standard_leg_old_version" params="parent self:=${self} *origin">
+    <xacro:extra_module name = "leg${self}" parent = "${parent}" visible = "1"
+                        model_url = "package://hydrus/urdf/mesh/ver1/leg/standard_legs.dae" >
+      <xacro:insert_block name="origin" />
+      <inertial>
+        <!-- short leg:
+             <origin xyz="0.0 0.0 -0.055380" rpy="0 0 0"/>
+             <mass value="0.043000"/>
+             <inertia
+             ixx="0.000088" iyy="0.000088" izz="0.000000"
+             ixy="0.000000" ixz="0.000000" iyz="0.000000"/>
+        -->
+        <!-- standard leg: -->
+        <origin xyz="0.0 0.0 -0.093" rpy="0 0 0"/>
+        <mass value="0.047000"/>
+        <inertia
+            ixx="0.000259" iyy="0.000281" izz="0.000010"
+            ixy="0.000000" ixz="0.000000" iyz="0.000000"/>
+      </inertial>
+    </xacro:extra_module>
+  </xacro:macro>
+  <xacro:macro name="standard_leg_joint" params="parent self:=${self} *origin">
+    <xacro:extra_module name = "leg${self}" parent = "${parent}" visible = "1"
+                        model_url = "package://hydrus/urdf/mesh/ver2/leg/joint_leg.dae" >
+      <xacro:insert_block name="origin" />
+      <inertial>
+        <origin xyz="0.0 0.0005 -0.09521" rpy="0 0 0"/>
+        <mass value="0.0471"/>
+        <inertia
+            ixx="0.000251" iyy="0.000242" izz="0.000011"
+            ixy="0.000000" ixz="0.000000" iyz="0.000000"/>
+      </inertial>
+    </xacro:extra_module>
+  </xacro:macro>
+  <xacro:macro name="standard_leg_end" params="parent self:=${self} *origin">
+    <xacro:extra_module name = "leg${self}" parent = "${parent}" visible = "1"
+                        model_url = "package://hydrus/urdf/mesh/ver2/leg/end_leg.dae" >
+      <xacro:insert_block name="origin" />
+      <inertial>
+        <origin xyz="0.0 0.0005 -0.09411" rpy="0 0 0"/>
+        <mass value="0.0471"/>
+        <inertia
+            ixx="0.000251" iyy="0.000242" izz="0.000011"
+            ixy="0.000000" ixz="0.000000" iyz="0.000000"/>
+      </inertial>
+    </xacro:extra_module>
   </xacro:macro>
   <!-- friction -->

File: robots/hydrus/urdf/link.urdf.xacro (robot description, xacro)
@@ -3,43 +3,98 @@
     xmlns:xacro="http://www.ros.org/wiki/xacro" name="hydrusx_link" >
   <!-- D-H kai description(different from prof.nakamura) -->
-  <xacro:macro name="hydrusx_link" params="self child rotor_direction with_leg:=1 with_battery:=1">
-    <!-- link -->
-    <link name="link${self}">
-      <!-- head -->
-      <xacro:if value="${self == 1}">
-        <inertial>
-          <origin xyz="${link_length* 0.5 + 0.055120} 0.0 0.011580" rpy="0 0 0"/>
-          <mass value="0.566650"/>
-          <inertia
-              ixx="0.001804" iyy="0.017972" izz="0.019248"
-              ixy="0.000021" ixz="0.000372" iyz="0.000000"/>
-        </inertial>
-        <xacro:link_model type="head" />
-      </xacro:if>
-      <xacro:unless value="${self == 1}">
-        <!-- tail -->
-        <xacro:if value="${self == child}">
+  <xacro:macro name="hydrusx_link" params="links self rotor_direction with_leg:=1 with_battery:=1 old_version:=0">
+    <xacro:if value="${old_version == 1}">
+      <!-- link -->
+      <link name="link${self}">
+        <!-- head -->
+        <xacro:if value="${self == 1}">
           <inertial>
-            <origin xyz="${link_length * 0.5 + -0.013450} 0.0 0.012830" rpy="0 0 0"/>
-            <mass value="0.495530"/>
+            <origin xyz="${link_length* 0.5 + 0.055120} 0.0 0.011580" rpy="0 0 0"/>
+            <mass value="0.566650"/>
             <inertia
-                ixx="0.001758" iyy="0.013619" izz="0.014910"
-                ixy="0.000020" ixz="-0.000076" iyz="0.000000"/>
+                ixx="0.001804" iyy="0.017972" izz="0.019248"
+                ixy="0.000021" ixz="0.000372" iyz="0.000000"/>
           </inertial>
-          <xacro:link_model type="end" />
-        </xacro:if>
-        <xacro:unless value="${self == child}">
-          <!-- general -->
+          <xacro:link_model type="head" />
+        </xacro:if>
+        <xacro:unless value="${self == 1}">
+          <!-- tail -->
+          <xacro:if value="${self == links}">
+            <inertial>
+              <origin xyz="${link_length * 0.5 + -0.013450} 0.0 0.012830" rpy="0 0 0"/>
+              <mass value="0.495530"/>
+              <inertia
+                  ixx="0.001758" iyy="0.013619" izz="0.014910"
+                  ixy="0.000020" ixz="-0.000076" iyz="0.000000"/>
+            </inertial>
+            <xacro:link_model type="end" />
+          </xacro:if>
+          <xacro:unless value="${self == links}">
+            <!-- general -->
+            <inertial>
+              <origin xyz="${link_length * 0.5 + 0.038190} 0.0 0.010950" rpy="0 0 0"/>
+              <mass value="0.597720"/>
+              <inertia
+                  ixx="0.001828" iyy="0.021127" izz="0.022388"
+                  ixy="0.000021" ixz="0.000260" iyz="0.000000"/>
+            </inertial>
+            <xacro:link_model type="general" />
+          </xacro:unless>
+        </xacro:unless>
+      </link>
+    </xacro:if>
+    <xacro:unless value="${old_version == 1}">
+      <!-- link -->
+      <link name="link${self}">
+        <!-- head -->
+        <xacro:if value="${self == 1}">
           <inertial>
-            <origin xyz="${link_length * 0.5 + 0.038190} 0.0 0.010950" rpy="0 0 0"/>
-            <mass value="0.597720"/>
+            <origin xyz="${link_length* 0.5 + 0.057} 0.0 0.018" rpy="0 0 0"/>
+            <mass value="0.58712"/>
             <inertia
-                ixx="0.001828" iyy="0.021127" izz="0.022388"
-                ixy="0.000021" ixz="0.000260" iyz="0.000000"/>
+                ixx="0.00179" iyy="0.01605" izz="0.01714"
+                ixy="0.00000" ixz="0.00067" iyz="0.00000"/>
           </inertial>
-          <xacro:link_model type="general" />
-        </xacro:unless>
-      </xacro:unless>
-    </link>
+          <xacro:link_model type="1" />
+        </xacro:if>
+        <xacro:unless value="${self == 1}">
+          <!-- tail -->
+          <xacro:if value="${self == links}">
+            <inertial>
+              <origin xyz="${link_length * 0.5 -0.058} 0.0 0.0188" rpy="0 0 0"/>
+              <mass value="0.590"/>
+              <inertia
+                  ixx="0.00179" iyy="0.01581" izz="0.01692"
+                  ixy="0.00000" ixz="-0.00067" iyz="0.00000"/>
+            </inertial>
+            <xacro:link_model type="4" />
+          </xacro:if>
+          <xacro:unless value="${self == links}">
+            <!-- symetry -->
+            <xacro:if value="${self == links/2}">
+              <inertial>
+                <origin xyz="${link_length * 0.5} 0.0 0.01287" rpy="0 0 0"/>
+                <mass value="0.55744"/>
+                <inertia
+                    ixx="0.00171" iyy="0.01727" izz="0.01844"
+                    ixy="0.00000" ixz="0.00001" iyz="0.00000"/>
+              </inertial>
+              <xacro:link_model type="2" />
+            </xacro:if>
+            <!-- general -->
+            <xacro:unless value="${self == links/2}">
+              <inertial>
+                <origin xyz="${link_length * 0.5 - 0.0317} 0.0 0.01836" rpy="0 0 0"/>
+                <mass value="0.63453"/>
+                <inertia
+                    ixx="0.00182" iyy="0.02232" izz="0.02254"
+                    ixy="0.00000" ixz="-0.00077" iyz="0.00000"/>
+              </inertial>
+              <xacro:link_model type="3" />
+            </xacro:unless>
+          </xacro:unless>
+        </xacro:unless>
+      </link>
+    </xacro:unless>
     <xacro:damping_factor link ="link${self}"/>
     <!-- rotor -->
@@ -72,6 +127,7 @@
     <!-- use default battery: -->
     <xacro:if value="${with_battery == 1}">
+      <!-- note: use the same configuration between new and old version -->
       <xacro:extra_module name = "bat${self}" parent = "link${self}" visible = "1"
-                          model_url = "package://hydrus/urdf/mesh/modules/battery/VOLTON-PG-1300LP2-6s.stl" scale="0.001">
+                          model_url = "package://hydrus/urdf/mesh/ver1/modules/battery/VOLTON-PG-1300LP2-6s.stl" scale="0.001">
         <origin xyz="${link_length/2} 0.0 -0.048" rpy="${pi/2} 0 0"/>
         <inertial>
@@ -88,26 +144,47 @@
       <!-- head -->
       <xacro:if value="${self == 1}">
-        <xacro:standard_leg parent = "link${self}" >
-          <origin xyz="${head_leg_offset} 0.0 0" rpy="0 0 0"/>
-        </xacro:standard_leg>
+        <xacro:if value="${old_version == 1}">
+          <xacro:standard_leg_old_version parent = "link${self}" >
+            <origin xyz="${head_leg_offset_old_version} 0.0 0" rpy="0 0 0"/>
+          </xacro:standard_leg_old_version>
+        </xacro:if>
+        <xacro:unless value="${old_version == 1}">
+          <xacro:standard_leg_end parent = "link${self}" >
+            <origin xyz="${head_leg_offset} 0.0 0" rpy="0 0 0"/>
+          </xacro:standard_leg_end>
+        </xacro:unless>
       </xacro:if>
       <xacro:unless value="${self == 1}">
-        <xacro:standard_leg parent = "link${self}" >
-          <origin xyz="${general_leg_offset} 0.0 0" rpy="0 0 0"/>
-        </xacro:standard_leg>
+        <xacro:if value="${old_version == 1}">
+        <xacro:standard_leg_old_version parent = "link${self}" >
+          <origin xyz="${general_leg_offset_old_version} 0.0 0" rpy="0 0 0"/>
+        </xacro:standard_leg_old_version>
+        </xacro:if>
+        <xacro:unless value="${old_version == 1}">
+          <xacro:standard_leg_joint parent = "link${self}" >
+            <origin xyz="0.0 0.0 0" rpy="0 0 0"/>
+          </xacro:standard_leg_joint>
+        </xacro:unless>
         <!-- tail -->
-        <xacro:if value="${self == child}">
-          <xacro:standard_leg parent = "link${self}" self= "${self + 1}" >
-            <origin xyz="${end_leg_offset} 0.0 0" rpy="0 0 0"/>
-          </xacro:standard_leg>
+        <xacro:if value="${self == links}">
+          <xacro:if value="${old_version == 1}">
+            <xacro:standard_leg_old_version parent = "link${self}" self= "${self + 1}" >
+              <origin xyz="${end_leg_offset_old_version} 0.0 0" rpy="0 0 0"/>
+            </xacro:standard_leg_old_version>
+          </xacro:if>
+          <xacro:unless value="${old_version == 1}">
+            <xacro:standard_leg_end parent = "link${self}" self= "${self + 1}" >
+              <origin xyz="${end_leg_offset} 0.0 0" rpy="0 0 0"/>
+            </xacro:standard_leg_end>
+          </xacro:unless>
         </xacro:if>
       </xacro:unless>
     </xacro:if>
     <!-- joint -->
-    <xacro:unless value="${self == child}">
+    <xacro:unless value="${self == links}">
       <joint name="joint${self}" type="revolute">
         <limit effort="10.0" lower="${-pi/2}" upper="${pi/2}" velocity="0.5"/>
         <parent link="link${self}"/>
-        <child link="link${child}"/>
+        <child link="link${self+1}"/>
         <origin rpy="0 0 0" xyz="${link_length} 0 0"/>
         <axis xyz="0 0 1"/>
@@ -135,5 +212,5 @@
     </xacro:if>
     <!-- hardware interface -->
-    <xacro:unless value="${self == child}">
+    <xacro:unless value="${self == links}">
       <transmission name="joint_tran${self}">
         <type>transmission_interface/SimpleTransmission</type>
