Commit message: - Refactor the config file structure - Update the servo and motor model for hydrus mbzirc version

File: robots/hydrus/robots/quad/mbzirc_default_mode_201907/robot.urdf.xacro (robot description, xacro)
@@ -69,8 +69,8 @@
     <origin xyz="${link_length/2 - 0.1855} 0.0 -0.0626" rpy="${pi} 0 0"/>
     <inertial>
-      <origin xyz="-0.0083 0.0 -0.001" rpy="0 0 0"/>
-      <mass value="0.032"/>
+      <origin xyz="-0.008 0.0 0.0" rpy="0 0 0"/>
+      <mass value="0.025"/>
       <inertia
-          ixx="0.000012" iyy="0.00001" izz="0.00001"
+          ixx="0.00001" iyy="0.000006" izz="0.00001"
           ixy="0.000000" ixz="0.000000" iyz="0.000000"/>
     </inertial>
