Commit message: temp

File: robots/hydrus/robots/quad/tx2_rs_t265_201906/robot.urdf.xacro (robot description, xacro)
@@ -78,5 +78,4 @@
   <!-- end: leddar one -->
   <!-- 2.2 gps -->
-  <!--
   <xacro:extra_module name = "gps" parent = "link2" visible = "1"
                       model_url = "package://hydrus/urdf/mesh/sensor/gps_ublox_m8n.dae">
@@ -101,5 +100,4 @@
     </inertial>
     </xacro:extra_module>
-  -->
   <!-- end: gps -->
   <!-- 2.3  side-view  and downwards realsense t265 -->
@@ -144,9 +142,9 @@
     <parent link="link3"/>
     <child link="usb_hub"/>
-    <origin xyz="${55 * 0.001} 0 ${-100 * 0.001}" rpy="0 0 0"/>
+    <origin xyz="${40 * 0.001} 0 ${-100 * 0.001}" rpy="0 0 0"/>
   </joint>
   <link name="usb_hub">
     <inertial>
-      <mass value = "${(27.1 + 2 * 9.3) * 0.001}" />
+      <mass value = "${(16.8 + 2 * 9.3) * 0.001}" />
       <origin xyz="0 0 0" rpy="0 0 0"/>
       <inertia
@@ -158,5 +156,5 @@
       <origin rpy="0 0 0" xyz="0 0 0"/>
       <geometry>
-        <box size="0.004 0.05 0.03" />
+        <box size="0.03 0.015 0.02" />
       </geometry>
       <material name="Black">
