Commit message: [Temp] Refactor the tilt mode, which can hold variable tilting angle.

File: robots/hydrus/robots/quad/tilt_10deg_201907/robot.gazebo.xacro (robot description, xacro)
@@ -3,5 +3,5 @@
     xmlns:xacro="http://www.ros.org/wiki/xacro" name="hydrusx" >
   <!-- robot urdf -->
-  <xacro:include filename="$(find hydrus)/robots/quad/mbzirc_tilt_mode_201907/robot.urdf.xacro" />
+  <xacro:include filename="$(find hydrus)/robots/quad/tilt_10deg_201907/robot.urdf.xacro" />
   <!-- gazebo plugin for default controller and sensors -->
   <xacro:include filename="$(find hydrus)/robots/default.gazebo.xacro" />

File: robots/hydrus/robots/quad/tilt_10deg_201907/robot.urdf.xacro (robot description, xacro)
@@ -5,8 +5,8 @@
   <xacro:include filename="$(find hydrus)/urdf/common.xacro" />
   <xacro:include filename="$(find hydrus)/urdf/link.urdf.xacro" />
-  <xacro:hydrusx_link links="4" self="1" rotor_direction="-1" with_battery = "0" tilt_mode="1" />
-  <xacro:hydrusx_link links="4" self="2" rotor_direction="1"  with_battery = "0" tilt_mode="1"/>
-  <xacro:hydrusx_link links="4" self="3" rotor_direction="-1" with_battery = "0" tilt_mode="1"/>
-  <xacro:hydrusx_link links="4" self="4" rotor_direction="1"  with_battery = "0" tilt_mode="1"/>
+  <xacro:hydrusx_link links="4" self="1" rotor_direction="-1" with_battery = "0" tilt_mode="1" tilt_angle="10" />
+  <xacro:hydrusx_link links="4" self="2" rotor_direction="1"  with_battery = "0" tilt_mode="1" tilt_angle="10"/>
+  <xacro:hydrusx_link links="4" self="3" rotor_direction="-1" with_battery = "0" tilt_mode="1" tilt_angle="10"/>
+  <xacro:hydrusx_link links="4" self="4" rotor_direction="1"  with_battery = "0" tilt_mode="1" tilt_angle="10"/>
   <!-- special battery arrangement -->
   <xacro:extra_module name = "bat1" parent = "link1" visible = "1"

File: robots/hydrus/urdf/common.xacro (robot description, xacro)
@@ -11,11 +11,9 @@
   <xacro:property name="general_leg_offset_old_version" value="0.05" />
   <xacro:property name="end_leg_offset_old_version" value="0.5355" />
-  <!-- tilt propeller mode -->
-  <xacro:property name="tilt_angle" value=" 0.34906" />
   <!-- collision model parameter -->
   <xacro:property name="leg_collision_model_height" value="0.1715" />
   <!-- dynamics -->
   <xacro:property name="max_force" value="18" /> <!-- [N] -->
-  <xacro:macro name="link_model" params="type with_leg:=${with_leg} old_version:=${old_version} tilt_mode:=${tilt_mode}">
+  <xacro:macro name="link_model" params="type with_leg:=${with_leg} old_version:=${old_version} tilt_mode:=${tilt_mode} tilt_angle:=${tilt_angle}">
     <!-- for fcl in planning -->
     <collision>
@@ -44,5 +42,5 @@
         <geometry>
           <xacro:if value="${tilt_mode == 1}">
-            <mesh filename="package://hydrus/urdf/mesh/ver2/link/tilt_link${type}.dae"/>
+            <mesh filename="package://hydrus/urdf/mesh/ver2/link/tilt_${tilt_angle}deg_link${type}.dae"/>
           </xacro:if>
           <xacro:unless value="${tilt_mode == 1}">

File: robots/hydrus/urdf/link.urdf.xacro (robot description, xacro)
@@ -3,5 +3,5 @@
     xmlns:xacro="http://www.ros.org/wiki/xacro" name="hydrusx_link" >
   <!-- D-H kai description(different from prof.nakamura) -->
-  <xacro:macro name="hydrusx_link" params="links self rotor_direction with_leg:=1 with_battery:=1 old_version:=0 tilt_mode:=0">
+  <xacro:macro name="hydrusx_link" params="links self rotor_direction with_leg:=1 with_battery:=1 old_version:=0 tilt_mode:=0 tilt_angle:=0">
     <xacro:if value="${old_version == 1}">
       <!-- link -->
@@ -148,5 +148,5 @@
       <child link="thrust${self}"/>
       <xacro:if value="${tilt_mode == 1}">
-        <origin rpy="0 ${-rotor_direction * tilt_angle} 0" xyz="${link_length* 0.5} 0 0.045"/>
+        <origin rpy="0 ${-rotor_direction * tilt_angle * pi / 180.0} 0" xyz="${link_length* 0.5} 0 0.045"/>
       </xacro:if>
       <xacro:unless value="${tilt_mode == 1}">
