Commit message: Add robot namespace for rosnde, rostopic, rosparam, urdf, etc, to enable the mutiple robot bringup in one single rosmaster, and gazebo. Also rename several varaibles in control system to improve the readability.

File: aerial_robot_simulation/xacro/spinal.gazebo.xacro (robot description, xacro)
@@ -6,5 +6,5 @@
     <gazebo>
       <plugin name="gazebo_ros_control" filename="libgazebo_ros_control.so">
-        <robotNamespace>/${robot_name}</robotNamespace>
+        <robotNamespace>${robot_name}</robotNamespace>
         <robotSimType>gazebo_ros_control/AerialRobotHWSim</robotSimType>
       </plugin>
@@ -111,8 +111,9 @@
     <gazebo>
       <plugin name="gps_controller" filename="libhector_gazebo_ros_gps.so">
+        <robotNamespace>${robot_name}</robotNamespace>
         <updateRate>5.0</updateRate>
         <bodyName>${gps_frame}</bodyName>
-        <topicName>/fix</topicName>
-        <velocityTopicName>/fix_velocity</velocityTopicName>
+        <topicName>sim/gps/fix</topicName>
+        <velocityTopicName>sim/gps/velocity</velocityTopicName>
       </plugin>
     </gazebo>

File: robots/dragon/robots/quad/euclid_201709.gazebo.xacro (robot description, xacro)
@@ -2,8 +2,9 @@
 <robot
     xmlns:xacro="http://www.ros.org/wiki/xacro" name="dragon" >
+  <xacro:arg name="robot_name" default="dragon" />
   <!-- robot urdf -->
   <xacro:include filename="$(find dragon)/robots/quad/euclid_201709.urdf.xacro" />
   <!-- gazebo plugin for default controller and sensors -->
   <xacro:include filename="$(find aerial_robot_simulation)/xacro/spinal.gazebo.xacro" />
-  <xacro:gazebo_spinal robot_name="dragon" mag_frame="fc" />
+  <xacro:gazebo_spinal robot_name="$(arg robot_name)" mag_frame="fc" />
 </robot>

File: robots/dragon/robots/quad/euclid_201709.urdf.xacro (robot description, xacro)
@@ -1,5 +1,5 @@
 <?xml version="1.0"?>
 <robot
-    xmlns:xacro="http://www.ros.org/wiki/xacro" name="hydrusx" >
+    xmlns:xacro="http://www.ros.org/wiki/xacro" name="hydrus" >
   <!-- temporary -->
   <xacro:include filename="$(find dragon)/urdf/dragon_common.xacro" />

File: robots/hydrus/robots/quad/default_mode_201907/robot.gazebo.xacro (robot description, xacro)
@@ -1,9 +1,10 @@
 <?xml version="1.0"?>
 <robot
-    xmlns:xacro="http://www.ros.org/wiki/xacro" name="hydrusx" >
+    xmlns:xacro="http://www.ros.org/wiki/xacro" name="hydrus" >
+  <xacro:arg name="robot_name" default="hydrus" />
   <!-- robot urdf -->
   <xacro:include filename="$(find hydrus)/robots/quad/default_mode_201907/robot.urdf.xacro" />
   <!-- gazebo plugin for default controller and sensors -->
   <xacro:include filename="$(find aerial_robot_simulation)/xacro/spinal.gazebo.xacro" />
-  <xacro:gazebo_spinal robot_name="hydrusx" />
+  <xacro:gazebo_spinal robot_name="$(arg robot_name)" />
 </robot>

File: robots/hydrus/robots/quad/default_mode_201907/robot.urdf.xacro (robot description, xacro)
@@ -1,12 +1,12 @@
 <?xml version="1.0"?>
 <robot
-    xmlns:xacro="http://www.ros.org/wiki/xacro" name="hydrusx" >
+    xmlns:xacro="http://www.ros.org/wiki/xacro" name="hydrus" >
   <!-- basic kinematics model -->
   <xacro:include filename="$(find hydrus)/urdf/common.xacro" />
   <xacro:include filename="$(find hydrus)/urdf/link.urdf.xacro" />
-  <xacro:hydrusx_link links="4" self="1" rotor_direction="-1" with_battery = "0" />
-  <xacro:hydrusx_link links="4" self="2" rotor_direction="1"  with_battery = "0" />
-  <xacro:hydrusx_link links="4" self="3" rotor_direction="-1" with_battery = "0" />
-  <xacro:hydrusx_link links="4" self="4" rotor_direction="1"  with_battery = "0" />
+  <xacro:hydrus_link links="4" self="1" rotor_direction="-1" with_battery = "0" />
+  <xacro:hydrus_link links="4" self="2" rotor_direction="1"  with_battery = "0" />
+  <xacro:hydrus_link links="4" self="3" rotor_direction="-1" with_battery = "0" />
+  <xacro:hydrus_link links="4" self="4" rotor_direction="1"  with_battery = "0" />
   <!-- special battery arrangement -->
   <xacro:extra_module name = "bat1" parent = "link1" visible = "1"

File: robots/hydrus/robots/quad/old_model_tx2_rs_t265_201906/robot.gazebo.xacro (robot description, xacro)
@@ -1,9 +1,10 @@
 <?xml version="1.0"?>
 <robot
-    xmlns:xacro="http://www.ros.org/wiki/xacro" name="hydrusx" >
+    xmlns:xacro="http://www.ros.org/wiki/xacro" name="hydrus" >
+  <xacro:arg name="robot_name" default="hydrus" />
   <!-- robot urdf -->
   <xacro:include filename="$(find hydrus)/robots/quad/old_model_tx2_rs_t265_201906/robot.urdf.xacro" />
   <!-- gazebo plugin for default controller and sensors -->
   <xacro:include filename="$(find aerial_robot_simulation)/xacro/spinal.gazebo.xacro" />
-  <xacro:gazebo_spinal robot_name="hydrusx" />
+  <xacro:gazebo_spinal robot_name="$(arg robot_name)" />
 </robot>

File: robots/hydrus/robots/quad/old_model_tx2_rs_t265_201906/robot.urdf.xacro (robot description, xacro)
@@ -1,13 +1,13 @@
 <?xml version="1.0"?>
 <robot
-    xmlns:xacro="http://www.ros.org/wiki/xacro" name="hydrusx" >
+    xmlns:xacro="http://www.ros.org/wiki/xacro" name="hydrus" >
   <!-- basic kinematics model -->
   <m_f_rate value="-0.0182" /> <!-- overwrite -->
   <xacro:include filename="$(find hydrus)/urdf/common.xacro" />
   <xacro:include filename="$(find hydrus)/urdf/link.urdf.xacro" />
-  <xacro:hydrusx_link links="4" self="1" rotor_direction="-1" with_battery = "0" old_version = "1" />
-  <xacro:hydrusx_link links="4" self="2" rotor_direction="1"  with_battery = "0" old_version = "1" />
-  <xacro:hydrusx_link links="4" self="3" rotor_direction="-1" with_battery = "0" old_version = "1" />
-  <xacro:hydrusx_link links="4" self="4" rotor_direction="1"  with_battery = "0" old_version = "1" />
+  <xacro:hydrus_link links="4" self="1" rotor_direction="-1" with_battery = "0" old_version = "1" />
+  <xacro:hydrus_link links="4" self="2" rotor_direction="1"  with_battery = "0" old_version = "1" />
+  <xacro:hydrus_link links="4" self="3" rotor_direction="-1" with_battery = "0" old_version = "1" />
+  <xacro:hydrus_link links="4" self="4" rotor_direction="1"  with_battery = "0" old_version = "1" />
   <!-- special battery arrangement -->
   <xacro:extra_module name = "bat1" parent = "link1" visible = "1"

File: robots/hydrus/robots/quad/old_model_tx2_zed_201810/robot.gazebo.xacro (robot description, xacro)
@@ -1,10 +1,11 @@
 <?xml version="1.0"?>
 <robot
-    xmlns:xacro="http://www.ros.org/wiki/xacro" name="hydrusx" >
+    xmlns:xacro="http://www.ros.org/wiki/xacro" name="hydrus" >
+  <xacro:arg name="robot_name" default="hydrus" />
   <!-- robot urdf -->
   <xacro:include filename="$(find hydrus)/robots/quad/old_model_tx2_zed_201810/robot.urdf.xacro" />
   <!-- gazebo plugin for default controller and sensors -->
   <xacro:include filename="$(find aerial_robot_simulation)/xacro/spinal.gazebo.xacro" />
-  <xacro:gazebo_spinal robot_name="hydrusx" />
+  <xacro:gazebo_spinal robot_name="$(arg robot_name)" />
   <!-- sensors -->
   <!-- 1. stereo camera: depth, color based on left camera -->
@@ -53,4 +54,5 @@
       </camera>
       <plugin name="depth_camera" filename="libgazebo_ros_openni_kinect.so">
+        <robotNamespace>$(arg robot_name)</robotNamespace>
         <baseline>0.06</baseline>
         <alwaysOn>true</alwaysOn>

File: robots/hydrus/robots/quad/old_model_tx2_zed_201810/robot.urdf.xacro (robot description, xacro)
@@ -1,13 +1,13 @@
 <?xml version="1.0"?>
 <robot
-    xmlns:xacro="http://www.ros.org/wiki/xacro" name="hydrusx" >
+    xmlns:xacro="http://www.ros.org/wiki/xacro" name="hydrus" >
   <!-- basic kinematics model -->
   <m_f_rate value="-0.0182" /> <!-- overwrite -->
   <xacro:include filename="$(find hydrus)/urdf/common.xacro" />
   <xacro:include filename="$(find hydrus)/urdf/link.urdf.xacro" />
-  <xacro:hydrusx_link links="4" self="1" rotor_direction="-1" with_battery = "0" old_version = "1" />
-  <xacro:hydrusx_link links="4" self="2" rotor_direction="1"  with_battery = "0" old_version = "1" />
-  <xacro:hydrusx_link links="4" self="3" rotor_direction="-1" with_battery = "0" old_version = "1" />
-  <xacro:hydrusx_link links="4" self="4" rotor_direction="1"  with_battery = "0" old_version = "1" />
+  <xacro:hydrus_link links="4" self="1" rotor_direction="-1" with_battery = "0" old_version = "1" />
+  <xacro:hydrus_link links="4" self="2" rotor_direction="1"  with_battery = "0" old_version = "1" />
+  <xacro:hydrus_link links="4" self="3" rotor_direction="-1" with_battery = "0" old_version = "1" />
+  <xacro:hydrus_link links="4" self="4" rotor_direction="1"  with_battery = "0" old_version = "1" />
   <!-- special battery arrangement -->
   <xacro:extra_module name = "bat1" parent = "link1" visible = "1"

File: robots/hydrus/robots/quad/tilt_10deg_201907/robot.gazebo.xacro (robot description, xacro)
@@ -1,9 +1,10 @@
 <?xml version="1.0"?>
 <robot
-    xmlns:xacro="http://www.ros.org/wiki/xacro" name="hydrusx" >
+    xmlns:xacro="http://www.ros.org/wiki/xacro" name="hydrus" >
+  <xacro:arg name="robot_name" default="hydrus" />
   <!-- robot urdf -->
   <xacro:include filename="$(find hydrus)/robots/quad/tilt_10deg_201907/robot.urdf.xacro" />
   <!-- gazebo plugin for default controller and sensors -->
   <xacro:include filename="$(find aerial_robot_simulation)/xacro/spinal.gazebo.xacro" />
-  <xacro:gazebo_spinal robot_name="hydrusx" />
+  <xacro:gazebo_spinal robot_name="$(arg robot_name)" />
 </robot>

File: robots/hydrus/robots/quad/tilt_10deg_201907/robot.urdf.xacro (robot description, xacro)
@@ -1,12 +1,12 @@
 <?xml version="1.0"?>
 <robot
-    xmlns:xacro="http://www.ros.org/wiki/xacro" name="hydrusx" >
+    xmlns:xacro="http://www.ros.org/wiki/xacro" name="hydrus" >
   <!-- basic kinematics model -->
   <xacro:include filename="$(find hydrus)/urdf/common.xacro" />
   <xacro:include filename="$(find hydrus)/urdf/link.urdf.xacro" />
-  <xacro:hydrusx_link links="4" self="1" rotor_direction="-1" with_battery = "0" tilt_mode="1" tilt_angle="10" />
-  <xacro:hydrusx_link links="4" self="2" rotor_direction="1"  with_battery = "0" tilt_mode="1" tilt_angle="10"/>
-  <xacro:hydrusx_link links="4" self="3" rotor_direction="-1" with_battery = "0" tilt_mode="1" tilt_angle="10"/>
-  <xacro:hydrusx_link links="4" self="4" rotor_direction="1"  with_battery = "0" tilt_mode="1" tilt_angle="10"/>
+  <xacro:hydrus_link links="4" self="1" rotor_direction="-1" with_battery = "0" tilt_mode="1" tilt_angle="10" />
+  <xacro:hydrus_link links="4" self="2" rotor_direction="1"  with_battery = "0" tilt_mode="1" tilt_angle="10"/>
+  <xacro:hydrus_link links="4" self="3" rotor_direction="-1" with_battery = "0" tilt_mode="1" tilt_angle="10"/>
+  <xacro:hydrus_link links="4" self="4" rotor_direction="1"  with_battery = "0" tilt_mode="1" tilt_angle="10"/>
   <!-- special battery arrangement -->
   <xacro:extra_module name = "bat1" parent = "link1" visible = "1"

File: robots/hydrus/robots/quad/tilt_20deg_201907/robot.gazebo.xacro (robot description, xacro)
@@ -1,9 +1,10 @@
 <?xml version="1.0"?>
 <robot
-    xmlns:xacro="http://www.ros.org/wiki/xacro" name="hydrusx" >
+    xmlns:xacro="http://www.ros.org/wiki/xacro" name="hydrus" >
+  <xacro:arg name="robot_name" default="hydrus" />
   <!-- robot urdf -->
   <xacro:include filename="$(find hydrus)/robots/quad/tilt_20deg_201907/robot.urdf.xacro" />
   <!-- gazebo plugin for default controller and sensors -->
   <xacro:include filename="$(find aerial_robot_simulation)/xacro/spinal.gazebo.xacro" />
-  <xacro:gazebo_spinal robot_name="hydrusx" />
+  <xacro:gazebo_spinal robot_name="$(arg robot_name)" />
 </robot>

File: robots/hydrus/robots/quad/tilt_20deg_201907/robot.urdf.xacro (robot description, xacro)
@@ -1,12 +1,12 @@
 <?xml version="1.0"?>
 <robot
-    xmlns:xacro="http://www.ros.org/wiki/xacro" name="hydrusx" >
+    xmlns:xacro="http://www.ros.org/wiki/xacro" name="hydrus" >
   <!-- basic kinematics model -->
   <xacro:include filename="$(find hydrus)/urdf/common.xacro" />
   <xacro:include filename="$(find hydrus)/urdf/link.urdf.xacro" />
-  <xacro:hydrusx_link links="4" self="1" rotor_direction="-1" with_battery = "0" tilt_mode="1" tilt_angle="20" />
-  <xacro:hydrusx_link links="4" self="2" rotor_direction="1"  with_battery = "0" tilt_mode="1" tilt_angle="20"/>
-  <xacro:hydrusx_link links="4" self="3" rotor_direction="-1" with_battery = "0" tilt_mode="1" tilt_angle="20"/>
-  <xacro:hydrusx_link links="4" self="4" rotor_direction="1"  with_battery = "0" tilt_mode="1" tilt_angle="20"/>
+  <xacro:hydrus_link links="4" self="1" rotor_direction="-1" with_battery = "0" tilt_mode="1" tilt_angle="20" />
+  <xacro:hydrus_link links="4" self="2" rotor_direction="1"  with_battery = "0" tilt_mode="1" tilt_angle="20"/>
+  <xacro:hydrus_link links="4" self="3" rotor_direction="-1" with_battery = "0" tilt_mode="1" tilt_angle="20"/>
+  <xacro:hydrus_link links="4" self="4" rotor_direction="1"  with_battery = "0" tilt_mode="1" tilt_angle="20"/>
   <!-- special battery arrangement -->
   <xacro:extra_module name = "bat1" parent = "link1" visible = "1"

File: robots/hydrus/urdf/common.xacro (robot description, xacro)
@@ -1,5 +1,5 @@
 <?xml version="1.0"?>
 <robot
-    xmlns:xacro="http://www.ros.org/wiki/xacro" name="hydrusx_common" >
+    xmlns:xacro="http://www.ros.org/wiki/xacro" name="hydrus_common" >
   <!-- general attribute -->
   <baselink name="fc" />

File: robots/hydrus/urdf/link.urdf.xacro (robot description, xacro)
@@ -1,7 +1,7 @@
 <?xml version="1.0"?>
 <robot
-    xmlns:xacro="http://www.ros.org/wiki/xacro" name="hydrusx_link" >
+    xmlns:xacro="http://www.ros.org/wiki/xacro" name="hydrus_link" >
   <!-- D-H kai description(different from prof.nakamura) -->
-  <xacro:macro name="hydrusx_link" params="links self rotor_direction with_leg:=1 with_battery:=1 old_version:=0 tilt_mode:=0 tilt_angle:=0">
+  <xacro:macro name="hydrus_link" params="links self rotor_direction with_leg:=1 with_battery:=1 old_version:=0 tilt_mode:=0 tilt_angle:=0">
     <xacro:if value="${old_version == 1}">
       <!-- link -->

File: robots/hydrus_xi/robots/hex/xavier201811.gazebo.xacro (robot description, xacro)
@@ -2,7 +2,8 @@
 <robot
     xmlns:xacro="http://www.ros.org/wiki/xacro" name="hydrus_xi" >
+  <xacro:arg name="robot_name" default="hydrus_xi" />
   <xacro:include filename="$(find hydrus_xi)/robots/hex/xavier201811.urdf.xacro" />
   <!-- gazebo plugin for default controller and sensors -->
   <xacro:include filename="$(find aerial_robot_simulation)/xacro/spinal.gazebo.xacro" />
-  <xacro:gazebo_spinal robot_name="hydrus_xi" mag_frame="fc" />
+  <xacro:gazebo_spinal robot_name="$(arg robot_name)" mag_frame="fc" />
 </robot>

File: robots/hydrus_xi/robots/hex_branch/xavier201811.gazebo.xacro (robot description, xacro)
@@ -2,7 +2,8 @@
 <robot
     xmlns:xacro="http://www.ros.org/wiki/xacro" name="hydrus_xi" >
+  <xacro:arg name="robot_name" default="hydrus_xi" />
   <xacro:include filename="$(find hydrus_xi)/robots/hex_branch/xavier201811.urdf.xacro" />
   <!-- gazebo plugin for default controller and sensors -->
   <xacro:include filename="$(find aerial_robot_simulation)/xacro/spinal.gazebo.xacro" />
-  <xacro:gazebo_spinal robot_name="hydrus_xi" mag_frame="fc" />
+  <xacro:gazebo_spinal robot_name="$(arg robot_name)" mag_frame="fc" />
 </robot>

File: robots/hydrus_xi/robots/hex_branch/xavier_hokuyo.gazebo.xacro (robot description, xacro)
@@ -2,7 +2,8 @@
 <robot
     xmlns:xacro="http://www.ros.org/wiki/xacro" name="hydrus_xi" >
+  <xacro:arg name="robot_name" default="hydrus_xi" />
   <xacro:include filename="$(find hydrus_xi)/robots/hex_branch/xavier_hokuyo.urdf.xacro" />
   <!-- gazebo plugin for default controller and sensors -->
   <xacro:include filename="$(find aerial_robot_simulation)/xacro/spinal.gazebo.xacro" />
-  <xacro:gazebo_spinal robot_name="hydrus_xi" mag_frame="fc" />
+  <xacro:gazebo_spinal robot_name="$(arg robot_name)" mag_frame="fc" />
 </robot>

File: robots/hydrus_xi/urdf/branch_type_link.urdf.xacro (robot description, xacro)
@@ -47,5 +47,5 @@
       <child link="link${child1}"/>
       <origin rpy="0 0 0" xyz="0.1555 0.0 0.015"/>
-      <axis xyz="1 0 0"/>
+      <axis xyz="0 0 1"/>
       <dynamics damping="0.8" friction="0.0"/>
     </joint>
@@ -55,5 +55,5 @@
       <child link="link${child2}"/>
       <origin rpy="0 0 ${pi * 2.0 / 3.0}" xyz="-0.07775 0.13467 0.015"/>
-      <axis xyz="1 0 0"/>
+      <axis xyz="0 0 1"/>
       <dynamics damping="0.8" friction="0.0"/>
     </joint>
@@ -63,5 +63,5 @@
       <child link="link${child3}"/>
       <origin rpy="0 0 ${pi * 4.0 / 3.0}" xyz="-0.07775 -0.13467 0.015"/>
-      <axis xyz="1 0 0"/>
+      <axis xyz="0 0 1"/>
       <dynamics damping="0.8" friction="0.0"/>
     </joint>
