Commit message: update for painter demo

File: aerial_robot_simulation/xacro/block.xacro (robot description, xacro)
@@ -2,7 +2,7 @@
 <robot
     xmlns:xacro="http://www.ros.org/wiki/xacro" name="block" >
-  <xacro:property name="block_x" value="0.5"/>
+  <xacro:property name="block_x" value="1.0"/>
   <xacro:property name="block_y" value="0.3"/>
-  <xacro:property name="block_z" value="0.2"/>
+  <xacro:property name="block_z" value="2.0"/>
   <xacro:property name="mass" value="0.4"/>
   <link name="block">

File: robots/delta/robots/quad/20240722/delta.urdf.xacro (robot description, xacro)
@@ -290,5 +290,6 @@
     <inertial>
       <origin xyz="0.0815 0 0" rpy="0 0 0"/>
-      <mass value="0.222"/>
+      <!-- mass is thrust link + painter -->
+      <mass value="${0.222 + 0.081}"/>
       <!-- this inertia value is 10 times bigger than the real one -->
       <!-- to avoid the instability in gazebo -->
@@ -350,202 +351,3 @@
     </actuator>
   </transmission>
-  <!-- 3 soft_airframe_2 -->
-  <!-- soft_link -->
-  <joint name="soft_joint4" type="fixed">
-    <parent link="gimbal_link5"/>
-    <child link="soft_link4"/>
-    <origin xyz="0.147 0 0" rpy="0 0 0"/>
-  </joint>
-  <joint name="soft_joint5" type="revolute">
-    <limit effort="5.0" lower="${-pi/2}" upper="${pi/2}" velocity="0.5"/>
-    <parent link="soft_link4"/>
-    <child link="soft_link5"/>
-    <origin xyz="0.2215 0 0" rpy="0 0 0"/>
-    <axis xyz="0 0 1"/>
-    <dynamics damping="0.4" friction="0.1"/>
-  </joint>
-  <joint name="soft_joint6" type="revolute">
-    <limit effort="5.0" lower="${-pi/2}" upper="${pi/2}" velocity="0.5"/>
-    <parent link="soft_link5"/>
-    <child link="soft_link6"/>
-    <origin xyz="0.235 0 0" rpy="0 0 0"/>
-    <axis xyz="0 0 1"/>
-    <dynamics damping="0.4" friction="0.1"/>
-  </joint>
-  <link name="soft_link4">
-    <inertial>
-      <origin xyz="0.101 0.000002 0.018960" rpy="0 0 0"/>
-      <mass value="${0.059 + 0.157}"/>
-      <inertia
-          ixx="0.00013185" ixy="-0.00000146" ixz="0.00000096"
-          iyy="0.00055113" iyz="-0.00000218"
-          izz="0.00050648"/>
-    </inertial>
-    <visual>
-      <geometry>
-        <box size="0.2215 0.03 0.04"/>
-      </geometry>
-      <origin xyz="0.11075 0 0.02" rpy="0 0 0"/>
-    </visual>
-  </link>
-  <gazebo reference="soft_link4">
-    <mu1>0.1</mu1>
-    <mu2>0.1</mu2>
-  </gazebo>
-  <xacro:damping_factor link="soft_link4"/>
-  <link name="soft_link5">
-    <inertial>
-      <origin xyz="0.118 0.000002 0.019998" rpy="0 0 0"/>
-      <mass value="0.118"/>
-      <inertia
-          ixx="0.00007941" ixy="0.00000218" ixz="0.0"
-          iyy="0.00065133" iyz="0.0"
-          izz="0.00062639"/>
-    </inertial>
-    <visual>
-      <geometry>
-        <box size="0.235 0.03 0.04"/>
-      </geometry>
-      <origin xyz="0.1175 0.000002 0.019998" rpy="0 0 0"/>
-    </visual>
-  </link>
-  <gazebo reference="soft_link5">
-    <mu1>0.1</mu1>
-    <mu2>0.1</mu2>
-  </gazebo>
-  <xacro:damping_factor link="soft_link5"/>
-  <link name="soft_link6">
-    <inertial>
-      <origin xyz="0.10740316 0.0 0.003" rpy="0 0 0"/>
-      <mass value="0.059"/>
-      <inertia
-          ixx="0.00005433" ixy="0.00000033" ixz="0.0"
-          iyy="0.00047358" iyz="-0.00000369"
-          izz="0.00046011"/>
-    </inertial>
-    <visual>
-      <geometry>
-        <box size="0.1175 0.03 0.04"/>
-      </geometry>
-      <origin xyz="0.05875 0 0.02" rpy="0 0 0"/>
-    </visual>
-  </link>
-  <gazebo reference="soft_link6">
-    <mu1>0.1</mu1>
-    <mu2>0.1</mu2>
-  </gazebo>
-  <xacro:damping_factor link="soft_link6"/>
-  <transmission name="soft_joint_tran_5">
-    <type>transmission_interface/SimpleTransmission</type>
-    <joint name="soft_joint5">
-      <hardwareInterface>hardware_interface/EffortJointInterface</hardwareInterface>
-    </joint>
-    <actuator name="soft_joint_servo5">
-      <hardwareInterface>hardware_interface/EffortJointInterface</hardwareInterface>
-      <mechanicalReduction>1</mechanicalReduction>
-    </actuator>
-  </transmission>
-  <transmission name="soft_joint_tran_6">
-    <type>transmission_interface/SimpleTransmission</type>
-    <joint name="soft_joint6">
-      <hardwareInterface>hardware_interface/EffortJointInterface</hardwareInterface>
-    </joint>
-    <actuator name="soft_joint_servo6">
-      <hardwareInterface>hardware_interface/EffortJointInterface</hardwareInterface>
-      <mechanicalReduction>1</mechanicalReduction>
-    </actuator>
-  </transmission>
-  <!-- dummy_link -->
-  <joint name="dummy_joint1" type="revolute">
-    <limit effort="5.0" lower="${-pi/2}" upper="${pi/2}" velocity="0.5"/>
-    <parent link="soft_link4"/>
-    <child link="dummy_link1"/>
-    <origin xyz="0 0 0" rpy="0 0 0"/>
-    <axis xyz="0 0 1"/>
-    <dynamics damping="0.9" friction="0.1"/>
-  </joint>
-  <joint name="dummy_joint2" type="revolute">
-    <limit effort="5.0" lower="${-pi/2}" upper="${pi/2}" velocity="0.5"/>
-    <parent link="soft_link4"/>
-    <child link="dummy_link2"/>
-    <origin xyz="0 0 0" rpy="0 0 0"/>
-    <axis xyz="0 0 1"/>
-    <dynamics damping="0.9" friction="0.1"/>
-  </joint>
-  <link name="dummy_link1">
-    <inertial>
-      <origin xyz="0 0 0" rpy="0 0 0"/>
-      <mass value="0.0001"/>
-      <!-- this is for avoiding error in gazebo -->
-      <!-- <inertia
-          ixx="0.001" ixy="0.0" ixz="0.0"
-          iyy="0.001" iyz="0.0"
-          izz="0.002"/> -->
-      <inertia
-          ixx="0.00001" ixy="0.0" ixz="0.0"
-          iyy="0.00001" iyz="0.0"
-          izz="0.00002"/>
-    </inertial>
-  </link>
-  <link name="dummy_link2">
-    <inertial>
-      <origin xyz="0 0 0" rpy="0 0 0"/>
-      <mass value="0.0001"/>
-      <!-- this is for avoiding error in gazebo -->
-      <!-- <inertia
-          ixx="0.001" ixy="0.0" ixz="0.0"
-          iyy="0.001" iyz="0.0"
-          izz="0.002"/> -->
-      <inertia
-          ixx="0.00001" ixy="0.0" ixz="0.0"
-          iyy="0.00001" iyz="0.0"
-          izz="0.00002"/>
-    </inertial>
-  </link>
-  <transmission name="dummy_joint_tran_1">
-    <type>transmission_interface/SimpleTransmission</type>
-    <joint name="dummy_joint1">
-      <hardwareInterface>hardware_interface/EffortJointInterface</hardwareInterface>
-    </joint>
-    <actuator name="dummy_joint_servo1">
-      <hardwareInterface>hardware_interface/EffortJointInterface</hardwareInterface>
-      <mechanicalReduction>1</mechanicalReduction>
-    </actuator>
-  </transmission>
-  <transmission name="dummy_joint_tran_2">
-    <type>transmission_interface/SimpleTransmission</type>
-    <joint name="dummy_joint2">
-      <hardwareInterface>hardware_interface/EffortJointInterface</hardwareInterface>
-    </joint>
-    <actuator name="dummy_joint_servo2">
-      <hardwareInterface>hardware_interface/EffortJointInterface</hardwareInterface>
-      <mechanicalReduction>1</mechanicalReduction>
-    </actuator>
-  </transmission>
-  <!-- leg -->
-  <link name="leg7">
-    <inertial>
-      <origin xyz="0.0 0.0 -0.093" rpy="0 0 0"/>
-      <mass value="0.051000"/>
-      <inertia
-          ixx="0.000122" iyy="0.000133" izz="0.000012"
-          ixy="0.000000" ixz="0.000000" iyz="0.000000"/>
-    </inertial>
-    <visual>
-      <geometry>
-        <box size="0.02 0.02 -0.15"/>
-      </geometry>
-      <origin xyz="0.01 0.01 -0.075" rpy="0 0 0"/>
-    </visual>
-  </link>
-  <gazebo reference="leg7">
-    <mu1>0.1</mu1>
-    <mu2>0.1</mu2>
-  </gazebo>
-  <xacro:damping_factor link="leg7"/>
-  <joint name="leg_joint_soft2" type="fixed">
-    <parent link="soft_link6"/>
-    <child link="leg7"/>
-    <origin xyz="0.1 0 0" rpy="0 0 0"/>
-  </joint>
 </robot>

File: robots/delta/urdf/20240722/head.urdf.xacro (robot description, xacro)
@@ -7,5 +7,7 @@
       <inertial>
         <origin xyz="0.27442477 -0.04145571 0.00766623" rpy="0 0 0"/>
-        <mass value="0.80165566"/>
+        <!-- <mass value="0.80165566"/> -->
+        <!-- Styrofoam is removed -->
+        <mass value="${0.80165566 - 0.216}"/>
         <inertia
              ixx="0.00393460" iyy="0.02769902" izz="0.03031993"

File: robots/delta/urdf/20240722/middle.urdf.xacro (robot description, xacro)
@@ -7,5 +7,5 @@
       <inertial>
         <origin xyz="0.29984170 -0.04053992 0.00751982" rpy="0 0 0"/>
-        <mass value="0.81525662"/>
+        <mass value="${0.81525662 - 0.216}"/>
         <inertia
              ixx="0.00398803" iyy="0.02991643" izz="0.03256914"

File: robots/delta/urdf/20240722/tail.urdf.xacro (robot description, xacro)
@@ -7,5 +7,5 @@
       <inertial>
         <origin xyz="0.26112729 -0.04939508 0.00100978" rpy="0 0 0"/>
-        <mass value="0.66898892"/>
+        <mass value="${0.66898892 - 0.216}"/>
         <inertia
              ixx="0.00346166"  iyy="0.02400775"  izz="0.02657264"
