Commit message: Modify the robot model and files for hydrus_xi quad type

File: robots/hydrus_xi/robots/quad/default.urdf.xacro (robot description, xacro)
@@ -8,3 +8,16 @@
   <xacro:hydrus_xi_link self="3" child="4" rotor_direction="1" link_type="middle"/>
   <xacro:hydrus_xi_link self="4" child="4" rotor_direction="-1"  link_type="end"/>
+  #### flight controller ####
+  <xacro:extra_module name = "fc" parent = "link2" visible = "1"
+                      model_url = "package://hydrus_xi/urdf/mesh/modules/flight_controller/quad/fc.dae">
+    <origin xyz="0.5451 -0.006 -0.032" rpy="0 0 0"/>
+    <inertial>
+      <mass value = "0.0436" />
+      <origin xyz="0.0 0.006 0.0" rpy="0 0 0"/>
+      <inertia
+          ixx="0.00001" ixy="0.0" ixz="0.0"
+          iyy="0.00001" iyz="0.0"
+          izz="0.00002"/>
+    </inertial>
+  </xacro:extra_module>
 </robot>

File: robots/hydrus_xi/robots/quad/upboard202007.gazebo.xacro (robot description, xacro)
@@ -2,5 +2,5 @@
 <robot
     xmlns:xacro="http://www.ros.org/wiki/xacro" name="hydrus_xi" >
-  <xacro:include filename="$(find hydrus_xi)/robots/quad/only_fc.urdf.xacro" />
+  <xacro:include filename="$(find hydrus_xi)/robots/quad/upboard202007.urdf.xacro" />
   <!-- gazebo plugin for default controller and sensors -->
   <xacro:include filename="$(find aerial_robot_simulation)/xacro/spinal.gazebo.xacro" />

File: robots/hydrus_xi/robots/quad/upboard202007.urdf.xacro (robot description, xacro)
@@ -3,11 +3,11 @@
     xmlns:xacro="http://www.ros.org/wiki/xacro" name="hydrus_xi" >
   <xacro:include filename="$(find hydrus_xi)/robots/quad/default.urdf.xacro" />
-  #### flight controller ####
-  <xacro:extra_module name = "fc" parent = "link2" visible = "1"
-                      model_url = "package://hydrus_xi/urdf/mesh/modules/flight_controller/fc.dae">
-    <origin xyz="0.5396 -0.0044 -0.02847" rpy="0 0 0"/>
+  #### pc ####
+  <xacro:extra_module name = "pc" parent = "link3" visible = "1"
+                      model_url = "package://hydrus_xi/urdf/mesh/modules/pc/quad/upboard.dae">
+    <origin xyz="0.087 0 -0.029" rpy="${pi} 0 ${pi}"/>
     <inertial>
-      <mass value = "0.021" />
-      <origin xyz="0.01389 0.00526 0.0049" rpy="0 0 0"/>
+      <mass value = "0.138" />
+      <origin xyz="0.0 0.0 0.0" rpy="0 0 0"/>
       <inertia
           ixx="0.00001" ixy="0.0" ixz="0.0"
