Commit message: Clean up xacro files

File: robots/hydrus/urdf/common.xacro (robot description, xacro)
@@ -2,5 +2,4 @@
 <robot
     xmlns:xacro="http://www.ros.org/wiki/xacro" name="hydrusx_common" >
-  <xacro:property name="pi" value="3.1415926535897931" />
   <!-- kinematics [m] -->
   <xacro:property name="link_length" value=".6" />

Commit message: Add new nonliner control method for the under-actuated hydrus model (i.e. quad/penta)

File: robots/hydrus/urdf/common.xacro (robot description, xacro)
@@ -11,4 +11,5 @@
   <xacro:property name="general_leg_offset_old_version" value="0.05" />
   <xacro:property name="end_leg_offset_old_version" value="0.5355" />
+  <xacro:property name="tilt_angle" value="0.2" />
   <!-- collision model parameter -->
   <xacro:property name="leg_collision_model_height" value="0.1715" />

File: robots/hydrus/urdf/link.urdf.xacro (robot description, xacro)
@@ -103,5 +103,5 @@
       <parent link="link${self}"/>
       <child link="thrust${self}"/>
-      <origin rpy="0 0 0" xyz="${link_length* 0.5} 0 0"/>
+      <origin rpy="0 ${rotor_direction * tilt_angle} 0" xyz="${link_length* 0.5} 0 0"/>
       <axis xyz="0 0 ${rotor_direction}"/>
     </joint>
@@ -119,5 +119,5 @@
         <origin rpy="0 0 0" xyz="0 0 0"/>
         <geometry>
-          <cylinder length="0.1" radius="${protector_radius + 0.01}"/>
+          <cylinder length="0.1" radius="${protector_radius -0.1}"/>
         </geometry>
       </collision>

Commit message: temp

File: robots/hydrus/urdf/common.xacro (robot description, xacro)
@@ -11,5 +11,5 @@
   <xacro:property name="general_leg_offset_old_version" value="0.05" />
   <xacro:property name="end_leg_offset_old_version" value="0.5355" />
-  <xacro:property name="tilt_angle" value="0.2" />
+  <xacro:property name="tilt_angle" value="0.0" />
   <!-- collision model parameter -->
   <xacro:property name="leg_collision_model_height" value="0.1715" />

File: robots/hydrus_xi/robots/quad/default.urdf.xacro (robot description, xacro)
@@ -4,7 +4,7 @@
   <xacro:include filename="$(find hydrus_xi)/urdf/common.xacro" />
   <xacro:include filename="$(find hydrus_xi)/urdf/link.urdf.xacro" />
-  <xacro:hydrus_xi_link self="1" child="2" rotor_direction="-1" link_type="head"/>
-  <xacro:hydrus_xi_link self="2" child="3" rotor_direction="1"  link_type="general"/>
-  <xacro:hydrus_xi_link self="3" child="4" rotor_direction="-1" link_type="general"/>
-  <xacro:hydrus_xi_link self="4" child="4" rotor_direction="1"  link_type="end"/>
+  <xacro:hydrus_xi_link self="1" child="2" rotor_direction="1" link_type="head"/>
+  <xacro:hydrus_xi_link self="2" child="3" rotor_direction="-1"  link_type="general"/>
+  <xacro:hydrus_xi_link self="3" child="4" rotor_direction="1" link_type="general"/>
+  <xacro:hydrus_xi_link self="4" child="4" rotor_direction="-1"  link_type="end"/>
 </robot>

File: robots/hydrus_xi/urdf/common.xacro (robot description, xacro)
@@ -8,5 +8,5 @@
   <xacro:property name="fc_x_offset" value="0.566"/>
   <xacro:property name="fc_z_offset" value="-0.021"/>
-  <xacro:property name="thrust_tilt_angle" value="0.34906585039"/> <!-- 20deg -->
+  <xacro:property name="thrust_tilt_angle" value="0.2"/> <!-- 20deg:0.3491 -->
   <xacro:property name="rotor_radius" value=".0178"/>
   <!-- mass [Kg] -->

File: robots/hydrus_xi/urdf/link.urdf.xacro (robot description, xacro)
@@ -122,6 +122,6 @@
     </xacro:unless>
     #### gimbal joint ####
-    <joint name="gimbal${self}" type="revolute">
-      <limit effort="3.1" lower="-3.1415" upper="3.1415" velocity="0.5"/>
+    <joint name="gimbal${self}" type="continuous">
+      <limit effort="3.1" velocity="${pi}"/>
       <parent link="link${self}"/>
       <child link="gimbal_link${self}"/>

Commit message: Add fixed tilt propeller model for hydrus quad type

File: robots/hydrus/urdf/common.xacro (robot description, xacro)
@@ -11,10 +11,11 @@
   <xacro:property name="general_leg_offset_old_version" value="0.05" />
   <xacro:property name="end_leg_offset_old_version" value="0.5355" />
-  <xacro:property name="tilt_angle" value="0.0" />
+  <!-- tilt propeller mode -->
+  <xacro:property name="tilt_angle" value=" 0.34906" />
   <!-- collision model parameter -->
   <xacro:property name="leg_collision_model_height" value="0.1715" />
   <!-- dynamics -->
   <xacro:property name="max_force" value="18" /> <!-- [N] -->
-  <xacro:macro name="link_model" params="type with_leg:=${with_leg} old_version:=${old_version}">
+  <xacro:macro name="link_model" params="type with_leg:=${with_leg} old_version:=${old_version} tilt_mode:=${tilt_mode}">
     <!-- for fcl in planning -->
     <collision>
@@ -42,5 +43,10 @@
         <origin rpy="0 0 0" xyz="${link_length* 0.5} 0 0"/>
         <geometry>
-          <mesh filename="package://hydrus/urdf/mesh/ver2/link//link${type}.dae"/>
+          <xacro:if value="${tilt_mode == 1}">
+            <mesh filename="package://hydrus/urdf/mesh/ver2/link/tilt_link${type}.dae"/>
+          </xacro:if>
+          <xacro:unless value="${tilt_mode == 1}">
+            <mesh filename="package://hydrus/urdf/mesh/ver2/link/link${type}.dae"/>
+          </xacro:unless>
         </geometry>
       </xacro:unless>

File: robots/hydrus/urdf/link.urdf.xacro (robot description, xacro)
@@ -3,5 +3,5 @@
     xmlns:xacro="http://www.ros.org/wiki/xacro" name="hydrusx_link" >
   <!-- D-H kai description(different from prof.nakamura) -->
-  <xacro:macro name="hydrusx_link" params="links self rotor_direction with_leg:=1 with_battery:=1 old_version:=0">
+  <xacro:macro name="hydrusx_link" params="links self rotor_direction with_leg:=1 with_battery:=1 old_version:=0 tilt_mode:=0">
     <xacro:if value="${old_version == 1}">
       <!-- link -->
@@ -49,11 +49,22 @@
         <!-- head -->
         <xacro:if value="${self == 1}">
-          <inertial>
-            <origin xyz="${link_length* 0.5 + 0.057} 0.0 0.018" rpy="0 0 0"/>
-            <mass value="0.58712"/>
-            <inertia
-                ixx="0.00179" iyy="0.01605" izz="0.01714"
-                ixy="0.00000" ixz="0.00067" iyz="0.00000"/>
-          </inertial>
+          <xacro:if value="${tilt_mode == 1}">
+            <inertial>
+              <origin xyz="${link_length* 0.5 + 0.056} 0.0 0.02577" rpy="0 0 0"/>
+              <mass value="0.61442"/>
+              <inertia
+                  ixx="0.002" iyy="0.01634" izz="0.01723"
+                  ixy="0.00000" ixz="0.00045" iyz="0.00000"/>
+            </inertial>
+          </xacro:if>
+          <xacro:unless value="${tilt_mode == 1}">
+            <inertial>
+              <origin xyz="${link_length* 0.5 + 0.057} 0.0 0.018" rpy="0 0 0"/>
+              <mass value="0.58712"/>
+              <inertia
+                  ixx="0.00179" iyy="0.01605" izz="0.01714"
+                  ixy="0.00000" ixz="0.00067" iyz="0.00000"/>
+            </inertial>
+          </xacro:unless>
           <xacro:link_model type="1" />
         </xacro:if>
@@ -61,11 +72,22 @@
           <!-- tail -->
           <xacro:if value="${self == links}">
-            <inertial>
-              <origin xyz="${link_length * 0.5 -0.058} 0.0 0.0188" rpy="0 0 0"/>
-              <mass value="0.590"/>
-              <inertia
-                  ixx="0.00179" iyy="0.01581" izz="0.01692"
-                  ixy="0.00000" ixz="-0.00067" iyz="0.00000"/>
-            </inertial>
+            <xacro:if value="${tilt_mode == 1}">
+              <inertial>
+                <origin xyz="${link_length* 0.5 - 0.0576} 0.0 0.0258" rpy="0 0 0"/>
+                <mass value="0.616"/>
+                <inertia
+                    ixx="0.002" iyy="0.0161" izz="0.016992"
+                    ixy="0.00000" ixz="0.00000" iyz="0.00000"/>
+              </inertial>
+            </xacro:if>
+            <xacro:unless value="${tilt_mode == 1}">
+              <inertial>
+                <origin xyz="${link_length * 0.5 -0.058} 0.0 0.0188" rpy="0 0 0"/>
+                <mass value="0.590"/> <!-- +DCDC -->
+                <inertia
+                    ixx="0.00179" iyy="0.01581" izz="0.01692"
+                    ixy="0.00000" ixz="-0.00067" iyz="0.00000"/>
+              </inertial>
+            </xacro:unless>
             <xacro:link_model type="4" />
           </xacro:if>
@@ -73,22 +95,44 @@
             <!-- symetry -->
             <xacro:if value="${self == links/2}">
-              <inertial>
-                <origin xyz="${link_length * 0.5} 0.0 0.01287" rpy="0 0 0"/>
-                <mass value="0.55744"/>
-                <inertia
-                    ixx="0.00171" iyy="0.01727" izz="0.01844"
-                    ixy="0.00000" ixz="0.00001" iyz="0.00000"/>
-              </inertial>
+              <xacro:if value="${tilt_mode == 1}">
+                <inertial>
+                  <origin xyz="${link_length* 0.5 - 0.0005} 0.0 0.0204" rpy="0 0 0"/>
+                  <mass value="0.58312"/>
+                  <inertia
+                      ixx="0.002" iyy="0.01752" izz="0.018447"
+                      ixy="0.00000" ixz="0.00000" iyz="0.00000"/>
+                </inertial>
+              </xacro:if>
+              <xacro:unless value="${tilt_mode == 1}">
+                <inertial>
+                  <origin xyz="${link_length * 0.5} 0.0 0.01287" rpy="0 0 0"/>
+                  <mass value="0.55744"/>
+                  <inertia
+                      ixx="0.00171" iyy="0.01727" izz="0.01844"
+                      ixy="0.00000" ixz="0.00001" iyz="0.00000"/>
+                </inertial>
+              </xacro:unless>
               <xacro:link_model type="2" />
             </xacro:if>
             <!-- general -->
             <xacro:unless value="${self == links/2}">
-              <inertial>
-                <origin xyz="${link_length * 0.5 - 0.0317} 0.0 0.01836" rpy="0 0 0"/>
-                <mass value="0.63453"/>
-                <inertia
-                    ixx="0.00182" iyy="0.02232" izz="0.02254"
-                    ixy="0.00000" ixz="-0.00077" iyz="0.00000"/>
-              </inertial>
+              <xacro:if value="${tilt_mode == 1}">
+                <inertial>
+                  <origin xyz="${link_length* 0.5 - 0.03} 0.0 0.025" rpy="0 0 0"/>
+                  <mass value="0.66183"/>
+                  <inertia
+                      ixx="0.002" iyy="0.021851" izz="0.022718"
+                      ixy="0.00000" ixz="0.00000" iyz="0.00000"/>
+                </inertial>
+              </xacro:if>
+              <xacro:unless value="${tilt_mode == 1}">
+                <inertial>
+                  <origin xyz="${link_length * 0.5 - 0.0317} 0.0 0.01836" rpy="0 0 0"/>
+                  <mass value="0.63453"/>
+                  <inertia
+                      ixx="0.00182" iyy="0.02232" izz="0.02254"
+                      ixy="0.00000" ixz="-0.00077" iyz="0.00000"/>
+                </inertial>
+              </xacro:unless>
               <xacro:link_model type="3" />
             </xacro:unless>
@@ -103,5 +147,10 @@
       <parent link="link${self}"/>
       <child link="thrust${self}"/>
-      <origin rpy="0 ${rotor_direction * tilt_angle} 0" xyz="${link_length* 0.5} 0 0"/>
+      <xacro:if value="${tilt_mode == 1}">
+        <origin rpy="0 ${-rotor_direction * tilt_angle} 0" xyz="${link_length* 0.5} 0 0.045"/>
+      </xacro:if>
+      <xacro:unless value="${tilt_mode == 1}">
+        <origin rpy="0 0 0" xyz="${link_length* 0.5} 0 0"/>
+      </xacro:unless>
       <axis xyz="0 0 ${rotor_direction}"/>
     </joint>

Commit message: Implement robot model and transform control (lqi gain generator) for tilted hydrus model.

File: robots/hydrus/urdf/common.xacro (robot description, xacro)
@@ -15,5 +15,5 @@
   <!-- dynamics -->
   <xacro:property name="max_force" value="18" /> <!-- [N] -->
-  <xacro:macro name="link_model" params="type with_leg:=${with_leg} old_version:=${old_version}">
+  <xacro:macro name="link_model" params="type with_leg:=${with_leg} old_version:=${old_version} tilt_mode:=${tilt_mode} tilt_angle:=${tilt_angle}">
     <!-- for fcl in planning -->
     <collision>
@@ -41,5 +41,10 @@
         <origin rpy="0 0 0" xyz="${link_length* 0.5} 0 0"/>
         <geometry>
-          <mesh filename="package://hydrus/urdf/mesh/ver2/link//link${type}.dae"/>
+          <xacro:if value="${tilt_mode == 1}">
+            <mesh filename="package://hydrus/urdf/mesh/ver2/link/tilt_${tilt_angle}deg_link${type}.dae"/>
+          </xacro:if>
+          <xacro:unless value="${tilt_mode == 1}">
+            <mesh filename="package://hydrus/urdf/mesh/ver2/link/link${type}.dae"/>
+          </xacro:unless>
         </geometry>
       </xacro:unless>

File: robots/hydrus/urdf/link.urdf.xacro (robot description, xacro)
@@ -3,5 +3,5 @@
     xmlns:xacro="http://www.ros.org/wiki/xacro" name="hydrusx_link" >
   <!-- D-H kai description(different from prof.nakamura) -->
-  <xacro:macro name="hydrusx_link" params="links self rotor_direction with_leg:=1 with_battery:=1 old_version:=0">
+  <xacro:macro name="hydrusx_link" params="links self rotor_direction with_leg:=1 with_battery:=1 old_version:=0 tilt_mode:=0 tilt_angle:=0">
     <xacro:if value="${old_version == 1}">
       <!-- link -->
@@ -49,11 +49,22 @@
         <!-- head -->
         <xacro:if value="${self == 1}">
-          <inertial>
-            <origin xyz="${link_length* 0.5 + 0.057} 0.0 0.018" rpy="0 0 0"/>
-            <mass value="0.58712"/>
-            <inertia
-                ixx="0.00179" iyy="0.01605" izz="0.01714"
-                ixy="0.00000" ixz="0.00067" iyz="0.00000"/>
-          </inertial>
+          <xacro:if value="${tilt_mode == 1}">
+            <inertial>
+              <origin xyz="${link_length* 0.5 + 0.056} 0.0 0.02577" rpy="0 0 0"/>
+              <mass value="0.61442"/>
+              <inertia
+                  ixx="0.002" iyy="0.01634" izz="0.01723"
+                  ixy="0.00000" ixz="0.00045" iyz="0.00000"/>
+            </inertial>
+          </xacro:if>
+          <xacro:unless value="${tilt_mode == 1}">
+            <inertial>
+              <origin xyz="${link_length* 0.5 + 0.057} 0.0 0.018" rpy="0 0 0"/>
+              <mass value="0.58712"/>
+              <inertia
+                  ixx="0.00179" iyy="0.01605" izz="0.01714"
+                  ixy="0.00000" ixz="0.00067" iyz="0.00000"/>
+            </inertial>
+          </xacro:unless>
           <xacro:link_model type="1" />
         </xacro:if>
@@ -61,11 +72,22 @@
           <!-- tail -->
           <xacro:if value="${self == links}">
-            <inertial>
-              <origin xyz="${link_length * 0.5 -0.058} 0.0 0.0188" rpy="0 0 0"/>
-              <mass value="0.590"/>
-              <inertia
-                  ixx="0.00179" iyy="0.01581" izz="0.01692"
-                  ixy="0.00000" ixz="-0.00067" iyz="0.00000"/>
-            </inertial>
+            <xacro:if value="${tilt_mode == 1}">
+              <inertial>
+                <origin xyz="${link_length* 0.5 - 0.0576} 0.0 0.0258" rpy="0 0 0"/>
+                <mass value="0.616"/>
+                <inertia
+                    ixx="0.002" iyy="0.0161" izz="0.016992"
+                    ixy="0.00000" ixz="0.00000" iyz="0.00000"/>
+              </inertial>
+            </xacro:if>
+            <xacro:unless value="${tilt_mode == 1}">
+              <inertial>
+                <origin xyz="${link_length * 0.5 -0.058} 0.0 0.0188" rpy="0 0 0"/>
+                <mass value="0.590"/> <!-- +DCDC -->
+                <inertia
+                    ixx="0.00179" iyy="0.01581" izz="0.01692"
+                    ixy="0.00000" ixz="-0.00067" iyz="0.00000"/>
+              </inertial>
+            </xacro:unless>
             <xacro:link_model type="4" />
           </xacro:if>
@@ -73,22 +95,44 @@
             <!-- symetry -->
             <xacro:if value="${self == links/2}">
-              <inertial>
-                <origin xyz="${link_length * 0.5} 0.0 0.01287" rpy="0 0 0"/>
-                <mass value="0.55744"/>
-                <inertia
-                    ixx="0.00171" iyy="0.01727" izz="0.01844"
-                    ixy="0.00000" ixz="0.00001" iyz="0.00000"/>
-              </inertial>
+              <xacro:if value="${tilt_mode == 1}">
+                <inertial>
+                  <origin xyz="${link_length* 0.5 - 0.0005} 0.0 0.0204" rpy="0 0 0"/>
+                  <mass value="0.58312"/>
+                  <inertia
+                      ixx="0.002" iyy="0.01752" izz="0.018447"
+                      ixy="0.00000" ixz="0.00000" iyz="0.00000"/>
+                </inertial>
+              </xacro:if>
+              <xacro:unless value="${tilt_mode == 1}">
+                <inertial>
+                  <origin xyz="${link_length * 0.5} 0.0 0.01287" rpy="0 0 0"/>
+                  <mass value="0.55744"/>
+                  <inertia
+                      ixx="0.00171" iyy="0.01727" izz="0.01844"
+                      ixy="0.00000" ixz="0.00001" iyz="0.00000"/>
+                </inertial>
+              </xacro:unless>
               <xacro:link_model type="2" />
             </xacro:if>
             <!-- general -->
             <xacro:unless value="${self == links/2}">
-              <inertial>
-                <origin xyz="${link_length * 0.5 - 0.0317} 0.0 0.01836" rpy="0 0 0"/>
-                <mass value="0.63453"/>
-                <inertia
-                    ixx="0.00182" iyy="0.02232" izz="0.02254"
-                    ixy="0.00000" ixz="-0.00077" iyz="0.00000"/>
-              </inertial>
+              <xacro:if value="${tilt_mode == 1}">
+                <inertial>
+                  <origin xyz="${link_length* 0.5 - 0.03} 0.0 0.025" rpy="0 0 0"/>
+                  <mass value="0.66183"/>
+                  <inertia
+                      ixx="0.002" iyy="0.021851" izz="0.022718"
+                      ixy="0.00000" ixz="0.00000" iyz="0.00000"/>
+                </inertial>
+              </xacro:if>
+              <xacro:unless value="${tilt_mode == 1}">
+                <inertial>
+                  <origin xyz="${link_length * 0.5 - 0.0317} 0.0 0.01836" rpy="0 0 0"/>
+                  <mass value="0.63453"/>
+                  <inertia
+                      ixx="0.00182" iyy="0.02232" izz="0.02254"
+                      ixy="0.00000" ixz="-0.00077" iyz="0.00000"/>
+                </inertial>
+              </xacro:unless>
               <xacro:link_model type="3" />
             </xacro:unless>
@@ -103,5 +147,10 @@
       <parent link="link${self}"/>
       <child link="thrust${self}"/>
-      <origin rpy="0 0 0" xyz="${link_length* 0.5} 0 0"/>
+      <xacro:if value="${tilt_mode == 1}">
+        <origin rpy="0 ${-rotor_direction * tilt_angle * pi / 180.0} 0" xyz="${link_length* 0.5} 0 0.045"/>
+      </xacro:if>
+      <xacro:unless value="${tilt_mode == 1}">
+        <origin rpy="0 0 0" xyz="${link_length* 0.5} 0 0"/>
+      </xacro:unless>
       <axis xyz="0 0 ${rotor_direction}"/>
     </joint>
@@ -129,6 +178,6 @@
       <!-- note: use the same configuration between new and old version -->
       <xacro:extra_module name = "bat${self}" parent = "link${self}" visible = "1"
-                          model_url = "package://hydrus/urdf/mesh/ver1/modules/battery/VOLTON-PG-1300LP2-6s.stl" scale="0.001">
-        <origin xyz="${link_length/2} 0.0 -0.048" rpy="${pi/2} 0 0"/>
+                          model_url = "package://hydrus/urdf/mesh/battery/VOLTON-PG-1300LP2-6s.stl" scale="0.001">
+        <origin xyz="${link_length/2} 0.0 -0.048" rpy="0 0 0"/>
         <inertial>
           <origin xyz="0 0 0" rpy="0 0 0"/>

Commit message: [hydrus] add mesh file for 15inch prop model

File: robots/hydrus/urdf/common.xacro (robot description, xacro)
@@ -20,5 +20,5 @@
   <xacro:property name="max_force" value="20.0" /> <!-- [N] -->
   <xacro:property name="min_force" value="1.0" /> <!-- [N] -->
-  <xacro:macro name="link_model" params="type with_leg:=${with_leg} old_version:=${old_version} tilt_mode:=${tilt_mode} tilt_angle:=${tilt_angle}">
+  <xacro:macro name="link_model" params="type with_leg:=${with_leg} old_version:=${old_version} tilt_mode:=${tilt_mode} tilt_angle:=${tilt_angle} prop_15inch:=${prop_15inch}">
     <!-- for fcl in planning -->
     <collision>
@@ -47,5 +47,10 @@
         <geometry>
           <xacro:if value="${tilt_mode == 1}">
-            <mesh filename="package://hydrus/urdf/mesh/ver2/link/tilt_${tilt_angle}deg_link${type}.dae"/>
+            <xacro:if value="${prop_15inch == 1}">
+              <mesh filename="package://hydrus/urdf/mesh/ver2/link/tilt_${tilt_angle}deg_15inch_link${type}.dae"/>
+            </xacro:if>
+            <xacro:unless value="${prop_15inch == 1}">
+              <mesh filename="package://hydrus/urdf/mesh/ver2/link/tilt_${tilt_angle}deg_link${type}.dae"/>
+            </xacro:unless>
           </xacro:if>
           <xacro:unless value="${tilt_mode == 1}">
