Commit message: [Bug] the wrong path of the standard battery

File: robots/hydrus/urdf/link.urdf.xacro (robot description, xacro)
@@ -178,6 +178,6 @@
       <!-- note: use the same configuration between new and old version -->
       <xacro:extra_module name = "bat${self}" parent = "link${self}" visible = "1"
-                          model_url = "package://hydrus/urdf/mesh/ver1/modules/battery/VOLTON-PG-1300LP2-6s.stl" scale="0.001">
-        <origin xyz="${link_length/2} 0.0 -0.048" rpy="${pi/2} 0 0"/>
+                          model_url = "package://hydrus/urdf/mesh/battery/VOLTON-PG-1300LP2-6s.stl" scale="0.001">
+        <origin xyz="${link_length/2} 0.0 -0.048" rpy="0 0 0"/>
         <inertial>
           <origin xyz="0 0 0" rpy="0 0 0"/>

Commit message: Fix the wrong radius of propeller protector

File: robots/hydrus/urdf/link.urdf.xacro (robot description, xacro)
@@ -168,5 +168,5 @@
         <origin rpy="0 0 0" xyz="0 0 0"/>
         <geometry>
-          <cylinder length="0.1" radius="${protector_radius -0.1}"/>
+          <cylinder length="0.1" radius="${protector_radius + 0.01}"/>
         </geometry>
       </collision>

Commit message: added oct and multi model with torsion suppression control

File: robots/hydrus/urdf/link.urdf.xacro (robot description, xacro)
@@ -3,5 +3,12 @@
     xmlns:xacro="http://www.ros.org/wiki/xacro" name="hydrus_link" >
   <!-- D-H kai description(different from prof.nakamura) -->
-  <xacro:macro name="hydrus_link" params="links self rotor_direction with_leg:=1 with_battery:=1 old_version:=0 tilt_mode:=0 tilt_angle:=0">
+  <xacro:macro name="hydrus_link" params="links self rotor_direction with_leg:=1 with_battery:=1 old_version:=0 tilt_mode:=0 tilt_angle:=0 vibrate:=0 fix_rotor:=0">
+  <xacro:if value="${vibrate==1}">
+    <xacro:property name="link_inertial_pos" value="0.25"/>
+  </xacro:if>
+  <xacro:unless value="${vibrate==1}">
+    <xacro:property name="link_inertial_pos" value="0.5"/>
+  </xacro:unless>
+  <xacro:property name="link_half_mass_for_dummy" value="0.3"/>
     <xacro:if value="${old_version == 1}">
       <!-- link -->
@@ -10,6 +17,6 @@
         <xacro:if value="${self == 1}">
           <inertial>
-            <origin xyz="${link_length* 0.5 + 0.055120} 0.0 0.011580" rpy="0 0 0"/>
-            <mass value="0.566650"/>
+            <origin xyz="${link_length* link_inertial_pos + 0.055120} 0.0 0.011580" rpy="0 0 0"/>
+            <mass value="${0.566650-link_half_mass_for_dummy*vibrate}"/>
             <inertia
                 ixx="0.001804" iyy="0.017972" izz="0.019248"
@@ -22,6 +29,6 @@
           <xacro:if value="${self == links}">
             <inertial>
-              <origin xyz="${link_length * 0.5 + -0.013450} 0.0 0.012830" rpy="0 0 0"/>
-              <mass value="0.495530"/>
+              <origin xyz="${link_length * link_inertial_pos + -0.013450} 0.0 0.012830" rpy="0 0 0"/>
+              <mass value="${0.495530-link_half_mass_for_dummy*vibrate}"/>
               <inertia
                   ixx="0.001758" iyy="0.013619" izz="0.014910"
@@ -33,6 +40,6 @@
             <!-- general -->
             <inertial>
-              <origin xyz="${link_length * 0.5 + 0.038190} 0.0 0.010950" rpy="0 0 0"/>
-              <mass value="0.597720"/>
+              <origin xyz="${link_length * link_inertial_pos + 0.038190} 0.0 0.010950" rpy="0 0 0"/>
+              <mass value="${0.597720-link_half_mass_for_dummy*vibrate}"/>
               <inertia
                   ixx="0.001828" iyy="0.021127" izz="0.022388"
@@ -51,6 +58,6 @@
           <xacro:if value="${tilt_mode == 1}">
             <inertial>
-              <origin xyz="${link_length* 0.5 + 0.056} 0.0 0.02577" rpy="0 0 0"/>
-              <mass value="0.61442"/>
+              <origin xyz="${link_length* link_inertial_pos + 0.056} 0.0 0.02577" rpy="0 0 0"/>
+              <mass value="${0.61442-0.3*vibrate}"/>
               <inertia
                   ixx="0.002" iyy="0.01634" izz="0.01723"
@@ -60,6 +67,6 @@
           <xacro:unless value="${tilt_mode == 1}">
             <inertial>
-              <origin xyz="${link_length* 0.5 + 0.057} 0.0 0.018" rpy="0 0 0"/>
-              <mass value="0.58712"/>
+              <origin xyz="${link_length* link_inertial_pos + 0.057} 0.0 0.018" rpy="0 0 0"/>
+              <mass value="${0.58712-link_half_mass_for_dummy*vibrate}"/>
               <inertia
                   ixx="0.00179" iyy="0.01605" izz="0.01714"
@@ -74,6 +81,6 @@
             <xacro:if value="${tilt_mode == 1}">
               <inertial>
-                <origin xyz="${link_length* 0.5 - 0.0576} 0.0 0.0258" rpy="0 0 0"/>
-                <mass value="0.616"/>
+                <origin xyz="${link_length* link_inertial_pos - 0.0576} 0.0 0.0258" rpy="0 0 0"/>
+                <mass value="${0.616-link_half_mass_for_dummy*vibrate}"/>
                 <inertia
                     ixx="0.002" iyy="0.0161" izz="0.016992"
@@ -83,6 +90,6 @@
             <xacro:unless value="${tilt_mode == 1}">
               <inertial>
-                <origin xyz="${link_length * 0.5 -0.058} 0.0 0.0188" rpy="0 0 0"/>
-                <mass value="0.590"/> <!-- +DCDC -->
+                <origin xyz="${link_length * link_inertial_pos -0.058} 0.0 0.0188" rpy="0 0 0"/>
+                <mass value="${0.590-link_half_mass_for_dummy*vibrate}"/> <!-- +DCDC -->
                 <inertia
                     ixx="0.00179" iyy="0.01581" izz="0.01692"
@@ -97,6 +104,6 @@
               <xacro:if value="${tilt_mode == 1}">
                 <inertial>
-                  <origin xyz="${link_length* 0.5 - 0.0005} 0.0 0.0204" rpy="0 0 0"/>
-                  <mass value="0.58312"/>
+                  <origin xyz="${link_length* link_inertial_pos - 0.0005} 0.0 0.0204" rpy="0 0 0"/>
+                  <mass value="${0.58312-link_half_mass_for_dummy*vibrate}"/>
                   <inertia
                       ixx="0.002" iyy="0.01752" izz="0.018447"
@@ -106,6 +113,6 @@
               <xacro:unless value="${tilt_mode == 1}">
                 <inertial>
-                  <origin xyz="${link_length * 0.5} 0.0 0.01287" rpy="0 0 0"/>
-                  <mass value="0.55744"/>
+                  <origin xyz="${link_length * link_inertial_pos} 0.0 0.01287" rpy="0 0 0"/>
+                  <mass value="${0.55744-link_half_mass_for_dummy*vibrate}"/>
                   <inertia
                       ixx="0.00171" iyy="0.01727" izz="0.01844"
@@ -119,6 +126,6 @@
               <xacro:if value="${tilt_mode == 1}">
                 <inertial>
-                  <origin xyz="${link_length* 0.5 - 0.03} 0.0 0.025" rpy="0 0 0"/>
-                  <mass value="0.66183"/>
+                  <origin xyz="${link_length* link_inertial_pos - 0.03} 0.0 0.025" rpy="0 0 0"/>
+                  <mass value="${0.66183-link_half_mass_for_dummy*vibrate}"/>
                   <inertia
                       ixx="0.002" iyy="0.021851" izz="0.022718"
@@ -128,6 +135,6 @@
               <xacro:unless value="${tilt_mode == 1}">
                 <inertial>
-                  <origin xyz="${link_length * 0.5 - 0.0317} 0.0 0.01836" rpy="0 0 0"/>
-                  <mass value="0.63453"/>
+                  <origin xyz="${link_length * link_inertial_pos - 0.0317} 0.0 0.01836" rpy="0 0 0"/>
+                  <mass value="${0.63453-link_half_mass_for_dummy*vibrate}"/>
                   <inertia
                       ixx="0.00182" iyy="0.02232" izz="0.02254"
@@ -143,5 +150,11 @@
     <xacro:damping_factor link ="link${self}"/>
     <!-- rotor -->
-    <joint name="rotor${self}" type="continuous">
+    <xacro:if value="${fix_rotor == 1}">
+      <xacro:property name="rotor_joint_type" value="fixed"/>
+    </xacro:if>
+    <xacro:unless value="${fix_rotor == 1}">
+      <xacro:property name="rotor_joint_type" value="continuous"/>
+    </xacro:unless>
+    <joint name="rotor${self}" type="${rotor_joint_type}">
       <limit effort="100.0" lower="${min_force}" upper="${max_force}" velocity="0.5"/>
       <parent link="link${self}"/>
@@ -232,9 +245,35 @@
     <!-- joint -->
     <xacro:unless value="${self == links}">
+      <xacro:if value="${vibrate == 1}">
+        <link name="torsion_dummy${self}">
+          <inertial>
+            <origin xyz="${link_length*0.25} 0 0.012" rpy="0 0 0"/>
+            <mass value="${link_half_mass_for_dummy}"/>
+            <inertia
+                ixx="0.001828" iyy="0.021127" izz="0.022388"
+                ixy="0.000021" ixz="0.000260" iyz="0.000000"/>
+          </inertial>
+        </link>
+        <joint name="torsion${self}" type="revolute">
+          <limit effort="100.0" lower="${-pi/6}" upper="${pi/6}" velocity="1"/>
+          <parent link="link${self}"/>
+          <child link="torsion_dummy${self}"/>
+          <origin rpy="0 0 0" xyz="${link_length/2} 0 0"/>
+          <axis xyz="1 0 0"/>
+          <dynamics damping="0.9" friction="0.05"/>
+        </joint>
+      </xacro:if>
       <joint name="joint${self}" type="revolute">
         <limit effort="10.0" lower="${-pi/2}" upper="${pi/2}" velocity="0.5"/>
-        <parent link="link${self}"/>
-        <child link="link${self+1}"/>
-        <origin rpy="0 0 0" xyz="${link_length} 0 0"/>
+        <xacro:unless value="${vibrate == 1}">
+          <parent link="link${self}"/>
+          <child link="link${self+1}"/>
+          <origin rpy="0 0 0" xyz="${link_length} 0 0"/>
+        </xacro:unless>
+        <xacro:if value="${vibrate == 1}">
+          <parent link="torsion_dummy${self}"/>
+          <child link="link${self+1}"/>
+          <origin rpy="0 0 0" xyz="${link_length*0.5} 0 0"/>
+        </xacro:if>
         <axis xyz="0 0 1"/>
         <dynamics damping="0.9" friction="0.05"/>

Commit message: [hydrus] add prop_15inch arg in link.urdf.xacro

File: robots/hydrus/urdf/link.urdf.xacro (robot description, xacro)
@@ -3,5 +3,5 @@
     xmlns:xacro="http://www.ros.org/wiki/xacro" name="hydrus_link" >
   <!-- D-H kai description(different from prof.nakamura) -->
-  <xacro:macro name="hydrus_link" params="links self rotor_direction with_leg:=1 with_battery:=1 old_version:=0 tilt_mode:=0 tilt_angle:=0">
+  <xacro:macro name="hydrus_link" params="links self rotor_direction with_leg:=1 with_battery:=1 old_version:=0 tilt_mode:=0 tilt_angle:=0 prop_15inch:=0">
     <xacro:if value="${old_version == 1}">
       <!-- link -->
@@ -148,5 +148,10 @@
       <child link="thrust${self}"/>
       <xacro:if value="${tilt_mode == 1}">
-        <origin rpy="0 ${-rotor_direction * tilt_angle * pi / 180.0} 0" xyz="${link_length* 0.5} 0 0.045"/>
+        <xacro:if value="${prop_15inch == 1}">
+          <origin rpy="0 ${-rotor_direction * tilt_angle * pi / 180.0} 0" xyz="${link_length* 0.5 + 0.01944 * rotor_direction} 0 0.05395"/>
+        </xacro:if>
+        <xacro:unless value="${prop_15inch == 1}">
+          <origin rpy="0 ${-rotor_direction * tilt_angle * pi / 180.0} 0" xyz="${link_length* 0.5} 0 0.045"/>
+        </xacro:unless>
       </xacro:if>
       <xacro:unless value="${tilt_mode == 1}">

Commit message: [hydrus] add tilt_10deg_15inch_202106 model

File: robots/hydrus/urdf/link.urdf.xacro (robot description, xacro)
@@ -50,11 +50,22 @@
         <xacro:if value="${self == 1}">
           <xacro:if value="${tilt_mode == 1}">
-            <inertial>
-              <origin xyz="${link_length* 0.5 + 0.056} 0.0 0.02577" rpy="0 0 0"/>
-              <mass value="0.61442"/>
-              <inertia
-                  ixx="0.002" iyy="0.01634" izz="0.01723"
-                  ixy="0.00000" ixz="0.00045" iyz="0.00000"/>
-            </inertial>
+            <xacro:if value="${prop_15inch == 1}">
+              <inertial>
+                <origin xyz="${link_length* 0.5 + 0.05056} 0.0 0.02733" rpy="0 0 0"/>
+                <mass value="0.61741"/>
+                <inertia
+                    ixx="0.00222" iyy="0.01679" izz="0.01773"
+                    ixy="-0.00006" ixz="0.00027" iyz="0.00001"/>
+              </inertial>
+            </xacro:if>
+            <xacro:unless value="${prop_15inch == 1}">
+              <inertial>
+                <origin xyz="${link_length* 0.5 + 0.056} 0.0 0.02577" rpy="0 0 0"/>
+                <mass value="0.61442"/>
+                <inertia
+                    ixx="0.002" iyy="0.01634" izz="0.01723"
+                    ixy="0.00000" ixz="0.00045" iyz="0.00000"/>
+              </inertial>
+            </xacro:unless>
           </xacro:if>
           <xacro:unless value="${tilt_mode == 1}">
@@ -73,11 +84,22 @@
           <xacro:if value="${self == links}">
             <xacro:if value="${tilt_mode == 1}">
-              <inertial>
-                <origin xyz="${link_length* 0.5 - 0.0576} 0.0 0.0258" rpy="0 0 0"/>
-                <mass value="0.616"/>
-                <inertia
-                    ixx="0.002" iyy="0.0161" izz="0.016992"
-                    ixy="0.00000" ixz="0.00000" iyz="0.00000"/>
-              </inertial>
+              <xacro:if value="${prop_15inch == 1}">
+                <inertial>
+                  <origin xyz="${link_length* 0.5 - 0.051759} 0.0 0.027370" rpy="0 0 0"/>
+                  <mass value="0.61502"/>
+                  <inertia
+                      ixx="0.002217" iyy="0.016559" izz="0.017499"
+                      ixy="-0.000061" ixz="-0.000265" iyz="-0.000012"/>
+                </inertial>
+              </xacro:if>
+              <xacro:unless value="${prop_15inch == 1}">
+                <inertial>
+                  <origin xyz="${link_length* 0.5 - 0.0576} 0.0 0.0258" rpy="0 0 0"/>
+                  <mass value="0.616"/>
+                  <inertia
+                      ixx="0.002" iyy="0.0161" izz="0.016992"
+                      ixy="0.00000" ixz="0.00000" iyz="0.00000"/>
+                </inertial>
+              </xacro:unless>
             </xacro:if>
             <xacro:unless value="${tilt_mode == 1}">
@@ -96,11 +118,22 @@
             <xacro:if value="${self == links/2}">
               <xacro:if value="${tilt_mode == 1}">
-                <inertial>
-                  <origin xyz="${link_length* 0.5 - 0.0005} 0.0 0.0204" rpy="0 0 0"/>
-                  <mass value="0.58312"/>
-                  <inertia
-                      ixx="0.002" iyy="0.01752" izz="0.018447"
-                      ixy="0.00000" ixz="0.00000" iyz="0.00000"/>
-                </inertial>
+                <xacro:if value="${prop_15inch == 1}">
+                  <inertial>
+                    <origin xyz="${link_length* 0.5 + 0.004047} 0.0 0.022092" rpy="0 0 0"/>
+                    <mass value="0.586111"/>
+                    <inertia
+                        ixx="0.002188" iyy="0.017570" izz="0.018535"
+                        ixy="-0.000069" ixz="0.000118" iyz="-0.000012"/>
+                  </inertial>
+                </xacro:if>
+                <xacro:unless value="${prop_15inch == 1}">
+                  <inertial>
+                    <origin xyz="${link_length* 0.5 - 0.0005} 0.0 0.0204" rpy="0 0 0"/>
+                    <mass value="0.58312"/>
+                    <inertia
+                        ixx="0.002" iyy="0.01752" izz="0.018447"
+                        ixy="0.00000" ixz="0.00000" iyz="0.00000"/>
+                  </inertial>
+                </xacro:unless>
               </xacro:if>
               <xacro:unless value="${tilt_mode == 1}">
@@ -118,5 +151,15 @@
             <xacro:unless value="${self == links/2}">
               <xacro:if value="${tilt_mode == 1}">
-                <inertial>
+                <xacro:if value="${prop_15inch == 1}">
+                  <inertial>
+                  <origin xyz="${link_length* 0.5 - 0.033997} 0.0 0.026303" rpy="0 0 0"/>
+                  <mass value="0.664819"/>
+                  <inertia
+                      ixx="0.002256" iyy="0.021753" izz="0.022667"
+                      ixy="-0.000062" ixz="-0.000716" iyz="0.000011"/>
+                  </inertial>
+                </xacro:if>
+                <xacro:unless value="${prop_15inch == 1}">
+                  <inertial>
                   <origin xyz="${link_length* 0.5 - 0.03} 0.0 0.025" rpy="0 0 0"/>
                   <mass value="0.66183"/>
@@ -124,5 +167,6 @@
                       ixx="0.002" iyy="0.021851" izz="0.022718"
                       ixy="0.00000" ixz="0.00000" iyz="0.00000"/>
-                </inertial>
+                  </inertial>
+                </xacro:unless>
               </xacro:if>
               <xacro:unless value="${tilt_mode == 1}">

Commit message: [merge][build OK] merge origin master for estimation for livox

File: robots/hydrus/urdf/link.urdf.xacro (robot description, xacro)
@@ -200,5 +200,5 @@
       </xacro:if>
       <xacro:unless value="${tilt_mode == 1}">
-        <origin rpy="0 0 0" xyz="${link_length* 0.5} 0 0"/>
+        <origin rpy="0 0 0" xyz="${link_length* 0.5} 0 0.013"/>
       </xacro:unless>
       <axis xyz="0 0 ${rotor_direction}"/>
@@ -220,4 +220,15 @@
         </geometry>
       </collision>
+      <visual>
+        <origin rpy="0 0 0" xyz="0 0 0.032"/>
+        <geometry>
+          <xacro:if value="${rotor_direction == 1}">
+            <mesh filename="package://hydrus/urdf/mesh/propeller/T-motor-CF-14inch-CCW.dae"/>
+          </xacro:if>
+          <xacro:if value="${rotor_direction == -1}">
+            <mesh filename="package://hydrus/urdf/mesh/propeller/T-motor-CF-14inch-CW.dae"/>
+          </xacro:if>
+        </geometry>
+      </visual>
     </link>
     <xacro:damping_factor link ="thrust${self}"/>
