Commit message: add parent and root arg in dragn_link.urdf.xacro

File: robots/dragon/robots/quad/euclid_201709.urdf.xacro (robot description, xacro)
@@ -5,7 +5,7 @@
   <xacro:include filename="$(find dragon)/urdf/dragon_common.xacro" />
   <xacro:include filename="$(find dragon)/urdf/dragon_link.urdf.xacro" />
-  <xacro:dragon_module self="1" child="2" baselink="false" />
-  <xacro:dragon_module self="2" child="3" baselink="true" />
-  <xacro:dragon_module self="3" child="4" baselink="false" />
-  <xacro:dragon_module self="4" child="4" baselink="false" />
+  <xacro:dragon_module self="1" child="2" baselink="false" root="true" />
+  <xacro:dragon_module self="2" child="3" baselink="true" root="false" />
+  <xacro:dragon_module self="3" child="4" baselink="false" root="false" />
+  <xacro:dragon_module self="4" child="4" baselink="false" root="false" />
 </robot>

File: robots/dragon/urdf/dragon_link.urdf.xacro (robot description, xacro)
@@ -3,5 +3,5 @@
     xmlns:xacro="http://www.ros.org/wiki/xacro" name="dragon_link" >
   <!-- D-H kai description(different from prof.nakamura) -->
-  <xacro:macro name="dragon_module" params="self child baselink">
+  <xacro:macro name="dragon_module" params="self child:=-1 parent:=-1 root baselink">
     <!-- link -->
     <link name="link${self}">
@@ -200,9 +200,15 @@
     <xacro:damping_factor link ="thrust${self}"/>
     <!-- joint -->
-    <xacro:unless value="${self == child}">
+    <xacro:unless value="${self == child or self == parent}">
       <joint name="joint${self}_pitch" type="revolute">
         <limit effort="10.0" lower="${-pi/2}" upper="${pi/2}" velocity="0.1"/>
-        <parent link="link${self}"/>
-        <child link="inter_joint${self}"/>
+        <xacro:if value="${parent > 0}">
+          <parent link="inter_joint${self}"/>
+          <child link="link${self}"/>
+        </xacro:if>
+        <xacro:if value="${child > 0}">
+          <parent link="link${self}"/>
+          <child link="inter_joint${self}"/>
+        </xacro:if>
         <origin rpy="0 0 0" xyz="${link_length} 0 0"/>
         <axis xyz="0 1 0"/>
@@ -228,6 +234,12 @@
       <joint name="joint${self}_yaw" type="revolute">
         <limit effort="10.0" lower="${-pi/2}" upper="${pi/2}" velocity="0.1"/>
-        <parent link="inter_joint${self}"/>
-        <child link="link${child}"/>
+        <xacro:if value="${child > 0}">
+          <parent link="inter_joint${self}"/>
+          <child link="link${child}"/>
+        </xacro:if>
+        <xacro:if value="${parent > 0}">
+          <parent link="link${parent}"/>
+          <child link="inter_joint${self}"/>
+        </xacro:if>
         <origin rpy="0 0 0" xyz="${2 * inter_joint_x_offset} 0 0"/>
         <axis xyz="0 0 1"/>
@@ -239,5 +251,5 @@
       </gazebo>
     </xacro:unless>
-    <xacro:if value="${self == 1}">
+    <xacro:if value="${root}">
       <!-- dummy root link for KDL -->
       <link name="root">
@@ -278,5 +290,5 @@
     </xacro:if>
     <!-- hardware interface -->
-    <xacro:unless value="${self == child}">
+    <xacro:if value="${self != child and self != parent}">
       <transmission name="joint${self}_pitch_tran">
         <type>transmission_interface/SimpleTransmission</type>
@@ -303,5 +315,5 @@
         </actuator>
       </transmission>
-    </xacro:unless>
+    </xacro:if>
     <transmission name="gimbal${self}_roll_tran">
       <type>transmission_interface/SimpleTransmission</type>
