Commit message: [DRAGON][Localization][Livox] add livox MID360 for Fast LIO

File: robots/dragon/robots/quad/vim4_202311.urdf.xacro (robot description, xacro)
@@ -9,3 +9,25 @@
   <xacro:dragon_module self="3" child="4" baselink="false" />
   <xacro:dragon_module self="4" child="4" baselink="false" />
+  <!-- Livox MID360 -->
+  <xacro:extra_module name = "livox_mid360" parent = "link3" visible = "1"
+                      model_url = "package://dragon/urdf/mesh/sensor/livox_mid360.dae" >
+    <origin xyz="${link_length/2 - 0.109} 0.0 0.06592" rpy="0 0 ${-pi/2}"/>
+    <inertial>
+      <origin xyz="${-3.43 * 0.001} ${2.47 * 0.001} ${-10.27 * 0.001}" rpy="0 0 0"/>
+      <mass value="0.313"/>
+      <inertia
+          ixx="0.00027" iyy="0.00032" izz="0.00028"
+          ixy="0.0" ixz="0.00006" iyz="0.0"/>
+    </inertial>
+  </xacro:extra_module>
+  <xacro:extra_module name = "lidar_imu" parent = "livox_mid360" visible = "0" >
+    <origin xyz="0.011 0.02329 ${-0.02592 + 0.047 -0.04412}" rpy="0 0 0"/>
+    <inertial>
+      <origin xyz="0 0 0" rpy="0 0 0"/>
+      <mass value="0"/>
+      <inertia
+          ixx="0.0" iyy="0.0" izz="0.0"
+          ixy="0.0" ixz="0.0" iyz="0.0"/>
+    </inertial>
+  </xacro:extra_module>
 </robot>

File: robots/dragon/urdf/dragon_common.xacro (robot description, xacro)
@@ -42,4 +42,22 @@
     </visual>
   </xacro:macro>
+  <xacro:macro name="extra_module" params="name parent *origin *inertial visible:=0 model_url:=1 scale:=1">
+    <joint name="${parent}2${name}" type="fixed">
+      <parent link="${parent}"/>
+      <child link="${name}"/>
+      <xacro:insert_block name="origin" />
+    </joint>
+    <link name="${name}">
+      <xacro:insert_block name="inertial" />
+      <xacro:if value="${visible == 1}">
+        <visual>
+          <origin rpy="0 0 0" xyz="0 0 0"/>
+          <geometry>
+            <mesh filename="${model_url}" scale= "${scale} ${scale} ${scale}"/>
+          </geometry>
+        </visual>
+      </xacro:if>
+    </link>
+  </xacro:macro>
   <!-- friction -->
   <xacro:macro name="friction" params="self">
