Commit message: [Dragon][v1.5] update the urdf to include the livox model

File: robots/dragon/robots/quad/v1_5_202601.urdf.xacro (robot description, xacro)
@@ -8,3 +8,25 @@
   <xacro:dragon_module self="3" child="4" baselink="false" battery="true"/>
   <xacro:dragon_module self="4" child="4" baselink="false" battery="true"/>
+  <!-- Livox MID360 -->
+  <xacro:extra_module name = "livox_mid360" parent = "link2" visible = "1"
+                      model_url = "package://dragon/urdf/v1_5/mesh/sensor/livox_mid360_v1_5.stl" >
+    <origin xyz="0.132 0.0 0.05592" rpy="0 0 0"/>
+    <inertial>
+      <origin xyz="0.0068 0.0 -0.0066" rpy="0 0 0"/>
+      <mass value="0.2988"/>
+      <inertia
+          ixx="0.00018" iyy="0.00068" izz="0.00061"
+          ixy="0.0" ixz="-0.0001" iyz="0.0"/>
+    </inertial>
+  </xacro:extra_module>
+  <xacro:extra_module name = "lidar_imu" parent = "livox_mid360" visible = "0" >
+    <origin xyz="0.011 0.02329 ${-0.02592 + 0.047 -0.04412}" rpy="0 0 0"/>
+    <inertial>
+      <origin xyz="0 0 0" rpy="0 0 0"/>
+      <mass value="0"/>
+      <inertia
+          ixx="0.0" iyy="0.0" izz="0.0"
+          ixy="0.0" ixz="0.0" iyz="0.0"/>
+    </inertial>
+  </xacro:extra_module>
 </robot>

File: robots/dragon/robots/quad/v1_5_202601_no_bat.urdf.xacro (robot description, xacro)
@@ -2,4 +2,5 @@
 <robot
     xmlns:xacro="http://www.ros.org/wiki/xacro" name="dragon" >
+  <!-- robot urdf -->
   <xacro:include filename="$(find dragon)/urdf/v1_5/dragon_common.xacro" />
   <xacro:include filename="$(find dragon)/urdf/v1_5/dragon_link.urdf.xacro" />
@@ -8,3 +9,25 @@
   <xacro:dragon_module self="3" child="4" baselink="false" battery="false"/>
   <xacro:dragon_module self="4" child="4" baselink="false" battery="false"/>
+  <!-- Livox MID360 -->
+  <xacro:extra_module name = "livox_mid360" parent = "link2" visible = "1"
+                      model_url = "package://dragon/urdf/v1_5/mesh/sensor/livox_mid360_v1_5.stl" >
+    <origin xyz="0.132 0.0 0.05592" rpy="0 0 0"/>
+    <inertial>
+      <origin xyz="0.0068 0.0 -0.0066" rpy="0 0 0"/>
+      <mass value="0.2988"/>
+      <inertia
+          ixx="0.00018" iyy="0.00068" izz="0.00061"
+          ixy="0.0" ixz="-0.0001" iyz="0.0"/>
+    </inertial>
+  </xacro:extra_module>
+  <xacro:extra_module name = "lidar_imu" parent = "livox_mid360" visible = "0" >
+    <origin xyz="0.011 0.02329 ${-0.02592 + 0.047 -0.04412}" rpy="0 0 0"/>
+    <inertial>
+      <origin xyz="0 0 0" rpy="0 0 0"/>
+      <mass value="0"/>
+      <inertia
+          ixx="0.0" iyy="0.0" izz="0.0"
+          ixy="0.0" ixz="0.0" iyz="0.0"/>
+    </inertial>
+  </xacro:extra_module>
 </robot>
