Commit message: add roll pitch topic

File: robots/assemble_quadrotors/urdf/assemble_dual_quadrotors_female.urdf.xacro (robot description, xacro)
@@ -111,8 +111,12 @@
       <mass value = "0.6757" />
       <origin xyz="0 0 0" rpy="0 0 0"/>
+      <!-- <inertia -->
+      <!--     ixx="0.002125" ixy="0.00001389" ixz="0.00060374" -->
+      <!--     iyy="0.005992" iyz="-0.00000414" -->
+      <!--     izz="0.007684"/> -->
       <inertia
-          ixx="0.002281" ixy="0.0003799" ixz="0.00060374"
-          iyy="0.005992" iyz="0.00005686"
-          izz="0.007840"/>
+          ixx="0.00210931" ixy="-0.00000293" ixz="0.00048177"
+          iyy="0.00506536" iyz="-0.00000639"
+          izz="0.00677356"/>
     </inertial>
     <visual>

Commit message: work around female, male and whole models

File: robots/assemble_quadrotors/urdf/assemble_dual_quadrotors_female.urdf.xacro (robot description, xacro)
@@ -8,5 +8,5 @@
   <xacro:property name="pos_bound" value="${0.22628}" />
   <xacro:property name="center_dis" value="${0.393}" />
-  <xacro:property name="rotor_z" value="${0.025}" />
+  <xacro:property name="rotor_z" value="${0.050}" />
   <xacro:property name="opt_pich_1" value="${0.523525}" />
   <xacro:property name="opt_yaw_1" value="${0.73108}" />

File: robots/assemble_quadrotors/urdf/assemble_dual_quadrotors_male.urdf.xacro (robot description, xacro)
@@ -8,5 +8,5 @@
   <xacro:property name="pos_bound" value="${0.22628}" />
   <xacro:property name="center_dis" value="${0.393}" />
-  <xacro:property name="rotor_z" value="${0.025}" />
+  <xacro:property name="rotor_z" value="${0.05}" />
   <xacro:property name="opt_pich_1" value="${0.523525}" />
   <xacro:property name="opt_yaw_1" value="${0.73108}" />

File: robots/assemble_quadrotors/urdf/assemble_dual_quadrotors_whole.urdf.xacro (robot description, xacro)
@@ -8,5 +8,5 @@
   <xacro:property name="pos_bound" value="${0.22628}" />
   <xacro:property name="center_dis" value="${0.393}" />
-  <xacro:property name="rotor_z" value="${0.025}" />
+  <xacro:property name="rotor_z" value="${0.050}" />
   <xacro:property name="opt_pich_1" value="${0.523525}" />
   <xacro:property name="opt_yaw_1" value="${0.73108}" />

Commit message: work around for unit flight stability

File: robots/assemble_quadrotors/urdf/assemble_dual_quadrotors_female.urdf.xacro (robot description, xacro)
@@ -57,5 +57,5 @@
       <inertial>
         <origin xyz="0 0 0" rpy="0 0 0"/>
-        <mass value="0.0091"/>
+        <mass value="0.0052"/>
         <inertia
             ixx="0.00000807" ixy="0.0" ixz="0.0"
@@ -67,8 +67,8 @@
         <geometry>
           <xacro:if value="${direction == 1}">
-            <mesh filename="package://assemble_quadrotors/urdf/mesh/6_inchi_propeller.dae" />
+            <mesh filename="package://assemble_quadrotors/urdf/mesh/5_inchi_propeller.STL" />
           </xacro:if>
           <xacro:unless value="${direction == 1}">
-	    <mesh filename="package://assemble_quadrotors/urdf/mesh/6_inchi_propeller.dae" />
+	    <mesh filename="package://assemble_quadrotors/urdf/mesh/5_inchi_propeller.STL" />
           </xacro:unless>
         </geometry>
@@ -109,19 +109,15 @@
   <link name="main_body">
     <inertial>
-      <mass value = "0.6757" />
-      <origin xyz="0 0 0" rpy="0 0 0"/>
-      <!-- <inertia -->
-      <!--     ixx="0.002125" ixy="0.00001389" ixz="0.00060374" -->
-      <!--     iyy="0.005992" iyz="-0.00000414" -->
-      <!--     izz="0.007684"/> -->
+      <mass value = "0.75397839" />
+      <origin xyz="0 0 0 " rpy="0 0 0"/>
       <inertia
-          ixx="0.00210931" ixy="-0.00000293" ixz="0.00048177"
-          iyy="0.00506536" iyz="-0.00000639"
-          izz="0.00677356"/>
+          ixx="0.00558137" ixy="-0.00014117" ixz="-0.00047401"
+          iyy="0.00776130" iyz="0.00003630"
+          izz="0.01172792"/>
     </inertial>
     <visual>
       <origin rpy="0 0 0" xyz="0 0 0"/>
       <geometry>
-        <mesh filename="package://assemble_quadrotors/urdf/mesh/assemble_dual_quadrotors_female_body.dae" />
+        <mesh filename="package://assemble_quadrotors/urdf/mesh/Assemble_dual_quadrotors_v3_female.STL" />
       </geometry>
     </visual>
@@ -146,7 +142,7 @@
   </xacro:extra_module>
   <!-- propellers -->
-  <xacro:propeller_module id = "1" x = "${-pos_bound/2}" y = "${-pos_bound/2}" z = "${rotor_z}" pich = "${opt_pich_1}" yaw = "${opt_yaw_1}" direction = "1" />
-  <xacro:propeller_module id = "2" x = "${pos_bound/2}" y = "${-pos_bound/2}" z = "${rotor_z}" pich = "${opt_pich_2}" yaw = "${opt_yaw_2}"  direction = "-1" />
-  <xacro:propeller_module id = "3" x = "${pos_bound/2}" y = "${pos_bound/2}" z = "${rotor_z}"  pich = "${opt_pich_3}" yaw = "${opt_yaw_3}" direction = "1" />
-  <xacro:propeller_module id = "4" x = "${-pos_bound/2}" y = "${pos_bound/2}" z = "${rotor_z}"  pich = "${opt_pich_4}" yaw = "${opt_yaw_4}"  direction = "-1" />
+  <xacro:propeller_module id = "1" x = "-0.1044" y = "-0.12014" z = "0.05402" pich = "${opt_pich_4}" yaw = "${opt_yaw_4}" direction = "1" />
+  <xacro:propeller_module id = "2" x = "0.10705" y = "-0.10827" z = "0.05946" pich = "${opt_pich_3}" yaw = "${opt_yaw_3}"  direction = "-1" />
+  <xacro:propeller_module id = "3" x = "0.10474" y = "0.10579" z = "0.05404"  pich = "${opt_pich_2}" yaw = "${opt_yaw_2}" direction = "1" />
+  <xacro:propeller_module id = "4" x = "-0.10757" y = "0.12281" z = "0.05404"  pich = "${opt_pich_1}" yaw = "${opt_yaw_1}"  direction = "-1" />
 </robot>

File: robots/assemble_quadrotors/urdf/assemble_dual_quadrotors_male.urdf.xacro (robot description, xacro)
@@ -67,8 +67,8 @@
         <geometry>
           <xacro:if value="${direction == 1}">
-            <mesh filename="package://assemble_quadrotors/urdf/mesh/6_inchi_propeller.dae" />
+            <mesh filename="package://assemble_quadrotors/urdf/mesh/5_inchi_propeller.STL" />
           </xacro:if>
           <xacro:unless value="${direction == 1}">
-	    <mesh filename="package://assemble_quadrotors/urdf/mesh/6_inchi_propeller.dae" />
+	    <mesh filename="package://assemble_quadrotors/urdf/mesh/5_inchi_propeller.STL" />
           </xacro:unless>
         </geometry>
@@ -109,15 +109,16 @@
   <link name="main_body">
     <inertial>
-      <mass value = "0.6583" />
+      <!-- <mass value = "0.79154967" /> -->
+      <mass value = "0.79154967" />
       <origin xyz="0 0 0" rpy="0 0 0"/>
       <inertia
-          ixx="0.002127" ixy="-0.00001259" ixz="-0.0005813"
-          iyy="0.005264" iyz="0.00000375"
-          izz="0.006936"/>
+          ixx="0.00565753" ixy="-0.00012094" ixz="0.00049859"
+          iyy="0.00763738" iyz="0.00003798"
+          izz="0.01152518"/>
     </inertial>
     <visual>
       <origin rpy="0 0 0" xyz="0 0 0"/>
       <geometry>
-        <mesh filename="package://assemble_quadrotors/urdf/mesh/assemble_dual_quadrotors_male_body.dae" />
+        <mesh filename="package://assemble_quadrotors/urdf/mesh/Assemble_dual_quadrotors_v3_male.STL"/>
       </geometry>
     </visual>

File: robots/assemble_quadrotors/urdf/assemble_dual_quadrotors_whole.urdf.xacro (robot description, xacro)
@@ -11,10 +11,18 @@
   <xacro:property name="opt_pich_1" value="${0.523525}" />
   <xacro:property name="opt_yaw_1" value="${0.73108}" />
+  <!-- <xacro:property name="opt_pich_2" value="${0.523535}" /> -->
+  <!-- <xacro:property name="opt_yaw_2" value="${-2.08113}" /> -->
+  <!-- <xacro:property name="opt_pich_3" value="${0.523595}" /> -->
+  <!-- <xacro:property name="opt_yaw_3" value="${2.4662}" /> -->
+  <!-- <xacro:property name="opt_pich_4" value="${0.348489}" /> -->
+  <!-- <xacro:property name="opt_yaw_4" value="${-0.673131}" /> -->
+  <xacro:property name="opt_pich_1" value="${0.45}" />
+  <xacro:property name="opt_yaw_1" value="${0.73108}" />
   <xacro:property name="opt_pich_2" value="${0.523535}" />
   <xacro:property name="opt_yaw_2" value="${-2.08113}" />
-  <xacro:property name="opt_pich_3" value="${0.523595}" />
-  <xacro:property name="opt_yaw_3" value="${2.4662}" />
-  <xacro:property name="opt_pich_4" value="${0.348489}" />
-  <xacro:property name="opt_yaw_4" value="${-0.673131}" />
+  <xacro:property name="opt_pich_3" value="${0.523535}" />
+  <xacro:property name="opt_yaw_3" value="${2.08113}" />
+  <xacro:property name="opt_pich_4" value="${0.45}" />
+  <xacro:property name="opt_yaw_4" value="${-0.73108}" />
   <!-- dynamics -->
   <m_f_rate value="-0.006" /> <!-- drag torque rate, the true value should be -0.006 -->
@@ -57,5 +65,5 @@
       <inertial>
         <origin xyz="0 0 0" rpy="0 0 0"/>
-        <mass value="0.0091"/>
+        <mass value="0.0052"/>
         <inertia
             ixx="0.00000807" ixy="0.0" ixz="0.0"
@@ -67,8 +75,8 @@
         <geometry>
           <xacro:if value="${direction == 1}">
-            <mesh filename="package://assemble_quadrotors/urdf/mesh/6_inchi_propeller.dae" />
+            <mesh filename="package://assemble_quadrotors/urdf/mesh/5_inchi_propeller.STL" />
           </xacro:if>
           <xacro:unless value="${direction == 1}">
-	    <mesh filename="package://assemble_quadrotors/urdf/mesh/6_inchi_propeller.dae" />
+	    <mesh filename="package://assemble_quadrotors/urdf/mesh/5_inchi_propeller.STL" />
           </xacro:unless>
         </geometry>
@@ -109,15 +117,15 @@
   <link name="main_body">
     <inertial>
-      <mass value = "1.3341" />
+      <mass value = "1.54552806" />
       <origin xyz="0 0 0" rpy="0 0 0"/>
       <inertia
-          ixx="0.00425385" ixy="-0.00002899" ixz="-0.00001228"
-          iyy="0.04648" iyz="0.00000789"
-          izz="0.04984"/>
+          ixx="0.01124041" ixy="-0.00026951" ixz="-0.00026951"
+          iyy="0.06648421" iyz="0.00007432"
+          izz="0.07433712"/>
     </inertial>
     <visual>
       <origin rpy="0 0 0" xyz="0 0 0"/>
       <geometry>
-        <mesh filename="package://assemble_quadrotors/urdf/mesh/assemble_dual_quadrotors_whole_body.dae" />
+        <mesh filename="package://assemble_quadrotors/urdf/mesh/Assemble_dual_quadrotors_v3_whole.STL"/>
       </geometry>
     </visual>
@@ -142,11 +150,19 @@
   </xacro:extra_module>
   <!-- propellers -->
-  <xacro:propeller_module id = "1" x = "${center_dis/2-pos_bound/2}" y = "${-pos_bound/2}" z = "${rotor_z}" pich = "${opt_pich_1}" yaw = "${opt_yaw_1}" direction = "1" />
-  <xacro:propeller_module id = "2" x = "${center_dis/2+pos_bound/2}" y = "${-pos_bound/2}" z = "${rotor_z}" pich = "${opt_pich_2}" yaw = "${opt_yaw_2}"  direction = "-1" />
-  <xacro:propeller_module id = "3" x = "${center_dis/2+ pos_bound/2}" y = "${pos_bound/2}" z = "${rotor_z}"  pich = "${opt_pich_3}" yaw = "${opt_yaw_3}" direction = "1" />
-  <xacro:propeller_module id = "4" x = "${center_dis/2 -pos_bound/2}" y = "${pos_bound/2}" z = "${rotor_z}"  pich = "${opt_pich_4}" yaw = "${opt_yaw_4}"  direction = "-1" />
-  <xacro:propeller_module id = "5" x = "${-center_dis/2+pos_bound/2}" y = "${pos_bound/2}" z = "${rotor_z}"  pich = "${opt_pich_1}" yaw = "${-opt_yaw_1}" direction = "1" />
-  <xacro:propeller_module id = "6" x = "${-center_dis/2-pos_bound/2}" y = "${pos_bound/2}" z = "${rotor_z}"  pich = "${opt_pich_2}" yaw = "${-opt_yaw_2}" direction = "-1" />
-  <xacro:propeller_module id = "7" x = "${-center_dis/2-pos_bound/2}" y = "${-pos_bound/2}" z = "${rotor_z}"   pich = "${opt_pich_3}" yaw = "${-opt_yaw_3}" direction = "1" />
-  <xacro:propeller_module id = "8" x = "${-center_dis/2+pos_bound/2}" y = "${-pos_bound/2}" z = "${rotor_z}"  pich = "${opt_pich_4}" yaw = "${-opt_yaw_4}"  direction = "-1" />
+  <!-- <xacro:propeller_module id = "1" x = "0.09099" y = "-0.10578" z = "0.0521" pich = "${opt_pich_1}" yaw = "${opt_yaw_1}" direction = "1" /> -->
+  <!-- <xacro:propeller_module id = "2" x = "0.30329" y = "-0.1228" z = "0.0521" pich = "${opt_pich_2}" yaw = "${opt_yaw_2}"  direction = "-1" /> -->
+  <!-- <xacro:propeller_module id = "3" x = "0.30012" y = "0.12015" z = "0.0521"  pich = "${opt_pich_3}" yaw = "${opt_yaw_3}" direction = "1" /> -->
+  <!-- <xacro:propeller_module id = "4" x = "0.0886" y = "0.10827" z = "0.05752"  pich = "${opt_pich_4}" yaw = "${opt_yaw_4}"  direction = "-1" /> -->
+  <!-- <xacro:propeller_module id = "5" x = "-0.09099" y = "0.10578" z = "0.0521"  pich = "${-opt_pich_1}" yaw = "${opt_yaw_1}" direction = "1" /> -->
+  <!-- <xacro:propeller_module id = "6" x = "-0.30329" y = "0.1228" z = "0.0521"  pich = "${-opt_pich_2}" yaw = "${opt_yaw_2}" direction = "-1" /> -->
+  <!-- <xacro:propeller_module id = "7" x = "-0.30012" y = "-0.12015" z = "0.0521"  pich = "${-opt_pich_3}" yaw = "${opt_yaw_3}" direction = "1" /> -->
+  <!-- <xacro:propeller_module id = "8" x = "-0.0886" y = "-0.10827" z = "0.05752"  pich = "${-opt_pich_4}" yaw = "${opt_yaw_4}"  direction = "-1" /> -->
+  <xacro:propeller_module id = "1" x = "0.09" y = "-0.107" z = "0.0521" pich = "${opt_pich_1}" yaw = "${opt_yaw_1}" direction = "1" />
+  <xacro:propeller_module id = "2" x = "0.3" y = "-0.12" z = "0.0521" pich = "${opt_pich_2}" yaw = "${opt_yaw_2}"  direction = "-1" />
+  <xacro:propeller_module id = "3" x = "0.3" y = "0.12" z = "0.0521"  pich = "${opt_pich_3}" yaw = "${opt_yaw_3}" direction = "1" />
+  <xacro:propeller_module id = "4" x = "0.09" y = "0.107" z = "0.0521"  pich = "${opt_pich_4}" yaw = "${opt_yaw_4}"  direction = "-1" />
+  <xacro:propeller_module id = "5" x = "-0.09" y = "0.107" z = "0.0521"  pich = "${-opt_pich_1}" yaw = "${opt_yaw_1}" direction = "1" />
+  <xacro:propeller_module id = "6" x = "-0.3" y = "0.12" z = "0.0521"  pich = "${-opt_pich_2}" yaw = "${opt_yaw_2}" direction = "-1" />
+  <xacro:propeller_module id = "7" x = "-0.3" y = "-0.12" z = "0.0521"  pich = "${-opt_pich_3}" yaw = "${opt_yaw_3}" direction = "1" />
+  <xacro:propeller_module id = "8" x = "-0.09" y = "-0.107" z = "0.0521"  pich = "${-opt_pich_4}" yaw = "${opt_yaw_4}"  direction = "-1" />
 </robot>
