Commit message: add agile_multirotor folder
change gitignore

File: robots/assemble_quadrotors/urdf/assemble_dual_quadrotor_test.urdf.xacro (robot description, xacro)
@@ -21,4 +21,6 @@
   <xacro:property name="max_force" value="15.0" /> <!-- [N] -->
   <xacro:property name="min_force" value="0.0" /> <!-- [N] -->
+  <!-- obstacle [m] -->
+  <!-- <xacro:property name="sphere1_r" value="${1.00}" /> -->
   <!-- friction -->
   <xacro:macro name="damping_factor" params="link">
@@ -100,4 +102,14 @@
     </inertial>
   </link>
+    <!-- <link name="obstacle_root">
+    <inertial>
+      <origin xyz="0 0 0" rpy="0 0 0"/>
+      <mass value="0.00001"/>
+      <inertia
+          ixx="0.000001" ixy="0.0" ixz="0.0"
+          iyy="0.000001" iyz="0.0"
+          izz="0.000002"/>
+    </inertial>
+  </link> -->
   <joint name="root_joint" type="fixed">
     <parent link="root"/>
@@ -106,4 +118,11 @@
     <axis xyz="0 0 1"/>
   </joint>
+  <!-- <joint name="root_obstacle" type="fixed">
+    <parent link="obstacle_root"/>
+    <child link="sphere_body"/>
+    <origin rpy="0 0 0" xyz="1 0 0"/>
+    <axis xyz="0 0 1"/>
+  </joint>  -->
+  <!-- if connected, the sphere moves depending on the sphere -->
   <!-- main_body -->
   <link name="main_body">
@@ -119,6 +138,6 @@
       <origin rpy="0 0 0" xyz="0 0 0"/>
       <geometry>
+      </geometry>
         <mesh filename="package://assemble_quadrotors/urdf/mesh/Assemble_fixed_parts_test.STL" />
-      </geometry>
     </visual>
     <collision>
@@ -129,4 +148,27 @@
     </collision>
   </link>
+  <!-- sphere obstacle -->
+  <!-- <link name="sphere_body">
+    <inertial>
+      <mass value = "0.01" />
+      <origin xyz="0 0 0" rpy="0 0 0"/>
+      <inertia
+          ixx="0.001" ixy="0.0000" ixz="0.0000"
+          iyy="0.001" iyz="0.00000"
+          izz="0.001"/>
+    </inertial>
+    <visual>
+      <origin rpy="0 0 0" xyz="1 0 1"/>
+      <geometry>
+         <sphere radius="0.2"/>
+      </geometry>
+    </visual>
+    <collision>
+      <origin rpy="0 0 0" xyz="1 0 1"/>
+      <geometry>
+         <sphere radius="0.2"/>
+      </geometry>
+    </collision>
+  </link> -->
   <!-- spinal -->
   <xacro:extra_module name = "fc" parent = "main_body" visible = "0" >
