Commit message: [Tiger] refactor the URDF model for walk mode

File: robots/tiger/robots/octo/tiger_v1_base.urdf.xacro (robot description, xacro)
@@ -3,14 +3,14 @@
     xmlns:xacro="http://www.ros.org/wiki/xacro" name="tiger_v1" >
   <xacro:include filename="$(find tiger)/urdf/v1/link.urdf.xacro" />
-  <xacro:macro name="tiger_v1" params="battery:=1 leg:=1">
+  <xacro:macro name="tiger_v1" params="battery:=1 leg:=1 end_leg:=1">
     <xacro:tiger_center_link child1="1" child2="3" child3="5" child4="7" leg="${leg}"/>
     <xacro:tiger_link self="1" child="2" link_type="general" battery="${battery}" leg="${leg}"/>
-    <xacro:tiger_link self="2" child="2" link_type="end"     battery="${battery}" leg="${leg}"/>
+    <xacro:tiger_link self="2" child="2" link_type="end"     battery="${battery}" leg="${end_leg}"/>
     <xacro:tiger_link self="3" child="4" link_type="general" battery="${battery}" leg="${leg}"/>
-    <xacro:tiger_link self="4" child="4" link_type="end"     battery="${battery}" leg="${leg}"/>
+    <xacro:tiger_link self="4" child="4" link_type="end"     battery="${battery}" leg="${end_leg}"/>
     <xacro:tiger_link self="5" child="6" link_type="general" battery="${battery}" leg="${leg}"/>
-    <xacro:tiger_link self="6" child="6" link_type="end"     battery="${battery}" leg="${leg}"/>
+    <xacro:tiger_link self="6" child="6" link_type="end"     battery="${battery}" leg="${end_leg}"/>
     <xacro:tiger_link self="7" child="8" link_type="general" battery="${battery}" leg="${leg}"/>
-    <xacro:tiger_link self="8" child="8" link_type="end"     battery="${battery}" leg="${leg}"/>
+    <xacro:tiger_link self="8" child="8" link_type="end"     battery="${battery}" leg="${end_leg}"/>
   </xacro:macro>
 </robot>

File: robots/tiger/robots/octo/v1_leg/robot.urdf.xacro (robot description, xacro)
@@ -2,12 +2,33 @@
 <robot
     xmlns:xacro="http://www.ros.org/wiki/xacro" name="tiger" >
-  <xacro:include filename="$(find tiger)/robots/octo/v1_default/robot.urdf.xacro" />
-  <xacro:property name="foot_radius" value="0.04"/>
-  <xacro:property name="foot_mass" value="0.02"/>
+  <xacro:include filename="$(find tiger)/robots/octo/tiger_v1_base.urdf.xacro" />
+  <xacro:tiger_v1 end_leg="false" />
+  #### flight controller ####
+  <xacro:extra_module name = "fc" parent = "center_link" visible = "1"
+                      model_url = "package://tiger/urdf/v1/mesh/board/spinal.dae">
+    <origin xyz="-0.0129 -0.0044 0.0398284" rpy="0 0 0"/>
+    <inertial>
+      <mass value="0.0354160"/>
+      <origin xyz="0.0128576 0.0044678 -0.0226530" rpy="0 0 0"/>
+      <inertia
+          ixx="0.0000225" iyy="0.0000225" izz="0.0000346"
+          ixy="-0.0000001" iyz="0.0000000" ixz="0.0000000" />
+    </inertial>
+  </xacro:extra_module>
+  <xacro:extra_module name = "pc" parent = "center_link" visible = "0">
+    <origin xyz="0 0.089888 0.002" rpy="${pi/2} 0 0"/>
+    <inertial>
+      <mass value="0.1411331"/>
+      <origin xyz="0.0008915 0.0304136 0.0271590" rpy="0 0 0"/>
+      <inertia
+          ixx="0.0000768" iyy="0.0001380" izz="0.0001493"
+          ixy="0.0000018" iyz="0.0000071" ixz="-0.0000024" />
+    </inertial>
+  </xacro:extra_module>
   <xacro:macro name="foot_ball" params="parent">
-    <joint name="${parent}2${parent}_foot" type="revolute">
+    <joint name="${parent}2${parent}_foot" type="fixed">
       <parent link="${parent}"/>
       <child link="${parent}_foot"/>
-      <origin xyz="${general_link_length - 0.0115} 0 0" rpy="0 0 0"/>
+      <origin xyz="0.5115 0 0" rpy="0 0 0"/>
       <limit lower="0" upper="0" effort="100" velocity="100"/>
       <axis xyz="0 0 1" />
@@ -15,20 +36,19 @@
     <link name="${parent}_foot">
       <inertial>
-        <mass value="${foot_mass}"/>
-        <origin xyz="0 0 0" rpy="0 0 0"/>
+        <mass value="0.09"/>
+        <origin xyz="0.007 0 0" rpy="0 0 0"/>
         <inertia
-            ixx="${0.4 * foot_mass * foot_radius * foot_radius}"
-            iyy="${0.4 * foot_mass * foot_radius * foot_radius}"
-            izz="${0.4 * foot_mass * foot_radius * foot_radius}"
+            ixx="0.000055" iyy="0.000047" izz="0.000055"
             ixy="0" iyz="0" ixz="0"/>
       </inertial>
       <visual>
         <origin xyz="0 0 0" rpy="0 0 0"/>
-        <geometry> <sphere radius="${foot_radius}"/> </geometry>
-        <material name="black">  <color rgba="0 0 0 1"/> </material>
+	<geometry>
+          <mesh filename="package://tiger/urdf/v1/mesh/leg/leg_cap.dae"/>
+	</geometry>
       </visual>
       <collision>
         <origin xyz="0 0 0" rpy="0 0 0"/>
-        <geometry> <sphere radius="${foot_radius}"/> </geometry>
+        <geometry> <sphere radius="0.04"/> </geometry>
       </collision>
     </link>
