Commit message: [Tiger][WIP] improve the stand performance

File: robots/tiger/urdf/v1/link.urdf.xacro (robot description, xacro)
@@ -45,5 +45,5 @@
     <xacro:damping_factor link="joint_junction_link${self}"/>
     <joint name="joint${self}_pitch" type="revolute">
-      <limit effort="${max_joint_torque}" lower="${-pi/2}" upper="${pi/2}" velocity="${max_joint_vel}"/>
+      <limit effort="${max_joint_torque}" lower="${-pi/2 - 0.34}" upper="${pi/2 + 0.34}" velocity="${max_joint_vel}"/>
       <parent link="joint_junction_link${self}"/>
       <child link="${child}"/>
@@ -113,5 +113,5 @@
     #### joints ####
     <joint name="joint${child1}_yaw" type="revolute">
-      <limit effort="${max_joint_torque}" lower="${-pi/2}" upper="${pi/2}" velocity="${max_joint_vel}"/>
+      <limit effort="${max_joint_torque}" lower="${-pi/2 - 0.34}" upper="${pi/2 + 0.34}" velocity="${max_joint_vel}"/>
       <parent link="center_link"/>
       <child link="joint_junction_link${child1}"/>
@@ -121,5 +121,5 @@
     </joint>
     <joint name="joint${child2}_yaw" type="revolute">
-      <limit effort="${max_joint_torque}" lower="${-pi/2}" upper="${pi/2}" velocity="${max_joint_vel}"/>
+      <limit effort="${max_joint_torque}" lower="${-pi/2 - 0.34}" upper="${pi/2 + 0.34}" velocity="${max_joint_vel}"/>
       <parent link="center_link"/>
       <child link="joint_junction_link${child2}"/>
@@ -129,5 +129,5 @@
     </joint>
     <joint name="joint${child3}_yaw" type="revolute">
-      <limit effort="${max_joint_torque}" lower="${-pi/2}" upper="${pi/2}" velocity="${max_joint_vel}"/>
+      <limit effort="${max_joint_torque}" lower="${-pi/2 - 0.34}" upper="${pi/2 + 0.34}" velocity="${max_joint_vel}"/>
       <parent link="center_link"/>
       <child link="joint_junction_link${child3}"/>
@@ -137,5 +137,5 @@
     </joint>
     <joint name="joint${child4}_yaw" type="revolute">
-      <limit effort="${max_joint_torque}" lower="${-pi/2}" upper="${pi/2}" velocity="${max_joint_vel}"/>
+      <limit effort="${max_joint_torque}" lower="${-pi/2 - 0.34}" upper="${pi/2 + 0.34}" velocity="${max_joint_vel}"/>
       <parent link="center_link"/>
       <child link="joint_junction_link${child4}"/>
@@ -265,5 +265,5 @@
     <xacro:unless value="${self == child}">
       <joint name="joint${child}_yaw" type="revolute">
-        <limit effort="${max_joint_torque}" lower="${-pi/2}" upper="${pi}" velocity="${max_joint_vel}"/>
+        <limit effort="${max_joint_torque}" lower="${-pi/2 - 0.34}" upper="${pi/2 + 0.34}" velocity="${max_joint_vel}"/>
         <parent link="link${self}"/>
         <child link="joint_junction_link${child}"/>
