Commit message: [trirotor] add dae of baselink of trirotor

File: robots/trirotor/urdf/trirotor.urdf.xacro (robot description, xacro)
@@ -31,5 +31,5 @@
       <visual>
         <geometry>
-          <mesh filename="package://trirotor/urdf/mesh/kxr_flight_trirotor_base_link.STL" scale="0.001 0.001 0.001"/>
+          <mesh filename="package://trirotor/urdf/mesh/kxr_flight_trirotor_base_link.dae" scale="0.001 0.001 0.001"/>
           <origin rpy="0 0 0" xyz="0 0 0"/>
         </geometry>
