Commit message: [birotor] add dae of thruster and baselink

File: robots/birotor/urdf/birotor.urdf.xacro (robot description, xacro)
@@ -16,10 +16,10 @@
     <joint name="root_joint" type="fixed">
       <parent link="root"/>
-      <child link="fc"/>
+      <child link="base_link"/>
       <origin rpy="0 0 0" xyz="0 0 0"/>
       <axis xyz="0 0 1"/>
     </joint>
     ## link
-    <link name="fc">
+    <link name="base_link">
       <inertial>
         <origin xyz="0 0 0" rpy="0 0 0"/>
@@ -31,5 +31,5 @@
       <visual>
         <geometry>
-          <mesh filename="package://birotor/urdf/mesh/kxr_flight_unit_base_link.STL" scale="0.001 0.001 0.001"/>
+          <mesh filename="package://birotor/urdf/mesh/kxr_flight_unit_base_link.dae" scale="0.001 0.001 0.001"/>
           <origin rpy="0 0 0" xyz="0 0 0"/>
         </geometry>
@@ -42,9 +42,25 @@
       </collision>
     </link>
-    <xacro:damping_factor link="fc"/>
+    <xacro:damping_factor link="base_link"/>
+    <link name="fc">
+      <inertial>
+        <origin xyz="0 0 0" rpy="0 0 0"/>
+        <mass value="0.00001"/>
+        <inertia
+            ixx="0.000001" ixy="0.0" ixz="0.0"
+            iyy="0.000001" iyz="0.0"
+            izz="0.000002"/>
+      </inertial>
+    </link>
+    <joint name="fc_joint" type="fixed">
+      <child link="fc"/>
+      <parent link="base_link"/>
+      <origin rpy="0 0 0" xyz="0 0 0"/>
+      <axis xyz="0 0 1"/>
+    </joint>
     ## joints
-    <joint name="joint${child1}" type="revolute">
+    <joint name="gimbal${child1}" type="revolute">
       <limit effort="6.6" lower="-1.57" upper="1.57" velocity="3.0"/>
-      <parent link="fc"/>
+      <parent link="base_link"/>
       <child link="gimbal_link${child1}"/>
       <origin rpy="0 0 0" xyz="0 0.154 0.051"/>
@@ -52,7 +68,7 @@
       <dynamics damping="0.8" friction="0.0"/>
     </joint>
-    <joint name="joint${child2}" type="revolute">
+    <joint name="gimbal${child2}" type="revolute">
       <limit effort="6.6" lower="-1.57" upper="1.57" velocity="3.0"/>
-      <parent link="fc"/>
+      <parent link="base_link"/>
       <child link="gimbal_link${child2}"/>
       <origin rpy="0 0 0" xyz="0 -0.154 0.051"/>
@@ -63,5 +79,5 @@
     <transmission name="joint_tran${child1}">
       <type>transmission_interface/SimpleTransmission</type>
-      <joint name="joint${child1}">
+      <joint name="gimbal${child1}">
         <hardwareInterface>hardware_interface/EffortJointInterface</hardwareInterface>
       </joint>
@@ -73,5 +89,5 @@
     <transmission name="joint_tran${child2}">
       <type>transmission_interface/SimpleTransmission</type>
-      <joint name="joint${child2}">
+      <joint name="gimbal${child2}">
         <hardwareInterface>hardware_interface/EffortJointInterface</hardwareInterface>
       </joint>
@@ -81,5 +97,5 @@
       </actuator>
     </transmission>
-    <xacro:friction self="fc"/>
+    <xacro:friction self="base_link"/>
   </xacro:macro>
   <xacro:macro name="birotor_thrust_link" params="self rotor_direction">
@@ -103,5 +119,5 @@
         <origin rpy="0 0 ${pi/2 - pi/2 * rotor_direction}" xyz="0.0 0.0 0.0"/>
         <geometry>
-          <mesh filename="package://birotor/urdf/mesh/thrust_link_left_straight.STL" scale="0.001 0.001 0.001"/>
+          <mesh filename="package://birotor/urdf/mesh/thrust_link_left_straight.dae" scale="0.001 0.001 0.001"/>
         </geometry>
       </visual>

Commit message: [birotor][urdf] update parameters of urdf

File: robots/birotor/urdf/birotor.urdf.xacro (robot description, xacro)
@@ -23,9 +23,9 @@
     <link name="base_link">
       <inertial>
-        <origin xyz="0 0 0" rpy="0 0 0"/>
-        <mass value="0.970304"/>
+        <origin xyz="0 0 -0.034417" rpy="0 0 0"/>
+        <mass value="0.942442"/>
         <inertia
-            ixx="0.011445" iyy="0.011444" izz="0.021712"
-            ixy="-0.000000" ixz="-0.000000" iyz="0.000000"/>
+            ixx="0.015351" iyy="0.002766" izz="0.013177"
+            ixy="-0.000002" ixz="-0.000024" iyz="0.000002"/>
       </inertial>
       <visual>
@@ -104,9 +104,9 @@
     <link name="gimbal_link${self}">
       <inertial>
-        <origin xyz="0 0 0" rpy="0 0 0"/>
-        <mass value="0.237140"/>
+        <origin xyz="0 ${rotor_direction * 0.0835} 0" rpy="0 0 0"/>
+        <mass value="0.250950"/>
         <inertia
-            ixx="0.004029" iyy="0.003369" izz="0.006515"
-            ixy="-0.000000" ixz="-0.001310" iyz="0.000000"/>
+            ixx="0.001920" iyy="0.000249" izz="0.013177"
+            ixy="0.000002" ixz="-0.000024" iyz="0.000002"/>
       </inertial>
       <collision>

Commit message: [birotor] update mass of urdf

File: robots/birotor/urdf/birotor.urdf.xacro (robot description, xacro)
@@ -139,5 +139,5 @@
       <inertial>
         <origin xyz="0 0 0" rpy="0 0 0"/>
-        <mass value="0.2"/>
+        <mass value="0.00001"/>
         <inertia
             ixx="0.001" ixy="0.0" ixz="0.0"

Commit message: [birotor] fix coordinate and add fixed frame of gimbal in urdf

File: robots/birotor/urdf/birotor.urdf.xacro (robot description, xacro)
@@ -3,5 +3,6 @@
     xmlns:xacro="http://www.ros.org/wiki/xacro" name="birotor_link" >
   <xacro:macro name="birotor_center_link" params="child1 child2">
-    ## dummy
+    ## link
+    #### root link (vitrual) ####
     <link name="root">
       <inertial>
@@ -9,72 +10,105 @@
         <mass value="0.00001"/>
         <inertia
-            ixx="0.000001" ixy="0.0" ixz="0.0"
-            iyy="0.000001" iyz="0.0"
-            izz="0.000001"/>
-      </inertial>
-    </link>
+            ixx="0.000001" iyy="0.000001" izz="0.000001"
+            ixy="0.000000" ixz="0.000000" iyz="0.000000"/>
+      </inertial>
+    </link>
+    #### base link ####
+    <link name="base_link">
+      <inertial>
+        <origin xyz="0 0 -0.034417" rpy="0 0 0"/>
+        <mass value="0.942442"/>
+        <inertia
+            ixx="0.015351" iyy="0.002766" izz="0.013177"
+            ixy="-0.000002" ixz="-0.000024" iyz="0.000002"/>
+      </inertial>
+      <visual>
+        <geometry>
+          <mesh filename="package://birotor/urdf/mesh/kxr_flight_unit_base_link.dae" scale="0.001 0.001 0.001"/>
+          <origin xyz="0 0 0" rpy="0 0 0"/>
+        </geometry>
+      </visual>
+      <collision>
+        <origin xyz="0 0 0" rpy="0 0 0"/>
+        <geometry>
+          <box size="0.1 0.3 0.21"/>
+        </geometry>
+      </collision>
+    </link>
+    <xacro:damping_factor link="base_link"/>
+    #### rotor coord link (virtual)####
+    <link name="rotor_coord${child1}">
+      <inertial>
+        <origin xyz="0 0 0" rpy="0 0 0"/>
+        <mass value="0.00001"/>
+        <inertia
+            ixx="0.000001" iyy="0.000001" izz="0.000001"
+            ixy="0.000000" ixz="0.000000" iyz="0.000000"/>
+      </inertial>
+    </link>
+    <link name="rotor_coord${child2}">
+      <inertial>
+        <origin xyz="0 0 0" rpy="0 0 0"/>
+        <mass value="0.00001"/>
+        <inertia
+            ixx="0.000001" iyy="0.000001" izz="0.000001"
+            ixy="0.000000" ixz="0.000000" iyz="0.000000"/>
+      </inertial>
+    </link>
+    #### fcu frame ####
+    <link name="fc">
+      <inertial>
+        <origin xyz="0 0 0" rpy="0 0 0"/>
+        <mass value="0.00001"/>
+        <inertia
+            ixx="0.000001" iyy="0.000001" izz="0.000001"
+            ixy="0.000000" ixz="0.000000" iyz="0.000000"/>
+      </inertial>
+    </link>
+    ## joints ##
+    #### fixed frames (virtual) ####
     <joint name="root_joint" type="fixed">
       <parent link="root"/>
       <child link="base_link"/>
-      <origin rpy="0 0 0" xyz="0 0 0"/>
-      <axis xyz="0 0 1"/>
-    </joint>
-    ## link
-    <link name="base_link">
-      <inertial>
-        <origin xyz="0 0 -0.034417" rpy="0 0 0"/>
-        <mass value="0.942442"/>
-        <inertia
-            ixx="0.015351" iyy="0.002766" izz="0.013177"
-            ixy="-0.000002" ixz="-0.000024" iyz="0.000002"/>
-      </inertial>
-      <visual>
-        <geometry>
-          <mesh filename="package://birotor/urdf/mesh/kxr_flight_unit_base_link.dae" scale="0.001 0.001 0.001"/>
-          <origin rpy="0 0 0" xyz="0 0 0"/>
-        </geometry>
-      </visual>
-      <collision>
-        <origin xyz="0 0 0" rpy="0 0 0"/>
-        <geometry>
-          <box size="0.1 0.3 0.21"/>
-        </geometry>
-      </collision>
-    </link>
-    <xacro:damping_factor link="base_link"/>
-    <link name="fc">
-      <inertial>
-        <origin xyz="0 0 0" rpy="0 0 0"/>
-        <mass value="0.00001"/>
-        <inertia
-            ixx="0.000001" ixy="0.0" ixz="0.0"
-            iyy="0.000001" iyz="0.0"
-            izz="0.000002"/>
-      </inertial>
-    </link>
+      <origin xyz="0 0 0" rpy="0 0 0"/>
+      <axis xyz="0 0 1"/>
+    </joint>
     <joint name="fc_joint" type="fixed">
+      <parent link="base_link"/>
       <child link="fc"/>
+      <origin xyz="0 0 0" rpy="0 0 0"/>
+      <axis xyz="0 0 1"/>
+    </joint>
+    #### rotor coord link joint (virtual) ####
+    <joint name="rotor_coord_joint${child1}" type="fixed">
+      <parent link="base_link" />
+      <child link="rotor_coord${child1}"/>
+      <origin xyz="0 0.154 0.051" rpy="0 0 ${pi/2}"/>
+      <axis xyz="0 0 1"/>
+    </joint>
+    <joint name="rotor_coord_joint${child2}" type="fixed">
       <parent link="base_link"/>
-      <origin rpy="0 0 0" xyz="0 0 0"/>
-      <axis xyz="0 0 1"/>
-    </joint>
-    ## joints
+      <child link="rotor_coord${child2}"/>
+      <origin xyz="0 -0.154 0.051" rpy="0 0 ${-pi/2}"/>
+      <axis xyz="0 0 1"/>
+    </joint>
+    #### gimbal link joint ####
     <joint name="gimbal${child1}" type="revolute">
       <limit effort="6.6" lower="-1.57" upper="1.57" velocity="3.0"/>
-      <parent link="base_link"/>
+      <parent link="rotor_coord${child1}"/>
       <child link="gimbal_link${child1}"/>
-      <origin rpy="0 0 0" xyz="0 0.154 0.051"/>
-      <axis xyz="0 1 0"/>
+      <origin xyz="0 0 0" rpy="0 0 0"/>
+      <axis xyz="1 0 0"/>
       <dynamics damping="0.8" friction="0.0"/>
     </joint>
     <joint name="gimbal${child2}" type="revolute">
       <limit effort="6.6" lower="-1.57" upper="1.57" velocity="3.0"/>
-      <parent link="base_link"/>
+      <parent link="rotor_coord${child2}"/>
       <child link="gimbal_link${child2}"/>
-      <origin rpy="0 0 0" xyz="0 -0.154 0.051"/>
-      <axis xyz="0 1 0"/>
+      <origin xyz="0 0 0" rpy="0 0 0"/>
+      <axis xyz="1 0 0"/>
       <dynamics damping="0.8" friction="0.0"/>
     </joint>
-    #### hardware interface ####
+    ## hardware interface ##
     <transmission name="joint_tran${child1}">
       <type>transmission_interface/SimpleTransmission</type>
@@ -101,8 +135,8 @@
   <xacro:macro name="birotor_thrust_link" params="self rotor_direction">
     ## link
-    #### rotor parent link (virtual) ####
+    #### rotor link  ####
     <link name="gimbal_link${self}">
       <inertial>
-        <origin xyz="0 ${rotor_direction * 0.0835} 0" rpy="0 0 0"/>
+        <origin xyz="0.0835 0 0" rpy="0 0 0"/>
         <mass value="0.250950"/>
         <inertia
@@ -110,19 +144,19 @@
             ixy="0.000002" ixz="-0.000024" iyz="0.000002"/>
       </inertial>
+      <visual>
+        <origin xyz="0 0 0" rpy="0 0 ${-pi/2}"/>
+        <geometry>
+          <mesh filename="package://birotor/urdf/mesh/thrust_link_left_straight.dae" scale="0.001 0.001 0.001"/>
+        </geometry>
+      </visual>
       <collision>
-        <origin xyz="0 ${rotor_direction * 0.0835} 0" rpy="0 0 0"/>
+        <origin xyz="0.0835 0 0" rpy="0 0 0"/>
         <geometry>
           <cylinder radius="0.1" length="0.1"/>
         </geometry>
       </collision>
-      <visual>
-        <origin rpy="0 0 ${pi/2 - pi/2 * rotor_direction}" xyz="0.0 0.0 0.0"/>
-        <geometry>
-          <mesh filename="package://birotor/urdf/mesh/thrust_link_left_straight.dae" scale="0.001 0.001 0.001"/>
-        </geometry>
-      </visual>
     </link>
     <xacro:damping_factor link="gimbal_link${self}"/>
-    ## rotor parent link (virtual)
+    #### rotor parent link (virtual) ####
     <link name="rotor_parent${self}">
       <inertial>
@@ -130,10 +164,9 @@
         <mass value="0.00001"/>
         <inertia
-            ixx="0.000001" ixy="0.0" ixz="0.0"
-            iyy="0.000001" iyz="0.0"
-            izz="0.000001"/>
-      </inertial>
-    </link>
-    ## thrust link (virtual)
+            ixx="0.000001" iyy="0.000001" izz="0.000001"
+            ixy="0.000000" ixz="0.000000" iyz="0.000000"/>
+      </inertial>
+    </link>
+    #### thrust link (virtual) ####
     <link name="thrust${self}">
       <inertial>
@@ -141,17 +174,16 @@
         <mass value="0.00001"/>
         <inertia
-            ixx="0.001" ixy="0.0" ixz="0.0"
-            iyy="0.001" iyz="0.0"
-            izz="0.001"/>
+            ixx="0.000001" iyy="0.000001" izz="0.000001"
+            ixy="0.000000" ixz="0.000000" iyz="0.000000"/>
       </inertial>
     </link>
     <xacro:damping_factor link="thrust${self}"/>
-    #### joints ####
+    ## joints ##
     #### rotor parent link joint (virtual) ####
     <joint name="rotor_parent_link_joint${self}" type="fixed">
       <parent link="gimbal_link${self}"/>
       <child link="rotor_parent${self}"/>
-      <origin rpy="0 0 0" xyz="0 ${rotor_direction * 0.0835} 0"/>
-      <axis xyz="0 0 ${rotor_direction}"/>
+      <origin xyz="0.0835 0 0" rpy="0 0 0"/>
+      <axis xyz="0 0 1"/>
     </joint>
     #### rotor joint (virtual) ####
@@ -163,4 +195,5 @@
       <axis xyz="0 0 ${rotor_direction}"/>
     </joint>
+    #### hardware interface ####
     <transmission name="rotor_tran${self}">
       <type>transmission_interface/SimpleTransmission</type>
