Commit message: [Gimbalrotor][Controller&Model] Workaound new controling and modeling method using local coordinates of each thrust.

File: robots/gimbalrotor/urdf/gimbalrotor.urdf.xacro (robot description, xacro)
@@ -59,78 +59,69 @@
       <axis xyz="0 0 1"/>
     </joint>
-    ## joints
-    <joint name="gimbal${child1}" type="revolute">
-      <limit effort="6.6" lower="-1.57" upper="1.57" velocity="3.0"/>
-      <parent link="base_link"/>
-      <child link="gimbal_link${child1}"/>
-      <origin rpy="0 0 0" xyz="0 0.1 0.051"/>
-      <axis xyz="0 1 0"/>
-      <dynamics damping="0.8" friction="0.0"/>
-    </joint>
-    <joint name="gimbal${child2}" type="revolute">
-      <limit effort="6.6" lower="-1.57" upper="1.57" velocity="3.0"/>
-      <parent link="base_link"/>
-      <child link="gimbal_link${child2}"/>
-      <origin rpy="0 0 0" xyz="0 -0.1 0.051"/>
-      <axis xyz="0 1 0"/>
-      <dynamics damping="0.8" friction="0.0"/>
-    </joint>
-    <joint name="gimbal${child3}" type="revolute">
-      <limit effort="6.6" lower="-1.57" upper="1.57" velocity="3.0"/>
-      <parent link="base_link"/>
-      <child link="gimbal_link${child3}"/>
-      <origin rpy="0 0 ${pi/2}" xyz="-0.1 0 0.051"/>
-      <axis xyz="0 1 0"/>
-      <dynamics damping="0.8" friction="0.0"/>
-    </joint>
-    <joint name="gimbal${child4}" type="revolute">
-      <limit effort="6.6" lower="-1.57" upper="1.57" velocity="3.0"/>
-      <parent link="base_link"/>
-      <child link="gimbal_link${child4}"/>
-      <origin rpy="0 0 ${pi/2}" xyz="0.1 0 0.051"/>
-      <axis xyz="0 1 0"/>
-      <dynamics damping="0.8" friction="0.0"/>
-    </joint>
-    #### hardware interface ####
-    <transmission name="joint_tran${child1}">
-      <type>transmission_interface/SimpleTransmission</type>
-      <joint name="gimbal${child1}">
-        <hardwareInterface>hardware_interface/EffortJointInterface</hardwareInterface>
-      </joint>
-      <actuator name="servo${child1}">
-        <hardwareInterface>hardware_interface/EffortJointInterface</hardwareInterface>
-        <mechanicalReduction>1</mechanicalReduction>
-      </actuator>
-    </transmission>
-    <transmission name="joint_tran${child2}">
-      <type>transmission_interface/SimpleTransmission</type>
-      <joint name="gimbal${child2}">
-        <hardwareInterface>hardware_interface/EffortJointInterface</hardwareInterface>
-      </joint>
-      <actuator name="servo${child2}">
-        <hardwareInterface>hardware_interface/EffortJointInterface</hardwareInterface>
-        <mechanicalReduction>1</mechanicalReduction>
-      </actuator>
-    </transmission>
-    <transmission name="joint_tran${child3}">
-      <type>transmission_interface/SimpleTransmission</type>
-      <joint name="gimbal${child3}">
-        <hardwareInterface>hardware_interface/EffortJointInterface</hardwareInterface>
-      </joint>
-      <actuator name="servo${child3}">
-        <hardwareInterface>hardware_interface/EffortJointInterface</hardwareInterface>
-        <mechanicalReduction>1</mechanicalReduction>
-      </actuator>
-    </transmission>
-    <transmission name="joint_tran${child4}">
-      <type>transmission_interface/SimpleTransmission</type>
-      <joint name="gimbal${child4}">
-        <hardwareInterface>hardware_interface/EffortJointInterface</hardwareInterface>
-      </joint>
-      <actuator name="servo${child4}">
-        <hardwareInterface>hardware_interface/EffortJointInterface</hardwareInterface>
-        <mechanicalReduction>1</mechanicalReduction>
-      </actuator>
-    </transmission>
+    ## dummy gimbal parrents
+    <link name="gimbal_parent${child1}">
+      <inertial>
+        <origin rpy="0 0 0" xyz="0 0 0"/>
+        <mass value="0.00001"/>
+        <inertia
+            ixx="0.000001" ixy="0.0" ixz="0.0"
+            iyy="0.000001" iyz="0.0"
+            izz="0.000001"/>
+      </inertial>
+    </link>
+    <joint name="base_joint${child1}" type="fixed">
+      <parent link="base_link"/>
+      <child link="gimbal_parent${child1}"/>
+      <origin rpy="0 0 -${pi/4}" xyz="0.1 -0.1 0.051"/>
+      <axis xyz="0 0 1"/>
+    </joint>
+    <link name="gimbal_parent${child2}">
+      <inertial>
+        <origin rpy="0 0 0" xyz="0 0 0"/>
+        <mass value="0.00001"/>
+        <inertia
+            ixx="0.000001" ixy="0.0" ixz="0.0"
+            iyy="0.000001" iyz="0.0"
+            izz="0.000001"/>
+      </inertial>
+    </link>
+    <joint name="base_joint${child2}" type="fixed">
+      <parent link="base_link"/>
+      <child link="gimbal_parent${child2}"/>
+      <origin rpy="0 0 ${pi/4}" xyz="0.1 0.1 0.051"/>
+      <axis xyz="0 0 1"/>
+    </joint>
+    <link name="gimbal_parent${child3}">
+      <inertial>
+        <origin rpy="0 0 0" xyz="0 0 0"/>
+        <mass value="0.00001"/>
+        <inertia
+            ixx="0.000001" ixy="0.0" ixz="0.0"
+            iyy="0.000001" iyz="0.0"
+            izz="0.000001"/>
+      </inertial>
+    </link>
+    <joint name="base_joint${child3}" type="fixed">
+      <parent link="base_link"/>
+      <child link="gimbal_parent${child3}"/>
+      <origin rpy="0 0 ${pi*3/4}" xyz="-0.1 0.1 0.051"/>
+      <axis xyz="0 0 1"/>
+    </joint>
+    <link name="gimbal_parent${child4}">
+      <inertial>
+        <origin rpy="0 0 0" xyz="0 0 0"/>
+        <mass value="0.00001"/>
+        <inertia
+            ixx="0.000001" ixy="0.0" ixz="0.0"
+            iyy="0.000001" iyz="0.0"
+            izz="0.000001"/>
+      </inertial>
+    </link>
+    <joint name="base_joint${child4}" type="fixed">
+      <parent link="base_link"/>
+      <child link="gimbal_parent${child4}"/>
+      <origin rpy="0 0 ${pi*5/4}" xyz="-0.1 -0.1 0.051"/>
+      <axis xyz="0 0 1"/>
+    </joint>
     <xacro:friction self="base_link"/>
   </xacro:macro>
@@ -140,5 +131,5 @@
     <link name="gimbal_link${self}">
       <inertial>
-        <origin xyz="0 ${rotor_direction * 0.0835} 0" rpy="0 0 0"/>
+        <origin xyz="0.0835 0 0" rpy="0 0 0"/>
         <mass value="0.250950"/>
         <inertia
@@ -147,13 +138,13 @@
       </inertial>
       <collision>
-        <origin xyz="0 ${rotor_direction * 0.0835} 0" rpy="0 0 0"/>
-        <geometry>
-          <cylinder radius="0.05" length="0.1"/>
+        <origin xyz="0.0835 0 0" rpy="0 0 0"/>
+        <geometry>
+          <cylinder radius="0.0835" length="0.1"/>
         </geometry>
       </collision>
       <visual>
-        <origin xyz="0 ${rotor_direction * 0.0835} 0" rpy="0 0 0"/>
-        <geometry>
-          <cylinder radius="0.05" length="0.1"/>
+        <origin xyz="0.0835 0 0" rpy="0 0 0"/>
+        <geometry>
+          <cylinder radius="0.0835" length="0.1"/>
         </geometry>
       </visual>
@@ -184,9 +175,28 @@
     <xacro:damping_factor link="thrust${self}"/>
     #### joints ####
+    #### gimbal joints ####
+    <joint name="gimbal${self}" type="revolute">
+      <limit effort="6.6" lower="-1.57" upper="1.57" velocity="3.0"/>
+      <parent link="gimbal_parent${self}"/>
+      <child link="gimbal_link${self}"/>
+      <origin rpy="0 0 0" xyz="0 0 0"/>
+      <axis xyz="1 0 0"/>
+      <dynamics damping="0.8" friction="0.0"/>
+    </joint>
+    <transmission name="joint_tran${self}">
+      <type>transmission_interface/SimpleTransmission</type>
+      <joint name="gimbal${self}">
+        <hardwareInterface>hardware_interface/EffortJointInterface</hardwareInterface>
+      </joint>
+      <actuator name="servo${self}">
+        <hardwareInterface>hardware_interface/EffortJointInterface</hardwareInterface>
+        <mechanicalReduction>1</mechanicalReduction>
+      </actuator>
+    </transmission>
     #### rotor parent link joint (virtual) ####
     <joint name="rotor_parent_link_joint${self}" type="fixed">
       <parent link="gimbal_link${self}"/>
       <child link="rotor_parent${self}"/>
-      <origin rpy="0 0 0" xyz="0 ${rotor_direction * 0.0835} 0"/>
+      <origin rpy="0 0 0" xyz="0.0835 0 0"/>
       <axis xyz="0 0 ${rotor_direction}"/>
     </joint>

Commit message: [Gimbalrotor][URDF]add urdf model of ant module

File: robots/gimbalrotor/urdf/gimbalrotor.urdf.xacro (robot description, xacro)
@@ -23,20 +23,20 @@
     <link name="base_link">
       <inertial>
-        <origin xyz="0.0 0 0.0" rpy="0 0 0"/>
-        <mass value="1.037"/>
-        <inertia
-            ixx="0.004606" iyy="0.005835" izz="0.009493"
-            ixy="-0.00000" ixz="-0.000036" iyz="0.00000"/>
-      </inertial>
-      <visual>
-        <origin xyz="0 0 0" rpy="0 0 0"/>
-        <geometry>
-          <box size="0.2 0.2 0.05"/>
-        </geometry>
-      </visual>
-      <collision>
-        <origin xyz="0 0 0" rpy="0 0 0"/>
-        <geometry>
-          <box size="0.2 0.2 0.05"/>
+        <origin xyz="0.0 0.0 0.0165" rpy="0 0 0"/>
+        <mass value="0.1753"/>
+        <inertia
+            ixx="0.0004" iyy="0.0004" izz="0.0008"
+            ixy="0.00000" ixz="0.0000" iyz="0.00000"/>
+      </inertial>
+      <visual>
+        <origin xyz="0 0 0" rpy="0 0 0"/>
+        <geometry>
+          <mesh filename="package://gimbalrotor/urdf/mesh/base_link.STL"/>
+        </geometry>
+      </visual>
+      <collision>
+        <origin xyz="0 0 0" rpy="0 0 0"/>
+        <geometry>
+          <box size="0.25 0.25 0.035"/>
         </geometry>
       </collision>
@@ -59,67 +59,115 @@
       <axis xyz="0 0 1"/>
     </joint>
-    ## dummy gimbal parrents
-    <link name="gimbal_parent${child1}">
-      <inertial>
-        <origin rpy="0 0 0" xyz="0 0 0"/>
-        <mass value="0.00001"/>
-        <inertia
-            ixx="0.000001" ixy="0.0" ixz="0.0"
-            iyy="0.000001" iyz="0.0"
-            izz="0.000001"/>
-      </inertial>
-    </link>
-    <joint name="base_joint${child1}" type="fixed">
-      <parent link="base_link"/>
-      <child link="gimbal_parent${child1}"/>
-      <origin rpy="0 0 -${pi/4}" xyz="0.1 -0.1 0.051"/>
-      <axis xyz="0 0 1"/>
-    </joint>
-    <link name="gimbal_parent${child2}">
-      <inertial>
-        <origin rpy="0 0 0" xyz="0 0 0"/>
-        <mass value="0.00001"/>
-        <inertia
-            ixx="0.000001" ixy="0.0" ixz="0.0"
-            iyy="0.000001" iyz="0.0"
-            izz="0.000001"/>
-      </inertial>
-    </link>
-    <joint name="base_joint${child2}" type="fixed">
-      <parent link="base_link"/>
-      <child link="gimbal_parent${child2}"/>
-      <origin rpy="0 0 ${pi/4}" xyz="0.1 0.1 0.051"/>
-      <axis xyz="0 0 1"/>
-    </joint>
-    <link name="gimbal_parent${child3}">
-      <inertial>
-        <origin rpy="0 0 0" xyz="0 0 0"/>
-        <mass value="0.00001"/>
-        <inertia
-            ixx="0.000001" ixy="0.0" ixz="0.0"
-            iyy="0.000001" iyz="0.0"
-            izz="0.000001"/>
-      </inertial>
-    </link>
-    <joint name="base_joint${child3}" type="fixed">
-      <parent link="base_link"/>
-      <child link="gimbal_parent${child3}"/>
-      <origin rpy="0 0 ${pi*3/4}" xyz="-0.1 0.1 0.051"/>
-      <axis xyz="0 0 1"/>
-    </joint>
-    <link name="gimbal_parent${child4}">
-      <inertial>
-        <origin rpy="0 0 0" xyz="0 0 0"/>
-        <mass value="0.00001"/>
-        <inertia
-            ixx="0.000001" ixy="0.0" ixz="0.0"
-            iyy="0.000001" iyz="0.0"
-            izz="0.000001"/>
-      </inertial>
-    </link>
-    <joint name="base_joint${child4}" type="fixed">
-      <parent link="base_link"/>
-      <child link="gimbal_parent${child4}"/>
-      <origin rpy="0 0 ${pi*5/4}" xyz="-0.1 -0.1 0.051"/>
+    ## rotor arms
+    <link name="rotor_arm${child1}">
+      <inertial>
+        <origin xyz="0.0486 0 0.0161" rpy="0 0 0"/>
+        <mass value="0.088"/>
+        <inertia
+            ixx="0.000001" ixy="0.0" ixz="0.0"
+            iyy="0.0001" iyz="0.0"
+            izz="0.0001"/>
+      </inertial>
+      <visual>
+        <origin xyz="0 0 0" rpy="0 0 0"/>
+        <geometry>
+          <mesh filename="package://gimbalrotor/urdf/mesh/rotor_arm.STL"/>
+        </geometry>
+      </visual>
+      <collision>
+        <origin xyz="0 0 0" rpy="0 0 0"/>
+        <geometry>
+          <box size="0.131 0.0325 0.065"/>
+        </geometry>
+      </collision>
+    </link>
+    <joint name="base_arm_joint${child1}" type="fixed">
+      <parent link="base_link"/>
+      <child link="rotor_arm${child1}"/>
+      <origin rpy="0 0 ${pi/4}" xyz="0.051 0.051 0.0"/>
+      <axis xyz="0 0 1"/>
+    </joint>
+    <link name="rotor_arm${child2}">
+      <inertial>
+        <origin xyz="0.0486 0 0.0161" rpy="0 0 0"/>
+        <mass value="0.088"/>
+        <inertia
+            ixx="0.000001" ixy="0.0" ixz="0.0"
+            iyy="0.0001" iyz="0.0"
+            izz="0.0001"/>
+      </inertial>
+      <visual>
+        <origin xyz="0 0 0" rpy="0 0 0"/>
+        <geometry>
+          <mesh filename="package://gimbalrotor/urdf/mesh/rotor_arm.STL"/>
+        </geometry>
+      </visual>
+      <collision>
+        <origin xyz="0 0 0" rpy="0 0 0"/>
+        <geometry>
+          <box size="0.131 0.0325 0.065"/>
+        </geometry>
+      </collision>
+    </link>
+    <joint name="base_arm_joint${child2}" type="fixed">
+      <parent link="base_link"/>
+      <child link="rotor_arm${child2}"/>
+      <origin rpy="0 0 ${pi*3.0/4.0}" xyz="-0.051 0.051 0.0"/>
+      <axis xyz="0 0 1"/>
+    </joint>
+    <link name="rotor_arm${child3}">
+      <inertial>
+        <origin xyz="0.0486 0 0.0161" rpy="0 0 0"/>
+        <mass value="0.088"/>
+        <inertia
+            ixx="0.000001" ixy="0.0" ixz="0.0"
+            iyy="0.0001" iyz="0.0"
+            izz="0.0001"/>
+      </inertial>
+      <visual>
+        <origin xyz="0 0 0" rpy="0 0 0"/>
+        <geometry>
+          <mesh filename="package://gimbalrotor/urdf/mesh/rotor_arm.STL"/>
+        </geometry>
+      </visual>
+      <collision>
+        <origin xyz="0 0 0" rpy="0 0 0"/>
+        <geometry>
+          <box size="0.131 0.0325 0.065"/>
+        </geometry>
+      </collision>
+    </link>
+    <joint name="base_arm_joint${child3}" type="fixed">
+      <parent link="base_link"/>
+      <child link="rotor_arm${child3}"/>
+      <origin rpy="0 0 ${pi*5.0/4.0}" xyz="-0.051 -0.051 0.0"/>
+      <axis xyz="0 0 1"/>
+    </joint>
+    <link name="rotor_arm${child4}">
+      <inertial>
+        <origin xyz="0.0486 0 0.0161" rpy="0 0 0"/>
+        <mass value="0.088"/>
+        <inertia
+            ixx="0.000001" ixy="0.0" ixz="0.0"
+            iyy="0.0001" iyz="0.0"
+            izz="0.0001"/>
+      </inertial>
+      <visual>
+        <origin xyz="0 0 0" rpy="0 0 0"/>
+        <geometry>
+          <mesh filename="package://gimbalrotor/urdf/mesh/rotor_arm.STL"/>
+        </geometry>
+      </visual>
+      <collision>
+        <origin xyz="0 0 0" rpy="0 0 0"/>
+        <geometry>
+          <box size="0.131 0.0325 0.065"/>
+        </geometry>
+      </collision>
+    </link>
+    <joint name="base_arm_joint${child4}" type="fixed">
+      <parent link="base_link"/>
+      <child link="rotor_arm${child4}"/>
+      <origin rpy="0 0 ${-pi/4.0}" xyz="0.051 -0.051 0.0"/>
       <axis xyz="0 0 1"/>
     </joint>
@@ -131,20 +179,20 @@
     <link name="gimbal_link${self}">
       <inertial>
-        <origin xyz="0.0835 0 0" rpy="0 0 0"/>
-        <mass value="0.250950"/>
-        <inertia
-            ixx="0.001920" iyy="0.000249" izz="0.013177"
-            ixy="0.000002" ixz="-0.000024" iyz="0.000002"/>
-      </inertial>
-      <collision>
-        <origin xyz="0.0835 0 0" rpy="0 0 0"/>
-        <geometry>
-          <cylinder radius="0.0835" length="0.1"/>
-        </geometry>
-      </collision>
-      <visual>
-        <origin xyz="0.0835 0 0" rpy="0 0 0"/>
-        <geometry>
-          <cylinder radius="0.0835" length="0.1"/>
+        <origin xyz="0.018 0.00 0.00438" rpy="0 0 0"/>
+        <mass value="0.1095"/>
+        <inertia
+            ixx="0.00002989" iyy="0.00002848" izz="0.0002698"
+            ixy="0.0000" ixz="-0.0000" iyz="0.00000"/>
+      </inertial>
+      <collision>
+        <origin xyz="0.0 0 0" rpy="0 0 0"/>
+        <geometry>
+          <cylinder radius="0.018" length="0.033"/>
+        </geometry>
+      </collision>
+      <visual>
+        <origin xyz="0 0 0" rpy="0 0 0"/>
+        <geometry>
+          <mesh filename="package://gimbalrotor/urdf/mesh/rotor_module.STL"/>
         </geometry>
       </visual>
@@ -178,7 +226,7 @@
     <joint name="gimbal${self}" type="revolute">
       <limit effort="6.6" lower="-1.57" upper="1.57" velocity="3.0"/>
-      <parent link="gimbal_parent${self}"/>
+      <parent link="rotor_arm${self}"/>
       <child link="gimbal_link${self}"/>
-      <origin rpy="0 0 0" xyz="0 0 0"/>
+      <origin rpy="0 0 0" xyz="0.077 0 0.0385"/>
       <axis xyz="1 0 0"/>
       <dynamics damping="0.8" friction="0.0"/>
@@ -198,5 +246,5 @@
       <parent link="gimbal_link${self}"/>
       <child link="rotor_parent${self}"/>
-      <origin rpy="0 0 0" xyz="0.0835 0 0"/>
+      <origin rpy="0 0 0" xyz="0.018 0.00 0.00438"/>
       <axis xyz="0 0 ${rotor_direction}"/>
     </joint>

Commit message: [Gimbalrotor][URDF]modified gimbalrotor urdf

File: robots/gimbalrotor/urdf/gimbalrotor.urdf.xacro (robot description, xacro)
@@ -30,5 +30,5 @@
       </inertial>
       <visual>
-        <origin xyz="0 0 0" rpy="0 0 0"/>
+        <origin xyz="0 0 -0.0165" rpy="0 0 0"/>
         <geometry>
           <mesh filename="package://gimbalrotor/urdf/mesh/base_link.STL"/>
@@ -107,5 +107,5 @@
         <geometry>
           <box size="0.131 0.0325 0.065"/>
-        </geometry>
+        </geometry>p
       </collision>
     </link>

Commit message: [Gimbalrotor][URDF]modified upper limit angle of gimbal joint for KRS-3304R2

File: robots/gimbalrotor/urdf/gimbalrotor.urdf.xacro (robot description, xacro)
@@ -225,5 +225,5 @@
     #### gimbal joints ####
     <joint name="gimbal${self}" type="revolute">
-      <limit effort="6.6" lower="-1.57" upper="1.57" velocity="3.0"/>
+      <limit effort="6.6" lower="-2.0" upper="2.0" velocity="3.0"/>
       <parent link="rotor_arm${self}"/>
       <child link="gimbal_link${self}"/>
