Commit message: [agile quadrotor] update the configuration for quadorotor in gazebo

File: robots/agile_multirotor/urdf/quadrotor.gazebo.xacro (robot description, xacro)
@@ -11,4 +11,17 @@
     <mu1>0.1</mu1>
     <mu2>0.1</mu2>
+    <material>Gazebo/Red</material>
+  </gazebo>
+  <gazebo reference="thrust1">
+    <material>Gazebo/Black</material>
+  </gazebo>
+  <gazebo reference="thrust2">
+    <material>Gazebo/Black</material>
+  </gazebo>
+  <gazebo reference="thrust3">
+    <material>Gazebo/Black</material>
+  </gazebo>
+  <gazebo reference="thrust4">
+    <material>Gazebo/Black</material>
   </gazebo>
 </robot>

Commit message: [agile quadrotor] add obstacle world spawner and collision detection

File: robots/agile_multirotor/urdf/quadrotor.gazebo.xacro (robot description, xacro)
@@ -2,5 +2,5 @@
 <robot
     xmlns:xacro="http://www.ros.org/wiki/xacro" name="quadrotor" >
-  <xacro:arg name="robot_name" default="quadrotor" />
+  <xacro:arg name="robot_name" default="multirotor" />
   <!-- robot urdf -->
   <xacro:include filename="$(find agile_multirotor)/urdf/quadrotor.urdf.xacro" />
@@ -25,3 +25,75 @@
     <material>Gazebo/Black</material>
   </gazebo>
+  <!-- sensors -->
+  <!-- 1. stereo camera: depth, color camera -->
+  <xacro:extra_module name = "rgbd_camera_frame" parent = "main_body">
+    <origin xyz="0.13 0.0 0.0" rpy="0 0 0"/>
+    <inertial>
+      <mass value = "0.00001" />
+      <origin xyz="0 0 0" rpy="0 0 0"/>
+      <inertia
+          ixx="0.000001" ixy="0.0" ixz="0.0"
+          iyy="0.000001" iyz="0.0"
+          izz="0.000002"/>
+    </inertial>
+  </xacro:extra_module>
+  <xacro:extra_module name = "rgbd_camera_optical_frame" parent = "rgbd_camera_frame">
+    <origin xyz="0 0 0" rpy="${-pi / 2} 0 ${-pi / 2}"/>
+    <inertial>
+      <mass value = "0.00001" />
+      <origin xyz="0 0 0" rpy="0 0 0"/>
+      <inertia
+          ixx="0.000001" ixy="0.0" ixz="0.0"
+          iyy="0.000001" iyz="0.0"
+          izz="0.000002"/>
+    </inertial>
+  </xacro:extra_module>
+  <!-- gazebo plugin -->
+  <gazebo reference="rgbd_camera_frame">
+    <sensor type="depth" name="rgbd_depth_camera">
+      <update_rate>20.0</update_rate>
+      <camera name="head">
+        <horizontal_fov>1.57</horizontal_fov>
+        <image>
+          <width>1280</width>
+          <height>720</height>
+          <format>RGB</format>
+        </image>
+        <clip>
+          <near>0.02</near>
+          <far>300</far>
+        </clip>
+        <noise>
+          <type>gaussian</type>
+          <mean>0.0</mean>
+          <stddev>0.007</stddev>
+        </noise>
+      </camera>
+      <plugin name="depth_camera" filename="libgazebo_ros_openni_kinect.so">
+        <robotNamespace>$(arg robot_name)</robotNamespace>
+        <baseline>0.06</baseline>
+        <alwaysOn>true</alwaysOn>
+        <updateRate>0.0</updateRate>
+        <cameraName>rgbd</cameraName>
+        <imageTopicName>rgb/image_rect_color</imageTopicName>
+        <cameraInfoTopicName>rgb/camera_info</cameraInfoTopicName>
+        <depthImageTopicName>depth/depth_registered</depthImageTopicName>
+        <depthImageInfoTopicName>depth/camera_info</depthImageInfoTopicName>
+        <pointCloudTopicName>point_cloud/cloud_registered</pointCloudTopicName>
+        <frameName>rgbd_camera_optical_frame</frameName>
+        <pointCloudCutoff>0.05</pointCloudCutoff>
+        <pointCloudCutoffMax>10.0</pointCloudCutoffMax>
+        <distortionK1>0</distortionK1>
+        <distortionK2>0</distortionK2>
+        <distortionK3>0</distortionK3>
+        <distortionT1>0</distortionT1>
+        <distortionT2>0</distortionT2>
+        <CxPrime>0</CxPrime>
+        <Cx>0</Cx>
+        <Cy>0</Cy>
+        <focalLength>0</focalLength>
+        <hackBaseline>0</hackBaseline>
+      </plugin>
+    </sensor>
+  </gazebo>
 </robot>

Commit message: [Agile Multirotor] add virtual hokuyo 2D LiDAR model

File: robots/agile_multirotor/urdf/quadrotor.gazebo.xacro (robot description, xacro)
@@ -97,3 +97,39 @@
     </sensor>
   </gazebo>
+  <!-- hokuyo -->
+  <xacro:property name="ray_count" default="1081" />
+  <xacro:property name="max_angle" default="135" />
+  <gazebo reference="laser_frame">
+    <sensor type="ray" name="laser">
+      <always_on>true</always_on>
+      <update_rate>40</update_rate>
+      <pose>0 0 0 0 0 0</pose>
+      <visualize>false</visualize>
+      <ray>
+        <scan>
+          <horizontal>
+            <samples>${ray_count}</samples>
+            <resolution>1</resolution>
+            <min_angle>${-max_angle * M_PI/180}</min_angle>
+            <max_angle>${max_angle * M_PI/180}</max_angle>
+          </horizontal>
+        </scan>
+        <range>
+          <min>0.1</min>
+          <max>20.0</max>
+          <resolution>0.01</resolution>
+        </range>
+        <noise>
+          <type>gaussian</type>
+          <mean>0.0</mean>
+          <stddev>0.004</stddev>
+        </noise>
+      </ray>
+      <plugin name="gazebo_ros_laser_controller" filename="libgazebo_ros_laser.so">
+        <robotNamespace>$(arg robot_name)</robotNamespace>
+        <topicName>scan</topicName>
+        <frameName>laser_frame</frameName>
+      </plugin>
+    </sensor>
+  </gazebo>
 </robot>

File: robots/agile_multirotor/urdf/quadrotor.urdf.xacro (robot description, xacro)
@@ -121,7 +121,7 @@
     <!-- collision is not sphere to be able to  -->
     <collision>
-      <origin rpy="0 0 0" xyz="0 0 0"/>
+      <origin rpy="0 0 0" xyz="0 0 -0.05"/>
       <geometry>
-        <box size="0.3525 0.26 0.092" />
+        <box size="0.3525 0.26 0.04" />
       </geometry>
     </collision>
@@ -144,3 +144,8 @@
   <xacro:propeller_module id = "3" x = "${pos_bound/2}" y = "${pos_bound/2}" z = "${rotor_z}"  pich = "${opt_pich_3}" yaw = "${opt_yaw_3}" direction = "1" />
   <xacro:propeller_module id = "4" x = "${-pos_bound/2}" y = "${pos_bound/2}" z = "${rotor_z}"  pich = "${opt_pich_4}" yaw = "${opt_yaw_4}"  direction = "-1" />
+  <!-- hokuyo 2D LiDAR -->
+  <xacro:include filename="$(find hector_sensors_description)/urdf/hokuyo_utm30lx.urdf.xacro" />
+  <xacro:hokuyo_utm30lx_model name="laser" parent="main_body">
+    <origin xyz="0.0 0.0 0.06" rpy="0 0 0"/>
+  </xacro:hokuyo_utm30lx_model>
 </robot>

Commit message: [multirotor][hydrus] visualization for robomech poster

File: robots/agile_multirotor/urdf/quadrotor.gazebo.xacro (robot description, xacro)
@@ -11,4 +11,7 @@
     <mu1>1.0</mu1>
     <mu2>1.0</mu2>
+    <material>Gazebo/GreyTransparent</material>
+  </gazebo>
+  <gazebo reference="dummy_body_visualize">
     <material>Gazebo/Red</material>
   </gazebo>

File: robots/agile_multirotor/urdf/quadrotor.urdf.xacro (robot description, xacro)
@@ -38,10 +38,10 @@
       <xacro:insert_block name="inertial" />
       <xacro:if value="${visible == 1}">
-        <visual>
+        <!-- <visual>
           <origin rpy="0 0 0" xyz="0 0 0"/>
           <geometry>
             <mesh filename="${model_url}" scale= "${scale} ${scale} ${scale}"/>
           </geometry>
-        </visual>
+        </visual> -->
       </xacro:if>
     </link>
@@ -65,10 +65,10 @@
             izz="0.00001612"/>
       </inertial>
-      <visual>
+      <!-- <visual>
         <origin rpy="0 0 0" xyz="0 0 0"/>
         <geometry>
 	    <mesh filename="package://agile_multirotor/urdf/mesh/5_inch_propeller.stl" />
         </geometry>
-      </visual>
+      </visual> -->
     </link>
     <xacro:damping_factor link ="thrust${id}"/>
@@ -130,4 +130,25 @@
     </collision>
   </link>
+  <link name="dummy_body_visualize">
+    <inertial>
+      <mass value = "0.0001" />
+      <origin xyz="0 0 0 " rpy="0 0 0"/>
+      <inertia
+          ixx="0.000001" ixy="0.0000" ixz="0.0000"
+          iyy="0.000001" iyz="0.00000"
+          izz="0.000001"/>
+    </inertial>
+    <visual>
+      <origin rpy="0 0 0" xyz="0 0 0"/>
+      <geometry>
+       <mesh filename="package://agile_multirotor/urdf/mesh/quadrotor.stl" />
+      </geometry>
+    </visual>
+  </link>
+  <joint name="dummy_joint_2" type="fixed">
+    <parent link="main_body"/>
+    <child link="dummy_body_visualize"/>
+    <origin rpy="0 0 0" xyz="0.0 0.0 0.0"/>
+  </joint>
   <!-- spinal -->
   <xacro:extra_module name = "fc" parent = "main_body" visible = "0" >

File: robots/hydrus/robots/quad/default_mode_201907/robot.gazebo.xacro (robot description, xacro)
@@ -8,3 +8,9 @@
   <xacro:include filename="$(find aerial_robot_simulation)/xacro/spinal.gazebo.xacro" />
   <xacro:gazebo_spinal robot_name="$(arg robot_name)" />
+  <gazebo reference="dummy_body">
+    <material>Gazebo/GreyTransparent</material>
+  </gazebo>
+    <gazebo reference="dummy_body_visualize">
+    <material>Gazebo/Red</material>
+  </gazebo>
 </robot>

File: robots/hydrus/robots/quad/default_mode_201907/robot.urdf.xacro (robot description, xacro)
@@ -10,5 +10,5 @@
   <xacro:hydrus_link links="4" self="4" rotor_direction="1"  with_battery = "0" />
   <!-- special battery arrangement -->
-  <xacro:extra_module name = "bat1" parent = "link1" visible = "0"
+  <xacro:extra_module name = "bat1" parent = "link1" visible = "1"
                       model_url = "package://hydrus/urdf/mesh/battery/Kypom-3000-6s.dae" >
     <origin xyz="${link_length/2} 0.0 -0.048" rpy="0 0 0"/>
@@ -21,5 +21,5 @@
     </inertial>
   </xacro:extra_module>
-  <xacro:extra_module name = "bat2" parent = "link4" visible = "0"
+  <xacro:extra_module name = "bat2" parent = "link4" visible = "1"
                       model_url = "package://hydrus/urdf/mesh/battery/Kypom-3000-6s.dae" >
     <origin xyz="${link_length/2} 0.0 -0.048" rpy="0 0 0"/>
@@ -35,5 +35,5 @@
   <!-- 1.  processor -->
   <!-- 1.1 flight controller -->
-  <xacro:extra_module name = "fc" parent = "link2" visible = "0"
+  <xacro:extra_module name = "fc" parent = "link2" visible = "1"
                       model_url = "package://hydrus/urdf/mesh/ver2/flight_controller/spinal.dae"> <!-- same with intel euclid -->
     <origin xyz="${link_length / 2 + 0.2221} ${-4.4*0.001} 0.02135" rpy="0 0 0"/>
@@ -50,5 +50,5 @@
   <!-- 1.2 processor: jetson tx2 -->
   <!-- confirm the inertial parameter with real machine -->
-  <xacro:extra_module name = "pc" parent = "link3" visible = "0"
+  <xacro:extra_module name = "pc" parent = "link3" visible = "1"
                       model_url = "package://hydrus/urdf/mesh/ver2/processor/jetson_tx2_unit.dae" >
     <origin xyz="${link_length / 2 - 0.23775} 0.0 ${-0.01}" rpy="0 0 0"/>
@@ -101,5 +101,8 @@
   </xacro:extra_module>
   <!-- end: gps -->
-  <xacro:property name="body_radius" value=".50" />
+  <xacro:property name="body_radius" value="0.50" />
+  <material name="Dummy_body_color">
+    <color rgba="1.0 1.0 1.0 0.5"/>
+  </material>
   <link name="dummy_body">
     <inertial>
@@ -116,4 +119,5 @@
         <cylinder length="0.30" radius="${body_radius}"/>
       </geometry>
+      <material name="Dummy_body_color"/>
     </visual>
     <collision>
@@ -124,8 +128,31 @@
     </collision>
   </link>
-  <joint name="dummy_joint" type="fixed">
+  <joint name="dummy_joint_1" type="fixed">
     <parent link="link1"/>
     <child link="dummy_body"/>
     <origin rpy="0 0 0" xyz="${link_length* 0.5} ${link_length* 0.5} 0.0"/>
   </joint>
+   <link name="dummy_body_visualize">
+    <inertial>
+      <mass value = "0.0001" />
+      <origin xyz="0 0 0 " rpy="0 0 0"/>
+      <inertia
+          ixx="0.000001" ixy="0.0000" ixz="0.0000"
+          iyy="0.000001" iyz="0.00000"
+          izz="0.000001"/>
+    </inertial>
+    <visual>
+      <origin rpy="0 0 0" xyz="0 0 0"/>
+      <geometry>
+       <mesh
+        scale="2 2 2"
+        filename="package://agile_multirotor/urdf/mesh/quadrotor.stl" />
+      </geometry>
+    </visual>
+  </link>
+  <joint name="dummy_joint_2" type="fixed">
+    <parent link="link1"/>
+    <child link="dummy_body_visualize"/>
+    <origin rpy="0 0 0" xyz="${link_length* 0.5} ${link_length* 0.5} 0.0"/>
+  </joint>
 </robot>

File: robots/hydrus/urdf/common.xacro (robot description, xacro)
@@ -36,5 +36,5 @@
       </xacro:unless>
     </collision>
-    <visual>
+    <!-- <visual>
       <xacro:if value="${old_version == 1}">
         <origin rpy="0 0 0" xyz="${link_length* 0.5} 0 0"/>
@@ -59,5 +59,5 @@
         </geometry>
       </xacro:unless>
-    </visual>
+    </visual> -->
   </xacro:macro>
   <xacro:macro name="extra_module" params="name parent *origin *inertial visible:=0 model_url:=1 scale:=1">
@@ -70,10 +70,10 @@
       <xacro:insert_block name="inertial" />
       <xacro:if value="${visible == 1}">
-        <visual>
+        <!-- <visual>
           <origin rpy="0 0 0" xyz="0 0 0"/>
           <geometry>
             <mesh filename="${model_url}" scale= "${scale} ${scale} ${scale}"/>
           </geometry>
-        </visual>
+        </visual> -->
       </xacro:if>
     </link>
