Commit message: create collision_detection to get obstacle information from topic

File: robots/agile_multirotor/urdf/quadrotor.urdf.xacro (robot description, xacro)
@@ -121,6 +121,7 @@
     <collision>
       <origin rpy="0 0 0" xyz="0 0 0"/>
+      <!-- real quadrotor's size -->
       <geometry>
-        <box size="0.3525 0.26 0.092" />
+        <sphere radius="0.47"/>
       </geometry>
     </collision>

Commit message: make collision detection node

File: robots/agile_multirotor/urdf/quadrotor.urdf.xacro (robot description, xacro)
@@ -119,9 +119,9 @@
       </geometry>
     </visual>
+    <!-- collision is not sphere to be able to  -->
     <collision>
       <origin rpy="0 0 0" xyz="0 0 0"/>
-      <!-- real quadrotor's size -->
       <geometry>
-        <sphere radius="0.47"/>
+        <box size="0.3525 0.26 0.092" />
       </geometry>
     </collision>

Commit message: update urdf file to be the same parameter as the real quadrotor

File: robots/agile_multirotor/urdf/quadrotor.urdf.xacro (robot description, xacro)
@@ -106,10 +106,10 @@
   <link name="main_body">
     <inertial>
-      <mass value = "0.58229687" />
-      <origin xyz="-0.001214 0.00090575 -0.00144420" rpy="0 0 0"/>
+      <mass value = "0.807" />
+      <origin xyz="-0.0006654 0.0005569 -0.007939" rpy="0 0 0"/>
       <inertia
-          ixx="0.00371935" ixy="0.0000" ixz="0.0000"
-          iyy="0.00414867" iyz="0.00000"
-          izz="0.00745213"/>
+          ixx="0.004284" ixy="0.0000" ixz="0.0000"
+          iyy="0.004642" iyz="0.00000"
+          izz="0.007742"/>
     </inertial>
     <visual>
@@ -147,5 +147,5 @@
   <xacro:include filename="$(find hector_sensors_description)/urdf/hokuyo_utm30lx.urdf.xacro" />
   <xacro:hokuyo_utm30lx_model name="laser" parent="main_body">
-    <origin xyz="0.0 0.0 0.06" rpy="0 0 0"/>
+    <origin xyz="0.0 0.0 0.076" rpy="0 0 0"/>
   </xacro:hokuyo_utm30lx_model>
 </robot>

Commit message: change gazebo setting to show the size easily

File: robots/agile_multirotor/urdf/quadrotor.urdf.xacro (robot description, xacro)
@@ -116,12 +116,15 @@
       <origin rpy="0 0 0" xyz="0 0 0"/>
       <geometry>
-	<mesh filename="package://agile_multirotor/urdf/mesh/quadrotor.stl" />
+	<!-- <mesh filename="package://agile_multirotor/urdf/mesh/quadrotor.stl" /> -->
+        <cylinder length="0.3" radius="0.48"/>
       </geometry>
     </visual>
     <!-- collision is not sphere to be able to  -->
     <collision>
-      <origin rpy="0 0 0" xyz="0 0 -0.05"/>
+      <origin rpy="0 0 0" xyz="0 0 0.00"/>
       <geometry>
-        <box size="0.3525 0.26 0.04" />
+        <!-- <box size="0.3525 0.26 0.04" /> -->
+        <!-- length should be smaller not to collide to myself -->
+        <cylinder length="0.04" radius="0.50"/>
       </geometry>
     </collision>

Commit message: [change parameter] change the mass and inertia for long leg quadrotor model

File: robots/agile_multirotor/urdf/quadrotor.urdf.xacro (robot description, xacro)
@@ -106,10 +106,10 @@
   <link name="main_body">
     <inertial>
-      <mass value = "0.807" />
+      <mass value = "0.842" />
       <origin xyz="-0.0006654 0.0005569 -0.007939" rpy="0 0 0"/>
       <inertia
-          ixx="0.004284" ixy="0.0000" ixz="0.0000"
-          iyy="0.004642" iyz="0.00000"
-          izz="0.007742"/>
+          ixx="0.005272" ixy="0.0000" ixz="0.0000"
+          iyy="0.005809" iyz="0.00000"
+          izz="0.007425"/>
     </inertial>
     <visual>

Commit message: [Param Change] chage the mass parameter of the urdf file

File: robots/agile_multirotor/urdf/quadrotor.urdf.xacro (robot description, xacro)
@@ -106,10 +106,10 @@
   <link name="main_body">
     <inertial>
-      <mass value = "0.842" />
+      <mass value = "0.793" />
       <origin xyz="-0.0006654 0.0005569 -0.007939" rpy="0 0 0"/>
       <inertia
-          ixx="0.005272" ixy="0.0000" ixz="0.0000"
-          iyy="0.005809" iyz="0.00000"
-          izz="0.007425"/>
+          ixx="0.00664" ixy="0.0000" ixz="0.0000"
+          iyy="0.00714" iyz="0.00000"
+          izz="0.00916"/>
     </inertial>
     <visual>

Commit message: with weight and small difference of inertia

File: robots/agile_multirotor/urdf/quadrotor.urdf.xacro (robot description, xacro)
@@ -106,10 +106,10 @@
   <link name="main_body">
     <inertial>
-      <mass value = "0.793" />
+      <mass value = "1.056" />
       <origin xyz="-0.0006654 0.0005569 -0.007939" rpy="0 0 0"/>
       <inertia
-          ixx="0.00664" ixy="0.0000" ixz="0.0000"
-          iyy="0.00714" iyz="0.00000"
-          izz="0.00916"/>
+          ixx="0.01464" ixy="0.0000" ixz="0.0000"
+          iyy="0.01518" iyz="0.00000"
+          izz="0.01602"/>
     </inertial>
     <visual>

Commit message: change the radius of the visual of the quadrotor from 0.48 to 0.50

File: robots/agile_multirotor/urdf/quadrotor.urdf.xacro (robot description, xacro)
@@ -117,5 +117,5 @@
       <geometry>
 	<!-- <mesh filename="package://agile_multirotor/urdf/mesh/quadrotor.stl" /> -->
-        <cylinder length="0.3" radius="0.48"/>
+        <cylinder length="0.3" radius="0.50"/>
       </geometry>
     </visual>

Commit message: set the length of the cylinder of the collision is 0.005 to be the same length of the cylinder of the real quadrotor

File: robots/agile_multirotor/urdf/quadrotor.urdf.xacro (robot description, xacro)
@@ -126,5 +126,5 @@
         <!-- <box size="0.3525 0.26 0.04" /> -->
         <!-- length should be smaller not to collide to myself -->
-        <cylinder length="0.04" radius="0.50"/>
+        <cylinder length="0.005" radius="0.50"/>
       </geometry>
     </collision>

Commit message: change the main_body mass parameter with enclosure

File: robots/agile_multirotor/urdf/quadrotor.urdf.xacro (robot description, xacro)
@@ -106,5 +106,5 @@
   <link name="main_body">
     <inertial>
-      <mass value = "0.793" />
+      <mass value = "0.829" />
       <origin xyz="-0.0006654 0.0005569 -0.007939" rpy="0 0 0"/>
       <inertia

Commit message: change the mass for the new frame of the quadrotor

File: robots/agile_multirotor/urdf/quadrotor.urdf.xacro (robot description, xacro)
@@ -106,5 +106,5 @@
   <link name="main_body">
     <inertial>
-      <mass value = "0.829" />
+      <mass value = "0.847" />
       <origin xyz="-0.0006654 0.0005569 -0.007939" rpy="0 0 0"/>
       <inertia

Commit message: set the large quadrotor run w/o obstacles in long field

File: robots/agile_multirotor/urdf/quadrotor.urdf.xacro (robot description, xacro)
@@ -106,10 +106,10 @@
   <link name="main_body">
     <inertial>
-      <mass value = "1.11" />
+      <mass value = "1.30" />
       <origin xyz="-0.0006654 0.0005569 -0.007939" rpy="0 0 0"/>
       <inertia
-          ixx="0.02075" ixy="0.0000" ixz="0.0000"
-          iyy="0.02129" iyz="0.00000"
-          izz="0.03180"/>
+          ixx="0.04" ixy="0.0000" ixz="0.0000"
+          iyy="0.04" iyz="0.00000"
+          izz="0.06"/>
     </inertial>
     <visual>

Commit message: set the gain and the simulator for the small quadrotor

File: robots/agile_multirotor/urdf/quadrotor.urdf.xacro (robot description, xacro)
@@ -106,10 +106,10 @@
   <link name="main_body">
     <inertial>
-      <mass value = "1.30" />
+      <mass value = "0.847" />
       <origin xyz="-0.0006654 0.0005569 -0.007939" rpy="0 0 0"/>
       <inertia
-          ixx="0.04" ixy="0.0000" ixz="0.0000"
-          iyy="0.04" iyz="0.00000"
-          izz="0.06"/>
+          ixx="0.00664" ixy="0.0000" ixz="0.0000"
+          iyy="0.00714" iyz="0.00000"
+          izz="0.00916"/>
     </inertial>
     <visual>
@@ -117,5 +117,5 @@
       <geometry>
 	<!-- <mesh filename="package://agile_multirotor/urdf/mesh/quadrotor.stl" /> -->
-        <cylinder length="0.3" radius="0.50"/>
+        <cylinder length="0.3" radius="0.25"/>
       </geometry>
     </visual>
@@ -126,5 +126,5 @@
         <!-- <box size="0.3525 0.26 0.04" /> -->
         <!-- length should be smaller not to collide to myself -->
-        <cylinder length="0.005" radius="0.50"/>
+        <cylinder length="0.005" radius="0.25"/>
       </geometry>
     </collision>

Commit message: change mass from real quadrotor, and inertia from solidworks for new version

File: robots/agile_multirotor/urdf/quadrotor.urdf.xacro (robot description, xacro)
@@ -106,10 +106,10 @@
   <link name="main_body">
     <inertial>
-      <mass value = "0.847" />
+      <mass value = "0.852" />
       <origin xyz="-0.0006654 0.0005569 -0.007939" rpy="0 0 0"/>
       <inertia
-          ixx="0.00664" ixy="0.0000" ixz="0.0000"
-          iyy="0.00714" iyz="0.00000"
-          izz="0.00916"/>
+          ixx="0.00525" ixy="0.0000" ixz="0.0000"
+          iyy="0.00590" iyz="0.00000"
+          izz="0.00928"/>
     </inertial>
     <visual>

Commit message: [VISUALIZE] set tree shadow as false, and set collision check as r=0.325

File: robots/agile_multirotor/urdf/quadrotor.urdf.xacro (robot description, xacro)
@@ -117,5 +117,5 @@
       <geometry>
 	<!-- <mesh filename="package://agile_multirotor/urdf/mesh/quadrotor.stl" /> -->
-        <cylinder length="0.3" radius="0.25"/>
+        <cylinder length="0.3" radius="0.325"/>
       </geometry>
     </visual>
@@ -126,5 +126,5 @@
         <!-- <box size="0.3525 0.26 0.04" /> -->
         <!-- length should be smaller not to collide to myself -->
-        <cylinder length="0.005" radius="0.25"/>
+        <cylinder length="0.005" radius="0.325"/>
       </geometry>
     </collision>

Commit message: [agile_multirotor] change mass parameter for jetson version body

File: robots/agile_multirotor/urdf/quadrotor.urdf.xacro (robot description, xacro)
@@ -106,5 +106,5 @@
   <link name="main_body">
     <inertial>
-      <mass value = "0.852" />
+      <mass value = "0.985" />
       <origin xyz="-0.0006654 0.0005569 -0.007939" rpy="0 0 0"/>
       <inertia

Commit message: [agile_multirotor] set livox config to quadrotor.urdf

File: robots/agile_multirotor/urdf/quadrotor.urdf.xacro (robot description, xacro)
@@ -163,4 +163,15 @@
     </inertial>
   </xacro:extra_module>
+  <!-- livox mid360 -->
+  <xacro:extra_module name = "lidar_imu" parent = "main_body" visible = "0" > <!-- should be IMU frame -->
+    <origin xyz="${0.011} ${0.02329} ${0.0425 + 0.047 - 0.04412}" rpy="0 0 0"/> <!-- TODO: the true pos -->
+    <inertial>
+      <mass value = "00" />
+      <origin xyz="0 0 0" rpy="0 0 0"/>
+      <inertia
+          ixx="0.0" ixy="0.0" ixz="0.0"
+          iyy="0.0" iyz="0.0" izz="0.0"/>
+    </inertial>
+  </xacro:extra_module>
   <!-- propellers -->
   <xacro:propeller_module id = "1" x = "${-pos_bound/2}" y = "${-pos_bound/2}" z = "${rotor_z}" pich = "${opt_pich_1}" yaw = "${opt_yaw_1}" direction = "1" />

Commit message: [agile_multirotor] set true lidar_imu position based on real quadrotor

File: robots/agile_multirotor/urdf/quadrotor.urdf.xacro (robot description, xacro)
@@ -165,5 +165,5 @@
   <!-- livox mid360 -->
   <xacro:extra_module name = "lidar_imu" parent = "main_body" visible = "0" > <!-- should be IMU frame -->
-    <origin xyz="${0.011} ${0.02329} ${0.0425 + 0.047 - 0.04412}" rpy="0 0 0"/> <!-- TODO: the true pos -->
+    <origin xyz="${0.0} ${0.0} ${0.103 + 0.047 - 0.04412}" rpy="0 0 0"/> <!-- TODO: the true pos -->
     <inertial>
       <mass value = "00" />

Commit message: [agile_multirotor] set correct mass param based on real whole weight

File: robots/agile_multirotor/urdf/quadrotor.urdf.xacro (robot description, xacro)
@@ -106,5 +106,5 @@
   <link name="main_body">
     <inertial>
-      <mass value = "0.985" />
+      <mass value = "0.833" />
       <origin xyz="-0.0006654 0.0005569 -0.007939" rpy="0 0 0"/>
       <inertia

Commit message: [debug][agile_multirotor] correct lidar_imu position based on manta document

File: robots/agile_multirotor/urdf/quadrotor.urdf.xacro (robot description, xacro)
@@ -165,5 +165,5 @@
   <!-- livox mid360 -->
   <xacro:extra_module name = "lidar_imu" parent = "main_body" visible = "0" > <!-- should be IMU frame -->
-    <origin xyz="${0.0} ${0.0} ${0.103 + 0.047 - 0.04412}" rpy="0 0 0"/> <!-- TODO: the true pos -->
+    <origin xyz="${0.011} ${0.02329} ${0.103 + 0.047 - 0.04412}" rpy="0 0 0"/> <!-- TODO: the true pos -->
     <inertial>
       <mass value = "00" />

Commit message: [agile_multirotor][urdf] add battery urdf with information of mass

File: robots/agile_multirotor/urdf/quadrotor.urdf.xacro (robot description, xacro)
@@ -174,4 +174,15 @@
     </inertial>
   </xacro:extra_module>
+    <!-- battery -->
+  <xacro:extra_module name = "battery" parent = "main_body" visible = "0" > <!-- should be IMU frame -->
+    <origin xyz="0 0 -0.050" rpy="0 0 0"/> <!-- TODO: the true pos -->
+    <inertial>
+      <mass value = "0.270" />
+      <origin xyz="0 0 0" rpy="0 0 0"/>
+      <inertia
+          ixx="0.0" ixy="0.0" ixz="0.0"
+          iyy="0.0" iyz="0.0" izz="0.0"/>
+    </inertial>
+  </xacro:extra_module>
   <!-- propellers -->
   <xacro:propeller_module id = "1" x = "${-pos_bound/2}" y = "${-pos_bound/2}" z = "${rotor_z}" pich = "${opt_pich_1}" yaw = "${opt_yaw_1}" direction = "1" />

Commit message: [agile_multirotor] reset livox and battery urdf file from solidworks file

File: robots/agile_multirotor/urdf/quadrotor.urdf.xacro (robot description, xacro)
@@ -167,9 +167,9 @@
     <origin xyz="${0.011} ${0.02329} ${0.103 + 0.047 - 0.04412}" rpy="0 0 0"/> <!-- TODO: the true pos -->
     <inertial>
-      <mass value = "00" />
-      <origin xyz="0 0 0" rpy="0 0 0"/>
+      <mass value = "0.262" />
+      <origin xyz="-0.011 -0.02329 0.04412" rpy="0 0 0"/>
       <inertia
-          ixx="0.0" ixy="0.0" ixz="0.0"
-          iyy="0.0" iyz="0.0" izz="0.0"/>
+          ixx="0.00111" ixy="0.0" ixz="0.0"
+          iyy="0.00125" iyz="0.0" izz="0.00122"/>
     </inertial>
   </xacro:extra_module>
@@ -181,6 +181,6 @@
       <origin xyz="0 0 0" rpy="0 0 0"/>
       <inertia
-          ixx="0.0" ixy="0.0" ixz="0.0"
-          iyy="0.0" iyz="0.0" izz="0.0"/>
+          ixx="0.000407" ixy="0.0" ixz="0.0"
+          iyy="0.000438" iyz="0.0" izz="0.000048"/>
     </inertial>
   </xacro:extra_module>

Commit message: [agile_multirotor] show agile_flight obstacle radius from 0.325 to 0.30 to pass through walls

File: robots/agile_multirotor/urdf/quadrotor.urdf.xacro (robot description, xacro)
@@ -126,5 +126,5 @@
         <!-- <box size="0.3525 0.26 0.04" /> -->
         <!-- length should be smaller not to collide to myself -->
-        <cylinder length="0.005" radius="0.325"/>
+        <cylinder length="0.005" radius="0.30"/>
       </geometry>
     </collision>
