Commit message: [Ants] add docking mech plugin to urdf

File: robots/gimbalrotor/robots/quad/gimbalrotor.gazebo.xacro (robot description, xacro)
@@ -7,3 +7,20 @@
   <xacro:include filename="$(find aerial_robot_simulation)/xacro/spinal.gazebo.xacro" />
   <xacro:gazebo_spinal robot_name="$(arg robot_name)" mag_frame="fc" />
+  <!-- gazebo plugin for docking mech -->
+  <gazebo>
+    <plugin name="gazebo_grasp_fix" filename="libgazebo_grasp_fix.so">
+      <arm>
+        <arm_name>docking_mech</arm_name>
+        <palm_link>dummy_palm</palm_link>
+        <gripper_link>dummy_gripper</gripper_link>
+      </arm>
+      <forces_angle_tolerance>90</forces_angle_tolerance>
+      <update_rate>50</update_rate>
+      <grip_count_threshold>0</grip_count_threshold>
+      <max_grip_count>1</max_grip_count>
+      <release_tolerance>1</release_tolerance>
+      <disable_collisions_on_attach>false</disable_collisions_on_attach>
+      <contact_topic>__default_topic__</contact_topic>
+    </plugin>
+  </gazebo>
 </robot>

File: robots/gimbalrotor/robots/quad/gimbalrotor.urdf.xacro (robot description, xacro)
@@ -9,3 +9,70 @@
   <xacro:gimbalrotor_thrust_link self="3" rotor_direction="1"/>
   <xacro:gimbalrotor_thrust_link self="4" rotor_direction="-1"/>
+  ##### dummy grasp links ####
+  <joint name="base_dummy_arm_joint" type="fixed">
+    <parent link="base_link"/>
+    <child link="dummy_arm"/>
+    <origin xyz="0.22 0 0.1455" rpy="0 0 0"/>
+  </joint>
+  <link name="dummy_arm">
+    <inertial>
+      <mass value = "0.01" />
+      <origin xyz="0.05 0 0" rpy="0 0 0"/>
+      <inertia
+          ixx="0.0001" ixy="0.0000" ixz="0.0000"
+          iyy="0.0001" iyz="0.0000" izz="0.0001"/>
+    </inertial>
+  </link>
+  <joint name="dummy_arm_palm_joint" type="revolute">
+    <parent link="dummy_arm"/>
+    <child link="dummy_palm"/>
+    <origin xyz="0.02 0 0" rpy="0 0 0"/>
+    <axis xyz="1 0 0"/>
+    <limit lower="0" upper="0" effort="0" velocity="0"/>
+    <dynamics damping="0.2" friction="0.02"/>
+  </joint>
+  <link name="dummy_palm">
+    <inertial>
+      <mass value = "0.001" />
+      <origin xyz="0 0 0" rpy="0 0 0"/>
+      <inertia
+          ixx="0.0001" ixy="0.0000" ixz="0.0000"
+          iyy="0.0001" iyz="0.0000" izz="0.0001"/>
+    </inertial>
+    <collision>
+      <origin xyz="0 0 0" rpy="0 0 0"/>
+      <geometry>
+        <box size="0.04 0.04 0.04"/>
+      </geometry>
+    </collision>
+  </link>
+  <joint name="dummy_palm_gripper_joint" type="revolute">
+    <parent link="dummy_palm"/>
+    <child link="dummy_gripper"/>
+    <origin xyz="0 0 0" rpy="0 0 0"/>
+    <axis xyz="1 0 0"/>
+    <limit lower="0" upper="0" effort="0" velocity="0"/>
+    <dynamics damping="0.2" friction="0.02"/>
+  </joint>
+  <link name="dummy_gripper">
+    <inertial>
+      <mass value = "0.001" />
+      <origin xyz="0.0 0 0" rpy="0 0 0"/>
+      <inertia
+          ixx="0.0001" ixy="0.0000" ixz="0.0000"
+          iyy="0.0001" iyz="0.0000" izz="0.0001"/>
+    </inertial>
+    <collision>
+      <origin xyz="0 0 0" rpy="0 0 0"/>
+      <geometry>
+        <box size="0.04 0.04 0.04"/>
+      </geometry>
+    </collision>
+    <visual>
+      <origin xyz="0 0 0" rpy="0.0 0 0"/>
+      <geometry>
+        <box size="0.04 0.04 0.04"/>
+      </geometry>
+    </visual>
+  </link>
 </robot>

Commit message: [Gimbalrotor] remove needless files and portions for normal gimbalrotor.

File: robots/gimbalrotor/robots/quad/gimbalrotor.gazebo.xacro (robot description, xacro)
@@ -7,20 +7,3 @@
   <xacro:include filename="$(find aerial_robot_simulation)/xacro/spinal.gazebo.xacro" />
   <xacro:gazebo_spinal robot_name="$(arg robot_name)" mag_frame="fc" />
-  <!-- gazebo plugin for docking mech -->
-  <gazebo>
-    <plugin name="gazebo_grasp_fix" filename="libgazebo_grasp_fix.so">
-      <arm>
-        <arm_name>docking_mech</arm_name>
-        <palm_link>dummy_palm</palm_link>
-        <gripper_link>dummy_gripper</gripper_link>
-      </arm>
-      <forces_angle_tolerance>90</forces_angle_tolerance>
-      <update_rate>50</update_rate>
-      <grip_count_threshold>0</grip_count_threshold>
-      <max_grip_count>1</max_grip_count>
-      <release_tolerance>1</release_tolerance>
-      <disable_collisions_on_attach>false</disable_collisions_on_attach>
-      <contact_topic>__default_topic__</contact_topic>
-    </plugin>
-  </gazebo>
 </robot>

File: robots/gimbalrotor/robots/quad/gimbalrotor.urdf.xacro (robot description, xacro)
@@ -9,70 +9,3 @@
   <xacro:gimbalrotor_thrust_link self="3" rotor_direction="1"/>
   <xacro:gimbalrotor_thrust_link self="4" rotor_direction="-1"/>
-  ##### dummy grasp links ####
-  <joint name="base_dummy_arm_joint" type="fixed">
-    <parent link="base_link"/>
-    <child link="dummy_arm"/>
-    <origin xyz="0.22 0 0.1455" rpy="0 0 0"/>
-  </joint>
-  <link name="dummy_arm">
-    <inertial>
-      <mass value = "0.01" />
-      <origin xyz="0.05 0 0" rpy="0 0 0"/>
-      <inertia
-          ixx="0.0001" ixy="0.0000" ixz="0.0000"
-          iyy="0.0001" iyz="0.0000" izz="0.0001"/>
-    </inertial>
-  </link>
-  <joint name="dummy_arm_palm_joint" type="revolute">
-    <parent link="dummy_arm"/>
-    <child link="dummy_palm"/>
-    <origin xyz="0.02 0 0" rpy="0 0 0"/>
-    <axis xyz="1 0 0"/>
-    <limit lower="0" upper="0" effort="0" velocity="0"/>
-    <dynamics damping="0.2" friction="0.02"/>
-  </joint>
-  <link name="dummy_palm">
-    <inertial>
-      <mass value = "0.001" />
-      <origin xyz="0 0 0" rpy="0 0 0"/>
-      <inertia
-          ixx="0.0001" ixy="0.0000" ixz="0.0000"
-          iyy="0.0001" iyz="0.0000" izz="0.0001"/>
-    </inertial>
-    <collision>
-      <origin xyz="0 0 0" rpy="0 0 0"/>
-      <geometry>
-        <box size="0.04 0.04 0.04"/>
-      </geometry>
-    </collision>
-  </link>
-  <joint name="dummy_palm_gripper_joint" type="revolute">
-    <parent link="dummy_palm"/>
-    <child link="dummy_gripper"/>
-    <origin xyz="0 0 0" rpy="0 0 0"/>
-    <axis xyz="1 0 0"/>
-    <limit lower="0" upper="0" effort="0" velocity="0"/>
-    <dynamics damping="0.2" friction="0.02"/>
-  </joint>
-  <link name="dummy_gripper">
-    <inertial>
-      <mass value = "0.001" />
-      <origin xyz="0.0 0 0" rpy="0 0 0"/>
-      <inertia
-          ixx="0.0001" ixy="0.0000" ixz="0.0000"
-          iyy="0.0001" iyz="0.0000" izz="0.0001"/>
-    </inertial>
-    <collision>
-      <origin xyz="0 0 0" rpy="0 0 0"/>
-      <geometry>
-        <box size="0.04 0.04 0.04"/>
-      </geometry>
-    </collision>
-    <visual>
-      <origin xyz="0 0 0" rpy="0.0 0 0"/>
-      <geometry>
-        <box size="0.04 0.04 0.04"/>
-      </geometry>
-    </visual>
-  </link>
 </robot>
