Commit message: [hydrus_gripper] set mass as the uruav_graphene battery

File: robots/hydrus_gripper/urdf/fixed_link.urdf.xacro (robot description, xacro)
@@ -141,5 +141,5 @@
         <inertial>
           <origin xyz="0 0 0" rpy="0 0 0"/>
-          <mass value="0.194"/>
+          <mass value="0.158"/>
           <inertia
               ixx="0.00005" iyy="0.00012" izz="0.00011"
