Commit message: [COLLISION CHECK BY CYLINDER] run in 90 deg's hydrus & collision check is conducted on any size of the cylinder

File: robots/hydrus/robots/quad/default_mode_201907/robot.urdf.xacro (robot description, xacro)
@@ -10,5 +10,5 @@
   <xacro:hydrus_link links="4" self="4" rotor_direction="1"  with_battery = "0" />
   <!-- special battery arrangement -->
-  <xacro:extra_module name = "bat1" parent = "link1" visible = "1"
+  <xacro:extra_module name = "bat1" parent = "link1" visible = "0"
                       model_url = "package://hydrus/urdf/mesh/battery/Kypom-3000-6s.dae" >
     <origin xyz="${link_length/2} 0.0 -0.048" rpy="0 0 0"/>
@@ -21,5 +21,5 @@
     </inertial>
   </xacro:extra_module>
-  <xacro:extra_module name = "bat2" parent = "link4" visible = "1"
+  <xacro:extra_module name = "bat2" parent = "link4" visible = "0"
                       model_url = "package://hydrus/urdf/mesh/battery/Kypom-3000-6s.dae" >
     <origin xyz="${link_length/2} 0.0 -0.048" rpy="0 0 0"/>
@@ -35,5 +35,5 @@
   <!-- 1.  processor -->
   <!-- 1.1 flight controller -->
-  <xacro:extra_module name = "fc" parent = "link2" visible = "1"
+  <xacro:extra_module name = "fc" parent = "link2" visible = "0"
                       model_url = "package://hydrus/urdf/mesh/ver2/flight_controller/spinal.dae"> <!-- same with intel euclid -->
     <origin xyz="${link_length / 2 + 0.2221} ${-4.4*0.001} 0.02135" rpy="0 0 0"/>
@@ -50,5 +50,5 @@
   <!-- 1.2 processor: jetson tx2 -->
   <!-- confirm the inertial parameter with real machine -->
-  <xacro:extra_module name = "pc" parent = "link3" visible = "1"
+  <xacro:extra_module name = "pc" parent = "link3" visible = "0"
                       model_url = "package://hydrus/urdf/mesh/ver2/processor/jetson_tx2_unit.dae" >
     <origin xyz="${link_length / 2 - 0.23775} 0.0 ${-0.01}" rpy="0 0 0"/>
@@ -65,5 +65,5 @@
   <!-- 2.  sensor -->
   <!-- 2.1 leddar one -->
-  <xacro:extra_module name = "leddarone" parent = "link3" visible = "1"
+  <xacro:extra_module name = "leddarone" parent = "link3" visible = "0"
                       model_url = "package://hydrus/urdf/mesh/sensor/leddar_one_tx2_attached_mode.dae">
     <origin xyz="${link_length/2 - 0.1855} 0.0 -0.0626" rpy="${pi} 0 0"/>
@@ -78,5 +78,5 @@
   <!-- end: leddar one -->
   <!-- 2.2 gps -->
-  <xacro:extra_module name = "gps" parent = "link2" visible = "1"
+  <xacro:extra_module name = "gps" parent = "link2" visible = "0"
                       model_url = "package://hydrus/urdf/mesh/sensor/gps_ublox_m8n.dae">
     <origin xyz="${link_length/2 + 0.1925} 0.0 0.152" rpy="0 0 0"/>
@@ -101,3 +101,30 @@
   </xacro:extra_module>
   <!-- end: gps -->
+  <link name="dummy_body">
+    <inertial>
+      <mass value = "0.0001" />
+      <origin xyz="0 0 0 " rpy="0 0 0"/>
+      <inertia
+          ixx="0.000001" ixy="0.0000" ixz="0.0000"
+          iyy="0.000001" iyz="0.00000"
+          izz="0.000001"/>
+    </inertial>
+    <visual>
+      <origin rpy="0 0 0" xyz="0 0 0"/>
+      <geometry>
+        <cylinder length="0.30" radius="0.50"/>
+      </geometry>
+    </visual>
+    <collision>
+        <origin rpy="0 0 0" xyz="0 0 0"/>
+        <geometry>
+          <cylinder length="0.02" radius="0.50"/>
+        </geometry>
+    </collision>
+  </link>
+  <joint name="dummy_joint" type="fixed">
+    <parent link="link1"/>
+    <child link="dummy_body"/>
+    <origin rpy="0 0 0" xyz="${link_length* 0.5} ${link_length* 0.5} 0.0"/>
+  </joint>
 </robot>

File: robots/hydrus/urdf/link.urdf.xacro (robot description, xacro)
@@ -16,5 +16,5 @@
                 ixy="0.000021" ixz="0.000372" iyz="0.000000"/>
           </inertial>
-          <xacro:link_model type="head" />
+          <!-- <xacro:link_model type="head" /> -->
         </xacro:if>
         <xacro:unless value="${self == 1}">
@@ -28,5 +28,5 @@
                   ixy="0.000020" ixz="-0.000076" iyz="0.000000"/>
             </inertial>
-            <xacro:link_model type="end" />
+            <!-- <xacro:link_model type="end" /> -->
           </xacro:if>
           <xacro:unless value="${self == links}">
@@ -39,5 +39,5 @@
                   ixy="0.000021" ixz="0.000260" iyz="0.000000"/>
             </inertial>
-            <xacro:link_model type="general" />
+            <!-- <xacro:link_model type="general" /> -->
           </xacro:unless>
         </xacro:unless>
@@ -78,5 +78,5 @@
             </inertial>
           </xacro:unless>
-          <xacro:link_model type="1" />
+          <!-- <xacro:link_model type="1" /> -->
         </xacro:if>
         <xacro:unless value="${self == 1}">
@@ -112,5 +112,5 @@
               </inertial>
             </xacro:unless>
-            <xacro:link_model type="4" />
+            <!-- <xacro:link_model type="4" /> -->
           </xacro:if>
           <xacro:unless value="${self == links}">
@@ -146,5 +146,5 @@
                 </inertial>
               </xacro:unless>
-              <xacro:link_model type="2" />
+              <!-- <xacro:link_model type="2" /> -->
             </xacro:if>
             <!-- general -->
@@ -179,5 +179,5 @@
                 </inertial>
               </xacro:unless>
-              <xacro:link_model type="3" />
+              <!-- <xacro:link_model type="3" /> -->
             </xacro:unless>
           </xacro:unless>
@@ -214,10 +214,10 @@
             izz="0.00002"/>
       </inertial>
-      <collision>
+      <!-- <collision>
         <origin rpy="0 0 0" xyz="0 0 0"/>
         <geometry>
           <cylinder length="0.1" radius="${protector_radius + 0.01}"/>
         </geometry>
-      </collision>
+      </collision> -->
     </link>
     <xacro:damping_factor link ="thrust${self}"/>

Commit message: [refactoring] set variable body_radius

File: robots/hydrus/robots/quad/default_mode_201907/robot.urdf.xacro (robot description, xacro)
@@ -101,4 +101,5 @@
   </xacro:extra_module>
   <!-- end: gps -->
+  <xacro:property name="body_radius" value=".50" />
   <link name="dummy_body">
     <inertial>
@@ -113,5 +114,5 @@
       <origin rpy="0 0 0" xyz="0 0 0"/>
       <geometry>
-        <cylinder length="0.30" radius="0.50"/>
+        <cylinder length="0.30" radius="${body_radius}"/>
       </geometry>
     </visual>
@@ -119,5 +120,5 @@
         <origin rpy="0 0 0" xyz="0 0 0"/>
         <geometry>
-          <cylinder length="0.02" radius="0.50"/>
+          <cylinder length="0.02" radius="${body_radius}"/>
         </geometry>
     </collision>

Commit message: [visualize] change urdf file to show it is hydrus simulation

File: robots/hydrus/robots/quad/default_mode_201907/robot.urdf.xacro (robot description, xacro)
@@ -121,10 +121,10 @@
       <material name="Dummy_body_color"/>
     </visual>
-    <collision>
+    <!-- <collision>
         <origin rpy="0 0 0" xyz="0 0 0"/>
         <geometry>
           <cylinder length="0.02" radius="${body_radius}"/>
         </geometry>
-    </collision>
+    </collision> -->
   </link>
   <joint name="dummy_joint_1" type="fixed">
@@ -133,5 +133,5 @@
     <origin rpy="0 0 0" xyz="${link_length* 0.5} ${link_length* 0.5} 0.0"/>
   </joint>
-   <link name="dummy_body_visualize">
+   <!-- <link name="dummy_body_visualize">
     <inertial>
       <mass value = "0.0001" />
@@ -155,4 +155,4 @@
     <child link="dummy_body_visualize"/>
     <origin rpy="0 0 0" xyz="${link_length* 0.5} ${link_length* 0.5} 0.0"/>
-  </joint>
+  </joint> -->
 </robot>

File: robots/hydrus/urdf/common.xacro (robot description, xacro)
@@ -36,5 +36,5 @@
       </xacro:unless>
     </collision>
-    <!-- <visual>
+    <visual>
       <xacro:if value="${old_version == 1}">
         <origin rpy="0 0 0" xyz="${link_length* 0.5} 0 0"/>
@@ -59,5 +59,5 @@
         </geometry>
       </xacro:unless>
-    </visual> -->
+    </visual>
   </xacro:macro>
   <xacro:macro name="extra_module" params="name parent *origin *inertial visible:=0 model_url:=1 scale:=1">

File: robots/hydrus/urdf/link.urdf.xacro (robot description, xacro)
@@ -16,5 +16,5 @@
                 ixy="0.000021" ixz="0.000372" iyz="0.000000"/>
           </inertial>
-          <!-- <xacro:link_model type="head" /> -->
+          <xacro:link_model type="head" />
         </xacro:if>
         <xacro:unless value="${self == 1}">
@@ -28,5 +28,5 @@
                   ixy="0.000020" ixz="-0.000076" iyz="0.000000"/>
             </inertial>
-            <!-- <xacro:link_model type="end" /> -->
+            <xacro:link_model type="end" />
           </xacro:if>
           <xacro:unless value="${self == links}">
@@ -39,5 +39,5 @@
                   ixy="0.000021" ixz="0.000260" iyz="0.000000"/>
             </inertial>
-            <!-- <xacro:link_model type="general" /> -->
+            <xacro:link_model type="general" />
           </xacro:unless>
         </xacro:unless>
@@ -78,5 +78,5 @@
             </inertial>
           </xacro:unless>
-          <!-- <xacro:link_model type="1" /> -->
+          <xacro:link_model type="1" />
         </xacro:if>
         <xacro:unless value="${self == 1}">
@@ -112,5 +112,5 @@
               </inertial>
             </xacro:unless>
-            <!-- <xacro:link_model type="4" /> -->
+            <xacro:link_model type="4" />
           </xacro:if>
           <xacro:unless value="${self == links}">
@@ -146,5 +146,5 @@
                 </inertial>
               </xacro:unless>
-              <!-- <xacro:link_model type="2" /> -->
+              <xacro:link_model type="2" />
             </xacro:if>
             <!-- general -->
@@ -179,5 +179,5 @@
                 </inertial>
               </xacro:unless>
-              <!-- <xacro:link_model type="3" /> -->
+              <xacro:link_model type="3" />
             </xacro:unless>
           </xacro:unless>
@@ -214,10 +214,10 @@
             izz="0.00002"/>
       </inertial>
-      <!-- <collision>
+      <collision>
         <origin rpy="0 0 0" xyz="0 0 0"/>
         <geometry>
           <cylinder length="0.1" radius="${protector_radius + 0.01}"/>
         </geometry>
-      </collision> -->
+      </collision>
     </link>
     <xacro:damping_factor link ="thrust${self}"/>

Commit message: prep for merge with hydrus/gripper_model/spinal/uauav_graphene
checkout following file:
- aerial_robot_control/
- aerial_robot_estimation/
- aerial_robot aerial_robot_model/
- robots/
- aerial_robot_base/
- aerial_robot_simulation/
- aerial_robot_msgs/

File: robots/hydrus/robots/quad/default_mode_201907/robot.urdf.xacro (robot description, xacro)
@@ -65,5 +65,5 @@
   <!-- 2.  sensor -->
   <!-- 2.1 leddar one -->
-  <xacro:extra_module name = "leddarone" parent = "link3" visible = "1"
+  <xacro:extra_module name = "leddarone" parent = "link3" visible = "0"
                       model_url = "package://hydrus/urdf/mesh/sensor/leddar_one_tx2_attached_mode.dae">
     <origin xyz="${link_length/2 - 0.1855} 0.0 -0.0626" rpy="${pi} 0 0"/>
@@ -78,5 +78,5 @@
   <!-- end: leddar one -->
   <!-- 2.2 gps -->
-  <xacro:extra_module name = "gps" parent = "link2" visible = "1"
+  <xacro:extra_module name = "gps" parent = "link2" visible = "0"
                       model_url = "package://hydrus/urdf/mesh/sensor/gps_ublox_m8n.dae">
     <origin xyz="${link_length/2 + 0.1925} 0.0 0.152" rpy="0 0 0"/>
@@ -101,3 +101,58 @@
   </xacro:extra_module>
   <!-- end: gps -->
+  <xacro:property name="body_radius" value="0.50" />
+  <material name="Dummy_body_color">
+    <color rgba="1.0 1.0 1.0 0.5"/>
+  </material>
+  <link name="dummy_body">
+    <inertial>
+      <mass value = "0.0001" />
+      <origin xyz="0 0 0 " rpy="0 0 0"/>
+      <inertia
+          ixx="0.000001" ixy="0.0000" ixz="0.0000"
+          iyy="0.000001" iyz="0.00000"
+          izz="0.000001"/>
+    </inertial>
+    <visual>
+      <origin rpy="0 0 0" xyz="0 0 0"/>
+      <geometry>
+        <cylinder length="0.30" radius="${body_radius}"/>
+      </geometry>
+      <material name="Dummy_body_color"/>
+    </visual>
+    <!-- <collision>
+        <origin rpy="0 0 0" xyz="0 0 0"/>
+        <geometry>
+          <cylinder length="0.02" radius="${body_radius}"/>
+        </geometry>
+    </collision> -->
+  </link>
+  <joint name="dummy_joint_1" type="fixed">
+    <parent link="link1"/>
+    <child link="dummy_body"/>
+    <origin rpy="0 0 0" xyz="${link_length* 0.5} ${link_length* 0.5} 0.0"/>
+  </joint>
+   <!-- <link name="dummy_body_visualize">
+    <inertial>
+      <mass value = "0.0001" />
+      <origin xyz="0 0 0 " rpy="0 0 0"/>
+      <inertia
+          ixx="0.000001" ixy="0.0000" ixz="0.0000"
+          iyy="0.000001" iyz="0.00000"
+          izz="0.000001"/>
+    </inertial>
+    <visual>
+      <origin rpy="0 0 0" xyz="0 0 0"/>
+      <geometry>
+       <mesh
+        scale="2 2 2"
+        filename="package://agile_multirotor/urdf/mesh/quadrotor.stl" />
+      </geometry>
+    </visual>
+  </link>
+  <joint name="dummy_joint_2" type="fixed">
+    <parent link="link1"/>
+    <child link="dummy_body_visualize"/>
+    <origin rpy="0 0 0" xyz="${link_length* 0.5} ${link_length* 0.5} 0.0"/>
+  </joint> -->
 </robot>

File: robots/hydrus/urdf/common.xacro (robot description, xacro)
@@ -70,10 +70,10 @@
       <xacro:insert_block name="inertial" />
       <xacro:if value="${visible == 1}">
-        <visual>
+        <!-- <visual>
           <origin rpy="0 0 0" xyz="0 0 0"/>
           <geometry>
             <mesh filename="${model_url}" scale= "${scale} ${scale} ${scale}"/>
           </geometry>
-        </visual>
+        </visual> -->
       </xacro:if>
     </link>

File: robots/hydrus/urdf/link.urdf.xacro (robot description, xacro)
@@ -243,36 +243,36 @@
       <xacro:if value="${self == 1}">
         <xacro:if value="${old_version == 1}">
-          <xacro:standard_leg_old_version parent = "link${self}" >
+          <!-- <xacro:standard_leg_old_version parent = "link${self}" >
             <origin xyz="${head_leg_offset_old_version} 0.0 0" rpy="0 0 0"/>
-          </xacro:standard_leg_old_version>
+          </xacro:standard_leg_old_version> -->
         </xacro:if>
         <xacro:unless value="${old_version == 1}">
-          <xacro:standard_leg_end parent = "link${self}" >
+          <!-- <xacro:standard_leg_end parent = "link${self}" >
             <origin xyz="${head_leg_offset} 0.0 0" rpy="0 0 0"/>
-          </xacro:standard_leg_end>
+          </xacro:standard_leg_end> -->
         </xacro:unless>
       </xacro:if>
       <xacro:unless value="${self == 1}">
         <xacro:if value="${old_version == 1}">
-        <xacro:standard_leg_old_version parent = "link${self}" >
+        <!-- <xacro:standard_leg_old_version parent = "link${self}" >
           <origin xyz="${general_leg_offset_old_version} 0.0 0" rpy="0 0 0"/>
-        </xacro:standard_leg_old_version>
+        </xacro:standard_leg_old_version> -->
         </xacro:if>
         <xacro:unless value="${old_version == 1}">
-          <xacro:standard_leg_joint parent = "link${self}" >
+          <!-- <xacro:standard_leg_joint parent = "link${self}" >
             <origin xyz="0.0 0.0 0" rpy="0 0 0"/>
-          </xacro:standard_leg_joint>
+          </xacro:standard_leg_joint> -->
         </xacro:unless>
         <!-- tail -->
         <xacro:if value="${self == links}">
           <xacro:if value="${old_version == 1}">
-            <xacro:standard_leg_old_version parent = "link${self}" self= "${self + 1}" >
+            <!-- <xacro:standard_leg_old_version parent = "link${self}" self= "${self + 1}" >
               <origin xyz="${end_leg_offset_old_version} 0.0 0" rpy="0 0 0"/>
-            </xacro:standard_leg_old_version>
+            </xacro:standard_leg_old_version> -->
           </xacro:if>
           <xacro:unless value="${old_version == 1}">
-            <xacro:standard_leg_end parent = "link${self}" self= "${self + 1}" >
+            <!-- <xacro:standard_leg_end parent = "link${self}" self= "${self + 1}" >
               <origin xyz="${end_leg_offset} 0.0 0" rpy="0 0 0"/>
-            </xacro:standard_leg_end>
+            </xacro:standard_leg_end> -->
           </xacro:unless>
         </xacro:if>
