Commit message: update parameter in yaml and urdf file

File: robots/mini_quadrotor/urdf/infratable/robot.urdf.xacro (robot description, xacro)
@@ -6,7 +6,7 @@
   <thrust_link name="thrust" />
   <!-- kinematics [m] -->
-  <xacro:property name="rotor_x" value="0.070" />
-  <xacro:property name="rotor_y" value="0.086" />
-  <xacro:property name="rotor_z" value="0.026" />
+  <xacro:property name="rotor_x" value="0.090" />
+  <xacro:property name="rotor_y" value="0.090" />
+  <xacro:property name="rotor_z" value="0.055" />
   <!-- dynamics -->
   <m_f_rate value="-0.011" /> <!-- drag torque rate -->
@@ -96,5 +96,5 @@
   <link name="main_body">
     <inertial>
-      <mass value = "0.432" />
+      <mass value = "0.910" />
       <origin xyz="0 0 0.017" rpy="0 0 0"/>
       <inertia
@@ -139,7 +139,7 @@
   </xacro:extra_module>
   <!-- propellers -->
-  <xacro:propeller_module id = "1" x = "${-rotor_x}" y = "${-rotor_y}" z = "${rotor_z}" direction = "-1" />
-  <xacro:propeller_module id = "2" x = "${rotor_x}" y = "${-rotor_y}" z = "${rotor_z}" direction = "1" />
-  <xacro:propeller_module id = "3" x = "${rotor_x}" y = "${rotor_y}" z = "${rotor_z}" direction = "-1" />
-  <xacro:propeller_module id = "4" x = "${-rotor_x}" y = "${rotor_y}" z = "${rotor_z}"  direction = "1" />
+  <xacro:propeller_module id = "1" x = "${-rotor_x}" y = "${-rotor_y}" z = "${rotor_z}" direction = "1" />
+  <xacro:propeller_module id = "2" x = "${rotor_x}" y = "${-rotor_y}" z = "${rotor_z}" direction = "-1" />
+  <xacro:propeller_module id = "3" x = "${rotor_x}" y = "${rotor_y}" z = "${rotor_z}" direction = "1" />
+  <xacro:propeller_module id = "4" x = "${-rotor_x}" y = "${rotor_y}" z = "${rotor_z}"  direction = "-1" />
 </robot>

Commit message: change the param and gain

File: robots/mini_quadrotor/urdf/infratable/robot.urdf.xacro (robot description, xacro)
@@ -8,5 +8,6 @@
   <xacro:property name="rotor_x" value="0.090" />
   <xacro:property name="rotor_y" value="0.090" />
-  <xacro:property name="rotor_z" value="0.055" />
+  <xacro:property name="rotor_z" value="0.060" />
+  <!-- <xacro:property name="rotor_z" value="0.055" /> -->
   <!-- dynamics -->
   <m_f_rate value="-0.011" /> <!-- drag torque rate -->

Commit message: change the param of mass value

File: robots/mini_quadrotor/urdf/infratable/robot.urdf.xacro (robot description, xacro)
@@ -97,5 +97,5 @@
   <link name="main_body">
     <inertial>
-      <mass value = "0.910" />
+      <mass value = "1.45" />
       <origin xyz="0 0 0.017" rpy="0 0 0"/>
       <inertia

Commit message: change the rotor_z param

File: robots/mini_quadrotor/urdf/infratable/robot.urdf.xacro (robot description, xacro)
@@ -8,6 +8,7 @@
   <xacro:property name="rotor_x" value="0.090" />
   <xacro:property name="rotor_y" value="0.090" />
-  <xacro:property name="rotor_z" value="0.060" />
+  <!-- <xacro:property name="rotor_z" value="0.330" /> -->
   <!-- <xacro:property name="rotor_z" value="0.055" /> -->
+  <xacro:property name="rotor_z" value="0.180" />
   <!-- dynamics -->
   <m_f_rate value="-0.011" /> <!-- drag torque rate -->
