Commit message: [Beetle] refacotr beetle urdf using rotor arm macro.

File: robots/beetle/urdf/beetle.urdf.xacro (robot description, xacro)
@@ -59,69 +59,30 @@
       <axis xyz="0 0 1"/>
     </joint>
+    ## rotor arm macro
+    <xacro:macro name="dummy_rotor_arm" params="id x y z yaw">
+      ## link
+      <link name="rotor_arm${id}">
+        <inertial>
+          <origin xyz="0 0 0" rpy="0 0 0"/>
+          <mass value="0.0001"/>
+          <inertia
+              ixx="0.000001" ixy="0.0" ixz="0.0"
+              iyy="0.0001" iyz="0.0"
+              izz="0.0001"/>
+        </inertial>
+      </link>
+      ## joint
+      <joint name="base_arm_joint${id}" type="fixed">
+        <parent link="base_link"/>
+        <child link="rotor_arm${id}"/>
+        <origin rpy="0 0 ${yaw}" xyz="${x} ${y} ${z}"/>
+        <axis xyz="0 0 1"/>
+      </joint>
+    </xacro:macro>
     ## dummy rotor arms
-    <link name="rotor_arm${child1}">
-      <inertial>
-        <origin xyz="0 0 0" rpy="0 0 0"/>
-        <mass value="0.0001"/>
-        <inertia
-            ixx="0.000001" ixy="0.0" ixz="0.0"
-            iyy="0.0001" iyz="0.0"
-            izz="0.0001"/>
-      </inertial>
-    </link>
-    <joint name="base_arm_joint${child1}" type="fixed">
-      <parent link="base_link"/>
-      <child link="rotor_arm${child1}"/>
-      <origin rpy="0 0 ${pi/4}" xyz="0.12488 0.12509 0.1185"/>
-      <axis xyz="0 0 1"/>
-    </joint>
-    <link name="rotor_arm${child2}">
-      <inertial>
-        <origin xyz="0.0486 0 0.0161" rpy="0 0 0"/>
-        <mass value="0.0001"/>
-        <inertia
-            ixx="0.000001" ixy="0.0" ixz="0.0"
-            iyy="0.0001" iyz="0.0"
-            izz="0.0001"/>
-      </inertial>
-    </link>
-    <joint name="base_arm_joint${child2}" type="fixed">
-      <parent link="base_link"/>
-      <child link="rotor_arm${child2}"/>
-      <origin rpy="0 0 ${pi*3.0/4.0}" xyz="-0.12488 0.12509 0.1185"/>
-      <axis xyz="0 0 1"/>
-    </joint>
-    <link name="rotor_arm${child3}">
-      <inertial>
-        <origin xyz="0.0486 0 0.0161" rpy="0 0 0"/>
-        <mass value="0.0001"/>
-        <inertia
-            ixx="0.000001" ixy="0.0" ixz="0.0"
-            iyy="0.0001" iyz="0.0"
-            izz="0.0001"/>
-      </inertial>
-    </link>
-    <joint name="base_arm_joint${child3}" type="fixed">
-      <parent link="base_link"/>
-      <child link="rotor_arm${child3}"/>
-      <origin rpy="0 0 ${pi*5.0/4.0}" xyz="-0.12488 -0.12509 0.1185"/>
-      <axis xyz="0 0 1"/>
-    </joint>
-    <link name="rotor_arm${child4}">
-      <inertial>
-        <origin xyz="0.0486 0 0.0161" rpy="0 0 0"/>
-        <mass value="0.0001"/>
-        <inertia
-            ixx="0.000001" ixy="0.0" ixz="0.0"
-            iyy="0.0001" iyz="0.0"
-            izz="0.0001"/>
-      </inertial>
-    </link>
-    <joint name="base_arm_joint${child4}" type="fixed">
-      <parent link="base_link"/>
-      <child link="rotor_arm${child4}"/>
-      <origin rpy="0 0 ${-pi/4.0}" xyz="0.12488 -0.12509 0.1185"/>
-      <axis xyz="0 0 1"/>
-    </joint>
+    <xacro:dummy_rotor_arm id = "${child1}" x = "0.12488" y="0.12509" z = "0.1185" yaw = "${pi/4.0}"/>
+    <xacro:dummy_rotor_arm id = "${child2}" x = "-0.12488" y="0.12509" z = "0.1185" yaw = "${pi*3.0/4.0}"/>
+    <xacro:dummy_rotor_arm id = "${child3}" x = "-0.12488" y="-0.12509" z = "0.1185" yaw = "${pi*5.0/4.0}"/>
+    <xacro:dummy_rotor_arm id = "${child4}" x = "0.12488" y="-0.12509" z = "0.1185" yaw = "${-pi/4.0}"/>
     <xacro:friction self="base_link"/>
   </xacro:macro>

Commit message: [Beetle] add a variable frame on the contact point.

File: robots/beetle/urdf/beetle.urdf.xacro (robot description, xacro)
@@ -30,5 +30,5 @@
       </inertial>
       <visual>
-        <origin xyz="0 0 0" rpy="0 0 0"/>
+        <origin xyz="0 0 0" rpy="0 0 3.141592"/>
         <geometry>
           <mesh filename="package://beetle/urdf/mesh/base_link.dae"/>
@@ -85,4 +85,21 @@
     <xacro:dummy_rotor_arm id = "${child3}" x = "-0.12488" y="-0.12509" z = "0.1185" yaw = "${pi*5.0/4.0}"/>
     <xacro:dummy_rotor_arm id = "${child4}" x = "0.12488" y="-0.12509" z = "0.1185" yaw = "${-pi/4.0}"/>
+    ## dummy link for the contact point coordinate
+      <link name="contact_point">
+        <inertial>
+          <origin xyz="0 0 0" rpy="0 0 0"/>
+          <mass value="0.0001"/>
+          <inertia
+              ixx="0.000001" ixy="0.0" ixz="0.0"
+              iyy="0.0001" iyz="0.0"
+              izz="0.0001"/>
+        </inertial>
+      </link>
+      <joint name="cp_base_joint" type="fixed">
+        <parent link="base_link"/>
+        <child link="contact_point"/>
+        <origin rpy="0 0 0" xyz="0.26 0 0"/>
+        <axis xyz="0 0 1"/>
+      </joint>
     <xacro:friction self="base_link"/>
   </xacro:macro>

Commit message: [Beetle][test] modified urdf for test module

File: robots/beetle/urdf/beetle.urdf.xacro (robot description, xacro)
@@ -23,9 +23,9 @@
     <link name="base_link">
       <inertial>
-        <origin xyz="-0.0081803 0.0 0.1184962" rpy="0 0 0"/>
-        <mass value="1.82"/>
-        <inertia
-            ixx="0.0511797" iyy="0.0835848" izz="0.1010814"
-            ixy="-0.0000001" ixz="-0.0015934" iyz="0.0000027"/>
+        <origin xyz="0.0048861 0.0001638 0.1407979" rpy="0 0 0"/>
+        <mass value="2.24"/>
+        <inertia
+            ixx="0.0466335" iyy="0.0763754" izz="0.1025914"
+            ixy="-0.0000023" ixz="-0.0007664" iyz="-0.0000396"/>
       </inertial>
       <visual>
@@ -109,9 +109,9 @@
     <link name="gimbal_link${self}">
       <inertial>
-        <origin xyz="0.02284089 0.0 0.00720578" rpy="0 0 0"/>
-        <mass value="0.1333"/>
-        <inertia
-            ixx="0.00005310" iyy="0.00005269" izz="0.00005333"
-            ixy="-0.00000001" ixz="0.00000064" iyz="0.00000"/>
+        <origin xyz="0.02239457 0.0 0.00766902" rpy="0 0 0"/>
+        <mass value="0.15429"/>
+        <inertia
+            ixx="0.00006797" iyy="0.00006788" izz="0.00007058"
+            ixy="0.00000001" ixz="0.00000122" iyz="0.00000"/>
       </inertial>
       <collision>

Commit message: [Beetle][Test] modified robot's urdf for test version

File: robots/beetle/urdf/beetle.urdf.xacro (robot description, xacro)
@@ -23,8 +23,8 @@
     <link name="base_link">
       <inertial>
-        <origin xyz="0.0048861 0.0001638 0.1407979" rpy="0 0 0"/>
-        <mass value="2.24"/>
-        <inertia
-            ixx="0.0466335" iyy="0.0763754" izz="0.1025914"
+        <origin xyz="0.0050550 0.0002059 0.1416011" rpy="0 0 0"/>
+        <mass value="2.3422286"/>
+        <inertia
+            ixx="0.0445802" iyy="0.0743446" izz="0.0988890"
             ixy="-0.0000023" ixz="-0.0007664" iyz="-0.0000396"/>
       </inertial>
@@ -144,5 +144,5 @@
       <inertial>
         <origin xyz="0 0 0" rpy="0 0 0"/>
-        <mass value="0.00001"/>
+        <mass value="0.005"/>
         <inertia
             ixx="0.001" ixy="0.0" ixz="0.0"

Commit message: [Beetle] modified urdf as to value

File: robots/beetle/urdf/beetle.urdf.xacro (robot description, xacro)
@@ -23,9 +23,9 @@
     <link name="base_link">
       <inertial>
-        <origin xyz="0.0050550 0.0002059 0.1416011" rpy="0 0 0"/>
-        <mass value="2.3422286"/>
-        <inertia
-            ixx="0.0445802" iyy="0.0743446" izz="0.0988890"
-            ixy="-0.0000023" ixz="-0.0007664" iyz="-0.0000396"/>
+        <origin xyz="-0.0071465 -0.0009129 0.1378714" rpy="0 0 0"/>
+        <mass value="2.7463823"/>
+        <inertia
+            ixx="0.0524891" iyy="0.0892659" izz="0.1190375"
+            ixy="-0.0002672" ixz="-0.0008904" iyz="0.0000968"/>
       </inertial>
       <visual>
@@ -81,8 +81,8 @@
     </xacro:macro>
     ## dummy rotor arms
-    <xacro:dummy_rotor_arm id = "${child1}" x = "0.12488" y="0.12509" z = "0.1185" yaw = "${pi/4.0}"/>
-    <xacro:dummy_rotor_arm id = "${child2}" x = "-0.12488" y="0.12509" z = "0.1185" yaw = "${pi*3.0/4.0}"/>
-    <xacro:dummy_rotor_arm id = "${child3}" x = "-0.12488" y="-0.12509" z = "0.1185" yaw = "${pi*5.0/4.0}"/>
-    <xacro:dummy_rotor_arm id = "${child4}" x = "0.12488" y="-0.12509" z = "0.1185" yaw = "${-pi/4.0}"/>
+    <xacro:dummy_rotor_arm id = "${child1}" x = "0.12129" y="0.12150" z = "0.1185" yaw = "${pi/4.0}"/>
+    <xacro:dummy_rotor_arm id = "${child2}" x = "-0.12129" y="0.12150" z = "0.1185" yaw = "${pi*3.0/4.0}"/>
+    <xacro:dummy_rotor_arm id = "${child3}" x = "-0.12129" y="-0.12150" z = "0.1185" yaw = "${pi*5.0/4.0}"/>
+    <xacro:dummy_rotor_arm id = "${child4}" x = "0.12129" y="-0.12150" z = "0.1185" yaw = "${-pi/4.0}"/>
     ## dummy link for the contact point coordinate
       <link name="contact_point">
@@ -109,9 +109,9 @@
     <link name="gimbal_link${self}">
       <inertial>
-        <origin xyz="0.02239457 0.0 0.00766902" rpy="0 0 0"/>
-        <mass value="0.15429"/>
-        <inertia
-            ixx="0.00006797" iyy="0.00006788" izz="0.00007058"
-            ixy="0.00000001" ixz="0.00000122" iyz="0.00000"/>
+        <origin xyz="0.0223521 0.0 0.00776312" rpy="0 0 0"/>
+        <mass value="0.15944"/>
+        <inertia
+            ixx="0.00007458" iyy="0.00007325" izz="0.00007756"
+            ixy="0.00000001" ixz="0.00000084" iyz="0.00000001"/>
       </inertial>
       <collision>

Commit message: [Beetle][urdf] add battery model

File: robots/beetle/urdf/beetle.urdf.xacro (robot description, xacro)
@@ -23,9 +23,9 @@
     <link name="base_link">
       <inertial>
-        <origin xyz="-0.0071465 -0.0009129 0.1378714" rpy="0 0 0"/>
-        <mass value="2.7463823"/>
-        <inertia
-            ixx="0.0524891" iyy="0.0892659" izz="0.1190375"
-            ixy="-0.0002672" ixz="-0.0008904" iyz="0.0000968"/>
+        <origin xyz="-0.0071144 -0.0004661 0.1372857" rpy="0 0 0"/>
+        <mass value="2.7703823"/>
+        <inertia
+            ixx="0.0527268" iyy="0.0895178" izz="0.1192811"
+            ixy="-0.0001722" ixz="-0.0008599" iyz="0.0000395"/>
       </inertial>
       <visual>

Commit message: [Beetle][urdf] modified inertia info of base link.

File: robots/beetle/urdf/beetle.urdf.xacro (robot description, xacro)
@@ -23,9 +23,9 @@
     <link name="base_link">
       <inertial>
-        <origin xyz="-0.0071144 -0.0004661 0.1372857" rpy="0 0 0"/>
+        <origin xyz="0.0071144 0.0004661 0.1372857" rpy="0 0 0"/>
         <mass value="2.7703823"/>
         <inertia
             ixx="0.0527268" iyy="0.0895178" izz="0.1192811"
-            ixy="-0.0001722" ixz="-0.0008599" iyz="0.0000395"/>
+            ixy="-0.0001722" ixz="0.0008599" iyz="0.0000395"/>
       </inertial>
       <visual>
