Commit message: [beetle-art][URDF][Config]: update visual model; update IMU position; update rotor position

File: robots/beetle/urdf/beetle-art.urdf.xacro (robot description, xacro)
@@ -30,5 +30,5 @@
       </inertial>
       <visual>
-        <origin xyz="0 0 0" rpy="0 0 3.141592"/>
+        <origin xyz="0 0 0" rpy="0 0 0"/>
         <geometry>
           <mesh filename="package://beetle/urdf/mesh/base_link_beetle_art.dae"/>
@@ -56,5 +56,5 @@
       <child link="fc"/>
       <parent link="base_link"/>
-      <origin rpy="0 0 0" xyz="0 0 0.12947"/>
+      <origin rpy="0 0 0" xyz="-0.0175 -0.0015 0.12947"/>  # should be aligned with the position of IMU
       <axis xyz="0 0 1"/>
     </joint>
@@ -176,5 +176,5 @@
       <parent link="gimbal_link${self}"/>
       <child link="rotor_parent${self}"/>
-      <origin rpy="0 0 0" xyz="0.018 0.00 0.00438"/>
+      <origin rpy="0 0 0" xyz="0.02335 0.0 0.0"/>
       <axis xyz="0 0 ${rotor_direction}"/>
     </joint>
