Commit message: [beetle-art-omni][URDF] update /root, /base_link, /fc

File: robots/beetle/urdf/beetle-art-omni.urdf.xacro (robot description, xacro)
@@ -17,5 +17,5 @@
       <parent link="root"/>
       <child link="base_link"/>
-      <origin rpy="0 0 0" xyz="0 0 0"/>
+      <origin rpy="0 0 0" xyz="0 0 0.099"/>
       <axis xyz="0 0 1"/>
     </joint>
@@ -23,9 +23,9 @@
     <link name="base_link">
       <inertial>
-        <origin xyz="0.00001058 0.00029285 0.00900796" rpy="0 0 0"/>
-        <mass value="1.9328"/>
-        <inertia
-            ixx="0.01443196" iyy="0.01374647" izz="0.01963902"
-            ixy="-0.00000627" ixz="0.00009049" iyz="0.00006575"/>
+        <origin xyz="0.00001050 0.00029063 0.00895728" rpy="0 0 0"/>
+        <mass value="1.9614"/>
+        <inertia
+            ixx="0.01465916" iyy="0.01396881" izz="0.01999070"
+            ixy="-0.00000632" ixz="0.00009113" iyz="0.00006625"/>
       </inertial>
       <visual>
@@ -36,7 +36,7 @@
       </visual>
       <collision>
-        <origin xyz="0 0 0.1205" rpy="0 0 0"/>
-        <geometry>
-          <box size="0.52 0.52 0.241"/>
+        <origin xyz="0 0 0.0385" rpy="0 0 0"/>
+        <geometry>
+          <box size="0.35 0.35 0.275"/>
         </geometry>
       </collision>
@@ -56,5 +56,5 @@
       <child link="fc"/>
       <parent link="base_link"/>
-      <origin rpy="0 0 0" xyz="-0.0175 -0.0015 0.12947"/>  # should be aligned with the position of IMU
+      <origin rpy="0 0 0" xyz="-0.0175 -0.0015 0.06647"/>  # should be aligned with the position of IMU
       <axis xyz="0 0 1"/>
     </joint>

Commit message: [beetle-art-omni][URDF] update rotor arms and gimbal links.

File: robots/beetle/urdf/beetle-art-omni.urdf.xacro (robot description, xacro)
@@ -81,25 +81,25 @@
     </xacro:macro>
     ## dummy rotor arms
-    <xacro:dummy_rotor_arm id = "${child1}" x = "0.121218" y="0.121572" z = "0.1185" yaw = "${pi/4.0}"/>
-    <xacro:dummy_rotor_arm id = "${child2}" x = "-0.121218" y="0.121572" z = "0.1185" yaw = "${pi*3.0/4.0}"/>
-    <xacro:dummy_rotor_arm id = "${child3}" x = "-0.121218" y="-0.121572" z = "0.1185" yaw = "${pi*5.0/4.0}"/>
-    <xacro:dummy_rotor_arm id = "${child4}" x = "0.121218" y="-0.121572" z = "0.1185" yaw = "${-pi/4.0}"/>
+    <xacro:dummy_rotor_arm id = "${child1}" x = "0.17938" y="0.17938" z = "0.0171" yaw = "${pi*1.0/4.0}"/>
+    <xacro:dummy_rotor_arm id = "${child2}" x = "-0.17938" y="0.17938" z = "0.0171" yaw = "${pi*3.0/4.0}"/>
+    <xacro:dummy_rotor_arm id = "${child3}" x = "-0.17938" y="-0.17938" z = "0.0171" yaw = "${pi*5.0/4.0}"/>
+    <xacro:dummy_rotor_arm id = "${child4}" x = "0.17938" y="-0.17938" z = "0.0171" yaw = "${-pi*1.0/4.0}"/>
     ## dummy link for the contact point coordinate
-      <link name="contact_point">
-        <inertial>
-          <origin xyz="0 0 0" rpy="0 0 0"/>
-          <mass value="0.0001"/>
-          <inertia
-              ixx="0.000001" ixy="0.0" ixz="0.0"
-              iyy="0.0001" iyz="0.0"
-              izz="0.0001"/>
-        </inertial>
-      </link>
-      <joint name="cp_base_joint" type="fixed">
-        <parent link="base_link"/>
-        <child link="contact_point"/>
-        <origin rpy="0 0 0" xyz="0.26 0 0"/>
-        <axis xyz="0 0 1"/>
-      </joint>
+    <link name="contact_point">
+      <inertial>
+        <origin xyz="0 0 0" rpy="0 0 0"/>
+        <mass value="0.0001"/>
+        <inertia
+                ixx="0.000001" ixy="0.0" ixz="0.0"
+                iyy="0.0001" iyz="0.0"
+                izz="0.0001"/>
+      </inertial>
+    </link>
+    <joint name="cp_base_joint" type="fixed">
+      <parent link="base_link"/>
+      <child link="contact_point"/>
+      <origin rpy="0 0 0" xyz="0.26 0 0"/>
+      <axis xyz="0 0 1"/>
+    </joint>
     <xacro:friction self="base_link"/>
   </xacro:macro>
@@ -109,14 +109,14 @@
     <link name="gimbal_link${self}">
       <inertial>
-        <origin xyz="0.02239457 0.0 0.00766902" rpy="0 0 0"/>
-        <mass value="0.15429"/>
-        <inertia
-            ixx="0.00006797" iyy="0.00006788" izz="0.00007058"
-            ixy="0.00000001" ixz="0.00000122" iyz="0.00000"/>
+        <origin xyz="0.02085225 0.0 -0.01276312" rpy="0 0 0"/>
+        <mass value="0.15944"/>
+        <inertia
+            ixx="0.00007281" iyy="0.00007289" izz="0.00007635"
+            ixy="0.0" ixz="0.0" iyz="0.0"/>
       </inertial>
       <collision>
-        <origin xyz="0.0 0 0" rpy="0 0 0"/>
-        <geometry>
-          <cylinder radius="0.02" length="0.033"/>
+        <origin xyz="0.06 0 0" rpy="0 0 0"/>
+        <geometry>
+          <box size="0.11 0.11 0.05"/>
         </geometry>
       </collision>
@@ -155,5 +155,5 @@
     #### gimbal joints ####
     <joint name="gimbal${self}" type="revolute">
-      <limit effort="6.6" lower="-1.57" upper="1.57" velocity="3.0"/>
+      <limit effort="6.6" lower="-3.141593" upper="3.141593" velocity="3.0"/>
       <parent link="rotor_arm${self}"/>
       <child link="gimbal_link${self}"/>
@@ -162,5 +162,5 @@
       <dynamics damping="0.8" friction="0.0"/>
     </joint>
-    <transmission name="joint_tran${self}">1.570796
+    <transmission name="joint_tran${self}">3.141593
       <type>transmission_interface/SimpleTransmission</type>
       <joint name="gimbal${self}">
@@ -176,5 +176,5 @@
       <parent link="gimbal_link${self}"/>
       <child link="rotor_parent${self}"/>
-      <origin rpy="0 0 0" xyz="0.02335 0.0 0.0"/>
+      <origin rpy="0 0 0" xyz="0.02185 0.0 0.0"/>
       <axis xyz="0 0 ${rotor_direction}"/>
     </joint>

Commit message: [beetle-omni][URDF]: delete unused code

File: robots/beetle/urdf/beetle-art-omni.urdf.xacro (robot description, xacro)
@@ -85,21 +85,4 @@
     <xacro:dummy_rotor_arm id = "${child3}" x = "-0.17938" y="-0.17938" z = "0.0171" yaw = "${pi*5.0/4.0}"/>
     <xacro:dummy_rotor_arm id = "${child4}" x = "0.17938" y="-0.17938" z = "0.0171" yaw = "${-pi*1.0/4.0}"/>
-    ## dummy link for the contact point coordinate
-    <link name="contact_point">
-      <inertial>
-        <origin xyz="0 0 0" rpy="0 0 0"/>
-        <mass value="0.0001"/>
-        <inertia
-                ixx="0.000001" ixy="0.0" ixz="0.0"
-                iyy="0.0001" iyz="0.0"
-                izz="0.0001"/>
-      </inertial>
-    </link>
-    <joint name="cp_base_joint" type="fixed">
-      <parent link="base_link"/>
-      <child link="contact_point"/>
-      <origin rpy="0 0 0" xyz="0.26 0 0"/>
-      <axis xyz="0 0 1"/>
-    </joint>
     <xacro:friction self="base_link"/>
   </xacro:macro>

Commit message: [Beetle-Art-Omni-W-Guard]: update dae model; update URDF; update yaml file with Physical Params.

File: robots/beetle/urdf/beetle-art-omni.urdf.xacro (robot description, xacro)
@@ -23,14 +23,14 @@
     <link name="base_link">
       <inertial>
-        <origin xyz="0.00001050 0.00029063 0.00895728" rpy="0 0 0"/>
-        <mass value="1.9614"/>
+        <origin xyz="0.00000845 0.00023419 0.02260762" rpy="0 0 0"/>
+        <mass value="2.3096"/>
         <inertia
-            ixx="0.01465916" iyy="0.01396881" izz="0.01999070"
-            ixy="-0.00000632" ixz="0.00009113" iyz="0.00006625"/>
+            ixx="0.03155716" iyy="0.03084096" izz="0.03900553"
+            ixy="-0.00000599" ixz="0.00008620" iyz="0.00005548"/>
       </inertial>
       <visual>
         <origin xyz="0 0 0" rpy="0 0 0"/>
         <geometry>
-          <mesh filename="package://beetle/urdf/mesh/base_link_beetle_art_omni.dae"/>
+          <mesh filename="package://beetle/urdf/mesh/base_link_beetle_art_omni_w_guard.dae"/>
         </geometry>
       </visual>

File: robots/beetle/urdf/common.xacro (robot description, xacro)
@@ -5,5 +5,5 @@
   <baselink name="fc" />
   <thrust_link name="thrust" />
-  <m_f_rate value="-0.0172" /> <!-- drug torque rate -->
+  <m_f_rate value="-0.0165" /> <!-- drug torque rate -->
   <xacro:property name="max_force" value="30.0" /> <!-- [N] -->
   <xacro:property name="min_force" value="1.0" /> <!-- [N] -->

Commit message: [URDF][Beetle-Omni]: remove the axis parameter for fixed type joint

File: robots/beetle/urdf/beetle-art-omni.urdf.xacro (robot description, xacro)
@@ -57,5 +57,4 @@
       <parent link="base_link"/>
       <origin rpy="0 0 0" xyz="-0.0175 -0.0015 0.06647"/>  # should be aligned with the position of IMU
-      <axis xyz="0 0 1"/>
     </joint>
     ## rotor arm macro
@@ -77,5 +76,4 @@
         <child link="rotor_arm${id}"/>
         <origin rpy="0 0 ${yaw}" xyz="${x} ${y} ${z}"/>
-        <axis xyz="0 0 1"/>
       </joint>
     </xacro:macro>
@@ -160,5 +158,4 @@
       <child link="rotor_parent${self}"/>
       <origin rpy="0 0 0" xyz="0.02185 0.0 0.0"/>
-      <axis xyz="0 0 ${rotor_direction}"/>
     </joint>
     #### rotor joint (virtual) ####

Commit message: [URDF][Beetle-Omni]: change "base_link" to "main_body" to avoid misunderstanding. The name "baselink" (no underscore _) has been assigned to "fc" in common.xacro, which will be used in estimation.

File: robots/beetle/urdf/beetle-art-omni.urdf.xacro (robot description, xacro)
@@ -1,25 +1,9 @@
 <?xml version="1.0"?>
-<robot
-    xmlns:xacro="http://www.ros.org/wiki/xacro" name="beetle_link" >
+<robot xmlns:xacro="http://www.ros.org/wiki/xacro" name="beetle_link" >
   <xacro:macro name="beetle_center_link" params="child1 child2 child3 child4">
     ## dummy
-    <link name="root">
-      <inertial>
-        <origin xyz="0 0 0" rpy="0 0 0"/>
-        <mass value="0.00001"/>
-        <inertia
-            ixx="0.000001" ixy="0.0" ixz="0.0"
-            iyy="0.000001" iyz="0.0"
-            izz="0.000001"/>
-      </inertial>
-    </link>
-    <joint name="root_joint" type="fixed">
-      <parent link="root"/>
-      <child link="base_link"/>
-      <origin rpy="0 0 0" xyz="0 0 0.099"/>
-      <axis xyz="0 0 1"/>
-    </joint>
-    ## link
-    <link name="base_link">
+    <link name="root"/>
+    ## main body
+    <link name="main_body">
       <inertial>
         <origin xyz="0.00000845 0.00023419 0.02260762" rpy="0 0 0"/>
@@ -32,5 +16,5 @@
         <origin xyz="0 0 0" rpy="0 0 0"/>
         <geometry>
-          <mesh filename="package://beetle/urdf/mesh/base_link_beetle_art_omni_w_guard.dae"/>
+          <mesh filename="package://beetle/urdf/mesh/main_body_beetle_art_omni_w_guard.dae"/>
         </geometry>
       </visual>
@@ -42,5 +26,10 @@
       </collision>
     </link>
-    <xacro:damping_factor link="base_link"/>
+    <joint name="root_joint" type="fixed">
+      <parent link="root"/>
+      <child link="main_body"/>
+      <origin rpy="0 0 0" xyz="0 0 0"/>
+    </joint>
+    ## fc: flight controller. Note that "baselink" is assigned to "fc" in common.xacro by default
     <link name="fc">
       <inertial>
@@ -55,5 +44,5 @@
     <joint name="fc_joint" type="fixed">
       <child link="fc"/>
-      <parent link="base_link"/>
+      <parent link="main_body"/>
       <origin rpy="0 0 0" xyz="-0.0175 -0.0015 0.06647"/>  # should be aligned with the position of IMU
     </joint>
@@ -73,5 +62,5 @@
       ## joint
       <joint name="base_arm_joint${id}" type="fixed">
-        <parent link="base_link"/>
+        <parent link="main_body"/>
         <child link="rotor_arm${id}"/>
         <origin rpy="0 0 ${yaw}" xyz="${x} ${y} ${z}"/>
@@ -83,5 +72,5 @@
     <xacro:dummy_rotor_arm id = "${child3}" x = "-0.17938" y="-0.17938" z = "0.0171" yaw = "${pi*5.0/4.0}"/>
     <xacro:dummy_rotor_arm id = "${child4}" x = "0.17938" y="-0.17938" z = "0.0171" yaw = "${-pi*1.0/4.0}"/>
-    <xacro:friction self="base_link"/>
+    <xacro:friction self="main_body"/>
   </xacro:macro>
   <xacro:macro name="beetle_thrust_link" params="self rotor_direction">

File: robots/beetle/urdf/common.xacro (robot description, xacro)
@@ -1,9 +1,8 @@
 <?xml version="1.0"?>
-<robot
-    xmlns:xacro="http://www.ros.org/wiki/xacro" name="beetle_common" >
+<robot xmlns:xacro="http://www.ros.org/wiki/xacro" name="beetle_common" >
   <!-- general attribute -->
   <baselink name="fc" />
   <thrust_link name="thrust" />
-  <m_f_rate value="-0.0165" /> <!-- drug torque rate -->
+  <m_f_rate value="-0.0165" /> <!-- drag torque rate -->
   <xacro:property name="max_force" value="30.0" /> <!-- [N] -->
   <xacro:property name="min_force" value="1.0" /> <!-- [N] -->
