Commit message: [delta] update urdfs for 10inch prop model

File: robots/delta/robots/20240117_10inch/rolling.gazebo.xacro (robot description, xacro)
@@ -3,5 +3,5 @@
     xmlns:xacro="http://www.ros.org/wiki/xacro" name="delta" >
   <xacro:arg name="robot_name" default="delta" />
-  <xacro:include filename="$(find delta)/robots/20231013_frame/rolling.urdf.xacro" />
+  <xacro:include filename="$(find delta)/robots/20240117_10inch/rolling.urdf.xacro" />
   <!-- gazebo plugin for default controller and sensors -->
   <xacro:include filename="$(find aerial_robot_simulation)/xacro/spinal.gazebo.xacro" />

File: robots/delta/robots/20240117_10inch/rolling.urdf.xacro (robot description, xacro)
@@ -2,8 +2,8 @@
 <robot
     xmlns:xacro="http://www.ros.org/wiki/xacro" name="delta" >
-  <xacro:include filename="$(find delta)/urdf/20231013_frame/rolling_link.urdf.xacro" />
+  <xacro:include filename="$(find delta)/urdf/20240117_10inch/rolling_link.urdf.xacro" />
   <xacro:include filename="$(find delta)/urdf/common.xacro" />
-  <xacro:delta_module self="1" child="2" rotor_direction="1"  battery="false"/>
-  <xacro:delta_module self="2" child="3" rotor_direction="-1" battery="false"/>
-  <xacro:delta_module self="3" child="3" rotor_direction="1"  battery="false"/>
+  <xacro:delta_module self="1" child="2" rotor_direction="1"  battery="true"/>
+  <xacro:delta_module self="2" child="3" rotor_direction="-1" battery="true"/>
+  <xacro:delta_module self="3" child="3" rotor_direction="1"  battery="true"/>
 </robot>

File: robots/delta/urdf/20240117_10inch/battery.urdf.xacro (robot description, xacro)
@@ -13,5 +13,5 @@
       <visual>
         <geometry>
-          <mesh filename="package://delta/urdf/mesh/20231013_frame/battery_module.dae" />
+          <mesh filename="package://delta/urdf/mesh/20240117_10inch/battery_module.dae" />
         </geometry>
       </visual>

File: robots/delta/urdf/20240117_10inch/link1.urdf.xacro (robot description, xacro)
@@ -13,5 +13,5 @@
       <visual>
         <geometry>
-          <mesh filename="package://delta/urdf/mesh/20231013_frame/link1_base.dae" />
+          <mesh filename="package://delta/urdf/mesh/20240117_10inch/link1_base.dae" />
         </geometry>
       </visual>
@@ -33,5 +33,5 @@
       <visual>
         <geometry>
-          <mesh filename="package://delta/urdf/mesh/20231013_frame/link1_gimbal.dae" />
+          <mesh filename="package://delta/urdf/mesh/20240117_10inch/link1_gimbal.dae" />
         </geometry>
       </visual>

File: robots/delta/urdf/20240117_10inch/link2.urdf.xacro (robot description, xacro)
@@ -13,5 +13,5 @@
       <visual>
         <geometry>
-          <mesh filename="package://delta/urdf/mesh/20231013_frame/link2_base.dae" />
+          <mesh filename="package://delta/urdf/mesh/20240117_10inch/link2_base.dae" />
         </geometry>
       </visual>
@@ -33,5 +33,5 @@
       <visual>
         <geometry>
-          <mesh filename="package://delta/urdf/mesh/20231013_frame/link2_gimbal.dae" />
+          <mesh filename="package://delta/urdf/mesh/20240117_10inch/link2_gimbal.dae" />
         </geometry>
       </visual>

File: robots/delta/urdf/20240117_10inch/link3.urdf.xacro (robot description, xacro)
@@ -13,5 +13,5 @@
       <visual>
         <geometry>
-          <mesh filename="package://delta/urdf/mesh/20231013_frame/link3_base.dae" />
+          <mesh filename="package://delta/urdf/mesh/20240117_10inch/link3_base.dae" />
         </geometry>
       </visual>
@@ -33,5 +33,5 @@
       <visual>
         <geometry>
-          <mesh filename="package://delta/urdf/mesh/20231013_frame/link3_gimbal.dae" />
+          <mesh filename="package://delta/urdf/mesh/20240117_10inch/link3_gimbal.dae" />
         </geometry>
       </visual>

File: robots/delta/urdf/20240117_10inch/rolling_link.urdf.xacro (robot description, xacro)
@@ -2,8 +2,8 @@
 <robot
     xmlns:xacro="http://www.ros.org/wiki/xacro" name="delta_link" >
-  <xacro:include filename="$(find delta)/urdf/20231013_frame/link1.urdf.xacro" />
-  <xacro:include filename="$(find delta)/urdf/20231013_frame/link2.urdf.xacro" />
-  <xacro:include filename="$(find delta)/urdf/20231013_frame/link3.urdf.xacro" />
-  <xacro:include filename="$(find delta)/urdf/20231013_frame/battery.urdf.xacro" />
+  <xacro:include filename="$(find delta)/urdf/20240117_10inch/link1.urdf.xacro" />
+  <xacro:include filename="$(find delta)/urdf/20240117_10inch/link2.urdf.xacro" />
+  <xacro:include filename="$(find delta)/urdf/20240117_10inch/link3.urdf.xacro" />
+  <xacro:include filename="$(find delta)/urdf/20240117_10inch/battery.urdf.xacro" />
   <xacro:macro name="delta_module" params="self child rotor_direction battery">
     <!-- dummy root link for KDL -->
