Commit message: [delta] add new battery type and separate thrust information in urdf for different type of prop

File: robots/delta/robots/20240117_10inch/rolling.urdf.xacro (robot description, xacro)
@@ -4,6 +4,9 @@
   <xacro:include filename="$(find delta)/urdf/20240117_10inch/rolling_link.urdf.xacro" />
   <xacro:include filename="$(find delta)/urdf/common.xacro" />
-  <xacro:delta_module self="1" child="2" rotor_direction="1"  battery="true"/>
-  <xacro:delta_module self="2" child="3" rotor_direction="-1" battery="true"/>
-  <xacro:delta_module self="3" child="3" rotor_direction="1"  battery="true"/>
+  <!-- battery: 1 = 6S ZIPPY 3000 (blue)              -->
+  <!-- battery: 2 = 6S Turningy high lipo (silver) x1 -->
+  <!-- battery: 3 = 6S Turningy high lipo (silver) x2 -->
+  <xacro:delta_module self="1" child="2" rotor_direction="1"  battery="2"/>
+  <xacro:delta_module self="2" child="3" rotor_direction="-1" battery="2"/>
+  <xacro:delta_module self="3" child="3" rotor_direction="1"  battery="2"/>
 </robot>

File: robots/delta/urdf/20231013_frame/rolling_link.urdf.xacro (robot description, xacro)
@@ -6,4 +6,5 @@
   <xacro:include filename="$(find delta)/urdf/20231013_frame/link3.urdf.xacro" />
   <xacro:include filename="$(find delta)/urdf/20231013_frame/battery.urdf.xacro" />
+  <xacro:include filename="$(find delta)/urdf/20231013_frame/thrust.urdf.xacro" />
   <xacro:macro name="delta_module" params="self child rotor_direction battery">
     <!-- dummy root link for KDL -->

File: robots/delta/urdf/20240117_10inch/battery.urdf.xacro (robot description, xacro)
@@ -2,4 +2,5 @@
 <robot
     xmlns:xacro="http://www.ros.org/wiki/xacro" name="battery" >
+  <!-- 6S ZIPPY 3000 6S (blue) -->
   <xacro:macro name="battery" params="index">
     <link name="battery${index}">
@@ -18,3 +19,37 @@
     </link>
   </xacro:macro>
+  <!-- 6S Turningy high lipo 1300 (silver) x1 -->
+  <xacro:macro name="high_lipo_single" params="index">
+    <link name="high_lipo_single${index}">
+      <inertial>
+        <origin xyz="0.04390043 -0.02150000 0.00000000" rpy="0 0 0"/>
+        <mass value="0.22649093"/>
+        <inertia
+            ixx="0.00005005"  iyy="0.00017334"  izz="0.00016934"
+            ixy="-0.00000034" ixz="0.00000000"  iyz="0.00000000"/>
+      </inertial>
+      <visual>
+        <geometry>
+          <mesh filename="package://delta/urdf/mesh/20240117_10inch/high_lipo_single_module.STL" />
+        </geometry>
+      </visual>
+    </link>
+  </xacro:macro>
+  <!-- 6S Turningy high lipo 1300 (silver) x2 -->
+  <xacro:macro name="high_lipo_double" params="index">
+    <link name="high_lipo_double${index}">
+      <inertial>
+        <origin xyz="0.4390043 0.00000000 0.00000000" rpy="0 0 0"/>
+        <mass value="0.45298185"/>
+        <inertia
+            ixx="0.00044266" iyy="0.00068125"  izz="0.00034667"
+            ixy="0.00000000" ixz="0.00000000" iyz="-0.00000000"/>
+      </inertial>
+      <visual>
+        <geometry>
+          <mesh filename="package://delta/urdf/mesh/20240117_10inch/high_lipo_double_module.STL" />
+        </geometry>
+      </visual>
+    </link>
+  </xacro:macro>
 </robot>

File: robots/delta/urdf/20240117_10inch/rolling_link.urdf.xacro (robot description, xacro)
@@ -6,4 +6,5 @@
   <xacro:include filename="$(find delta)/urdf/20240117_10inch/link3.urdf.xacro" />
   <xacro:include filename="$(find delta)/urdf/20240117_10inch/battery.urdf.xacro" />
+  <xacro:include filename="$(find delta)/urdf/20240117_10inch/thrust.urdf.xacro" />
   <xacro:macro name="delta_module" params="self child rotor_direction battery">
     <!-- dummy root link for KDL -->
@@ -88,5 +89,5 @@
     </xacro:unless>
     <!-- battery -->
-    <xacro:if value="${battery}">
+    <xacro:if value="${battery == 1}">
       <xacro:battery index="${self}"/>
       <joint name="battery_joint${self}" type="fixed">
@@ -101,4 +102,36 @@
         <xacro:if value="${self == 3}">
           <origin xyz="0.3535 0 0"/>
+        </xacro:if>
+      </joint>
+    </xacro:if>
+    <xacro:if value="${battery == 2}">
+      <xacro:high_lipo_single index="${self}"/>
+      <joint name="battery_joint${self}" type="fixed">
+        <parent link="link${self}"/>
+        <child link="high_lipo_single${self}"/>
+        <xacro:if value="${self == 1}">
+          <origin xyz="0.28 0 0"/>
+        </xacro:if>
+        <xacro:if value="${self == 2}">
+          <origin xyz="0.3135 0 0"/>
+        </xacro:if>
+        <xacro:if value="${self == 3}">
+          <origin xyz="0.3135 0 0"/>
+        </xacro:if>
+      </joint>
+    </xacro:if>
+    <xacro:if value="${battery == 3}">
+      <xacro:high_lipo_double index="${self}"/>
+      <joint name="battery_joint${self}" type="fixed">
+        <parent link="link${self}"/>
+        <child link="high_lipo_double${self}"/>
+        <xacro:if value="${self == 1}">
+          <origin xyz="0.310 0 0"/>
+        </xacro:if>
+        <xacro:if value="${self == 2}">
+          <origin xyz="0.3435 0 0"/>
+        </xacro:if>
+        <xacro:if value="${self == 3}">
+          <origin xyz="0.3435 0 0"/>
         </xacro:if>
       </joint>

File: robots/delta/urdf/common.xacro (robot description, xacro)
@@ -5,7 +5,4 @@
   <baselink name="fc" />
   <thrust_link name="thrust" />
-  <m_f_rate value="-0.0142" /> <!-- drug torque rate -->
-  <xacro:property name="max_force" value="22.0" /> <!-- [N] -->
-  <xacro:property name="min_force" value="0.0" /> <!-- [N] -->
   <!-- friction -->
   <xacro:macro name="friction" params="link">

Commit message: [delta][urdf] add new battery type: high lipo single under side of the link

File: robots/delta/robots/20240117_10inch/rolling.urdf.xacro (robot description, xacro)
@@ -7,6 +7,6 @@
   <!-- battery: 2 = 6S Turningy high lipo (silver) x1 -->
   <!-- battery: 3 = 6S Turningy high lipo (silver) x2 -->
-  <xacro:delta_module self="1" child="2" rotor_direction="1"  battery="2"/>
-  <xacro:delta_module self="2" child="3" rotor_direction="-1" battery="2"/>
-  <xacro:delta_module self="3" child="3" rotor_direction="1"  battery="2"/>
+  <xacro:delta_module self="1" child="2" rotor_direction="1"  battery="4"/>
+  <xacro:delta_module self="2" child="3" rotor_direction="-1" battery="4"/>
+  <xacro:delta_module self="3" child="3" rotor_direction="1"  battery="4"/>
 </robot>

File: robots/delta/urdf/20240117_10inch/battery.urdf.xacro (robot description, xacro)
@@ -19,5 +19,5 @@
     </link>
   </xacro:macro>
-  <!-- 6S Turningy high lipo 1300 (silver) x1 -->
+  <!-- 6S Turningy high lipo 1300 (silver) x1 outer side of the link-->
   <xacro:macro name="high_lipo_single" params="index">
     <link name="high_lipo_single${index}">
@@ -53,3 +53,20 @@
     </link>
   </xacro:macro>
+  <!-- 6S Turningy high lipo 1300 (silver) x1 under side of the link -->
+  <xacro:macro name="high_lipo_single_under" params="index">
+    <link name="high_lipo_single${index}">
+      <inertial>
+        <origin xyz="0.4390043 0.00000000 -0.02750000" rpy="0 0 0"/>
+        <mass value="0.22649093"/>
+        <inertia
+            ixx="0.00005005"  iyy="0.00016934"  izz="0.00017334"
+            ixy="0.00000000" ixz="-0.00000034" iyz="-0.00000000"/>
+      </inertial>
+      <visual>
+        <geometry>
+          <mesh filename="package://delta/urdf/mesh/20240117_10inch/high_lipo_single_module_under.STL" />
+        </geometry>
+      </visual>
+    </link>
+  </xacro:macro>
 </robot>

File: robots/delta/urdf/20240117_10inch/rolling_link.urdf.xacro (robot description, xacro)
@@ -126,4 +126,20 @@
         <parent link="link${self}"/>
         <child link="high_lipo_double${self}"/>
+        <xacro:if value="${self == 1}">
+          <origin xyz="0.310 0 0"/>
+        </xacro:if>
+        <xacro:if value="${self == 2}">
+          <origin xyz="0.3435 0 0"/>
+        </xacro:if>
+        <xacro:if value="${self == 3}">
+          <origin xyz="0.3435 0 0"/>
+        </xacro:if>
+      </joint>
+    </xacro:if>
+    <xacro:if value="${battery == 4}">
+      <xacro:high_lipo_single_under index="${self}"/>
+      <joint name="battery_joint${self}" type="fixed">
+        <parent link="link${self}"/>
+        <child link="high_lipo_single${self}"/>
         <xacro:if value="${self == 1}">
           <origin xyz="0.310 0 0"/>

Commit message: [delta][urdf] update battery models

File: robots/delta/robots/20240117_10inch/rolling.urdf.xacro (robot description, xacro)
@@ -5,6 +5,8 @@
   <xacro:include filename="$(find delta)/urdf/common.xacro" />
   <!-- battery: 1 = 6S ZIPPY 3000 (blue)              -->
-  <!-- battery: 2 = 6S Turningy high lipo (silver) x1 -->
-  <!-- battery: 3 = 6S Turningy high lipo (silver) x2 -->
+  <!-- battery: 2 = 6S Turningy high lipo (silver) x1 inner side -->
+  <!-- battery: 3 = 6S Turningy high lipo (silver) x1 outer side -->
+  <!-- battery: 4 = 6S Turningy high lipo (silver) x1 under side -->
+  <!-- battery: 5 = 6S Turningy high lipo (silver) x2 -->
   <xacro:delta_module self="1" child="2" rotor_direction="1"  battery="4"/>
   <xacro:delta_module self="2" child="3" rotor_direction="-1" battery="4"/>

File: robots/delta/urdf/20240117_10inch/battery.urdf.xacro (robot description, xacro)
@@ -19,9 +19,26 @@
     </link>
   </xacro:macro>
-  <!-- 6S Turningy high lipo 1300 (silver) x1 outer side of the link-->
-  <xacro:macro name="high_lipo_single" params="index">
+  <!-- 6S Turningy high lipo 1300 (silver) x1 inner side of the link -->
+  <xacro:macro name="high_lipo_single_inner" params="index">
     <link name="high_lipo_single${index}">
       <inertial>
-        <origin xyz="0.04390043 -0.02150000 0.00000000" rpy="0 0 0"/>
+        <origin xyz="0.04390043 0.02750000 0.00000000 " rpy="0 0 0"/>
+        <mass value="0.22649093"/>
+        <inertia
+            ixx="0.00005005" iyy="0.00017334"  izz="0.00016934"
+            ixy="0.00000034" ixz="0.00000000" iyz="-0.00000000"/>
+      </inertial>
+      <visual>
+        <geometry>
+          <mesh filename="package://delta/urdf/mesh/20240117_10inch/high_lipo_single_module_inner.stl" />
+        </geometry>
+      </visual>
+    </link>
+  </xacro:macro>
+  <!-- 6S Turningy high lipo 1300 (silver) x1 outer side of the link-->
+  <xacro:macro name="high_lipo_single_outer" params="index">
+    <link name="high_lipo_single${index}">
+      <inertial>
+        <origin xyz="0.04490043 -0.02150000 0.00000000" rpy="0 0 0"/>
         <mass value="0.22649093"/>
         <inertia
@@ -31,5 +48,22 @@
       <visual>
         <geometry>
-          <mesh filename="package://delta/urdf/mesh/20240117_10inch/high_lipo_single_module.stl" />
+          <mesh filename="package://delta/urdf/mesh/20240117_10inch/high_lipo_single_module_outer.stl" />
+        </geometry>
+      </visual>
+    </link>
+  </xacro:macro>
+  <!-- 6S Turningy high lipo 1300 (silver) x1 under side of the link -->
+  <xacro:macro name="high_lipo_single_under" params="index">
+    <link name="high_lipo_single${index}">
+      <inertial>
+        <origin xyz="0.04390043 0.00000000 -0.02750000" rpy="0 0 0"/>
+        <mass value="0.22649093"/>
+        <inertia
+            ixx="0.00005005"  iyy="0.00016934"  izz="0.00017334"
+            ixy="0.00000000" ixz="-0.00000034" iyz="-0.00000000"/>
+      </inertial>
+      <visual>
+        <geometry>
+          <mesh filename="package://delta/urdf/mesh/20240117_10inch/high_lipo_single_module_under.stl" />
         </geometry>
       </visual>
@@ -53,20 +87,3 @@
     </link>
   </xacro:macro>
-  <!-- 6S Turningy high lipo 1300 (silver) x1 under side of the link -->
-  <xacro:macro name="high_lipo_single_under" params="index">
-    <link name="high_lipo_single${index}">
-      <inertial>
-        <origin xyz="0.04390043 0.00000000 -0.02750000" rpy="0 0 0"/>
-        <mass value="0.22649093"/>
-        <inertia
-            ixx="0.00005005"  iyy="0.00016934"  izz="0.00017334"
-            ixy="0.00000000" ixz="-0.00000034" iyz="-0.00000000"/>
-      </inertial>
-      <visual>
-        <geometry>
-          <mesh filename="package://delta/urdf/mesh/20240117_10inch/high_lipo_single_module_under.STL" />
-        </geometry>
-      </visual>
-    </link>
-  </xacro:macro>
 </robot>

File: robots/delta/urdf/20240117_10inch/rolling_link.urdf.xacro (robot description, xacro)
@@ -89,4 +89,9 @@
     </xacro:unless>
     <!-- battery -->
+    <!-- battery: 1 = 6S ZIPPY 3000 (blue)              -->
+    <!-- battery: 2 = 6S Turningy high lipo (silver) x1 inner side -->
+    <!-- battery: 3 = 6S Turningy high lipo (silver) x1 outer side -->
+    <!-- battery: 4 = 6S Turningy high lipo (silver) x1 under side -->
+    <!-- battery: 5 = 6S Turningy high lipo (silver) x2 -->
     <xacro:if value="${battery == 1}">
       <xacro:battery index="${self}"/>
@@ -106,9 +111,25 @@
     </xacro:if>
     <xacro:if value="${battery == 2}">
-      <xacro:high_lipo_single index="${self}"/>
+      <xacro:high_lipo_single_inner index="${self}"/>
       <joint name="battery_joint${self}" type="fixed">
         <parent link="link${self}"/>
         <child link="high_lipo_single${self}"/>
         <xacro:if value="${self == 1}">
+          <origin xyz="0.32 0 0"/>
+        </xacro:if>
+        <xacro:if value="${self == 2}">
+          <origin xyz="0.3535 0 0"/>
+        </xacro:if>
+        <xacro:if value="${self == 3}">
+          <origin xyz="0.3535 0 0"/>
+        </xacro:if>
+      </joint>
+    </xacro:if>
+    <xacro:if value="${battery == 3}">
+      <xacro:high_lipo_single_outer index="${self}"/>
+      <joint name="battery_joint${self}" type="fixed">
+        <parent link="link${self}"/>
+        <child link="high_lipo_single${self}"/>
+        <xacro:if value="${self == 1}">
           <origin xyz="0.28 0 0"/>
         </xacro:if>
@@ -118,20 +139,4 @@
         <xacro:if value="${self == 3}">
           <origin xyz="0.3135 0 0"/>
-        </xacro:if>
-      </joint>
-    </xacro:if>
-    <xacro:if value="${battery == 3}">
-      <xacro:high_lipo_double index="${self}"/>
-      <joint name="battery_joint${self}" type="fixed">
-        <parent link="link${self}"/>
-        <child link="high_lipo_double${self}"/>
-        <xacro:if value="${self == 1}">
-          <origin xyz="0.310 0 0"/>
-        </xacro:if>
-        <xacro:if value="${self == 2}">
-          <origin xyz="0.3435 0 0"/>
-        </xacro:if>
-        <xacro:if value="${self == 3}">
-          <origin xyz="0.3435 0 0"/>
         </xacro:if>
       </joint>
@@ -142,4 +147,20 @@
         <parent link="link${self}"/>
         <child link="high_lipo_single${self}"/>
+        <xacro:if value="${self == 1}">
+          <origin xyz="0.310 0 0"/>
+        </xacro:if>
+        <xacro:if value="${self == 2}">
+          <origin xyz="0.3435 0 0"/>
+        </xacro:if>
+        <xacro:if value="${self == 3}">
+          <origin xyz="0.3435 0 0"/>
+        </xacro:if>
+      </joint>
+    </xacro:if>
+    <xacro:if value="${battery == 5}">
+      <xacro:high_lipo_double index="${self}"/>
+      <joint name="battery_joint${self}" type="fixed">
+        <parent link="link${self}"/>
+        <child link="high_lipo_double${self}"/>
         <xacro:if value="${self == 1}">
           <origin xyz="0.310 0 0"/>
