Commit message: [delta][urdf] update battery model

File: robots/delta/robots/20240117_10inch/rolling.urdf.xacro (robot description, xacro)
@@ -4,11 +4,7 @@
   <xacro:include filename="$(find delta)/urdf/20240117_10inch/rolling_link.urdf.xacro" />
   <xacro:include filename="$(find delta)/urdf/common.xacro" />
-  <!-- battery: 1 = 6S ZIPPY 3000 (blue)              -->
-  <!-- battery: 2 = 6S Turningy high lipo (silver) x1 inner side -->
-  <!-- battery: 3 = 6S Turningy high lipo (silver) x1 outer side -->
-  <!-- battery: 4 = 6S Turningy high lipo (silver) x1 under side -->
-  <!-- battery: 5 = 6S Turningy high lipo (silver) x2 -->
-  <xacro:delta_module self="1" child="2" rotor_direction="1"  battery="4"/>
-  <xacro:delta_module self="2" child="3" rotor_direction="-1" battery="4"/>
-  <xacro:delta_module self="3" child="3" rotor_direction="1"  battery="4"/>
+  <!-- battery: 1 = 6S Turningy high lipo (silver) x1 -->
+  <xacro:delta_module self="1" child="2" rotor_direction="1"  battery="1"/>
+  <xacro:delta_module self="2" child="3" rotor_direction="-1" battery="1"/>
+  <xacro:delta_module self="3" child="3" rotor_direction="1"  battery="1"/>
 </robot>

File: robots/delta/urdf/20240117_10inch/battery.urdf.xacro (robot description, xacro)
@@ -19,68 +19,17 @@
     </link>
   </xacro:macro>
-  <!-- 6S Turningy high lipo 1300 (silver) x1 inner side of the link -->
-  <xacro:macro name="high_lipo_single_inner" params="index">
+  <!-- 6S Turningy high lipo 1300 (silver) x1 -->
+  <xacro:macro name="high_lipo_single" params="index">
     <link name="high_lipo_single${index}">
       <inertial>
-        <origin xyz="0.04390043 0.02750000 0.00000000 " rpy="0 0 0"/>
+        <origin xyz="0.04390043 0.00000000 0.01150000 " rpy="0 0 0"/>
         <mass value="0.22649093"/>
         <inertia
-            ixx="0.00005005" iyy="0.00017334"  izz="0.00016934"
-            ixy="0.00000034" ixz="0.00000000" iyz="-0.00000000"/>
+            ixx="0.00005005" iyy="0.00016934"  izz="0.00017334"
+            ixy="0.00000000" ixz="0.00000034" iyz="-0.00000000"/>
       </inertial>
       <visual>
         <geometry>
-          <mesh filename="package://delta/urdf/mesh/20240117_10inch/high_lipo_single_module_inner.stl" />
-        </geometry>
-      </visual>
-    </link>
-  </xacro:macro>
-  <!-- 6S Turningy high lipo 1300 (silver) x1 outer side of the link-->
-  <xacro:macro name="high_lipo_single_outer" params="index">
-    <link name="high_lipo_single${index}">
-      <inertial>
-        <origin xyz="0.04490043 -0.02150000 0.00000000" rpy="0 0 0"/>
-        <mass value="0.22649093"/>
-        <inertia
-            ixx="0.00005005"  iyy="0.00017334"  izz="0.00016934"
-            ixy="-0.00000034" ixz="0.00000000"  iyz="0.00000000"/>
-      </inertial>
-      <visual>
-        <geometry>
-          <mesh filename="package://delta/urdf/mesh/20240117_10inch/high_lipo_single_module_outer.stl" />
-        </geometry>
-      </visual>
-    </link>
-  </xacro:macro>
-  <!-- 6S Turningy high lipo 1300 (silver) x1 under side of the link -->
-  <xacro:macro name="high_lipo_single_under" params="index">
-    <link name="high_lipo_single${index}">
-      <inertial>
-        <origin xyz="0.04390043 0.00000000 -0.02750000" rpy="0 0 0"/>
-        <mass value="0.22649093"/>
-        <inertia
-            ixx="0.00005005"  iyy="0.00016934"  izz="0.00017334"
-            ixy="0.00000000" ixz="-0.00000034" iyz="-0.00000000"/>
-      </inertial>
-      <visual>
-        <geometry>
-          <mesh filename="package://delta/urdf/mesh/20240117_10inch/high_lipo_single_module_under.stl" />
-        </geometry>
-      </visual>
-    </link>
-  </xacro:macro>
-  <!-- 6S Turningy high lipo 1300 (silver) x2 -->
-  <xacro:macro name="high_lipo_double" params="index">
-    <link name="high_lipo_double${index}">
-      <inertial>
-        <origin xyz="0.04390043 0.00000000 0.00000000" rpy="0 0 0"/>
-        <mass value="0.45298185"/>
-        <inertia
-            ixx="0.00044266" iyy="0.00068125"  izz="0.00034667"
-            ixy="0.00000000" ixz="0.00000000" iyz="-0.00000000"/>
-      </inertial>
-      <visual>
-        <geometry>
-          <mesh filename="package://delta/urdf/mesh/20240117_10inch/high_lipo_double_module.stl" />
+          <mesh filename="package://delta/urdf/mesh/20240117_10inch/high_lipo_single_module.STL" />
         </geometry>
       </visual>

File: robots/delta/urdf/20240117_10inch/rolling_link.urdf.xacro (robot description, xacro)
@@ -89,86 +89,18 @@
     </xacro:unless>
     <!-- battery -->
-    <!-- battery: 1 = 6S ZIPPY 3000 (blue)              -->
-    <!-- battery: 2 = 6S Turningy high lipo (silver) x1 inner side -->
-    <!-- battery: 3 = 6S Turningy high lipo (silver) x1 outer side -->
-    <!-- battery: 4 = 6S Turningy high lipo (silver) x1 under side -->
-    <!-- battery: 5 = 6S Turningy high lipo (silver) x2 -->
+    <!-- battery: 1 = 6S Turningy high lipo (silver) x1 -->
     <xacro:if value="${battery == 1}">
-      <xacro:battery index="${self}"/>
-      <joint name="battery_joint${self}" type="fixed">
-        <parent link="link${self}"/>
-        <child link="battery${self}"/>
-        <xacro:if value="${self == 1}">
-          <origin xyz="0.32 0 0"/>
-        </xacro:if>
-        <xacro:if value="${self == 2}">
-          <origin xyz="0.3535 0 0"/>
-        </xacro:if>
-        <xacro:if value="${self == 3}">
-          <origin xyz="0.3535 0 0"/>
-        </xacro:if>
-      </joint>
-    </xacro:if>
-    <xacro:if value="${battery == 2}">
-      <xacro:high_lipo_single_inner index="${self}"/>
+      <xacro:high_lipo_single index="${self}"/>
       <joint name="battery_joint${self}" type="fixed">
         <parent link="link${self}"/>
         <child link="high_lipo_single${self}"/>
         <xacro:if value="${self == 1}">
-          <origin xyz="0.32 0 0"/>
+          <origin xyz="0.37192 -0.029 0" rpy="${pi / 2} 0 ${-pi / 2}"/>
         </xacro:if>
         <xacro:if value="${self == 2}">
-          <origin xyz="0.3535 0 0"/>
+          <origin xyz="0.40542 -0.029 0" rpy="${pi / 2} 0 ${-pi / 2}"/>
         </xacro:if>
         <xacro:if value="${self == 3}">
-          <origin xyz="0.3535 0 0"/>
-        </xacro:if>
-      </joint>
-    </xacro:if>
-    <xacro:if value="${battery == 3}">
-      <xacro:high_lipo_single_outer index="${self}"/>
-      <joint name="battery_joint${self}" type="fixed">
-        <parent link="link${self}"/>
-        <child link="high_lipo_single${self}"/>
-        <xacro:if value="${self == 1}">
-          <origin xyz="0.28 0 0"/>
-        </xacro:if>
-        <xacro:if value="${self == 2}">
-          <origin xyz="0.3135 0 0"/>
-        </xacro:if>
-        <xacro:if value="${self == 3}">
-          <origin xyz="0.3135 0 0"/>
-        </xacro:if>
-      </joint>
-    </xacro:if>
-    <xacro:if value="${battery == 4}">
-      <xacro:high_lipo_single_under index="${self}"/>
-      <joint name="battery_joint${self}" type="fixed">
-        <parent link="link${self}"/>
-        <child link="high_lipo_single${self}"/>
-        <xacro:if value="${self == 1}">
-          <origin xyz="0.310 0 0"/>
-        </xacro:if>
-        <xacro:if value="${self == 2}">
-          <origin xyz="0.3435 0 0"/>
-        </xacro:if>
-        <xacro:if value="${self == 3}">
-          <origin xyz="0.3435 0 0"/>
-        </xacro:if>
-      </joint>
-    </xacro:if>
-    <xacro:if value="${battery == 5}">
-      <xacro:high_lipo_double index="${self}"/>
-      <joint name="battery_joint${self}" type="fixed">
-        <parent link="link${self}"/>
-        <child link="high_lipo_double${self}"/>
-        <xacro:if value="${self == 1}">
-          <origin xyz="0.310 0 0"/>
-        </xacro:if>
-        <xacro:if value="${self == 2}">
-          <origin xyz="0.3435 0 0"/>
-        </xacro:if>
-        <xacro:if value="${self == 3}">
-          <origin xyz="0.3435 0 0"/>
+          <origin xyz="0.40542 -0.029 0" rpy="${pi / 2} 0 ${-pi / 2}"/>
         </xacro:if>
       </joint>
