Commit message: [delta] workaround to calculate real contact point based on cog state

File: robots/delta/urdf/20240117_10inch/link1.urdf.xacro (robot description, xacro)
@@ -37,4 +37,19 @@
       </visual>
     </link>
+    <link name="link1_center">
+      <inerial>
+        <origin xyz="0 0 0"/>
+          <mass value="0.00001"/>
+          <inertia
+              ixx="0.000001" ixy="0.0" ixz="0.0"
+              iyy="0.000001" iyz="0.0"
+              izz="0.000001"/>
+      </inerial>
+    </link>
+    <joint name="link1_center_joint" type="fixed">
+      <parent link="link1"/>
+      <child link="link1_center"/>
+      <origin xyz="0.23025 0.15228 0" rpy="0 0 ${pi}"/>
+    </joint>
   </xacro:macro>
 </robot>

File: robots/delta/urdf/20240117_10inch/link2.urdf.xacro (robot description, xacro)
@@ -37,4 +37,19 @@
       </visual>
     </link>
+    <link name="link2_center">
+      <inerial>
+        <origin xyz="0 0 0"/>
+          <mass value="0.00001"/>
+          <inertia
+              ixx="0.000001" ixy="0.0" ixz="0.0"
+              iyy="0.000001" iyz="0.0"
+              izz="0.000001"/>
+      </inerial>
+    </link>
+    <joint name="link2_center_joint" type="fixed">
+      <parent link="link2"/>
+      <child link="link2_center"/>
+      <origin xyz="0.26375 0.15228 0" rpy="0 0 ${pi}"/>
+    </joint>
   </xacro:macro>
 </robot>

File: robots/delta/urdf/20240117_10inch/link3.urdf.xacro (robot description, xacro)
@@ -37,4 +37,19 @@
       </visual>
     </link>
+    <link name="link3_center">
+      <inerial>
+        <origin xyz="0 0 0"/>
+          <mass value="0.00001"/>
+          <inertia
+              ixx="0.000001" ixy="0.0" ixz="0.0"
+              iyy="0.000001" iyz="0.0"
+              izz="0.000001"/>
+      </inerial>
+    </link>
+    <joint name="link3_center_joint" type="fixed">
+      <parent link="link3"/>
+      <child link="link3_center"/>
+      <origin xyz="0.26375 0.15228 0" rpy="0 0 ${pi}"/>
+    </joint>
   </xacro:macro>
 </robot>
