Commit message: [delta][urdf] fix mesh path

File: robots/delta/urdf/20240117_10inch/battery.urdf.xacro (robot description, xacro)
@@ -31,5 +31,5 @@
       <visual>
         <geometry>
-          <mesh filename="package://delta/urdf/mesh/20240117_10inch/high_lipo_single_module.STL" />
+          <mesh filename="package://delta/urdf/mesh/20240117_10inch/high_lipo_single_module.stl" />
         </geometry>
       </visual>
@@ -48,5 +48,5 @@
       <visual>
         <geometry>
-          <mesh filename="package://delta/urdf/mesh/20240117_10inch/high_lipo_double_module.STL" />
+          <mesh filename="package://delta/urdf/mesh/20240117_10inch/high_lipo_double_module.stl" />
         </geometry>
       </visual>

Commit message: [delta] fix origin of battery in urdf

File: robots/delta/urdf/20240117_10inch/battery.urdf.xacro (robot description, xacro)
@@ -40,5 +40,5 @@
     <link name="high_lipo_double${index}">
       <inertial>
-        <origin xyz="0.4390043 0.00000000 0.00000000" rpy="0 0 0"/>
+        <origin xyz="0.04390043 0.00000000 0.00000000" rpy="0 0 0"/>
         <mass value="0.45298185"/>
         <inertia
@@ -57,5 +57,5 @@
     <link name="high_lipo_single${index}">
       <inertial>
-        <origin xyz="0.4390043 0.00000000 -0.02750000" rpy="0 0 0"/>
+        <origin xyz="0.04390043 0.00000000 -0.02750000" rpy="0 0 0"/>
         <mass value="0.22649093"/>
         <inertia

Commit message: [delta][urdf] modify mesh extension for mujoco model generation

File: robots/delta/urdf/20240117_10inch/battery.urdf.xacro (robot description, xacro)
@@ -31,5 +31,5 @@
       <visual>
         <geometry>
-          <mesh filename="package://delta/urdf/mesh/20240117_10inch/high_lipo_single_module.STL" />
+          <mesh filename="package://delta/urdf/mesh/20240117_10inch/high_lipo_single_module.stl" />
         </geometry>
       </visual>
