Commit message: [delta][control] workaround to get rotor tile from urdf

File: robots/delta/urdf/20240117_10inch/rolling_link.urdf.xacro (robot description, xacro)
@@ -147,11 +147,11 @@
       <axis xyz="0 0 1"/>
       <xacro:if value="${self == 1}">
-        <origin xyz="0 0 0" rpy="0 -0.125 0"/>
+        <origin xyz="0 0 0" rpy="0 ${rotor_tilt1} 0"/>
       </xacro:if>
       <xacro:if value="${self == 2}">
-        <origin xyz="0 0 0" rpy="0 0.146 0"/>
+        <origin xyz="0 0 0" rpy="0 ${rotor_tilt2} 0"/>
       </xacro:if>
       <xacro:if value="${self == 3}">
-        <origin xyz="0 0 0" rpy="0 0.083 0"/>
+        <origin xyz="0 0 0" rpy="0 ${rotor_tilt3} 0"/>
       </xacro:if>
     </joint>

File: robots/delta/urdf/20240117_10inch/thrust.urdf.xacro (robot description, xacro)
@@ -5,3 +5,9 @@
   <xacro:property name="max_force" value="28.2" /> <!-- [N] -->
   <xacro:property name="min_force" value="0.0" /> <!-- [N] -->
+  <rotor_tilt1 value="-0.125"/>
+  <rotor_tilt2  value="0.146"/>
+  <rotor_tilt3  value="0.083"/>
+  <xacro:property name="rotor_tilt1" value="-0.125"/>
+  <xacro:property name="rotor_tilt2" value="0.146"/>
+  <xacro:property name="rotor_tilt3" value="0.083"/>
 </robot>
