Commit message: [delta] update urdf

File: robots/delta/urdf/20240207_new_armor/link1.urdf.xacro (robot description, xacro)
@@ -5,9 +5,9 @@
     <link name="link1">
       <inertial>
-        <origin xyz="0.29073125 -0.04875364 0.00356353" rpy="0 0 0"/>
-        <mass value="1.04062549"/>
+        <origin xyz="0.28794398 -0.04712329 0.00347969" rpy="0 0 0"/>
+        <mass value="1.08222549"/>
         <inertia
-            ixx="0.00487578"  iyy="0.03111063" izz="0.03370272"
-            ixy="-0.00077066" ixz="0.00156790" iyz="0.00018086" />
+             ixx="0.00498184" iyy="0.03252549" izz="0.03516989"
+            ixy="-0.00088064" ixz="0.00165575" iyz="0.00017753" />
       </inertial>
       <visual>
@@ -25,9 +25,9 @@
     <link name="gimbal_link1">
       <inertial>
-        <origin xyz="0.00936905 -0.00000232 0.01002430" rpy="0 0 0"/>
-        <mass value="0.26465910"/>
+        <origin xyz="0.00944096 -0.00000223 0.01141561" rpy="0 0 0"/>
+        <mass value="0.27443334"/>
         <inertia
-            ixx="0.00062925"  iyy="0.00070169"  izz="0.00017410"
-            ixy="0.00000004"  ixz="-0.00017063" iyz="0.00000004" />
+            ixx="0.00066652"  iyy="0.00074131" izz="0.00017798"
+            ixy="0.00000004" ixz="-0.00017867" iyz="0.00000005" />
       </inertial>
       <visual>

File: robots/delta/urdf/20240207_new_armor/link2.urdf.xacro (robot description, xacro)
@@ -5,9 +5,9 @@
     <link name="link2">
       <inertial>
-        <origin xyz="0.29447929 -0.04304240 0.00219467" rpy="0 0 0"/>
-        <mass value="1.17603627"/>
+        <origin xyz="0.29247546 -0.04173228 0.00214003" rpy="0 0 0"/>
+        <mass value="1.21919627"/>
         <inertia
-            ixx="0.00529347"  iyy="0.03954260" izz="0.04242468"
-            ixy="-0.00230287" ixz="0.00207827" iyz="0.00011471" />
+             ixx="0.00538607" iyy="0.04105715" izz="0.04397541"
+            ixy="-0.00237976" ixz="0.00218016" iyz="0.00011267" />
       </inertial>
       <visual>
@@ -25,9 +25,9 @@
     <link name="gimbal_link2">
       <inertial>
-        <origin xyz="0.01251605 -0.00000228 0.01144490" rpy="0 0 0"/>
-        <mass value="0.26844267"/>
+        <origin xyz="0.01205240 -0.00000221 0.01260343" rpy="0 0 0"/>
+        <mass value="0.27751558"/>
         <inertia
-            ixx="0.00065559"  iyy="0.00071177"  izz="0.00015907"
-            ixy="0.00000004"  ixz="-0.00013895" iyz="0.00000005"/>
+            ixx="0.00068946"  iyy="0.00075023" izz="0.00016497"
+            ixy="0.00000004" ixz="-0.00015101" iyz="0.00000005"/>
       </inertial>
       <visual>

File: robots/delta/urdf/20240207_new_armor/link3.urdf.xacro (robot description, xacro)
@@ -5,9 +5,9 @@
     <link name="link3">
       <inertial>
-        <origin xyz="0.29414327 -0.05513197 -0.00624486" rpy="0 0 0"/>
-        <mass value="0.91687816"/>
+        <origin xyz="0.29164273 -0.05294374 -0.00632002" rpy="0 0 0"/>
+        <mass value="0.95975816"/>
         <inertia
-            ixx="0.00464612"  iyy="0.03077571"  izz="0.03297254"
-            ixy="-0.00234213" ixz="0.00008767" iyz="-0.00031567" />
+             ixx="0.00478040"  iyy="0.03231099"  izz="0.03458590"
+            ixy="-0.00244503"  ixz="0.00009334" iyz="-0.00032114" />
       </inertial>
       <visual>
@@ -25,9 +25,9 @@
     <link name="gimbal_link3">
       <inertial>
-        <origin xyz="0.00925022 -0.00000236 0.01013816" rpy="0 0 0"/>
-        <mass value="0.26494712"/>
+        <origin xyz="0.00935372 -0.00000228 0.01150070" rpy="0 0 0"/>
+        <mass value="0.27464497"/>
         <inertia
-            ixx="0.00063135" iyy="0.00070447"  izz="0.00017487"
-            ixy="0.00000004" ixz="-0.00017210" iyz="0.00000004" />
+            ixx="0.00066816"  iyy="0.00074345"  izz="0.00017856"
+            ixy="0.00000004" ixz="-0.00017982"  iyz="0.00000005" />
       </inertial>
       <visual>

File: robots/delta/urdf/20240207_new_armor/thrust.urdf.xacro (robot description, xacro)
@@ -5,9 +5,9 @@
   <xacro:property name="max_force" value="28.2" /> <!-- [N] -->
   <xacro:property name="min_force" value="0.0" /> <!-- [N] -->
-  <rotor_tilt1 value="-0.0876"/>
-  <rotor_tilt2  value="0.217"/>
-  <rotor_tilt3 value="-0.0975"/>
-  <xacro:property name="rotor_tilt1" value="-0.0876"/>
-  <xacro:property name="rotor_tilt2" value="0.217"/>
-  <xacro:property name="rotor_tilt3" value="-0.0975"/>
+  <rotor_tilt1 value="-0.0727822"/>
+  <rotor_tilt2  value="0.178982"/>
+  <rotor_tilt3 value="-0.0802372"/>
+  <xacro:property name="rotor_tilt1" value="-0.0727822"/>
+  <xacro:property name="rotor_tilt2" value="0.178982"/>
+  <xacro:property name="rotor_tilt3" value="-0.0802372"/>
 </robot>
