Commit message: [delta] update motor info: gemfan 9inch 3wing

File: robots/delta/urdf/20240207_new_armor/thrust.urdf.xacro (robot description, xacro)
@@ -2,6 +2,6 @@
 <robot
     xmlns:xacro="http://www.ros.org/wiki/xacro" name="delta_common" >
-  <m_f_rate value="-0.0146" /> <!-- drug torque rate -->
-  <xacro:property name="max_force" value="28.2" /> <!-- [N] -->
+  <m_f_rate value="-0.0156" /> <!-- drug torque rate -->
+  <xacro:property name="max_force" value="26.5" /> <!-- [N] -->
   <xacro:property name="min_force" value="0.0" /> <!-- [N] -->
   <rotor_tilt1 value="-0.0727822"/>
