Commit message: [Bi][NMPC]: add URDF model; add the initial version for NMPC controller, build successfully, but run with error.

File: robots/gimbalrotor/robots/bi/gimbalrotor.gazebo.xacro (robot description, xacro)
@@ -1,7 +1,7 @@
 <?xml version="1.0"?>
 <robot
-    xmlns:xacro="http://www.ros.org/wiki/xacro" name="beetle" >
-  <xacro:arg name="robot_name" default="beetle" />
-  <xacro:include filename="$(find beetle)/robots/beetle-art.urdf.xacro" />
+    xmlns:xacro="http://www.ros.org/wiki/xacro" name="gimbalrotor" >
+  <xacro:arg name="robot_name" default="gimbalrotor" />
+  <xacro:include filename="$(find gimbalrotor)/robots/bi/gimbalrotor.urdf.xacro" />
   <!-- gazebo plugin for default controller and sensors -->
   <xacro:include filename="$(find aerial_robot_simulation)/xacro/spinal.gazebo.xacro" />

File: robots/gimbalrotor/urdf/bi/common.xacro (robot description, xacro)
@@ -1,10 +1,10 @@
 <?xml version="1.0"?>
 <robot
-    xmlns:xacro="http://www.ros.org/wiki/xacro" name="beetle_common" >
+    xmlns:xacro="http://www.ros.org/wiki/xacro" name="birotor_common" >
   <!-- general attribute -->
   <baselink name="fc" />
   <thrust_link name="thrust" />
   <m_f_rate value="-0.0172" /> <!-- drug torque rate -->
-  <xacro:property name="max_force" value="30.0" /> <!-- [N] -->
+  <xacro:property name="max_force" value="18.0" /> <!-- [N] -->
   <xacro:property name="min_force" value="1.0" /> <!-- [N] -->
   <!-- friction -->
