Commit message: [hydrus_gripper] set correst jetson processor's mass

File: robots/hydrus_gripper/robots/robot.urdf.xacro (robot description, xacro)
@@ -46,5 +46,5 @@
     <origin xyz="${link_length / 2 + 0.2845} 0.011 0.016" rpy="0 0 ${pi}"/>
     <inertial>
-      <mass value = "0.120" />  <!-- TODO: set the correct mass -->
+      <mass value = "0.148" />
       <origin xyz="${21 * 0.001} ${4 * 0.001} ${12 * 0.001}" rpy="0 0 0"/>
       <inertia

Commit message: [hydrus_gripper] set hokuyo_pos to observe self body

File: robots/hydrus_gripper/robots/robot.urdf.xacro (robot description, xacro)
@@ -119,5 +119,5 @@
   <xacro:include filename="$(find hector_sensors_description)/urdf/hokuyo_utm30lx.urdf.xacro" />
   <xacro:hokuyo_utm30lx_model name="laser" parent="link3">
-    <origin xyz="0.0 0.0 0.12" rpy="0 0 0"/>
+    <origin xyz="0.0 0.0 0.20" rpy="0 0 0"/>
   </xacro:hokuyo_utm30lx_model>
 </robot>

Commit message: [hydrus_gripper][WIP] debug of stop observation in moving obstacle

File: robots/hydrus_gripper/robots/robot.urdf.xacro (robot description, xacro)
@@ -119,5 +119,5 @@
   <xacro:include filename="$(find hector_sensors_description)/urdf/hokuyo_utm30lx.urdf.xacro" />
   <xacro:hokuyo_utm30lx_model name="laser" parent="link3">
-    <origin xyz="0.0 0.0 0.20" rpy="0 0 0"/>
+    <origin xyz="0.0 0.0 0.30" rpy="0 0 0"/>
   </xacro:hokuyo_utm30lx_model>
 </robot>

Commit message: [hydrus_gripper][debug] same as direction as hokuyo and CoG direction

File: robots/hydrus_gripper/robots/robot.urdf.xacro (robot description, xacro)
@@ -119,5 +119,5 @@
   <xacro:include filename="$(find hector_sensors_description)/urdf/hokuyo_utm30lx.urdf.xacro" />
   <xacro:hokuyo_utm30lx_model name="laser" parent="link3">
-    <origin xyz="0.0 0.0 0.30" rpy="0 0 0"/>
+    <origin xyz="0.0 0.0 0.30" rpy="0 0 -1.57"/>
   </xacro:hokuyo_utm30lx_model>
 </robot>

Commit message: [hydrus_gripper] set different origin to fit real hokuyo config

File: robots/hydrus_gripper/robots/robot.urdf.xacro (robot description, xacro)
@@ -119,5 +119,5 @@
   <xacro:include filename="$(find hector_sensors_description)/urdf/hokuyo_utm30lx.urdf.xacro" />
   <xacro:hokuyo_utm30lx_model name="laser" parent="link3">
-    <origin xyz="0.0 0.0 0.30" rpy="0 0 -1.57"/>
+    <origin xyz="0.23 0.23 0.27" rpy="0 0 -1.57"/>
   </xacro:hokuyo_utm30lx_model>
 </robot>

Commit message: [hydrus_gripper] show obstacle setting to fit hokuyo estimation result

File: robots/hydrus_gripper/robots/robot.urdf.xacro (robot description, xacro)
@@ -119,5 +119,5 @@
   <xacro:include filename="$(find hector_sensors_description)/urdf/hokuyo_utm30lx.urdf.xacro" />
   <xacro:hokuyo_utm30lx_model name="laser" parent="link3">
-    <origin xyz="0.23 0.23 0.27" rpy="0 0 -1.57"/>
+    <origin xyz="0.18 0.23 0.27" rpy="0 0 -1.57"/>
   </xacro:hokuyo_utm30lx_model>
 </robot>
