Commit message: [hydrus_gripper] set hydrus obstacle hokuyo setting for obstacle estimation

File: robots/hydrus_gripper/robots/robot.gazebo.xacro (robot description, xacro)
@@ -125,3 +125,39 @@
     </sensor>
   </gazebo>
+  <!-- hokuyo -->
+  <xacro:property name="ray_count" default="1081" />
+  <xacro:property name="max_angle" default="135" />
+  <gazebo reference="laser_frame">
+    <sensor type="ray" name="laser">
+      <always_on>true</always_on>
+      <update_rate>40</update_rate>
+      <pose>0 0 0 0 0 0</pose>
+      <visualize>false</visualize>
+      <ray>
+        <scan>
+          <horizontal>
+            <samples>${ray_count}</samples>
+            <resolution>1</resolution>
+            <min_angle>${-max_angle * M_PI/180}</min_angle>
+            <max_angle>${max_angle * M_PI/180}</max_angle>
+          </horizontal>
+        </scan>
+        <range>
+          <min>0.1</min>
+          <max>20.0</max>
+          <resolution>0.01</resolution>
+        </range>
+        <noise>
+          <type>gaussian</type>
+          <mean>0.0</mean>
+          <stddev>0.004</stddev>
+        </noise>
+      </ray>
+      <plugin name="gazebo_ros_laser_controller" filename="libgazebo_ros_laser.so">
+        <robotNamespace>$(arg robot_name)</robotNamespace>
+        <topicName>scan</topicName>
+        <frameName>multirotor/laser_frame</frameName>
+      </plugin>
+    </sensor>
+  </gazebo>
 </robot>

File: robots/hydrus_gripper/robots/robot.urdf.xacro (robot description, xacro)
@@ -117,3 +117,7 @@
     </actuator>
   </transmission>
+  <xacro:include filename="$(find hector_sensors_description)/urdf/hokuyo_utm30lx.urdf.xacro" />
+  <xacro:hokuyo_utm30lx_model name="laser" parent="link3">
+    <origin xyz="0.0 0.0 0.12" rpy="0 0 0"/>
+  </xacro:hokuyo_utm30lx_model>
 </robot>

Commit message: [hydrus_gripper] update urdf: disable realsense and hokuyo

File: robots/hydrus_gripper/robots/robot.gazebo.xacro (robot description, xacro)
@@ -7,157 +7,157 @@
   <xacro:include filename="$(find aerial_robot_simulation)/xacro/spinal.gazebo.xacro" />
   <xacro:gazebo_spinal robot_name="hydrus" />
-  <!-- gazebo for Realsense D435 -->
-  <!--  The following values model the aluminum peripherial case for the
-        D435 camera, with the camera joint represented by the actual
-        peripherial camera tripod mount -->
-  <xacro:property name="d435_cam_depth_to_left_ir_offset" value="0.0"/>
-  <xacro:property name="d435_cam_depth_to_right_ir_offset" value="-0.050"/>
-  <xacro:property name="d435_cam_depth_to_color_offset" value="0.015"/>
-  <xacro:property name="d435_cam_width" value="0.090"/>
-  <xacro:property name="d435_cam_height" value="0.025"/>
-  <xacro:property name="d435_cam_depth" value="0.02505"/>
-  <xacro:property name="d435_cam_mount_from_center_offset" value="0.0149"/>
-  <!--  The following offset is relative the the physical D435 camera peripherial
-        camera tripod mount -->
-  <xacro:property name="d435_cam_depth_px" value="${d435_cam_mount_from_center_offset}"/>
-  <xacro:property name="d435_cam_depth_py" value="0.0175"/>
-  <xacro:property name="d435_cam_depth_pz" value="${d435_cam_height/2}"/>
-  <material name="aluminum">
-    <color rgba="0.5 0.5 0.5 1"/>
-  </material>
-  <!-- camera depth joints and links -->
-  <joint name="rs_d435_depth_joint" type="fixed">
-    <origin xyz="0 0 0" rpy="0 0 0"/>
-    <parent link="rs_d435_link"/>
-    <child link="rs_d435_depth_frame" />
-  </joint>
-  <link name="rs_d435_depth_frame"/>
-  <joint name="rs_d435_depth_optical_joint" type="fixed">
-    <origin xyz="0 0 0" rpy="${-pi/2} 0 ${-pi/2}" />
-    <parent link="rs_d435_depth_frame" />
-    <child link="rs_d435_depth_optical_frame" />
-  </joint>
-  <link name="rs_d435_depth_optical_frame"/>
-  <!-- camera left IR joints and links -->
-  <joint name="rs_d435_left_ir_joint" type="fixed">
-    <origin xyz="0 ${d435_cam_depth_to_left_ir_offset} 0" rpy="0 0 0" />
-    <parent link="rs_d435_depth_frame" />
-    <child link="rs_d435_left_ir_frame" />
-  </joint>
-  <link name="rs_d435_left_ir_frame"/>
-  <joint name="rs_d435_left_ir_optical_joint" type="fixed">
-    <origin xyz="0 0 0" rpy="${-pi/2} 0 ${-pi/2}" />
-    <parent link="rs_d435_left_ir_frame" />
-    <child link="rs_d435_left_ir_optical_frame" />
-  </joint>
-  <link name="rs_d435_left_ir_optical_frame"/>
-  <!-- camera right IR joints and links -->
-  <joint name="rs_d435_right_ir_joint" type="fixed">
-    <origin xyz="0 ${d435_cam_depth_to_right_ir_offset} 0" rpy="0 0 0" />
-    <parent link="rs_d435_depth_frame" />
-    <child link="rs_d435_right_ir_frame" />
-  </joint>
-  <link name="rs_d435_right_ir_frame"/>
-  <joint name="rs_d435_right_ir_optical_joint" type="fixed">
-    <origin xyz="0 0 0" rpy="${-pi/2} 0 ${-pi/2}" />
-    <parent link="rs_d435_right_ir_frame" />
-    <child link="rs_d435_right_ir_optical_frame" />
-  </joint>
-  <link name="rs_d435_right_ir_optical_frame"/>
-  <!-- camera color joints and links -->
-  <joint name="rs_d435_color_joint" type="fixed">
-    <origin xyz="0 ${d435_cam_depth_to_color_offset} 0" rpy="0 0 0" />
-    <parent link="rs_d435_depth_frame" />
-    <child link="rs_d435_color_frame" />
-  </joint>
-  <link name="rs_d435_color_frame"/>
-  <joint name="rs_d435_color_optical_joint" type="fixed">
-    <origin xyz="0 0 0" rpy="${-pi/2} 0 ${-pi/2}" />
-    <parent link="rs_d435_color_frame" />
-    <child link="rs_d435_color_optical_frame" />
-  </joint>
-  <link name="rs_d435_color_optical_frame"/>
-  <!-- gazebo plugin -->
-  <gazebo reference="rs_d435_color_frame">
-    <sensor type="depth" name="rs_d435_camera">
-      <update_rate>20.0</update_rate>
-      <camera name="head">
-	<horizontal_fov>1.59174</horizontal_fov>
-	<!--vertical_fov>1.14319</vertical_fov-->
-	<image>
-	  <width>1280</width>
-	  <height>720</height>
-	  <format>RGB</format>
-	</image>
-	<clip>
-	  <near>0.02</near>
-	  <far>300</far>
-	</clip>
-	<noise>
-	  <type>gaussian</type>
-	  <mean>0.0</mean>
-	  <stddev>0.007</stddev>
-	</noise>
-      </camera>
-      <plugin name="depth_camera" filename="libgazebo_ros_openni_kinect.so">
-	<baseline>0.06</baseline>
-	<alwaysOn>true</alwaysOn>
-	<updateRate>0.0</updateRate>
-	<cameraName>rs_d435</cameraName>
-	<imageTopicName>color/image_rect_color</imageTopicName>
-	<cameraInfoTopicName>color/camera_info</cameraInfoTopicName>
-	<depthImageCameraInfoTopicName>aligned_depth_to_color/camera_info</depthImageCameraInfoTopicName>
-	<depthImageTopicName>aligned_depth_to_color/image_raw</depthImageTopicName>
-	<pointCloudTopicName>depth_registered/points</pointCloudTopicName>
-	<frameName>rs_d435_color_optical_frame</frameName>
-	<pointCloudCutoff>0.05</pointCloudCutoff>
-	<distortionK1>0</distortionK1>
-	<distortionK2>0</distortionK2>
-	<distortionK3>0</distortionK3>
-	<distortionT1>0</distortionT1>
-	<distortionT2>0</distortionT2>
-	<CxPrime>0</CxPrime>
-	<Cx>0</Cx>
-	<Cy>0</Cy>
-	<focalLength>0</focalLength>
-	<hackBaseline>0</hackBaseline>
-      </plugin>
-    </sensor>
-  </gazebo>
-  <!-- hokuyo -->
-  <xacro:property name="ray_count" default="1081" />
-  <xacro:property name="max_angle" default="135" />
-  <gazebo reference="laser_frame">
-    <sensor type="ray" name="laser">
-      <always_on>true</always_on>
-      <update_rate>40</update_rate>
-      <pose>0 0 0 0 0 0</pose>
-      <visualize>false</visualize>
-      <ray>
-        <scan>
-          <horizontal>
-            <samples>${ray_count}</samples>
-            <resolution>1</resolution>
-            <min_angle>${-max_angle * M_PI/180}</min_angle>
-            <max_angle>${max_angle * M_PI/180}</max_angle>
-          </horizontal>
-        </scan>
-        <range>
-          <min>0.1</min>
-          <max>20.0</max>
-          <resolution>0.01</resolution>
-        </range>
-        <noise>
-          <type>gaussian</type>
-          <mean>0.0</mean>
-          <stddev>0.004</stddev>
-        </noise>
-      </ray>
-      <plugin name="gazebo_ros_laser_controller" filename="libgazebo_ros_laser.so">
-        <robotNamespace>$(arg robot_name)</robotNamespace>
-        <topicName>scan</topicName>
-        <frameName>hydrus/laser_frame</frameName>
-      </plugin>
-    </sensor>
-  </gazebo>
+  <!-- <!-\- gazebo for Realsense D435 -\-> -->
+  <!-- <!-\-  The following values model the aluminum peripherial case for the -->
+  <!--       D435 camera, with the camera joint represented by the actual -->
+  <!--       peripherial camera tripod mount -\-> -->
+  <!-- <xacro:property name="d435_cam_depth_to_left_ir_offset" value="0.0"/> -->
+  <!-- <xacro:property name="d435_cam_depth_to_right_ir_offset" value="-0.050"/> -->
+  <!-- <xacro:property name="d435_cam_depth_to_color_offset" value="0.015"/> -->
+  <!-- <xacro:property name="d435_cam_width" value="0.090"/> -->
+  <!-- <xacro:property name="d435_cam_height" value="0.025"/> -->
+  <!-- <xacro:property name="d435_cam_depth" value="0.02505"/> -->
+  <!-- <xacro:property name="d435_cam_mount_from_center_offset" value="0.0149"/> -->
+  <!-- <!-\-  The following offset is relative the the physical D435 camera peripherial -->
+  <!--       camera tripod mount -\-> -->
+  <!-- <xacro:property name="d435_cam_depth_px" value="${d435_cam_mount_from_center_offset}"/> -->
+  <!-- <xacro:property name="d435_cam_depth_py" value="0.0175"/> -->
+  <!-- <xacro:property name="d435_cam_depth_pz" value="${d435_cam_height/2}"/> -->
+  <!-- <material name="aluminum"> -->
+  <!--   <color rgba="0.5 0.5 0.5 1"/> -->
+  <!-- </material> -->
+  <!-- <!-\- camera depth joints and links -\-> -->
+  <!-- <joint name="rs_d435_depth_joint" type="fixed"> -->
+  <!--   <origin xyz="0 0 0" rpy="0 0 0"/> -->
+  <!--   <parent link="rs_d435_link"/> -->
+  <!--   <child link="rs_d435_depth_frame" /> -->
+  <!-- </joint> -->
+  <!-- <link name="rs_d435_depth_frame"/> -->
+  <!-- <joint name="rs_d435_depth_optical_joint" type="fixed"> -->
+  <!--   <origin xyz="0 0 0" rpy="${-pi/2} 0 ${-pi/2}" /> -->
+  <!--   <parent link="rs_d435_depth_frame" /> -->
+  <!--   <child link="rs_d435_depth_optical_frame" /> -->
+  <!-- </joint> -->
+  <!-- <link name="rs_d435_depth_optical_frame"/> -->
+  <!-- <!-\- camera left IR joints and links -\-> -->
+  <!-- <joint name="rs_d435_left_ir_joint" type="fixed"> -->
+  <!--   <origin xyz="0 ${d435_cam_depth_to_left_ir_offset} 0" rpy="0 0 0" /> -->
+  <!--   <parent link="rs_d435_depth_frame" /> -->
+  <!--   <child link="rs_d435_left_ir_frame" /> -->
+  <!-- </joint> -->
+  <!-- <link name="rs_d435_left_ir_frame"/> -->
+  <!-- <joint name="rs_d435_left_ir_optical_joint" type="fixed"> -->
+  <!--   <origin xyz="0 0 0" rpy="${-pi/2} 0 ${-pi/2}" /> -->
+  <!--   <parent link="rs_d435_left_ir_frame" /> -->
+  <!--   <child link="rs_d435_left_ir_optical_frame" /> -->
+  <!-- </joint> -->
+  <!-- <link name="rs_d435_left_ir_optical_frame"/> -->
+  <!-- <!-\- camera right IR joints and links -\-> -->
+  <!-- <joint name="rs_d435_right_ir_joint" type="fixed"> -->
+  <!--   <origin xyz="0 ${d435_cam_depth_to_right_ir_offset} 0" rpy="0 0 0" /> -->
+  <!--   <parent link="rs_d435_depth_frame" /> -->
+  <!--   <child link="rs_d435_right_ir_frame" /> -->
+  <!-- </joint> -->
+  <!-- <link name="rs_d435_right_ir_frame"/> -->
+  <!-- <joint name="rs_d435_right_ir_optical_joint" type="fixed"> -->
+  <!--   <origin xyz="0 0 0" rpy="${-pi/2} 0 ${-pi/2}" /> -->
+  <!--   <parent link="rs_d435_right_ir_frame" /> -->
+  <!--   <child link="rs_d435_right_ir_optical_frame" /> -->
+  <!-- </joint> -->
+  <!-- <link name="rs_d435_right_ir_optical_frame"/> -->
+  <!-- <!-\- camera color joints and links -\-> -->
+  <!-- <joint name="rs_d435_color_joint" type="fixed"> -->
+  <!--   <origin xyz="0 ${d435_cam_depth_to_color_offset} 0" rpy="0 0 0" /> -->
+  <!--   <parent link="rs_d435_depth_frame" /> -->
+  <!--   <child link="rs_d435_color_frame" /> -->
+  <!-- </joint> -->
+  <!-- <link name="rs_d435_color_frame"/> -->
+  <!-- <joint name="rs_d435_color_optical_joint" type="fixed"> -->
+  <!--   <origin xyz="0 0 0" rpy="${-pi/2} 0 ${-pi/2}" /> -->
+  <!--   <parent link="rs_d435_color_frame" /> -->
+  <!--   <child link="rs_d435_color_optical_frame" /> -->
+  <!-- </joint> -->
+  <!-- <link name="rs_d435_color_optical_frame"/> -->
+  <!-- <!-\- gazebo plugin -\-> -->
+  <!-- <gazebo reference="rs_d435_color_frame"> -->
+  <!--   <sensor type="depth" name="rs_d435_camera"> -->
+  <!--     <update_rate>20.0</update_rate> -->
+  <!--     <camera name="head"> -->
+  <!--       <horizontal_fov>1.59174</horizontal_fov> -->
+  <!--       <!-\-vertical_fov>1.14319</vertical_fov-\-> -->
+  <!--       <image> -->
+  <!--         <width>1280</width> -->
+  <!--         <height>720</height> -->
+  <!--         <format>RGB</format> -->
+  <!--       </image> -->
+  <!--       <clip> -->
+  <!--         <near>0.02</near> -->
+  <!--         <far>300</far> -->
+  <!--       </clip> -->
+  <!--       <noise> -->
+  <!--         <type>gaussian</type> -->
+  <!--         <mean>0.0</mean> -->
+  <!--         <stddev>0.007</stddev> -->
+  <!--       </noise> -->
+  <!--     </camera> -->
+  <!--     <plugin name="depth_camera" filename="libgazebo_ros_openni_kinect.so"> -->
+  <!--       <baseline>0.06</baseline> -->
+  <!--       <alwaysOn>true</alwaysOn> -->
+  <!--       <updateRate>0.0</updateRate> -->
+  <!--       <cameraName>rs_d435</cameraName> -->
+  <!--       <imageTopicName>color/image_rect_color</imageTopicName> -->
+  <!--       <cameraInfoTopicName>color/camera_info</cameraInfoTopicName> -->
+  <!--       <depthImageCameraInfoTopicName>aligned_depth_to_color/camera_info</depthImageCameraInfoTopicName> -->
+  <!--       <depthImageTopicName>aligned_depth_to_color/image_raw</depthImageTopicName> -->
+  <!--       <pointCloudTopicName>depth_registered/points</pointCloudTopicName> -->
+  <!--       <frameName>rs_d435_color_optical_frame</frameName> -->
+  <!--       <pointCloudCutoff>0.05</pointCloudCutoff> -->
+  <!--       <distortionK1>0</distortionK1> -->
+  <!--       <distortionK2>0</distortionK2> -->
+  <!--       <distortionK3>0</distortionK3> -->
+  <!--       <distortionT1>0</distortionT1> -->
+  <!--       <distortionT2>0</distortionT2> -->
+  <!--       <CxPrime>0</CxPrime> -->
+  <!--       <Cx>0</Cx> -->
+  <!--       <Cy>0</Cy> -->
+  <!--       <focalLength>0</focalLength> -->
+  <!--       <hackBaseline>0</hackBaseline> -->
+  <!--     </plugin> -->
+  <!--   </sensor> -->
+  <!-- </gazebo> -->
+  <!-- <!-\- hokuyo -\-> -->
+  <!-- <xacro:property name="ray_count" default="1081" /> -->
+  <!-- <xacro:property name="max_angle" default="135" /> -->
+  <!-- <gazebo reference="laser_frame"> -->
+  <!--   <sensor type="ray" name="laser"> -->
+  <!--     <always_on>true</always_on> -->
+  <!--     <update_rate>40</update_rate> -->
+  <!--     <pose>0 0 0 0 0 0</pose> -->
+  <!--     <visualize>false</visualize> -->
+  <!--     <ray> -->
+  <!--       <scan> -->
+  <!--         <horizontal> -->
+  <!--           <samples>${ray_count}</samples> -->
+  <!--           <resolution>1</resolution> -->
+  <!--           <min_angle>${-max_angle * M_PI/180}</min_angle> -->
+  <!--           <max_angle>${max_angle * M_PI/180}</max_angle> -->
+  <!--         </horizontal> -->
+  <!--       </scan> -->
+  <!--       <range> -->
+  <!--         <min>0.1</min> -->
+  <!--         <max>20.0</max> -->
+  <!--         <resolution>0.01</resolution> -->
+  <!--       </range> -->
+  <!--       <noise> -->
+  <!--         <type>gaussian</type> -->
+  <!--         <mean>0.0</mean> -->
+  <!--         <stddev>0.004</stddev> -->
+  <!--       </noise> -->
+  <!--     </ray> -->
+  <!--     <plugin name="gazebo_ros_laser_controller" filename="libgazebo_ros_laser.so"> -->
+  <!--       <robotNamespace>$(arg robot_name)</robotNamespace> -->
+  <!--       <topicName>scan</topicName> -->
+  <!--       <frameName>hydrus/laser_frame</frameName> -->
+  <!--     </plugin> -->
+  <!--   </sensor> -->
+  <!-- </gazebo> -->
 </robot>

File: robots/hydrus_gripper/robots/robot.urdf.xacro (robot description, xacro)
@@ -57,67 +57,67 @@
   <!-- 2. Realsense D435 -->
   <!-- TODO: accurate intertia parameters and position -->
-  <xacro:extra_module name = "rs_d435_mount" parent = "link2" visible = "1"
-                      model_url = "package://hydrus_gripper/urdf/mesh/modules/sensor/rs_d435_unit2.STL">
-    <origin xyz="${link_length / 2} 0 0" rpy="0 0 0"/>
-    <inertial>
-      <mass value = "0.0" />
-      <origin xyz="0 0 0" rpy="0 0 0"/>
-      <inertia
-          ixx="0.0" ixy="0.0" ixz="0.0"
-          iyy="0.0" iyz="0.0" izz="0.0"/>
-    </inertial>
-  </xacro:extra_module>
-  <joint name="rs_d435_servo_joint" type="revolute">
-    <limit effort="0.2" lower="0" upper="1.8" velocity="0.1"/>
-    <parent link="link2"/>
-    <child link="rs_d435_servo"/>
-    <origin xyz="${link_length / 2 + 0.20395} 0.02495 -0.038" rpy="0 0 ${pi/4}"/>
-    <axis xyz="-1 0 0"/>
-    <dynamics damping="0.01" friction="0.0"/>
-  </joint>
-  <link name="rs_d435_servo">
-    <inertial>
-      <mass value = "0" />
-      <origin xyz="0 0 0" rpy="0 0 0"/>
-      <inertia
-          ixx="0.0" ixy="0.0" ixz="0.0"
-          iyy="0.0" iyz="0.0" izz="0.0"/>
-    </inertial>
-  </link>
-  <xacro:extra_module name = "rs_d435_unit" parent = "rs_d435_servo" visible = "1" model_url = "package://hydrus_gripper/urdf/mesh/modules/sensor/rs_d435_unit1.STL">
-    <origin xyz="0.05275 0.01005 0" rpy="0 0 ${pi / 2}"/>
-    <inertial>
-      <mass value = "0.124" /> <!-- includes usb cable, servo, mounts -->
-      <origin xyz="-0.01005 0 0" rpy="0 0 0"/>
-      <inertia
-          ixx="0.0001" iyy="0.0001" izz="0.0002"
-          ixy="0" ixz="0" iyz="0"/>
-    </inertial>
-  </xacro:extra_module>
-  <!-- rs_d435_link is the parrent of sensors' frame, identical to rs_d435_left_ir_frame  -->
-  <xacro:extra_module name = "rs_d435_link" parent = "rs_d435_unit" visible = "0" >
-    <origin xyz="-0.008 0.0175 0 " rpy="0 0 0"/>
-    <inertial>
-      <mass value = "0.0" />
-      <origin xyz="0 0 0" rpy="0 0 0"/>
-      <inertia
-          ixx="0.0" ixy="0.0" ixz="0.0"
-          iyy="0.0" iyz="0.0"
-          izz="0.0"/>
-    </inertial>
-  </xacro:extra_module>
-  <transmission name="rs_d435_servo_joint_tran">
-    <type>transmission_interface/SimpleTransmission</type>
-    <joint name="rs_d435_servo_joint">
-      <hardwareInterface>hardware_interface/EffortJointInterface</hardwareInterface>
-    </joint>
-    <actuator name="rs_d435_servo_joint">
-      <hardwareInterface>hardware_interface/EffortJointInterface</hardwareInterface>
-      <mechanicalReduction>1</mechanicalReduction>
-    </actuator>
-  </transmission>
-  <xacro:include filename="$(find hector_sensors_description)/urdf/hokuyo_utm30lx.urdf.xacro" />
-  <xacro:hokuyo_utm30lx_model name="laser" parent="link3">
-    <origin xyz="0.18 0.23 0.27" rpy="0 0 -1.57"/>
-  </xacro:hokuyo_utm30lx_model>
+  <!-- <xacro:extra_module name = "rs_d435_mount" parent = "link2" visible = "1" -->
+  <!--                     model_url = "package://hydrus_gripper/urdf/mesh/modules/sensor/rs_d435_unit2.STL"> -->
+  <!--   <origin xyz="${link_length / 2} 0 0" rpy="0 0 0"/> -->
+  <!--   <inertial> -->
+  <!--     <mass value = "0.0" /> -->
+  <!--     <origin xyz="0 0 0" rpy="0 0 0"/> -->
+  <!--     <inertia -->
+  <!--         ixx="0.0" ixy="0.0" ixz="0.0" -->
+  <!--         iyy="0.0" iyz="0.0" izz="0.0"/> -->
+  <!--   </inertial> -->
+  <!-- </xacro:extra_module> -->
+  <!-- <joint name="rs_d435_servo_joint" type="revolute"> -->
+  <!--   <limit effort="0.2" lower="0" upper="1.8" velocity="0.1"/> -->
+  <!--   <parent link="link2"/> -->
+  <!--   <child link="rs_d435_servo"/> -->
+  <!--   <origin xyz="${link_length / 2 + 0.20395} 0.02495 -0.038" rpy="0 0 ${pi/4}"/> -->
+  <!--   <axis xyz="-1 0 0"/> -->
+  <!--   <dynamics damping="0.01" friction="0.0"/> -->
+  <!-- </joint> -->
+  <!-- <link name="rs_d435_servo"> -->
+  <!--   <inertial> -->
+  <!--     <mass value = "0" /> -->
+  <!--     <origin xyz="0 0 0" rpy="0 0 0"/> -->
+  <!--     <inertia -->
+  <!--         ixx="0.0" ixy="0.0" ixz="0.0" -->
+  <!--         iyy="0.0" iyz="0.0" izz="0.0"/> -->
+  <!--   </inertial> -->
+  <!-- </link> -->
+  <!-- <xacro:extra_module name = "rs_d435_unit" parent = "rs_d435_servo" visible = "1" model_url = "package://hydrus_gripper/urdf/mesh/modules/sensor/rs_d435_unit1.STL"> -->
+  <!--   <origin xyz="0.05275 0.01005 0" rpy="0 0 ${pi / 2}"/> -->
+  <!--   <inertial> -->
+  <!--     <mass value = "0.124" /> <!-\- includes usb cable, servo, mounts -\-> -->
+  <!--     <origin xyz="-0.01005 0 0" rpy="0 0 0"/> -->
+  <!--     <inertia -->
+  <!--         ixx="0.0001" iyy="0.0001" izz="0.0002" -->
+  <!--         ixy="0" ixz="0" iyz="0"/> -->
+  <!--   </inertial> -->
+  <!-- </xacro:extra_module> -->
+  <!-- <!-\- rs_d435_link is the parrent of sensors' frame, identical to rs_d435_left_ir_frame  -\-> -->
+  <!-- <xacro:extra_module name = "rs_d435_link" parent = "rs_d435_unit" visible = "0" > -->
+  <!--   <origin xyz="-0.008 0.0175 0 " rpy="0 0 0"/> -->
+  <!--   <inertial> -->
+  <!--     <mass value = "0.0" /> -->
+  <!--     <origin xyz="0 0 0" rpy="0 0 0"/> -->
+  <!--     <inertia -->
+  <!--         ixx="0.0" ixy="0.0" ixz="0.0" -->
+  <!--         iyy="0.0" iyz="0.0" -->
+  <!--         izz="0.0"/> -->
+  <!--   </inertial> -->
+  <!-- </xacro:extra_module> -->
+  <!-- <transmission name="rs_d435_servo_joint_tran"> -->
+  <!--   <type>transmission_interface/SimpleTransmission</type> -->
+  <!--   <joint name="rs_d435_servo_joint"> -->
+  <!--     <hardwareInterface>hardware_interface/EffortJointInterface</hardwareInterface> -->
+  <!--   </joint> -->
+  <!--   <actuator name="rs_d435_servo_joint"> -->
+  <!--     <hardwareInterface>hardware_interface/EffortJointInterface</hardwareInterface> -->
+  <!--     <mechanicalReduction>1</mechanicalReduction> -->
+  <!--   </actuator> -->
+  <!-- </transmission> -->
+  <!-- <xacro:include filename="$(find hector_sensors_description)/urdf/hokuyo_utm30lx.urdf.xacro" /> -->
+  <!-- <xacro:hokuyo_utm30lx_model name="laser" parent="link3"> -->
+  <!--   <origin xyz="0.18 0.23 0.27" rpy="0 0 -1.57"/> -->
+  <!-- </xacro:hokuyo_utm30lx_model> -->
 </robot>
