Commit message: [Ninja] modified some structure of urdf

File: robots/ninja/robots/ninja.gazebo.xacro (robot description, xacro)
@@ -7,4 +7,72 @@
   <xacro:include filename="$(find aerial_robot_simulation)/xacro/spinal.gazebo.xacro" />
   <xacro:gazebo_spinal robot_name="$(arg robot_name)" mag_frame="fc" />
+  ##### dummy grasp links ####
+  <link name="dummy_arm">
+    <inertial>
+      <mass value = "0.01" />
+      <origin xyz="0.1 0 0" rpy="0 0 0"/>
+      <inertia
+          ixx="0.0011" ixy="0.0000" ixz="0.0001"
+          iyy="0.0011" iyz="0.0000" izz="0.0011"/>
+    </inertial>
+  </link>
+  <joint name="base_dummy_arm_joint" type="fixed">
+    <parent link="yaw_dock_link"/>
+    <child link="dummy_arm"/>
+    <origin xyz="0.0 0 0" rpy="0 0 0"/>
+    <axis xyz="1 0 0"/>
+  </joint>
+  <joint name="dummy_arm_palm_joint" type="revolute">
+    <parent link="dummy_arm"/>
+    <child link="dummy_palm"/>
+    <origin xyz="0.0 0 0" rpy="0 0 0"/>
+    <axis xyz="1 0 0"/>
+    <limit lower="0" upper="0" effort="0" velocity="0"/>
+    <dynamics damping="0.2" friction="0.02"/>
+  </joint>
+  <link name="dummy_palm">
+    <inertial>
+      <mass value = "0.001" />
+      <origin xyz="0 0 0" rpy="0 0 0"/>
+      <inertia
+          ixx="0.0001" ixy="0.0000" ixz="0.0000"
+          iyy="0.0001" iyz="0.0000" izz="0.0001"/>
+    </inertial>
+    <collision>
+      <origin xyz="0 0 0" rpy="0 0 0"/>
+      <geometry>
+        <box size="0.06 0.06 0.06"/>
+      </geometry>
+    </collision>
+  </link>
+  <joint name="dummy_palm_gripper_joint" type="revolute">
+    <parent link="dummy_palm"/>
+    <child link="dummy_gripper"/>
+    <origin xyz="0 0 0" rpy="0 0 0"/>
+    <axis xyz="1 0 0"/>
+    <limit lower="0" upper="0" effort="0" velocity="0"/>
+    <dynamics damping="0.2" friction="0.02"/>
+  </joint>
+  <link name="dummy_gripper">
+    <inertial>
+      <mass value = "0.001" />
+      <origin xyz="0.0 0 0" rpy="0 0 0"/>
+      <inertia
+          ixx="0.0001" ixy="0.0000" ixz="0.0000"
+          iyy="0.0001" iyz="0.0000" izz="0.0001"/>
+    </inertial>
+    <collision>
+      <origin xyz="0 0 0" rpy="0 0 0"/>
+      <geometry>
+        <box size="0.05 0.05 0.05"/>
+      </geometry>
+    </collision>
+    <visual>
+      <origin xyz="0 0 0" rpy="0.0 0 0"/>
+      <geometry>
+        <box size="0.05 0.05 0.05"/>
+      </geometry>
+    </visual>
+  </link>
   <!-- gazebo plugin for docking mech -->
   <gazebo>

File: robots/ninja/robots/ninja.urdf.xacro (robot description, xacro)
@@ -11,72 +11,4 @@
   <xacro:ninja_docking_mech_pitch/>
   <xacro:ninja_tail_link/>
-  ##### dummy grasp links ####
-  <link name="dummy_arm">
-    <inertial>
-      <mass value = "0.01" />
-      <origin xyz="0.1 0 0" rpy="0 0 0"/>
-      <inertia
-          ixx="0.0011" ixy="0.0000" ixz="0.0001"
-          iyy="0.0011" iyz="0.0000" izz="0.0011"/>
-    </inertial>
-  </link>
-  <joint name="base_dummy_arm_joint" type="fixed">
-    <parent link="yaw_dock_link"/>
-    <child link="dummy_arm"/>
-    <origin xyz="0.0 0 0" rpy="0 0 0"/>
-    <axis xyz="1 0 0"/>
-  </joint>
-  <joint name="dummy_arm_palm_joint" type="revolute">
-    <parent link="dummy_arm"/>
-    <child link="dummy_palm"/>
-    <origin xyz="0.0 0 0" rpy="0 0 0"/>
-    <axis xyz="1 0 0"/>
-    <limit lower="0" upper="0" effort="0" velocity="0"/>
-    <dynamics damping="0.2" friction="0.02"/>
-  </joint>
-  <link name="dummy_palm">
-    <inertial>
-      <mass value = "0.001" />
-      <origin xyz="0 0 0" rpy="0 0 0"/>
-      <inertia
-          ixx="0.0001" ixy="0.0000" ixz="0.0000"
-          iyy="0.0001" iyz="0.0000" izz="0.0001"/>
-    </inertial>
-    <collision>
-      <origin xyz="0 0 0" rpy="0 0 0"/>
-      <geometry>
-        <box size="0.06 0.06 0.06"/>
-      </geometry>
-    </collision>
-  </link>
-  <joint name="dummy_palm_gripper_joint" type="revolute">
-    <parent link="dummy_palm"/>
-    <child link="dummy_gripper"/>
-    <origin xyz="0 0 0" rpy="0 0 0"/>
-    <axis xyz="1 0 0"/>
-    <limit lower="0" upper="0" effort="0" velocity="0"/>
-    <dynamics damping="0.2" friction="0.02"/>
-  </joint>
-  <link name="dummy_gripper">
-    <inertial>
-      <mass value = "0.001" />
-      <origin xyz="0.0 0 0" rpy="0 0 0"/>
-      <inertia
-          ixx="0.0001" ixy="0.0000" ixz="0.0000"
-          iyy="0.0001" iyz="0.0000" izz="0.0001"/>
-    </inertial>
-    <collision>
-      <origin xyz="0 0 0" rpy="0 0 0"/>
-      <geometry>
-        <box size="0.05 0.05 0.05"/>
-      </geometry>
-    </collision>
-    <visual>
-      <origin xyz="0 0 0" rpy="0.0 0 0"/>
-      <geometry>
-        <box size="0.05 0.05 0.05"/>
-      </geometry>
-    </visual>
-  </link>
   ## dummy link for the contact point coordinate
   <link name="contact_point">

Commit message: [Ninja] update urdf to new version

File: robots/ninja/robots/ninja.gazebo.xacro (robot description, xacro)
@@ -10,9 +10,9 @@
   <link name="dummy_arm">
     <inertial>
-      <mass value = "0.01" />
+      <mass value = "0.001" />
       <origin xyz="0.1 0 0" rpy="0 0 0"/>
       <inertia
-          ixx="0.0011" ixy="0.0000" ixz="0.0001"
-          iyy="0.0011" iyz="0.0000" izz="0.0011"/>
+          ixx="0.00011" ixy="0.0000" ixz="0.00001"
+          iyy="0.00011" iyz="0.0000" izz="0.00011"/>
     </inertial>
   </link>
@@ -20,5 +20,5 @@
     <parent link="yaw_dock_link"/>
     <child link="dummy_arm"/>
-    <origin xyz="0.0 0 0" rpy="0 0 0"/>
+    <origin xyz="0.017 0 -0.025" rpy="0 0 0"/>
     <axis xyz="1 0 0"/>
   </joint>
@@ -42,5 +42,5 @@
       <origin xyz="0 0 0" rpy="0 0 0"/>
       <geometry>
-        <box size="0.06 0.06 0.06"/>
+        <box size="0.01 0.01 0.01"/>
       </geometry>
     </collision>
@@ -65,13 +65,13 @@
       <origin xyz="0 0 0" rpy="0 0 0"/>
       <geometry>
-        <box size="0.05 0.05 0.05"/>
+        <box size="0.01 0.01 0.01"/>
       </geometry>
     </collision>
-    <visual>
-      <origin xyz="0 0 0" rpy="0.0 0 0"/>
-      <geometry>
-        <box size="0.05 0.05 0.05"/>
-      </geometry>
-    </visual>
+    <!-- <visual> -->
+    <!--   <origin xyz="0 0 0" rpy="0.0 0 0"/> -->
+    <!--   <geometry> -->
+    <!--     <box size="0.05 0.05 0.05"/> -->
+    <!--   </geometry> -->
+    <!-- </visual> -->
   </link>
   <!-- gazebo plugin for docking mech -->

File: robots/ninja/robots/ninja.urdf.xacro (robot description, xacro)
@@ -10,5 +10,5 @@
   <xacro:ninja_docking_mech_yaw/>
   <xacro:ninja_docking_mech_pitch/>
-  <xacro:ninja_tail_link/>
+  <xacro:battery/>
   ## dummy link for the contact point coordinate
   <link name="contact_point">

File: robots/ninja/urdf/ninja.urdf.xacro (robot description, xacro)
@@ -23,20 +23,20 @@
     <link name="main_body">
       <inertial>
-        <origin xyz="0.2237 0.0050 0.0126" rpy="0 0 0"/>
-        <mass value="0.74"/>
-        <inertia
-            ixx="0.0011933" iyy="0.0157954" izz="0.0157066"
-            ixy="-0.0008036" ixz="0.0002441" iyz="0.0000132"/>
-      </inertial>
-      <visual>
-        <origin xyz="0 0 0" rpy="0 0 0"/>
-       <geometry>
-          <mesh filename="package://ninja/urdf/mesh/main_link.dae" scale="0.001 0.001 0.001"/>
+        <origin xyz="-0.08759215 -0.00288270 -0.01603775" rpy="0 0 0"/>
+        <mass value="1.23541002"/>
+        <inertia
+            ixx="0.00525317" iyy="0.04243332" izz="0.04586890"
+            ixy="0.00128324" ixz="0.00066518" iyz="-0.00004431"/>
+      </inertial>
+      <visual>
+        <origin xyz="0 0 0" rpy="0 0 0"/>
+        <geometry>
+          <mesh filename="package://ninja/urdf/mesh/mainbody.dae" scale="1 1 1"/>
         </geometry>
       </visual>
       <collision>
-        <origin xyz="0.2 0 0" rpy="0 0 0"/>
-        <geometry>
-          <box size="0.4 0.3 0.222"/>
+        <origin xyz="-0.12 0 -0.052" rpy="0 0 0"/>
+        <geometry>
+          <box size="0.30 0.3065 0.104"/>
         </geometry>
       </collision>
@@ -56,5 +56,5 @@
       <child link="fc"/>
       <parent link="main_body"/>
-      <origin rpy="0 0 0" xyz="0.33 0 0.067"/>
+      <origin rpy="0 0 0" xyz="-0.04695 0 0.0369"/>
       <axis xyz="0 0 1"/>
     </joint>
@@ -73,5 +73,5 @@
       <parent link="main_body"/>
       <child link="rotor_arm${child1}"/>
-      <origin rpy="0 0 ${pi/2}" xyz="0.329 0.065 0.018"/>
+      <origin rpy="0 0 ${pi/2}" xyz="0.008 0.02725 -0.0165"/>
       <axis xyz="0 0 1"/>
     </joint>
@@ -89,5 +89,5 @@
       <parent link="main_body"/>
       <child link="rotor_arm${child2}"/>
-      <origin rpy="0 0 ${-pi/2}" xyz="0.329 -0.065 0.018"/>
+      <origin rpy="0 0 ${-pi/2}" xyz="0.008 -0.02725 -0.0165"/>
       <axis xyz="0 0 1"/>
     </joint>
@@ -103,7 +103,7 @@
     </link>
     <joint name="base_arm_joint${child3}" type="fixed">
-      <parent link="tail_link"/>
+      <parent link="main_body"/>
       <child link="rotor_arm${child3}"/>
-      <origin rpy="0 0 0" xyz="0.076 0 0.0145"/>
+      <origin rpy="0 0 ${pi}" xyz="-0.0625 0 -0.0165"/>
       <axis xyz="0 0 1"/>
     </joint>
@@ -114,22 +114,22 @@
     <link name="yaw_dock_link">
       <inertial>
-        <origin xyz="0.007 0 -0.038" rpy="0 0 0"/>
-        <mass value="0.081"/>
-        <inertia
-            ixx="0.00022881" iyy="0.00022121" izz="0.0"
-            ixy="0.0" ixz="0.00002107" iyz="0.00000009"/>
-      </inertial>
-      <visual>
-        <origin xyz="0 0 0" rpy="0 0 0"/>
-        <geometry>
-          <mesh filename="package://ninja/urdf/mesh/head_link.dae" scale="0.001 0.001 0.001"/>
-        </geometry>
-      </visual>
-      <collision>
-        <origin xyz="0 0 0" rpy="0 0 0"/>
-        <geometry>
-          <box size="0.05 0.05 0.05"/>
-        </geometry>
-      </collision>
+        <origin xyz="0.05327516 -0.00002577 -0.02332311" rpy="0 0 0"/>
+        <mass value="0.21349624"/>
+        <inertia
+            ixx="0.00060141" iyy="0.00047550" izz="0.00067084"
+            ixy="0.00000015" ixz="-0.00001907" iyz="-0.00010342"/>
+      </inertial>
+      <visual>
+        <origin xyz="0 0 0" rpy="${pi/2} 0 0"/>
+        <geometry>
+          <mesh filename="package://ninja/urdf/mesh/female_dock_mech.dae" scale="1 1 1"/>
+        </geometry>
+      </visual>
+      <!-- <collision> -->
+      <!--   <origin xyz="0 0 0" rpy="0 0 0"/> -->
+      <!--   <geometry> -->
+      <!--     <box size="0.05 0.05 0.05"/> -->
+      <!--   </geometry> -->
+      <!-- </collision> -->
     </link>
     <xacro:damping_factor link="yaw_dock_link"/>
@@ -138,5 +138,5 @@
       <parent link="main_body"/>
       <child link="yaw_dock_link"/>
-      <origin rpy="0 0 0" xyz="0.41 0 0.018"/>
+      <origin rpy="0 0 0" xyz="0.1935 0 0.0085"/>
       <axis xyz="0 0 1"/>
       <dynamics damping="0.8" friction="0.0"/>
@@ -165,34 +165,6 @@
       <parent link="yaw_dock_link"/>
       <child link="yaw_connect_point"/>
-      <origin rpy="0 0 0" xyz="0.025 0 0"/>
-      <axis xyz="0 0 1"/>
-    </joint>
-  </xacro:macro>
-  <xacro:macro name="ninja_tail_link">
-    <!-- tail -->
-    <link name="tail_link">
-      <inertial>
-        <origin xyz="0.0356 -0.00294 0.00267" rpy="0 0 0"/>
-        <mass value="0.1212457"/>
-        <inertia
-            ixx="0.0000575" ixy="0.0000127" ixz="0.0000036"
-            iyy="0.0000946" iyz="0.0000010"
-            izz="0.0001120"/>
-      </inertial>
-      <visual>
-        <origin xyz="0 0 0" rpy="0 0 0"/>
-        <geometry>
-          <mesh filename="package://ninja/urdf/mesh/tail_link.dae" scale="1 1 1"/>
-        </geometry>
-      </visual>
-    </link>
-    <xacro:damping_factor link="tail_link"/>
-    <joint name="tail_joint" type="fixed">
-      <limit effort="6.6" lower="-1.57" upper="1.57" velocity="0.2"/>
-      <parent link="main_body"/>
-      <child link="tail_link"/>
-      <origin rpy="0 0 ${pi}" xyz="-0.02 0 0.018"/>
-      <axis xyz="0 1 0"/>
-      <dynamics damping="0.8" friction="0.0"/>
+      <origin rpy="0 0 0" xyz="0.037 0 -0.025"/>
+      <axis xyz="0 0 1"/>
     </joint>
   </xacro:macro>
@@ -220,9 +192,9 @@
     <link name="gimbal_link${self}">
       <inertial>
-       <origin xyz="0.074 0.044 0.0" rpy="0 0 0"/>
-        <mass value="0.124"/>
-        <inertia
-            ixx="0.00080131" iyy="0.00021920" izz="0.00099608"
-            ixy="0.00012557" ixz="0.00000026" iyz="-0.00000061"/>
+       <origin xyz="0.12 0.029 0.0000178" rpy="0 0 0"/>
+        <mass value="0.18778"/>
+        <inertia
+            ixx="0.00119072" iyy="0.00041760" izz="0.00154581"
+            ixy="0.00012643" ixz=" -0.00000030" iyz="-0.00000017"/>
       </inertial>
       <visual>
@@ -239,5 +211,5 @@
       <parent link="gimbal_link${self}"/>
       <child link="rotor_parent${self}"/>
-      <origin rpy="0 0 0" xyz="0.112 0.0877 0"/>
+      <origin rpy="0 0 0" xyz="0.162845 0.0735 0"/>
       <axis xyz="0 1 0"/>
     </joint>
@@ -292,5 +264,5 @@
       <parent link="rotor_parent${self}"/>
       <child link="thrust${self}"/>
-      <origin rpy="0 0 0" xyz="0 -0.088 0.02"/>
+      <origin rpy="0 0 0" xyz="0 -0.0835 0.025"/>
       <axis xyz="0 0 ${rotor_direction}"/>
     </joint>
@@ -310,20 +282,20 @@
     <link name="pitch_dock_link">
       <inertial>
-        <origin xyz="0.007 0 -0.038" rpy="0 0 0"/>
-        <mass value="0.081"/>
-        <inertia
-            ixx="0.00022881" iyy="0.00022121" izz="0.0"
-            ixy="0.0" ixz="0.00002107" iyz="0.00000009"/>
-      </inertial>
-      <visual>
-        <origin xyz="0 0 0" rpy="0 0 0"/>
-        <geometry>
-          <mesh filename="package://ninja/urdf/mesh/head_link.dae" scale="0.001 0.001 0.001"/>
+        <origin xyz="-0.07842366 0.02368423 -0.00011723" rpy="0 0 0"/>
+        <mass value="0.28876670"/>
+        <inertia
+            ixx="0.00036857" iyy="0.00079765" izz="0.00084052"
+            ixy="-0.00002766" ixz="-0.00000557" iyz="-0.00000287"/>
+      </inertial>
+      <visual>
+        <origin xyz="0 0 0" rpy="${pi} ${pi} 0"/>
+        <geometry>
+          <mesh filename="package://ninja/urdf/mesh/male_dock_mech.dae" scale="1 1 1"/>
         </geometry>
       </visual>
       <collision>
-        <origin xyz="0 0 0" rpy="0 0 0"/>
-        <geometry>
-          <box size="0.05 0.05 0.05"/>
+        <origin xyz="-${0.1531/2} 0.025 0" rpy="0 0 0"/>
+        <geometry>
+          <box size="0.1531 0.064 0.064"/>
         </geometry>
       </collision>
@@ -334,5 +306,5 @@
       <parent link="main_body"/>
       <child link="pitch_dock_link"/>
-      <origin rpy="0 0 0" xyz="-0.32 0 0.018"/>
+      <origin rpy="0 0 0" xyz="-0.434658 -0.025 -0.0165"/>
       <axis xyz="0 1 0"/>
       <dynamics damping="0.8" friction="0.0"/>
@@ -361,7 +333,53 @@
       <parent link="pitch_dock_link"/>
       <child link="pitch_connect_point"/>
-      <origin rpy="0 0 0" xyz="-0.025 0 0"/>
-      <axis xyz="0 0 1"/>
-    </joint>
+      <origin rpy="0 0 0" xyz="-0.1531 0.025 0"/>
+      <axis xyz="0 0 1"/>
+    </joint>
+  </xacro:macro>
+  <xacro:macro name="battery">
+    <joint name="battry_1_joint" type="fixed">
+      <parent link="main_body"/>
+      <child link="battery_1"/>
+      <origin rpy="-${pi/2} 0 ${pi}" xyz="-0.00891 0.0399 -0.069"/>
+      <axis xyz="0 0 0"/>
+    </joint>
+    <link name="battery_1">
+      <inertial>
+       <origin xyz="0.12 0.029 0.0000178" rpy="0 0 0"/>
+        <mass value="0.18778"/>
+        <inertia
+            ixx="0.00119072" iyy="0.00041760" izz="0.00154581"
+            ixy="0.00012643" ixz=" -0.00000030" iyz="-0.00000017"/>
+      </inertial>
+      <visual>
+        <origin xyz="0 0 0" rpy="0 0 0"/>
+        <geometry>
+          <mesh filename="package://ninja/urdf/mesh/battery.dae" scale="1 1 1"/>
+        </geometry>
+      </visual>
+    </link>
+    <xacro:damping_factor link="battery_1"/>
+    <joint name="battry_2_joint" type="fixed">
+      <parent link="main_body"/>
+      <child link="battery_2"/>
+      <origin rpy="${-pi/2} 0 0" xyz="-0.00891 -0.0399 -0.069"/>
+      <axis xyz="0 0 0"/>
+    </joint>
+    <link name="battery_2">
+      <inertial>
+       <origin xyz="0 0.0 00.01700000" rpy="0 0 0"/>
+        <mass value="0.40700000"/>
+        <inertia
+            ixx="0.00010170" iyy="0.00060259" izz="0.00062827"
+            ixy="0.000" ixz=" 0.000000" iyz="0.0000"/>
+      </inertial>
+      <visual>
+        <origin xyz="0 0 0" rpy="0 0 0"/>
+        <geometry>
+          <mesh filename="package://ninja/urdf/mesh/battery.dae" scale="1 1 1"/>
+        </geometry>
+      </visual>
+    </link>
+    <xacro:damping_factor link="battery_2"/>
   </xacro:macro>
 </robot>

Commit message: [Ninja][urdf] modified collision setting of docking mechanism

File: robots/ninja/robots/ninja.gazebo.xacro (robot description, xacro)
@@ -65,13 +65,7 @@
       <origin xyz="0 0 0" rpy="0 0 0"/>
       <geometry>
-        <box size="0.01 0.01 0.01"/>
+        <box size="0.04 0.01 0.01"/>
       </geometry>
     </collision>
-    <!-- <visual> -->
-    <!--   <origin xyz="0 0 0" rpy="0.0 0 0"/> -->
-    <!--   <geometry> -->
-    <!--     <box size="0.05 0.05 0.05"/> -->
-    <!--   </geometry> -->
-    <!-- </visual> -->
   </link>
   <!-- gazebo plugin for docking mech -->

Commit message: [Ninja][URDF] Modified docking_mech collision.

File: robots/ninja/robots/ninja.gazebo.xacro (robot description, xacro)
@@ -20,5 +20,5 @@
     <parent link="yaw_dock_link"/>
     <child link="dummy_arm"/>
-    <origin xyz="0.017 0 -0.025" rpy="0 0 0"/>
+    <origin xyz="0.132 0 -0.025" rpy="0 0 0"/>
     <axis xyz="1 0 0"/>
   </joint>
@@ -39,4 +39,10 @@
           iyy="0.0001" iyz="0.0000" izz="0.0001"/>
     </inertial>
+    <visual>
+      <origin xyz="0 0 0" rpy="0 0 0"/>
+      <geometry>
+        <box size="0.01 0.01 0.01"/>
+      </geometry>
+    </visual>
     <collision>
       <origin xyz="0 0 0" rpy="0 0 0"/>
@@ -62,4 +68,10 @@
           iyy="0.0001" iyz="0.0000" izz="0.0001"/>
     </inertial>
+    <visual>
+      <origin xyz="0 0 0" rpy="0 0 0"/>
+      <geometry>
+        <box size="0.04 0.01 0.01"/>
+      </geometry>
+    </visual>
     <collision>
       <origin xyz="0 0 0" rpy="0 0 0"/>

File: robots/ninja/urdf/ninja.urdf.xacro (robot description, xacro)
@@ -124,14 +124,14 @@
       <visual>
         <origin xyz="0 0 0" rpy="${pi/2} 0 0"/>
-        <geometry>
+       <geometry>
           <mesh filename="package://ninja/urdf/mesh/male_dock_mech.dae" scale="1 1 1"/>
         </geometry>
       </visual>
-      <collision>
-        <origin xyz="0 0.0 0" rpy="${pi/2} 0 0"/>
-        <geometry>
-          <box size="0.1531 0.064 0.064"/>
-        </geometry>
-      </collision>
+      <!-- <collision> -->
+      <!--   <origin xyz="0 0.0 0" rpy="${pi/2} 0 0"/> -->
+      <!--   <geometry> -->
+      <!--     <box size="0.1531 0.064 0.064"/> -->
+      <!--   </geometry> -->
+      <!-- </collision> -->
     </link>
     <xacro:damping_factor link="yaw_dock_link"/>
@@ -316,10 +316,10 @@
         </geometry>
       </visual>
-      <!-- <collision> -->
-      <!--   <origin xyz="0 0 0" rpy="0 0 0"/> -->
-      <!--   <geometry> -->
-      <!--     <box size="0.05 0.05 0.05"/> -->
-      <!--   </geometry> -->
-      <!-- </collision> -->
+      <collision>
+        <origin xyz="-0.02 0.025 0" rpy="0 0 0"/>
+        <geometry>
+          <box size="0.04 0.04 0.04"/>
+        </geometry>
+      </collision>
     </link>
     <xacro:damping_factor link="pitch_dock_link"/>

Commit message: [Ninja][URDF][Sim] Modified docking mech size in simulation.

File: robots/ninja/robots/ninja.gazebo.xacro (robot description, xacro)
@@ -20,5 +20,5 @@
     <parent link="yaw_dock_link"/>
     <child link="dummy_arm"/>
-    <origin xyz="0.132 0 -0.025" rpy="0 0 0"/>
+    <origin xyz="0.132 0 -0.030" rpy="0 0 0"/>
     <axis xyz="1 0 0"/>
   </joint>
@@ -71,5 +71,5 @@
       <origin xyz="0 0 0" rpy="0 0 0"/>
       <geometry>
-        <box size="0.04 0.01 0.01"/>
+        <box size="0.02 0.01 0.01"/>
       </geometry>
     </visual>
@@ -77,5 +77,5 @@
       <origin xyz="0 0 0" rpy="0 0 0"/>
       <geometry>
-        <box size="0.04 0.01 0.01"/>
+        <box size="0.02 0.01 0.01"/>
       </geometry>
     </collision>
