Commit message: [Ninja] install new docking mechanism to enable transformation

File: robots/ninja/robots/ninja.urdf.xacro (robot description, xacro)
@@ -8,25 +8,27 @@
   <xacro:ninja_gimbal_link self="2" rotor_direction="-1"/>
   <xacro:ninja_gimbal_link self="3" rotor_direction="-1"/>
-  <xacro:ninja_head_link/>
+  <xacro:ninja_docking_mech_yaw/>
+  <xacro:ninja_docking_mech_pitch/>
   <xacro:ninja_tail_link/>
   ##### dummy grasp links ####
-  <joint name="base_dummy_arm_joint" type="fixed">
-    <parent link="tail_link"/>
-    <child link="dummy_arm"/>
-    <origin xyz="0.3 0 0" rpy="0 0 ${pi}"/>
-  </joint>
   <link name="dummy_arm">
     <inertial>
       <mass value = "0.01" />
-      <origin xyz="0.05 0 0" rpy="0 0 0"/>
+      <origin xyz="0.1 0 0" rpy="0 0 0"/>
       <inertia
-          ixx="0.0001" ixy="0.0000" ixz="0.0000"
-          iyy="0.0001" iyz="0.0000" izz="0.0001"/>
+          ixx="0.0011" ixy="0.0000" ixz="0.0001"
+          iyy="0.0011" iyz="0.0000" izz="0.0011"/>
     </inertial>
   </link>
+  <joint name="base_dummy_arm_joint" type="fixed">
+    <parent link="yaw_dock_link"/>
+    <child link="dummy_arm"/>
+    <origin xyz="0.0 0 0" rpy="0 0 0"/>
+    <axis xyz="1 0 0"/>
+  </joint>
   <joint name="dummy_arm_palm_joint" type="revolute">
     <parent link="dummy_arm"/>
     <child link="dummy_palm"/>
-    <origin xyz="0.02 0 0" rpy="0 0 0"/>
+    <origin xyz="0.0 0 0" rpy="0 0 0"/>
     <axis xyz="1 0 0"/>
     <limit lower="0" upper="0" effort="0" velocity="0"/>
@@ -44,5 +46,5 @@
       <origin xyz="0 0 0" rpy="0 0 0"/>
       <geometry>
-        <box size="0.04 0.04 0.04"/>
+        <box size="0.06 0.06 0.06"/>
       </geometry>
     </collision>
@@ -67,5 +69,5 @@
       <origin xyz="0 0 0" rpy="0 0 0"/>
       <geometry>
-        <box size="0.04 0.04 0.04"/>
+        <box size="0.05 0.05 0.05"/>
       </geometry>
     </collision>
@@ -73,5 +75,5 @@
       <origin xyz="0 0 0" rpy="0.0 0 0"/>
       <geometry>
-        <box size="0.04 0.04 0.04"/>
+        <box size="0.05 0.05 0.05"/>
       </geometry>
     </visual>

File: robots/ninja/urdf/ninja.urdf.xacro (robot description, xacro)
@@ -110,7 +110,7 @@
    <xacro:friction self="base_link"/>
   </xacro:macro>
-  <xacro:macro name="ninja_head_link">
-    <!-- head -->
-    <link name="head_link">
+  <xacro:macro name="ninja_docking_mech_yaw">
+    <!-- yaw -->
+    <link name="yaw_dock_link">
       <inertial>
         <origin xyz="0.007 0 -0.038" rpy="0 0 0"/>
@@ -133,19 +133,19 @@
       </collision>
     </link>
-    <xacro:damping_factor link="head_link"/>
-    <joint name="head_joint" type="revolute">
-      <limit effort="6.6" lower="-3.14" upper="3.14" velocity="3.0"/>
-      <parent link="base_link"/>
-      <child link="head_link"/>
+    <xacro:damping_factor link="yaw_dock_link"/>
+    <joint name="yaw_dock_joint" type="revolute">
+      <limit effort="6.6" lower="-3.14" upper="3.14" velocity="0.5"/>
+      <parent link="base_link"/>
+      <child link="yaw_dock_link"/>
       <origin rpy="0 0 0" xyz="0.41 0 0.018"/>
       <axis xyz="0 0 1"/>
       <dynamics damping="0.8" friction="0.0"/>
     </joint>
-    <transmission name="head_joint_tran">
-      <type>transmission_interface/SimpleTransmission</type>
-      <joint name="head_joint">
-        <hardwareInterface>hardware_interface/EffortJointInterface</hardwareInterface>
-      </joint>
-      <actuator name="head_servo">
+    <transmission name="yaw_dockjoint_tran">
+      <type>transmission_interface/SimpleTransmission</type>
+      <joint name="yaw_dock_joint">
+        <hardwareInterface>hardware_interface/EffortJointInterface</hardwareInterface>
+      </joint>
+      <actuator name="yaw_dock_servo">
         <hardwareInterface>hardware_interface/EffortJointInterface</hardwareInterface>
         <mechanicalReduction>1</mechanicalReduction>
@@ -172,6 +172,6 @@
     </link>
     <xacro:damping_factor link="tail_link"/>
-    <joint name="tail_joint" type="revolute">
-      <limit effort="6.6" lower="-1.57" upper="1.57" velocity="3.0"/>
+    <joint name="tail_joint" type="fixed">
+      <limit effort="6.6" lower="-1.57" upper="1.57" velocity="0.5"/>
       <parent link="base_link"/>
       <child link="tail_link"/>
@@ -180,14 +180,4 @@
       <dynamics damping="0.8" friction="0.0"/>
     </joint>
-    <transmission name="tail_joint_tran">
-      <type>transmission_interface/SimpleTransmission</type>
-      <joint name="tail_joint">
-        <hardwareInterface>hardware_interface/EffortJointInterface</hardwareInterface>
-      </joint>
-      <actuator name="tail_servo">
-        <hardwareInterface>hardware_interface/EffortJointInterface</hardwareInterface>
-        <mechanicalReduction>1</mechanicalReduction>
-      </actuator>
-    </transmission>
   </xacro:macro>
   <xacro:macro name="ninja_gimbal_link" params="self rotor_direction">
@@ -300,3 +290,46 @@
     </transmission>
   </xacro:macro>
+  <xacro:macro name="ninja_docking_mech_pitch">
+    <!-- pitch -->
+    <link name="pitch_dock_link">
+      <inertial>
+        <origin xyz="0.007 0 -0.038" rpy="0 0 0"/>
+        <mass value="0.081"/>
+        <inertia
+            ixx="0.00022881" iyy="0.00022121" izz="0.0"
+            ixy="0.0" ixz="0.00002107" iyz="0.00000009"/>
+      </inertial>
+      <visual>
+        <origin xyz="0 0 0" rpy="0 0 0"/>
+        <geometry>
+          <mesh filename="package://ninja/urdf/mesh/head_link.dae" scale="0.001 0.001 0.001"/>
+        </geometry>
+      </visual>
+      <collision>
+        <origin xyz="0 0 0" rpy="0 0 0"/>
+        <geometry>
+          <box size="0.05 0.05 0.05"/>
+        </geometry>
+      </collision>
+    </link>
+    <xacro:damping_factor link="pitch_dock_link"/>
+    <joint name="pitch_dock_joint" type="revolute">
+      <limit effort="6.6" lower="-3.14" upper="3.14" velocity="0.5"/>
+      <parent link="tail_link"/>
+      <child link="pitch_dock_link"/>
+      <origin rpy="0 0 0" xyz="0.3 0 0"/>
+      <axis xyz="0 1 0"/>
+      <dynamics damping="0.8" friction="0.0"/>
+    </joint>
+    <transmission name="pitch_dockjoint_tran">
+      <type>transmission_interface/SimpleTransmission</type>
+      <joint name="pitch_dock_joint">
+        <hardwareInterface>hardware_interface/EffortJointInterface</hardwareInterface>
+      </joint>
+      <actuator name="pitch_dock_servo">
+        <hardwareInterface>hardware_interface/EffortJointInterface</hardwareInterface>
+        <mechanicalReduction>1</mechanicalReduction>
+      </actuator>
+    </transmission>
+  </xacro:macro>
 </robot>

Commit message: [Ninja] workaroud to develop new navigation method based on Forward Kinematics.

File: robots/ninja/robots/ninja.urdf.xacro (robot description, xacro)
@@ -23,5 +23,5 @@
   </link>
   <joint name="cp_base_joint" type="fixed">
-    <parent link="base_link"/>
+    <parent link="main_body"/>
     <child link="contact_point"/>
     <origin rpy="0 0 0" xyz="0.26 0 0"/>

File: robots/ninja/urdf/ninja.urdf.xacro (robot description, xacro)
@@ -16,10 +16,10 @@
     <joint name="root_joint" type="fixed">
       <parent link="root"/>
-      <child link="base_link"/>
+      <child link="main_body"/>
       <origin rpy="0 0 0" xyz="0 0 0"/>
       <axis xyz="0 0 1"/>
     </joint>
     ## link
-    <link name="base_link">
+    <link name="main_body">
       <inertial>
         <origin xyz="0.2237 0.0050 0.0126" rpy="0 0 0"/>
@@ -42,5 +42,5 @@
       </collision>
     </link>
-    <xacro:damping_factor link="base_link"/>
+    <xacro:damping_factor link="main_body"/>
     <link name="fc">
       <inertial>
@@ -55,5 +55,5 @@
     <joint name="fc_joint" type="fixed">
       <child link="fc"/>
-      <parent link="base_link"/>
+      <parent link="main_body"/>
       <origin rpy="0 0 0" xyz="0.33 0 0.067"/>
       <axis xyz="0 0 1"/>
@@ -71,5 +71,5 @@
     </link>
     <joint name="base_arm_joint${child1}" type="fixed">
-      <parent link="base_link"/>
+      <parent link="main_body"/>
       <child link="rotor_arm${child1}"/>
       <origin rpy="0 0 ${pi/2}" xyz="0.329 0.065 0.018"/>
@@ -87,5 +87,5 @@
     </link>
     <joint name="base_arm_joint${child2}" type="fixed">
-      <parent link="base_link"/>
+      <parent link="main_body"/>
       <child link="rotor_arm${child2}"/>
       <origin rpy="0 0 ${-pi/2}" xyz="0.329 -0.065 0.018"/>
@@ -108,5 +108,5 @@
       <axis xyz="0 0 1"/>
     </joint>
-   <xacro:friction self="base_link"/>
+   <xacro:friction self="main_body"/>
   </xacro:macro>
   <xacro:macro name="ninja_docking_mech_yaw">
@@ -136,5 +136,5 @@
     <joint name="yaw_dock_joint" type="revolute">
       <limit effort="6.6" lower="-3.14" upper="3.14" velocity="0.5"/>
-      <parent link="base_link"/>
+      <parent link="main_body"/>
       <child link="yaw_dock_link"/>
       <origin rpy="0 0 0" xyz="0.41 0 0.018"/>
@@ -152,4 +152,20 @@
       </actuator>
     </transmission>
+    <link name="yaw_connect_point">
+      <inertial>
+        <origin xyz="0 0 0" rpy="0 0 0"/>
+        <mass value="0.0001"/>
+        <inertia
+            ixx="0.000001" ixy="0.0" ixz="0.0"
+            iyy="0.000001" iyz="0.0"
+            izz="0.000001"/>
+      </inertial>
+    </link>
+    <joint name="yaw_connect_point_joint" type="fixed">
+      <parent link="yaw_dock_link"/>
+      <child link="yaw_connect_point"/>
+      <origin rpy="0 0 0" xyz="0.025 0 0"/>
+      <axis xyz="0 0 1"/>
+    </joint>
   </xacro:macro>
   <xacro:macro name="ninja_tail_link">
@@ -174,5 +190,5 @@
     <joint name="tail_joint" type="fixed">
       <limit effort="6.6" lower="-1.57" upper="1.57" velocity="0.5"/>
-      <parent link="base_link"/>
+      <parent link="main_body"/>
       <child link="tail_link"/>
       <origin rpy="0 0 ${pi}" xyz="-0.02 0 0.018"/>
@@ -316,5 +332,5 @@
     <joint name="pitch_dock_joint" type="revolute">
       <limit effort="6.6" lower="-3.14" upper="3.14" velocity="0.5"/>
-      <parent link="base_link"/>
+      <parent link="main_body"/>
       <child link="pitch_dock_link"/>
       <origin rpy="0 0 0" xyz="-0.32 0 0"/>
@@ -332,4 +348,20 @@
       </actuator>
     </transmission>
+    <link name="pitch_connect_point">
+      <inertial>
+        <origin xyz="0 0 0" rpy="0 0 0"/>
+        <mass value="0.0001"/>
+        <inertia
+            ixx="0.000001" ixy="0.0" ixz="0.0"
+            iyy="0.000001" iyz="0.0"
+            izz="0.000001"/>
+      </inertial>
+    </link>
+    <joint name="pitch_connect_point_joint" type="fixed">
+      <parent link="pitch_dock_link"/>
+      <child link="pitch_connect_point"/>
+      <origin rpy="0 0 0" xyz="-0.025 0 0"/>
+      <axis xyz="0 0 1"/>
+    </joint>
   </xacro:macro>
 </robot>

Commit message: [Ninja][Estimation] Workaround using onboard localization using Livox.

File: robots/ninja/robots/ninja.urdf.xacro (robot description, xacro)
@@ -10,5 +10,6 @@
   <xacro:ninja_docking_mech_yaw/>
   <xacro:ninja_docking_mech_pitch/>
-  <xacro:battery/>
+  <!-- <xacro:battery/> -->
+  <xacro:livox/>
   ## dummy link for the contact point coordinate
   <link name="contact_point">

File: robots/ninja/urdf/common.xacro (robot description, xacro)
@@ -20,3 +20,21 @@
     </gazebo>
   </xacro:macro>
+  <xacro:macro name="extra_module" params="name parent *origin *inertial visible:=0 model_url:=1 scale:=1">
+    <joint name="${parent}2${name}" type="fixed">
+      <parent link="${parent}"/>
+      <child link="${name}"/>
+      <xacro:insert_block name="origin" />
+    </joint>
+    <link name="${name}">
+      <xacro:insert_block name="inertial" />
+      <xacro:if value="${visible == 1}">
+        <visual>
+          <origin rpy="0 0 0" xyz="0 0 0"/>
+          <geometry>
+            <mesh filename="${model_url}" scale= "${scale} ${scale} ${scale}"/>
+          </geometry>
+        </visual>
+      </xacro:if>
+    </link>
+  </xacro:macro>
 </robot>

File: robots/ninja/urdf/ninja.urdf.xacro (robot description, xacro)
@@ -415,3 +415,16 @@
     <xacro:damping_factor link="battery_2"/>
   </xacro:macro>
+  <!-- livox mid360 -->
+  <xacro:macro name="livox">
+    <xacro:extra_module name = "lidar_imu" parent = "main_body" visible = "0" > <!-- should be IMU frame -->
+      <origin xyz="${-0.053 + 0.011} ${0.02329} ${0.046 + 0.025}" rpy="0 0 0"/>
+      <inertial>
+	<mass value = "0.262" />
+	<origin xyz="0 0 0.0038" rpy="0 0 0"/>
+	<inertia
+            ixx="0.000122" ixy="0.0" ixz="0.0"
+            iyy="0.000132" iyz="0.0" izz="0.000131"/>
+      </inertial>
+    </xacro:extra_module>
+  </xacro:macro>
 </robot>

Commit message: [Ninja][urdf] Add 1300mAh battery urdf

File: robots/ninja/robots/ninja.urdf.xacro (robot description, xacro)
@@ -10,5 +10,6 @@
   <xacro:ninja_docking_mech_yaw/>
   <xacro:ninja_docking_mech_pitch/>
-  <!-- <xacro:battery/> -->
+  <!-- <xacro:battery_3000mAh/> -->
+  <xacro:battery_1300mAh/>
   <xacro:livox/>
   ## dummy link for the contact point coordinate

File: robots/ninja/urdf/ninja.urdf.xacro (robot description, xacro)
@@ -367,5 +367,6 @@
     </joint>
   </xacro:macro>
-  <xacro:macro name="battery">
+  ## battery 3000mAh
+  <xacro:macro name="battery_3000mAh">
     <joint name="battry_1_joint" type="fixed">
       <parent link="main_body"/>
@@ -411,4 +412,59 @@
           <mesh filename="package://ninja/urdf/mesh/battery.dae" scale="1 1 1"/>
         </geometry>
+      </visual>
+    </link>
+    <xacro:damping_factor link="battery_2"/>
+  </xacro:macro>
+    ## battery 1300mAh
+  <xacro:macro name="battery_1300mAh">
+    <joint name="battry_1_joint" type="fixed">
+      <parent link="main_body"/>
+      <child link="battery_1"/>
+      <origin rpy="0 0 ${pi/2-0.977}" xyz="-0.10215 -0.07574 -0.04"/>
+      <axis xyz="0 0 0"/>
+    </joint>
+    <link name="battery_1">
+      <inertial>
+        <origin xyz="-0.00161235  0.0 -0.01674383" rpy="0 0 0"/>
+        <mass value="0.19795108"/>
+        <inertia
+            ixx = "0.00004618" ixy = "0.00000000" ixz = "0.00000000"
+            iyx = "0.00000000" iyy = "0.00010688" iyz = "0.00000000"
+            izx = "0.00000000" izy = "0.00000000" izz = "0.00011601"/>
+      </inertial>
+      <visual>
+        <origin xyz="0 0 0" rpy="0 0 0"/>
+        <geometry>
+          <box size="0.076 0.04 0.0335"/>
+        </geometry>
+        <material name="blue">
+          <color rgba="0.0 0.0 1.0 1.0"/>
+        </material>
+      </visual>
+    </link>
+    <xacro:damping_factor link="battery_1"/>
+    <joint name="battry_2_joint" type="fixed">
+      <parent link="main_body"/>
+      <child link="battery_2"/>
+      <origin rpy="0 0 -${pi/2-0.977}" xyz="-0.10215 0.07574 -0.04"/>
+      <axis xyz="0 0 0"/>
+    </joint>
+    <link name="battery_2">
+      <inertial>
+        <origin xyz="-0.00161235  0.0 -0.01674383" rpy="0 0 0"/>
+        <mass value="0.19795108"/>
+        <inertia
+            ixx = "0.00004618" ixy = "0.00000000" ixz = "0.00000000"
+            iyx = "0.00000000" iyy = "0.00010688" iyz = "0.00000000"
+            izx = "0.00000000" izy = "0.00000000" izz = "0.00011601"/>
+      </inertial>
+      <visual>
+        <origin xyz="0 0 0" rpy="0 0 0"/>
+        <geometry>
+          <box size="0.076 0.04 0.0335"/>
+        </geometry>
+        <material name="blue">
+          <color rgba="0.0 0.0 1.0 1.0"/>
+        </material>
       </visual>
     </link>
