Commit message: [NewPack][beetle_omni]: move URDF and related xml files

File: robots/beetle_omni/robots/beetle_art_omni.gazebo.xacro (robot description, xacro)
@@ -2,5 +2,5 @@
 <robot xmlns:xacro="http://www.ros.org/wiki/xacro" name="beetle-art-omni" >
   <!-- robot itself -->
-  <xacro:include filename="$(find beetle)/robots/beetle-art-omni.urdf.xacro" />
+  <xacro:include filename="$(find beetle_omni)/robots/beetle_art_omni.urdf.xacro" />
   <!-- gazebo plugin for default controller and sensors -->
   <xacro:include filename="$(find aerial_robot_simulation)/xacro/spinal.gazebo.xacro" />

File: robots/beetle_omni/urdf/beetle_art_omni.urdf.xacro (robot description, xacro)
@@ -16,5 +16,5 @@
         <origin xyz="0 0 0" rpy="0 0 0"/>
         <geometry>
-          <mesh filename="package://beetle/urdf/mesh/main_body_beetle_art_omni_w_guard.dae"/>
+          <mesh filename="package://beetle_omni/urdf/mesh/main_body_beetle_art_omni_w_guard.dae"/>
         </geometry>
       </visual>
@@ -94,5 +94,5 @@
         <origin xyz="0 0 0" rpy="0 0 0"/>
         <geometry>
-          <mesh filename="package://beetle/urdf/mesh/omni_rotor_module.dae"/>
+          <mesh filename="package://beetle_omni/urdf/mesh/omni_rotor_module.dae"/>
         </geometry>
       </visual>
