Commit message: chore: update mesh and xacro

File: robots/gimbalrotor/urdf/ynltilt/gimbalrotor.urdf.xacro (robot description, xacro)
@@ -23,9 +23,9 @@
     <link name="base_link">
       <inertial>
-        <origin xyz="0.00006 0.0001 0.00289" rpy="0 0 0"/>
-        <mass value="0.700"/>
-        <inertia
-            ixx="0.00726123" iyy="0.00729525" izz="0.01289551"
-            ixy="0.00000" ixz="0.0000" iyz="0.00000"/>
+        <origin xyz="0.001 0.00007 0.00275" rpy="0 0 0"/>
+        <mass value="0.958"/>
+        <inertia
+            ixx="0.01097918" iyy="0.01101753" izz="0.01953502"
+            ixy="-0.00000048" ixz="0.0000" iyz="0.00000"/>
       </inertial>
       <visual>
@@ -73,5 +73,5 @@
       <parent link="base_link"/>
       <child link="rotor_arm${child1}"/>
-      <origin rpy="0 0 ${pi*5.0/4.0}" xyz="-0.13711 -0.13711 0.04225"/>
+      <origin rpy="0 0 ${pi*5.0/4.0}" xyz="-0.13576 -0.13576 0.0495"/>
       <axis xyz="0 0 1"/>
     </joint>
@@ -89,5 +89,5 @@
       <parent link="base_link"/>
       <child link="rotor_arm${child2}"/>
-      <origin rpy="0 0 ${-pi/4.0}" xyz="0.13711 -0.13711 0.04225"/>
+      <origin rpy="0 0 ${-pi/4.0}" xyz="0.13576 -0.13576 0.0495"/>
       <axis xyz="0 0 1"/>
     </joint>
@@ -105,5 +105,5 @@
       <parent link="base_link"/>
       <child link="rotor_arm${child3}"/>
-      <origin rpy="0 0 ${pi/4.0}" xyz="0.13711 0.13711 0.04225"/>
+      <origin rpy="0 0 ${pi/4.0}" xyz="0.13576 0.13576 0.0495"/>
       <axis xyz="0 0 1"/>
     </joint>
@@ -121,5 +121,5 @@
       <parent link="base_link"/>
       <child link="rotor_arm${child4}"/>
-      <origin rpy="0 0 ${pi*3.0/4.0}" xyz="-0.13711 0.13711 0.04225"/>
+      <origin rpy="0 0 ${pi*3.0/4.0}" xyz="-0.13576 0.13576 0.0495"/>
       <axis xyz="0 0 1"/>
     </joint>

Commit message: feat: added lidar frame in ynltilt urdf

File: robots/gimbalrotor/urdf/ynltilt/gimbalrotor.urdf.xacro (robot description, xacro)
@@ -222,3 +222,31 @@
     </transmission>
   </xacro:macro>
+  <xacro:macro name="extra_module" params="name parent *origin *inertial visible:=0 model_url:=1 scale:=1">
+    <joint name="${parent}2${name}" type="fixed">
+      <parent link="${parent}"/>
+      <child link="${name}"/>
+      <xacro:insert_block name="origin" />
+    </joint>
+    <link name="${name}">
+      <xacro:insert_block name="inertial" />
+      <xacro:if value="${visible == 1}">
+        <visual>
+          <origin rpy="0 0 0" xyz="0 0 0"/>
+          <geometry>
+            <mesh filename="${model_url}" scale= "${scale} ${scale} ${scale}"/>
+          </geometry>
+        </visual>
+      </xacro:if>
+    </link>
+  </xacro:macro>
+  <xacro:extra_module name = "lidar_imu" parent = "base_link" visible = "0" > <!-- should be IMU frame -->
+    <origin xyz="${0.0} ${0.0} ${0.145}" rpy="0 0 ${pi/2.0}"/> <!-- TODO: the true pos -->
+    <inertial>
+      <mass value = "00" />
+      <origin xyz="0 0 0" rpy="0 0 0"/>
+      <inertia
+          ixx="0.0" ixy="0.0" ixz="0.0"
+          iyy="0.0" iyz="0.0" izz="0.0"/>
+    </inertial>
+  </xacro:extra_module>
 </robot>

Commit message: kamada temp

File: robots/gimbalrotor/urdf/ynltilt/gimbalrotor.urdf.xacro (robot description, xacro)
@@ -22,11 +22,21 @@
     ## link
     <link name="base_link">
-      <inertial>
-        <origin xyz="0.001 0.00007 0.00275" rpy="0 0 0"/>
-        <mass value="0.958"/>
-        <inertia
-            ixx="0.01097918" iyy="0.01101753" izz="0.01953502"
-            ixy="-0.00000048" ixz="0.0000" iyz="0.00000"/>
-      </inertial>
+    ## inertial of no attachment
+      <inertial>
+        <origin xyz="0.00009021 -0.00005299 0.04639014" rpy="0 0 0"/>
+        <mass value="1.16544411"/>
+        <inertia
+            ixx="0.01251517" iyy="0.01254829" izz="0.01920936"
+            ixy="-0.00000046" ixz="-0.00000278" iyz="-0.00001104"/>
+      </inertial>
+    ## inertial with pruning tools
+      <!-- <inertial> -->
+      <!--   <origin xyz="0.05514 0.00149 0.03734" rpy="0 0 0"/> -->
+      <!--   <mass value="1.38734"/> -->
+      <!--   <inertia -->
+      <!--       ixx="0.01325195352" ixy="0.00068117226" ixz="-0.00359026615" -->
+      <!--       iyx="0.00068117226" iyy="0.03735952771" iyz="-0.00013486816" -->
+      <!--       izx="-0.00359026615" izy="-0.00013486186" izz="0.04350508718"/> -->
+      <!-- </inertial> -->
       <visual>
         <origin xyz="0 0 -0.0" rpy="0 0 0"/>
@@ -131,10 +141,10 @@
     <link name="gimbal_link${self}">
       <inertial>
-        <origin xyz="0.018 0.00 0.00438" rpy="0 0 0"/>
-        <mass value="0.1095"/>
-        <inertia
-            ixx="0.00002989" ixy="0.0000"     ixz="-0.0000"
-                             iyy="0.00002848" iyz="0.00000"
-                                              izz="0.0002698"
+        <origin xyz="0.0412 0.00 0.0184" rpy="0 0 0"/>
+        <mass value="0.14"/>
+        <inertia
+            ixx="0.00003614" ixy="0.0000"     ixz="0.00000471"
+                             iyy="0.00004251" iyz="0.00000"
+                                              izz="0.00002946"
         />
       </inertial>
@@ -241,5 +251,5 @@
   </xacro:macro>
   <xacro:extra_module name = "lidar_imu" parent = "base_link" visible = "0" > <!-- should be IMU frame -->
-    <origin xyz="${0.0} ${0.0} ${0.145}" rpy="0 0 ${pi/2.0}"/> <!-- TODO: the true pos -->
+    <origin xyz="${0.0} ${0.0} ${0.145}" rpy="0 0 ${-pi/2.0}"/> <!-- TODO: the true pos -->
     <inertial>
       <mass value = "00" />

Commit message: Essam: commented the prunning system in urdf

File: robots/gimbalrotor/urdf/ynltilt/gimbalrotor.urdf.xacro (robot description, xacro)
@@ -22,6 +22,5 @@
     ## link
     <link name="base_link">
-    ## inertial of no attachment
-      <inertial>
+      <!-- <inertial>
         <origin xyz="0.00009021 -0.00005299 0.04639014" rpy="0 0 0"/>
         <mass value="1.16544411"/>
@@ -29,14 +28,13 @@
             ixx="0.01251517" iyy="0.01254829" izz="0.01920936"
             ixy="-0.00000046" ixz="-0.00000278" iyz="-0.00001104"/>
-      </inertial>
-    ## inertial with pruning tools
-      <!-- <inertial> -->
-      <!--   <origin xyz="0.05514 0.00149 0.03734" rpy="0 0 0"/> -->
-      <!--   <mass value="1.38734"/> -->
-      <!--   <inertia -->
-      <!--       ixx="0.01325195352" ixy="0.00068117226" ixz="-0.00359026615" -->
-      <!--       iyx="0.00068117226" iyy="0.03735952771" iyz="-0.00013486816" -->
-      <!--       izx="-0.00359026615" izy="-0.00013486186" izz="0.04350508718"/> -->
-      <!-- </inertial> -->
+      </inertial> -->
+      <inertial>
+        <origin xyz="0.05984 0.00138 0.03247" rpy="0 0 0"/>
+        <mass value="1.43147"/>
+        <inertia
+            ixx="0.01393149076" ixy="0.00059865083" ixz="-0.00538129912"
+            iyx="-0.00059865083" iyy="0.03783180404" iyz="-0.00018635030"
+            izx="-0.00538129912" izy="-0.00018635030" izz="0.04319444852"/>
+      </inertial>
       <visual>
         <origin xyz="0 0 -0.0" rpy="0 0 0"/>
