Commit message: [beetle-omni] change launch file and urdf to choose either fork or ball end effector.

File: robots/beetle_omni/urdf/beetle_art_omni.urdf.xacro (robot description, xacro)
@@ -7,14 +7,14 @@
     <link name="main_body">
       <inertial>
-        <origin xyz="0.00000845 0.00023419 0.02260762" rpy="0 0 0"/>
-        <mass value="2.3096"/>
-        <inertia
-            ixx="0.03155716" iyy="0.03084096" izz="0.03900553"
-            ixy="-0.00000599" ixz="0.00008620" iyz="0.00005548"/>
-      </inertial>
-      <visual>
-        <origin xyz="0 0 0" rpy="0 0 0"/>
-        <geometry>
-          <mesh filename="package://beetle_omni/urdf/mesh/main_body_beetle_art_omni_w_guard.dae"/>
+        <origin xyz="0.00000847 0.00023741 0.01491666" rpy="0 0 0"/>
+        <mass value="2.27739"/>
+        <inertia
+            ixx="0.02747704" iyy="0.02676088" izz="0.04047304"
+            ixy="-0.00000599" ixz="0.00009626" iyz="0.00006750"/>
+      </inertial>
+      <visual>
+        <origin xyz="0 0 0" rpy="0 0 0"/>
+        <geometry>
+          <mesh filename="package://beetle_omni/urdf/mesh/main_body_beetle_omni_w_guard.dae"/>
         </geometry>
       </visual>
@@ -174,3 +174,61 @@
   <xacro:beetle_thrust_link self="3" rotor_direction="1"/>
   <xacro:beetle_thrust_link self="4" rotor_direction="-1"/>
+<!-- ============ End Effector =============== -->
+  <!-- Define a parameter to choose the end effector type: "fork" or "ball" -->
+  <xacro:arg name="end_effector" default="fork" />
+  <xacro:property name="end_effector" value="$(arg end_effector)" />
+  <!-- Define the "end" link, which is positioned 0.3m along the Z axis relative to main_body -->
+  <link name="end">
+    <!-- Optionally, you can add inertial, collision, and visual information here -->
+  </link>
+  <joint name="main_body_to_end" type="fixed">
+    <parent link="main_body"/>
+    <child link="end"/>
+    <origin xyz="0 0 0.1725" rpy="0 0 0"/>
+  </joint>
+  <!-- Conditionally create the fork or ball link based on the parameter value -->
+  <xacro:if value="${end_effector == 'fork'}">
+    <!-- Define the fork link with mesh visualization -->
+    <link name="fork">
+      <inertial>
+        <origin xyz="0.00000000 0.06681059 -0.00005783" rpy="0 0 0"/>
+        <mass value="0.140"/>
+        <inertia
+                ixx="0.00040632" iyy="0.00053824" izz="0.00040617"
+                ixy="0.00000000" ixz="0.00000000" iyz="0.00000000"/>
+      </inertial>
+      <visual>
+        <geometry>
+          <mesh filename="package://beetle_omni/urdf/mesh/end_effector_fork.dae" scale="1 1 1"/>
+        </geometry>
+      </visual>
+    </link>
+    <joint name="end_to_fork" type="fixed">
+      <parent link="end"/>
+      <child link="fork"/>
+      <origin xyz="0 0 0" rpy="1.570796 0 -1.570796"/>
+    </joint>
+  </xacro:if>
+  <xacro:if value="${end_effector == 'ball'}">
+    <!-- Define the ball link with mesh visualization -->
+    <link name="ball">
+      <inertial>
+        <origin xyz="0.00000000 0.08052689 0.00000000" rpy="0 0 0"/>
+        <mass value="0.1030"/>
+        <inertia
+                ixx="0.00020646" iyy="0.00008167" izz="0.00020646"
+                ixy="0.00000000" ixz="0.00000000" iyz="0.00000000"/>
+      </inertial>
+      <visual>
+        <geometry>
+          <mesh filename="package://beetle_omni/urdf/mesh/end_effector_origin_ball.dae" scale="1 1 1"/>
+        </geometry>
+      </visual>
+    </link>
+    <joint name="end_to_ball" type="fixed">
+      <parent link="end"/>
+      <child link="ball"/>
+      <origin xyz="0 0 0" rpy="1.570796 0 0"/>
+    </joint>
+  </xacro:if>
 </robot>

Commit message: [beetle-omni] support brush end-effector now

File: robots/beetle_omni/urdf/beetle_art_omni.urdf.xacro (robot description, xacro)
@@ -232,3 +232,25 @@
     </joint>
   </xacro:if>
+  <xacro:if value="${end_effector == 'brush'}">
+    <!-- Define the brush link with mesh visualization -->
+    <link name="brush">
+      <inertial>
+        <origin xyz="0.00000000 0.06565796 -0.00001172" rpy="0 0 0"/>
+        <mass value="0.100"/>
+        <inertia
+                ixx="0.00019687" iyy="0.00013173" izz="0.00019689"
+                ixy="0.00000000" ixz="0.00000000" iyz="0.00000000"/>
+      </inertial>
+      <visual>
+        <geometry>
+          <mesh filename="package://beetle_omni/urdf/mesh/end_effector_brush.dae" scale="1 1 1"/>
+        </geometry>
+      </visual>
+    </link>
+    <joint name="end_to_brush" type="fixed">
+      <parent link="end"/>
+      <child link="brush"/>
+      <origin xyz="0 0 0" rpy="0 0 0"/>
+    </joint>
+  </xacro:if>
 </robot>

Commit message: [beetle-omni]: change the limitation of servo angle from +-180 deg to +-225deg according to hardware. change the max degree in traj. as well.

File: robots/beetle_omni/urdf/beetle_art_omni.urdf.xacro (robot description, xacro)
@@ -125,5 +125,5 @@
     #### gimbal joints ####
     <joint name="gimbal${self}" type="revolute">
-      <limit effort="6.6" lower="-3.141593" upper="3.141593" velocity="3.0"/>
+      <limit effort="6.6" lower="-3.926991" upper="3.926991" velocity="3.0"/>
       <parent link="rotor_arm${self}"/>
       <child link="gimbal_link${self}"/>

Commit message: [urdf]: update end_effector_ball 3d model

File: robots/beetle_omni/urdf/beetle_art_omni.urdf.xacro (robot description, xacro)
@@ -222,5 +222,5 @@
       <visual>
         <geometry>
-          <mesh filename="package://beetle_omni/urdf/mesh/end_effector_origin_ball.dae" scale="1 1 1"/>
+          <mesh filename="package://beetle_omni/urdf/mesh/end_effector_ball.dae" scale="1 1 1"/>
         </geometry>
       </visual>
@@ -229,5 +229,5 @@
       <parent link="end"/>
       <child link="ball"/>
-      <origin xyz="0 0 0" rpy="1.570796 0 0"/>
+      <origin xyz="0 0 0" rpy="0 0 1.570796"/>
     </joint>
   </xacro:if>
@@ -251,5 +251,5 @@
       <parent link="end"/>
       <child link="brush"/>
-      <origin xyz="0 0 0" rpy="0 0 0"/>
+      <origin xyz="0 0 0" rpy="0 0 1.570796"/>
     </joint>
   </xacro:if>

Commit message: [urdf]: add wrench_sensor and add one option called sensor_ball

File: robots/beetle_omni/urdf/beetle_art_omni.urdf.xacro (robot description, xacro)
@@ -232,4 +232,45 @@
     </joint>
   </xacro:if>
+  <xacro:if value="${end_effector == 'sensor_ball'}">
+    <!-- Define the ball link with mesh visualization -->
+    <link name="ball">
+      <inertial>
+        <origin xyz="0.00000000 0.08052689 0.00000000" rpy="0 0 0"/>
+        <mass value="0.1030"/>
+        <inertia
+                ixx="0.00020646" iyy="0.00008167" izz="0.00020646"
+                ixy="0.00000000" ixz="0.00000000" iyz="0.00000000"/>
+      </inertial>
+      <visual>
+        <geometry>
+          <mesh filename="package://beetle_omni/urdf/mesh/end_effector_ball.dae" scale="1 1 1"/>
+        </geometry>
+      </visual>
+    </link>
+    <link name="wrench_sensor">
+      <inertial>
+        <origin xyz="-0.00941317 0.00000000 -0.01652886" rpy="0 0 0"/>
+        <mass value="0.285"/>
+        <inertia
+                ixx="0.00008773" iyy="0.00012377" izz="0.00016573"
+                ixy="0.00000000" ixz="0.00000328" iyz="0.00000000"/>
+      </inertial>
+      <visual>
+        <geometry>
+          <mesh filename="package://beetle_omni/urdf/mesh/wrench_sensor_pfs055ya501u6.dae" scale="1 1 1"/>
+        </geometry>
+      </visual>
+    </link>
+    <joint name="end_to_sensor" type="fixed">
+      <parent link="end"/>
+      <child link="wrench_sensor"/>
+      <origin xyz="0 0 0.031" rpy="0 0 0"/>
+    </joint>
+    <joint name="sensor_to_ball" type="fixed">
+      <parent link="wrench_sensor"/>
+      <child link="ball"/>
+      <origin xyz="0 0 0" rpy="0 0 1.570796"/>
+    </joint>
+  </xacro:if>
   <xacro:if value="${end_effector == 'brush'}">
     <!-- Define the brush link with mesh visualization -->

Commit message: [beetle-omni][urdf]: rename coordinate frames; add one contact frame

File: robots/beetle_omni/urdf/beetle_art_omni.urdf.xacro (robot description, xacro)
@@ -174,20 +174,20 @@
   <xacro:beetle_thrust_link self="3" rotor_direction="1"/>
   <xacro:beetle_thrust_link self="4" rotor_direction="-1"/>
-<!-- ============ End Effector =============== -->
-  <!-- Define a parameter to choose the end effector type: "fork" or "ball" -->
-  <xacro:arg name="end_effector" default="fork" />
-  <xacro:property name="end_effector" value="$(arg end_effector)" />
-  <!-- Define the "end" link, which is positioned 0.3m along the Z axis relative to main_body -->
-  <link name="end">
-    <!-- Optionally, you can add inertial, collision, and visual information here -->
-  </link>
-  <joint name="main_body_to_end" type="fixed">
+  <!-- ============ End‑Effector (EE) =============== -->
+  <!-- Select EE type:  fork | ball | sensor_ball | brush -->
+  <xacro:arg name="end_effector" default="fork"/>
+  <xacro:property name="end_effector" value="$(arg end_effector)"/>
+  <!-- Fixed the flange that all tools attach to -->
+  <link name="ee_mount"/>
+  <joint name="body_to_ee_mount" type="fixed">
     <parent link="main_body"/>
-    <child link="end"/>
+    <child link="ee_mount"/>
     <origin xyz="0 0 0.1725" rpy="0 0 0"/>
   </joint>
-  <!-- Conditionally create the fork or ball link based on the parameter value -->
+  <!-- Tool‑agnostic contact frame (pose set inside each branch) -->
+  <link name="ee_contact"/>
+  <!-- ############# Fork tool ############# -->
   <xacro:if value="${end_effector == 'fork'}">
-    <!-- Define the fork link with mesh visualization -->
+    <!-- Tool geometry -->
     <link name="fork">
       <inertial>
@@ -204,12 +204,19 @@
       </visual>
     </link>
-    <joint name="end_to_fork" type="fixed">
-      <parent link="end"/>
+    <!-- Mount fork to the flange -->
+    <joint name="ee_mount_to_fork" type="fixed">
+      <parent link="ee_mount"/>
       <child link="fork"/>
       <origin xyz="0 0 0" rpy="1.570796 0 -1.570796"/>
     </joint>
+    <!-- Contact point for the fork tips -->
+    <joint name="fork_to_ee_contact" type="fixed">
+      <parent link="fork"/>
+      <child link="ee_contact"/>
+      <origin xyz="0.07 0 0" rpy="0 0 0"/>
+    </joint>
   </xacro:if>
+  <!-- ############# Ball tool ############# -->
   <xacro:if value="${end_effector == 'ball'}">
-    <!-- Define the ball link with mesh visualization -->
     <link name="ball">
       <inertial>
@@ -226,13 +233,41 @@
       </visual>
     </link>
-    <joint name="end_to_ball" type="fixed">
-      <parent link="end"/>
+    <joint name="ee_mount_to_ball" type="fixed">
+      <parent link="ee_mount"/>
       <child link="ball"/>
       <origin xyz="0 0 0" rpy="0 0 1.570796"/>
     </joint>
+    <!-- Contact point at the ball’s center -->
+    <joint name="ball_to_ee_contact" type="fixed">
+      <parent link="ball"/>
+      <child link="ee_contact"/>
+      <origin xyz="0 0 0.03" rpy="0 0 0"/>
+    </joint>
   </xacro:if>
+  <!-- ############# Sensor‑ball tool ############# -->
   <xacro:if value="${end_effector == 'sensor_ball'}">
-    <!-- Define the ball link with mesh visualization -->
+    <!-- Wrench sensor -->
+    <link name="wrench_sensor">
+      <inertial>
+        <origin xyz="-0.00941317 0.00000000 -0.01652886" rpy="0 0 0"/>
+        <mass value="0.285"/>
+        <inertia
+                ixx="0.00008773" iyy="0.00012377" izz="0.00016573"
+                ixy="0.00000000" ixz="0.00000328" iyz="0.00000000"/>
+      </inertial>
+      <visual>
+        <geometry>
+          <mesh filename="package://beetle_omni/urdf/mesh/wrench_sensor_pfs055ya501u6.dae" scale="1 1 1"/>
+        </geometry>
+      </visual>
+    </link>
+    <joint name="ee_mount_to_sensor" type="fixed">
+      <parent link="ee_mount"/>
+      <child link="wrench_sensor"/>
+      <origin xyz="0 0 0.031" rpy="0 0 0"/>
+    </joint>
+    <!-- Ball attached to the sensor -->
     <link name="ball">
+      <!-- (same as plain ball) -->
       <inertial>
         <origin xyz="0.00000000 0.08052689 0.00000000" rpy="0 0 0"/>
@@ -248,23 +283,4 @@
       </visual>
     </link>
-    <link name="wrench_sensor">
-      <inertial>
-        <origin xyz="-0.00941317 0.00000000 -0.01652886" rpy="0 0 0"/>
-        <mass value="0.285"/>
-        <inertia
-                ixx="0.00008773" iyy="0.00012377" izz="0.00016573"
-                ixy="0.00000000" ixz="0.00000328" iyz="0.00000000"/>
-      </inertial>
-      <visual>
-        <geometry>
-          <mesh filename="package://beetle_omni/urdf/mesh/wrench_sensor_pfs055ya501u6.dae" scale="1 1 1"/>
-        </geometry>
-      </visual>
-    </link>
-    <joint name="end_to_sensor" type="fixed">
-      <parent link="end"/>
-      <child link="wrench_sensor"/>
-      <origin xyz="0 0 0.031" rpy="0 0 0"/>
-    </joint>
     <joint name="sensor_to_ball" type="fixed">
       <parent link="wrench_sensor"/>
@@ -272,7 +288,13 @@
       <origin xyz="0 0 0" rpy="0 0 1.570796"/>
     </joint>
+    <!-- Contact point at ball tip -->
+    <joint name="ball_to_ee_contact" type="fixed">
+      <parent link="ball"/>
+      <child link="ee_contact"/>
+      <origin xyz="0 0 -0.03" rpy="0 0 0"/>
+    </joint>
   </xacro:if>
+  <!-- ############# Brush tool ############# -->
   <xacro:if value="${end_effector == 'brush'}">
-    <!-- Define the brush link with mesh visualization -->
     <link name="brush">
       <inertial>
@@ -289,9 +311,15 @@
       </visual>
     </link>
-    <joint name="end_to_brush" type="fixed">
-      <parent link="end"/>
+    <joint name="ee_mount_to_brush" type="fixed">
+      <parent link="ee_mount"/>
       <child link="brush"/>
       <origin xyz="0 0 0" rpy="0 0 1.570796"/>
     </joint>
+    <!-- Contact frame at the bristle tip -->
+    <joint name="brush_to_ee_contact" type="fixed">
+      <parent link="brush"/>
+      <child link="ee_contact"/>
+      <origin xyz="0 0 0.04" rpy="0 0 0"/>
+    </joint>
   </xacro:if>
 </robot>

Commit message: [beetle-omni][urdf]: update the info of all end-effectors; change the position of the contact frame to the correct one.

File: robots/beetle_omni/urdf/beetle_art_omni.urdf.xacro (robot description, xacro)
@@ -208,5 +208,5 @@
       <parent link="ee_mount"/>
       <child link="fork"/>
-      <origin xyz="0 0 0" rpy="1.570796 0 -1.570796"/>
+      <origin xyz="0 0 0" rpy="0 0 0"/>
     </joint>
     <!-- Contact point for the fork tips -->
@@ -214,5 +214,5 @@
       <parent link="fork"/>
       <child link="ee_contact"/>
-      <origin xyz="0.07 0 0" rpy="0 0 0"/>
+      <origin xyz="0 0 0.104" rpy="0 0 0"/>
     </joint>
   </xacro:if>
@@ -236,5 +236,5 @@
       <parent link="ee_mount"/>
       <child link="ball"/>
-      <origin xyz="0 0 0" rpy="0 0 1.570796"/>
+      <origin xyz="0 0 0" rpy="0 0 0"/>
     </joint>
     <!-- Contact point at the ball’s center -->
@@ -242,5 +242,5 @@
       <parent link="ball"/>
       <child link="ee_contact"/>
-      <origin xyz="0 0 0.03" rpy="0 0 0"/>
+      <origin xyz="0 0 0.11" rpy="0 0 0"/>
     </joint>
   </xacro:if>
@@ -286,5 +286,5 @@
       <parent link="wrench_sensor"/>
       <child link="ball"/>
-      <origin xyz="0 0 0" rpy="0 0 1.570796"/>
+      <origin xyz="0 0 0" rpy="0 0 0"/>
     </joint>
     <!-- Contact point at ball tip -->
@@ -292,5 +292,5 @@
       <parent link="ball"/>
       <child link="ee_contact"/>
-      <origin xyz="0 0 -0.03" rpy="0 0 0"/>
+      <origin xyz="0 0 0.11" rpy="0 0 0"/>
     </joint>
   </xacro:if>
@@ -314,5 +314,5 @@
       <parent link="ee_mount"/>
       <child link="brush"/>
-      <origin xyz="0 0 0" rpy="0 0 1.570796"/>
+      <origin xyz="0 0 0" rpy="0 0 0"/>
     </joint>
     <!-- Contact frame at the bristle tip -->
@@ -320,5 +320,5 @@
       <parent link="brush"/>
       <child link="ee_contact"/>
-      <origin xyz="0 0 0.04" rpy="0 0 0"/>
+      <origin xyz="0 0 0.144" rpy="0 0 0"/>
     </joint>
   </xacro:if>
