Commit message: [robots/amoeba/servo.yaml] add an actuator

File: robots/amoeba/urdf/amoeba.urdf.xacro (robot description, xacro)
@@ -46,34 +46,98 @@
       <parent link="main_body"/>
       <origin rpy="0 0 0" xyz="-0.0175 -0.0015 0.06347"/>  # should be aligned with the position of IMU
-      # changed from omni to amoeba
-    </joint>
-    ## rotor arm macro
-    <xacro:macro name="dummy_rotor_arm" params="id x y z yaw">
+      <!-- changed from omni to amoeba -->
+    </joint>
+    ## female rotor arm macro
+    <xacro:macro name="dummy_rotor_arm_f" params="id x y z yaw">
       ## dummy rotor arm link (virtual anchor point)
-      <link name="rotor_arm${id}">
+      <link name="rotor_arm_f_${id}">
         <inertial>
           <origin xyz="0 0 0" rpy="0 0 0"/>
-          <mass value="0.0001"/>
+          <mass value="0.0000001"/>
           <inertia
-              ixx="0.000001" ixy="0.0" ixz="0.0"
-              iyy="0.0001" iyz="0.0"
-              izz="0.0001"/>
+              ixx="0.0000001" ixy="0.0" ixz="0.0"
+              iyy="0.0000001" iyz="0.0"
+              izz="0.0000001"/>
         </inertial>
       </link>
       ## joint from main body to dummy rotor arm
-      <joint name="base_arm_joint${id}" type="fixed">
+      <joint name="base_arm_joint_f_${id}" type="fixed">
         <parent link="main_body"/>
-        <child link="rotor_arm${id}"/>
+        <child link="rotor_arm_f_${id}"/>
         <origin rpy="0 0 ${yaw}" xyz="${x} ${y} ${z}"/>
       </joint>
-      ## extendable arm link
+      ## female extendable arm link
       <link name="extendable${id}">
         <inertial>
-          <origin xyz="0.05 0 0" rpy="0 0 0"/>
-          <mass value="0.2"/>
+          <origin xyz="-0.0916461 -0.000000 -0.0011561" rpy="0 0 0"/>
+          <mass value="0.1110974"/>
           <inertia
-              ixx="0.001" ixy="0.0" ixz="0.0"
-              iyy="0.002" iyz="0.0"
-              izz="0.002"/>
+              ixx="0.0000192" ixy="0.0" ixz="0.0000010"
+              iyy="0.0013666" iyz="0.0"
+              izz="0.0013682"/>
+        </inertial>
+        <visual>
+          <origin xyz="0 0 0" rpy="0 0 0"/>
+          <geometry>
+            <mesh filename="package://amoeba/urdf/mesh/amoeba_arm_out.dae"/>
+          </geometry>
+        </visual>
+        <!-- the motor_case's limit pin is 87mm from the servo -->
+        <collision>
+          <origin xyz="-0.0435 0 0" rpy="0 0 0"/>
+          <geometry>
+            <box size="0.087 0.02 0.02"/>
+          </geometry>
+        </collision>
+      </link>
+      ## prismatic joint for extendable arm
+      <joint name="extendable_joint_f_${id}" type="prismatic">
+        <parent link="rotor_arm_f_${id}"/>
+        <child link="extendable${id}"/>
+        <origin rpy="0 0 0" xyz="0 0 0"/>
+        <axis xyz="1 0 0"/>
+        <limit effort="100.0" lower="-0.1" upper="0.1" velocity="0.1"/>
+        <dynamics damping="1.0" friction="0.1"/>
+      </joint>
+      ## transmission for extendable joint
+      <transmission name="extendable_tran_f_${id}">
+        <type>transmission_interface/SimpleTransmission</type>
+        <joint name="extendable_joint_f_${id}">
+          <hardwareInterface>hardware_interface/EffortJointInterface</hardwareInterface>
+        </joint>
+        <actuator name="extendable_actuator_f_${id}">
+          <hardwareInterface>hardware_interface/EffortJointInterface</hardwareInterface>
+          <mechanicalReduction>1</mechanicalReduction>
+        </actuator>
+      </transmission>
+    </xacro:macro>
+    ## male rotor arm macro
+    <xacro:macro name="dummy_rotor_arm_m" params="id x y z yaw">
+      ## dummy rotor arm link (virtual anchor point)
+      <link name="rotor_arm_m_${id}">
+        <inertial>
+          <origin xyz="0 0 0" rpy="0 0 0"/>
+          <mass value="0.0000001"/>
+          <inertia
+              ixx="0.0000001" ixy="0.0" ixz="0.0"
+              iyy="0.0000001" iyz="0.0"
+              izz="0.0000001"/>
+        </inertial>
+      </link>
+      ## joint from main body to dummy rotor arm
+      <joint name="base_arm_joint_m_${id}" type="fixed">
+        <parent link="main_body"/>
+        <child link="rotor_arm_m_${id}"/>
+        <origin rpy="0 0 ${yaw}" xyz="${x} ${y} ${z}"/>
+      </joint>
+      ## extendable arm link male
+      <link name="extendable${id}">
+        <inertial>
+          <origin xyz="-0.0930395 -0.000002 -0.0011329" rpy="0 0 0"/>
+          <mass value="0.1142974"/>
+          <inertia
+              ixx="0.0000195" ixy="0.0000001" ixz="0.0000011"
+              iyy="0.0014420" iyz="0.0"
+              izz="0.0014439"/>
         </inertial>
         <visual>
@@ -83,27 +147,28 @@
           </geometry>
         </visual>
+        <!-- the motor_case's limit pin is 87mm from the servo -->
         <collision>
-          <origin xyz="0.05 0 0" rpy="0 0 0"/>
+          <origin xyz="-0.0435 0 0" rpy="0 0 0"/>
           <geometry>
-            <box size="0.1 0.02 0.02"/>
+            <box size="0.087 0.02 0.02"/>
           </geometry>
         </collision>
       </link>
       ## prismatic joint for extendable arm
-      <joint name="extendable_joint${id}" type="prismatic">
-        <parent link="rotor_arm${id}"/>
+      <joint name="extendable_joint_m_${id}" type="prismatic">
+        <parent link="rotor_arm_m_${id}"/>
         <child link="extendable${id}"/>
         <origin rpy="0 0 0" xyz="0 0 0"/>
         <axis xyz="1 0 0"/>
-        <limit effort="100.0" lower="0.0" upper="0.2" velocity="0.1"/>
+        <limit effort="100.0" lower="-0.1" upper="0.1" velocity="0.1"/>
         <dynamics damping="1.0" friction="0.1"/>
       </joint>
       ## transmission for extendable joint
-      <transmission name="extendable_tran${id}">
+      <transmission name="extendable_tran_m_${id}">
         <type>transmission_interface/SimpleTransmission</type>
-        <joint name="extendable_joint${id}">
+        <joint name="extendable_joint_m_${id}">
           <hardwareInterface>hardware_interface/EffortJointInterface</hardwareInterface>
         </joint>
-        <actuator name="extendable_actuator${id}">
+        <actuator name="extendable_actuator_m_${id}">
           <hardwareInterface>hardware_interface/EffortJointInterface</hardwareInterface>
           <mechanicalReduction>1</mechanicalReduction>
@@ -112,8 +177,8 @@
     </xacro:macro>
     ## dummy rotor arms
-    <xacro:dummy_rotor_arm id = "${child1}" x = "0.198956" y="0.198956" z = "0.0154" yaw = "${pi*1.0/4.0}"/>
-    <xacro:dummy_rotor_arm id = "${child2}" x = "-0.198956" y="0.198956" z = "0.0154" yaw = "${pi*3.0/4.0}"/>
-    <xacro:dummy_rotor_arm id = "${child3}" x = "-0.198956" y="-0.198956" z = "0.0154" yaw = "${pi*5.0/4.0}"/>
-    <xacro:dummy_rotor_arm id = "${child4}" x = "0.198956" y="-0.198956" z = "0.0154" yaw = "${-pi*1.0/4.0}"/>
+    <xacro:dummy_rotor_arm_f id = "${child1}" x = " 0.198956" y=" 0.198956" z = "0.0154" yaw = "${pi*1.0/4.0}"/>
+    <xacro:dummy_rotor_arm_m id = "${child2}" x = "-0.198956" y=" 0.198956" z = "0.0154" yaw = "${pi*3.0/4.0}"/>
+    <xacro:dummy_rotor_arm_f id = "${child3}" x = "-0.198956" y="-0.198956" z = "0.0154" yaw = "${pi*5.0/4.0}"/>
+    <xacro:dummy_rotor_arm_m id = "${child4}" x = " 0.198956" y="-0.198956" z = "0.0154" yaw = "${-pi*1.0/4.0}"/>
     <xacro:friction self="main_body"/>
   </xacro:macro>
@@ -172,5 +237,5 @@
       <parent link="extendable${self}"/>
       <child link="gimbal_link${self}"/>
-      <origin rpy="0 0 0" xyz="0.1 0 0"/>
+      <origin rpy="0 0 0" xyz="0.0 0 0"/>
       <axis xyz="1 0 0"/>
       <dynamics damping="0.8" friction="0.0"/>

File: robots/amoeba_fix/urdf/beetle_art_omni.urdf.xacro (robot description, xacro)
@@ -133,5 +133,5 @@
       <dynamics damping="0.8" friction="0.0"/>
     </joint>
-    <transmission name="joint_tran${self}">3.141593
+    <transmission name="joint_tran${self}">
       <type>transmission_interface/SimpleTransmission</type>
       <joint name="gimbal${self}">

Commit message: [amoeba/urdf] fix gazebo bug

File: robots/amoeba/urdf/amoeba.urdf.xacro (robot description, xacro)
@@ -48,25 +48,24 @@
       <!-- changed from omni to amoeba -->
     </joint>
-    ## female rotor arm macro
-    <xacro:macro name="dummy_rotor_arm_f" params="id x y z yaw">
+      <xacro:macro name="dummy_rotor_arm" params="id x y z yaw">
       ## dummy rotor arm link (virtual anchor point)
-      <link name="rotor_arm_f_${id}">
+      <link name="rotor_arm${id}">
         <inertial>
           <origin xyz="0 0 0" rpy="0 0 0"/>
-          <mass value="0.0000001"/>
+          <mass value="0.00001"/>
           <inertia
-              ixx="0.0000001" ixy="0.0" ixz="0.0"
-              iyy="0.0000001" iyz="0.0"
-              izz="0.0000001"/>
+              ixx="0.000001" ixy="0.0" ixz="0.0"
+              iyy="0.000001" iyz="0.0"
+              izz="0.000001"/>
         </inertial>
       </link>
       ## joint from main body to dummy rotor arm
-      <joint name="base_arm_joint_f_${id}" type="fixed">
+      <joint name="base_arm_joint${id}" type="fixed">
         <parent link="main_body"/>
-        <child link="rotor_arm_f_${id}"/>
+        <child link="rotor_arm${id}"/>
         <origin rpy="0 0 ${yaw}" xyz="${x} ${y} ${z}"/>
       </joint>
       ## female extendable arm link
-      <link name="extendable${id}">
+      <link name="chain_link${id}">
         <inertial>
           <origin xyz="-0.0916461 -0.000000 -0.0011561" rpy="0 0 0"/>
@@ -77,10 +76,4 @@
               izz="0.0013682"/>
         </inertial>
-        <visual>
-          <origin xyz="0 0 0" rpy="0 0 0"/>
-          <geometry>
-            <mesh filename="package://amoeba/urdf/mesh/amoeba_arm_out.dae"/>
-          </geometry>
-        </visual>
         <!-- the motor_case's limit pin is 87mm from the servo -->
         <collision>
@@ -90,85 +83,28 @@
           </geometry>
         </collision>
+        <visual>
+          <origin xyz="0 0 0" rpy="0 0 0"/>
+          <geometry>
+            <mesh filename="package://amoeba/urdf/mesh/amoeba_arm_out.dae"/>
+          </geometry>
+        </visual>
       </link>
-      ## prismatic joint for extendable arm
-      <joint name="extendable_joint_f_${id}" type="prismatic">
-        <parent link="rotor_arm_f_${id}"/>
-        <child link="extendable${id}"/>
+      <xacro:damping_factor link="chain_link${id}"/>
+      ## prismatic joint for chain_link arm
+      <joint name="extendable_joint${id}" type="prismatic">
+        <limit effort="100.0" lower="-0.1" upper="0.1" velocity="0.01"/>
+        <parent link="rotor_arm${id}"/>
+        <child link="chain_link${id}"/>
         <origin rpy="0 0 0" xyz="0 0 0"/>
         <axis xyz="1 0 0"/>
-        <limit effort="100.0" lower="-0.1" upper="0.1" velocity="0.1"/>
         <dynamics damping="1.0" friction="0.1"/>
       </joint>
       ## transmission for extendable joint
-      <transmission name="extendable_tran_f_${id}">
+      <transmission name="extendable_tran${id}">
         <type>transmission_interface/SimpleTransmission</type>
-        <joint name="extendable_joint_f_${id}">
+        <joint name="extendable_joint${id}">
           <hardwareInterface>hardware_interface/EffortJointInterface</hardwareInterface>
         </joint>
-        <actuator name="extendable_actuator_f_${id}">
-          <hardwareInterface>hardware_interface/EffortJointInterface</hardwareInterface>
-          <mechanicalReduction>1</mechanicalReduction>
-        </actuator>
-      </transmission>
-    </xacro:macro>
-    ## male rotor arm macro
-    <xacro:macro name="dummy_rotor_arm_m" params="id x y z yaw">
-      ## dummy rotor arm link (virtual anchor point)
-      <link name="rotor_arm_m_${id}">
-        <inertial>
-          <origin xyz="0 0 0" rpy="0 0 0"/>
-          <mass value="0.0000001"/>
-          <inertia
-              ixx="0.0000001" ixy="0.0" ixz="0.0"
-              iyy="0.0000001" iyz="0.0"
-              izz="0.0000001"/>
-        </inertial>
-      </link>
-      ## joint from main body to dummy rotor arm
-      <joint name="base_arm_joint_m_${id}" type="fixed">
-        <parent link="main_body"/>
-        <child link="rotor_arm_m_${id}"/>
-        <origin rpy="0 0 ${yaw}" xyz="${x} ${y} ${z}"/>
-      </joint>
-      ## extendable arm link male
-      <link name="extendable${id}">
-        <inertial>
-          <origin xyz="-0.0930395 -0.000002 -0.0011329" rpy="0 0 0"/>
-          <mass value="0.1142974"/>
-          <inertia
-              ixx="0.0000195" ixy="0.0000001" ixz="0.0000011"
-              iyy="0.0014420" iyz="0.0"
-              izz="0.0014439"/>
-        </inertial>
-        <visual>
-          <origin xyz="0 0 0" rpy="0 0 0"/>
-          <geometry>
-            <mesh filename="package://amoeba/urdf/mesh/amoeba_arm_in.dae"/>
-          </geometry>
-        </visual>
-        <!-- the motor_case's limit pin is 87mm from the servo -->
-        <collision>
-          <origin xyz="-0.0435 0 0" rpy="0 0 0"/>
-          <geometry>
-            <box size="0.087 0.02 0.02"/>
-          </geometry>
-        </collision>
-      </link>
-      ## prismatic joint for extendable arm
-      <joint name="extendable_joint_m_${id}" type="prismatic">
-        <parent link="rotor_arm_m_${id}"/>
-        <child link="extendable${id}"/>
-        <origin rpy="0 0 0" xyz="0 0 0"/>
-        <axis xyz="1 0 0"/>
-        <limit effort="100.0" lower="-0.1" upper="0.1" velocity="0.1"/>
-        <dynamics damping="1.0" friction="0.1"/>
-      </joint>
-      ## transmission for extendable joint
-      <transmission name="extendable_tran_m_${id}">
-        <type>transmission_interface/SimpleTransmission</type>
-        <joint name="extendable_joint_m_${id}">
-          <hardwareInterface>hardware_interface/EffortJointInterface</hardwareInterface>
-        </joint>
-        <actuator name="extendable_actuator_m_${id}">
+        <actuator name="extendable_actuator${id}">
           <hardwareInterface>hardware_interface/EffortJointInterface</hardwareInterface>
           <mechanicalReduction>1</mechanicalReduction>
@@ -177,8 +113,8 @@
     </xacro:macro>
     ## dummy rotor arms
-    <xacro:dummy_rotor_arm_f id = "${child1}" x = " 0.198956" y=" 0.198956" z = "0.0154" yaw = "${pi*1.0/4.0}"/>
-    <xacro:dummy_rotor_arm_m id = "${child2}" x = "-0.198956" y=" 0.198956" z = "0.0154" yaw = "${pi*3.0/4.0}"/>
-    <xacro:dummy_rotor_arm_f id = "${child3}" x = "-0.198956" y="-0.198956" z = "0.0154" yaw = "${pi*5.0/4.0}"/>
-    <xacro:dummy_rotor_arm_m id = "${child4}" x = " 0.198956" y="-0.198956" z = "0.0154" yaw = "${-pi*1.0/4.0}"/>
+    <xacro:dummy_rotor_arm id = "${child1}" x = " 0.198956" y=" 0.198956" z = "0.0154" yaw = "${pi*1.0/4.0}"/>
+    <xacro:dummy_rotor_arm id = "${child2}" x = "-0.198956" y=" 0.198956" z = "0.0154" yaw = "${pi*3.0/4.0}"/>
+    <xacro:dummy_rotor_arm id = "${child3}" x = "-0.198956" y="-0.198956" z = "0.0154" yaw = "${pi*5.0/4.0}"/>
+    <xacro:dummy_rotor_arm id = "${child4}" x = " 0.198956" y="-0.198956" z = "0.0154" yaw = "${-pi*1.0/4.0}"/>
     <xacro:friction self="main_body"/>
   </xacro:macro>
@@ -235,5 +171,5 @@
     <joint name="gimbal${self}" type="revolute">
       <limit effort="6.6" lower="-3.926991" upper="3.926991" velocity="3.0"/>
-      <parent link="extendable${self}"/>
+      <parent link="chain_link${self}"/>
       <child link="gimbal_link${self}"/>
       <origin rpy="0 0 0" xyz="0.0 0 0"/>

Commit message: [robot/amoeba]update model to coarse one[planning] robot going circle and transform at same time

File: robots/amoeba/urdf/amoeba.urdf.xacro (robot description, xacro)
@@ -7,9 +7,9 @@
     <link name="main_body">
       <inertial>
-        <origin xyz="-0.0002494 0.0002857 0.0310495" rpy="0 0 0"/>
+        <origin xyz="-0.00034267 0.00045403 0.03598886" rpy="0 0 0"/>
         <mass value="1.9660957"/>
         <inertia
-            ixx="0.018188022" iyy="0.018172157" izz="0.022508471"
-            ixy="-0.00006050" ixz="0.00012987" iyz="0.00007583"/>
+            ixx="0.00874381" iyy="0.00872797" izz="0.00460590"
+            ixy="0.00000741" ixz="0.00013082" iyz="0.00007583"/>
       </inertial>
       <visual>
@@ -20,7 +20,7 @@
       </visual>
       <collision>
-        <origin xyz="0 0 0.0385" rpy="0 0 0"/>
-        <geometry>
-          <box size="0.35 0.35 0.275"/>
+        <origin xyz="0 0 0.0385" rpy="0 0 ${pi/4}"/>
+        <geometry>
+          <box size="0.12 0.12 0.275"/>
         </geometry>
       </collision>

Commit message: [robot/amoeba] change base_link mass

File: robots/amoeba/urdf/amoeba.urdf.xacro (robot description, xacro)
@@ -8,5 +8,5 @@
       <inertial>
         <origin xyz="-0.00034267 0.00045403 0.03598886" rpy="0 0 0"/>
-        <mass value="1.9660957"/>
+        <mass value="1.23731225"/>
         <inertia
             ixx="0.00874381" iyy="0.00872797" izz="0.00460590"

Commit message: [amoeba/urdf] update mass with wire [amoeba_fix/config] show mass

File: robots/amoeba/urdf/amoeba.urdf.xacro (robot description, xacro)
@@ -7,8 +7,8 @@
     <link name="main_body">
       <inertial>
-        <origin xyz="-0.00034267 0.00045403 0.03598886" rpy="0 0 0"/>
-        <mass value="1.23731225"/>
-        <inertia
-            ixx="0.00874381" iyy="0.00872797" izz="0.00460590"
+        <origin xyz="-0.00027907 0.00036976 0.03599093" rpy="0 0 0"/>
+        <mass value="1.51931225"/>
+        <inertia
+            ixx="0.00913984" iyy="0.00912399" izz="0.00466230"
             ixy="0.00000741" ixz="0.00013082" iyz="0.00007583"/>
       </inertial>

Commit message: [robot/amoeba] add percher

File: robots/amoeba/urdf/amoeba.urdf.xacro (robot description, xacro)
@@ -123,4 +123,34 @@
         </actuator>
       </transmission>
+      ## percher link (only for chain_link 1 and 3)
+      <xacro:if value="${id == 1 or id == 3}">
+        <link name="percher${id}">
+          <inertial>
+            <origin xyz="0.07203636 -0.00070189 0.00924944" rpy="0 0 0"/>
+            <mass value="0.23213"/>
+            <inertia
+                ixx="0.00093823" ixy="-0.00002851" ixz="0.00044947"
+                iyy="0.00455027" iyz="-0.00000728"
+                izz="0.00451444"/>
+          </inertial>
+          <visual>
+            <origin xyz="0 0 0" rpy="0 0 0"/>
+            <geometry>
+              <mesh filename="package://amoeba/urdf/mesh/percher.dae"/>
+            </geometry>
+          </visual>
+          <collision>
+            <origin xyz="0.2 0 0.1" rpy="0 0 0"/>
+            <geometry>
+              <box size="0.1 0.35 0.05"/>
+            </geometry>
+          </collision>
+        </link>
+        <joint name="percher_install${id}" type="fixed">
+          <parent link="chain_link${id}"/>
+          <child link="percher${id}"/>
+          <origin rpy="0 0 0" xyz="0 0 0"/>
+        </joint>
+      </xacro:if>
     </xacro:macro>
     ## dummy rotor arms

Commit message: [robot/amoeba] change to sidemount battery 2.46kg base

File: robots/amoeba/urdf/amoeba.urdf.xacro (robot description, xacro)
@@ -7,9 +7,9 @@
     <link name="main_body">
       <inertial>
-        <origin xyz="-0.00027907 0.00036976 0.03599093" rpy="0 0 0"/>
-        <mass value="1.51931225"/>
-        <inertia
-            ixx="0.00913984" iyy="0.00912399" izz="0.00466230"
-            ixy="0.00000741" ixz="0.00013082" iyz="0.00007583"/>
+        <origin xyz="-0.00017970 0.00022844 0.06412770" rpy="0 0 0"/>
+        <mass value="2.45965596"/>
+        <inertia
+            ixx="0.02794065" iyy="0.02190286" izz="0.01108005"
+            ixy="0.00000780" ixz="0.00014208" iyz="0.00007584"/>
       </inertial>
       <visual>

Commit message: [robot] use 1300ma 6s, 1.95kg

File: robots/amoeba/urdf/amoeba.urdf.xacro (robot description, xacro)
@@ -7,9 +7,9 @@
     <link name="main_body">
       <inertial>
-        <origin xyz="-0.00017970 0.00022844 0.06412770" rpy="0 0 0"/>
-        <mass value="2.45965596"/>
-        <inertia
-            ixx="0.02794065" iyy="0.02190286" izz="0.01108005"
-            ixy="0.00000780" ixz="0.00014208" iyz="0.00007584"/>
+        <origin xyz="-0.00027191 0.00028756 0.04712130" rpy="0 0 0"/>
+        <mass value="1.95374926"/>
+        <inertia
+            ixx="0.01533519" iyy="0.01278624" izz="0.00741448"
+            ixy="0.00000757" ixz="0.00013253" iyz="0.00007584"/>
       </inertial>
       <visual>

Commit message: [robot/amoeba]cancel battery try take off

File: robots/amoeba/urdf/amoeba.urdf.xacro (robot description, xacro)
@@ -7,9 +7,9 @@
     <link name="main_body">
       <inertial>
-        <origin xyz="-0.00027191 0.00028756 0.04712130" rpy="0 0 0"/>
-        <mass value="1.95374926"/>
-        <inertia
-            ixx="0.01533519" iyy="0.01278624" izz="0.00741448"
-            ixy="0.00000757" ixz="0.00013253" iyz="0.00007584"/>
+        <origin xyz="-0.00027907 0.00036976 0.03599093" rpy="0 0 0"/>
+        <mass value="1.51931225"/>
+        <inertia
+            ixx="0.00913984" iyy="0.00912399" izz="0.00466230"
+            ixy="0.00000741" ixz="0.00013082" iyz="0.00007583"/>
       </inertial>
       <visual>
