Commit message: [Ninja][URDF] change the parent link of pitch_docking_mechanism to baselink

File: robots/ninja/urdf/ninja.urdf.xacro (robot description, xacro)
@@ -316,7 +316,7 @@
     <joint name="pitch_dock_joint" type="revolute">
       <limit effort="6.6" lower="-3.14" upper="3.14" velocity="0.5"/>
-      <parent link="tail_link"/>
+      <parent link="base_link"/>
       <child link="pitch_dock_link"/>
-      <origin rpy="0 0 0" xyz="0.3 0 0"/>
+      <origin rpy="0 0 0" xyz="-0.32 0 0"/>
       <axis xyz="0 1 0"/>
       <dynamics damping="0.8" friction="0.0"/>

Commit message: [Ninja][Navigation] workaournd implimentation of transforming feature

File: robots/ninja/urdf/ninja.urdf.xacro (robot description, xacro)
@@ -135,5 +135,5 @@
     <xacro:damping_factor link="yaw_dock_link"/>
     <joint name="yaw_dock_joint" type="revolute">
-      <limit effort="6.6" lower="-3.14" upper="3.14" velocity="0.5"/>
+      <limit effort="6.6" lower="-3.14" upper="3.14" velocity="0.2"/>
       <parent link="main_body"/>
       <child link="yaw_dock_link"/>
@@ -189,5 +189,5 @@
     <xacro:damping_factor link="tail_link"/>
     <joint name="tail_joint" type="fixed">
-      <limit effort="6.6" lower="-1.57" upper="1.57" velocity="0.5"/>
+      <limit effort="6.6" lower="-1.57" upper="1.57" velocity="0.2"/>
       <parent link="main_body"/>
       <child link="tail_link"/>
@@ -331,8 +331,8 @@
     <xacro:damping_factor link="pitch_dock_link"/>
     <joint name="pitch_dock_joint" type="revolute">
-      <limit effort="6.6" lower="-3.14" upper="3.14" velocity="0.5"/>
+      <limit effort="6.6" lower="-3.14" upper="3.14" velocity="0.2"/>
       <parent link="main_body"/>
       <child link="pitch_dock_link"/>
-      <origin rpy="0 0 0" xyz="-0.32 0 0"/>
+      <origin rpy="0 0 0" xyz="-0.32 0 0.018"/>
       <axis xyz="0 1 0"/>
       <dynamics damping="0.8" friction="0.0"/>

Commit message: [Ninja][model] modified urdf model to correct version

File: robots/ninja/urdf/ninja.urdf.xacro (robot description, xacro)
@@ -211,5 +211,5 @@
       <parent link="gimbal_link${self}"/>
       <child link="rotor_parent${self}"/>
-      <origin rpy="0 0 0" xyz="0.162845 0.0735 0"/>
+      <origin rpy="0 0 0" xyz="0.162845 0.09285 0"/>
       <axis xyz="0 1 0"/>
     </joint>
@@ -235,7 +235,7 @@
       </inertial>
       <visual>
-        <origin xyz="0 0 0" rpy="0 0 ${-pi/2}"/>
-        <geometry>
-          <mesh filename="package://ninja/urdf/mesh/rotor_link_CW.dae" scale="1 1 1"/>
+        <origin xyz="0 -0.09285 0" rpy="0 0 ${pi}"/>
+        <geometry>
+          <mesh filename="package://ninja/urdf/mesh/5inch_edf.dae" scale="1 1 1"/>
         </geometry>
       </visual>
@@ -264,5 +264,5 @@
       <parent link="rotor_parent${self}"/>
       <child link="thrust${self}"/>
-      <origin rpy="0 0 0" xyz="0 -0.0835 0.025"/>
+      <origin rpy="0 0 0" xyz="0 -0.09285 0.025"/>
       <axis xyz="0 0 ${rotor_direction}"/>
     </joint>

Commit message: [Ninja][URDF] modfied inertial value

File: robots/ninja/urdf/ninja.urdf.xacro (robot description, xacro)
@@ -23,11 +23,12 @@
     <link name="main_body">
       <inertial>
-        <origin xyz="-0.08759215 -0.00288270 -0.01603775" rpy="0 0 0"/>
-        <mass value="1.23541002"/>
-        <inertia
-            ixx="0.00525317" iyy="0.04243332" izz="0.04586890"
-            ixy="0.00128324" ixz="0.00066518" iyz="-0.00004431"/>
-      </inertial>
-      <visual>
+        <origin xyz="-0.08989427 -0.00260694 -0.01604721" rpy="0 0 0"/>
+        <mass value="1.32590383"/>
+        <inertia
+            ixx = "0.00565938" ixy = "0.00127382" ixz = "0.00065740"
+            iyx = "0.00127382" iyy = "0.04578657" iyz = "-0.00004725"
+            izx = "0.00065q740" izy = "-0.00004725" izz = "0.04949468"/>
+      </inertial>
+        <visual>
         <origin xyz="0 0 0" rpy="0 0 0"/>
         <geometry>
@@ -114,9 +115,10 @@
     <link name="yaw_dock_link">
       <inertial>
-        <origin xyz="0.05327516 -0.00002577 -0.02332311" rpy="0 0 0"/>
-        <mass value="0.21349624"/>
-        <inertia
-            ixx="0.00060141" iyy="0.00047550" izz="0.00067084"
-            ixy="0.00000015" ixz="-0.00001907" iyz="-0.00010342"/>
+        <origin xyz="0.06781112 -0.00002493 -0.02345044" rpy="0 0 0"/>
+        <mass value="0.21443253"/>
+        <inertia
+            ixx = "0.00093162" ixy = "0.00000022" ixz = "-0.00002253"
+            iyx = "0.00000022" iyy = "0.00071768" iyz = "-0.00010593"
+            izx = "-0.00002253" izy = "-0.00010593" izz = "0.00091594"/>
       </inertial>
       <visual>
@@ -192,9 +194,10 @@
     <link name="gimbal_link${self}">
       <inertial>
-       <origin xyz="0.12 0.029 0.0000178" rpy="0 0 0"/>
-        <mass value="0.18778"/>
-        <inertia
-            ixx="0.00119072" iyy="0.00041760" izz="0.00154581"
-            ixy="0.00012643" ixz=" -0.00000030" iyz="-0.00000017"/>
+       <origin xyz="0.12245044 0.03129270 0.00001719" rpy="0 0 0"/>
+        <mass value="0.19445396"/>
+        <inertia
+            ixx = "0.00119253" ixy = "0.00015756" ixz = "-0.00000029"
+            iyx = "0.00015756" iyy = "0.00043864" iyz = "-0.00000018"
+            izx = "-0.00000029" izy = "-0.00000018" izz = "0.00156562"/>
       </inertial>
       <visual>
@@ -282,9 +285,10 @@
     <link name="pitch_dock_link">
       <inertial>
-        <origin xyz="-0.07842366 0.02368423 -0.00011723" rpy="0 0 0"/>
-        <mass value="0.28876670"/>
-        <inertia
-            ixx="0.00036857" iyy="0.00079765" izz="0.00084052"
-            ixy="-0.00002766" ixz="-0.00000557" iyz="-0.00000287"/>
+        <origin xyz="-0.06961517 0.02389743 -0.00688546" rpy="0 0 0"/>
+        <mass value="0.30174800"/>
+        <inertia
+            ixx = "0.00119253" ixy = "0.00015756" ixz = "-0.00000029"
+            iyx = "0.00015756" iyy = "0.00043864" iyz = "-0.00000018"
+            izx = "-0.00000029" izy = "-0.00000018" izz = "0.00156562"/>
       </inertial>
       <visual>

Commit message: [Ninja][URDF] modified inertial parameters of real-machine

File: robots/ninja/urdf/ninja.urdf.xacro (robot description, xacro)
@@ -28,7 +28,7 @@
             ixx = "0.00565938" ixy = "0.00127382" ixz = "0.00065740"
             iyx = "0.00127382" iyy = "0.04578657" iyz = "-0.00004725"
-            izx = "0.00065q740" izy = "-0.00004725" izz = "0.04949468"/>
-      </inertial>
-        <visual>
+            izx = "0.00065740" izy = "-0.00004725" izz = "0.04949468"/>
+      </inertial>
+      <visual>
         <origin xyz="0 0 0" rpy="0 0 0"/>
         <geometry>
@@ -288,7 +288,7 @@
         <mass value="0.30174800"/>
         <inertia
-            ixx = "0.00119253" ixy = "0.00015756" ixz = "-0.00000029"
-            iyx = "0.00015756" iyy = "0.00043864" iyz = "-0.00000018"
-            izx = "-0.00000029" izy = "-0.00000018" izz = "0.00156562"/>
+            ixx = "0.00053278" ixy = "-0.00002216" ixz = "0.00003995"
+            iyx = "-0.00002216" iyy = "0.00065740" iyz = "-0.00000804"
+            izx = "0.00003995" izy = "-0.00000804" izz = "0.00073599"/>
       </inertial>
       <visual>

Commit message: [Ninja][URDF] correct battery inertial

File: robots/ninja/urdf/ninja.urdf.xacro (robot description, xacro)
@@ -350,9 +350,9 @@
     <link name="battery_1">
       <inertial>
-       <origin xyz="0.12 0.029 0.0000178" rpy="0 0 0"/>
-        <mass value="0.18778"/>
-        <inertia
-            ixx="0.00119072" iyy="0.00041760" izz="0.00154581"
-            ixy="0.00012643" ixz=" -0.00000030" iyz="-0.00000017"/>
+        <origin xyz="0 0.0 00.01700000" rpy="0 0 0"/>
+        <mass value="0.40700000"/>
+        <inertia
+            ixx="0.00010170" iyy="0.00060259" izz="0.00062827"
+            ixy="0.000" ixz=" 0.000000" iyz="0.0000"/>
       </inertial>
       <visual>
@@ -372,5 +372,5 @@
     <link name="battery_2">
       <inertial>
-       <origin xyz="0 0.0 00.01700000" rpy="0 0 0"/>
+        <origin xyz="0 0.0 00.01700000" rpy="0 0 0"/>
         <mass value="0.40700000"/>
         <inertia

Commit message: [Ninja][URDF] update urdf model

File: robots/ninja/urdf/ninja.urdf.xacro (robot description, xacro)
@@ -23,10 +23,10 @@
     <link name="main_body">
       <inertial>
-        <origin xyz="-0.08989427 -0.00260694 -0.01604721" rpy="0 0 0"/>
-        <mass value="1.32590383"/>
-        <inertia
-            ixx = "0.00565938" ixy = "0.00127382" ixz = "0.00065740"
-            iyx = "0.00127382" iyy = "0.04578657" iyz = "-0.00004725"
-            izx = "0.00065740" izy = "-0.00004725" izz = "0.04949468"/>
+        <origin xyz="-0.08859352 -0.00340645 -0.01623433" rpy="0 0 0"/>
+        <mass value="1.41458199"/>
+        <inertia
+            ixx = "0.00677420" ixy = "0.00173147" ixz = "0.00081701"
+            iyx = "0.00173147" iyy = "0.05074341" iyz = "-0.00005705"
+            izx = "0.00081701" izy = "-0.00005705" izz = "0.05529837"/>
       </inertial>
       <visual>
@@ -115,15 +115,15 @@
     <link name="yaw_dock_link">
       <inertial>
-        <origin xyz="0.06781112 -0.00002493 -0.02345044" rpy="0 0 0"/>
-        <mass value="0.21443253"/>
-        <inertia
-            ixx = "0.00093162" ixy = "0.00000022" ixz = "-0.00002253"
-            iyx = "0.00000022" iyy = "0.00071768" iyz = "-0.00010593"
-            izx = "-0.00002253" izy = "-0.00010593" izz = "0.00091594"/>
+        <origin xyz="0.06974525 0.00038438 -0.02390949" rpy="0 0 0"/>
+        <mass value="0.30727535"/>
+        <inertia
+            ixx = "0.00056834" ixy = "-0.00000383" ixz = "-0.00002348"
+            iyx = "-0.00000383" iyy = "0.00074609" iyz = "-0.00000529"
+            izx = "-0.00002348" izy = "-0.00000529" izz = "0.00067836"/>
       </inertial>
       <visual>
         <origin xyz="0 0 0" rpy="${pi/2} 0 0"/>
         <geometry>
-          <mesh filename="package://ninja/urdf/mesh/female_dock_mech.dae" scale="1 1 1"/>
+          <mesh filename="package://ninja/urdf/mesh/male_dock_mech.dae" scale="1 1 1"/>
         </geometry>
       </visual>
@@ -137,5 +137,5 @@
     <xacro:damping_factor link="yaw_dock_link"/>
     <joint name="yaw_dock_joint" type="revolute">
-      <limit effort="6.6" lower="-3.14" upper="3.14" velocity="0.2"/>
+      <limit effort="10" lower="-3.14" upper="3.14" velocity="0.2"/>
       <parent link="main_body"/>
       <child link="yaw_dock_link"/>
@@ -167,5 +167,5 @@
       <parent link="yaw_dock_link"/>
       <child link="yaw_connect_point"/>
-      <origin rpy="0 0 0" xyz="0.037 0 -0.025"/>
+      <origin rpy="0 0 0" xyz="0.1531 0 -0.025"/>
       <axis xyz="0 0 1"/>
     </joint>
@@ -195,5 +195,5 @@
       <inertial>
        <origin xyz="0.12245044 0.03129270 0.00001719" rpy="0 0 0"/>
-        <mass value="0.19445396"/>
+       <mass value="0.19445396"/>
         <inertia
             ixx = "0.00119253" ixy = "0.00015756" ixz = "-0.00000029"
@@ -230,10 +230,10 @@
     <link name="rotor_parent${self}">
       <inertial>
-        <origin xyz="0.09 0 0" rpy="0 0 ${-pi/2}"/>
-        <mass value="0.220"/>
-        <inertia
-            ixx="0.0002011" ixy="0.0000001" ixz="0.0000003"
-            iyy="0.0004337" iyz="0.0"
-            izz="0.0005261"/>
+        <origin xyz="-0.0000209 -0.0725606 0.0007205" rpy="0 0 0"/>
+        <mass value="0.2051889"/>
+        <inertia
+            ixx = "0.0004283" ixy = "0.0000000" ixz = "0.0000001"
+            iyx = "0.0000000" iyy = "0.0002249" iyz = "-0.0000001"
+            izx = "0.0000001" izy = "-0.0000001" izz = "0.0005545"/>
       </inertial>
       <visual>
@@ -285,15 +285,15 @@
     <link name="pitch_dock_link">
       <inertial>
-        <origin xyz="-0.06961517 0.02389743 -0.00688546" rpy="0 0 0"/>
-        <mass value="0.30174800"/>
-        <inertia
-            ixx = "0.00053278" ixy = "-0.00002216" ixz = "0.00003995"
-            iyx = "-0.00002216" iyy = "0.00065740" iyz = "-0.00000804"
-            izx = "0.00003995" izy = "-0.00000804" izz = "0.00073599"/>
+        <origin xyz="-0.05345739 0.02283891 0.00003454" rpy="0 0 0"/>
+        <mass value="0.15375166"/>
+        <inertia
+            ixx = "0.00044124" ixy = "-0.00001776" ixz = "0.00000015"
+            iyx = "-0.00001776" iyy = "0.00046036" iyz = "-0.00006736"
+            izx = "0.00000015" izy = "-0.00006736" izz = "0.00038793"/>
       </inertial>
       <visual>
         <origin xyz="0 0 0" rpy="${pi} ${pi} 0"/>
         <geometry>
-          <mesh filename="package://ninja/urdf/mesh/male_dock_mech.dae" scale="1 1 1"/>
+          <mesh filename="package://ninja/urdf/mesh/female_dock_mech.dae" scale="1 1 1"/>
         </geometry>
       </visual>
@@ -307,5 +307,5 @@
     <xacro:damping_factor link="pitch_dock_link"/>
     <joint name="pitch_dock_joint" type="revolute">
-      <limit effort="6.6" lower="-3.14" upper="3.14" velocity="0.2"/>
+      <limit effort="10" lower="-3.14" upper="3.14" velocity="0.2"/>
       <parent link="main_body"/>
       <child link="pitch_dock_link"/>
@@ -337,5 +337,5 @@
       <parent link="pitch_dock_link"/>
       <child link="pitch_connect_point"/>
-      <origin rpy="0 0 0" xyz="-0.1531 0.025 0"/>
+      <origin rpy="0 0 0" xyz="-0.037 0.025 0"/>
       <axis xyz="0 0 1"/>
     </joint>
@@ -345,14 +345,15 @@
       <parent link="main_body"/>
       <child link="battery_1"/>
-      <origin rpy="-${pi/2} 0 ${pi}" xyz="-0.00891 0.0399 -0.069"/>
+      <origin rpy="0 0 ${pi/2-0.977}" xyz="-0.10215 -0.07574 -0.04"/>
       <axis xyz="0 0 0"/>
     </joint>
     <link name="battery_1">
       <inertial>
-        <origin xyz="0 0.0 00.01700000" rpy="0 0 0"/>
-        <mass value="0.40700000"/>
-        <inertia
-            ixx="0.00010170" iyy="0.00060259" izz="0.00062827"
-            ixy="0.000" ixz=" 0.000000" iyz="0.0000"/>
+        <origin xyz="0.0 0.0 -0.019" rpy="0 0 0"/>
+        <mass value="0.44600000"/>
+        <inertia
+            ixx = "0.00012215" ixy = "0.00000000" ixz = "0.00000000"
+            iyx = "0.00000000" iyy = "0.00067139" iyz = "0.00000000"
+            izx = "0.00000000" izy = "0.00000000" izz = "0.00068918"/>
       </inertial>
       <visual>
@@ -367,14 +368,15 @@
       <parent link="main_body"/>
       <child link="battery_2"/>
-      <origin rpy="${-pi/2} 0 0" xyz="-0.00891 -0.0399 -0.069"/>
+      <origin rpy="0 0 -${pi/2-0.977}" xyz="-0.10215 0.07574 -0.04"/>
       <axis xyz="0 0 0"/>
     </joint>
     <link name="battery_2">
       <inertial>
-        <origin xyz="0 0.0 00.01700000" rpy="0 0 0"/>
-        <mass value="0.40700000"/>
-        <inertia
-            ixx="0.00010170" iyy="0.00060259" izz="0.00062827"
-            ixy="0.000" ixz=" 0.000000" iyz="0.0000"/>
+        <origin xyz="0.0 0.0 -0.01900000" rpy="0 0 0"/>
+        <mass value="0.44600000"/>
+        <inertia
+            ixx = "0.00012215" ixy = "0.00000000" ixz = "0.00000000"
+            iyx = "0.00000000" iyy = "0.00067139" iyz = "0.00000000"
+            izx = "0.00000000" izy = "0.00000000" izz = "0.00068918"/>
       </inertial>
       <visual>

Commit message: [Ninja][URDF] Corrected gimbal_link inertia.

File: robots/ninja/urdf/ninja.urdf.xacro (robot description, xacro)
@@ -128,14 +128,14 @@
         </geometry>
       </visual>
-      <!-- <collision> -->
-      <!--   <origin xyz="0 0 0" rpy="0 0 0"/> -->
-      <!--   <geometry> -->
-      <!--     <box size="0.05 0.05 0.05"/> -->
-      <!--   </geometry> -->
-      <!-- </collision> -->
+      <collision>
+        <origin xyz="0 0.0 0" rpy="${pi/2} 0 0"/>
+        <geometry>
+          <box size="0.1531 0.064 0.064"/>
+        </geometry>
+      </collision>
     </link>
     <xacro:damping_factor link="yaw_dock_link"/>
     <joint name="yaw_dock_joint" type="revolute">
-      <limit effort="10" lower="-3.14" upper="3.14" velocity="0.2"/>
+      <limit effort="6.6" lower="-3.14" upper="3.14" velocity="0.2"/>
       <parent link="main_body"/>
       <child link="yaw_dock_link"/>
@@ -194,6 +194,16 @@
     <link name="gimbal_link${self}">
       <inertial>
-       <origin xyz="0.12245044 0.03129270 0.00001719" rpy="0 0 0"/>
-       <mass value="0.19445396"/>
+        <xacro:if value="${self==1}">
+          <origin xyz="0.12245044 -0.03129270 -0.00001719" rpy="${pi} 0 0"/>
+          <mass value="0.19445396"/>
+        </xacro:if>
+        <xacro:if value="${self==2}">
+          <origin xyz="0.12245044 0.03129270 0.00001719" rpy="0 0 0"/>
+          <mass value="0.19445396"/>
+        </xacro:if>
+        <xacro:if value="${self==3}">
+          <origin xyz="0.12245044 -0.03129270 -0.00001719" rpy="${pi} 0 0"/>
+          <mass value="0.19445396"/>
+        </xacro:if>
         <inertia
             ixx = "0.00119253" ixy = "0.00015756" ixz = "-0.00000029"
@@ -202,5 +212,13 @@
       </inertial>
       <visual>
-        <origin xyz="0 0 0" rpy="0 0 0"/>
+        <xacro:if value="${self==1}">
+          <origin xyz="0 0 0" rpy="0 0 0"/>
+        </xacro:if>
+        <xacro:if value="${self==2}">
+          <origin xyz="0 0 0" rpy="${pi} 0 0"/>
+        </xacro:if>
+        <xacro:if value="${self==3}">
+          <origin xyz="0 0 0" rpy="0 0 0"/>
+        </xacro:if>
         <geometry>
           <mesh filename="package://ninja/urdf/mesh/gimbal_link.dae" scale="1 1 1"/>
@@ -298,14 +316,14 @@
         </geometry>
       </visual>
-      <collision>
-        <origin xyz="-${0.1531/2} 0.025 0" rpy="0 0 0"/>
-        <geometry>
-          <box size="0.1531 0.064 0.064"/>
-        </geometry>
-      </collision>
+      <!-- <collision> -->
+      <!--   <origin xyz="0 0 0" rpy="0 0 0"/> -->
+      <!--   <geometry> -->
+      <!--     <box size="0.05 0.05 0.05"/> -->
+      <!--   </geometry> -->
+      <!-- </collision> -->
     </link>
     <xacro:damping_factor link="pitch_dock_link"/>
     <joint name="pitch_dock_joint" type="revolute">
-      <limit effort="10" lower="-3.14" upper="3.14" velocity="0.2"/>
+      <limit effort="20" lower="-3.14" upper="3.14" velocity="0.2"/>
       <parent link="main_body"/>
       <child link="pitch_dock_link"/>

Commit message: [Ninja][URDF]Chnage model innertia and mesh to the one with magnet.

File: robots/ninja/urdf/ninja.urdf.xacro (robot description, xacro)
@@ -115,23 +115,23 @@
     <link name="yaw_dock_link">
       <inertial>
-        <origin xyz="0.06974525 0.00038438 -0.02390949" rpy="0 0 0"/>
-        <mass value="0.30727535"/>
-        <inertia
-            ixx = "0.00056834" ixy = "-0.00000383" ixz = "-0.00002348"
-            iyx = "-0.00000383" iyy = "0.00074609" iyz = "-0.00000529"
-            izx = "-0.00002348" izy = "-0.00000529" izz = "0.00067836"/>
-      </inertial>
-      <visual>
-        <origin xyz="0 0 0" rpy="${pi/2} 0 0"/>
+        <origin xyz="0.07864928 0.00031794 -0.02812152" rpy="0 0 0"/>
+        <mass value="0.37142798"/>
+        <inertia
+           ixx ="0.00056278" ixy ="-0.00000715" ixz ="-0.00002624"
+          iyx ="-0.00000715" iyy ="0.00095271" iyz ="0.00000729"
+          izx ="-0.00002624" izy ="0.00000729" izz ="0.00089334"/>
+      </inertial>
+      <visual>
+        <origin xyz="0 0 0" rpy="0 0 0"/>
        <geometry>
           <mesh filename="package://ninja/urdf/mesh/male_dock_mech.dae" scale="1 1 1"/>
         </geometry>
       </visual>
-      <!-- <collision> -->
-      <!--   <origin xyz="0 0.0 0" rpy="${pi/2} 0 0"/> -->
-      <!--   <geometry> -->
-      <!--     <box size="0.1531 0.064 0.064"/> -->
-      <!--   </geometry> -->
-      <!-- </collision> -->
+      <collision>
+        <origin xyz="0 0.0 0" rpy="${pi/2} 0 0"/>
+        <geometry>
+          <box size="0.1531 0.064 0.064"/>
+        </geometry>
+      </collision>
     </link>
     <xacro:damping_factor link="yaw_dock_link"/>
@@ -140,5 +140,5 @@
       <parent link="main_body"/>
       <child link="yaw_dock_link"/>
-      <origin rpy="0 0 0" xyz="0.1935 0 0.0085"/>
+      <origin rpy="0 0 0" xyz="0.1935 0 0.0125"/>
       <axis xyz="0 0 1"/>
       <dynamics damping="0.8" friction="0.0"/>
@@ -167,5 +167,5 @@
       <parent link="yaw_dock_link"/>
       <child link="yaw_connect_point"/>
-      <origin rpy="0 0 0" xyz="0.1531 0 -0.025"/>
+      <origin rpy="0 0 0" xyz="0.14085 0 -0.025"/>
       <axis xyz="0 0 1"/>
     </joint>
@@ -303,10 +303,10 @@
     <link name="pitch_dock_link">
       <inertial>
-        <origin xyz="-0.05345739 0.02283891 0.00003454" rpy="0 0 0"/>
-        <mass value="0.15375166"/>
-        <inertia
-            ixx = "0.00044124" ixy = "-0.00001776" ixz = "0.00000015"
-            iyx = "-0.00001776" iyy = "0.00046036" iyz = "-0.00006736"
-            izx = "0.00000015" izy = "-0.00006736" izz = "0.00038793"/>
+        <origin xyz="-0.05014456 0.02319253 0.00002876" rpy="0 0 0"/>
+        <mass value="0.18383088"/>
+        <inertia
+            ixx ="0.00040471" ixy ="-0.00001666" ixz ="0.00000013"
+            iyx ="-0.00001666" iyy ="0.00042839" iyz ="-0.00005920"
+            izx ="0.00000013" izy ="-0.00005920" izz ="0.00036811"/>
       </inertial>
       <visual>

Commit message: [Ninja][URDF] Update female mech inertia.

File: robots/ninja/urdf/ninja.urdf.xacro (robot description, xacro)
@@ -303,10 +303,10 @@
     <link name="pitch_dock_link">
       <inertial>
-        <origin xyz="-0.05014456 0.02319253 0.00002876" rpy="0 0 0"/>
-        <mass value="0.18383088"/>
-        <inertia
-            ixx ="0.00040471" ixy ="-0.00001666" ixz ="0.00000013"
-            iyx ="-0.00001666" iyy ="0.00042839" iyz ="-0.00005920"
-            izx ="0.00000013" izy ="-0.00005920" izz ="0.00036811"/>
+        <origin xyz="-0.05087327 0.02329154 0.00017464" rpy="0 0 0"/>
+        <mass value="0.19583088"/>
+        <inertia
+            ixx ="0.00044711" ixy ="-0.00001684" ixz ="-0.00000107"
+            iyx ="-0.00001684" iyy ="0.00047285" iyz ="-0.00007906"
+            izx ="-0.00000107" izy ="-0.00007906" izz = "0.00038353"/>
       </inertial>
       <visual>

Commit message: [Ninja][URDF] Modified yaw_connect_point position.

File: robots/ninja/urdf/ninja.urdf.xacro (robot description, xacro)
@@ -167,5 +167,5 @@
       <parent link="yaw_dock_link"/>
       <child link="yaw_connect_point"/>
-      <origin rpy="0 0 0" xyz="0.14085 0 -0.025"/>
+      <origin rpy="0 0 0" xyz="0.14085 0 -0.030"/>
       <axis xyz="0 0 1"/>
     </joint>
