Commit message: [Ninja][URDF] update dock mech inertia.

File: robots/ninja/urdf/ninja.urdf.xacro (robot description, xacro)
@@ -115,10 +115,10 @@
     <link name="yaw_dock_link">
       <inertial>
-        <origin xyz="0.07864928 0.00031794 -0.02812152" rpy="0 0 0"/>
-        <mass value="0.37142798"/>
-        <inertia
-           ixx ="0.00056278" ixy ="-0.00000715" ixz ="-0.00002624"
-          iyx ="-0.00000715" iyy ="0.00095271" iyz ="0.00000729"
-          izx ="-0.00002624" izy ="0.00000729" izz ="0.00089334"/>
+        <origin xyz="0.07707992 0.00034225 -0.02807178" rpy="0 0 0"/>
+        <mass value="0.33699537"/>
+        <inertia
+            ixx = "0.00047120" ixy = "-0.00000696" ixz = "-0.00002605"
+            iyx = "-0.00000696" iyy = "0.00089048" iyz = "0.00000963"
+            izx = "-0.00002605" izy = "0.00000963" izz = "0.00082655"/>
       </inertial>
       <visual>
@@ -303,10 +303,10 @@
     <link name="pitch_dock_link">
       <inertial>
-        <origin xyz="-0.05087327 0.02329154 0.00017464" rpy="0 0 0"/>
-        <mass value="0.19583088"/>
-        <inertia
-            ixx ="0.00044711" ixy ="-0.00001684" ixz ="-0.00000107"
-            iyx ="-0.00001684" iyy ="0.00047285" iyz ="-0.00007906"
-            izx ="-0.00000107" izy ="-0.00007906" izz = "0.00038353"/>
+        <origin xyz="-0.04795875 0.02306659 0.00003088" rpy="0 0 0"/>
+        <mass value="0.17183088"/>
+        <inertia
+            ixx = "0.00035938" ixy = "-0.00001594" ixz = "0.00000012"
+            iyx = "-0.00001594" iyy = "0.00038919" iyz = "0.00006568"
+            izx = "0.00000012" izy = "0.00006568" izz = "0.00032884"/>
       </inertial>
       <visual>

Commit message: [Ninja][urdf] Change the inertia of gimbal pitch link

File: robots/ninja/urdf/ninja.urdf.xacro (robot description, xacro)
@@ -247,11 +247,19 @@
     ## rotor parent link
     <link name="rotor_parent${self}">
-      <inertial>
-        <origin xyz="-0.0000209 -0.0725606 0.0007205" rpy="0 0 0"/>
-        <mass value="0.2051889"/>
-        <inertia
-            ixx = "0.0004283" ixy = "0.0000000" ixz = "0.0000001"
-            iyx = "0.0000000" iyy = "0.0002249" iyz = "-0.0000001"
-            izx = "0.0000001" izy = "-0.0000001" izz = "0.0005545"/>
+      <!-- <inertial> -->
+      <!--   <origin xyz="-0.0000209 -0.0725606 0.0007205" rpy="0 0 0"/> -->
+      <!--   <mass value="0.2051889"/> -->
+      <!--   <inertia -->
+      <!--       ixx = "0.0004283" ixy = "0.0000000" ixz = "0.0000001" -->
+      <!--       iyx = "0.0000000" iyy = "0.0002249" iyz = "-0.0000001" -->
+      <!--       izx = "0.0000001" izy = "-0.0000001" izz = "0.0005545"/> -->
+      <!-- </inertial> -->
+      <inertial>
+        <origin xyz="0.00000000 -0.07234801 0.00062937" rpy="0 0 0"/>
+        <mass value="0.17219070"/>
+        <inertia
+            ixx = "0.00035073" ixy = "0.00000000" ixz = "0.00000000"
+            iyx = "0.00000000" iyy = "0.00017156" iyz = "-0.00000012"
+            izx = "0.00000000" izy = "-0.00000012" izz = "0.00044377"/>
       </inertial>
       <visual>

Commit message: [Ninja][urdf] Modified positions of 1300mAh batteries.

File: robots/ninja/urdf/ninja.urdf.xacro (robot description, xacro)
@@ -421,5 +421,5 @@
       <parent link="main_body"/>
       <child link="battery_1"/>
-      <origin rpy="0 0 ${pi/2-0.977}" xyz="-0.10215 -0.07574 -0.04"/>
+      <origin rpy="0 0 0" xyz="-0.21 -0.15 -0.04"/>
       <axis xyz="0 0 0"/>
     </joint>
@@ -447,5 +447,5 @@
       <parent link="main_body"/>
       <child link="battery_2"/>
-      <origin rpy="0 0 -${pi/2-0.977}" xyz="-0.10215 0.07574 -0.04"/>
+      <origin rpy="0 0 0" xyz="-0.21 0.15 -0.04"/>
       <axis xyz="0 0 0"/>
     </joint>
