Commit message: fix inertial matrix more correctly

File: robots/hugmy/urdf/robot.urdf.xacro (robot description, xacro)
@@ -6,9 +6,11 @@
   <thrust_link name="thrust" />
   <!-- kinematics [m] -->
-  <xacro:property name="rotor_x" value="0.070" />
-  <xacro:property name="rotor_y" value="0.086" />
-  <xacro:property name="rotor_z" value="0.026" />
+  <xacro:property name="rotor_x" value="0.08479" />
+  <xacro:property name="rotor_y" value="0.08479" />
+  <!-- <xacro:property name="rotor_z" value="0.330" /> -->
+  <!-- <xacro:property name="rotor_z" value="0.055" /> -->
+  <xacro:property name="rotor_z" value="0.0024" />
   <!-- dynamics -->
-  <m_f_rate value="-0.011" /> <!-- drag torque rate -->
+  <m_f_rate value="-0.0068" /> <!-- drag torque rate -->
   <xacro:property name="max_force" value="8.0" /> <!-- [N] -->
   <xacro:property name="min_force" value="0.0" /> <!-- [N] -->
@@ -58,5 +60,5 @@
         <origin rpy="0 0 0" xyz="0 0 0"/>
         <geometry>
-          <mesh filename="package://mini_quadrotor/urdf/mesh/prop_5inch.dae" />
+          <mesh filename="package://hugmy/urdf/mesh/prop_5inch.dae" />
         </geometry>
       </visual>
@@ -96,15 +98,15 @@
   <link name="main_body">
     <inertial>
-      <mass value = "0.432" />
-      <origin xyz="0 0 0.017" rpy="0 0 0"/>
+      <mass value = "1.286" />
+      <origin xyz="0.0001458 -0.00117927 0.00925351" rpy="0 0 0"/>
       <inertia
-          ixx="0.0021" ixy="0" ixz="0"
-          iyy="0.0015" iyz="0"
-          izz="0.0032"/>
+          ixx="0.00915711" ixy="0.00000019" ixz="-0.00001262"
+          iyy="0.00910525" iyz="0.00004832"
+          izz="0.01525601"/>
     </inertial>
     <visual>
       <origin rpy="0 0 0" xyz="0 0 0"/>
       <geometry>
-        <mesh filename="package://mini_quadrotor/urdf/mesh/main_body.dae" />
+        <mesh filename="package://hugmy/urdf/mesh/hugmy.dae" />
       </geometry>
     </visual>
@@ -128,5 +130,5 @@
   </xacro:extra_module>
   <!-- battery -->
-  <xacro:extra_module name = "battery" parent = "main_body" visible = "1" model_url = "package://mini_quadrotor/urdf/mesh/turnigy_3S_2200mAh.dae" >
+  <xacro:extra_module name = "battery" parent = "main_body" visible = "1" model_url = "package://hugmy/urdf/mesh/turnigy_3S_2200mAh.dae" >
     <origin xyz="0.0105 0 -0.012" rpy="0 0 0"/>
     <inertial>
@@ -134,5 +136,5 @@
       <origin xyz="0 0 0" rpy="0 0 0"/>
       <inertia
-          ixx="0.0002" ixy="0.0" ixz="0.0"
+          ixx="0.0" ixy="0.0" ixz="0.0"
           iyy="0.0002" iyz="0.0" izz="0.0002"/>
     </inertial>

File: robots/mini_quadrotor/urdf/infratable/robot.urdf.xacro (robot description, xacro)
@@ -6,11 +6,11 @@
   <thrust_link name="thrust" />
   <!-- kinematics [m] -->
-  <xacro:property name="rotor_x" value="0.090" />
-  <xacro:property name="rotor_y" value="0.090" />
+  <xacro:property name="rotor_x" value="0.08479" />
+  <xacro:property name="rotor_y" value="0.08479" />
   <!-- <xacro:property name="rotor_z" value="0.330" /> -->
   <!-- <xacro:property name="rotor_z" value="0.055" /> -->
-  <xacro:property name="rotor_z" value="0.180" />
+  <xacro:property name="rotor_z" value="0.0024" />
   <!-- dynamics -->
-  <m_f_rate value="-0.011" /> <!-- drag torque rate -->
+  <m_f_rate value="-0.0068" /> <!-- drag torque rate -->
   <xacro:property name="max_force" value="8.0" /> <!-- [N] -->
   <xacro:property name="min_force" value="0.0" /> <!-- [N] -->
@@ -99,9 +99,9 @@
     <inertial>
       <mass value = "1.45" />
-      <origin xyz="0 0 0.017" rpy="0 0 0"/>
+      <origin xyz="0.0001458 -0.00117927 0.00925351" rpy="0 0 0"/>
       <inertia
-          ixx="0.0021" ixy="0" ixz="0"
-          iyy="0.0015" iyz="0"
-          izz="0.0032"/>
+          ixx="0.00934471" ixy="0.00000254" ixz="-0.00002280"
+          iyy="0.00939415" iyz="0.00000342"
+          izz="0.01536758"/>
     </inertial>
     <visual>

Commit message: update robot urdf of no face

File: robots/hugmy/urdf/robot.urdf.xacro (robot description, xacro)
@@ -99,9 +99,16 @@
     <inertial>
       <mass value = "1.286" />
-      <origin xyz="0.0001458 -0.00117927 0.00925351" rpy="0 0 0"/>
+      <!-- with eye module -->
+      <!-- <origin xyz="0.0001458 -0.00117927 0.00925351" rpy="0 0 0"/> -->
+      <origin xyz="0.00005399, 0.00050398, 0.06350617" rpy="0 0 0"/>
+      <!-- with eye module -->
+      <!-- <inertia -->
+      <!--     ixx="0.00915711" ixy="0.00000019" ixz="-0.00001262" -->
+      <!--     iyy="0.00910525" iyz="0.00004832" -->
+      <!--     izz="0.01525601"/> -->
       <inertia
-          ixx="0.00915711" ixy="0.00000019" ixz="-0.00001262"
-          iyy="0.00910525" iyz="0.00004832"
-          izz="0.01525601"/>
+          ixx="0.01486737" ixy="-0.00000799" ixz="-0.00000789"
+          iyy="0.01486369" iyz="-0.00004397"
+          izz="0.00624429"/>
     </inertial>
     <visual>

Commit message: adjust parameter

File: robots/hugmy/urdf/robot.urdf.xacro (robot description, xacro)
@@ -10,5 +10,5 @@
   <!-- <xacro:property name="rotor_z" value="0.330" /> -->
   <!-- <xacro:property name="rotor_z" value="0.055" /> -->
-  <xacro:property name="rotor_z" value="0.0024" />
+  <xacro:property name="rotor_z" value="0.044" />
   <!-- dynamics -->
   <m_f_rate value="-0.0068" /> <!-- drag torque rate -->
@@ -101,5 +101,5 @@
       <!-- with eye module -->
       <!-- <origin xyz="0.0001458 -0.00117927 0.00925351" rpy="0 0 0"/> -->
-      <origin xyz="0.00005399, 0.00050398, 0.06350617" rpy="0 0 0"/>
+      <origin xyz="0.00005399 0.00050398 0.06350617" rpy="0 0 0"/>
       <!-- with eye module -->
       <!-- <inertia -->
@@ -115,5 +115,5 @@
       <origin rpy="0 0 0" xyz="0 0 0"/>
       <geometry>
-        <mesh filename="package://hugmy/urdf/mesh/hugmy.dae" />
+        <mesh filename="package://hugmy/urdf/mesh/Inflatable_asm_with_all_module.STL" />
       </geometry>
     </visual>

Commit message: update main_body

File: robots/hugmy/urdf/robot.urdf.xacro (robot description, xacro)
@@ -101,5 +101,5 @@
       <!-- with eye module -->
       <!-- <origin xyz="0.0001458 -0.00117927 0.00925351" rpy="0 0 0"/> -->
-      <origin xyz="0.00005399 0.00050398 0.06350617" rpy="0 0 0"/>
+      <origin xyz="-0.00070411 -0.00014118 -0.00266031" rpy="0 0 0"/>
       <!-- with eye module -->
       <!-- <inertia -->
@@ -108,7 +108,7 @@
       <!--     izz="0.01525601"/> -->
       <inertia
-          ixx="0.01486737" ixy="-0.00000799" ixz="-0.00000789"
-          iyy="0.01486369" iyz="-0.00004397"
-          izz="0.00624429"/>
+          ixx="0.00917972" ixy="-0.00000174" ixz="-0.00002884"
+          iyy="0.00919131" iyz="-0.00000126"
+          izz="0.01521010"/>
     </inertial>
     <visual>

Commit message: update urdf

File: robots/hugmy/urdf/robot.urdf.xacro (robot description, xacro)
@@ -98,8 +98,8 @@
   <link name="main_body">
     <inertial>
-      <mass value = "1.286" />
+      <mass value = "1.176" />
       <!-- with eye module -->
       <!-- <origin xyz="0.0001458 -0.00117927 0.00925351" rpy="0 0 0"/> -->
-      <origin xyz="-0.00070411 -0.00014118 -0.00266031" rpy="0 0 0"/>
+      <origin xyz="-0.00187886 -0.00015416 0.00165752" rpy="0 0 0"/>
       <!-- with eye module -->
       <!-- <inertia -->
@@ -108,7 +108,7 @@
       <!--     izz="0.01525601"/> -->
       <inertia
-          ixx="0.00917972" ixy="-0.00000174" ixz="-0.00002884"
-          iyy="0.00919131" iyz="-0.00000126"
-          izz="0.01521010"/>
+          ixx="0.00659595" ixy="-0.00000357" ixz="-0.00010985"
+          iyy="0.00674188" iyz="-0.00000027"
+          izz="0.01039566"/>
     </inertial>
     <visual>

Commit message: add battery URDF model

File: robots/hugmy/urdf/robot.urdf.xacro (robot description, xacro)
@@ -8,6 +8,7 @@
   <xacro:property name="rotor_x" value="0.08479" />
   <xacro:property name="rotor_y" value="0.08479" />
-  <!-- <xacro:property name="rotor_z" value="0.330" /> -->
-  <!-- <xacro:property name="rotor_z" value="0.055" /> -->
+  <!-- simulation -->
+  <!-- <xacro:property name="rotor_z" value="-0.002" /> -->
+  <!-- real machine -->
   <xacro:property name="rotor_z" value="0.044" />
   <!-- dynamics -->
@@ -121,5 +122,5 @@
       <origin rpy="0 0 0" xyz="0 0 0"/>
       <geometry>
-        <box size="0.28 0.28 0.072" />
+        <box size="0.28 0.28 0.121" />
       </geometry>
     </collision>
@@ -137,14 +138,77 @@
   </xacro:extra_module>
   <!-- battery -->
-  <xacro:extra_module name = "battery" parent = "main_body" visible = "1" model_url = "package://hugmy/urdf/mesh/turnigy_3S_2200mAh.dae" >
-    <origin xyz="0.0105 0 -0.012" rpy="0 0 0"/>
-    <inertial>
-      <mass value = "0.188" />
-      <origin xyz="0 0 0" rpy="0 0 0"/>
-      <inertia
-          ixx="0.0" ixy="0.0" ixz="0.0"
-          iyy="0.0002" iyz="0.0" izz="0.0002"/>
-    </inertial>
-  </xacro:extra_module>
+  <!-- <xacro:extra_module name = "battery" parent = "main_body" visible = "1" model_url = "package://hugmy/urdf/mesh/turnigy_3S_2200mAh.dae" > -->
+  <!--   <origin xyz="0.0105 0 -0.012" rpy="0 0 0"/> -->
+  <!--   <inertial> -->
+  <!--     <mass value = "0.188" /> -->
+  <!--     <origin xyz="0 0 0" rpy="0 0 0"/> -->
+  <!--     <inertia -->
+  <!--         ixx="0.0" ixy="0.0" ixz="0.0" -->
+  <!--         iyy="0.0002" iyz="0.0" izz="0.0002"/> -->
+  <!--   </inertial> -->
+  <!-- </xacro:extra_module> -->
+  <link name = "battery_0">
+    <inertial>
+      <mass value = "0.108" />
+      <origin xyz="0 0 0" rpy="0 0 0"/>
+      <inertia
+          ixx="0.00001517" ixy="0.0" ixz="0.0"
+          iyy="0.00005450" iyz="0.0" izz="0.00004886"/>
+    </inertial>
+    <visual>
+      <origin rpy="0 0 0" xyz="0 0 0"/>
+      <geometry>
+        <mesh filename="package://hugmy/urdf/mesh/4S_1000mAh_battery.STL"/>
+        <box size="0.29 0.34 0.070" />
+      </geometry>
+    </visual>
+  </link>
+    <link name = "battery_1">
+    <inertial>
+      <mass value = "0.108" />
+      <origin xyz="0 0 0" rpy="0 0 0"/>
+      <inertia
+          ixx="0.00001517" ixy="0.0" ixz="0.0"
+          iyy="0.00005450" iyz="0.0" izz="0.00004886"/>
+    </inertial>
+    <visual>
+      <origin rpy="0 0 0" xyz="0 0 0"/>
+      <geometry>
+        <mesh filename="package://hugmy/urdf/mesh/4S_1000mAh_battery.STL"/>
+        <box size="0.070 0.023 0.034" />
+      </geometry>
+    </visual>
+  </link>
+  <!-- <link name = "battery_1"> -->
+  <!--   <inertial> -->
+  <!--     <mass value = "0.108" /> -->
+  <!--     <origin xyz="0 0 0" rpy="0 0 0"/> -->
+  <!--     <inertia -->
+  <!--         ixx="0.0" ixy="0.0" ixz="0.0" -->
+  <!--         iyy="0.0002" iyz="0.0" izz="0.0002"/> -->
+  <!--   </inertial> -->
+  <!--   <visual> -->
+  <!--     <origin rpy="0 0 0" xyz="0 0 0"/> -->
+  <!--     <geometry> -->
+  <!--       <mesh filename="package://hugmy/urdf/mesh/4S_1300mAh_battery.STL"/> -->
+  <!--       <box size="0.29 0.34 0.070" /> -->
+  <!--     </geometry> -->
+  <!--   </visual> -->
+  <!-- </link> -->
+  <joint name="battery_0_joint" type="fixed">
+      <parent link="main_body"/>
+      <child link="battery_0"/>
+      <origin rpy="0 0 ${-pi/4}" xyz="0.01202 0.01202 -0.0365"/>
+  </joint>
+  <joint name="battery_1_joint" type="fixed">
+      <parent link="main_body"/>
+      <child link="battery_1"/>
+      <origin rpy="0 0 ${-pi/4}" xyz="-0.01202 -0.01202 -0.0365"/>
+  </joint>
+  <!-- <joint name="battery_1_joint" type="fixed"> -->
+  <!--     <parent link="main_body"/> -->
+  <!--     <child link="battery_1"/> -->
+  <!--     <origin rpy="0 0 ${-pi/4}" xyz="-0.01025 -0.01025 -0.045"/> -->
+  <!-- </joint> -->
   <!-- propellers -->
   <xacro:propeller_module id = "1" x = "${rotor_x}" y = "${-rotor_y}" z = "${rotor_z}" direction = "-1" />

File: robots/hugmy/urdf/robot_ver2.urdf.xacro (robot description, xacro)
@@ -258,14 +258,67 @@
   </xacro:extra_module>
   <!-- battery -->
-  <xacro:extra_module name = "battery" parent = "main_body" visible = "1" model_url = "package://hugmy/urdf/mesh/turnigy_3S_2200mAh.dae" >
-    <origin xyz="0.0105 0 -0.012" rpy="0 0 0"/>
-    <inertial>
-      <mass value = "0.188" />
+  <link name = "battery_0">
+    <inertial>
+      <mass value = "0.108" />
       <origin xyz="0 0 0" rpy="0 0 0"/>
       <inertia
-          ixx="0.0" ixy="0.0" ixz="0.0"
-          iyy="0.0002" iyz="0.0" izz="0.0002"/>
-    </inertial>
-  </xacro:extra_module>
+          ixx="0.00001517" ixy="0.0" ixz="0.0"
+          iyy="0.00005450" iyz="0.0" izz="0.00004886"/>
+    </inertial>
+    <visual>
+      <origin rpy="0 0 0" xyz="0 0 0"/>
+      <geometry>
+        <mesh filename="package://hugmy/urdf/mesh/4S_1000mAh_battery.STL"/>
+        <box size="0.29 0.34 0.070" />
+      </geometry>
+    </visual>
+  </link>
+    <link name = "battery_1">
+    <inertial>
+      <mass value = "0.108" />
+      <origin xyz="0 0 0" rpy="0 0 0"/>
+      <inertia
+          ixx="0.00001517" ixy="0.0" ixz="0.0"
+          iyy="0.00005450" iyz="0.0" izz="0.00004886"/>
+    </inertial>
+    <visual>
+      <origin rpy="0 0 0" xyz="0 0 0"/>
+      <geometry>
+        <mesh filename="package://hugmy/urdf/mesh/4S_1000mAh_battery.STL"/>
+        <box size="0.070 0.023 0.034" />
+      </geometry>
+    </visual>
+  </link>
+  <!-- <link name = "battery_1"> -->
+  <!--   <inertial> -->
+  <!--     <mass value = "0.108" /> -->
+  <!--     <origin xyz="0 0 0" rpy="0 0 0"/> -->
+  <!--     <inertia -->
+  <!--         ixx="0.0" ixy="0.0" ixz="0.0" -->
+  <!--         iyy="0.0002" iyz="0.0" izz="0.0002"/> -->
+  <!--   </inertial> -->
+  <!--   <visual> -->
+  <!--     <origin rpy="0 0 0" xyz="0 0 0"/> -->
+  <!--     <geometry> -->
+  <!--       <mesh filename="package://hugmy/urdf/mesh/4S_1300mAh_battery.STL"/> -->
+  <!--       <box size="0.29 0.34 0.070" /> -->
+  <!--     </geometry> -->
+  <!--   </visual> -->
+  <!-- </link> -->
+  <joint name="battery_0_joint" type="fixed">
+      <parent link="main_body"/>
+      <child link="battery_0"/>
+      <origin rpy="0 0 ${-pi/4}" xyz="0.01202 0.01202 -0.0365"/>
+  </joint>
+  <joint name="battery_1_joint" type="fixed">
+      <parent link="main_body"/>
+      <child link="battery_1"/>
+      <origin rpy="0 0 ${-pi/4}" xyz="-0.01202 -0.01202 -0.0365"/>
+  </joint>
+  <!-- <joint name="battery_1_joint" type="fixed"> -->
+  <!--     <parent link="main_body"/> -->
+  <!--     <child link="battery_1"/> -->
+  <!--     <origin rpy="0 0 ${-pi/4}" xyz="-0.01025 -0.01025 -0.045"/> -->
+  <!-- </joint> -->
   <!-- propellers -->
   <xacro:propeller_module id = "1" x = "${rotor_x}" y = "${-rotor_y}" z = "${rotor_z}" direction = "-1" />

Commit message: change the battery from 1000mAh to 1300mAh

File: robots/hugmy/urdf/robot.urdf.xacro (robot description, xacro)
@@ -148,67 +148,88 @@
   <!--   </inertial> -->
   <!-- </xacro:extra_module> -->
-  <link name = "battery_0">
-    <inertial>
-      <mass value = "0.108" />
-      <origin xyz="0 0 0" rpy="0 0 0"/>
-      <inertia
-          ixx="0.00001517" ixy="0.0" ixz="0.0"
-          iyy="0.00005450" iyz="0.0" izz="0.00004886"/>
-    </inertial>
-    <visual>
-      <origin rpy="0 0 0" xyz="0 0 0"/>
-      <geometry>
-        <mesh filename="package://hugmy/urdf/mesh/4S_1000mAh_battery.STL"/>
-        <box size="0.29 0.34 0.070" />
-      </geometry>
-    </visual>
-  </link>
-    <link name = "battery_1">
-    <inertial>
-      <mass value = "0.108" />
-      <origin xyz="0 0 0" rpy="0 0 0"/>
-      <inertia
-          ixx="0.00001517" ixy="0.0" ixz="0.0"
-          iyy="0.00005450" iyz="0.0" izz="0.00004886"/>
-    </inertial>
-    <visual>
-      <origin rpy="0 0 0" xyz="0 0 0"/>
-      <geometry>
-        <mesh filename="package://hugmy/urdf/mesh/4S_1000mAh_battery.STL"/>
-        <box size="0.070 0.023 0.034" />
-      </geometry>
-    </visual>
-  </link>
-  <!-- <link name = "battery_1"> -->
+  <!-- <link name = "battery_0"> -->
   <!--   <inertial> -->
   <!--     <mass value = "0.108" /> -->
   <!--     <origin xyz="0 0 0" rpy="0 0 0"/> -->
   <!--     <inertia -->
-  <!--         ixx="0.0" ixy="0.0" ixz="0.0" -->
-  <!--         iyy="0.0002" iyz="0.0" izz="0.0002"/> -->
+  <!--         ixx="0.00001517" ixy="0.0" ixz="0.0" -->
+  <!--         iyy="0.00005450" iyz="0.0" izz="0.00004886"/> -->
   <!--   </inertial> -->
   <!--   <visual> -->
   <!--     <origin rpy="0 0 0" xyz="0 0 0"/> -->
   <!--     <geometry> -->
-  <!--       <mesh filename="package://hugmy/urdf/mesh/4S_1300mAh_battery.STL"/> -->
+  <!--       <mesh filename="package://hugmy/urdf/mesh/4S_1000mAh_battery.STL"/> -->
   <!--       <box size="0.29 0.34 0.070" /> -->
   <!--     </geometry> -->
   <!--   </visual> -->
   <!-- </link> -->
+  <!--   <link name = "battery_1"> -->
+  <!--   <inertial> -->
+  <!--     <mass value = "0.108" /> -->
+  <!--     <origin xyz="0 0 0" rpy="0 0 0"/> -->
+  <!--     <inertia -->
+  <!--         ixx="0.00001517" ixy="0.0" ixz="0.0" -->
+  <!--         iyy="0.00005450" iyz="0.0" izz="0.00004886"/> -->
+  <!--   </inertial> -->
+  <!--   <visual> -->
+  <!--     <origin rpy="0 0 0" xyz="0 0 0"/> -->
+  <!--     <geometry> -->
+  <!--       <mesh filename="package://hugmy/urdf/mesh/4S_1000mAh_battery.STL"/> -->
+  <!--       <box size="0.070 0.023 0.034" /> -->
+  <!--     </geometry> -->
+  <!--   </visual> -->
+  <!-- </link> -->
+  <link name = "battery_0">
+    <inertial>
+      <mass value = "0.134" />
+      <origin xyz="0 0 0" rpy="0 0 0"/>
+      <inertia
+          ixx="0.00001517" ixy="0.0" ixz="0.0"
+	  iyy="0.00005450" iyz="0.0" izz="0.00004886"/>
+    </inertial>
+    <visual>
+      <origin rpy="0 0 0" xyz="0 0 0"/>
+      <geometry>
+        <mesh filename="package://hugmy/urdf/mesh/4S_1300mAh_battery.STL"/>
+        <box size="0.29 0.34 0.070" />
+      </geometry>
+    </visual>
+  </link>
+  <link name = "battery_1">
+    <inertial>
+      <mass value = "0.134" />
+      <origin xyz="0 0 0" rpy="0 0 0"/>
+      <inertia
+	  ixx="0.00001517" ixy="0.0" ixz="0.0"
+	  iyy="0.00005450" iyz="0.0" izz="0.00004886"/>
+    </inertial>
+    <visual>
+      <origin rpy="0 0 0" xyz="0 0 0"/>
+      <geometry>
+        <mesh filename="package://hugmy/urdf/mesh/4S_1300mAh_battery.STL"/>
+        <box size="0.29 0.34 0.070" />
+      </geometry>
+    </visual>
+  </link>
+  <!-- <joint name="battery_0_joint" type="fixed"> -->
+  <!--     <parent link="main_body"/> -->
+  <!--     <child link="battery_0"/> -->
+  <!--     <origin rpy="0 0 ${-pi/4}" xyz="0.01202 0.01202 -0.0365"/> -->
+  <!-- </joint> -->
+  <!-- <joint name="battery_1_joint" type="fixed"> -->
+  <!--     <parent link="main_body"/> -->
+  <!--     <child link="battery_1"/> -->
+  <!--     <origin rpy="0 0 ${-pi/4}" xyz="-0.01202 -0.01202 -0.0365"/> -->
+  <!-- </joint> -->
   <joint name="battery_0_joint" type="fixed">
       <parent link="main_body"/>
       <child link="battery_0"/>
-      <origin rpy="0 0 ${-pi/4}" xyz="0.01202 0.01202 -0.0365"/>
+      <origin rpy="0 0 ${-pi/4}" xyz="0.01025 0.01025 -0.045"/>
   </joint>
   <joint name="battery_1_joint" type="fixed">
       <parent link="main_body"/>
       <child link="battery_1"/>
-      <origin rpy="0 0 ${-pi/4}" xyz="-0.01202 -0.01202 -0.0365"/>
+      <origin rpy="0 0 ${-pi/4}" xyz="-0.01025 -0.01025 -0.045"/>
   </joint>
-  <!-- <joint name="battery_1_joint" type="fixed"> -->
-  <!--     <parent link="main_body"/> -->
-  <!--     <child link="battery_1"/> -->
-  <!--     <origin rpy="0 0 ${-pi/4}" xyz="-0.01025 -0.01025 -0.045"/> -->
-  <!-- </joint> -->
   <!-- propellers -->
   <xacro:propeller_module id = "1" x = "${rotor_x}" y = "${-rotor_y}" z = "${rotor_z}" direction = "-1" />

Commit message: add robot urdf and param of hugmy with face and eye module

File: robots/hugmy/urdf/robot.urdf.xacro (robot description, xacro)
@@ -99,9 +99,8 @@
   <link name="main_body">
     <inertial>
-      <mass value = "1.176" />
       <!-- with eye module -->
+      <mass value = "1.238" />
       <!-- <origin xyz="0.0001458 -0.00117927 0.00925351" rpy="0 0 0"/> -->
-      <origin xyz="-0.00187886 -0.00015416 0.00165752" rpy="0 0 0"/>
-      <!-- with eye module -->
+      <origin xyz="0.00014259 -0.00116305 0.00198970" rpy="0 0 0"/>
       <!-- <inertia -->
       <!--     ixx="0.00915711" ixy="0.00000019" ixz="-0.00001262" -->
@@ -109,12 +108,22 @@
       <!--     izz="0.01525601"/> -->
       <inertia
-          ixx="0.00659595" ixy="-0.00000357" ixz="-0.00010985"
-          iyy="0.00674188" iyz="-0.00000027"
-          izz="0.01039566"/>
+          ixx="0.00601282" ixy="0.00000325" ixz="-0.00001709"
+          iyy="0.00596220" iyz="0.00002248"
+          izz="0.00952003"/>
+      <!-- without eye module -->
+      <!-- <mass value = "1.176" /> -->
+      <!-- <origin xyz="-0.00187886 -0.00015416 0.00165752" rpy="0 0 0"/> -->
+      <!-- <inertia -->
+      <!--     ixx="0.00659595" ixy="-0.00000357" ixz="-0.00010985" -->
+      <!--     iyy="0.00674188" iyz="-0.00000027" -->
+      <!--     izz="0.01039566"/> -->
     </inertial>
     <visual>
       <origin rpy="0 0 0" xyz="0 0 0"/>
       <geometry>
-        <mesh filename="package://hugmy/urdf/mesh/Inflatable_asm_with_all_module.STL" />
+        <!-- with eye module -->
+        <mesh filename="package://hugmy/urdf/mesh/hugmy.dae" />
+        <!-- without eye module -->
+        <!-- <mesh filename="package://hugmy/urdf/mesh/hugmy_2.dae" /> -->
       </geometry>
     </visual>
