Commit message: add morphing arm controller heading flie

File: robots/hugmy/urdf/robot_ver2.gazebo.xacro (robot description, xacro)
@@ -9,7 +9,17 @@
   <xacro:gazebo_spinal robot_name="$(arg robot_name)" />
   <gazebo reference="main_body">
-    <mu1>0.1</mu1>
-    <mu2>0.1</mu2>
+    <mu1>3.0</mu1>
+    <mu2>3.0</mu2>
   </gazebo>
+  <!-- <gazebo> -->
+  <!--   <plugin name="arm_thrust" filename="$(find hugmy)/devel/lib/libarm_thrust_plugin.so"> -->
+  <!--     <rotor_links> -->
+  <!--       <link>thrust1</link> -->
+  <!--       <link>thrust2</link> -->
+  <!--       <link>thrust3</link> -->
+  <!--       <link>thrust4</link> -->
+  <!--     </rotor_links> -->
+  <!--   </plugin> -->
+  <!-- </gazebo> -->
   <!-- link for cameras -->
   <joint name="realsence_link_joint" type="fixed">

File: robots/hugmy/urdf/robot_ver2.urdf.xacro (robot description, xacro)
@@ -118,5 +118,5 @@
       <origin rpy="0 0 0" xyz="0 0 0"/>
       <geometry>
-        <box size="0.28 0.28 0.072" />
+        <box size="0.1 0.1 0.1" />
       </geometry>
     </collision>
@@ -211,4 +211,6 @@
       <axis xyz="0 1 0"/>
       <limit lower="0" upper="0.8727" effort="10" velocity="1.0"/>
+      <!-- <dynamics damping="0.0005" friction="0.8"/> -->
+      <dynamics damping="0.002" friction="0.2"/>
     </joint>
     <joint name="joint_2_${id}" type="revolute">
@@ -218,4 +220,6 @@
       <axis xyz="0 1 0"/>
       <limit lower="0" upper="1.047" effort="10" velocity="1.0"/>
+      <!-- <dynamics damping="0.0005" friction="0.8"/> -->
+      <dynamics damping="0.002" friction="0.2"/>
     </joint>
     <joint name="joint_3_${id}" type="revolute">
@@ -225,11 +229,15 @@
       <axis xyz="0 1 0"/>
       <limit lower="0" upper="1.047" effort="10" velocity="1.0"/>
+      <!-- <dynamics damping="0.0005" friction="0.8"/> -->
+      <dynamics damping="0.002" friction="0.2"/>
     </joint>
     <joint name="joint_4_${id}" type="revolute">
       <parent link="link_rotor_${id}"/>
       <child link="link_4_${id}"/>
-    <origin rpy="0 0 0" xyz="${link_length_r} 0.00 0.00"/>
-    <axis xyz="0 1 0"/>
-    <limit lower="0" upper="1.047" effort="10" velocity="1.0"/>
+      <origin rpy="0 0 0" xyz="${link_length_r} 0.00 0.00"/>
+      <axis xyz="0 1 0"/>
+      <limit lower="0" upper="1.047" effort="10" velocity="1.0"/>
+      <!-- <dynamics damping="0.0005" friction="0.8"/> -->
+      <dynamics damping="0.002" friction="0.2"/>
     </joint>
     <joint name="joint_5_${id}" type="revolute">
