Commit message: add servo controller

File: robots/hugmy/urdf/robot_ver2.urdf.xacro (robot description, xacro)
@@ -239,5 +239,57 @@
       <axis xyz="0 1 0"/>
       <limit lower="0" upper="1.047" effort="10" velocity="1.0"/>
-    </joint>
+      <!-- <dynamics damping="0.0005" friction="0.8"/> -->
+      <dynamics damping="0.002" friction="0.2"/>
+    </joint>
+    <transmission name="joint_1_${id}_tran">
+      <type>transmission_interface/SimpleTransmission</type>
+      <joint name="joint_1_${id}">
+        <hardwareInterface>hardware_interface/EffortJointInterface</hardwareInterface>
+      </joint>
+      <actuator name="joint_1_${id}_servo">
+        <hardwareInterface>hardware_interface/EffortJointInterface</hardwareInterface>
+        <mechanicalReduction>1</mechanicalReduction>
+      </actuator>
+    </transmission>
+    <transmission name="joint_2_${id}_tran">
+      <type>transmission_interface/SimpleTransmission</type>
+      <joint name="joint_2_${id}">
+        <hardwareInterface>hardware_interface/EffortJointInterface</hardwareInterface>
+      </joint>
+      <actuator name="joint_2_${id}_servo">
+        <hardwareInterface>hardware_interface/EffortJointInterface</hardwareInterface>
+        <mechanicalReduction>1</mechanicalReduction>
+      </actuator>
+    </transmission>
+    <transmission name="joint_3_${id}_tran">
+      <type>transmission_interface/SimpleTransmission</type>
+      <joint name="joint_3_${id}">
+        <hardwareInterface>hardware_interface/EffortJointInterface</hardwareInterface>
+      </joint>
+      <actuator name="joint_3_${id}_servo">
+        <hardwareInterface>hardware_interface/EffortJointInterface</hardwareInterface>
+        <mechanicalReduction>1</mechanicalReduction>
+      </actuator>
+    </transmission>
+        <transmission name="joint_4_${id}_tran">
+      <type>transmission_interface/SimpleTransmission</type>
+      <joint name="joint_4_${id}">
+        <hardwareInterface>hardware_interface/EffortJointInterface</hardwareInterface>
+      </joint>
+      <actuator name="joint_4_${id}_servo">
+        <hardwareInterface>hardware_interface/EffortJointInterface</hardwareInterface>
+        <mechanicalReduction>1</mechanicalReduction>
+      </actuator>
+    </transmission>
+    <transmission name="joint_5_${id}_tran">
+      <type>transmission_interface/SimpleTransmission</type>
+      <joint name="joint_5_${id}">
+        <hardwareInterface>hardware_interface/EffortJointInterface</hardwareInterface>
+      </joint>
+      <actuator name="joint_5_${id}_servo">
+        <hardwareInterface>hardware_interface/EffortJointInterface</hardwareInterface>
+        <mechanicalReduction>1</mechanicalReduction>
+      </actuator>
+    </transmission>
   </xacro:macro>
   <!-- Main body links and repeated arms -->

Commit message: change the name of joints

File: robots/hugmy/urdf/robot_ver2.urdf.xacro (robot description, xacro)
@@ -45,5 +45,5 @@
     <joint name="rotor${id}" type="continuous">
       <limit effort="100.0" lower="${min_force}" upper="${max_force}" velocity="0.5"/>
-      <parent link="link_rotor_${id}"/>
+      <parent link="link_${id}_rotor"/>
       <child link="thrust${id}"/>
       <origin rpy="0 0 0" xyz="0.020 0.0175 0.0369"/>
@@ -124,5 +124,5 @@
   <xacro:macro name="arm_module" params="id base_offset">
     <!--link-->
-    <link name="link_1_${id}">
+    <link name="link_${id}_1">
       <inertial>
         <origin xyz="0.01174501 0.01750000 0.00608468" rpy="0 0 0"/>
@@ -140,5 +140,5 @@
       </visual>
     </link>
-    <link name="link_2_${id}">
+    <link name="link_${id}_2">
       <inertial>
         <origin xyz="0.01174501 0.01750000 0.00608468" rpy="0 0 0"/>
@@ -156,5 +156,5 @@
       </visual>
     </link>
-    <link name="link_rotor_${id}">
+    <link name="link_${id}_rotor">
       <inertial>
         <origin xyz="0.02005067 0.01755833 0.04034797" rpy="0 0 0"/>
@@ -172,5 +172,5 @@
       </visual>
     </link>
-    <link name="link_4_${id}">
+    <link name="link_${id}_4">
       <inertial>
         <origin xyz="0.01174501 0.01750000 0.00608468" rpy="0 0 0"/>
@@ -188,5 +188,5 @@
       </visual>
     </link>
-    <link name="link_end_${id}">
+    <link name="link_${id}_end">
       <inertial>
         <origin xyz="0.00910088 0.01750002 0.00845133" rpy="0 0 0"/>
@@ -205,7 +205,7 @@
     </link>
     <!-- joint -->
-    <joint name="joint_1_${id}" type="revolute">
+    <joint name="joint_${id}_1" type="revolute">
       <parent link="main_body"/>
-      <child link="link_1_${id}"/>
+      <child link="link_${id}_1"/>
       <origin rpy="0 0 ${pi/2 * (id+3)}" xyz="${base_offset}"/>
       <axis xyz="0 1 0"/>
@@ -214,7 +214,7 @@
       <dynamics damping="0.002" friction="0.2"/>
     </joint>
-    <joint name="joint_2_${id}" type="revolute">
-      <parent link="link_1_${id}"/>
-      <child link="link_2_${id}"/>
+    <joint name="joint_${id}_2" type="revolute">
+      <parent link="link_${id}_1"/>
+      <child link="link_${id}_2"/>
       <origin rpy="0 0 0" xyz="${link_length_n} 0.00 0.00"/>
       <axis xyz="0 1 0"/>
@@ -223,7 +223,7 @@
       <dynamics damping="0.002" friction="0.2"/>
     </joint>
-    <joint name="joint_3_${id}" type="revolute">
-      <parent link="link_2_${id}"/>
-      <child link="link_rotor_${id}"/>
+    <joint name="joint_${id}_3" type="revolute">
+      <parent link="link_${id}_2"/>
+      <child link="link_${id}_rotor"/>
       <origin rpy="0 0 0" xyz="${link_length_n} 0.00 0.00"/>
       <axis xyz="0 1 0"/>
@@ -232,7 +232,7 @@
       <dynamics damping="0.002" friction="0.2"/>
     </joint>
-    <joint name="joint_4_${id}" type="revolute">
-      <parent link="link_rotor_${id}"/>
-      <child link="link_4_${id}"/>
+    <joint name="joint_${id}_4" type="revolute">
+      <parent link="link_${id}_rotor"/>
+      <child link="link_${id}_4"/>
       <origin rpy="0 0 0" xyz="${link_length_r} 0.00 0.00"/>
       <axis xyz="0 1 0"/>
@@ -241,7 +241,7 @@
       <dynamics damping="0.002" friction="0.2"/>
     </joint>
-    <joint name="joint_5_${id}" type="revolute">
-      <parent link="link_4_${id}"/>
-      <child link="link_end_${id}"/>
+    <joint name="joint_${id}_5" type="revolute">
+      <parent link="link_${id}_4"/>
+      <child link="link_${id}_end"/>
       <origin rpy="0 0 0" xyz="${link_length_n} 0.00 0.00"/>
       <axis xyz="0 1 0"/>
@@ -250,50 +250,50 @@
       <dynamics damping="0.002" friction="0.2"/>
     </joint>
-    <transmission name="joint_1_${id}_tran">
-      <type>transmission_interface/SimpleTransmission</type>
-      <joint name="joint_1_${id}">
-        <hardwareInterface>hardware_interface/EffortJointInterface</hardwareInterface>
-      </joint>
-      <actuator name="joint_1_${id}_servo">
-        <hardwareInterface>hardware_interface/EffortJointInterface</hardwareInterface>
-        <mechanicalReduction>1</mechanicalReduction>
-      </actuator>
-    </transmission>
-    <transmission name="joint_2_${id}_tran">
-      <type>transmission_interface/SimpleTransmission</type>
-      <joint name="joint_2_${id}">
-        <hardwareInterface>hardware_interface/EffortJointInterface</hardwareInterface>
-      </joint>
-      <actuator name="joint_2_${id}_servo">
-        <hardwareInterface>hardware_interface/EffortJointInterface</hardwareInterface>
-        <mechanicalReduction>1</mechanicalReduction>
-      </actuator>
-    </transmission>
-    <transmission name="joint_3_${id}_tran">
-      <type>transmission_interface/SimpleTransmission</type>
-      <joint name="joint_3_${id}">
-        <hardwareInterface>hardware_interface/EffortJointInterface</hardwareInterface>
-      </joint>
-      <actuator name="joint_3_${id}_servo">
-        <hardwareInterface>hardware_interface/EffortJointInterface</hardwareInterface>
-        <mechanicalReduction>1</mechanicalReduction>
-      </actuator>
-    </transmission>
-        <transmission name="joint_4_${id}_tran">
-      <type>transmission_interface/SimpleTransmission</type>
-      <joint name="joint_4_${id}">
-        <hardwareInterface>hardware_interface/EffortJointInterface</hardwareInterface>
-      </joint>
-      <actuator name="joint_4_${id}_servo">
-        <hardwareInterface>hardware_interface/EffortJointInterface</hardwareInterface>
-        <mechanicalReduction>1</mechanicalReduction>
-      </actuator>
-    </transmission>
-    <transmission name="joint_5_${id}_tran">
-      <type>transmission_interface/SimpleTransmission</type>
-      <joint name="joint_5_${id}">
-        <hardwareInterface>hardware_interface/EffortJointInterface</hardwareInterface>
-      </joint>
-      <actuator name="joint_5_${id}_servo">
+    <transmission name="joint_${id}_1_tran">
+      <type>transmission_interface/SimpleTransmission</type>
+      <joint name="joint_${id}_1">
+        <hardwareInterface>hardware_interface/EffortJointInterface</hardwareInterface>
+      </joint>
+      <actuator name="joint_${id}_servo_1">
+        <hardwareInterface>hardware_interface/EffortJointInterface</hardwareInterface>
+        <mechanicalReduction>1</mechanicalReduction>
+      </actuator>
+    </transmission>
+    <transmission name="joint_${id}_2_tran">
+      <type>transmission_interface/SimpleTransmission</type>
+      <joint name="joint_${id}_2">
+        <hardwareInterface>hardware_interface/EffortJointInterface</hardwareInterface>
+      </joint>
+      <actuator name="joint_${id}_2_servo">
+        <hardwareInterface>hardware_interface/EffortJointInterface</hardwareInterface>
+        <mechanicalReduction>1</mechanicalReduction>
+      </actuator>
+    </transmission>
+    <transmission name="joint_${id}_3_tran">
+      <type>transmission_interface/SimpleTransmission</type>
+      <joint name="joint_${id}_3">
+        <hardwareInterface>hardware_interface/EffortJointInterface</hardwareInterface>
+      </joint>
+      <actuator name="joint_${id}_3_servo">
+        <hardwareInterface>hardware_interface/EffortJointInterface</hardwareInterface>
+        <mechanicalReduction>1</mechanicalReduction>
+      </actuator>
+    </transmission>
+        <transmission name="joint_${id}_4_tran">
+      <type>transmission_interface/SimpleTransmission</type>
+      <joint name="joint_${id}_4">
+        <hardwareInterface>hardware_interface/EffortJointInterface</hardwareInterface>
+      </joint>
+      <actuator name="joint_${id}_4_servo">
+        <hardwareInterface>hardware_interface/EffortJointInterface</hardwareInterface>
+        <mechanicalReduction>1</mechanicalReduction>
+      </actuator>
+    </transmission>
+    <transmission name="joint_${id}_5_tran">
+      <type>transmission_interface/SimpleTransmission</type>
+      <joint name="joint_${id}_5">
+        <hardwareInterface>hardware_interface/EffortJointInterface</hardwareInterface>
+      </joint>
+      <actuator name="joint_${id}_5_servo">
         <hardwareInterface>hardware_interface/EffortJointInterface</hardwareInterface>
         <mechanicalReduction>1</mechanicalReduction>

Commit message: fix urdf bug

File: robots/hugmy/urdf/robot_ver2.urdf.xacro (robot description, xacro)
@@ -208,5 +208,5 @@
       <parent link="main_body"/>
       <child link="link_${id}_1"/>
-      <origin rpy="0 0 ${pi/2 * (id+3)}" xyz="${base_offset}"/>
+      <origin rpy="0 0 ${-pi/4 -pi/2*(id-1)}" xyz="${base_offset}"/>
       <axis xyz="0 1 0"/>
       <limit lower="0" upper="0.8727" effort="10" velocity="1.0"/>
@@ -302,8 +302,12 @@
   </xacro:macro>
   <!-- Main body links and repeated arms -->
-  <xacro:arm_module id="1" base_offset="0.05391 -0.0175 -0.039"/>
-  <xacro:arm_module id="2" base_offset="0.0175 0.05391 -0.039"/>
-  <xacro:arm_module id="3" base_offset="-0.05391 0.0175 -0.039"/>
-  <xacro:arm_module id="4" base_offset="-0.0175 -0.05391 -0.039"/>
+  <!-- <xacro:arm_module id="1" base_offset="0.05391 -0.0175 -0.039"/> -->
+  <!-- <xacro:arm_module id="2" base_offset="0.0175 0.05391 -0.039"/> -->
+  <!-- <xacro:arm_module id="3" base_offset="-0.05391 0.0175 -0.039"/> -->
+  <!-- <xacro:arm_module id="4" base_offset="-0.0175 -0.05391 -0.039"/> -->
+  <xacro:arm_module id="1" base_offset=" 0.05391 -0.05391 -0.039"/>
+  <xacro:arm_module id="2" base_offset="-0.05391 -0.05391 -0.039"/>
+  <xacro:arm_module id="3" base_offset="-0.05391  0.05391 -0.039"/>
+  <xacro:arm_module id="4" base_offset=" 0.05391  0.05391 -0.039"/>
   <!-- spinal -->
   <xacro:extra_module name = "fc" parent = "main_body" visible = "0" >

Commit message: fix urdf model

File: robots/hugmy/urdf/robot_ver2.urdf.xacro (robot description, xacro)
@@ -47,5 +47,5 @@
       <parent link="link_${id}_rotor"/>
       <child link="thrust${id}"/>
-      <origin rpy="0 0 0" xyz="0.020 0.0175 0.0369"/>
+      <origin rpy="0 0 0" xyz="-0.020 0.000 0.0369"/>
       <!-- <origin rpy="0 0 0" xyz="${x} ${y} ${z}"/> -->
       <axis xyz="0 0 ${direction}"/>
@@ -126,15 +126,15 @@
     <link name="link_${id}_1">
       <inertial>
-        <origin xyz="0.01174501 0.01750000 0.00608468" rpy="0 0 0"/>
-        <mass value="0.00752930"/>
-        <inertia
-            ixx="0.00000411" ixy="0.00000155" ixz="0.00000051"
-            iyy="0.00000214" iyz="0.00000080"
-            izz="0.00000483"/>
-      </inertial>
-      <visual>
-        <origin rpy="0 0 0" xyz="0 0 0"/>
-        <geometry>
-        <mesh filename="package://hugmy/urdf/mesh/cable_carrier_normal.dae" />
+        <origin xyz="-0.01174501 0.0000000 0.00608468" rpy="0 0 0"/>
+        <mass value="0.00639991"/>
+        <inertia
+            ixx="0.00000153" ixy="0.00000000" ixz="-0.00000044"
+            iyy="0.00000182" iyz="0.00000000"
+            izz="0.00000214"/>
+      </inertial>
+      <visual>
+        <origin rpy="0 0 0" xyz="0 0 0"/>
+        <geometry>
+        <mesh filename="package://hugmy/urdf/mesh/cable_carrier_2.STL" />
         </geometry>
       </visual>
@@ -142,15 +142,15 @@
     <link name="link_${id}_2">
       <inertial>
-        <origin xyz="0.01174501 0.01750000 0.00608468" rpy="0 0 0"/>
-        <mass value="0.00752930"/>
-        <inertia
-            ixx="0.00000411" ixy="0.00000155" ixz="0.00000051"
-            iyy="0.00000214" iyz="0.00000080"
-            izz="0.00000483"/>
-      </inertial>
-      <visual>
-        <origin rpy="0 0 0" xyz="0 0 0"/>
-        <geometry>
-          <mesh filename="package://hugmy/urdf/mesh/cable_carrier_normal.dae" />
+        <origin xyz="-0.01174501 0.0000000 0.00608468" rpy="0 0 0"/>
+        <mass value="0.00639991"/>
+        <inertia
+            ixx="0.00000153" ixy="0.00000000" ixz="-0.00000044"
+            iyy="0.00000182" iyz="0.00000000"
+            izz="0.00000214"/>
+      </inertial>
+      <visual>
+        <origin rpy="0 0 0" xyz="0 0 0"/>
+        <geometry>
+        <mesh filename="package://hugmy/urdf/mesh/cable_carrier_2.STL" />
         </geometry>
       </visual>
@@ -158,10 +158,10 @@
     <link name="link_${id}_rotor">
       <inertial>
-        <origin xyz="0.02005067 0.01755833 0.04034797" rpy="0 0 0"/>
-        <mass value="0.11565729"/>
-        <inertia
-            ixx="0.00042229" ixy="0.00004075" ixz="0.00009327"
-            iyy="0.00043336" iyz="0.00008185"
-            izz="0.00034957"/>
+        <origin xyz="-0.01937864 -0.00057405 0.04048424" rpy="0 0 0"/>
+        <mass value="0.07114866"/>
+        <inertia
+            ixx="0.00026540" ixy="0.00000193" ixz="-0.00005391"
+            iyy="0.00029155" iyz="-0.00000277"
+            izz="0.00022726"/>
       </inertial>
       <visual>
@@ -174,15 +174,15 @@
     <link name="link_${id}_4">
       <inertial>
-        <origin xyz="0.01174501 0.01750000 0.00608468" rpy="0 0 0"/>
-        <mass value="0.00752930"/>
-        <inertia
-            ixx="0.00000411" ixy="0.00000155" ixz="0.00000051"
-            iyy="0.00000214" iyz="0.00000080"
-            izz="0.00000483"/>
-      </inertial>
-      <visual>
-        <origin rpy="0 0 0" xyz="0 0 0"/>
-        <geometry>
-        <mesh filename="package://hugmy/urdf/mesh/cable_carrier_normal.dae" />
+        <origin xyz="-0.01174501 0.0000000 0.00608468" rpy="0 0 0"/>
+        <mass value="0.00639991"/>
+        <inertia
+            ixx="0.00000153" ixy="0.00000000" ixz="-0.00000044"
+            iyy="0.00000182" iyz="0.00000000"
+            izz="0.00000214"/>
+      </inertial>
+      <visual>
+        <origin rpy="0 0 0" xyz="0 0 0"/>
+        <geometry>
+          <mesh filename="package://hugmy/urdf/mesh/cable_carrier_2.STL" />
         </geometry>
       </visual>
@@ -190,15 +190,15 @@
     <link name="link_${id}_end">
       <inertial>
-        <origin xyz="0.00910088 0.01750002 0.00845133" rpy="0 0 0"/>
-        <mass value="0.00505969"/>
-        <inertia
-            ixx="0.00000287" ixy="0.00000081" ixz="0.00000044"
-            iyy="0.00000126" iyz="0.00000075"
-          izz="0.00000283"/>
+        <origin xyz="-0.00910082 0.000000 0.00845129" rpy="0 0 0"/>
+        <mass value="0.00430071"/>
+        <inertia
+            ixx="0.00000112" ixy="0.00000000" ixz="-0.00000037"
+            iyy="0.00000107" iyz="0.00000000"
+            izz="0.00000109"/>
       </inertial>
     <visual>
       <origin rpy="0 0 0" xyz="0 0 0"/>
       <geometry>
-        <mesh filename="package://hugmy/urdf/mesh/cable_carrier_end.dae" />
+        <mesh filename="package://hugmy/urdf/mesh/cable_carrier_arm_end.STL" />
       </geometry>
     </visual>
@@ -208,6 +208,6 @@
       <parent link="main_body"/>
       <child link="link_${id}_1"/>
-      <origin rpy="0 0 ${-pi/4 -pi/2*(id-1)}" xyz="${base_offset}"/>
-      <axis xyz="0 1 0"/>
+      <origin rpy="0 0 ${3*pi/4 - pi/2*(id-1)}" xyz="${base_offset}"/>
+      <axis xyz="0 -1 0"/>
       <limit lower="0" upper="0.8727" effort="10" velocity="1.0"/>
       <!-- <dynamics damping="0.0005" friction="0.8"/> -->
@@ -217,6 +217,6 @@
       <parent link="link_${id}_1"/>
       <child link="link_${id}_2"/>
-      <origin rpy="0 0 0" xyz="${link_length_n} 0.00 0.00"/>
-      <axis xyz="0 1 0"/>
+      <origin rpy="0 0 0" xyz="-${link_length_n} 0.00 0.00"/>
+      <axis xyz="0 -1 0"/>
       <limit lower="0" upper="1.047" effort="10" velocity="1.0"/>
       <!-- <dynamics damping="0.0005" friction="0.8"/> -->
@@ -226,6 +226,6 @@
       <parent link="link_${id}_2"/>
       <child link="link_${id}_rotor"/>
-      <origin rpy="0 0 0" xyz="${link_length_n} 0.00 0.00"/>
-      <axis xyz="0 1 0"/>
+      <origin rpy="0 0 0" xyz="-${link_length_n} 0.00 0.00"/>
+      <axis xyz="0 -1 0"/>
       <limit lower="0" upper="1.047" effort="10" velocity="1.0"/>
       <!-- <dynamics damping="0.0005" friction="0.8"/> -->
@@ -235,6 +235,6 @@
       <parent link="link_${id}_rotor"/>
       <child link="link_${id}_4"/>
-      <origin rpy="0 0 0" xyz="${link_length_r} 0.00 0.00"/>
-      <axis xyz="0 1 0"/>
+      <origin rpy="0 0 0" xyz="-${link_length_r} 0.00 0.00"/>
+      <axis xyz="0 -1 0"/>
       <limit lower="0" upper="1.047" effort="10" velocity="1.0"/>
       <!-- <dynamics damping="0.0005" friction="0.8"/> -->
@@ -244,6 +244,6 @@
       <parent link="link_${id}_4"/>
       <child link="link_${id}_end"/>
-      <origin rpy="0 0 0" xyz="${link_length_n} 0.00 0.00"/>
-      <axis xyz="0 1 0"/>
+      <origin rpy="0 0 0" xyz="-${link_length_n} 0.00 0.00"/>
+      <axis xyz="0 -1 0"/>
       <limit lower="0" upper="1.047" effort="10" velocity="1.0"/>
       <!-- <dynamics damping="0.0005" friction="0.8"/> -->
@@ -306,8 +306,8 @@
   <!-- <xacro:arm_module id="3" base_offset="-0.05391 0.0175 -0.039"/> -->
   <!-- <xacro:arm_module id="4" base_offset="-0.0175 -0.05391 -0.039"/> -->
-  <xacro:arm_module id="1" base_offset=" 0.05391 -0.05391 -0.039"/>
-  <xacro:arm_module id="2" base_offset="-0.05391 -0.05391 -0.039"/>
-  <xacro:arm_module id="3" base_offset="-0.05391  0.05391 -0.039"/>
-  <xacro:arm_module id="4" base_offset=" 0.05391  0.05391 -0.039"/>
+  <xacro:arm_module id="1" base_offset=" 0.03812 -0.03812 -0.039"/>
+  <xacro:arm_module id="2" base_offset="-0.03812 -0.03812 -0.039"/>
+  <xacro:arm_module id="3" base_offset="-0.03812  0.03812 -0.039"/>
+  <xacro:arm_module id="4" base_offset=" 0.03812  0.03812 -0.039"/>
   <!-- spinal -->
   <xacro:extra_module name = "fc" parent = "main_body" visible = "0" >

Commit message: add main body with face

File: robots/hugmy/urdf/robot_ver2.urdf.xacro (robot description, xacro)
@@ -100,17 +100,40 @@
   </joint>
   <!-- main_body -->
+  <!-- <link name="main_body"> -->
+  <!--   <inertial> -->
+  <!--     <mass value = "0.698" /> -->
+  <!--     <origin xyz="0.00110883 0.00011825 0.00012320" rpy="0 0 0"/> -->
+  <!--     <inertia -->
+  <!--         ixx="0.00145773" ixy="-0.00000588" ixz="0.00002143" -->
+  <!--         iyy="0.00150029" iyz="-0.00004262" -->
+  <!--         izz="0.00061796"/> -->
+  <!--   </inertial> -->
+  <!--   <visual> -->
+  <!--     <origin rpy="0 0 0" xyz="0 0 0"/> -->
+  <!--     <geometry> -->
+  <!--       <mesh filename="package://hugmy/urdf/mesh/Inflatable_asm.STL" /> -->
+  <!--     </geometry> -->
+  <!--   </visual> -->
+  <!--   <collision> -->
+  <!--     <origin rpy="0 0 0" xyz="0 0 0"/> -->
+  <!--     <geometry> -->
+  <!--       <box size="0.1 0.1 0.1" /> -->
+  <!--     </geometry> -->
+  <!--   </collision> -->
+  <!-- </link> -->
+  <!-- main_body with face-->
   <link name="main_body">
     <inertial>
-      <mass value = "0.698" />
-      <origin xyz="0.00110883 0.00011825 0.00012320" rpy="0 0 0"/>
+      <mass value = "0.92157932" />
+      <origin xyz="-0.00348932 0.00065510 0.01200916" rpy="0 0 0"/>
       <inertia
-          ixx="0.00145773" ixy="-0.00000588" ixz="0.00002143"
-          iyy="0.00150029" iyz="-0.00004262"
-          izz="0.00061796"/>
+          ixx="0.00296732" ixy="-0.00002177" ixz="-0.00023771"
+          iyy="0.00303063" iyz="0.00005805"
+          izz="0.00110707"/>
     </inertial>
     <visual>
       <origin rpy="0 0 0" xyz="0 0 0"/>
       <geometry>
-        <mesh filename="package://hugmy/urdf/mesh/Inflatable_asm.STL" />
+        <mesh filename="package://hugmy/urdf/mesh/body_with_face.STL" />
       </geometry>
     </visual>

Commit message: fix the precise weight

File: robots/hugmy/urdf/robot_ver2.urdf.xacro (robot description, xacro)
@@ -125,5 +125,5 @@
   <link name="main_body">
     <inertial>
-      <mass value = "0.92157932" />
+      <mass value = "1.244" />
       <origin xyz="-0.00348932 0.00065510 0.01200916" rpy="0 0 0"/>
       <inertia
