Commit message: add controllers and others

File: robots/hydrus/robots/quad/soft_airframe_202509/robot.urdf.xacro (robot description, xacro)
@@ -102,7 +102,49 @@
   <!-- end: gps -->
   <!-- 3 soft_airframe -->
-  <link name="tail_link1"/>
-  <link name="tail_link2"/>
-  <link name="tail_link3"/>
+  <link name="tail_link1">
+    <inertial>
+      <origin xyz="0 0 0" rpy="0 0 0"/>
+      <mass value="0.001"/>
+      <inertia
+          ixx="0.001" ixy="0.0" ixz="0.0"
+          iyy="0.001" iyz="0.0"
+          izz="0.002"/>
+    </inertial>
+  </link>
+  <gazebo reference="tail_link1">
+    <mu1>0.1</mu1>
+    <mu2>0.1</mu2>
+  </gazebo>
+  <xacro:damping_factor link="tail_link1"/>
+  <link name="tail_link2">
+    <inertial>
+      <origin xyz="0 0 0" rpy="0 0 0"/>
+      <mass value="0.001"/>
+      <inertia
+          ixx="0.001" ixy="0.0" ixz="0.0"
+          iyy="0.001" iyz="0.0"
+          izz="0.002"/>
+    </inertial>
+  </link>
+  <gazebo reference="tail_link2">
+    <mu1>0.1</mu1>
+    <mu2>0.1</mu2>
+  </gazebo>
+  <xacro:damping_factor link="tail_link2"/>
+  <link name="tail_link3">
+    <inertial>
+      <origin xyz="0 0 0" rpy="0 0 0"/>
+      <mass value="0.001"/>
+      <inertia
+          ixx="0.001" ixy="0.0" ixz="0.0"
+          iyy="0.001" iyz="0.0"
+          izz="0.002"/>
+    </inertial>
+  </link>
+  <gazebo reference="tail_link3">
+    <mu1>0.1</mu1>
+    <mu2>0.1</mu2>
+  </gazebo>
+  <xacro:damping_factor link="tail_link3"/>
   <joint name="tail_joint1" type="fixed">
     <parent link="link4"/>
@@ -116,5 +158,5 @@
     <origin xyz="0 0 0" rpy="0 0 0"/>
     <axis xyz="0 0 1"/>
-    <dynamics damping="0.9" friction="0.05"/>
+    <dynamics damping="0.9" friction="0.1"/>
   </joint>
   <joint name="tail_joint3" type="revolute">
@@ -124,5 +166,25 @@
     <origin xyz="0 0 0" rpy="0 0 0"/>
     <axis xyz="0 0 1"/>
-    <dynamics damping="0.9" friction="0.05"/>
+    <dynamics damping="0.9" friction="0.1"/>
   </joint>
+  <transmission name="tail_joint_tran_2">
+    <type>transmission_interface/SimpleTransmission</type>
+    <joint name="tail_joint2">
+      <hardwareInterface>hardware_interface/EffortJointInterface</hardwareInterface>
+    </joint>
+    <actuator name="tail_joint_servo2">
+      <hardwareInterface>hardware_interface/EffortJointInterface</hardwareInterface>
+      <mechanicalReduction>1</mechanicalReduction>
+    </actuator>
+  </transmission>
+  <transmission name="tail_joint_tran_3">
+    <type>transmission_interface/SimpleTransmission</type>
+    <joint name="tail_joint3">
+      <hardwareInterface>hardware_interface/EffortJointInterface</hardwareInterface>
+    </joint>
+    <actuator name="tail_joint_servo3">
+      <hardwareInterface>hardware_interface/EffortJointInterface</hardwareInterface>
+      <mechanicalReduction>1</mechanicalReduction>
+    </actuator>
+  </transmission>
 </robot>

Commit message: added gimbal and rotor

File: robots/hydrus/robots/quad/soft_airframe_202509/robot.urdf.xacro (robot description, xacro)
@@ -102,7 +102,7 @@
   <!-- end: gps -->
   <!-- 3 soft_airframe -->
-  <link name="tail_link1">
-    <inertial>
-      <origin xyz="0 0 0" rpy="0 0 0"/>
+  <link name="soft_link1">
+    <inertial>
+      <origin xyz="${0.3 + 0.038190} 0.0 0.010950" rpy="0 0 0"/>
       <mass value="0.001"/>
       <inertia
@@ -112,10 +112,10 @@
     </inertial>
   </link>
-  <gazebo reference="tail_link1">
+  <gazebo reference="soft_link1">
     <mu1>0.1</mu1>
     <mu2>0.1</mu2>
   </gazebo>
-  <xacro:damping_factor link="tail_link1"/>
-  <link name="tail_link2">
+  <xacro:damping_factor link="soft_link1"/>
+  <link name="soft_link2">
     <inertial>
       <origin xyz="0 0 0" rpy="0 0 0"/>
@@ -127,10 +127,10 @@
     </inertial>
   </link>
-  <gazebo reference="tail_link2">
+  <gazebo reference="soft_link2">
     <mu1>0.1</mu1>
     <mu2>0.1</mu2>
   </gazebo>
-  <xacro:damping_factor link="tail_link2"/>
-  <link name="tail_link3">
+  <xacro:damping_factor link="soft_link2"/>
+  <link name="soft_link3">
     <inertial>
       <origin xyz="0 0 0" rpy="0 0 0"/>
@@ -142,46 +142,123 @@
     </inertial>
   </link>
-  <gazebo reference="tail_link3">
+  <gazebo reference="soft_link3">
     <mu1>0.1</mu1>
     <mu2>0.1</mu2>
   </gazebo>
-  <xacro:damping_factor link="tail_link3"/>
-  <joint name="tail_joint1" type="fixed">
+  <xacro:damping_factor link="soft_link3"/>
+  <joint name="soft_joint1" type="fixed">
     <parent link="link4"/>
-    <child link="tail_link1"/>
-    <origin xyz="0 0 0.5" rpy="0 0 0"/>
-  </joint>
-  <joint name="tail_joint2" type="revolute">
+    <child link="soft_link1"/>
+    <origin xyz="0.6 0 0.1" rpy="0 0 0"/>
+  </joint>
+  <joint name="soft_joint2" type="revolute">
     <limit effort="10.0" lower="${-pi/2}" upper="${pi/2}" velocity="0.5"/>
-    <parent link="tail_link1"/>
-    <child link="tail_link2"/>
-    <origin xyz="0 0 0" rpy="0 0 0"/>
+    <parent link="soft_link1"/>
+    <child link="soft_link2"/>
+    <origin xyz="0.1175 0 0" rpy="0 0 0"/>
     <axis xyz="0 0 1"/>
     <dynamics damping="0.9" friction="0.1"/>
   </joint>
-  <joint name="tail_joint3" type="revolute">
+  <joint name="soft_joint3" type="revolute">
     <limit effort="10.0" lower="${-pi/2}" upper="${pi/2}" velocity="0.5"/>
-    <parent link="tail_link2"/>
-    <child link="tail_link3"/>
-    <origin xyz="0 0 0" rpy="0 0 0"/>
+    <parent link="soft_link2"/>
+    <child link="soft_link3"/>
+    <origin xyz="0.235 0 0" rpy="0 0 0"/>
     <axis xyz="0 0 1"/>
     <dynamics damping="0.9" friction="0.1"/>
   </joint>
-  <transmission name="tail_joint_tran_2">
-    <type>transmission_interface/SimpleTransmission</type>
-    <joint name="tail_joint2">
-      <hardwareInterface>hardware_interface/EffortJointInterface</hardwareInterface>
-    </joint>
-    <actuator name="tail_joint_servo2">
-      <hardwareInterface>hardware_interface/EffortJointInterface</hardwareInterface>
-      <mechanicalReduction>1</mechanicalReduction>
-    </actuator>
-  </transmission>
-  <transmission name="tail_joint_tran_3">
-    <type>transmission_interface/SimpleTransmission</type>
-    <joint name="tail_joint3">
-      <hardwareInterface>hardware_interface/EffortJointInterface</hardwareInterface>
-    </joint>
-    <actuator name="tail_joint_servo3">
+  <transmission name="soft_joint_tran_2">
+    <type>transmission_interface/SimpleTransmission</type>
+    <joint name="soft_joint2">
+      <hardwareInterface>hardware_interface/EffortJointInterface</hardwareInterface>
+    </joint>
+    <actuator name="soft_joint_servo2">
+      <hardwareInterface>hardware_interface/EffortJointInterface</hardwareInterface>
+      <mechanicalReduction>1</mechanicalReduction>
+    </actuator>
+  </transmission>
+  <transmission name="soft_joint_tran_3">
+    <type>transmission_interface/SimpleTransmission</type>
+    <joint name="soft_joint3">
+      <hardwareInterface>hardware_interface/EffortJointInterface</hardwareInterface>
+    </joint>
+    <actuator name="soft_joint_servo3">
+      <hardwareInterface>hardware_interface/EffortJointInterface</hardwareInterface>
+      <mechanicalReduction>1</mechanicalReduction>
+    </actuator>
+  </transmission>
+  <!-- gimbal -->
+  <joint name="gimbal_joint1" type="continuous">
+    <limit effort="100.0" lower="1.0" upper="20.0" velocity="0.5"/>
+    <parent link="soft_link3"/>
+    <child link="gimbal_link1"/>
+    <origin rpy="0 0 0" xyz="0.1595 0 0"/>
+    <axis xyz="1 0 0"/>
+    <dynamics damping="0.9" friction="0.1"/>
+  </joint>
+  <link name="gimbal_link1">
+    <inertial>
+      <origin xyz="0 0 0" rpy="0 0 0"/>
+      <mass value="0.0001"/>
+      <inertia
+          ixx="0.00001" ixy="0.0" ixz="0.0"
+          iyy="0.00001" iyz="0.0"
+          izz="0.00002"/>
+    </inertial>
+    <collision>
+      <origin rpy="0 0 0" xyz="0 0 0"/>
+      <geometry>
+        <cylinder length="0.1" radius="0.11"/>
+      </geometry>
+    </collision>
+    <!-- <visual>
+      <origin rpy="0 0 0" xyz="0 0 0.032"/>
+    </visual> -->
+  </link>
+  <xacro:damping_factor link ="gimbal_link1"/>
+  <transmission name="gimbal_tran1">
+    <type>transmission_interface/SimpleTransmission</type>
+    <joint name="gimbal_joint1">
+      <hardwareInterface>hardware_interface/EffortJointInterface</hardwareInterface>
+    </joint>
+    <actuator name="gimbal_servo1">
+      <hardwareInterface>hardware_interface/EffortJointInterface</hardwareInterface>
+      <mechanicalReduction>1</mechanicalReduction>
+    </actuator>
+  </transmission>
+  <!-- rotor -->
+  <joint name="rotor5" type="continuous">
+    <limit effort="100.0" lower="1.0" upper="20.0" velocity="0.5"/>
+    <parent link="gimbal_link1"/>
+    <child link="thrust5"/>
+    <origin rpy="0 0 0" xyz="0.0735 0 0"/>
+    <axis xyz="0 0 1"/>
+  </joint>
+  <link name="thrust5">
+    <inertial>
+      <origin xyz="0 0 0" rpy="0 0 0"/>
+      <mass value="0.0001"/>
+      <inertia
+          ixx="0.00001" ixy="0.0" ixz="0.0"
+          iyy="0.00001" iyz="0.0"
+          izz="0.00002"/>
+    </inertial>
+    <collision>
+      <origin rpy="0 0 0" xyz="0 0 0"/>
+      <geometry>
+        <cylinder length="0.1" radius="0.11"/>
+      </geometry>
+    </collision>
+    <!-- <visual>
+      <origin rpy="0 0 0" xyz="0 0 0.032"/>
+    </visual> -->
+  </link>
+  <xacro:damping_factor link ="thrust5"/>
+  <transmission name="rotor_tran5">
+    <type>transmission_interface/SimpleTransmission</type>
+    <joint name="rotor5">
+      <hardwareInterface>hardware_interface/EffortJointInterface</hardwareInterface>
+    </joint>
+    <actuator name="rotor5">
       <hardwareInterface>hardware_interface/EffortJointInterface</hardwareInterface>
       <mechanicalReduction>1</mechanicalReduction>

Commit message: wip

File: robots/hydrus/robots/quad/soft_airframe_202509/robot.urdf.xacro (robot description, xacro)
@@ -104,10 +104,20 @@
   <link name="soft_link1">
     <inertial>
-      <origin xyz="${0.3 + 0.038190} 0.0 0.010950" rpy="0 0 0"/>
-      <mass value="0.001"/>
-      <inertia
-          ixx="0.001" ixy="0.0" ixz="0.0"
-          iyy="0.001" iyz="0.0"
-          izz="0.002"/>
+      <origin xyz="0.06875 0.000002 0.018960" rpy="0 0 0"/>
+      <mass value="${0.010*2 + 0.012}"/>
+      <!-- this is the original -->
+      <!-- <inertia
+          ixx="0.000064" ixy="0.0" ixz="0.000004"
+          iyy="0.0001555" iyz="0.0"
+          izz="0.000154"/> -->
+      <inertia
+          ixx="${0.00007117961/2}" ixy="0.0" ixz="0.000004"
+          iyy="${0.00017932677/2}" iyz="0.0"
+          izz="${0.00045111519/2}"/>
+      <!-- this one works -->
+      <!-- <inertia
+          ixx="0.001804" ixy="0.000021" ixz="0.000372"
+          iyy="0.017972"  iyz="0.000000"
+          izz="0.019248"/> -->
     </inertial>
   </link>
@@ -119,10 +129,21 @@
   <link name="soft_link2">
     <inertial>
-      <origin xyz="0 0 0" rpy="0 0 0"/>
-      <mass value="0.001"/>
-      <inertia
-          ixx="0.001" ixy="0.0" ixz="0.0"
-          iyy="0.001" iyz="0.0"
-          izz="0.002"/>
+      <origin xyz="0.1175 0.000002 0.019998" rpy="0 0 0"/>
+      <mass value="${0.010*5 + 0.012*2}"/>
+      <!-- <inertia
+          ixx="0.000123" ixy="0.0" ixz="0.0"
+          iyy="0.001" iyz="0.000758"
+          izz="0.000758"/> -->
+      <inertia
+          ixx="${0.00012174242/2}" ixy="0.0" ixz="0.0"
+          iyy="${0.00083236110/2}" iyz="0.0"
+          izz="${0.00082463843/2}"/>
+      <!-- <inertia
+        ixx="${0.00007117961/2}" ixy="0.0" ixz="0.000004"
+        iyy="${0.00017932677/2}" iyz="0.0"
+        izz="${0.00045111519/2}"/> -->
+      <!-- <inertia
+          ixx="0.001804" iyy="0.017972" izz="0.019248"
+          ixy="0.000021" ixz="0.000372" iyz="0.000000"/> -->
     </inertial>
   </link>
@@ -134,10 +155,22 @@
   <link name="soft_link3">
     <inertial>
-      <origin xyz="0 0 0" rpy="0 0 0"/>
-      <mass value="0.001"/>
-      <inertia
-          ixx="0.001" ixy="0.0" ixz="0.0"
-          iyy="0.001" iyz="0.0"
-          izz="0.002"/>
+      <origin xyz="0.10740316 0.0 0.003" rpy="0 0 0"/>
+      <mass value="${0.010*2 + 0.012 + 0.070}"/>
+      <!-- <inertia
+          ixx="0.000080" ixy="0.0" ixz="0.000027"
+          iyy="0.000357" iyz="0.0"
+          izz="0.000347"/> -->
+      <!-- the latest -->
+      <inertia
+          ixx="0.00005679" ixy="-0.000000031" ixz="-0.00002256"
+          iyy="0.00028149" iyz="0.000000005"
+          izz="0.00026759"/>
+      <!-- <inertia
+          ixx="${0.00012174242/2}" ixy="0.0" ixz="0.0"
+          iyy="${0.00083236110/2}" iyz="0.0"
+          izz="${0.00082463843/2}"/> -->
+      <!-- <inertia
+          ixx="0.001804" iyy="0.017972" izz="0.019248"
+          ixy="0.000021" ixz="0.000372" iyz="0.000000"/> -->
     </inertial>
   </link>
@@ -150,5 +183,5 @@
     <parent link="link4"/>
     <child link="soft_link1"/>
-    <origin xyz="0.6 0 0.1" rpy="0 0 0"/>
+    <origin xyz="0.6 0 0" rpy="0 0 0"/>
   </joint>
   <joint name="soft_joint2" type="revolute">
@@ -189,5 +222,5 @@
   </transmission>
   <!-- gimbal -->
-  <joint name="gimbal_joint1" type="continuous">
+  <!-- <joint name="gimbal_joint1" type="continuous">
     <limit effort="100.0" lower="1.0" upper="20.0" velocity="0.5"/>
     <parent link="soft_link3"/>
@@ -199,4 +232,45 @@
   <link name="gimbal_link1">
     <inertial>
+      <origin xyz="0.0815 0 0" rpy="0 0 0"/>
+      <mass value="0.159380"/>
+      <inertia
+          ixx="0.000171" ixy="0.0" ixz="0.0"
+          iyy="0.000244" iyz="0.0"
+          izz="0.000336"/>
+    </inertial>
+    <collision>
+      <origin xyz="0.0815 0 0" rpy="0 0 0"/>
+      <geometry>
+        <cylinder length="0.1" radius="0.11"/>
+      </geometry>
+    </collision>
+    <visual>
+      <origin xyz="0.0815 0 0" rpy="0 0 0"/>
+      <geometry>
+        <mesh filename="package://hydrus/urdf/mesh/propeller/5inch_propeller_duct_right_v2.dae"/>
+      </geometry>
+    </visual>
+  </link>
+  <xacro:damping_factor link ="gimbal_link1"/>
+  <transmission name="gimbal_tran1">
+    <type>transmission_interface/SimpleTransmission</type>
+    <joint name="gimbal_joint1">
+      <hardwareInterface>hardware_interface/EffortJointInterface</hardwareInterface>
+    </joint>
+    <actuator name="gimbal_servo1">
+      <hardwareInterface>hardware_interface/EffortJointInterface</hardwareInterface>
+      <mechanicalReduction>1</mechanicalReduction>
+    </actuator>
+  </transmission> -->
+  <!-- rotor -->
+  <!-- <joint name="rotor5" type="continuous">
+    <limit effort="100.0" lower="1.0" upper="20.0" velocity="0.5"/>
+    <parent link="gimbal_link1"/>
+    <child link="thrust5"/>
+    <origin rpy="0 0 0" xyz="0.0735 0 0"/>
+    <axis xyz="0 0 1"/>
+  </joint>
+  <link name="thrust5">
+    <inertial>
       <origin xyz="0 0 0" rpy="0 0 0"/>
       <mass value="0.0001"/>
@@ -212,45 +286,10 @@
       </geometry>
     </collision>
-    <!-- <visual>
-      <origin rpy="0 0 0" xyz="0 0 0.032"/>
-    </visual> -->
-  </link>
-  <xacro:damping_factor link ="gimbal_link1"/>
-  <transmission name="gimbal_tran1">
-    <type>transmission_interface/SimpleTransmission</type>
-    <joint name="gimbal_joint1">
-      <hardwareInterface>hardware_interface/EffortJointInterface</hardwareInterface>
-    </joint>
-    <actuator name="gimbal_servo1">
-      <hardwareInterface>hardware_interface/EffortJointInterface</hardwareInterface>
-      <mechanicalReduction>1</mechanicalReduction>
-    </actuator>
-  </transmission>
-  <!-- rotor -->
-  <joint name="rotor5" type="continuous">
-    <limit effort="100.0" lower="1.0" upper="20.0" velocity="0.5"/>
-    <parent link="gimbal_link1"/>
-    <child link="thrust5"/>
-    <origin rpy="0 0 0" xyz="0.0735 0 0"/>
-    <axis xyz="0 0 1"/>
-  </joint>
-  <link name="thrust5">
-    <inertial>
-      <origin xyz="0 0 0" rpy="0 0 0"/>
-      <mass value="0.0001"/>
-      <inertia
-          ixx="0.00001" ixy="0.0" ixz="0.0"
-          iyy="0.00001" iyz="0.0"
-          izz="0.00002"/>
-    </inertial>
-    <collision>
-      <origin rpy="0 0 0" xyz="0 0 0"/>
+    <visual>
+      <origin rpy="${pi/2} 0 0" xyz="-0.045 0.055 0.06"/>
       <geometry>
-        <cylinder length="0.1" radius="0.11"/>
+        <mesh filename="package://hydrus/urdf/mesh/propeller/TriBlade_5045.dae"/>
       </geometry>
-    </collision>
-    <!-- <visual>
-      <origin rpy="0 0 0" xyz="0 0 0.032"/>
-    </visual> -->
+    </visual>
   </link>
   <xacro:damping_factor link ="thrust5"/>
@@ -264,4 +303,4 @@
       <mechanicalReduction>1</mechanicalReduction>
     </actuator>
-  </transmission>
+  </transmission> -->
 </robot>

Commit message: worked in gazebo

File: robots/hydrus/robots/quad/soft_airframe_202509/robot.urdf.xacro (robot description, xacro)
@@ -106,18 +106,8 @@
       <origin xyz="0.06875 0.000002 0.018960" rpy="0 0 0"/>
       <mass value="${0.010*2 + 0.012}"/>
-      <!-- this is the original -->
-      <!-- <inertia
-          ixx="0.000064" ixy="0.0" ixz="0.000004"
-          iyy="0.0001555" iyz="0.0"
-          izz="0.000154"/> -->
-      <inertia
-          ixx="${0.00007117961/2}" ixy="0.0" ixz="0.000004"
-          iyy="${0.00017932677/2}" iyz="0.0"
-          izz="${0.00045111519/2}"/>
-      <!-- this one works -->
-      <!-- <inertia
-          ixx="0.001804" ixy="0.000021" ixz="0.000372"
-          iyy="0.017972"  iyz="0.000000"
-          izz="0.019248"/> -->
+      <inertia
+          ixx="0.00003988" ixy="0.0" ixz="0.0"
+          iyy="0.00010606" iyz="0.0"
+          izz="0.00010185"/>
     </inertial>
   </link>
@@ -131,19 +121,8 @@
       <origin xyz="0.1175 0.000002 0.019998" rpy="0 0 0"/>
       <mass value="${0.010*5 + 0.012*2}"/>
-      <!-- <inertia
-          ixx="0.000123" ixy="0.0" ixz="0.0"
-          iyy="0.001" iyz="0.000758"
-          izz="0.000758"/> -->
-      <inertia
-          ixx="${0.00012174242/2}" ixy="0.0" ixz="0.0"
-          iyy="${0.00083236110/2}" iyz="0.0"
-          izz="${0.00082463843/2}"/>
-      <!-- <inertia
-        ixx="${0.00007117961/2}" ixy="0.0" ixz="0.000004"
-        iyy="${0.00017932677/2}" iyz="0.0"
-        izz="${0.00045111519/2}"/> -->
-      <!-- <inertia
-          ixx="0.001804" iyy="0.017972" izz="0.019248"
-          ixy="0.000021" ixz="0.000372" iyz="0.000000"/> -->
+      <inertia
+          ixx="0.00006787" ixy="0.0" ixz="0.0"
+          iyy="0.00049831" iyz="0.0"
+          izz="0.00048990"/>
     </inertial>
   </link>
@@ -157,20 +136,8 @@
       <origin xyz="0.10740316 0.0 0.003" rpy="0 0 0"/>
       <mass value="${0.010*2 + 0.012 + 0.070}"/>
-      <!-- <inertia
-          ixx="0.000080" ixy="0.0" ixz="0.000027"
-          iyy="0.000357" iyz="0.0"
-          izz="0.000347"/> -->
-      <!-- the latest -->
       <inertia
           ixx="0.00005679" ixy="-0.000000031" ixz="-0.00002256"
           iyy="0.00028149" iyz="0.000000005"
           izz="0.00026759"/>
-      <!-- <inertia
-          ixx="${0.00012174242/2}" ixy="0.0" ixz="0.0"
-          iyy="${0.00083236110/2}" iyz="0.0"
-          izz="${0.00082463843/2}"/> -->
-      <!-- <inertia
-          ixx="0.001804" iyy="0.017972" izz="0.019248"
-          ixy="0.000021" ixz="0.000372" iyz="0.000000"/> -->
     </inertial>
   </link>
@@ -201,4 +168,7 @@
     <dynamics damping="0.9" friction="0.1"/>
   </joint>
+  <!-- <gazebo reference="soft_link3">
+    <stopCfm>1000</stopCfm>
+  </gazebo> -->
   <transmission name="soft_joint_tran_2">
     <type>transmission_interface/SimpleTransmission</type>
@@ -221,6 +191,27 @@
     </actuator>
   </transmission>
+  <!-- leg -->
+  <!-- <link name="leg6">
+    <inertial>
+      <origin xyz="0.0 0.0 -0.093" rpy="0 0 0"/>
+      <mass value="0.047000"/>
+      <inertia
+          ixx="0.000259" iyy="0.000281" izz="0.000010"
+          ixy="0.000000" ixz="0.000000" iyz="0.000000"/>
+    </inertial>
+  </link>
+  <gazebo reference="leg6">
+    <mu1>0.1</mu1>
+    <mu2>0.1</mu2>
+  </gazebo>
+  <xacro:damping_factor link="leg6"/>
+  <joint name="leg_joint_soft1" type="fixed">
+    <parent link="soft_link3"/>
+    <child link="leg6"/>
+    <origin xyz="0.1 0 0" rpy="0 0 0"/>
+  </joint>
+ -->
   <!-- gimbal -->
-  <!-- <joint name="gimbal_joint1" type="continuous">
+  <joint name="gimbal_joint1" type="continuous">
     <limit effort="100.0" lower="1.0" upper="20.0" velocity="0.5"/>
     <parent link="soft_link3"/>
@@ -233,14 +224,16 @@
     <inertial>
       <origin xyz="0.0815 0 0" rpy="0 0 0"/>
-      <mass value="0.159380"/>
-      <inertia
-          ixx="0.000171" ixy="0.0" ixz="0.0"
-          iyy="0.000244" iyz="0.0"
-          izz="0.000336"/>
+      <mass value="0.083"/>
+      <!-- this inertia value is 10 times bigger than the real one -->
+      <!-- to avoid the instability in gazebo -->
+      <inertia
+          ixx="0.0022661" ixy="0.0" ixz="0.0"
+          iyy="0.0015451" iyz="0.0"
+          izz="0.00032533"/>
     </inertial>
     <collision>
       <origin xyz="0.0815 0 0" rpy="0 0 0"/>
       <geometry>
-        <cylinder length="0.1" radius="0.11"/>
+        <cylinder length="0.1" radius="0.05"/>
       </geometry>
     </collision>
@@ -262,7 +255,7 @@
       <mechanicalReduction>1</mechanicalReduction>
     </actuator>
-  </transmission> -->
+  </transmission>
   <!-- rotor -->
-  <!-- <joint name="rotor5" type="continuous">
+  <joint name="rotor5" type="continuous">
     <limit effort="100.0" lower="1.0" upper="20.0" velocity="0.5"/>
     <parent link="gimbal_link1"/>
@@ -303,4 +296,4 @@
       <mechanicalReduction>1</mechanicalReduction>
     </actuator>
-  </transmission> -->
+  </transmission>
 </robot>
