Commit message: worked with the real robot

File: robots/hydrus/robots/quad/soft_airframe_202509/robot.urdf.xacro (robot description, xacro)
@@ -147,4 +147,19 @@
   </gazebo>
   <xacro:damping_factor link="soft_link3"/>
+  <link name="dummy_link">
+    <inertial>
+      <origin xyz="0 0 0" rpy="0 0 0"/>
+      <mass value="0.0001"/>
+      <inertia
+          ixx="0.00001" ixy="0.0" ixz="0.0"
+          iyy="0.00001" iyz="0.0"
+          izz="0.00002"/>
+    </inertial>
+  </link>
+  <gazebo reference="dummy_link">
+    <mu1>0.1</mu1>
+    <mu2>0.1</mu2>
+  </gazebo>
+  <xacro:damping_factor link="dummy_link"/>
   <joint name="soft_joint1" type="fixed">
     <parent link="link4"/>
@@ -171,4 +186,12 @@
     <stopCfm>1000</stopCfm>
   </gazebo> -->
+  <joint name="soft_joint4" type="revolute">
+    <limit effort="10.0" lower="${-pi/2}" upper="${pi/2}" velocity="0.5"/>
+    <parent link="soft_link3"/>
+    <child link="dummy_link"/>
+    <origin xyz="0.235 0 0" rpy="0 0 0"/>
+    <axis xyz="0 0 1"/>
+    <dynamics damping="0.9" friction="0.1"/>
+  </joint>
   <transmission name="soft_joint_tran_2">
     <type>transmission_interface/SimpleTransmission</type>
@@ -187,4 +210,14 @@
     </joint>
     <actuator name="soft_joint_servo3">
+      <hardwareInterface>hardware_interface/EffortJointInterface</hardwareInterface>
+      <mechanicalReduction>1</mechanicalReduction>
+    </actuator>
+  </transmission>
+  <transmission name="soft_joint_tran_4">
+    <type>transmission_interface/SimpleTransmission</type>
+    <joint name="soft_joint4">
+      <hardwareInterface>hardware_interface/EffortJointInterface</hardwareInterface>
+    </joint>
+    <actuator name="soft_joint_servo4">
       <hardwareInterface>hardware_interface/EffortJointInterface</hardwareInterface>
       <mechanicalReduction>1</mechanicalReduction>
@@ -257,12 +290,12 @@
   </transmission>
   <!-- rotor -->
-  <joint name="rotor5" type="continuous">
-    <limit effort="100.0" lower="1.0" upper="20.0" velocity="0.5"/>
+  <joint name="rt5" type="fixed">
+    <!-- <limit effort="100.0" lower="1.0" upper="20.0" velocity="0.5"/> -->
     <parent link="gimbal_link1"/>
-    <child link="thrust5"/>
+    <child link="th5"/>
     <origin rpy="0 0 0" xyz="0.0735 0 0"/>
     <axis xyz="0 0 1"/>
   </joint>
-  <link name="thrust5">
+  <link name="th5">
     <inertial>
       <origin xyz="0 0 0" rpy="0 0 0"/>
@@ -286,14 +319,14 @@
     </visual>
   </link>
-  <xacro:damping_factor link ="thrust5"/>
-  <transmission name="rotor_tran5">
-    <type>transmission_interface/SimpleTransmission</type>
-    <joint name="rotor5">
-      <hardwareInterface>RotorInterface</hardwareInterface>
-    </joint>
-    <actuator name="rotor5">
-      <hardwareInterface>RotorInterface</hardwareInterface>
-      <mechanicalReduction>1</mechanicalReduction>
-    </actuator>
-  </transmission>
+  <xacro:damping_factor link ="th5"/>
+  <!-- <transmission name="rotor_tran5"> -->
+  <!--   <type>transmission_interface/SimpleTransmission</type> -->
+  <!--   <joint name="rotor5"> -->
+  <!--     <hardwareInterface>RotorInterface</hardwareInterface> -->
+  <!--   </joint> -->
+  <!--   <actuator name="rotor5"> -->
+  <!--     <hardwareInterface>RotorInterface</hardwareInterface> -->
+  <!--     <mechanicalReduction>1</mechanicalReduction> -->
+  <!--   </actuator> -->
+  <!-- </transmission> -->
 </robot>

Commit message: modified urdf for flight

File: robots/hydrus/robots/quad/soft_airframe_202509/robot.urdf.xacro (robot description, xacro)
@@ -105,9 +105,14 @@
     <inertial>
       <origin xyz="0.06875 0.000002 0.018960" rpy="0 0 0"/>
-      <mass value="${0.010*2 + 0.012}"/>
+      <!-- <mass value="${0.010*2 + 0.012}"/>
       <inertia
           ixx="0.00003988" ixy="0.0" ixz="0.0"
           iyy="0.00010606" iyz="0.0"
-          izz="0.00010185"/>
+          izz="0.00010185"/> -->
+      <mass value="0.0001"/>
+      <inertia
+          ixx="0.00001" ixy="0.0" ixz="0.0"
+          iyy="0.00001" iyz="0.0"
+          izz="0.00002"/>
     </inertial>
   </link>
@@ -120,9 +125,14 @@
     <inertial>
       <origin xyz="0.1175 0.000002 0.019998" rpy="0 0 0"/>
-      <mass value="${0.010*5 + 0.012*2}"/>
+      <!-- <mass value="${0.010*5 + 0.012*2}"/>
       <inertia
           ixx="0.00006787" ixy="0.0" ixz="0.0"
           iyy="0.00049831" iyz="0.0"
-          izz="0.00048990"/>
+          izz="0.00048990"/> -->
+      <mass value="0.0001"/>
+      <inertia
+          ixx="0.00001" ixy="0.0" ixz="0.0"
+          iyy="0.00001" iyz="0.0"
+          izz="0.00002"/>
     </inertial>
   </link>
@@ -135,9 +145,14 @@
     <inertial>
       <origin xyz="0.10740316 0.0 0.003" rpy="0 0 0"/>
-      <mass value="${0.010*2 + 0.012 + 0.070}"/>
+      <!-- <mass value="${0.010*2 + 0.012 + 0.070}"/>
       <inertia
           ixx="0.00005679" ixy="-0.000000031" ixz="-0.00002256"
           iyy="0.00028149" iyz="0.000000005"
-          izz="0.00026759"/>
+          izz="0.00026759"/> -->
+      <mass value="0.0001"/>
+      <inertia
+          ixx="0.00001" ixy="0.0" ixz="0.0"
+          iyy="0.00001" iyz="0.0"
+          izz="0.00002"/>
     </inertial>
   </link>
@@ -257,11 +272,16 @@
     <inertial>
       <origin xyz="0.0815 0 0" rpy="0 0 0"/>
-      <mass value="0.083"/>
+      <!-- <mass value="0.083"/> -->
       <!-- this inertia value is 10 times bigger than the real one -->
       <!-- to avoid the instability in gazebo -->
-      <inertia
+      <!-- <inertia
           ixx="0.0022661" ixy="0.0" ixz="0.0"
           iyy="0.0015451" iyz="0.0"
-          izz="0.00032533"/>
+          izz="0.00032533"/> -->
+      <mass value="0.0001"/>
+      <inertia
+          ixx="0.00001" ixy="0.0" ixz="0.0"
+          iyy="0.00001" iyz="0.0"
+          izz="0.00002"/>
     </inertial>
     <collision>

Commit message: flight has been done

File: robots/hydrus/robots/quad/soft_airframe_202509/robot.urdf.xacro (robot description, xacro)
@@ -105,14 +105,9 @@
     <inertial>
       <origin xyz="0.06875 0.000002 0.018960" rpy="0 0 0"/>
-      <!-- <mass value="${0.010*2 + 0.012}"/>
+      <mass value="${0.010*2 + 0.012}"/>
       <inertia
           ixx="0.00003988" ixy="0.0" ixz="0.0"
           iyy="0.00010606" iyz="0.0"
-          izz="0.00010185"/> -->
-      <mass value="0.0001"/>
-      <inertia
-          ixx="0.00001" ixy="0.0" ixz="0.0"
-          iyy="0.00001" iyz="0.0"
-          izz="0.00002"/>
+          izz="0.00010185"/>
     </inertial>
   </link>
@@ -125,14 +120,9 @@
     <inertial>
       <origin xyz="0.1175 0.000002 0.019998" rpy="0 0 0"/>
-      <!-- <mass value="${0.010*5 + 0.012*2}"/>
+      <mass value="${0.010*5 + 0.012*2}"/>
       <inertia
           ixx="0.00006787" ixy="0.0" ixz="0.0"
           iyy="0.00049831" iyz="0.0"
-          izz="0.00048990"/> -->
-      <mass value="0.0001"/>
-      <inertia
-          ixx="0.00001" ixy="0.0" ixz="0.0"
-          iyy="0.00001" iyz="0.0"
-          izz="0.00002"/>
+          izz="0.00048990"/>
     </inertial>
   </link>
@@ -145,14 +135,9 @@
     <inertial>
       <origin xyz="0.10740316 0.0 0.003" rpy="0 0 0"/>
-      <!-- <mass value="${0.010*2 + 0.012 + 0.070}"/>
+      <mass value="${0.010*2 + 0.012 + 0.070}"/>
       <inertia
           ixx="0.00005679" ixy="-0.000000031" ixz="-0.00002256"
           iyy="0.00028149" iyz="0.000000005"
-          izz="0.00026759"/> -->
-      <mass value="0.0001"/>
-      <inertia
-          ixx="0.00001" ixy="0.0" ixz="0.0"
-          iyy="0.00001" iyz="0.0"
-          izz="0.00002"/>
+          izz="0.00026759"/>
     </inertial>
   </link>
@@ -272,16 +257,12 @@
     <inertial>
       <origin xyz="0.0815 0 0" rpy="0 0 0"/>
-      <!-- <mass value="0.083"/> -->
+      <mass value="0.173"/>
       <!-- this inertia value is 10 times bigger than the real one -->
       <!-- to avoid the instability in gazebo -->
-      <!-- <inertia
-          ixx="0.0022661" ixy="0.0" ixz="0.0"
-          iyy="0.0015451" iyz="0.0"
-          izz="0.00032533"/> -->
-      <mass value="0.0001"/>
-      <inertia
-          ixx="0.00001" ixy="0.0" ixz="0.0"
-          iyy="0.00001" iyz="0.0"
-          izz="0.00002"/>
+      <!-- this is the original now -->
+      <inertia
+          ixx="0.00022661" ixy="0.0" ixz="0.0"
+          iyy="0.00015451" iyz="0.0"
+          izz="0.000032533"/>
     </inertial>
     <collision>

Commit message: relatively stable urdf with all the servos

File: robots/hydrus/robots/quad/soft_airframe_202509/robot.urdf.xacro (robot description, xacro)
@@ -111,4 +111,10 @@
           izz="0.00010185"/>
     </inertial>
+    <visual>
+      <geometry>
+        <box size="0.1175 0.03 0.04"/>
+      </geometry>
+      <origin xyz="0.05875 0 0.02" rpy="0 0 0"/>
+    </visual>
   </link>
   <gazebo reference="soft_link1">
@@ -126,4 +132,10 @@
           izz="0.00048990"/>
     </inertial>
+    <visual>
+      <geometry>
+        <box size="0.235 0.03 0.04"/>
+      </geometry>
+      <origin xyz="0.1175 0.000002 0.019998" rpy="0 0 0"/>
+    </visual>
   </link>
   <gazebo reference="soft_link2">
@@ -141,4 +153,10 @@
           izz="0.00026759"/>
     </inertial>
+    <visual>
+      <geometry>
+        <box size="0.1175 0.03 0.04"/>
+      </geometry>
+      <origin xyz="0.05875 0 0.02" rpy="0 0 0"/>
+    </visual>
   </link>
   <gazebo reference="soft_link3">
@@ -149,11 +167,17 @@
   <link name="dummy_link">
     <inertial>
-      <origin xyz="0 0 0" rpy="0 0 0"/>
-      <mass value="0.0001"/>
-      <inertia
-          ixx="0.00001" ixy="0.0" ixz="0.0"
-          iyy="0.00001" iyz="0.0"
-          izz="0.00002"/>
-    </inertial>
+      <origin xyz="0 0 -0.02" rpy="0 0 0"/>
+      <mass value="0.01"/>
+      <inertia
+          ixx="0.001" ixy="0.0" ixz="0.0"
+          iyy="0.001" iyz="0.0"
+          izz="0.002"/>
+    </inertial>
+    <visual>
+      <geometry>
+        <box size="0.05 0.05 0.05"/>
+      </geometry>
+      <origin xyz="0 0 -0.02" rpy="0 0 0"/>
+    </visual>
   </link>
   <gazebo reference="dummy_link">
@@ -168,5 +192,5 @@
   </joint>
   <joint name="soft_joint2" type="revolute">
-    <limit effort="10.0" lower="${-pi/2}" upper="${pi/2}" velocity="0.5"/>
+    <limit effort="5.0" lower="${-pi/2}" upper="${pi/2}" velocity="0.5"/>
     <parent link="soft_link1"/>
     <child link="soft_link2"/>
@@ -176,5 +200,5 @@
   </joint>
   <joint name="soft_joint3" type="revolute">
-    <limit effort="10.0" lower="${-pi/2}" upper="${pi/2}" velocity="0.5"/>
+    <limit effort="5.0" lower="${-pi/2}" upper="${pi/2}" velocity="0.5"/>
     <parent link="soft_link2"/>
     <child link="soft_link3"/>
@@ -187,8 +211,8 @@
   </gazebo> -->
   <joint name="soft_joint4" type="revolute">
-    <limit effort="10.0" lower="${-pi/2}" upper="${pi/2}" velocity="0.5"/>
+    <limit effort="5.0" lower="${-pi/2}" upper="${pi/2}" velocity="0.5"/>
     <parent link="soft_link3"/>
     <child link="dummy_link"/>
-    <origin xyz="0.235 0 0" rpy="0 0 0"/>
+    <origin xyz="0 0 -0.02" rpy="0 0 0"/>
     <axis xyz="0 0 1"/>
     <dynamics damping="0.9" friction="0.1"/>
@@ -247,5 +271,5 @@
   <!-- gimbal -->
   <joint name="gimbal_joint1" type="continuous">
-    <limit effort="100.0" lower="1.0" upper="20.0" velocity="0.5"/>
+    <limit effort="5.0" lower="1.0" upper="20.0" velocity="0.5"/>
     <parent link="soft_link3"/>
     <child link="gimbal_link1"/>
@@ -260,16 +284,15 @@
       <!-- this inertia value is 10 times bigger than the real one -->
       <!-- to avoid the instability in gazebo -->
-      <!-- this is the original now -->
-      <inertia
-          ixx="0.00022661" ixy="0.0" ixz="0.0"
-          iyy="0.00015451" iyz="0.0"
-          izz="0.000032533"/>
-    </inertial>
-    <collision>
+      <inertia
+          ixx="0.0022661" ixy="0.0" ixz="0.0"
+          iyy="0.0015451" iyz="0.0"
+          izz="0.00032533"/>
+    </inertial>
+    <!-- <collision>
       <origin xyz="0.0815 0 0" rpy="0 0 0"/>
       <geometry>
         <cylinder length="0.1" radius="0.05"/>
       </geometry>
-    </collision>
+    </collision> -->
     <visual>
       <origin xyz="0.0815 0 0" rpy="0 0 0"/>
@@ -291,12 +314,12 @@
   </transmission>
   <!-- rotor -->
-  <joint name="rt5" type="fixed">
-    <!-- <limit effort="100.0" lower="1.0" upper="20.0" velocity="0.5"/> -->
+  <joint name="rotor5" type="continuous">
+    <limit effort="5.0" lower="1.0" upper="20.0" velocity="0.5"/>
     <parent link="gimbal_link1"/>
-    <child link="th5"/>
+    <child link="thrust5"/>
     <origin rpy="0 0 0" xyz="0.0735 0 0"/>
     <axis xyz="0 0 1"/>
   </joint>
-  <link name="th5">
+  <link name="thrust5">
     <inertial>
       <origin xyz="0 0 0" rpy="0 0 0"/>
@@ -307,10 +330,10 @@
           izz="0.00002"/>
     </inertial>
-    <collision>
+    <!-- <collision>
       <origin rpy="0 0 0" xyz="0 0 0"/>
       <geometry>
         <cylinder length="0.1" radius="0.11"/>
       </geometry>
-    </collision>
+    </collision> -->
     <visual>
       <origin rpy="${pi/2} 0 0" xyz="-0.045 0.055 0.06"/>
@@ -320,14 +343,14 @@
     </visual>
   </link>
-  <xacro:damping_factor link ="th5"/>
-  <!-- <transmission name="rotor_tran5"> -->
-  <!--   <type>transmission_interface/SimpleTransmission</type> -->
-  <!--   <joint name="rotor5"> -->
-  <!--     <hardwareInterface>RotorInterface</hardwareInterface> -->
-  <!--   </joint> -->
-  <!--   <actuator name="rotor5"> -->
-  <!--     <hardwareInterface>RotorInterface</hardwareInterface> -->
-  <!--     <mechanicalReduction>1</mechanicalReduction> -->
-  <!--   </actuator> -->
-  <!-- </transmission> -->
+  <xacro:damping_factor link ="thrust5"/>
+  <transmission name="rotor_tran5">
+    <type>transmission_interface/SimpleTransmission</type>
+    <joint name="rotor5">
+      <hardwareInterface>RotorInterface</hardwareInterface>
+    </joint>
+    <actuator name="rotor5">
+      <hardwareInterface>RotorInterface</hardwareInterface>
+      <mechanicalReduction>1</mechanicalReduction>
+    </actuator>
+  </transmission>
 </robot>

Commit message: two types of motor info

File: robots/hydrus/robots/quad/soft_airframe_202509/robot.urdf.xacro (robot description, xacro)
@@ -270,6 +270,6 @@
  -->
   <!-- gimbal -->
-  <joint name="gimbal_joint1" type="continuous">
-    <limit effort="5.0" lower="1.0" upper="20.0" velocity="0.5"/>
+  <joint name="gimbal_joint1" type="revolute">
+    <limit effort="5.0" lower="${-pi}" upper="${pi}" velocity="0.5"/>
     <parent link="soft_link3"/>
     <child link="gimbal_link1"/>
@@ -302,4 +302,8 @@
     </visual>
   </link>
+  <gazebo reference="gimbal_link1">
+    <mu1>0.1</mu1>
+    <mu2>0.1</mu2>
+  </gazebo>
   <xacro:damping_factor link ="gimbal_link1"/>
   <transmission name="gimbal_tran1">

Commit message: fixed the spinal position in urdf

File: robots/hydrus/robots/quad/soft_airframe_202509/robot.urdf.xacro (robot description, xacro)
@@ -37,5 +37,5 @@
   <xacro:extra_module name = "fc" parent = "link3" visible = "1"
                       model_url = "package://hydrus/urdf/mesh/ver2/flight_controller/spinal.dae"> <!-- same with intel euclid -->
-    <origin xyz="${link_length / 2 + 0.2221} ${-4.4*0.001} 0.02135" rpy="0 0 0"/>
+    <origin xyz="${link_length / 2 - 0.2221} ${-4.4*0.001} 0.02135" rpy="0 0 0"/>
     <inertial>
       <mass value = "0.05" />

Commit message: fix gimbal and reverse-torque

File: robots/hydrus/robots/quad/soft_airframe_202509/robot.urdf.xacro (robot description, xacro)
@@ -319,5 +319,5 @@
   <!-- rotor -->
   <joint name="rotor5" type="continuous">
-    <limit effort="5.0" lower="1.0" upper="20.0" velocity="0.5"/>
+    <limit effort="-0.0064" lower="1.0" upper="20.0" velocity="0.5"/>
     <parent link="gimbal_link1"/>
     <child link="thrust5"/>

File: robots/hydrus/urdf/link.urdf.xacro (robot description, xacro)
@@ -188,5 +188,5 @@
     <!-- rotor -->
     <joint name="rotor${self}" type="continuous">
-      <limit effort="0" lower="${min_force}" upper="${max_force}" velocity="0.5"/>
+      <limit effort="${0.0172 * rotor_direction}" lower="${min_force}" upper="${max_force}" velocity="0.5"/>
       <parent link="link${self}"/>
       <child link="thrust${self}"/>

Commit message: debugging

File: robots/hydrus/robots/quad/soft_airframe_202509/robot.urdf.xacro (robot description, xacro)
@@ -167,6 +167,6 @@
   <link name="dummy_link">
     <inertial>
-      <origin xyz="0 0 -0.02" rpy="0 0 0"/>
-      <mass value="0.01"/>
+      <origin xyz="0 0 0" rpy="0 0 0"/>
+      <mass value="0.0001"/>
       <inertia
           ixx="0.001" ixy="0.0" ixz="0.0"
@@ -214,5 +214,5 @@
     <parent link="soft_link3"/>
     <child link="dummy_link"/>
-    <origin xyz="0 0 -0.02" rpy="0 0 0"/>
+    <origin xyz="0.235 0 0" rpy="0 0 0"/>
     <axis xyz="0 0 1"/>
     <dynamics damping="0.9" friction="0.1"/>

Commit message: set urdf to original one

File: robots/hydrus/robots/quad/soft_airframe_202509/robot.urdf.xacro (robot description, xacro)
@@ -169,8 +169,13 @@
       <origin xyz="0 0 0" rpy="0 0 0"/>
       <mass value="0.0001"/>
-      <inertia
+      <!-- this is for avoiding error in gazebo -->
+      <!-- <inertia
           ixx="0.001" ixy="0.0" ixz="0.0"
           iyy="0.001" iyz="0.0"
-          izz="0.002"/>
+          izz="0.002"/> -->
+      <inertia
+          ixx="0.00001" ixy="0.0" ixz="0.0"
+          iyy="0.00001" iyz="0.0"
+          izz="0.00002"/>
     </inertial>
     <visual>
@@ -284,8 +289,13 @@
       <!-- this inertia value is 10 times bigger than the real one -->
       <!-- to avoid the instability in gazebo -->
-      <inertia
+      <!-- <inertia
           ixx="0.0022661" ixy="0.0" ixz="0.0"
           iyy="0.0015451" iyz="0.0"
-          izz="0.00032533"/>
+          izz="0.00032533"/> -->
+      <!-- original one -->
+      <inertia
+          ixx="0.00022661" ixy="0.0" ixz="0.0"
+          iyy="0.00015451" iyz="0.0"
+          izz="0.000032533"/>
     </inertial>
     <!-- <collision>

Commit message: added 4th servo for soft_link

File: robots/hydrus/robots/quad/soft_airframe_202509/robot.urdf.xacro (robot description, xacro)
@@ -147,5 +147,5 @@
     <inertial>
       <origin xyz="0.10740316 0.0 0.003" rpy="0 0 0"/>
-      <mass value="${0.010*2 + 0.012 + 0.070}"/>
+      <mass value="${0.010*2 + 0.012 + 0.070 + 0.016}"/>
       <inertia
           ixx="0.00005679" ixy="-0.000000031" ixz="-0.00002256"
@@ -191,4 +191,30 @@
   </gazebo>
   <xacro:damping_factor link="dummy_link"/>
+    <link name="dummy_link1">
+    <inertial>
+      <origin xyz="0 0 0" rpy="0 0 0"/>
+      <mass value="0.0001"/>
+      <!-- this is for avoiding error in gazebo -->
+      <!-- <inertia
+          ixx="0.001" ixy="0.0" ixz="0.0"
+          iyy="0.001" iyz="0.0"
+          izz="0.002"/> -->
+      <inertia
+          ixx="0.00001" ixy="0.0" ixz="0.0"
+          iyy="0.00001" iyz="0.0"
+          izz="0.00002"/>
+    </inertial>
+    <visual>
+      <geometry>
+        <box size="0.05 0.05 0.05"/>
+      </geometry>
+      <origin xyz="0 0 -0.02" rpy="0 0 0"/>
+    </visual>
+  </link>
+  <gazebo reference="dummy_link1">
+    <mu1>0.1</mu1>
+    <mu2>0.1</mu2>
+  </gazebo>
+  <xacro:damping_factor link="dummy_link1"/>
   <joint name="soft_joint1" type="fixed">
     <parent link="link4"/>
@@ -223,4 +249,12 @@
     <dynamics damping="0.9" friction="0.1"/>
   </joint>
+  <joint name="soft_joint5" type="revolute">
+    <limit effort="5.0" lower="${-pi/2}" upper="${pi/2}" velocity="0.5"/>
+    <parent link="soft_link3"/>
+    <child link="dummy_link1"/>
+    <origin xyz="0.235 0 0" rpy="0 0 0"/>
+    <axis xyz="0 0 1"/>
+    <dynamics damping="0.9" friction="0.1"/>
+  </joint>
   <transmission name="soft_joint_tran_2">
     <type>transmission_interface/SimpleTransmission</type>
@@ -249,4 +283,14 @@
     </joint>
     <actuator name="soft_joint_servo4">
+      <hardwareInterface>hardware_interface/EffortJointInterface</hardwareInterface>
+      <mechanicalReduction>1</mechanicalReduction>
+    </actuator>
+  </transmission>
+  <transmission name="soft_joint_tran_5">
+    <type>transmission_interface/SimpleTransmission</type>
+    <joint name="soft_joint5">
+      <hardwareInterface>hardware_interface/EffortJointInterface</hardwareInterface>
+    </joint>
+    <actuator name="soft_joint_servo5">
       <hardwareInterface>hardware_interface/EffortJointInterface</hardwareInterface>
       <mechanicalReduction>1</mechanicalReduction>

Commit message: add leg

File: robots/hydrus/robots/quad/soft_airframe_202509/robot.urdf.xacro (robot description, xacro)
@@ -298,12 +298,18 @@
   </transmission>
   <!-- leg -->
-  <!-- <link name="leg6">
+  <link name="leg6">
     <inertial>
       <origin xyz="0.0 0.0 -0.093" rpy="0 0 0"/>
-      <mass value="0.047000"/>
-      <inertia
-          ixx="0.000259" iyy="0.000281" izz="0.000010"
+      <mass value="0.051000"/>
+      <inertia
+          ixx="0.000122" iyy="0.000133" izz="0.000012"
           ixy="0.000000" ixz="0.000000" iyz="0.000000"/>
     </inertial>
+    <visual>
+      <geometry>
+        <box size="0.02 0.02 -0.15"/>
+      </geometry>
+      <origin xyz="0.01 0.01 -0.075" rpy="0 0 0"/>
+    </visual>
   </link>
   <gazebo reference="leg6">
@@ -317,5 +323,4 @@
     <origin xyz="0.1 0 0" rpy="0 0 0"/>
   </joint>
- -->
   <!-- gimbal -->
   <joint name="gimbal_joint1" type="revolute">

Commit message: fix mf_rate

File: robots/hydrus/robots/quad/soft_airframe_202509/robot.urdf.xacro (robot description, xacro)
@@ -378,9 +378,9 @@
   <!-- rotor -->
   <joint name="rotor5" type="continuous">
-    <limit effort="-0.0064" lower="1.0" upper="20.0" velocity="0.5"/>
+    <limit effort="0.0064" lower="1.0" upper="20.0" velocity="0.5"/>
     <parent link="gimbal_link1"/>
     <child link="thrust5"/>
     <origin rpy="0 0 0" xyz="0.0735 0 0"/>
-    <axis xyz="0 0 1"/>
+    <axis xyz="0 0 -1"/>
   </joint>
   <link name="thrust5">

File: robots/hydrus/urdf/link.urdf.xacro (robot description, xacro)
@@ -188,5 +188,5 @@
     <!-- rotor -->
     <joint name="rotor${self}" type="continuous">
-      <limit effort="${0.0172 * rotor_direction}" lower="${min_force}" upper="${max_force}" velocity="0.5"/>
+      <limit effort="0.0172" lower="${min_force}" upper="${max_force}" velocity="0.5"/>
       <parent link="link${self}"/>
       <child link="thrust${self}"/>
