Commit message: implement qp and able to change max_thrust

File: robots/hydrus/robots/quad/soft_airframe_202509/robot.urdf.xacro (robot description, xacro)
@@ -5,8 +5,8 @@
   <xacro:include filename="$(find hydrus)/urdf/common.xacro" />
   <xacro:include filename="$(find hydrus)/urdf/link.urdf.xacro" />
-  <xacro:hydrus_link links="4" self="1" rotor_direction="-1" with_battery = "0" tilt_mode="1" tilt_angle="20" />
-  <xacro:hydrus_link links="4" self="2" rotor_direction="1"  with_battery = "0" tilt_mode="1" tilt_angle="20" />
-  <xacro:hydrus_link links="4" self="3" rotor_direction="-1" with_battery = "0" tilt_mode="1" tilt_angle="20" />
-  <xacro:hydrus_link links="4" self="4" rotor_direction="1"  with_battery = "0" tilt_mode="1" tilt_angle="20" />
+  <xacro:hydrus_link links="4" self="1" rotor_direction="-1" with_battery = "0" tilt_mode="1" tilt_angle="20" max_force="20.0"/>
+  <xacro:hydrus_link links="4" self="2" rotor_direction="1"  with_battery = "0" tilt_mode="1" tilt_angle="20" max_force="20.0"/>
+  <xacro:hydrus_link links="4" self="3" rotor_direction="-1" with_battery = "0" tilt_mode="1" tilt_angle="20" max_force="20.0"/>
+  <xacro:hydrus_link links="4" self="4" rotor_direction="1"  with_battery = "0" tilt_mode="1" tilt_angle="20" max_force="20.0"/>
   <!-- special battery arrangement -->
   <xacro:extra_module name = "bat1" parent = "link1" visible = "1"

File: robots/hydrus/urdf/common.xacro (robot description, xacro)
@@ -18,5 +18,5 @@
   <!-- dynamics -->
   <m_f_rate value="-0.0172" /> <!-- drug torque rate -->
-  <xacro:property name="max_force" value="20.0" /> <!-- [N] -->
+  <!-- <xacro:property name="max_force" value="20.0" /> --> <!-- [N] -->
   <xacro:property name="min_force" value="1.0" /> <!-- [N] -->
   <xacro:macro name="link_model" params="type with_leg:=${with_leg} old_version:=${old_version} tilt_mode:=${tilt_mode} tilt_angle:=${tilt_angle} prop_15inch:=${prop_15inch}">

File: robots/hydrus/urdf/link.urdf.xacro (robot description, xacro)
@@ -3,5 +3,5 @@
     xmlns:xacro="http://www.ros.org/wiki/xacro" name="hydrus_link" >
   <!-- D-H kai description(different from prof.nakamura) -->
-  <xacro:macro name="hydrus_link" params="links self rotor_direction with_leg:=1 with_battery:=1 old_version:=0 tilt_mode:=0 tilt_angle:=0 prop_15inch:=0">
+  <xacro:macro name="hydrus_link" params="links self rotor_direction with_leg:=1 with_battery:=1 old_version:=0 tilt_mode:=0 tilt_angle:=0 prop_15inch:=0 max_force:=20.0">
     <xacro:if value="${old_version == 1}">
       <!-- link -->

Commit message: handle the case that thrust5 mocap is not updated

File: robots/hydrus/robots/quad/soft_airframe_202509/robot.urdf.xacro (robot description, xacro)
@@ -170,12 +170,12 @@
       <mass value="0.0001"/>
       <!-- this is for avoiding error in gazebo -->
-      <!-- <inertia
+      <inertia
           ixx="0.001" ixy="0.0" ixz="0.0"
           iyy="0.001" iyz="0.0"
-          izz="0.002"/> -->
-      <inertia
+          izz="0.002"/>
+      <!-- <inertia
           ixx="0.00001" ixy="0.0" ixz="0.0"
           iyy="0.00001" iyz="0.0"
-          izz="0.00002"/>
+          izz="0.00002"/> -->
     </inertial>
     <visual>
@@ -196,12 +196,12 @@
       <mass value="0.0001"/>
       <!-- this is for avoiding error in gazebo -->
-      <!-- <inertia
+      <inertia
           ixx="0.001" ixy="0.0" ixz="0.0"
           iyy="0.001" iyz="0.0"
-          izz="0.002"/> -->
-      <inertia
+          izz="0.002"/>
+      <!-- <inertia
           ixx="0.00001" ixy="0.0" ixz="0.0"
           iyy="0.00001" iyz="0.0"
-          izz="0.00002"/>
+          izz="0.00002"/> -->
     </inertial>
     <visual>
@@ -338,13 +338,13 @@
       <!-- this inertia value is 10 times bigger than the real one -->
       <!-- to avoid the instability in gazebo -->
-      <!-- <inertia
+      <inertia
           ixx="0.0022661" ixy="0.0" ixz="0.0"
           iyy="0.0015451" iyz="0.0"
-          izz="0.00032533"/> -->
+          izz="0.00032533"/>
       <!-- original one -->
-      <inertia
+      <!-- <inertia
           ixx="0.00022661" ixy="0.0" ixz="0.0"
           iyy="0.00015451" iyz="0.0"
-          izz="0.000032533"/>
+          izz="0.000032533"/> -->
     </inertial>
     <!-- <collision>

Commit message: revert the change of urdf and position_based_tail.py

File: robots/hydrus/robots/quad/soft_airframe_202509/robot.urdf.xacro (robot description, xacro)
@@ -170,12 +170,12 @@
       <mass value="0.0001"/>
       <!-- this is for avoiding error in gazebo -->
-      <inertia
+      <!-- <inertia
           ixx="0.001" ixy="0.0" ixz="0.0"
           iyy="0.001" iyz="0.0"
-          izz="0.002"/>
-      <!-- <inertia
+          izz="0.002"/> -->
+      <inertia
           ixx="0.00001" ixy="0.0" ixz="0.0"
           iyy="0.00001" iyz="0.0"
-          izz="0.00002"/> -->
+          izz="0.00002"/>
     </inertial>
     <visual>
@@ -196,12 +196,12 @@
       <mass value="0.0001"/>
       <!-- this is for avoiding error in gazebo -->
-      <inertia
+      <!-- <inertia
           ixx="0.001" ixy="0.0" ixz="0.0"
           iyy="0.001" iyz="0.0"
-          izz="0.002"/>
-      <!-- <inertia
+          izz="0.002"/> -->
+      <inertia
           ixx="0.00001" ixy="0.0" ixz="0.0"
           iyy="0.00001" iyz="0.0"
-          izz="0.00002"/> -->
+          izz="0.00002"/>
     </inertial>
     <visual>
@@ -338,13 +338,13 @@
       <!-- this inertia value is 10 times bigger than the real one -->
       <!-- to avoid the instability in gazebo -->
-      <inertia
+      <!-- <inertia
           ixx="0.0022661" ixy="0.0" ixz="0.0"
           iyy="0.0015451" iyz="0.0"
-          izz="0.00032533"/>
+          izz="0.00032533"/> -->
       <!-- original one -->
-      <!-- <inertia
+      <inertia
           ixx="0.00022661" ixy="0.0" ixz="0.0"
           iyy="0.00015451" iyz="0.0"
-          izz="0.000032533"/> -->
+          izz="0.000032533"/>
     </inertial>
     <!-- <collision>

Commit message: add servo to urdf

File: robots/hydrus/robots/quad/soft_airframe_202509/robot.urdf.xacro (robot description, xacro)
@@ -37,5 +37,5 @@
   <xacro:extra_module name = "fc" parent = "link3" visible = "1"
                       model_url = "package://hydrus/urdf/mesh/ver2/flight_controller/spinal.dae"> <!-- same with intel euclid -->
-    <origin xyz="${link_length / 2 - 0.2221} ${-4.4*0.001} 0.02135" rpy="0 0 0"/>
+    <origin xyz="${link_length / 2 - 0.2221} ${-4.4*0.001} -0.02135" rpy="0 0 0"/>
     <inertial>
       <mass value = "0.05" />
@@ -165,8 +165,8 @@
   </gazebo>
   <xacro:damping_factor link="soft_link3"/>
-  <link name="dummy_link">
-    <inertial>
-      <origin xyz="0 0 0" rpy="0 0 0"/>
-      <mass value="0.0001"/>
+  <link name="servo_link">
+    <inertial>
+      <origin xyz="0 0 0" rpy="0 0 0"/>
+      <mass value="0.064"/>
       <!-- this is for avoiding error in gazebo -->
       <!-- <inertia
@@ -175,7 +175,7 @@
           izz="0.002"/> -->
       <inertia
-          ixx="0.00001" ixy="0.0" ixz="0.0"
-          iyy="0.00001" iyz="0.0"
-          izz="0.00002"/>
+          ixx="0.000017" ixy="0.000003" ixz="-0.0000001"
+          iyy="0.000023" iyz="0.000000"
+          izz="0.000025"/>
     </inertial>
     <visual>
@@ -186,13 +186,13 @@
     </visual>
   </link>
-  <gazebo reference="dummy_link">
-    <mu1>0.1</mu1>
-    <mu2>0.1</mu2>
-  </gazebo>
-  <xacro:damping_factor link="dummy_link"/>
-    <link name="dummy_link1">
-    <inertial>
-      <origin xyz="0 0 0" rpy="0 0 0"/>
-      <mass value="0.0001"/>
+  <gazebo reference="servo_link">
+    <mu1>0.1</mu1>
+    <mu2>0.1</mu2>
+  </gazebo>
+  <xacro:damping_factor link="servo_link"/>
+  <link name="servo_link1">
+    <inertial>
+      <origin xyz="0 0 0" rpy="0 0 0"/>
+      <mass value="0.059"/>
       <!-- this is for avoiding error in gazebo -->
       <!-- <inertia
@@ -201,7 +201,7 @@
           izz="0.002"/> -->
       <inertia
-          ixx="0.00001" ixy="0.0" ixz="0.0"
-          iyy="0.00001" iyz="0.0"
-          izz="0.00002"/>
+          ixx="0.000016" ixy="-0.000003" ixz="0.000001"
+          iyy="0.000019" iyz="0.000000"
+          izz="0.000022"/>
     </inertial>
     <visual>
@@ -212,9 +212,9 @@
     </visual>
   </link>
-  <gazebo reference="dummy_link1">
-    <mu1>0.1</mu1>
-    <mu2>0.1</mu2>
-  </gazebo>
-  <xacro:damping_factor link="dummy_link1"/>
+  <gazebo reference="servo_link1">
+    <mu1>0.1</mu1>
+    <mu2>0.1</mu2>
+  </gazebo>
+  <xacro:damping_factor link="servo_link1"/>
   <joint name="soft_joint1" type="fixed">
     <parent link="link4"/>
@@ -243,7 +243,7 @@
   <joint name="soft_joint4" type="revolute">
     <limit effort="5.0" lower="${-pi/2}" upper="${pi/2}" velocity="0.5"/>
-    <parent link="soft_link3"/>
-    <child link="dummy_link"/>
-    <origin xyz="0.235 0 0" rpy="0 0 0"/>
+    <parent link="link4"/>
+    <child link="servo_link"/>
+    <origin xyz="0.5 0 0.01" rpy="0 0 0"/>
     <axis xyz="0 0 1"/>
     <dynamics damping="0.9" friction="0.1"/>
@@ -251,7 +251,7 @@
   <joint name="soft_joint5" type="revolute">
     <limit effort="5.0" lower="${-pi/2}" upper="${pi/2}" velocity="0.5"/>
-    <parent link="soft_link3"/>
-    <child link="dummy_link1"/>
-    <origin xyz="0.235 0 0" rpy="0 0 0"/>
+    <parent link="link4"/>
+    <child link="servo_link1"/>
+    <origin xyz="0.5 0 -0.01" rpy="0 0 0"/>
     <axis xyz="0 0 1"/>
     <dynamics damping="0.9" friction="0.1"/>

Commit message: add weight

File: robots/hydrus/robots/quad/soft_airframe_202509/robot.urdf.xacro (robot description, xacro)
@@ -168,5 +168,5 @@
     <inertial>
       <origin xyz="0 0 0" rpy="0 0 0"/>
-      <mass value="0.064"/>
+      <mass value="0.073"/>
       <!-- this is for avoiding error in gazebo -->
       <!-- <inertia
@@ -194,5 +194,5 @@
     <inertial>
       <origin xyz="0 0 0" rpy="0 0 0"/>
-      <mass value="0.059"/>
+      <mass value="0.068"/>
       <!-- this is for avoiding error in gazebo -->
       <!-- <inertia

Commit message: change the pos of spinal

File: robots/hydrus/robots/quad/soft_airframe_202509/robot.urdf.xacro (robot description, xacro)
@@ -37,5 +37,5 @@
   <xacro:extra_module name = "fc" parent = "link3" visible = "1"
                       model_url = "package://hydrus/urdf/mesh/ver2/flight_controller/spinal.dae"> <!-- same with intel euclid -->
-    <origin xyz="${link_length / 2 - 0.2221} ${-4.4*0.001} -0.02135" rpy="0 0 0"/>
+    <origin xyz="${link_length / 2 - 0.2221} ${-4.4*0.001} 0.02135" rpy="0 0 0"/>
     <inertial>
       <mass value = "0.05" />

Commit message: use udp

File: robots/hydrus/robots/quad/soft_airframe_202509/robot.urdf.xacro (robot description, xacro)
@@ -105,5 +105,5 @@
     <inertial>
       <origin xyz="0.06875 0.000002 0.018960" rpy="0 0 0"/>
-      <mass value="${0.010*2 + 0.012}"/>
+      <mass value="0.059"/>
       <inertia
           ixx="0.00003988" ixy="0.0" ixz="0.0"
@@ -126,5 +126,5 @@
     <inertial>
       <origin xyz="0.1175 0.000002 0.019998" rpy="0 0 0"/>
-      <mass value="${0.010*5 + 0.012*2}"/>
+      <mass value="0.118"/>
       <inertia
           ixx="0.00006787" ixy="0.0" ixz="0.0"
@@ -147,5 +147,5 @@
     <inertial>
       <origin xyz="0.10740316 0.0 0.003" rpy="0 0 0"/>
-      <mass value="${0.010*2 + 0.012 + 0.070 + 0.016}"/>
+      <mass value="${0.059 + 0.053}"/>
       <inertia
           ixx="0.00005679" ixy="-0.000000031" ixz="-0.00002256"
@@ -324,5 +324,5 @@
   </joint>
   <!-- gimbal -->
-  <joint name="gimbal_joint1" type="revolute">
+  <joint name="gimbal_joint1" type="fixed">
     <limit effort="5.0" lower="${-pi}" upper="${pi}" velocity="0.5"/>
     <parent link="soft_link3"/>
@@ -335,5 +335,5 @@
     <inertial>
       <origin xyz="0.0815 0 0" rpy="0 0 0"/>
-      <mass value="0.173"/>
+      <mass value="0.222"/>
       <!-- this inertia value is 10 times bigger than the real one -->
       <!-- to avoid the instability in gazebo -->
@@ -366,5 +366,5 @@
   </gazebo>
   <xacro:damping_factor link ="gimbal_link1"/>
-  <transmission name="gimbal_tran1">
+  <!-- <transmission name="gimbal_tran1">
     <type>transmission_interface/SimpleTransmission</type>
     <joint name="gimbal_joint1">
@@ -375,5 +375,5 @@
       <mechanicalReduction>1</mechanicalReduction>
     </actuator>
-  </transmission>
+  </transmission> -->
   <!-- rotor -->
   <joint name="rotor5" type="continuous">

Commit message: update urdf to correspond the new tail

File: robots/hydrus/robots/quad/soft_airframe_202509/robot.urdf.xacro (robot description, xacro)
@@ -102,12 +102,34 @@
   <!-- end: gps -->
   <!-- 3 soft_airframe -->
+  <!-- soft_link -->
+  <joint name="soft_joint1" type="fixed">
+    <parent link="link4"/>
+    <child link="soft_link1"/>
+    <origin xyz="0.6 0 0" rpy="0 0 0"/>
+  </joint>
+  <joint name="soft_joint2" type="revolute">
+    <limit effort="5.0" lower="${-pi/2}" upper="${pi/2}" velocity="0.5"/>
+    <parent link="soft_link1"/>
+    <child link="soft_link2"/>
+    <origin xyz="0.1175 0 0" rpy="0 0 0"/>
+    <axis xyz="0 0 1"/>
+    <dynamics damping="0.9" friction="0.1"/>
+  </joint>
+  <joint name="soft_joint3" type="revolute">
+    <limit effort="5.0" lower="${-pi/2}" upper="${pi/2}" velocity="0.5"/>
+    <parent link="soft_link2"/>
+    <child link="soft_link3"/>
+    <origin xyz="0.235 0 0" rpy="0 0 0"/>
+    <axis xyz="0 0 1"/>
+    <dynamics damping="0.9" friction="0.1"/>
+  </joint>
   <link name="soft_link1">
     <inertial>
-      <origin xyz="0.06875 0.000002 0.018960" rpy="0 0 0"/>
+      <origin xyz="0.064 0.000002 0.018960" rpy="0 0 0"/>
       <mass value="0.059"/>
       <inertia
-          ixx="0.00003988" ixy="0.0" ixz="0.0"
-          iyy="0.00010606" iyz="0.0"
-          izz="0.00010185"/>
+          ixx="0.00005433" ixy="0.00000033" ixz="0.0"
+          iyy="0.00047358" iyz="-0.00000369"
+          izz="0.00046011"/>
     </inertial>
     <visual>
@@ -125,10 +147,10 @@
   <link name="soft_link2">
     <inertial>
-      <origin xyz="0.1175 0.000002 0.019998" rpy="0 0 0"/>
+      <origin xyz="0.118 0.000002 0.019998" rpy="0 0 0"/>
       <mass value="0.118"/>
       <inertia
-          ixx="0.00006787" ixy="0.0" ixz="0.0"
-          iyy="0.00049831" iyz="0.0"
-          izz="0.00048990"/>
+          ixx="0.00007941" ixy="0.00000218" ixz="0.0"
+          iyy="0.00065133" iyz="0.0"
+          izz="0.00062639"/>
     </inertial>
     <visual>
@@ -147,9 +169,9 @@
     <inertial>
       <origin xyz="0.10740316 0.0 0.003" rpy="0 0 0"/>
-      <mass value="${0.059 + 0.053}"/>
-      <inertia
-          ixx="0.00005679" ixy="-0.000000031" ixz="-0.00002256"
-          iyy="0.00028149" iyz="0.000000005"
-          izz="0.00026759"/>
+      <mass value="0.059"/>
+      <inertia
+          ixx="0.00005433" ixy="0.00000033" ixz="0.0"
+          iyy="0.00047358" iyz="-0.00000369"
+          izz="0.00046011"/>
     </inertial>
     <visual>
@@ -165,4 +187,41 @@
   </gazebo>
   <xacro:damping_factor link="soft_link3"/>
+  <transmission name="soft_joint_tran_2">
+    <type>transmission_interface/SimpleTransmission</type>
+    <joint name="soft_joint2">
+      <hardwareInterface>hardware_interface/EffortJointInterface</hardwareInterface>
+    </joint>
+    <actuator name="soft_joint_servo2">
+      <hardwareInterface>hardware_interface/EffortJointInterface</hardwareInterface>
+      <mechanicalReduction>1</mechanicalReduction>
+    </actuator>
+  </transmission>
+  <transmission name="soft_joint_tran_3">
+    <type>transmission_interface/SimpleTransmission</type>
+    <joint name="soft_joint3">
+      <hardwareInterface>hardware_interface/EffortJointInterface</hardwareInterface>
+    </joint>
+    <actuator name="soft_joint_servo3">
+      <hardwareInterface>hardware_interface/EffortJointInterface</hardwareInterface>
+      <mechanicalReduction>1</mechanicalReduction>
+    </actuator>
+  </transmission>
+  <!-- dummy_link -->
+  <joint name="soft_joint4" type="revolute">
+    <limit effort="5.0" lower="${-pi/2}" upper="${pi/2}" velocity="0.5"/>
+    <parent link="link4"/>
+    <child link="servo_link"/>
+    <origin xyz="0.5 0 0.01" rpy="0 0 0"/>
+    <axis xyz="0 0 1"/>
+    <dynamics damping="0.9" friction="0.1"/>
+  </joint>
+  <joint name="soft_joint5" type="revolute">
+    <limit effort="5.0" lower="${-pi/2}" upper="${pi/2}" velocity="0.5"/>
+    <parent link="link4"/>
+    <child link="servo_link1"/>
+    <origin xyz="0.5 0 -0.01" rpy="0 0 0"/>
+    <axis xyz="0 0 1"/>
+    <dynamics damping="0.9" friction="0.1"/>
+  </joint>
   <link name="servo_link">
     <inertial>
@@ -175,7 +234,7 @@
           izz="0.002"/> -->
       <inertia
-          ixx="0.000017" ixy="0.000003" ixz="-0.0000001"
-          iyy="0.000023" iyz="0.000000"
-          izz="0.000025"/>
+          ixx="0.000023" ixy="0.000003" ixz="-0.0000001"
+          iyy="0.000044" iyz="0.000000"
+          izz="0.000043"/>
     </inertial>
     <visual>
@@ -201,7 +260,7 @@
           izz="0.002"/> -->
       <inertia
-          ixx="0.000016" ixy="-0.000003" ixz="0.000001"
-          iyy="0.000019" iyz="0.000000"
-          izz="0.000022"/>
+          ixx="0.000022" ixy="-0.000003" ixz="0.000001"
+          iyy="0.000042" iyz="0.000000"
+          izz="0.000041"/>
     </inertial>
     <visual>
@@ -217,64 +276,4 @@
   </gazebo>
   <xacro:damping_factor link="servo_link1"/>
-  <joint name="soft_joint1" type="fixed">
-    <parent link="link4"/>
-    <child link="soft_link1"/>
-    <origin xyz="0.6 0 0" rpy="0 0 0"/>
-  </joint>
-  <joint name="soft_joint2" type="revolute">
-    <limit effort="5.0" lower="${-pi/2}" upper="${pi/2}" velocity="0.5"/>
-    <parent link="soft_link1"/>
-    <child link="soft_link2"/>
-    <origin xyz="0.1175 0 0" rpy="0 0 0"/>
-    <axis xyz="0 0 1"/>
-    <dynamics damping="0.9" friction="0.1"/>
-  </joint>
-  <joint name="soft_joint3" type="revolute">
-    <limit effort="5.0" lower="${-pi/2}" upper="${pi/2}" velocity="0.5"/>
-    <parent link="soft_link2"/>
-    <child link="soft_link3"/>
-    <origin xyz="0.235 0 0" rpy="0 0 0"/>
-    <axis xyz="0 0 1"/>
-    <dynamics damping="0.9" friction="0.1"/>
-  </joint>
-  <!-- <gazebo reference="soft_link3">
-    <stopCfm>1000</stopCfm>
-  </gazebo> -->
-  <joint name="soft_joint4" type="revolute">
-    <limit effort="5.0" lower="${-pi/2}" upper="${pi/2}" velocity="0.5"/>
-    <parent link="link4"/>
-    <child link="servo_link"/>
-    <origin xyz="0.5 0 0.01" rpy="0 0 0"/>
-    <axis xyz="0 0 1"/>
-    <dynamics damping="0.9" friction="0.1"/>
-  </joint>
-  <joint name="soft_joint5" type="revolute">
-    <limit effort="5.0" lower="${-pi/2}" upper="${pi/2}" velocity="0.5"/>
-    <parent link="link4"/>
-    <child link="servo_link1"/>
-    <origin xyz="0.5 0 -0.01" rpy="0 0 0"/>
-    <axis xyz="0 0 1"/>
-    <dynamics damping="0.9" friction="0.1"/>
-  </joint>
-  <transmission name="soft_joint_tran_2">
-    <type>transmission_interface/SimpleTransmission</type>
-    <joint name="soft_joint2">
-      <hardwareInterface>hardware_interface/EffortJointInterface</hardwareInterface>
-    </joint>
-    <actuator name="soft_joint_servo2">
-      <hardwareInterface>hardware_interface/EffortJointInterface</hardwareInterface>
-      <mechanicalReduction>1</mechanicalReduction>
-    </actuator>
-  </transmission>
-  <transmission name="soft_joint_tran_3">
-    <type>transmission_interface/SimpleTransmission</type>
-    <joint name="soft_joint3">
-      <hardwareInterface>hardware_interface/EffortJointInterface</hardwareInterface>
-    </joint>
-    <actuator name="soft_joint_servo3">
-      <hardwareInterface>hardware_interface/EffortJointInterface</hardwareInterface>
-      <mechanicalReduction>1</mechanicalReduction>
-    </actuator>
-  </transmission>
   <transmission name="soft_joint_tran_4">
     <type>transmission_interface/SimpleTransmission</type>
@@ -348,13 +347,7 @@
           izz="0.000032533"/>
     </inertial>
-    <!-- <collision>
+    <visual>
       <origin xyz="0.0815 0 0" rpy="0 0 0"/>
       <geometry>
-        <cylinder length="0.1" radius="0.05"/>
-      </geometry>
-    </collision> -->
-    <visual>
-      <origin xyz="0.0815 0 0" rpy="0 0 0"/>
-      <geometry>
         <mesh filename="package://hydrus/urdf/mesh/propeller/5inch_propeller_duct_right_v2.dae"/>
       </geometry>
@@ -366,14 +359,4 @@
   </gazebo>
   <xacro:damping_factor link ="gimbal_link1"/>
-  <!-- <transmission name="gimbal_tran1">
-    <type>transmission_interface/SimpleTransmission</type>
-    <joint name="gimbal_joint1">
-      <hardwareInterface>hardware_interface/EffortJointInterface</hardwareInterface>
-    </joint>
-    <actuator name="gimbal_servo1">
-      <hardwareInterface>hardware_interface/EffortJointInterface</hardwareInterface>
-      <mechanicalReduction>1</mechanicalReduction>
-    </actuator>
-  </transmission> -->
   <!-- rotor -->
   <joint name="rotor5" type="continuous">
@@ -393,10 +376,4 @@
           izz="0.00002"/>
     </inertial>
-    <!-- <collision>
-      <origin rpy="0 0 0" xyz="0 0 0"/>
-      <geometry>
-        <cylinder length="0.1" radius="0.11"/>
-      </geometry>
-    </collision> -->
     <visual>
       <origin rpy="${pi/2} 0 0" xyz="-0.045 0.055 0.06"/>
