Commit message: [mini quadrotor] update the model with livox lidar, which is the same with Yunong's branch.

File: robots/mini_quadrotor/urdf/robot.urdf.xacro (robot description, xacro)
@@ -1,11 +1,11 @@
 <?xml version="1.0"?>
 <robot
-    xmlns:xacro="http://www.ros.org/wiki/xacro" name="module_quadrotor" >
+        xmlns:xacro="http://www.ros.org/wiki/xacro" name="module_quadrotor" >
   <!-- general attribute -->
   <baselink name="fc" />
   <thrust_link name="thrust" />
   <!-- kinematics [m] -->
-  <xacro:property name="rotor_x" value="0.070" />
-  <xacro:property name="rotor_y" value="0.086" />
+  <xacro:property name="rotor_x" value="0.085" />
+  <xacro:property name="rotor_y" value="0.085" />
   <xacro:property name="rotor_z" value="0.026" />
   <!-- dynamics -->
@@ -51,7 +51,7 @@
         <mass value="0.0091"/>
         <inertia
-            ixx="0.00000807" ixy="0.0" ixz="0.0"
-            iyy="0.00000807" iyz="0.0"
-            izz="0.00001612"/>
+                ixx="0.00000807" ixy="0.0" ixz="0.0"
+                iyy="0.00000807" iyz="0.0"
+                izz="0.00001612"/>
       </inertial>
       <visual>
@@ -82,7 +82,7 @@
       <mass value="0.00001"/>
       <inertia
-          ixx="0.000001" ixy="0.0" ixz="0.0"
-          iyy="0.000001" iyz="0.0"
-          izz="0.000002"/>
+              ixx="0.000001" ixy="0.0" ixz="0.0"
+              iyy="0.000001" iyz="0.0"
+              izz="0.000002"/>
     </inertial>
   </link>
@@ -96,15 +96,15 @@
   <link name="main_body">
     <inertial>
-      <mass value = "0.432" />
-      <origin xyz="0 0 0.017" rpy="0 0 0"/>
+      <mass value = "0.832" />
+      <origin xyz="0.002 0 ${0.028 - 0.002}" rpy="0 0 0"/> <!-- TODO: true cog pos -->
       <inertia
-          ixx="0.0021" ixy="0" ixz="0"
-          iyy="0.0015" iyz="0"
-          izz="0.0032"/>
+              ixx="0.0030" ixy="0" ixz="0"
+              iyy="0.0030" iyz="0"
+              izz="0.0045"/>
     </inertial>
     <visual>
       <origin rpy="0 0 0" xyz="0 0 0"/>
       <geometry>
-        <mesh filename="package://mini_quadrotor/urdf/mesh/main_body.dae" />
+        <mesh filename="package://mini_quadrotor/urdf/mesh/main_body_livox.dae" />
       </geometry>
     </visual>
@@ -118,22 +118,43 @@
   <!-- spinal -->
   <xacro:extra_module name = "fc" parent = "main_body" visible = "0" >
-    <origin xyz="0 0 0" rpy="0 0 0"/>
+    <origin xyz="-0.012 -0.003 0.023" rpy="0 0 0"/>
     <inertial>
       <mass value = "00" />
       <origin xyz="0 0 0" rpy="0 0 0"/>
       <inertia
-          ixx="0.0" ixy="0.0" ixz="0.0"
-          iyy="0.0" iyz="0.0" izz="0.0"/>
+              ixx="0.0" ixy="0.0" ixz="0.0"
+              iyy="0.0" iyz="0.0" izz="0.0"/>
+    </inertial>
+  </xacro:extra_module>
+  <!-- livox mid360 -->
+  <xacro:extra_module name = "lidar_imu" parent = "main_body" visible = "0" > <!-- should be IMU frame -->
+    <origin xyz="${0.011} ${0.02329} ${0.0425 + 0.047 - 0.04412}" rpy="0 0 0"/> <!-- TODO: the true pos -->
+    <inertial>
+      <mass value = "00" />
+      <origin xyz="0 0 0" rpy="0 0 0"/>
+      <inertia
+              ixx="0.0" ixy="0.0" ixz="0.0"
+              iyy="0.0" iyz="0.0" izz="0.0"/>
+    </inertial>
+  </xacro:extra_module>
+  <xacro:extra_module name = "livox_link" parent = "main_body" visible = "0" >
+    <origin xyz="0 0 ${0.0425 + 0.047}" rpy="0 0 0"/>
+    <inertial>
+      <mass value = "0" />
+      <origin xyz="0 0 0" rpy="0 0 0"/>
+      <inertia
+              ixx="0.0" ixy="0.0" ixz="0.0"
+              iyy="0.0" iyz="0.0" izz="0.0"/>
     </inertial>
   </xacro:extra_module>
   <!-- battery -->
   <xacro:extra_module name = "battery" parent = "main_body" visible = "1" model_url = "package://mini_quadrotor/urdf/mesh/turnigy_3S_2200mAh.dae" >
-    <origin xyz="0.0105 0 -0.012" rpy="0 0 0"/>
+    <origin xyz="0.0 0 -0.035" rpy="${pi/2} 0 0"/>
     <inertial>
       <mass value = "0.188" />
       <origin xyz="0 0 0" rpy="0 0 0"/>
       <inertia
-          ixx="0.0" ixy="0.0" ixz="0.0"
-          iyy="0.0002" iyz="0.0" izz="0.0002"/>
+              ixx="0.0" ixy="0.0" ixz="0.0"
+              iyy="0.0002" iyz="0.0" izz="0.0002"/>
     </inertial>
   </xacro:extra_module>

Commit message: [mini_quadrotor] update

File: robots/mini_quadrotor/urdf/robot.urdf.xacro (robot description, xacro)
@@ -138,14 +138,14 @@
   </xacro:extra_module>
   <!-- livox mid360 -->
-  <xacro:extra_module name = "lidar_imu" parent = "main_body" visible = "0" > <!-- should be IMU frame -->
-    <origin xyz="${0.011} ${0.02329} ${0.0425 + 0.047 - 0.04412}" rpy="0 0 0"/> <!-- TODO: the true pos -->
-    <inertial>
-      <mass value = "00" />
-      <origin xyz="0 0 0" rpy="0 0 0"/>
-      <inertia
-          ixx="0.0" ixy="0.0" ixz="0.0"
-          iyy="0.0" iyz="0.0" izz="0.0"/>
-    </inertial>
-  </xacro:extra_module>
+  <!-- <xacro:extra_module name = "lidar_imu" parent = "main_body" visible = "0" > <!-\- should be IMU frame -\-> -->
+  <!--   <origin xyz="${0.011} ${0.02329} ${0.0425 + 0.047 - 0.04412}" rpy="0 0 0"/> <!-\- TODO: the true pos -\-> -->
+  <!--   <inertial> -->
+  <!--     <mass value = "00" /> -->
+  <!--     <origin xyz="0 0 0" rpy="0 0 0"/> -->
+  <!--     <inertia -->
+  <!--         ixx="0.0" ixy="0.0" ixz="0.0" -->
+  <!--         iyy="0.0" iyz="0.0" izz="0.0"/> -->
+  <!--   </inertial> -->
+  <!-- </xacro:extra_module> -->
   <!-- battery -->
   <xacro:extra_module name = "battery" parent = "main_body" visible = "1" model_url = "package://mini_quadrotor/urdf/mesh/turnigy_3S_2200mAh.dae" >
