Commit message: Update the mass parameter of dragon

File: robots/dragon/urdf/dragon_link.urdf.xacro (robot description, xacro)
@@ -10,5 +10,5 @@
         <inertial>
           <origin xyz="${link_length* 0.5 + 89.07 * 0.001} ${-6.90 * 0.001} ${-25.71 * 0.001}" rpy="0 0 0"/>
-          <mass value="0.7694" />
+          <mass value="0.7746" />
           <inertia
               ixx="0.0014" iyy="0.0144" izz="0.0137"
@@ -22,5 +22,5 @@
           <inertial>
             <origin xyz="${link_length* 0.5 + 24.31 * 0.001} ${-0.12 * 0.001} ${-18.98 * 0.001}" rpy="0 0 0"/>
-            <mass value="0.7669" />
+            <mass value="0.7721" />
             <inertia
                 ixx="0.0014" iyy="0.0146" izz="0.0134"
@@ -34,5 +34,5 @@
             <inertial>
             <origin xyz="${link_length* 0.5 + 34.31 * 0.001} ${-1.41 * 0.001} ${-12.73 * 0.001}" rpy="0 0 0"/>
-            <mass value="1.0337" />
+            <mass value="1.0389" />
             <inertia
                 ixx="0.0019" iyy="0.0206" izz="0.0197"
@@ -45,5 +45,5 @@
             <inertial>
               <origin xyz="${link_length* 0.5 + 48.08 * 0.001} ${-5.92 * 0.001} ${-15.22 * 0.001}" rpy="0 0 0"/>
-              <mass value="0.9099" />
+              <mass value="0.9151" />
               <inertia
                   ixx="0.0017" iyy="0.0188" izz="0.0179"

Commit message: Add the fc(attached with imu and fcu) frame to provide better kinematics from cog to baselink, also, update the configuration to set the baselink to fc

File: robots/dragon/urdf/dragon_link.urdf.xacro (robot description, xacro)
@@ -198,4 +198,23 @@
       </joint>
     </xacro:if>
+    <!-- set the fcu frame -->
+    <xacro:if value="${baselink}">
+      <link name="fc">
+        <inertial>
+          <origin xyz="0 0 0" rpy="0 0 0"/>
+          <mass value="0.00001"/>
+          <inertia
+              ixx="0.000001" ixy="0.0" ixz="0.0"
+              iyy="0.000001" iyz="0.0"
+              izz="0.000002"/>
+        </inertial>
+      </link>
+      <joint name="fc_joint" type="fixed">
+        <child link="fc"/>
+        <parent link="link${self}"/>
+        <origin rpy="0 0 0" xyz="0.343 0 0.034"/>
+        <axis xyz="0 0 1"/>
+      </joint>
+    </xacro:if>
     <!-- hardware interface -->
     <xacro:unless value="${self == child}">

Commit message: Change the damping rate of joint servo to be higher

File: robots/dragon/urdf/dragon_link.urdf.xacro (robot description, xacro)
@@ -139,5 +139,5 @@
         <origin rpy="0 0 0" xyz="${link_length} 0 0"/>
         <axis xyz="0 1 0"/>
-        <dynamics damping="0.8" friction="0.05"/>
+        <dynamics damping="0.9" friction="0.05"/>
       </joint>
       <!-- inter joint -->
@@ -171,5 +171,5 @@
         <origin rpy="0 0 0" xyz="${2 * inter_joint_x_offset} 0 0"/>
         <axis xyz="0 0 1"/>
-        <dynamics damping="0.8" friction="0.05"/>
+        <dynamics damping="0.9" friction="0.05"/>
       </joint>
       <gazebo reference="inter_joint${self}">

Commit message: Update dragon link model based on intel euclid version

File: robots/dragon/urdf/dragon_link.urdf.xacro (robot description, xacro)
@@ -12,6 +12,6 @@
           <mass value="0.7746" />
           <inertia
-              ixx="0.0014" iyy="0.0144" izz="0.0137"
-              ixy="-0.0009" ixz="-0.0018" iyz="0.0"/>
+              ixx="0.0014" iyy="0.0139" izz="0.0132"
+              ixy="-0.0009" ixz="-0.0017" iyz="0.0"/>
         </inertial>
         <xacro:link_model type="head_link" />
@@ -24,6 +24,6 @@
             <mass value="0.7721" />
             <inertia
-                ixx="0.0014" iyy="0.0146" izz="0.0134"
-                ixy="0.0" ixz="-0.0029" iyz="0.0"/>
+                ixx="0.0014" iyy="0.0142" izz="0.0129"
+                ixy="0.0" ixz="-0.0028" iyz="0.0"/>
           </inertial>
           <xacro:link_model type="end_link" />
@@ -34,8 +34,8 @@
             <inertial>
             <origin xyz="${link_length* 0.5 + 34.31 * 0.001} ${-1.41 * 0.001} ${-12.73 * 0.001}" rpy="0 0 0"/>
-            <mass value="1.0389" />
+            <mass value="1.0861" />
             <inertia
-                ixx="0.0019" iyy="0.0206" izz="0.0197"
-                ixy="-0.0014" ixz="-0.0027" iyz="0.0"/>
+                ixx="0.0022" iyy="0.0234" izz="0.0224"
+                ixy="-0.0016" ixz="-0.0036" iyz="0.0001"/>
             </inertial>
             <xacro:link_model type="baselink" />
@@ -47,6 +47,6 @@
               <mass value="0.9151" />
               <inertia
-                  ixx="0.0017" iyy="0.0188" izz="0.0179"
-                  ixy="-0.0009" ixz="-0.0028" iyz="0.0"/>
+                  ixx="0.0017" iyy="0.0184" izz="0.0174"
+                  ixy="-0.0009" ixz="-0.0027" iyz="0.0"/>
             </inertial>
             <xacro:link_model type="general_link" />

Commit message: Modified the joint speed

File: robots/dragon/urdf/dragon_link.urdf.xacro (robot description, xacro)
@@ -134,5 +134,5 @@
     <xacro:unless value="${self == child}">
       <joint name="joint${self}_pitch" type="revolute">
-        <limit effort="10.0" lower="-1.57" upper="1.57" velocity="0.5"/>
+        <limit effort="10.0" lower="-1.57" upper="1.57" velocity="0.1"/>
         <parent link="link${self}"/>
         <child link="inter_joint${self}"/>
@@ -166,5 +166,5 @@
       </link>
       <joint name="joint${self}_yaw" type="revolute">
-        <limit effort="10.0" lower="-1.57" upper="1.57" velocity="0.5"/>
+        <limit effort="10.0" lower="-1.57" upper="1.57" velocity="0.1"/>
         <parent link="inter_joint${self}"/>
         <child link="link${child}"/>

Commit message: Add the true thrust points of the dual-rotor gimbal module

File: robots/dragon/urdf/dragon_link.urdf.xacro (robot description, xacro)
@@ -122,9 +122,9 @@
       <limit effort="100.0" lower="0" upper="${max_force}" velocity="0.5"/>
       <parent link="gimbal${self}_pitch_module"/>
-      <child link="propeller${self}"/>
+      <child link="thrust${self}"/>
       <origin rpy="0 0 0" xyz="0 0 0"/>
       <axis xyz="0 0 1"/>
     </joint>
-    <link name="propeller${self}">
+    <link name="thrust${self}">
       <inertial>
         <origin xyz="0 0 0.1" rpy="0 0 0"/>
@@ -136,5 +136,38 @@
       </inertial>
     </link>
-    <xacro:damping_factor link ="propeller${self}"/>
+    <!-- special part of duct fun -->
+    <joint name="edf${self}_left_mount" type="fixed">
+      <child link="edf${self}_left"/>
+      <parent link="gimbal${self}_pitch_module"/>
+      <origin rpy="0 0 0" xyz="0 0.1115 0 "/>
+      <axis xyz="0 0 1"/>
+    </joint>
+    <link name="edf${self}_left">
+      <inertial>
+        <origin xyz="0 0 0" rpy="0 0 0"/>
+        <mass value="0.00001"/>
+        <inertia
+            ixx="0.000001" ixy="0.0" ixz="0.0"
+            iyy="0.000001" iyz="0.0"
+            izz="0.000002"/>
+      </inertial>
+    </link>
+    <joint name="edf${self}_right_mount" type="fixed">
+      <child link="edf${self}_right"/>
+      <parent link="gimbal${self}_pitch_module"/>
+      <origin rpy="0 0 0" xyz="0 -0.1115 0 "/>
+      <axis xyz="0 0 1"/>
+    </joint>
+    <link name="edf${self}_right">
+      <inertial>
+        <origin xyz="0 0 0" rpy="0 0 0"/>
+        <mass value="0.00001"/>
+        <inertia
+            ixx="0.000001" ixy="0.0" ixz="0.0"
+            iyy="0.000001" iyz="0.0"
+            izz="0.000002"/>
+      </inertial>
+    </link>
+    <xacro:damping_factor link ="thrust${self}"/>
     <!-- joint -->
     <xacro:unless value="${self == child}">

Commit message: Update the dragon model

File: robots/dragon/urdf/dragon_link.urdf.xacro (robot description, xacro)
@@ -9,10 +9,19 @@
       <xacro:if value="${self == 1}">
         <inertial>
-          <origin xyz="${link_length* 0.5 + 89.07 * 0.001} ${-6.90 * 0.001} ${-25.71 * 0.001}" rpy="0 0 0"/>
-          <mass value="0.7746" />
+          <origin xyz="${link_length* 0.5 + 14.03 * 0.001} ${-7.10 * 0.001} ${-24.66 * 0.001}" rpy="0 0 0"/>
+          <mass value="0.7485" />
           <inertia
-              ixx="0.0014" iyy="0.0139" izz="0.0132"
-              ixy="-0.0009" ixz="-0.0017" iyz="0.0"/>
+              ixx="0.0014" iyy="0.0154" izz="0.0147"
+              ixy="-0.0008" ixz="0.0006" iyz="0.0"/>
         </inertial>
+        <!-- old: zippy 3000mAh type
+             <inertial>
+             <origin xyz="${link_length* 0.5 + 89.07 * 0.001} ${-6.90 * 0.001} ${-25.71 * 0.001}" rpy="0 0 0"/>
+             <mass value="0.7746" />
+             <inertia
+             ixx="0.0014" iyy="0.0139" izz="0.0132"
+             ixy="-0.0009" ixz="-0.0017" iyz="0.0"/>
+             </inertial>
+        -->
         <xacro:link_model type="head_link" />
       </xacro:if>
@@ -21,10 +30,19 @@
         <xacro:if value="${self == child}">
           <inertial>
-            <origin xyz="${link_length* 0.5 + 24.31 * 0.001} ${-0.12 * 0.001} ${-18.98 * 0.001}" rpy="0 0 0"/>
-            <mass value="0.7721" />
+            <origin xyz="${link_length* 0.5 - 47.26 * 0.001} ${-0.12 * 0.001} ${-17.74 * 0.001}" rpy="0 0 0"/>
+            <mass value="0.7460" />
             <inertia
-                ixx="0.0014" iyy="0.0142" izz="0.0129"
-                ixy="0.0" ixz="-0.0028" iyz="0.0"/>
+                ixx="0.0014" iyy="0.0158" izz="0.0145"
+                ixy="0.0" ixz="-0.0006" iyz="0.0"/>
           </inertial>
+          <!-- old: zippy 3000mAh type
+               <inertial>
+               <origin xyz="${link_length* 0.5 + 24.31 * 0.001} ${-0.12 * 0.001} ${-18.98 * 0.001}" rpy="0 0 0"/>
+               <mass value="0.7721" />
+               <inertia
+               ixx="0.0014" iyy="0.0142" izz="0.0129"
+               ixy="0.0" ixz="-0.0028" iyz="0.0"/>
+               </inertial>
+          -->
           <xacro:link_model type="end_link" />
         </xacro:if>
@@ -33,10 +51,19 @@
           <xacro:if value="${baselink}">
             <inertial>
-            <origin xyz="${link_length* 0.5 + 34.31 * 0.001} ${-1.41 * 0.001} ${-12.73 * 0.001}" rpy="0 0 0"/>
-            <mass value="1.0861" />
-            <inertia
-                ixx="0.0022" iyy="0.0234" izz="0.0224"
-                ixy="-0.0016" ixz="-0.0036" iyz="0.0001"/>
+              <origin xyz="${link_length* 0.5 + 17.70 * 0.001} ${-5.98 * 0.001} ${-16.85 * 0.001}" rpy="0 0 0"/>
+              <mass value="1.0646" />
+              <inertia
+                  ixx="0.0021" iyy="0.0251" izz="0.0240"
+                  ixy="-0.0011" ixz="-0.0014" iyz="0.0"/>
             </inertial>
+            <!-- old: zippy 3000mAh type
+                 <inertial>
+                 <origin xyz="${link_length* 0.5 + 34.31 * 0.001} ${-1.41 * 0.001} ${-12.73 * 0.001}" rpy="0 0 0"/>
+                 <mass value="1.0861" />
+                 <inertia
+                 ixx="0.0022" iyy="0.0234" izz="0.0224"
+                 ixy="-0.0016" ixz="-0.0036" iyz="0.0001"/>
+                 </inertial>
+            -->
             <xacro:link_model type="baselink" />
           </xacro:if>
@@ -44,10 +71,19 @@
           <xacro:unless value="${baselink}">
             <inertial>
-              <origin xyz="${link_length* 0.5 + 48.08 * 0.001} ${-5.92 * 0.001} ${-15.22 * 0.001}" rpy="0 0 0"/>
-              <mass value="0.9151" />
+              <origin xyz="${link_length* 0.5 - 11.42 * 0.001} ${-6.06 * 0.001} ${-14.09 * 0.001}" rpy="0 0 0"/>
+              <mass value="0.8890" />
               <inertia
-                  ixx="0.0017" iyy="0.0184" izz="0.0174"
-                  ixy="-0.0009" ixz="-0.0027" iyz="0.0"/>
+                  ixx="0.0017" iyy="0.02" izz="0.019"
+                  ixy="-0.0009" ixz="-0.0004" iyz="0.0"/>
             </inertial>
+            <!-- old: zippy 3000mAh type
+                 <inertial>
+                 <origin xyz="${link_length* 0.5 + 48.08 * 0.001} ${-5.92 * 0.001} ${-15.22 * 0.001}" rpy="0 0 0"/>
+                 <mass value="0.9151" />
+                 <inertia
+                 ixx="0.0017" iyy="0.0184" izz="0.0174"
+                 ixy="-0.0009" ixz="-0.0027" iyz="0.0"/>
+                 </inertial>
+            -->
             <xacro:link_model type="general_link" />
           </xacro:unless>
@@ -67,10 +103,19 @@
     <link name="gimbal${self}_roll_module">
       <inertial>
-        <origin xyz="${gimbal_roll_x_offset - 17.20968 * 0.001} ${0.41439 * 0.001} ${15.61551 * 0.001}" rpy="0 0 0"/>
-        <mass value="0.44011" />
-        <inertia
-            ixx="0.0005" iyy="0.0007" izz="0.0003"
+        <origin xyz="${gimbal_roll_x_offset - 17.46431 * 0.001} ${0.42738 * 0.001} ${15.47344 * 0.001}" rpy="0 0 0"/>
+        <mass value="0.45058" />
+        <inertia
+            ixx="0.0005" iyy="0.0007" izz="0.0004"
             ixy="0" ixz="-0.0002" iyz="0.0"/>
       </inertial>
+      <!-- old: zippy 3000mAh type
+           <inertial>
+           <origin xyz="${gimbal_roll_x_offset - 17.20968 * 0.001} ${0.41439 * 0.001} ${15.61551 * 0.001}" rpy="0 0 0"/>
+           <mass value="0.44011" />
+           <inertia
+           ixx="0.0005" iyy="0.0007" izz="0.0003"
+           ixy="0" ixz="-0.0002" iyz="0.0"/>
+           </inertial>
+      -->
       <visual>
         <origin xyz="${gimbal_roll_x_offset} 0 0" rpy="0 0 0"/>

Commit message: Update the baselink module mass parameter

File: robots/dragon/urdf/dragon_link.urdf.xacro (robot description, xacro)
@@ -51,9 +51,9 @@
           <xacro:if value="${baselink}">
             <inertial>
-              <origin xyz="${link_length* 0.5 + 17.70 * 0.001} ${-5.98 * 0.001} ${-16.85 * 0.001}" rpy="0 0 0"/>
-              <mass value="1.0646" />
+              <origin xyz="${link_length* 0.5 + 18.74 * 0.001} ${-5.98 * 0.001} ${-17.04 * 0.001}" rpy="0 0 0"/>
+              <mass value="1.0717" />
               <inertia
-                  ixx="0.0021" iyy="0.0251" izz="0.0240"
-                  ixy="-0.0011" ixz="-0.0014" iyz="0.0"/>
+                  ixx="0.0021" iyy="0.0253" izz="0.0242"
+                  ixy="-0.0011" ixz="-0.0015" iyz="0.0"/>
             </inertial>
             <!-- old: zippy 3000mAh type

Commit message: Update the drogon model (the position change of intel euclid)

File: robots/dragon/urdf/dragon_link.urdf.xacro (robot description, xacro)
@@ -15,13 +15,4 @@
               ixy="-0.0008" ixz="0.0006" iyz="0.0"/>
         </inertial>
-        <!-- old: zippy 3000mAh type
-             <inertial>
-             <origin xyz="${link_length* 0.5 + 89.07 * 0.001} ${-6.90 * 0.001} ${-25.71 * 0.001}" rpy="0 0 0"/>
-             <mass value="0.7746" />
-             <inertia
-             ixx="0.0014" iyy="0.0139" izz="0.0132"
-             ixy="-0.0009" ixz="-0.0017" iyz="0.0"/>
-             </inertial>
-        -->
         <xacro:link_model type="head_link" />
       </xacro:if>
@@ -36,13 +27,4 @@
                 ixy="0.0" ixz="-0.0006" iyz="0.0"/>
           </inertial>
-          <!-- old: zippy 3000mAh type
-               <inertial>
-               <origin xyz="${link_length* 0.5 + 24.31 * 0.001} ${-0.12 * 0.001} ${-18.98 * 0.001}" rpy="0 0 0"/>
-               <mass value="0.7721" />
-               <inertia
-               ixx="0.0014" iyy="0.0142" izz="0.0129"
-               ixy="0.0" ixz="-0.0028" iyz="0.0"/>
-               </inertial>
-          -->
           <xacro:link_model type="end_link" />
         </xacro:if>
@@ -51,19 +33,10 @@
           <xacro:if value="${baselink}">
             <inertial>
-              <origin xyz="${link_length* 0.5 + 18.74 * 0.001} ${-5.98 * 0.001} ${-17.04 * 0.001}" rpy="0 0 0"/>
-              <mass value="1.0717" />
+              <origin xyz="${link_length* 0.5 + 9.75 * 0.001} ${-5.03 * 0.001} ${-14.39 * 0.001}" rpy="0 0 0"/>
+              <mass value="1.0697" />
               <inertia
-                  ixx="0.0021" iyy="0.0253" izz="0.0242"
-                  ixy="-0.0011" ixz="-0.0015" iyz="0.0"/>
+                  ixx="0.0019" iyy="0.0226" izz="0.0217"
+                  ixy="-0.0009" ixz="-0.0007" iyz="0.0"/>
             </inertial>
-            <!-- old: zippy 3000mAh type
-                 <inertial>
-                 <origin xyz="${link_length* 0.5 + 34.31 * 0.001} ${-1.41 * 0.001} ${-12.73 * 0.001}" rpy="0 0 0"/>
-                 <mass value="1.0861" />
-                 <inertia
-                 ixx="0.0022" iyy="0.0234" izz="0.0224"
-                 ixy="-0.0016" ixz="-0.0036" iyz="0.0001"/>
-                 </inertial>
-            -->
             <xacro:link_model type="baselink" />
           </xacro:if>
@@ -77,13 +50,4 @@
                   ixy="-0.0009" ixz="-0.0004" iyz="0.0"/>
             </inertial>
-            <!-- old: zippy 3000mAh type
-                 <inertial>
-                 <origin xyz="${link_length* 0.5 + 48.08 * 0.001} ${-5.92 * 0.001} ${-15.22 * 0.001}" rpy="0 0 0"/>
-                 <mass value="0.9151" />
-                 <inertia
-                 ixx="0.0017" iyy="0.0184" izz="0.0174"
-                 ixy="-0.0009" ixz="-0.0027" iyz="0.0"/>
-                 </inertial>
-            -->
             <xacro:link_model type="general_link" />
           </xacro:unless>
@@ -109,13 +73,4 @@
             ixy="0" ixz="-0.0002" iyz="0.0"/>
       </inertial>
-      <!-- old: zippy 3000mAh type
-           <inertial>
-           <origin xyz="${gimbal_roll_x_offset - 17.20968 * 0.001} ${0.41439 * 0.001} ${15.61551 * 0.001}" rpy="0 0 0"/>
-           <mass value="0.44011" />
-           <inertia
-           ixx="0.0005" iyy="0.0007" izz="0.0003"
-           ixy="0" ixz="-0.0002" iyz="0.0"/>
-           </inertial>
-      -->
       <visual>
         <origin xyz="${gimbal_roll_x_offset} 0 0" rpy="0 0 0"/>

Commit message: Fix the wrong place of color assignment for dragon model

File: robots/dragon/urdf/dragon_link.urdf.xacro (robot description, xacro)
@@ -77,6 +77,6 @@
         <geometry>
           <mesh filename="package://dragon/urdf/mesh/ducted_fan_gimbal_roll.stl" scale="0.001 0.001 0.001"/>
-          <material name="red"/>
         </geometry>
+        <material name="red"/>
       </visual>
       <collision>

Commit message: Fix the wrong offset of head link

File: robots/dragon/urdf/dragon_link.urdf.xacro (robot description, xacro)
@@ -9,5 +9,5 @@
       <xacro:if value="${self == 1}">
         <inertial>
-          <origin xyz="${link_length* 0.5 + 14.03 * 0.001} ${-7.10 * 0.001} ${-24.66 * 0.001}" rpy="0 0 0"/>
+          <origin xyz="${link_length* 0.5 + 20.63 * 0.001} ${-7.10 * 0.001} ${-24.66 * 0.001}" rpy="0 0 0"/>
           <mass value="0.7485" />
           <!-- bad problem: https://github.com/tongtybj/aerial_robot/issues/155
@@ -16,6 +16,6 @@
               ixy="-0.0008" ixz="0.0006" iyz="0.0"/> -->
           <inertia
-              ixx="0.00089834" iyy="0.0148345" izz="0.01457051"
-              ixy="0.00077224" ixz="-0.00087587" iyz="0.00011817"/>
+              ixx="0.00090734" iyy="0.01452037" izz="0.01426033"
+              ixy="0.00078582" ixz="-0.00090857" iyz="0.0001282"/>
         </inertial>
         <xacro:link_model type="head_link" />

Commit message: Update the collision model of dragon link, i.e., the padding model for dragon gimbal module

File: robots/dragon/urdf/dragon_link.urdf.xacro (robot description, xacro)
@@ -110,7 +110,7 @@
       <!-- cylinder collision geometry works well for FCL -->
       <collision>
-        <origin rpy="${pi/2} 0 0" xyz="${gimbal_roll_x_offset}  0 0"/>
+        <origin rpy="${pi/2} 0 0" xyz="0 0 0.02"/>
         <geometry>
-          <cylinder length="0.3" radius="0.08" />
+          <cylinder length="0.3" radius="0.09" />
         </geometry>
       </collision>

Commit message: Update the actuator limits for hydrus and dragon

File: robots/dragon/urdf/dragon_link.urdf.xacro (robot description, xacro)
@@ -195,5 +195,5 @@
     <xacro:unless value="${self == child}">
       <joint name="joint${self}_pitch" type="revolute">
-        <limit effort="10.0" lower="-1.57" upper="1.57" velocity="0.1"/>
+        <limit effort="10.0" lower="${-pi/2}" upper="${pi/2}" velocity="0.1"/>
         <parent link="link${self}"/>
         <child link="inter_joint${self}"/>
@@ -220,5 +220,5 @@
       </link>
       <joint name="joint${self}_yaw" type="revolute">
-        <limit effort="10.0" lower="-1.57" upper="1.57" velocity="0.1"/>
+        <limit effort="10.0" lower="${-pi/2}" upper="${pi/2}" velocity="0.1"/>
         <parent link="inter_joint${self}"/>
         <child link="link${child}"/>

File: robots/hydrus/urdf/link.urdf.xacro (robot description, xacro)
@@ -107,5 +107,5 @@
     <xacro:unless value="${self == child}">
       <joint name="joint${self}" type="revolute">
-        <limit effort="10.0" lower="-1.57" upper="1.57" velocity="0.5"/>
+        <limit effort="10.0" lower="${-pi/2}" upper="${pi/2}" velocity="0.5"/>
         <parent link="link${self}"/>
         <child link="link${child}"/>

Commit message: - Update the mass/inertial for dragon with bumpered spinal - Tune the p gain for pos xy control regarding to gimbal vectoring

File: robots/dragon/urdf/dragon_link.urdf.xacro (robot description, xacro)
@@ -42,5 +42,5 @@
             <inertial>
               <origin xyz="${link_length* 0.5 + 9.75 * 0.001} ${-5.03 * 0.001} ${-14.39 * 0.001}" rpy="0 0 0"/>
-              <mass value="1.0697" />
+              <mass value="1.092" />
               <!-- bad problem: https://github.com/tongtybj/aerial_robot/issues/155
               <inertia
@@ -266,5 +266,5 @@
         <child link="fc"/>
         <parent link="link${self}"/>
-        <origin rpy="0 0 0" xyz="0.343 0 0.034"/>
+        <origin rpy="0 0 0" xyz="0.330 -0.004 0.053"/>
         <axis xyz="0 0 1"/>
       </joint>

Commit message: Update the mass/inertial of baselink for dragon with bumpered spinal (version2)

File: robots/dragon/urdf/dragon_link.urdf.xacro (robot description, xacro)
@@ -41,6 +41,6 @@
           <xacro:if value="${baselink}">
             <inertial>
-              <origin xyz="${link_length* 0.5 + 9.75 * 0.001} ${-5.03 * 0.001} ${-14.39 * 0.001}" rpy="0 0 0"/>
-              <mass value="1.0697" />
+              <origin xyz="${link_length* 0.5 + 11.73 * 0.001} ${-4.91 * 0.001} ${-13.87 * 0.001}" rpy="0 0 0"/>
+              <mass value="1.096" />
               <!-- bad problem: https://github.com/tongtybj/aerial_robot/issues/155
               <inertia
@@ -266,5 +266,5 @@
         <child link="fc"/>
         <parent link="link${self}"/>
-        <origin rpy="0 0 0" xyz="0.343 0 0.034"/>
+        <origin rpy="0 0 0" xyz="0.316 -0.004 0.043"/>
         <axis xyz="0 0 1"/>
       </joint>
