Commit message: Update the mass/inertial of baselink for dragon with bumpered spinal (version2)

File: robots/dragon/urdf/dragon_link.urdf.xacro (robot description, xacro)
@@ -41,6 +41,6 @@
           <xacro:if value="${baselink}">
             <inertial>
-              <origin xyz="${link_length* 0.5 + 9.75 * 0.001} ${-5.03 * 0.001} ${-14.39 * 0.001}" rpy="0 0 0"/>
-              <mass value="1.092" />
+              <origin xyz="${link_length* 0.5 + 11.73 * 0.001} ${-4.91 * 0.001} ${-13.87 * 0.001}" rpy="0 0 0"/>
+              <mass value="1.096" />
               <!-- bad problem: https://github.com/tongtybj/aerial_robot/issues/155
               <inertia
@@ -266,5 +266,5 @@
         <child link="fc"/>
         <parent link="link${self}"/>
-        <origin rpy="0 0 0" xyz="0.330 -0.004 0.053"/>
+        <origin rpy="0 0 0" xyz="0.316 -0.004 0.043"/>
         <axis xyz="0 0 1"/>
       </joint>

Commit message: Update the inertial parameters since some components are changed in dragon

File: robots/dragon/urdf/dragon_link.urdf.xacro (robot description, xacro)
@@ -9,13 +9,9 @@
       <xacro:if value="${self == 1}">
         <inertial>
-          <origin xyz="${link_length* 0.5 + 20.63 * 0.001} ${-7.10 * 0.001} ${-24.66 * 0.001}" rpy="0 0 0"/>
-          <mass value="0.7485" />
-          <!-- bad problem: https://github.com/tongtybj/aerial_robot/issues/155
+          <origin xyz="${link_length* 0.5 + 18.25 * 0.001} ${-7.17 * 0.001} ${-25.73 * 0.001}" rpy="0 0 0"/>
+          <mass value="0.7408" />
           <inertia
-              ixx="0.0014" iyy="0.0154" izz="0.0147"
-              ixy="-0.0008" ixz="0.0006" iyz="0.0"/> -->
-          <inertia
-              ixx="0.0009" iyy="0.0146" izz="0.0143"
-              ixy="-0.0009" ixz="0.0002" iyz="0.0001"/>
+              ixx="0.00095" iyy="0.0143" izz="0.0139"
+              ixy="-0.00099" ixz="0.0003" iyz="0.0001"/>
         </inertial>
         <xacro:link_model type="head_link" />
@@ -25,13 +21,9 @@
         <xacro:if value="${self == child}">
           <inertial>
-            <origin xyz="${link_length* 0.5 - 47.26 * 0.001} ${-0.12 * 0.001} ${-17.74 * 0.001}" rpy="0 0 0"/>
-            <mass value="0.7460" />
-            <!-- bad problem: https://github.com/tongtybj/aerial_robot/issues/155
+            <origin xyz="${link_length* 0.5 - 45.44 * 0.001} ${-0.12 * 0.001} ${-18.74 * 0.001}" rpy="0 0 0"/>
+            <mass value="0.7383" />
             <inertia
-                ixx="0.0014" iyy="0.0158" izz="0.0145"
-                ixy="0.0" ixz="-0.0006" iyz="0.0"/> -->
-            <inertia
-                ixx="0.0012" iyy="0.0139" izz="0.0128"
-                ixy="0.0" ixz="0.0" iyz="0.0"/>
+                ixx="0.0012" iyy="0.0137" izz="0.0126"
+                ixy="0.0" ixz="0.0002" iyz="0.0"/>
           </inertial>
           <xacro:link_model type="end_link" />
@@ -41,13 +33,9 @@
           <xacro:if value="${baselink}">
             <inertial>
-              <origin xyz="${link_length* 0.5 + 11.73 * 0.001} ${-4.91 * 0.001} ${-13.87 * 0.001}" rpy="0 0 0"/>
-              <mass value="1.096" />
-              <!-- bad problem: https://github.com/tongtybj/aerial_robot/issues/155
+              <origin xyz="${link_length* 0.5 + 11.92 * 0.001} ${-4.98 * 0.001} ${-14.07 * 0.001}" rpy="0 0 0"/>
+              <mass value="1.07879" />
               <inertia
-                  ixx="0.0019" iyy="0.0226" izz="0.0217"
-                  ixy="-0.0009" ixz="-0.0007" iyz="0.0"/> -->
-              <inertia
-                  ixx="0.0017" iyy="0.0223" izz="0.0216"
-                  ixy="-0.0009" ixz="-0.0009" iyz="0.0001"/>
+                  ixx="0.0018" iyy="0.0219" izz="0.0211"
+                  ixy="-0.001" ixz="-0.0007" iyz="0.0001"/>
             </inertial>
             <xacro:link_model type="baselink" />
@@ -56,13 +44,9 @@
           <xacro:unless value="${baselink}">
             <inertial>
-              <origin xyz="${link_length* 0.5 - 11.42 * 0.001} ${-6.06 * 0.001} ${-14.09 * 0.001}" rpy="0 0 0"/>
-              <mass value="0.8890" />
-              <!-- bad problem: https://github.com/tongtybj/aerial_robot/issues/155
+              <origin xyz="${link_length* 0.5 - 11.75 * 0.001} ${-6.17 * 0.001} ${-15.04 * 0.001}" rpy="0 0 0"/>
+              <mass value="0.8729" />
               <inertia
-                  ixx="0.0017" iyy="0.02" izz="0.019"
-                  ixy="-0.0009" ixz="-0.0004" iyz="0.0"/> -->
-              <inertia
-                  ixx="0.0013" iyy="0.0194" izz="0.0188"
-                  ixy="-0.0008" ixz="0.0007" iyz="0.0"/>
+                  ixx="0.0015" iyy="0.0189" izz="0.0181"
+                  ixy="-0.0008" ixz="-0.0002" iyz="0.0001"/>
             </inertial>
             <xacro:link_model type="general_link" />
@@ -83,13 +67,8 @@
     <link name="gimbal${self}_roll_module">
       <inertial>
-        <origin xyz="${gimbal_roll_x_offset - 17.46431 * 0.001} ${0.42738 * 0.001} ${15.47344 * 0.001}" rpy="0 0 0"/>
-        <mass value="0.45058" />
-        <!-- bad problem: https://github.com/tongtybj/aerial_robot/issues/155
-        <inertia
-            ixx="0.0005" iyy="0.0007" izz="0.0004"
-            ixy="0" ixz="-0.0002" iyz="0.0"/>
-        -->
-        <inertia
-            ixx="0.0004" iyy="0.0005" izz="0.0003"
+        <origin xyz="${gimbal_roll_x_offset - 17.67 * 0.001} ${0.42 * 0.001} ${15.23 * 0.001}" rpy="0 0 0"/>
+        <mass value="0.4578" />
+        <inertia
+            ixx="0.0004" iyy="0.0004" izz="0.0002"
             ixy="0" ixz="-0.0003" iyz="0"/>
       </inertial>
@@ -127,8 +106,8 @@
     <link name="gimbal${self}_pitch_module">
       <inertial>
-        <origin xyz="0 ${0.47 * 0.001}  ${-7.38 * 0.001}" rpy="0 0 0"/>
-        <mass value=".4187" />
-        <inertia
-            ixx="0.0047" iyy="0.0002" izz="0.0047"
+        <origin xyz="0 ${0.46 * 0.001}  ${-7.3 * 0.001}" rpy="0 0 0"/>
+        <mass value="0.4235" />
+        <inertia
+            ixx="0.0048" iyy="0.0002" izz="0.0048"
             ixy="0.0" ixz="0.0" iyz="0.0"/>
       </inertial>

Commit message: Update the inertial parameters since some components are changed in dragon

File: robots/dragon/urdf/dragon_link.urdf.xacro (robot description, xacro)
@@ -9,13 +9,9 @@
       <xacro:if value="${self == 1}">
         <inertial>
-          <origin xyz="${link_length* 0.5 + 20.63 * 0.001} ${-7.10 * 0.001} ${-24.66 * 0.001}" rpy="0 0 0"/>
-          <mass value="0.7485" />
-          <!-- bad problem: https://github.com/JSKAerialRobot/aerial_robot/issues/155
+          <origin xyz="${link_length* 0.5 + 18.25 * 0.001} ${-7.17 * 0.001} ${-25.73 * 0.001}" rpy="0 0 0"/>
+          <mass value="0.7408" />
           <inertia
-              ixx="0.0014" iyy="0.0154" izz="0.0147"
-              ixy="-0.0008" ixz="0.0006" iyz="0.0"/> -->
-          <inertia
-              ixx="0.0009" iyy="0.0146" izz="0.0143"
-              ixy="-0.0009" ixz="0.0002" iyz="0.0001"/>
+              ixx="0.00095" iyy="0.0143" izz="0.0139"
+              ixy="-0.00099" ixz="0.0003" iyz="0.0001"/>
         </inertial>
         <xacro:link_model type="head_link" />
@@ -25,13 +21,9 @@
         <xacro:if value="${self == child}">
           <inertial>
-            <origin xyz="${link_length* 0.5 - 47.26 * 0.001} ${-0.12 * 0.001} ${-17.74 * 0.001}" rpy="0 0 0"/>
-            <mass value="0.7460" />
-            <!-- bad problem: https://github.com/JSKAerialRobot/aerial_robot/issues/155
+            <origin xyz="${link_length* 0.5 - 45.44 * 0.001} ${-0.12 * 0.001} ${-18.74 * 0.001}" rpy="0 0 0"/>
+            <mass value="0.7383" />
             <inertia
-                ixx="0.0014" iyy="0.0158" izz="0.0145"
-                ixy="0.0" ixz="-0.0006" iyz="0.0"/> -->
-            <inertia
-                ixx="0.0012" iyy="0.0139" izz="0.0128"
-                ixy="0.0" ixz="0.0" iyz="0.0"/>
+                ixx="0.0012" iyy="0.0137" izz="0.0126"
+                ixy="0.0" ixz="0.0002" iyz="0.0"/>
           </inertial>
           <xacro:link_model type="end_link" />
@@ -41,13 +33,9 @@
           <xacro:if value="${baselink}">
             <inertial>
-              <origin xyz="${link_length* 0.5 + 11.73 * 0.001} ${-4.91 * 0.001} ${-13.87 * 0.001}" rpy="0 0 0"/>
-              <mass value="1.096" />
-              <!-- bad problem: https://github.com/JSKAerialRobot/aerial_robot/issues/155
+              <origin xyz="${link_length* 0.5 + 11.92 * 0.001} ${-4.98 * 0.001} ${-14.07 * 0.001}" rpy="0 0 0"/>
+              <mass value="1.07879" />
               <inertia
-                  ixx="0.0019" iyy="0.0226" izz="0.0217"
-                  ixy="-0.0009" ixz="-0.0007" iyz="0.0"/> -->
-              <inertia
-                  ixx="0.0017" iyy="0.0223" izz="0.0216"
-                  ixy="-0.0009" ixz="-0.0009" iyz="0.0001"/>
+                  ixx="0.0018" iyy="0.0219" izz="0.0211"
+                  ixy="-0.001" ixz="-0.0007" iyz="0.0001"/>
             </inertial>
             <xacro:link_model type="baselink" />
@@ -56,13 +44,9 @@
           <xacro:unless value="${baselink}">
             <inertial>
-              <origin xyz="${link_length* 0.5 - 11.42 * 0.001} ${-6.06 * 0.001} ${-14.09 * 0.001}" rpy="0 0 0"/>
-              <mass value="0.8890" />
-              <!-- bad problem: https://github.com/JSKAerialRobot/aerial_robot/issues/155
+              <origin xyz="${link_length* 0.5 - 11.75 * 0.001} ${-6.17 * 0.001} ${-15.04 * 0.001}" rpy="0 0 0"/>
+              <mass value="0.8729" />
               <inertia
-                  ixx="0.0017" iyy="0.02" izz="0.019"
-                  ixy="-0.0009" ixz="-0.0004" iyz="0.0"/> -->
-              <inertia
-                  ixx="0.0013" iyy="0.0194" izz="0.0188"
-                  ixy="-0.0008" ixz="0.0007" iyz="0.0"/>
+                  ixx="0.0015" iyy="0.0189" izz="0.0181"
+                  ixy="-0.0008" ixz="-0.0002" iyz="0.0001"/>
             </inertial>
             <xacro:link_model type="general_link" />
@@ -83,13 +67,8 @@
     <link name="gimbal${self}_roll_module">
       <inertial>
-        <origin xyz="${gimbal_roll_x_offset - 17.46431 * 0.001} ${0.42738 * 0.001} ${15.47344 * 0.001}" rpy="0 0 0"/>
-        <mass value="0.45058" />
-        <!-- bad problem: https://github.com/JSKAerialRobot/aerial_robot/issues/155
-        <inertia
-            ixx="0.0005" iyy="0.0007" izz="0.0004"
-            ixy="0" ixz="-0.0002" iyz="0.0"/>
-        -->
-        <inertia
-            ixx="0.0004" iyy="0.0005" izz="0.0003"
+        <origin xyz="${gimbal_roll_x_offset - 17.67 * 0.001} ${0.42 * 0.001} ${15.23 * 0.001}" rpy="0 0 0"/>
+        <mass value="0.4578" />
+        <inertia
+            ixx="0.0004" iyy="0.0004" izz="0.0002"
             ixy="0" ixz="-0.0003" iyz="0"/>
       </inertial>
@@ -127,8 +106,8 @@
     <link name="gimbal${self}_pitch_module">
       <inertial>
-        <origin xyz="0 ${0.47 * 0.001}  ${-7.38 * 0.001}" rpy="0 0 0"/>
-        <mass value=".4187" />
-        <inertia
-            ixx="0.0047" iyy="0.0002" izz="0.0047"
+        <origin xyz="0 ${0.46 * 0.001}  ${-7.3 * 0.001}" rpy="0 0 0"/>
+        <mass value="0.4235" />
+        <inertia
+            ixx="0.0048" iyy="0.0002" izz="0.0048"
             ixy="0.0" ixz="0.0" iyz="0.0"/>
       </inertial>

Commit message: Implement the strict solver for the nonlinear vectoring force allocation problem by SLSQP (nlopt)
Complete:
- nonlinear allocation for hovering (only gravity, no torque) with both numerical / analytical gradient
- nonlinear allocation for target wrench with numerical gradient
- nonlinear allocation for target wrench with analytical gradient, but constant inertia (depreacated)
- nonlinear allocation for target wrench with analytical gradient

File: robots/dragon/urdf/dragon_link.urdf.xacro (robot description, xacro)
@@ -129,5 +129,5 @@
     <link name="thrust${self}">
       <inertial>
-        <origin xyz="0 0 0.1" rpy="0 0 0"/>
+        <origin xyz="0 0 0" rpy="0 0 0"/>
         <mass value="0.0001"/>
         <inertia

Commit message: fix dragon_link.urdf.xacro for head

File: robots/dragon/urdf/dragon_link.urdf.xacro (robot description, xacro)
@@ -84,4 +84,27 @@
     </link>
     <xacro:damping_factor link ="link${self}"/>
+    <link name="link${self}_edge">
+      <inertial>
+        <origin xyz="0 0 0" rpy="0 0 0"/>
+        <mass value="0.00001"/>
+        <inertia
+            ixx="0.000001" ixy="0.0" ixz="0.0"
+            iyy="0.000001" iyz="0.0"
+            izz="0.000002"/>
+      </inertial>
+    </link>
+    <joint name="link${self}_edge_fixed_joint" type="fixed">
+      <xacro:if value="${child > 0}">
+        <parent link="link${self}"/>
+        <child link="link${self}_edge"/>
+        <origin rpy="0 0 0" xyz="${link_length} 0 0"/>
+      </xacro:if>
+      <xacro:if value="${parent > 0}">
+        <parent link="link${self}_edge"/>
+        <child link="link${self}"/>
+        <origin rpy="0 0 0" xyz="${-1 * link_length} 0 0 "/>
+      </xacro:if>
+      <axis xyz="0 0 1"/>
+    </joint>
     <!-- gimbal roll -->
     <joint name="gimbal${self}_roll" type="revolute">
@@ -203,14 +226,16 @@
       <joint name="joint${self}_pitch" type="revolute">
         <limit effort="10.0" lower="${-pi/2}" upper="${pi/2}" velocity="0.1"/>
+        <xacro:if value="${child > 0}">
+          <parent link="link${self}_edge"/>
+          <child link="inter_joint${self}"/>
+          <origin rpy="0 0 0" xyz="0 0 0"/>
+          <axis xyz="0 1 0"/>
+        </xacro:if>
         <xacro:if value="${parent > 0}">
           <parent link="inter_joint${self}"/>
-          <child link="link${self}"/>
-        </xacro:if>
-        <xacro:if value="${child > 0}">
-          <parent link="link${self}"/>
-          <child link="inter_joint${self}"/>
-        </xacro:if>
-        <origin rpy="0 0 0" xyz="${link_length} 0 0"/>
-        <axis xyz="0 1 0"/>
+          <child link="link${self}_edge"/>
+          <origin rpy="0 0 0" xyz="${-2 * inter_joint_x_offset} 0 0"/>
+          <axis xyz="0 -1 0"/>
+        </xacro:if>
         <dynamics damping="0.9" friction="0.05"/>
       </joint>
@@ -226,5 +251,10 @@
         </inertial>
         <visual>
-          <origin rpy="0 0 0" xyz="${inter_joint_x_offset} 0 0"/>
+          <xacro:if value="${child > 0}">
+            <origin rpy="0 0 0" xyz="${inter_joint_x_offset} 0 0"/>
+          </xacro:if>
+          <xacro:if value="${parent > 0}">
+            <origin rpy="0 0 0" xyz="${-1 * inter_joint_x_offset} 0 0"/>
+          </xacro:if>
           <geometry>
             <mesh filename="package://dragon/urdf/mesh/inter_joint_junction.dae"/>
@@ -237,11 +267,13 @@
           <parent link="inter_joint${self}"/>
           <child link="link${child}"/>
+          <origin rpy="0 0 0" xyz="${2 * inter_joint_x_offset} 0 0"/>
+          <axis xyz="0 0 1"/>
         </xacro:if>
         <xacro:if value="${parent > 0}">
           <parent link="link${parent}"/>
           <child link="inter_joint${self}"/>
-        </xacro:if>
-        <origin rpy="0 0 0" xyz="${2 * inter_joint_x_offset} 0 0"/>
-        <axis xyz="0 0 1"/>
+          <origin rpy="0 0 0" xyz="0 0 0"/>
+          <axis xyz="0 0 -1"/>
+        </xacro:if>
         <dynamics damping="0.9" friction="0.05"/>
       </joint>

Commit message: [Dragon] update the dragon model for new thrust system

File: robots/dragon/urdf/dragon_link.urdf.xacro (robot description, xacro)
@@ -95,8 +95,8 @@
     <link name="gimbal${self}_roll_module">
       <inertial>
-        <origin xyz="${gimbal_roll_x_offset - 17.67 * 0.001} ${0.42 * 0.001} ${15.23 * 0.001}" rpy="0 0 0"/>
-        <mass value="0.4578" />
-        <inertia
-            ixx="0.0004" iyy="0.0005" izz="0.0003"
+        <origin xyz="${gimbal_roll_x_offset - 17.60 * 0.001} ${0.42 * 0.001} ${15.48 * 0.001}" rpy="0 0 0"/>
+        <mass value="0.4604" />
+        <inertia
+            ixx="0.0004" iyy="0.0004" izz="0.0003"
             ixy="0" ixz="-0.0003" iyz="0"/>
       </inertial>
@@ -134,8 +134,8 @@
     <link name="gimbal${self}_pitch_module">
       <inertial>
-        <origin xyz="0 ${0.46 * 0.001}  ${-7.3 * 0.001}" rpy="0 0 0"/>
-        <mass value="0.4235" />
-        <inertia
-            ixx="0.0048" iyy="0.0002" izz="0.0048"
+        <origin xyz="0 ${0.33 * 0.001}  ${-8.71 * 0.001}" rpy="0 0 0"/>
+        <mass value="0.5301" />
+        <inertia
+            ixx="0.0061" iyy="0.0001" izz="0.0061"
             ixy="0.0" ixz="0.0" iyz="0.0"/>
       </inertial>

Commit message: [Dragon] update the inerital paramter for dragon links, which shift to LiHV battery (6s 1300mAh) from Lipo.

File: robots/dragon/urdf/dragon_link.urdf.xacro (robot description, xacro)
@@ -9,4 +9,10 @@
       <xacro:if value="${self == 1}">
         <inertial>
+          <origin xyz="${link_length* 0.5 + 15.09 * 0.001} ${-6.67 * 0.001} ${-27.21 * 0.001}" rpy="0 0 0"/>
+          <mass value="0.7968" />
+          <inertia
+              ixx="0.00095" iyy="0.0151" izz="0.0148"
+              ixy="-0.00098" ixz="0.0003" iyz="0.0001"/>
+          <!--
           <origin xyz="${link_length* 0.5 + 18.25 * 0.001} ${-7.17 * 0.001} ${-25.73 * 0.001}" rpy="0 0 0"/>
           <mass value="0.7408" />
@@ -14,4 +20,5 @@
               ixx="0.00095" iyy="0.0143" izz="0.0139"
               ixy="-0.00099" ixz="0.0003" iyz="0.0001"/>
+          -->
         </inertial>
         <xacro:link_model type="head_link" />
@@ -21,4 +28,10 @@
         <xacro:if value="${self == child}">
           <inertial>
+            <origin xyz="${link_length* 0.5 - 44.26 * 0.001} ${-0.11 * 0.001} ${-20.72 * 0.001}" rpy="0 0 0"/>
+            <mass value="0.7943" />
+            <inertia
+                ixx="0.0012" iyy="0.0145" izz="0.0134"
+                ixy="0.0" ixz="0.0003" iyz="0.0000"/>
+            <!--
             <origin xyz="${link_length* 0.5 - 45.44 * 0.001} ${-0.12 * 0.001} ${-18.74 * 0.001}" rpy="0 0 0"/>
             <mass value="0.7383" />
@@ -26,4 +39,5 @@
                 ixx="0.0012" iyy="0.0137" izz="0.0126"
                 ixy="0.0" ixz="0.0002" iyz="0.0"/>
+            -->
           </inertial>
           <xacro:link_model type="end_link" />
@@ -33,4 +47,10 @@
           <xacro:if value="${baselink}">
             <inertial>
+              <origin xyz="${link_length* 0.5 + 9.54 * 0.001} ${-4.74 * 0.001} ${-15.68 * 0.001}" rpy="0 0 0"/>
+              <mass value="1.1348" />
+              <inertia
+                  ixx="0.0018" iyy="0.0228" izz="0.0219"
+                  ixy="-0.0009" ixz="-0.0006" iyz="0.0001"/>
+              <!--
               <origin xyz="${link_length* 0.5 + 11.92 * 0.001} ${-4.98 * 0.001} ${-14.07 * 0.001}" rpy="0 0 0"/>
               <mass value="1.07879" />
@@ -38,4 +58,5 @@
                   ixx="0.0018" iyy="0.0219" izz="0.0211"
                   ixy="-0.001" ixz="-0.0007" iyz="0.0001"/>
+              -->
             </inertial>
             <xacro:link_model type="baselink" />
@@ -44,4 +65,10 @@
           <xacro:unless value="${baselink}">
             <inertial>
+              <origin xyz="${link_length* 0.5 - 12.78 * 0.001} ${-5.80 * 0.001} ${-16.95 * 0.001}" rpy="0 0 0"/>
+              <mass value="0.9289" />
+              <inertia
+                  ixx="0.0015" iyy="0.0198" izz="0.0189"
+                  ixy="-0.0008" ixz="-0.0001" iyz="0.0001"/>
+              <!--
               <origin xyz="${link_length* 0.5 - 11.75 * 0.001} ${-6.17 * 0.001} ${-15.04 * 0.001}" rpy="0 0 0"/>
               <mass value="0.8729" />
@@ -49,4 +76,5 @@
                   ixx="0.0015" iyy="0.0189" izz="0.0181"
                   ixy="-0.0008" ixz="-0.0002" iyz="0.0001"/>
+              -->
             </inertial>
             <xacro:link_model type="general_link" />
@@ -129,5 +157,5 @@
     <link name="thrust${self}">
       <inertial>
-        <origin xyz="0 0 0.1" rpy="0 0 0"/>
+        <origin xyz="0 0 0" rpy="0 0 0"/>
         <mass value="0.0001"/>
         <inertia

Commit message: [dragon] fix urdf not to include rotor as joint

File: robots/dragon/urdf/dragon_link.urdf.xacro (robot description, xacro)
@@ -148,6 +148,6 @@
     </link>
     <!-- rotor -->
-    <joint name="rotor${self}" type="continuous">
-      <limit effort="100.0" lower="${min_force}" upper="${max_force}" velocity="0.5"/>
+    <joint name="rotor${self}" type="fixed">
+      <!-- <limit effort="100.0" lower="${min_force}" upper="${max_force}" velocity="0.5"/> -->
       <parent link="gimbal${self}_pitch_module"/>
       <child link="thrust${self}"/>
@@ -324,15 +324,15 @@
       </actuator>
     </transmission>
-    <transmission name="rotor${self}_tran">
-      <type>transmission_interface/SimpleTransmission</type>
-      <joint name="rotor${self}">
-        <hardwareInterface>RotorInterface</hardwareInterface>
-      </joint>
-      <actuator name="rotor${self}">
-        <hardwareInterface>RotorInterface</hardwareInterface>
-        <mechanicalReduction>1</mechanicalReduction>
-      </actuator>
-      </transmission>
-    <xacro:friction self ="${self}"/>
+    <!-- <transmission name="rotor${self}_tran"> -->
+    <!--   <type>transmission_interface/SimpleTransmission</type> -->
+    <!--   <joint name="rotor${self}"> -->
+    <!--     <hardwareInterface>RotorInterface</hardwareInterface> -->
+    <!--   </joint> -->
+    <!--   <actuator name="rotor${self}"> -->
+    <!--     <hardwareInterface>RotorInterface</hardwareInterface> -->
+    <!--     <mechanicalReduction>1</mechanicalReduction> -->
+    <!--   </actuator> -->
+    <!--   </transmission> -->
+    <!-- <xacro:friction self ="${self}"/> -->
   </xacro:macro>
 </robot>
