Commit message: Revert "[dragon] fix urdf not to include rotor as joint"
This reverts commit c18a8b07d3fc95acfbad47671238a8fee4504973.

File: robots/dragon/urdf/dragon_link.urdf.xacro (robot description, xacro)
@@ -148,6 +148,6 @@
     </link>
     <!-- rotor -->
-    <joint name="rotor${self}" type="fixed">
-      <!-- <limit effort="100.0" lower="${min_force}" upper="${max_force}" velocity="0.5"/> -->
+    <joint name="rotor${self}" type="continuous">
+      <limit effort="100.0" lower="${min_force}" upper="${max_force}" velocity="0.5"/>
       <parent link="gimbal${self}_pitch_module"/>
       <child link="thrust${self}"/>
@@ -324,15 +324,15 @@
       </actuator>
     </transmission>
-    <!-- <transmission name="rotor${self}_tran"> -->
-    <!--   <type>transmission_interface/SimpleTransmission</type> -->
-    <!--   <joint name="rotor${self}"> -->
-    <!--     <hardwareInterface>RotorInterface</hardwareInterface> -->
-    <!--   </joint> -->
-    <!--   <actuator name="rotor${self}"> -->
-    <!--     <hardwareInterface>RotorInterface</hardwareInterface> -->
-    <!--     <mechanicalReduction>1</mechanicalReduction> -->
-    <!--   </actuator> -->
-    <!--   </transmission> -->
-    <!-- <xacro:friction self ="${self}"/> -->
+    <transmission name="rotor${self}_tran">
+      <type>transmission_interface/SimpleTransmission</type>
+      <joint name="rotor${self}">
+        <hardwareInterface>RotorInterface</hardwareInterface>
+      </joint>
+      <actuator name="rotor${self}">
+        <hardwareInterface>RotorInterface</hardwareInterface>
+        <mechanicalReduction>1</mechanicalReduction>
+      </actuator>
+      </transmission>
+    <xacro:friction self ="${self}"/>
   </xacro:macro>
 </robot>
