Commit message: Correct the collsion model for dragon

File: robots/dragon/urdf/dragon_common.xacro (robot description, xacro)
@@ -25,5 +25,5 @@
       <origin rpy="0 0 0" xyz="${link_length* 0.5} 0 0"/>
       <geometry>
-        <box size="0.05 0.05 0.1686"/>
+        <box size="${link_length} 0.1 0.1686"/>
       </geometry>
     </collision>
@@ -39,6 +39,6 @@
   <xacro:macro name="friction" params="self">
     <gazebo reference="link${self}">
-      <mu1>0.2</mu1>
-      <mu2>0.2</mu2>
+      <mu1>0.0001</mu1>
+      <mu2>0.0001</mu2>
       <material>Gazebo/Black</material>
     </gazebo>

File: robots/dragon/urdf/dragon_link.urdf.xacro (robot description, xacro)
@@ -80,4 +80,10 @@
         </geometry>
       </visual>
+      <collision>
+        <origin rpy="0 0 0" xyz="${gimbal_roll_x_offset}  0 0"/>
+        <geometry>
+          <box size="0.1 0.3 0.1686"/>
+        </geometry>
+      </collision>
     </link>
     <gazebo reference="gimbal${self}_roll_module">
@@ -151,10 +157,4 @@
               ixy="0" ixz="0.0" iyz="0.0"/>
         </inertial>
-        <collision>
-          <origin rpy="0 0 0" xyz="${2 * inter_joint_x_offset} 0 0"/>
-          <geometry>
-            <cylinder length="0.1686" radius="0.011"/>
-          </geometry>
-        </collision>
         <visual>
           <origin rpy="0 0 0" xyz="${inter_joint_x_offset} 0 0"/>

Commit message: Update the dragon collision geometry to be more friendly for FCL

File: robots/dragon/urdf/dragon_common.xacro (robot description, xacro)
@@ -22,10 +22,19 @@
   <xacro:property name="max_force" value="30" /> <!-- [N] -->
   <xacro:macro name="link_model" params="type">
+    <!-- box collision geometry does not work well for FCL -->
     <collision>
-      <origin rpy="0 0 0" xyz="${link_length* 0.5} 0 0"/>
+    <origin rpy="0 0 0" xyz="${link_length* 0.5} 0 0"/>
+    <geometry>
+    <box size="${link_length} 0.15 0.1686"/>
+    </geometry>
+    </collision>
+    <!-- cylinder collision geometry works well for FCL
+    <collision>
+      <origin rpy="0 ${pi/2} 0" xyz="${link_length* 0.5} 0 0"/>
       <geometry>
-        <box size="${link_length} 0.1 0.1686"/>
+        <cylinder length="${link_length}" radius="0.06" />
       </geometry>
     </collision>
+    -->
     <visual>
       <origin rpy="0 0 0" xyz="${link_length* 0.5} 0 0"/>
@@ -39,6 +48,6 @@
   <xacro:macro name="friction" params="self">
     <gazebo reference="link${self}">
-      <mu1>0.0001</mu1>
-      <mu2>0.0001</mu2>
+      <mu1>0.2</mu1>
+      <mu2>0.2</mu2>
       <material>Gazebo/Black</material>
     </gazebo>

File: robots/dragon/urdf/dragon_link.urdf.xacro (robot description, xacro)
@@ -80,8 +80,17 @@
         <material name="red"/>
       </visual>
+      <!-- box collision not work good for FCL
       <collision>
         <origin rpy="0 0 0" xyz="${gimbal_roll_x_offset}  0 0"/>
         <geometry>
           <box size="0.1 0.3 0.1686"/>
+        </geometry>
+      </collision>
+      -->
+      <!-- cylinder collision geometry works well for FCL -->
+      <collision>
+        <origin rpy="${pi/2} 0 0" xyz="${gimbal_roll_x_offset}  0 0"/>
+        <geometry>
+          <cylinder length="0.3" radius="0.08" />
         </geometry>
       </collision>

Commit message: Update (Fix) the inertial matrix of each module (e.g. link, gimbal) to be suitable for the rull of URDF, that is based on the inertial frame (cog frame). Previous inertial matrix is with repecti to the link origin frame, which is the rule of Solid Edge.

File: robots/dragon/urdf/dragon_common.xacro (robot description, xacro)
@@ -40,6 +40,6 @@
   <xacro:macro name="friction" params="self">
     <gazebo reference="link${self}">
-      <mu1>0.2</mu1>
-      <mu2>0.2</mu2>
+      <mu1>0.4</mu1>
+      <mu2>0.4</mu2>
     </gazebo>
   </xacro:macro>

File: robots/dragon/urdf/dragon_link.urdf.xacro (robot description, xacro)
@@ -11,7 +11,11 @@
           <origin xyz="${link_length* 0.5 + 14.03 * 0.001} ${-7.10 * 0.001} ${-24.66 * 0.001}" rpy="0 0 0"/>
           <mass value="0.7485" />
+          <!-- bad problem: https://github.com/tongtybj/aerial_robot/issues/155
           <inertia
               ixx="0.0014" iyy="0.0154" izz="0.0147"
-              ixy="-0.0008" ixz="0.0006" iyz="0.0"/>
+              ixy="-0.0008" ixz="0.0006" iyz="0.0"/> -->
+          <inertia
+              ixx="0.00089834" iyy="0.0148345" izz="0.01457051"
+              ixy="0.00077224" ixz="-0.00087587" iyz="0.00011817"/>
         </inertial>
         <xacro:link_model type="head_link" />
@@ -23,7 +27,11 @@
             <origin xyz="${link_length* 0.5 - 47.26 * 0.001} ${-0.12 * 0.001} ${-17.74 * 0.001}" rpy="0 0 0"/>
             <mass value="0.7460" />
+            <!-- bad problem: https://github.com/tongtybj/aerial_robot/issues/155
             <inertia
                 ixx="0.0014" iyy="0.0158" izz="0.0145"
-                ixy="0.0" ixz="-0.0006" iyz="0.0"/>
+                ixy="0.0" ixz="-0.0006" iyz="0.0"/> -->
+            <inertia
+                ixx="${1.21645440 * 0.001}" iyy="${1.39001170 * 0.01}" izz="${1.28812312 * 0.01}"
+                ixy="${1.00390000 * 0.00001}" ixz="${1.17225120 * 0.001}" iyz="${2.89500000 * 0.000001}"/>
           </inertial>
           <xacro:link_model type="end_link" />
@@ -35,7 +43,11 @@
               <origin xyz="${link_length* 0.5 + 9.75 * 0.001} ${-5.03 * 0.001} ${-14.39 * 0.001}" rpy="0 0 0"/>
               <mass value="1.0697" />
+              <!-- bad problem: https://github.com/tongtybj/aerial_robot/issues/155
               <inertia
                   ixx="0.0019" iyy="0.0226" izz="0.0217"
-                  ixy="-0.0009" ixz="-0.0007" iyz="0.0"/>
+                  ixy="-0.0009" ixz="-0.0007" iyz="0.0"/> -->
+              <inertia
+                  ixx="${1.65168720 * 0.001}" iyy="${2.23498232 * 0.01}" izz="${2.16125712 * 0.01}"
+                  ixy="${8.74188000 * 0.0001}" ixz="${5.33822400 * 0.0001}" iyz="${7.75584000 * 0.00001}"/>
             </inertial>
             <xacro:link_model type="baselink" />
@@ -46,7 +58,11 @@
               <origin xyz="${link_length* 0.5 - 11.42 * 0.001} ${-6.06 * 0.001} ${-14.09 * 0.001}" rpy="0 0 0"/>
               <mass value="0.8890" />
+              <!-- bad problem: https://github.com/tongtybj/aerial_robot/issues/155
               <inertia
                   ixx="0.0017" iyy="0.02" izz="0.019"
-                  ixy="-0.0009" ixz="-0.0004" iyz="0.0"/>
+                  ixy="-0.0009" ixz="-0.0004" iyz="0.0"/> -->
+              <inertia
+                  ixx="${1.46927480 * 0.001}" iyy="${1.97395958 * 0.01}" izz="${1.88998884 * 0.01}"
+                  ixy="${9.65232800 * 0.0001}" ixz="${5.77743600 * 0.0001}" iyz="${9.10326000 * 0.00001}"/>
             </inertial>
             <xacro:link_model type="general_link" />
@@ -69,7 +85,12 @@
         <origin xyz="${gimbal_roll_x_offset - 17.46431 * 0.001} ${0.42738 * 0.001} ${15.47344 * 0.001}" rpy="0 0 0"/>
         <mass value="0.45058" />
+        <!-- bad problem: https://github.com/tongtybj/aerial_robot/issues/155
         <inertia
             ixx="0.0005" iyy="0.0007" izz="0.0004"
             ixy="0" ixz="-0.0002" iyz="0.0"/>
+        -->
+        <inertia
+            ixx="${4.49938835 * 0.0001}" iyy="${5.44075766 * 0.0001}" izz="${2.74350095 * 0.0001}"
+            ixy="${-3.56050862 * 0.000001}" ixz="${1.17396333 * 0.0001}" iyz="${1.01694621 * 0.00001}"/>
       </inertial>
       <visual>
@@ -109,5 +130,5 @@
         <mass value=".4187" />
         <inertia
-            ixx="0.0047" iyy="0.0002" izz="0.0047"
+            ixx="0.0047171" iyy="0.0001518" izz="0.0047442"
             ixy="0" ixz="0.0" iyz="0.0"/>
       </inertial>

Commit message: improve dragon mesh file

File: robots/dragon/urdf/dragon_common.xacro (robot description, xacro)
@@ -12,11 +12,4 @@
   <xacro:property name="gimbal_roll_x_offset" value="-0.01" />
   <xacro:property name="gimbal_pitch_z_offset" value="0.037" />
-  <!-- material color for rviz -->
-  <material name="black">
-    <color rgba="0 0 0 1"/>
-  </material>
-  <material name="red">
-    <color rgba="1 0 0 1"/>
-  </material>
   <!-- dynamics -->
   <xacro:property name="max_force" value="30" /> <!-- [N] -->
@@ -40,7 +33,6 @@
       <origin rpy="0 0 0" xyz="${link_length* 0.5} 0 0"/>
       <geometry>
-        <mesh filename="package://dragon/urdf/mesh/ducted_fan_${type}.stl" scale="0.001 0.001 0.001"/>
+        <mesh filename="package://dragon/urdf/mesh/ducted_fan_${type}.dae"/>
       </geometry>
-      <material name="black"/>
     </visual>
   </xacro:macro>
@@ -50,5 +42,4 @@
       <mu1>0.2</mu1>
       <mu2>0.2</mu2>
-      <material>Gazebo/Black</material>
     </gazebo>
   </xacro:macro>

File: robots/dragon/urdf/dragon_link.urdf.xacro (robot description, xacro)
@@ -76,7 +76,6 @@
         <origin xyz="${gimbal_roll_x_offset} 0 0" rpy="0 0 0"/>
         <geometry>
-          <mesh filename="package://dragon/urdf/mesh/ducted_fan_gimbal_roll.stl" scale="0.001 0.001 0.001"/>
+          <mesh filename="package://dragon/urdf/mesh/ducted_fan_gimbal_roll.dae"/>
         </geometry>
-        <material name="red"/>
       </visual>
       <!-- box collision not work good for FCL
@@ -96,7 +95,4 @@
       </collision>
     </link>
-    <gazebo reference="gimbal${self}_roll_module">
-      <material>Gazebo/Red</material>
-    </gazebo>
     <!-- gimbal pitch -->
     <joint name="gimbal${self}_pitch" type="revolute">
@@ -119,12 +115,8 @@
         <origin xyz="0 0 0" rpy="0 0 0"/>
         <geometry>
-          <mesh filename="package://dragon/urdf/mesh/ducted_fan_gimbal_pitch.stl" scale="0.001 0.001 0.001"/>
+          <mesh filename="package://dragon/urdf/mesh/ducted_fan_gimbal_pitch.dae"/>
         </geometry>
-        <material name="black"/>
       </visual>
     </link>
-    <gazebo reference="gimbal${self}_pitch_module">
-      <material>Gazebo/Black</material>
-    </gazebo>
     <!-- rotor -->
     <joint name="rotor${self}" type="continuous">
@@ -202,7 +194,6 @@
           <origin rpy="0 0 0" xyz="${inter_joint_x_offset} 0 0"/>
           <geometry>
-            <mesh filename="package://dragon/urdf/mesh/inter_joint_junction.stl" scale="0.001 0.001 0.001"/>
+            <mesh filename="package://dragon/urdf/mesh/inter_joint_junction.dae"/>
           </geometry>
-          <material name="red"/>
         </visual>
       </link>
@@ -218,5 +209,4 @@
         <mu1>0.2</mu1>
         <mu2>0.2</mu2>
-        <material>Gazebo/Red</material>
       </gazebo>
     </xacro:unless>

Commit message: Query rotor properties from urdf files: thrust min/max, m_f_rate

File: robots/dragon/urdf/dragon_common.xacro (robot description, xacro)
@@ -16,5 +16,7 @@
   <xacro:property name="gimbal_pitch_z_offset" value="0.037" />
   <!-- dynamics -->
+  <m_f_rate value="0" /> <!-- drug torque rate -->
   <xacro:property name="max_force" value="30" /> <!-- [N] -->
+  <xacro:property name="min_force" value="2" /> <!-- [N] -->
   <xacro:macro name="link_model" params="type">
     <!-- box collision geometry does not work well for FCL -->

File: robots/dragon/urdf/dragon_link.urdf.xacro (robot description, xacro)
@@ -142,5 +142,5 @@
     <!-- rotor -->
     <joint name="rotor${self}" type="continuous">
-      <limit effort="100.0" lower="0" upper="${max_force}" velocity="0.5"/>
+      <limit effort="100.0" lower="${min_force}" upper="${max_force}" velocity="0.5"/>
       <parent link="gimbal${self}_pitch_module"/>
       <child link="thrust${self}"/>

File: robots/hydrus/robots/quad/old_model_tx2_rs_t265_201906/robot.urdf.xacro (robot description, xacro)
@@ -3,4 +3,5 @@
     xmlns:xacro="http://www.ros.org/wiki/xacro" name="hydrusx" >
   <!-- basic kinematics model -->
+  <m_f_rate value="-0.0182" /> <!-- overwrite -->
   <xacro:include filename="$(find hydrus)/urdf/common.xacro" />
   <xacro:include filename="$(find hydrus)/urdf/link.urdf.xacro" />

File: robots/hydrus/robots/quad/old_model_tx2_zed_201810/robot.urdf.xacro (robot description, xacro)
@@ -3,4 +3,5 @@
     xmlns:xacro="http://www.ros.org/wiki/xacro" name="hydrusx" >
   <!-- basic kinematics model -->
+  <m_f_rate value="-0.0182" /> <!-- overwrite -->
   <xacro:include filename="$(find hydrus)/urdf/common.xacro" />
   <xacro:include filename="$(find hydrus)/urdf/link.urdf.xacro" />

File: robots/hydrus/urdf/common.xacro (robot description, xacro)
@@ -17,5 +17,7 @@
   <xacro:property name="leg_collision_model_height" value="0.1715" />
   <!-- dynamics -->
-  <xacro:property name="max_force" value="18" /> <!-- [N] -->
+  <m_f_rate value="-0.0172" /> <!-- drug torque rate -->
+  <xacro:property name="max_force" value="16.5" /> <!-- [N] -->
+  <xacro:property name="min_force" value="1.0" /> <!-- [N] -->
   <xacro:macro name="link_model" params="type with_leg:=${with_leg} old_version:=${old_version} tilt_mode:=${tilt_mode} tilt_angle:=${tilt_angle}">
     <!-- for fcl in planning -->

File: robots/hydrus/urdf/link.urdf.xacro (robot description, xacro)
@@ -144,5 +144,5 @@
     <!-- rotor -->
     <joint name="rotor${self}" type="continuous">
-      <limit effort="100.0" lower="0" upper="${max_force}" velocity="0.5"/> <!-- force range -->
+      <limit effort="100.0" lower="${min_force}" upper="${max_force}" velocity="0.5"/>
       <parent link="link${self}"/>
       <child link="thrust${self}"/>

File: robots/hydrus_xi/urdf/branch_type_link.urdf.xacro (robot description, xacro)
@@ -204,5 +204,5 @@
     #### rotor joint (virtual) ####
     <joint name="rotor${self}" type="continuous">
-     <limit effort="100.0" lower="0" upper="${max_force}" velocity="0.5"/>
+     <limit effort="100.0" lower="${min_force}" upper="${max_force}" velocity="0.5"/>
       <parent link="rotor_parent${self}"/>
       <child link="thrust${self}"/>

File: robots/hydrus_xi/urdf/common.xacro (robot description, xacro)
@@ -17,5 +17,7 @@
   <xacro:property name="bat_mass" value="0.193"/> <!-- 1300mAh -->
   <!-- dynamics -->
+  <m_f_rate value="-0.0182" /> <!-- MN4010KV475_Afro_15inch -->
   <xacro:property name="max_force" value="24"/> <!-- [N] -->
+  <xacro:property name="min_force" value="1"/> <!-- [N] -->
   <!-- collision -->
   <xacro:property name="collision_rotor_height" value="0.1" />

File: robots/hydrus_xi/urdf/link.urdf.xacro (robot description, xacro)
@@ -139,5 +139,5 @@
     #### rotor joint (virtual) ####
     <joint name="rotor${self}" type="continuous">
-     <limit effort="100.0" lower="0" upper="${max_force}" velocity="0.5"/>
+     <limit effort="100.0" lower="${min_force}" upper="${max_force}" velocity="0.5"/>
       <parent link="rotor_parent${self}"/>
       <child link="thrust${self}"/>

Commit message: [Dragon][Thrust] fix the wrong limitation of the thrust

File: robots/dragon/urdf/dragon_common.xacro (robot description, xacro)
@@ -17,5 +17,5 @@
   <!-- dynamics -->
   <m_f_rate value="0" /> <!-- drug torque rate -->
-  <xacro:property name="max_force" value="30" /> <!-- [N] -->
+  <xacro:property name="max_force" value="36" /> <!-- [N] -->
   <xacro:property name="min_force" value="2" /> <!-- [N] -->
   <xacro:macro name="link_model" params="type">
