Commit message: reduce max force

File: robots/delta/urdf/20240722/thrust.urdf.xacro (robot description, xacro)
@@ -3,5 +3,5 @@
     xmlns:xacro="http://www.ros.org/wiki/xacro" name="delta_common" >
   <m_f_rate value="-0.0156" /> <!-- drug torque rate -->
-  <xacro:property name="max_force" value="26.5" /> <!-- [N] -->
+  <xacro:property name="max_force" value="23.0" /> <!-- [N] -->
   <xacro:property name="min_force" value="0.0" /> <!-- [N] -->
 </robot>
