Commit message: [delta][quad] fixed rotor tilt and livox

File: robots/delta/robots/quad/20240722/delta.urdf.xacro (robot description, xacro)
@@ -4,8 +4,8 @@
   <xacro:include filename="$(find delta)/urdf/20240722/delta_link.urdf.xacro" />
   <xacro:include filename="$(find delta)/urdf/common.xacro" />
-  <xacro:delta_module self="1" child="2" rotor_direction="1" rotor_tilt="-0.0727822" battery="0"/>
-  <xacro:delta_module self="2" child="3" rotor_direction="-1" rotor_tilt="0.178982" battery="0"/>
-  <xacro:delta_module self="3" child="4" rotor_direction="1" rotor_tilt="-0.0802372"  battery="0"/>
-  <xacro:delta_module self="4" child="4" rotor_direction="-1" rotor_tilt="0.178982" battery="0"/>
+  <xacro:delta_module self="1" child="2" rotor_direction="1" rotor_tilt="0" battery="0"/>
+  <xacro:delta_module self="2" child="3" rotor_direction="-1" rotor_tilt="0" battery="0"/>
+  <xacro:delta_module self="3" child="4" rotor_direction="1" rotor_tilt="0"  battery="0"/>
+  <xacro:delta_module self="4" child="4" rotor_direction="-1" rotor_tilt="0" battery="0"/>
   <!-- dummy root link for KDL -->
   <link name="root">
@@ -47,5 +47,5 @@
   </xacro:extra_module>
   <!-- vio sensor -->
-  <xacro:extra_module name="lidar_imu_link" parent="link2" visible="1" model_url="package://delta/urdf/mesh/20240722/livox.dae" active="1">
+  <xacro:extra_module name="lidar_imu_link" parent="link2" visible="1" model_url="package://delta/urdf/mesh/20240722/livox.dae" active="0">
     <origin xyz="0.3635 -0.01 0" rpy="0 ${pi/2} ${-pi/2}"/>
     <inertial>
@@ -57,7 +57,7 @@
     </inertial>
   </xacro:extra_module>
-  <xacro:extra_module name="lidar_imu" parent="lidar_imu_link">
-    <origin xyz="0 0 0.03905" rpy="0 0 0"/>
-    <xacro:virtual_inertial/>
-  </xacro:extra_module>
+  <!-- <xacro:extra_module name="lidar_imu" parent="lidar_imu_link"> -->
+  <!--   <origin xyz="0 0 0.03905" rpy="0 0 0"/> -->
+  <!--   <xacro:virtual_inertial/> -->
+  <!-- </xacro:extra_module> -->
 </robot>

Commit message: integrate soft-airframe code into delta (fly in the simulation)

File: robots/delta/robots/quad/20240722/delta.urdf.xacro (robot description, xacro)
@@ -61,3 +61,319 @@
   <!--   <xacro:virtual_inertial/> -->
   <!-- </xacro:extra_module> -->
+  <!-- 3 soft_airframe -->
+  <link name="soft_link1">
+    <inertial>
+      <origin xyz="0.06875 0.000002 0.018960" rpy="0 0 0"/>
+      <mass value="${0.010*2 + 0.012}"/>
+      <inertia
+          ixx="0.00003988" ixy="0.0" ixz="0.0"
+          iyy="0.00010606" iyz="0.0"
+          izz="0.00010185"/>
+    </inertial>
+    <visual>
+      <geometry>
+        <box size="0.1175 0.03 0.04"/>
+      </geometry>
+      <origin xyz="0.05875 0 0.02" rpy="0 0 0"/>
+    </visual>
+  </link>
+  <gazebo reference="soft_link1">
+    <mu1>0.1</mu1>
+    <mu2>0.1</mu2>
+  </gazebo>
+  <xacro:damping_factor link="soft_link1"/>
+  <link name="soft_link2">
+    <inertial>
+      <origin xyz="0.1175 0.000002 0.019998" rpy="0 0 0"/>
+      <mass value="${0.010*5 + 0.012*2}"/>
+      <inertia
+          ixx="0.00006787" ixy="0.0" ixz="0.0"
+          iyy="0.00049831" iyz="0.0"
+          izz="0.00048990"/>
+    </inertial>
+    <visual>
+      <geometry>
+        <box size="0.235 0.03 0.04"/>
+      </geometry>
+      <origin xyz="0.1175 0.000002 0.019998" rpy="0 0 0"/>
+    </visual>
+  </link>
+  <gazebo reference="soft_link2">
+    <mu1>0.1</mu1>
+    <mu2>0.1</mu2>
+  </gazebo>
+  <xacro:damping_factor link="soft_link2"/>
+  <link name="soft_link3">
+    <inertial>
+      <origin xyz="0.10740316 0.0 0.003" rpy="0 0 0"/>
+      <mass value="${0.010*2 + 0.012 + 0.070 + 0.016}"/>
+      <inertia
+          ixx="0.00005679" ixy="-0.000000031" ixz="-0.00002256"
+          iyy="0.00028149" iyz="0.000000005"
+          izz="0.00026759"/>
+    </inertial>
+    <visual>
+      <geometry>
+        <box size="0.1175 0.03 0.04"/>
+      </geometry>
+      <origin xyz="0.05875 0 0.02" rpy="0 0 0"/>
+    </visual>
+  </link>
+  <gazebo reference="soft_link3">
+    <mu1>0.1</mu1>
+    <mu2>0.1</mu2>
+  </gazebo>
+  <xacro:damping_factor link="soft_link3"/>
+  <link name="servo_link">
+    <inertial>
+      <origin xyz="0 0 0" rpy="0 0 0"/>
+      <mass value="0.073"/>
+      <!-- this is for avoiding error in gazebo -->
+      <!-- <inertia
+          ixx="0.001" ixy="0.0" ixz="0.0"
+          iyy="0.001" iyz="0.0"
+          izz="0.002"/> -->
+      <inertia
+          ixx="0.000017" ixy="0.000003" ixz="-0.0000001"
+          iyy="0.000023" iyz="0.000000"
+          izz="0.000025"/>
+    </inertial>
+    <visual>
+      <geometry>
+        <box size="0.05 0.05 0.05"/>
+      </geometry>
+      <origin xyz="0 0 -0.02" rpy="0 0 0"/>
+    </visual>
+  </link>
+  <gazebo reference="servo_link">
+    <mu1>0.1</mu1>
+    <mu2>0.1</mu2>
+  </gazebo>
+  <xacro:damping_factor link="servo_link"/>
+  <link name="servo_link1">
+    <inertial>
+      <origin xyz="0 0 0" rpy="0 0 0"/>
+      <mass value="0.068"/>
+      <!-- this is for avoiding error in gazebo -->
+      <!-- <inertia
+          ixx="0.001" ixy="0.0" ixz="0.0"
+          iyy="0.001" iyz="0.0"
+          izz="0.002"/> -->
+      <inertia
+          ixx="0.000016" ixy="-0.000003" ixz="0.000001"
+          iyy="0.000019" iyz="0.000000"
+          izz="0.000022"/>
+    </inertial>
+    <visual>
+      <geometry>
+        <box size="0.05 0.05 0.05"/>
+      </geometry>
+      <origin xyz="0 0 -0.02" rpy="0 0 0"/>
+    </visual>
+  </link>
+  <gazebo reference="servo_link1">
+    <mu1>0.1</mu1>
+    <mu2>0.1</mu2>
+  </gazebo>
+  <xacro:damping_factor link="servo_link1"/>
+  <joint name="soft_joint1" type="fixed">
+    <parent link="link4"/>
+    <child link="soft_link1"/>
+    <origin xyz="0.6 0 0" rpy="0 0 0"/>
+  </joint>
+  <joint name="soft_joint2" type="revolute">
+    <limit effort="5.0" lower="${-pi/2}" upper="${pi/2}" velocity="0.5"/>
+    <parent link="soft_link1"/>
+    <child link="soft_link2"/>
+    <origin xyz="0.1175 0 0" rpy="0 0 0"/>
+    <axis xyz="0 0 1"/>
+    <dynamics damping="0.9" friction="0.1"/>
+  </joint>
+  <joint name="soft_joint3" type="revolute">
+    <limit effort="5.0" lower="${-pi/2}" upper="${pi/2}" velocity="0.5"/>
+    <parent link="soft_link2"/>
+    <child link="soft_link3"/>
+    <origin xyz="0.235 0 0" rpy="0 0 0"/>
+    <axis xyz="0 0 1"/>
+    <dynamics damping="0.9" friction="0.1"/>
+  </joint>
+  <!-- <gazebo reference="soft_link3">
+    <stopCfm>1000</stopCfm>
+  </gazebo> -->
+  <joint name="soft_joint4" type="revolute">
+    <limit effort="5.0" lower="${-pi/2}" upper="${pi/2}" velocity="0.5"/>
+    <parent link="link4"/>
+    <child link="servo_link"/>
+    <origin xyz="0.5 0 0.01" rpy="0 0 0"/>
+    <axis xyz="0 0 1"/>
+    <dynamics damping="0.9" friction="0.1"/>
+  </joint>
+  <joint name="soft_joint5" type="revolute">
+    <limit effort="5.0" lower="${-pi/2}" upper="${pi/2}" velocity="0.5"/>
+    <parent link="link4"/>
+    <child link="servo_link1"/>
+    <origin xyz="0.5 0 -0.01" rpy="0 0 0"/>
+    <axis xyz="0 0 1"/>
+    <dynamics damping="0.9" friction="0.1"/>
+  </joint>
+  <transmission name="soft_joint_tran_2">
+    <type>transmission_interface/SimpleTransmission</type>
+    <joint name="soft_joint2">
+      <hardwareInterface>hardware_interface/EffortJointInterface</hardwareInterface>
+    </joint>
+    <actuator name="soft_joint_servo2">
+      <hardwareInterface>hardware_interface/EffortJointInterface</hardwareInterface>
+      <mechanicalReduction>1</mechanicalReduction>
+    </actuator>
+  </transmission>
+  <transmission name="soft_joint_tran_3">
+    <type>transmission_interface/SimpleTransmission</type>
+    <joint name="soft_joint3">
+      <hardwareInterface>hardware_interface/EffortJointInterface</hardwareInterface>
+    </joint>
+    <actuator name="soft_joint_servo3">
+      <hardwareInterface>hardware_interface/EffortJointInterface</hardwareInterface>
+      <mechanicalReduction>1</mechanicalReduction>
+    </actuator>
+  </transmission>
+  <transmission name="soft_joint_tran_4">
+    <type>transmission_interface/SimpleTransmission</type>
+    <joint name="soft_joint4">
+      <hardwareInterface>hardware_interface/EffortJointInterface</hardwareInterface>
+    </joint>
+    <actuator name="soft_joint_servo4">
+      <hardwareInterface>hardware_interface/EffortJointInterface</hardwareInterface>
+      <mechanicalReduction>1</mechanicalReduction>
+    </actuator>
+  </transmission>
+  <transmission name="soft_joint_tran_5">
+    <type>transmission_interface/SimpleTransmission</type>
+    <joint name="soft_joint5">
+      <hardwareInterface>hardware_interface/EffortJointInterface</hardwareInterface>
+    </joint>
+    <actuator name="soft_joint_servo5">
+      <hardwareInterface>hardware_interface/EffortJointInterface</hardwareInterface>
+      <mechanicalReduction>1</mechanicalReduction>
+    </actuator>
+  </transmission>
+  <!-- leg -->
+  <link name="leg6">
+    <inertial>
+      <origin xyz="0.0 0.0 -0.093" rpy="0 0 0"/>
+      <mass value="0.051000"/>
+      <inertia
+          ixx="0.000122" iyy="0.000133" izz="0.000012"
+          ixy="0.000000" ixz="0.000000" iyz="0.000000"/>
+    </inertial>
+    <visual>
+      <geometry>
+        <box size="0.02 0.02 -0.15"/>
+      </geometry>
+      <origin xyz="0.01 0.01 -0.075" rpy="0 0 0"/>
+    </visual>
+  </link>
+  <gazebo reference="leg6">
+    <mu1>0.1</mu1>
+    <mu2>0.1</mu2>
+  </gazebo>
+  <xacro:damping_factor link="leg6"/>
+  <joint name="leg_joint_soft1" type="fixed">
+    <parent link="soft_link3"/>
+    <child link="leg6"/>
+    <origin xyz="0.1 0 0" rpy="0 0 0"/>
+  </joint>
+  <!-- gimbal -->
+  <joint name="gimbal_joint5" type="revolute">
+    <limit effort="5.0" lower="${-pi}" upper="${pi}" velocity="0.5"/>
+    <parent link="soft_link3"/>
+    <child link="gimbal_link5"/>
+    <origin rpy="0 0 0" xyz="0.1595 0 0"/>
+    <axis xyz="1 0 0"/>
+    <dynamics damping="0.9" friction="0.1"/>
+  </joint>
+  <link name="gimbal_link5">
+    <inertial>
+      <origin xyz="0.0815 0 0" rpy="0 0 0"/>
+      <mass value="0.173"/>
+      <!-- this inertia value is 10 times bigger than the real one -->
+      <!-- to avoid the instability in gazebo -->
+      <!-- <inertia
+          ixx="0.0022661" ixy="0.0" ixz="0.0"
+          iyy="0.0015451" iyz="0.0"
+          izz="0.00032533"/> -->
+      <!-- original one -->
+      <inertia
+          ixx="0.00022661" ixy="0.0" ixz="0.0"
+          iyy="0.00015451" iyz="0.0"
+          izz="0.000032533"/>
+    </inertial>
+    <!-- <collision>
+      <origin xyz="0.0815 0 0" rpy="0 0 0"/>
+      <geometry>
+        <cylinder length="0.1" radius="0.05"/>
+      </geometry>
+    </collision> -->
+    <visual>
+      <origin xyz="0.0815 0 0" rpy="0 0 0"/>
+      <geometry>
+        <mesh filename="package://delta/urdf/mesh/20240722/5inch_propeller_duct_right_v2.dae"/>
+      </geometry>
+    </visual>
+  </link>
+  <gazebo reference="gimbal_link5">
+    <mu1>0.1</mu1>
+    <mu2>0.1</mu2>
+  </gazebo>
+  <xacro:damping_factor link ="gimbal_link5"/>
+  <transmission name="gimbal_tran5">
+    <type>transmission_interface/SimpleTransmission</type>
+    <joint name="gimbal_joint5">
+      <hardwareInterface>hardware_interface/EffortJointInterface</hardwareInterface>
+    </joint>
+    <actuator name="gimbal_servo1">
+      <hardwareInterface>hardware_interface/EffortJointInterface</hardwareInterface>
+      <mechanicalReduction>1</mechanicalReduction>
+    </actuator>
+  </transmission>
+  <!-- rotor -->
+  <joint name="rotor5" type="continuous">
+    <limit effort="0.0064" lower="1.0" upper="20.0" velocity="0.5"/>
+    <parent link="gimbal_link5"/>
+    <child link="thrust5"/>
+    <origin rpy="0 0 0" xyz="0.0735 0 0"/>
+    <axis xyz="0 0 -1"/>
+  </joint>
+  <link name="thrust5">
+    <inertial>
+      <origin xyz="0 0 0" rpy="0 0 0"/>
+      <mass value="0.0001"/>
+      <inertia
+          ixx="0.00001" ixy="0.0" ixz="0.0"
+          iyy="0.00001" iyz="0.0"
+          izz="0.00002"/>
+    </inertial>
+    <!-- <collision>
+      <origin rpy="0 0 0" xyz="0 0 0"/>
+      <geometry>
+        <cylinder length="0.1" radius="0.11"/>
+      </geometry>
+    </collision> -->
+    <visual>
+      <origin rpy="${pi/2} 0 0" xyz="-0.045 0.055 0.06"/>
+      <geometry>
+        <mesh filename="package://delta/urdf/mesh/20240722/TriBlade_5045.dae"/>
+      </geometry>
+    </visual>
+  </link>
+  <xacro:damping_factor link ="thrust5"/>
+  <transmission name="rotor_tran5">
+    <type>transmission_interface/SimpleTransmission</type>
+    <joint name="rotor5">
+      <hardwareInterface>RotorInterface</hardwareInterface>
+    </joint>
+    <actuator name="rotor5">
+      <hardwareInterface>RotorInterface</hardwareInterface>
+      <mechanicalReduction>1</mechanicalReduction>
+    </actuator>
+  </transmission>
 </robot>

File: robots/delta/urdf/20240722/delta_link.urdf.xacro (robot description, xacro)
@@ -58,5 +58,5 @@
     <xacro:damping_factor link="thrust${self}" />
     <joint name="rotor${self}" type="continuous">
-      <limit effort="100.0" lower="${min_force}" upper="${max_force}" velocity="0.5"/>
+      <limit effort="-0.0156" lower="${min_force}" upper="${max_force}" velocity="0.5"/>
       <parent link="rotor_parent${self}"/>
       <child link="thrust${self}"/>

Commit message: change the new tail and remove gimbal

File: robots/delta/robots/quad/20240722/delta.urdf.xacro (robot description, xacro)
@@ -65,5 +65,5 @@
     <inertial>
       <origin xyz="0.06875 0.000002 0.018960" rpy="0 0 0"/>
-      <mass value="${0.010*2 + 0.012}"/>
+      <mass value="0.059"/>
       <inertia
           ixx="0.00003988" ixy="0.0" ixz="0.0"
@@ -86,5 +86,5 @@
     <inertial>
       <origin xyz="0.1175 0.000002 0.019998" rpy="0 0 0"/>
-      <mass value="${0.010*5 + 0.012*2}"/>
+      <mass value="0.118"/>
       <inertia
           ixx="0.00006787" ixy="0.0" ixz="0.0"
@@ -107,5 +107,5 @@
     <inertial>
       <origin xyz="0.10740316 0.0 0.003" rpy="0 0 0"/>
-      <mass value="${0.010*2 + 0.012 + 0.070 + 0.016}"/>
+      <mass value="${0.059 + 0.053}"/>
       <inertia
           ixx="0.00005679" ixy="-0.000000031" ixz="-0.00002256"
@@ -128,5 +128,5 @@
     <inertial>
       <origin xyz="0 0 0" rpy="0 0 0"/>
-      <mass value="0.073"/>
+      <mass value="0.064"/>
       <!-- this is for avoiding error in gazebo -->
       <!-- <inertia
@@ -154,5 +154,5 @@
     <inertial>
       <origin xyz="0 0 0" rpy="0 0 0"/>
-      <mass value="0.068"/>
+      <mass value="0.059"/>
       <!-- this is for avoiding error in gazebo -->
       <!-- <inertia
@@ -284,5 +284,5 @@
   </joint>
   <!-- gimbal -->
-  <joint name="gimbal_joint5" type="revolute">
+  <joint name="gimbal_joint5" type="fixed">
     <limit effort="5.0" lower="${-pi}" upper="${pi}" velocity="0.5"/>
     <parent link="soft_link3"/>
@@ -295,5 +295,5 @@
     <inertial>
       <origin xyz="0.0815 0 0" rpy="0 0 0"/>
-      <mass value="0.173"/>
+      <mass value="0.222"/>
       <!-- this inertia value is 10 times bigger than the real one -->
       <!-- to avoid the instability in gazebo -->
@@ -326,14 +326,4 @@
   </gazebo>
   <xacro:damping_factor link ="gimbal_link5"/>
-  <transmission name="gimbal_tran5">
-    <type>transmission_interface/SimpleTransmission</type>
-    <joint name="gimbal_joint5">
-      <hardwareInterface>hardware_interface/EffortJointInterface</hardwareInterface>
-    </joint>
-    <actuator name="gimbal_servo1">
-      <hardwareInterface>hardware_interface/EffortJointInterface</hardwareInterface>
-      <mechanicalReduction>1</mechanicalReduction>
-    </actuator>
-  </transmission>
   <!-- rotor -->
   <joint name="rotor5" type="continuous">
