Commit message: fly with closed loop

File: robots/delta/robots/quad/20240722/delta.urdf.xacro (robot description, xacro)
@@ -72,5 +72,5 @@
     <parent link="soft_link1"/>
     <child link="soft_link2"/>
-    <origin xyz="0.1175 0 0" rpy="0 0 0"/>
+    <origin xyz="0.1175 0 0" rpy="0 0 0.78"/>
     <axis xyz="0 0 1"/>
     <dynamics damping="0.2" friction="0.1"/>
@@ -80,5 +80,5 @@
     <parent link="soft_link2"/>
     <child link="soft_link3"/>
-    <origin xyz="0.235 0 0" rpy="0 0 0"/>
+    <origin xyz="0.235 0 0" rpy="0 0 0.78"/>
     <axis xyz="0 0 1"/>
     <dynamics damping="0.2" friction="0.1"/>
@@ -250,5 +250,5 @@
     <inertial>
       <origin xyz="0.0 0.0 -0.093" rpy="0 0 0"/>
-      <mass value="0.016000"/>
+      <mass value="0.051000"/>
       <inertia
           ixx="0.000122" iyy="0.000133" izz="0.000012"
@@ -362,5 +362,5 @@
     <parent link="soft_link4"/>
     <child link="soft_link5"/>
-    <origin xyz="0.1175 0 0" rpy="0 0 0"/>
+    <origin xyz="0.1175 0 0" rpy="0 0 0.78"/>
     <axis xyz="0 0 1"/>
     <dynamics damping="0.2" friction="0.1"/>
@@ -370,5 +370,5 @@
     <parent link="soft_link5"/>
     <child link="soft_link6"/>
-    <origin xyz="0.235 0 0" rpy="0 0 0"/>
+    <origin xyz="0.235 0 0" rpy="0 0 0.78"/>
     <axis xyz="0 0 1"/>
     <dynamics damping="0.2" friction="0.1"/>
@@ -537,5 +537,5 @@
   </transmission>
   <!-- leg -->
-  <link name="leg7">
+  <!-- <link name="leg7">
     <inertial>
       <origin xyz="0.0 0.0 -0.093" rpy="0 0 0"/>
@@ -561,4 +561,4 @@
     <child link="leg7"/>
     <origin xyz="0.1 0 0" rpy="0 0 0"/>
-  </joint>
+  </joint> -->
 </robot>

Commit message: add servo.yaml and servo_sim.yaml

File: robots/delta/robots/quad/20240722/delta.urdf.xacro (robot description, xacro)
@@ -168,5 +168,5 @@
   </transmission>
   <!-- dummy_link -->
-  <joint name="servo_joint1" type="revolute">
+  <joint name="servo_joint1" type="fixed">
     <limit effort="5.0" lower="${-pi/2}" upper="${pi/2}" velocity="0.5"/>
     <parent link="link4"/>
@@ -176,5 +176,5 @@
     <dynamics damping="0.9" friction="0.1"/>
   </joint>
-  <joint name="servo_joint2" type="revolute">
+  <joint name="servo_joint2" type="fixed">
     <limit effort="5.0" lower="${-pi/2}" upper="${pi/2}" velocity="0.5"/>
     <parent link="link4"/>
@@ -226,24 +226,4 @@
     </visual>
   </link>
-  <transmission name="servo_joint_tran_1">
-    <type>transmission_interface/SimpleTransmission</type>
-    <joint name="servo_joint1">
-      <hardwareInterface>hardware_interface/EffortJointInterface</hardwareInterface>
-    </joint>
-    <actuator name="servo_joint_servo1">
-      <hardwareInterface>hardware_interface/EffortJointInterface</hardwareInterface>
-      <mechanicalReduction>1</mechanicalReduction>
-    </actuator>
-  </transmission>
-  <transmission name="servo_joint_tran_2">
-    <type>transmission_interface/SimpleTransmission</type>
-    <joint name="servo_joint2">
-      <hardwareInterface>hardware_interface/EffortJointInterface</hardwareInterface>
-    </joint>
-    <actuator name="servo_joint_servo2">
-      <hardwareInterface>hardware_interface/EffortJointInterface</hardwareInterface>
-      <mechanicalReduction>1</mechanicalReduction>
-    </actuator>
-  </transmission>
   <!-- leg -->
   <link name="leg6">
@@ -458,5 +438,5 @@
   </transmission>
   <!-- dummy_link -->
-  <joint name="servo_joint3" type="revolute">
+  <joint name="servo_joint3" type="fixed">
     <limit effort="5.0" lower="${-pi/2}" upper="${pi/2}" velocity="0.5"/>
     <parent link="soft_link6"/>
@@ -466,5 +446,5 @@
     <dynamics damping="0.9" friction="0.1"/>
   </joint>
-  <joint name="servo_joint4" type="revolute">
+  <joint name="servo_joint4" type="fixed">
     <limit effort="5.0" lower="${-pi/2}" upper="${pi/2}" velocity="0.5"/>
     <parent link="soft_link6"/>
@@ -516,24 +496,4 @@
     </visual>
   </link>
-  <transmission name="servo_joint_tran_3">
-    <type>transmission_interface/SimpleTransmission</type>
-    <joint name="servo_joint3">
-      <hardwareInterface>hardware_interface/EffortJointInterface</hardwareInterface>
-    </joint>
-    <actuator name="servo_joint_servo1">
-      <hardwareInterface>hardware_interface/EffortJointInterface</hardwareInterface>
-      <mechanicalReduction>1</mechanicalReduction>
-    </actuator>
-  </transmission>
-  <transmission name="servo_joint_tran_4">
-    <type>transmission_interface/SimpleTransmission</type>
-    <joint name="servo_joint4">
-      <hardwareInterface>hardware_interface/EffortJointInterface</hardwareInterface>
-    </joint>
-    <actuator name="servo_joint_servo4">
-      <hardwareInterface>hardware_interface/EffortJointInterface</hardwareInterface>
-      <mechanicalReduction>1</mechanicalReduction>
-    </actuator>
-  </transmission>
   <!-- leg -->
   <!-- <link name="leg7">

Commit message: change soft_joint angle as transform

File: robots/delta/robots/quad/20240722/delta.urdf.xacro (robot description, xacro)
@@ -69,16 +69,16 @@
   </joint>
   <joint name="soft_joint2" type="revolute">
-    <limit effort="5.0" lower="${-pi/2}" upper="${pi/2}" velocity="0.5"/>
+    <limit effort="5.0" lower="${-pi}" upper="${pi}" velocity="0.5"/>
     <parent link="soft_link1"/>
     <child link="soft_link2"/>
-    <origin xyz="0.1175 0 0" rpy="0 0 0.78"/>
+    <origin xyz="0.1175 0 0" rpy="0 0 0"/>
     <axis xyz="0 0 1"/>
     <dynamics damping="0.2" friction="0.1"/>
   </joint>
   <joint name="soft_joint3" type="revolute">
-    <limit effort="5.0" lower="${-pi/2}" upper="${pi/2}" velocity="0.5"/>
+    <limit effort="5.0" lower="${-pi}" upper="${pi}" velocity="0.5"/>
     <parent link="soft_link2"/>
     <child link="soft_link3"/>
-    <origin xyz="0.235 0 0" rpy="0 0 0.78"/>
+    <origin xyz="0.235 0 0" rpy="0 0 0"/>
     <axis xyz="0 0 1"/>
     <dynamics damping="0.2" friction="0.1"/>
@@ -339,16 +339,16 @@
   </joint>
   <joint name="soft_joint5" type="revolute">
-    <limit effort="5.0" lower="${-pi/2}" upper="${pi/2}" velocity="0.5"/>
+    <limit effort="5.0" lower="${-pi}" upper="${pi}" velocity="0.5"/>
     <parent link="soft_link4"/>
     <child link="soft_link5"/>
-    <origin xyz="0.1175 0 0" rpy="0 0 0.78"/>
+    <origin xyz="0.1175 0 0" rpy="0 0 0"/>
     <axis xyz="0 0 1"/>
     <dynamics damping="0.2" friction="0.1"/>
   </joint>
   <joint name="soft_joint6" type="revolute">
-    <limit effort="5.0" lower="${-pi/2}" upper="${pi/2}" velocity="0.5"/>
+    <limit effort="5.0" lower="${-pi}" upper="${pi}" velocity="0.5"/>
     <parent link="soft_link5"/>
     <child link="soft_link6"/>
-    <origin xyz="0.235 0 0" rpy="0 0 0.78"/>
+    <origin xyz="0.235 0 0" rpy="0 0 0"/>
     <axis xyz="0 0 1"/>
     <dynamics damping="0.2" friction="0.1"/>

Commit message: succeeded in box hold demo

File: robots/delta/robots/quad/20240722/delta.urdf.xacro (robot description, xacro)
@@ -270,6 +270,5 @@
     <inertial>
       <origin xyz="0.0815 0 0" rpy="0 0 0"/>
-      <!-- mass is thrust link + painter -->
-      <mass value="${0.222 + 0.081}"/>
+      <mass value="${0.222}"/>
       <!-- this inertia value is 10 times bigger than the real one -->
       <!-- to avoid the instability in gazebo -->

Commit message: turn of rotor5

File: robots/delta/robots/quad/20240722/delta.urdf.xacro (robot description, xacro)
@@ -296,12 +296,12 @@
   <xacro:damping_factor link ="gimbal_link5"/>
   <!-- rotor -->
-  <joint name="rotor5" type="continuous">
+  <joint name="rt5" type="continuous">
     <limit effort="0.0064" lower="0.0" upper="20.0" velocity="0.5"/>
     <parent link="gimbal_link5"/>
-    <child link="thrust5"/>
+    <child link="th5"/>
     <origin rpy="0 0 0" xyz="0.0735 0 0"/>
     <axis xyz="0 0 -1"/>
   </joint>
-  <link name="thrust5">
+  <link name="th5">
     <inertial>
       <origin xyz="0 0 0" rpy="0 0 0"/>
@@ -319,15 +319,15 @@
     </visual>
   </link>
-  <xacro:damping_factor link ="thrust5"/>
-  <transmission name="rotor_tran5">
+  <xacro:damping_factor link ="th5"/>
+  <!-- <transmission name="rotor_tran5">
     <type>transmission_interface/SimpleTransmission</type>
-    <joint name="rotor5">
+    <joint name="rt5">
       <hardwareInterface>RotorInterface</hardwareInterface>
     </joint>
-    <actuator name="rotor5">
+    <actuator name="rt5">
       <hardwareInterface>RotorInterface</hardwareInterface>
       <mechanicalReduction>1</mechanicalReduction>
     </actuator>
-  </transmission>
+  </transmission> -->
   <!-- 3 soft_airframe_2 -->
   <!-- soft_link -->

Commit message: remove thrust5

File: robots/delta/robots/quad/20240722/delta.urdf.xacro (robot description, xacro)
@@ -259,5 +259,5 @@
   </joint>
   <!-- gimbal -->
-  <joint name="gimbal_joint5" type="fixed">
+  <!-- <joint name="gimbal_joint5" type="fixed">
     <limit effort="5.0" lower="${-pi}" upper="${pi}" velocity="0.5"/>
     <parent link="soft_link3"/>
@@ -266,9 +266,9 @@
     <axis xyz="1 0 0"/>
     <dynamics damping="0.9" friction="0.1"/>
-  </joint>
-  <link name="gimbal_link5">
+  </joint> -->
+  <!-- <link name="gimbal_link5">
     <inertial>
       <origin xyz="0.0815 0 0" rpy="0 0 0"/>
-      <mass value="${0.222}"/>
+      <mass value="${0.222}"/> -->
       <!-- this inertia value is 10 times bigger than the real one -->
       <!-- to avoid the instability in gazebo -->
@@ -278,5 +278,5 @@
           izz="0.00032533"/> -->
       <!-- original one -->
-      <inertia
+      <!-- <inertia
           ixx="0.00022661" ixy="0.0" ixz="0.0"
           iyy="0.00015451" iyz="0.0"
@@ -294,7 +294,7 @@
     <mu2>0.1</mu2>
   </gazebo>
-  <xacro:damping_factor link ="gimbal_link5"/>
+  <xacro:damping_factor link ="gimbal_link5"/> -->
   <!-- rotor -->
-  <joint name="rt5" type="continuous">
+  <!-- <joint name="rt5" type="continuous">
     <limit effort="0.0064" lower="0.0" upper="20.0" velocity="0.5"/>
     <parent link="gimbal_link5"/>
@@ -302,6 +302,6 @@
     <origin rpy="0 0 0" xyz="0.0735 0 0"/>
     <axis xyz="0 0 -1"/>
-  </joint>
-  <link name="th5">
+  </joint> -->
+  <!-- <link name="th5">
     <inertial>
       <origin xyz="0 0 0" rpy="0 0 0"/>
@@ -319,5 +319,5 @@
     </visual>
   </link>
-  <xacro:damping_factor link ="th5"/>
+  <xacro:damping_factor link ="th5"/> -->
   <!-- <transmission name="rotor_tran5">
     <type>transmission_interface/SimpleTransmission</type>
@@ -333,5 +333,5 @@
   <!-- soft_link -->
   <joint name="soft_joint4" type="fixed">
-    <parent link="gimbal_link5"/>
+    <parent link="soft_link3"/>
     <child link="soft_link4"/>
     <origin xyz="0.147 0 0" rpy="0 0 0"/>

Commit message: Revert "remove thrust5"
This reverts commit ed96abaea69035ca2d708218f2343af2efafad7e.

File: robots/delta/robots/quad/20240722/delta.urdf.xacro (robot description, xacro)
@@ -259,5 +259,5 @@
   </joint>
   <!-- gimbal -->
-  <!-- <joint name="gimbal_joint5" type="fixed">
+  <joint name="gimbal_joint5" type="fixed">
     <limit effort="5.0" lower="${-pi}" upper="${pi}" velocity="0.5"/>
     <parent link="soft_link3"/>
@@ -266,9 +266,9 @@
     <axis xyz="1 0 0"/>
     <dynamics damping="0.9" friction="0.1"/>
-  </joint> -->
-  <!-- <link name="gimbal_link5">
+  </joint>
+  <link name="gimbal_link5">
     <inertial>
       <origin xyz="0.0815 0 0" rpy="0 0 0"/>
-      <mass value="${0.222}"/> -->
+      <mass value="${0.222}"/>
       <!-- this inertia value is 10 times bigger than the real one -->
       <!-- to avoid the instability in gazebo -->
@@ -278,5 +278,5 @@
           izz="0.00032533"/> -->
       <!-- original one -->
-      <!-- <inertia
+      <inertia
           ixx="0.00022661" ixy="0.0" ixz="0.0"
           iyy="0.00015451" iyz="0.0"
@@ -294,7 +294,7 @@
     <mu2>0.1</mu2>
   </gazebo>
-  <xacro:damping_factor link ="gimbal_link5"/> -->
+  <xacro:damping_factor link ="gimbal_link5"/>
   <!-- rotor -->
-  <!-- <joint name="rt5" type="continuous">
+  <joint name="rt5" type="continuous">
     <limit effort="0.0064" lower="0.0" upper="20.0" velocity="0.5"/>
     <parent link="gimbal_link5"/>
@@ -302,6 +302,6 @@
     <origin rpy="0 0 0" xyz="0.0735 0 0"/>
     <axis xyz="0 0 -1"/>
-  </joint> -->
-  <!-- <link name="th5">
+  </joint>
+  <link name="th5">
     <inertial>
       <origin xyz="0 0 0" rpy="0 0 0"/>
@@ -319,5 +319,5 @@
     </visual>
   </link>
-  <xacro:damping_factor link ="th5"/> -->
+  <xacro:damping_factor link ="th5"/>
   <!-- <transmission name="rotor_tran5">
     <type>transmission_interface/SimpleTransmission</type>
@@ -333,5 +333,5 @@
   <!-- soft_link -->
   <joint name="soft_joint4" type="fixed">
-    <parent link="soft_link3"/>
+    <parent link="gimbal_link5"/>
     <child link="soft_link4"/>
     <origin xyz="0.147 0 0" rpy="0 0 0"/>

Commit message: Revert "turn of rotor5"
This reverts commit aa322a5b8074c7b9a13e7c2da12c5214ad2f4aaf.

File: robots/delta/robots/quad/20240722/delta.urdf.xacro (robot description, xacro)
@@ -296,12 +296,12 @@
   <xacro:damping_factor link ="gimbal_link5"/>
   <!-- rotor -->
-  <joint name="rt5" type="continuous">
+  <joint name="rotor5" type="continuous">
     <limit effort="0.0064" lower="0.0" upper="20.0" velocity="0.5"/>
     <parent link="gimbal_link5"/>
-    <child link="th5"/>
+    <child link="thrust5"/>
     <origin rpy="0 0 0" xyz="0.0735 0 0"/>
     <axis xyz="0 0 -1"/>
   </joint>
-  <link name="th5">
+  <link name="thrust5">
     <inertial>
       <origin xyz="0 0 0" rpy="0 0 0"/>
@@ -319,15 +319,15 @@
     </visual>
   </link>
-  <xacro:damping_factor link ="th5"/>
-  <!-- <transmission name="rotor_tran5">
+  <xacro:damping_factor link ="thrust5"/>
+  <transmission name="rotor_tran5">
     <type>transmission_interface/SimpleTransmission</type>
-    <joint name="rt5">
+    <joint name="rotor5">
       <hardwareInterface>RotorInterface</hardwareInterface>
     </joint>
-    <actuator name="rt5">
+    <actuator name="rotor5">
       <hardwareInterface>RotorInterface</hardwareInterface>
       <mechanicalReduction>1</mechanicalReduction>
     </actuator>
-  </transmission> -->
+  </transmission>
   <!-- 3 soft_airframe_2 -->
   <!-- soft_link -->
